Commit message: ft joint fixed

File: centauro_urdf/urdf/parts/centauro_arm.urdf.xacro (robot description, xacro)
@@ -221,5 +221,5 @@
 <!-- end-effector -->
 <!-- wrist pitch-->
-   <joint name="j_ft_${arm_num}" type="revolute">
+   <joint name="j_ft_${arm_num}" type="fixed">
       <parent link="arm${arm_num}_7"/>
       <child link="ft_arm${arm_num}"/>

Commit message: update in joint transform

File: centauro_urdf/urdf/parts/centauro_arm.urdf.xacro (robot description, xacro)
@@ -180,5 +180,5 @@
       <parent link="arm${arm_num}_2"/>
       <child link="arm${arm_num}_3"/>
-      <origin xyz="${Shoulder_3_Ox} ${Shoulder_3_Oy} ${Shoulder_3_Oz}" rpy="0.0 0.0 ${rot*0.274669}"/>
+      <origin xyz="${Shoulder_3_Ox} ${Shoulder_3_Oy} ${Shoulder_3_Oz}" rpy="0.0 0.0 ${rot*(-0.274669)}"/>
       <axis xyz="0 0 1" />
       <limit lower="${j_arm_3_lower[arm_num-1]}" upper="${j_arm_3_upper[arm_num-1]}" effort="${j_arm_3_torque[arm_num-1]}" velocity="${j_arm_3_velocity[arm_num-1]}"/>
@@ -216,5 +216,5 @@
       <parent link="arm${arm_num}_6"/>
       <child link="arm${arm_num}_7"/>
-      <origin xyz="${Wrist_3_Ox} ${rot*Wrist_3_Oy} ${Wrist_3_Oz}" rpy="0.0 0.0 ${-rot*0.0500815}"/>
+      <origin xyz="${Wrist_3_Ox} ${rot*Wrist_3_Oy} ${Wrist_3_Oz}" rpy="0.0 0.0 ${rot*(-0.0500815)}"/>
       <axis xyz="0 0 1"/>
       <limit lower="${j_arm_7_lower[arm_num-1]}" upper="${j_arm_7_upper[arm_num-1]}" effort="${j_arm_7_torque[arm_num-1]}" velocity="${j_arm_7_velocity[arm_num-1]}"/>

Commit message: checked joint transforms to be consistent with Homing

File: centauro_urdf/urdf/parts/centauro_arm.urdf.xacro (robot description, xacro)
@@ -160,6 +160,5 @@
       <child link="arm${arm_num}_1"/>
       <!--xacro:insert_block name="origin"/-->
-      <origin xyz="${Shoulder_1_Ox} ${rot*Shoulder_1_Oy} ${Shoulder_1_Oz}" rpy="0.0 0.520149 0.0"/>
-      <!--origin xyz="${Shoulder_1_Ox} ${rot*Shoulder_1_Oy} ${Shoulder_1_Oz}" rpy="0.0 1.520149 0.0"/-->
+      <origin xyz="${Shoulder_1_Ox} ${rot*Shoulder_1_Oy} ${Shoulder_1_Oz}" rpy="0.0 0.320865 0.0"/>
       <axis xyz="0 1 0"/>
       <limit lower="${j_arm_1_lower[arm_num-1]}" upper="${j_arm_1_upper[arm_num-1]}" effort="${j_arm_1_torque[arm_num-1]}" velocity="${j_arm_1_velocity[arm_num-1]}"/>
@@ -171,5 +170,5 @@
       <child link="arm${arm_num}_2"/>
       <!--origin xyz="${Shoulder_2_Ox} ${rot*Shoulder_2_Oy} ${Shoulder_2_Oz}" rpy="${rot*Shoulder_2_roll} ${Shoulder_2_pitch} ${Shoulder_2_yaw}"/-->
-      <origin xyz="${Shoulder_2_Ox} ${rot*Shoulder_2_Oy} ${Shoulder_2_Oz}" rpy="${rot*0.320865} 0.0 0.0"/>
+      <origin xyz="${Shoulder_2_Ox} ${rot*Shoulder_2_Oy} ${Shoulder_2_Oz}" rpy="${rot*0.520149} ${Shoulder_2_pitch} ${Shoulder_2_yaw}"/>
       <axis xyz="1 0 0" />
       <limit lower="${j_arm_2_lower[arm_num-1]}" upper="${j_arm_2_upper[arm_num-1]}" effort="${j_arm_2_torque[arm_num-1]}" velocity="${j_arm_2_velocity[arm_num-1]}"/>
