Commit message: adding armX_8 links to be the same as ballX

File: centauro_urdf/urdf/parts/ball.urdf.xacro (robot description, xacro)
@@ -33,4 +33,15 @@
 	<origin xyz="0 0 -0.07" rpy="0 0 0"/>
 </joint>
+<!-- add armX_8 link for legacy reasons (same as ballX) -->
+<joint name="j_ball${arm_num}_fixed" type="fixed">
+      <parent link="ball${arm_num}"/>
+      <child link="arm${arm_num}_8"/>
+</joint>
+<link name="arm${arm_num}_8">
+    <inertial>
+      <mass value="0"/>
+      <inertia ixx="0" ixy="0" ixz="0" iyy="0" iyz="0" izz="0"/>
+    </inertial>
+</link>
 </xacro:macro>
 </robot>

Commit message: arm*_8 to be at CoG, so as to control based on this

File: centauro_urdf/urdf/parts/ball.urdf.xacro (robot description, xacro)
@@ -37,4 +37,5 @@
       <parent link="ball${arm_num}"/>
       <child link="arm${arm_num}_8"/>
+      <origin xyz="${-1.0072498e-02*mmTom} ${3.7590658e-02*mmTom} ${1.9772332e+01*mmTom}" rpy="0 0 0"/>
 </joint>
 <link name="arm${arm_num}_8">
