Commit message: added simplified collision meshes for wheels

File: centauro_urdf/urdf/parts/centauro_leg.urdf.xacro (robot description, xacro)
@@ -118,10 +118,16 @@
          <material name="black"/>
       </visual>
-      <collision>
-               <origin xyz="0.0 0.0 0.0"  rpy="0.0 0.0 0.0"/>
-   <geometry>
-      <mesh filename="package://centauro_urdf/meshes/simple/wheel.stl" scale="0.001 ${0.001} 0.001" />
-   </geometry>
-      </collision>
+      <!--collision>
+      	<origin xyz="0.0 0.0 0.0"  rpy="0.0 0.0 0.0"/>
+   		<geometry>
+      			<mesh filename="package://centauro_urdf/meshes/simple/wheel.stl" scale="0.001 ${0.001} 0.001" />
+   		</geometry>
+      </collision-->
+	<collision>
+		<origin xyz="0 0 0" rpy="0 0 0"/>
+		<geometry>
+			<cylinder length="0.06" radius="${0.17/2.}"/>
+      		</geometry>
+	</collision>
 </link>
 <joint name="hip_yaw_${leg_num}" type="revolute">

Commit message: fixed wheel radius

File: centauro_urdf/urdf/parts/centauro_leg.urdf.xacro (robot description, xacro)
@@ -127,5 +127,5 @@
 		<origin xyz="0 0 0" rpy="0 0 0"/>
 		<geometry>
-			<cylinder length="0.06" radius="${0.17/2.}"/>
+			<cylinder length="0.06" radius="0.078"/>
       		</geometry>
 	</collision>

Commit message: first push

File: centauro_urdf/urdf/parts/centauro_leg.urdf.xacro (robot description, xacro)
@@ -131,4 +131,14 @@
 	</collision>
 </link>
+<!-- *****************************-->
+<link name="contact_${leg_num}">
+</link>
+<joint name="contact_joint_${leg_num}" type="fixed">
+	<parent link="ankle2_${leg_num}"/>
+	<child link="contact_${leg_num}"/>
+	<origin xyz="0 0 0.315" rpy="3.14159265 0 0"/>
+	<!--axis xyz="0 0 1" /-->
+</joint>
+<!-- ******************************** -->
 <joint name="hip_yaw_${leg_num}" type="revolute">
 	<parent link="pelvis"/>

Commit message: first push

File: centauro_urdf/urdf/parts/centauro_leg.urdf.xacro (robot description, xacro)
@@ -157,4 +157,14 @@
 </link>
 </xacro:unless>
+<!-- *****************************-->
+<link name="contact_${leg_num}">
+</link>
+<joint name="contact_joint_${leg_num}" type="fixed">
+	<parent link="ankle2_${leg_num}"/>
+	<child link="contact_${leg_num}"/>
+	<origin xyz="0 0 0.315" rpy="3.14159265 0 0"/>
+	<!--axis xyz="0 0 1" /-->
+</joint>
+<!-- ******************************** -->
 <joint name="hip_yaw_${leg_num}" type="revolute">
 	<parent link="pelvis"/>

Commit message: updated kinematics and mass properties from latest cad data

File: centauro_urdf/urdf/parts/centauro_leg.urdf.xacro (robot description, xacro)
@@ -2,37 +2,36 @@
 <robot xmlns:xacro="http://ros.org/wiki/xacro">
 <!-- macro legs -->
-<xacro:macro name="centauro_leg" params="leg_num origin_x origin_y">
+<xacro:macro name="centauro_leg" params="leg_num origin_x origin_y mirror">
 <link name="hip1_${leg_num}">
 	<inertial>
-		<origin xyz="${Leg_1_x} ${origin_x*origin_y*Leg_1_y} ${Leg_1_z}" />
+		<origin xyz="${Leg_1_x} ${mirror*Leg_1_y} ${Leg_1_z}" />
 		<mass value="${Leg_1_mass}"/> <!-- org: 2 -->
-		<inertia ixx="${Leg_1_xx}" ixy="${origin_x*origin_y*Leg_1_xy}" ixz="${Leg_1_xz}" iyy="${Leg_1_yy}" iyz="${origin_x*origin_y*Leg_1_yz}" izz="${Leg_1_zz}"/>
+		<inertia ixx="${Leg_1_xx}" ixy="${mirror*Leg_1_xy}" ixz="${Leg_1_xz}" iyy="${Leg_1_yy}" iyz="${mirror*Leg_1_yz}" izz="${Leg_1_zz}"/>
+	</inertial>
+   <visual>
+      <origin xyz="0.0 0.0 0.0"  rpy="0.0 0.0 0.0"/>
+      <geometry>
+         <mesh filename="package://centauro_urdf/meshes/v2/hip-yaw.stl" scale="0.001 ${mirror*0.001} 0.001" />
+      </geometry>
+      <material name="dark_grey"/>
+   </visual>
+   <collision>
+      <origin xyz="0.0 0.0 0.0"  rpy="0.0 0.0 ${origin_x*origin_y*(Leg_1_yaw-PI/2)-Leg_1_yaw+PI/2}"/>
+      <geometry>
+         <mesh filename="package://centauro_urdf/meshes/simple/hip-yaw.stl" scale="0.001 ${0.001} 0.001" />
+      </geometry>
+   </collision>
+</link>
+<link name="hip2_${leg_num}">
+	<inertial>
+		<origin xyz="${Leg_2_x} ${Leg_2_y} ${mirror*Leg_2_z}"/>
+		<mass value="${Leg_2_mass}"/> <!-- org: 4.5 -->
+		<inertia ixx="${Leg_2_xx}" ixy="${Leg_2_xy}" ixz="${mirror*Leg_2_xz}" iyy="${Leg_2_yy}" iyz="${mirror*Leg_2_yz}" izz="${Leg_2_zz}"/>
 		<!-- <inertia ixx="0.01" ixy="0.01" ixz="0.01" iyy="0.01" iyz="0.01" izz="0.01"/> -->
 	</inertial>
       <visual>
-         <origin xyz="0.0 0.0 0.0"  rpy="0.0 0.0 ${origin_x*origin_y*(Leg_1_yaw-PI/2)-Leg_1_yaw+PI/2}"/>
-   <geometry>
-      <mesh filename="package://centauro_urdf/meshes/hip-yaw.stl" scale="0.001 ${0.001} 0.001" />
-   </geometry>
-         <material name="dark_grey"/>
-      </visual>
-      <collision>
-         <origin xyz="0.0 0.0 0.0"  rpy="0.0 0.0 ${origin_x*origin_y*(Leg_1_yaw-PI/2)-Leg_1_yaw+PI/2}"/>
-   <geometry>
-      <mesh filename="package://centauro_urdf/meshes/simple/hip-yaw.stl" scale="0.001 ${0.001} 0.001" />
-   </geometry>
-      </collision>
-</link>
-<link name="hip2_${leg_num}">
-	<inertial>
-		<origin xyz="${Leg_2_x} ${Leg_2_y} ${Leg_2_z}"/>
-		<mass value="${Leg_2_mass}"/> <!-- org: 4.5 -->
-		<inertia ixx="${Leg_2_xx}" ixy="${Leg_2_xy}" ixz="${Leg_2_xz}" iyy="${Leg_2_yy}" iyz="${Leg_2_yz}" izz="${Leg_2_zz}"/>
-		<!-- <inertia ixx="0.01" ixy="0.01" ixz="0.01" iyy="0.01" iyz="0.01" izz="0.01"/> -->
-	</inertial>
-      <visual>
-         <origin xyz="0.0 0.0 0.0"  rpy="0.0 0.0 0.0"/>
-   <geometry>
-      <mesh filename="package://centauro_urdf/meshes/hip-pitch.stl" scale="0.001 ${0.001} 0.001" />
+         <origin xyz="0.0 0.0 0.0"  rpy="0.0 0.0 0.0"/>
+   <geometry>
+      <mesh filename="package://centauro_urdf/meshes/v2/hip-pitch.stl" scale="0.001 0.001 ${mirror*0.001}" />
    </geometry>
       </visual>
@@ -71,7 +70,7 @@
 <link name="knee_${leg_num}">
 	<inertial>
-		<origin xyz="${Leg_3_x} ${Leg_3_y} ${Leg_3_z}"/>
+		<origin xyz="${Leg_3_x} ${Leg_3_y} ${mirror*Leg_3_z}"/>
 		<mass value="${Leg_3_mass}"/>  <!-- org: 3.5, foot un modeled-->
-		<inertia ixx="${Leg_3_xx}" ixy="${Leg_3_xy}" ixz="${Leg_3_xz}" iyy="${Leg_3_yy}" iyz="${Leg_3_yz}" izz="${Leg_3_zz}"/>
+		<inertia ixx="${Leg_3_xx}" ixy="${Leg_3_xy}" ixz="${mirror*Leg_3_xz}" iyy="${Leg_3_yy}" iyz="${mirror*Leg_3_yz}" izz="${Leg_3_zz}"/>
 	<!--	<inertia ixx="0.01" ixy="0.01" ixz="0.01" iyy="0.01" iyz="0.01" izz="0.01"/>  -->
 	</inertial>
@@ -79,5 +78,5 @@
          <origin xyz="0.0 0.0 0.0"  rpy="0.0 0.0 0.0"/>
    <geometry>
-      <mesh filename="package://centauro_urdf/meshes/knee.stl" scale="0.001 ${0.001} 0.001" />
+      <mesh filename="package://centauro_urdf/meshes/v2/knee.stl" scale="0.001 0.001 ${mirror*0.001}" />
    </geometry>
          <material name="dark_grey"/>
@@ -92,7 +91,7 @@
 <link name="ankle1_${leg_num}">
 	<inertial>
-		<origin xyz="${Ankle_1_x} ${Ankle_1_y} ${Ankle_1_z}"/>
+		<origin xyz="${Ankle_1_x} ${Ankle_1_y} ${mirror*Ankle_1_z}"/>
 		<mass value="${Ankle_1_mass}"/>  <!-- org: 3.5, foot un modeled-->
-		<inertia ixx="${Ankle_1_xx}" ixy="${Ankle_1_xy}" ixz="${Ankle_1_xz}" iyy="${Ankle_1_yy}" iyz="${Ankle_1_yz}" izz="${Ankle_1_zz}"/>
+		<inertia ixx="${Ankle_1_xx}" ixy="${Ankle_1_xy}" ixz="${mirror*Ankle_1_xz}" iyy="${Ankle_1_yy}" iyz="${mirror*Ankle_1_yz}" izz="${Ankle_1_zz}"/>
 	<!--	<inertia ixx="0.01" ixy="0.01" ixz="0.01" iyy="0.01" iyz="0.01" izz="0.01"/>  -->
 	</inertial>
@@ -100,5 +99,5 @@
          <origin xyz="0.0 0.0 0.0"  rpy="0.0 0.0 0.0"/>
    <geometry>
-      <mesh filename="package://centauro_urdf/meshes/ankle-pitch.stl" scale="0.001 ${0.001} 0.001" />
+      <mesh filename="package://centauro_urdf/meshes/v2/ankle-pitch.stl" scale="0.001 0.001 ${mirror*0.001}" />
    </geometry>
       </visual>
@@ -112,12 +111,12 @@
 <link name="ankle2_${leg_num}">
 	<inertial>
-		<origin xyz="${Ankle_2_x} ${Ankle_2_y} ${Ankle_2_z}"/>
+		<origin xyz="${Ankle_2_x} ${mirror*Ankle_2_y} ${Ankle_2_z}"/>
 		<mass value="${Ankle_2_mass}"/>  <!-- org: 3.5, foot un modeled-->
-		<inertia ixx="${Ankle_2_xx}" ixy="${Ankle_2_xy}" ixz="${Ankle_2_xz}" iyy="${Ankle_2_yy}" iyz="${Ankle_2_yz}" izz="${Ankle_2_zz}"/>
-	</inertial>
-      <visual>
-         <origin xyz="0.0 0.0 0.0"  rpy="0.0 0.0 0.0"/>
-   <geometry>
-      <mesh filename="package://centauro_urdf/meshes/ankle-yaw.stl" scale="0.001 ${0.001} 0.001" />
+		<inertia ixx="${Ankle_2_xx}" ixy="${mirror*Ankle_2_xy}" ixz="${Ankle_2_xz}" iyy="${Ankle_2_yy}" iyz="${mirror*Ankle_2_yz}" izz="${Ankle_2_zz}"/>
+	</inertial>
+      <visual>
+         <origin xyz="0.0 0.0 0.0"  rpy="0.0 0.0 0.0"/>
+   <geometry>
+      <mesh filename="package://centauro_urdf/meshes/v2/ankle-yaw.stl" scale="0.001 ${origin_y*0.001} 0.001" />
    </geometry>
          <material name="dark_grey"/>
@@ -132,12 +131,12 @@
 <link name="wheel_${leg_num}">
 	<inertial>
-		<origin xyz="${Wheel_x} ${Wheel_y} ${Wheel_z}"/>
+		<origin xyz="${Wheel_x} ${Wheel_y} ${mirror*Wheel_z}"/>
 		<mass value="${Wheel_mass}"/>  <!-- org: 3.5, foot un modeled-->
-		<inertia ixx="${Wheel_xx}" ixy="${Wheel_xy}" ixz="${Wheel_xz}" iyy="${Wheel_yy}" iyz="${Wheel_yz}" izz="${Wheel_zz}"/>
-	</inertial>
-      <visual>
-         <origin xyz="0.0 0.0 0.0"  rpy="0.0 0.0 0.0"/>
-   <geometry>
-      <mesh filename="package://centauro_urdf/meshes/wheel.stl" scale="0.001 ${0.001} 0.001" />
+		<inertia ixx="${Wheel_xx}" ixy="${Wheel_xy}" ixz="${mirror*Wheel_xz}" iyy="${Wheel_yy}" iyz="${mirror*Wheel_yz}" izz="${Wheel_zz}"/>
+	</inertial>
+      <visual>
+         <origin xyz="0.0 0.0 0.0"  rpy="0.0 0.0 0.0"/>
+   <geometry>
+      <mesh filename="package://centauro_urdf/meshes/v2/wheel.stl" scale="0.001 0.001 ${mirror*0.001}" />
    </geometry>
          <material name="black"/>
@@ -170,14 +169,14 @@
 	<parent link="pelvis"/>
 	<child link="hip1_${leg_num}"/>
-	<origin xyz="${origin_x*Leg_1_Ox} ${origin_y*Leg_1_Oy} ${Leg_1_Oz}" rpy="${Leg_1_roll} ${Leg_1_pitch} ${PI/2-origin_x*PI/2+origin_x*origin_y*Leg_1_yaw}"/>
-	<axis xyz="0 0 1"/>
-        <limit lower="${hip_yaw_lower[leg_num-1]}" upper="${hip_yaw_upper[leg_num-1]}" effort="${motor_A_effort}" velocity="${motor_A_velocity}"/> <!-- 200 Nm, 1 rad/s-->
+	<origin xyz="${origin_x*Leg_1_Ox} ${origin_y*Leg_1_Oy} ${Leg_1_Oz}" rpy="${Leg_1_roll} ${Leg_1_pitch} ${Leg_1_yaw}"/>
+	<axis xyz="0 0 1"/>
+   <limit lower="${hip_yaw_lower[leg_num-1]}" upper="${hip_yaw_upper[leg_num-1]}" effort="${motor_A_effort}" velocity="${motor_A_velocity}"/> <!-- 200 Nm, 1 rad/s-->
 </joint>
 <joint name="hip_pitch_${leg_num}" type="revolute">
 	<parent link="hip1_${leg_num}"/>
 	<child link="hip2_${leg_num}"/>
-	<origin xyz="${Leg_2_Ox} ${Leg_2_Oy} ${Leg_2_Oz}" rpy="${Leg_2_roll} ${Leg_2_pitch} ${origin_x*origin_y*Leg_2_yaw-origin_x*origin_y*PI/2 + PI/2}"/>
-	<axis xyz="0 0 1"/>
-        <limit lower="${hip_pitch_lower[leg_num-1]}" upper="${hip_pitch_upper[leg_num-1]}" effort="${motor_A_effort}" velocity="${motor_A_velocity}"/> <!-- 200 Nm, 1 rad/s-->
+	<origin xyz="${Leg_2_Ox} ${mirror*Leg_2_Oy} ${Leg_2_Oz}" rpy="${Leg_2_roll} ${Leg_2_pitch} ${Leg_2_yaw}"/>
+	<axis xyz="0 0 1"/>
+   <limit lower="${hip_pitch_lower[leg_num-1]}" upper="${hip_pitch_upper[leg_num-1]}" effort="${motor_A_effort}" velocity="${motor_A_velocity}"/> <!-- 200 Nm, 1 rad/s-->
 </joint>
 <xacro:if  value="${USE_STICKS}">
@@ -194,12 +193,12 @@
 	<parent link="hip2_${leg_num}"/>
 	<child link="knee_${leg_num}"/>
-	<origin xyz="${Leg_3_Ox} ${Leg_3_Oy} ${Leg_3_Oz}" rpy="${Leg_3_roll} ${Leg_3_pitch} ${Leg_3_yaw}"/>
-	<axis xyz="0 0 1"/>
-        <limit lower="${knee_pitch_lower[leg_num-1]}" upper="${knee_pitch_upper[leg_num-1]}" effort="${motor_A_effort}" velocity="${motor_A_velocity}"/> <!-- 200 Nm, 1 rad/s-->
+	<origin xyz="${Leg_3_Ox} ${Leg_3_Oy} ${mirror*Leg_3_Oz}" rpy="${Leg_3_roll} ${Leg_3_pitch} ${Leg_3_yaw}"/>
+	<axis xyz="0 0 1"/>
+   <limit lower="${knee_pitch_lower[leg_num-1]}" upper="${knee_pitch_upper[leg_num-1]}" effort="${motor_A_effort}" velocity="${motor_A_velocity}"/> <!-- 200 Nm, 1 rad/s-->
 </joint>
 <joint name="ankle_pitch_${leg_num}" type="revolute">
 	<parent link="knee_${leg_num}"/>
 	<child link="ankle1_${leg_num}"/>
-	<origin xyz="${Ankle_1_Ox} ${Ankle_1_Oy} ${Ankle_1_Oz}" rpy="${Ankle_1_roll} ${Ankle_1_pitch} ${Ankle_1_yaw}"/>
+	<origin xyz="${Ankle_1_Ox} ${Ankle_1_Oy} ${mirror*Ankle_1_Oz}" rpy="${Ankle_1_roll} ${Ankle_1_pitch} ${Ankle_1_yaw}"/>
 	<axis xyz="0 0 1"/>
         <limit lower="${ankle_pitch_lower[leg_num-1]}" upper="${ankle_pitch_upper[leg_num-1]}" effort="${motor_B_effort}" velocity="${motor_B_velocity}"/> <!-- 98 Nm, 1 rad/s-->
@@ -208,5 +207,5 @@
 	<parent link="ankle1_${leg_num}"/>
 	<child link="ankle2_${leg_num}"/>
-	<origin xyz="${Ankle_2_Ox} ${Ankle_2_Oy} ${Ankle_2_Oz}" rpy="${Ankle_2_roll} ${Ankle_2_pitch} ${Ankle_2_yaw}"/>
+	<origin xyz="${Ankle_2_Ox} ${Ankle_2_Oy} ${mirror*Ankle_2_Oz}" rpy="${Ankle_2_roll} ${Ankle_2_pitch} ${Ankle_2_yaw}"/>
 	<axis xyz="0 0 1"/>
         <limit lower="${ankle_yaw_lower[leg_num-1]}" upper="${ankle_yaw_upper[leg_num-1]}" effort="${motor_C_effort}" velocity="${motor_C_velocity}"/>  <!-- 23 Nm, 1 rad/s-->
@@ -215,5 +214,5 @@
 	<parent link="ankle2_${leg_num}"/>
 	<child link="wheel_${leg_num}"/>
-	<origin xyz="${Wheel_Ox} ${Wheel_Oy} ${Wheel_Oz}" rpy="${Wheel_roll} ${Wheel_pitch} ${Wheel_yaw}"/>
+	<origin xyz="${Wheel_Ox} ${mirror*Wheel_Oy} ${Wheel_Oz}" rpy="${Wheel_roll} ${Wheel_pitch} ${Wheel_yaw}"/>
 	<axis xyz="0 0 1"/>
         <limit  effort="${motor_C_effort}" velocity="${motor_C_velocity}"/>  <!-- 23 Nm, 1 rad/s-->

File: centauro_urdf/urdf/parts/inertial_properties.urdf.xacro (robot description, xacro)
@@ -24,81 +24,81 @@
 <xacro:property name="Pelvis_mass" value=" 16.0975740000 "/>
 <!-- Center of Mass -->
-<xacro:property name="Leg_1_x" value=" 0.0102141990 "/>
-<xacro:property name="Leg_1_y" value=" 0.0183483590 "/>
-<xacro:property name="Leg_1_z" value=" 0.0380909870 "/>
-<!-- Inertia -->
-<xacro:property name="Leg_1_xx" value=" 0.0047439572 "/>
-<xacro:property name="Leg_1_yy" value=" 0.0040551878 "/>
-<xacro:property name="Leg_1_zz" value=" 0.0034146219 "/>
-<xacro:property name="Leg_1_xy" value=" -0.0005747047 "/>
-<xacro:property name="Leg_1_xz" value=" -0.0003784138 "/>
-<xacro:property name="Leg_1_yz" value=" -0.0007407508 "/>
-<!-- Mass -->
-<xacro:property name="Leg_1_mass" value=" 1.9194403000 "/>
-<!-- Center of Mass -->
-<xacro:property name="Leg_2_x" value=" 0.0000257966 "/>
-<xacro:property name="Leg_2_y" value=" 0.1810266000 "/>
-<xacro:property name="Leg_2_z" value=" 0.0856697560 "/>
-<!-- Inertia -->
-<xacro:property name="Leg_2_xx" value=" 0.0485186900 "/>
-<xacro:property name="Leg_2_yy" value=" 0.0042420550 "/>
-<xacro:property name="Leg_2_zz" value=" 0.0482558300 "/>
-<xacro:property name="Leg_2_xy" value=" -0.0000411894 "/>
-<xacro:property name="Leg_2_xz" value=" -0.0000168778 "/>
-<xacro:property name="Leg_2_yz" value=" 0.0032243188 "/>
-<!-- Mass -->
-<xacro:property name="Leg_2_mass" value=" 2.7264471000 "/>
-<!-- Center of Mass -->
-<xacro:property name="Leg_3_x" value="0.1088166700 "/>
-<xacro:property name="Leg_3_y" value="0.0001089081 "/>
-<xacro:property name="Leg_3_z" value="-0.0226389960 "/>
-<!-- Inertia -->
-<xacro:property name="Leg_3_xx" value=" 0.0030534242 "/>
-<xacro:property name="Leg_3_yy" value=" 0.0196033210 "/>
-<xacro:property name="Leg_3_zz" value=" 0.0198498170 "/>
-<xacro:property name="Leg_3_xy" value=" -0.0000422079 "/>
-<xacro:property name="Leg_3_xz" value=" 0.0013679297 "/>
-<xacro:property name="Leg_3_yz" value=" 0.0000069941 "/>
-<!-- Mass -->
-<xacro:property name="Leg_3_mass" value="1.9356754000 "/>
-<!-- Center of Mass -->
-<xacro:property name="Ankle_1_x" value=" 0.0321373180 "/>
-<xacro:property name="Ankle_1_y" value=" 0.0000973572 "/>
-<xacro:property name="Ankle_1_z" value=" -0.0044222206 "/>
-<!-- Inertia -->
-<xacro:property name="Ankle_1_xx" value=" 0.0015610452 "/>
-<xacro:property name="Ankle_1_yy" value=" 0.0037423211 "/>
-<xacro:property name="Ankle_1_zz" value=" 0.0038312442 "/>
-<xacro:property name="Ankle_1_xy" value=" 0.0000330597 "/>
-<xacro:property name="Ankle_1_xz" value=" -0.0001314174 "/>
-<xacro:property name="Ankle_1_yz" value=" -0.0000212589 "/>
-<!-- Mass -->
-<xacro:property name="Ankle_1_mass" value="1.2380744000 "/>
-<!-- Center of Mass -->
-<xacro:property name="Ankle_2_x" value=" 0.0004435803 "/>
-<xacro:property name="Ankle_2_y" value=" 0.0004389911 "/>
-<xacro:property name="Ankle_2_z" value=" 0.1939209200 "/>
-<!-- Inertia -->
-<xacro:property name="Ankle_2_xx" value=" 0.0049019475 "/>
-<xacro:property name="Ankle_2_yy" value=" 0.0038724162 "/>
-<xacro:property name="Ankle_2_zz" value=" 0.0021783198 "/>
-<xacro:property name="Ankle_2_xy" value=" 0.0000043032 "/>
-<xacro:property name="Ankle_2_xz" value=" 0.0000346491 "/>
-<xacro:property name="Ankle_2_yz" value=" 0.0000170990 "/>
-<!-- Mass -->
-<xacro:property name="Ankle_2_mass" value=" 1.1565926000 "/>
-<!-- Center of Mass -->
-<xacro:property name="Wheel_x" value=" 0.0000000000 "/>
-<xacro:property name="Wheel_y" value=" 0.000000 "/>
-<xacro:property name="Wheel_z" value=" 0.0024271906 "/>
-<!-- Inertia -->
-<xacro:property name="Wheel_xx" value=" 0.0046864297 "/>
-<xacro:property name="Wheel_yy" value=" 0.0046713489 "/>
-<xacro:property name="Wheel_zz" value=" 0.0053126029 "/>
-<xacro:property name="Wheel_xy" value=" 0.000000 "/>
-<xacro:property name="Wheel_xz" value=" 0.000000 "/>
-<xacro:property name="Wheel_yz" value=" 0.000000 "/>
-<!-- Mass -->
-<xacro:property name="Wheel_mass" value=" 1.7289003000 "/>
+<xacro:property name="Leg_1_x" value="${3.5958550e-01 * mmTom}"/>
+<xacro:property name="Leg_1_y" value="${-3.3338818e+01 * mmTom}"/>
+<xacro:property name="Leg_1_z" value="${-5.9190309e+01 * mmTom}"/>
+<!-- Inertia -->
+<xacro:property name="Leg_1_xx" value="${6.8405374e+03 * mm2Tom2}"/>
+<xacro:property name="Leg_1_yy" value="${2.6261815e+03 * mm2Tom2}"/>
+<xacro:property name="Leg_1_zz" value="${6.6933354e+03 * mm2Tom2}"/>
+<xacro:property name="Leg_1_xy" value="${-1.8572633e+01 * mm2Tom2}"/>
+<xacro:property name="Leg_1_xz" value="${-4.8325972e+01 * mm2Tom2}"/>
+<xacro:property name="Leg_1_yz" value="${-1.5642730e+02 * mm2Tom2}"/>
+<!-- Mass -->
+<xacro:property name="Leg_1_mass" value="${2.3349153e+00}"/>
+<!-- Center of Mass -->
+<xacro:property name="Leg_2_x" value="${-4.6285952e-03 * mmTom}"/>
+<xacro:property name="Leg_2_y" value="${-2.2140190e+02 * mmTom}"/>
+<xacro:property name="Leg_2_z" value="${-3.3166850e+01 * mmTom}"/>
+<!-- Inertia -->
+<xacro:property name="Leg_2_xx" value="${5.0469853e+04 * mm2Tom2}"/>
+<xacro:property name="Leg_2_yy" value="${8.1815970e+03 * mm2Tom2}"/>
+<xacro:property name="Leg_2_zz" value="${4.8213809e+04 * mm2Tom2}"/>
+<xacro:property name="Leg_2_xy" value="${-7.7849387e+00 * mm2Tom2}"/>
+<xacro:property name="Leg_2_xz" value="${9.2205810e+00 * mm2Tom2}"/>
+<xacro:property name="Leg_2_yz" value="${-5.9796848e+03 * mm2Tom2}"/>
+<!-- Mass -->
+<xacro:property name="Leg_2_mass" value="3.4572118e+00"/>
+<!-- Center of Mass -->
+<xacro:property name="Leg_3_x" value="${1.2063381e-01 * mmTom}"/>
+<xacro:property name="Leg_3_y" value="${1.4620674e+02 * mmTom}"/>
+<xacro:property name="Leg_3_z" value="${-2.9740711e+01 * mmTom}"/>
+<!-- Inertia -->
+<xacro:property name="Leg_3_xx" value="${1.8426403e+04 * mm2Tom2}"/>
+<xacro:property name="Leg_3_yy" value="${4.7685615e+03 * mm2Tom2}"/>
+<xacro:property name="Leg_3_zz" value="${1.7793722e+04 * mm2Tom2}"/>
+<xacro:property name="Leg_3_xy" value="${2.8226636e+01 * mm2Tom2}"/>
+<xacro:property name="Leg_3_xz" value="${2.9204348e+01 * mm2Tom2}"/>
+<xacro:property name="Leg_3_yz" value="${2.6407710e+03 * mm2Tom2}"/>
+<!-- Mass -->
+<xacro:property name="Leg_3_mass" value="2.1199315e+00"/>
+<!-- Center of Mass -->
+<xacro:property name="Ankle_1_x" value="${1.2360094e-01 * mmTom}"/>
+<xacro:property name="Ankle_1_y" value="${-6.2747120e+01 * mmTom}"/>
+<xacro:property name="Ankle_1_z" value="${4.9068453e+00 * mmTom}"/>
+<!-- Inertia -->
+<xacro:property name="Ankle_1_xx" value="${4.9928829e+03 * mm2Tom2}"/>
+<xacro:property name="Ankle_1_yy" value="${1.7621464e+03 * mm2Tom2}"/>
+<xacro:property name="Ankle_1_zz" value="${4.8706328e+03 * mm2Tom2}"/>
+<xacro:property name="Ankle_1_xy" value="${5.7623557e+00 * mm2Tom2}"/>
+<xacro:property name="Ankle_1_xz" value="${-1.9606394e+01 * mm2Tom2}"/>
+<xacro:property name="Ankle_1_yz" value="${-4.5315091e+02 * mm2Tom2}"/>
+<!-- Mass -->
+<xacro:property name="Ankle_1_mass" value="1.4023368e+00"/>
+<!-- Center of Mass -->
+<xacro:property name="Ankle_2_x" value="${1.8496706e+00 * mmTom}"/>
+<xacro:property name="Ankle_2_y" value="${5.1322371e-01 * mmTom}"/>
+<xacro:property name="Ankle_2_z" value="${-6.7309240e+01 * mmTom}"/>
+<!-- Inertia -->
+<xacro:property name="Ankle_2_xx" value="${7.3976286e+03 * mm2Tom2}"/>
+<xacro:property name="Ankle_2_yy" value="${5.4434358e+03 * mm2Tom2}"/>
+<xacro:property name="Ankle_2_zz" value="${4.3055053e+03 * mm2Tom2}"/>
+<xacro:property name="Ankle_2_xy" value="${-9.7557687e-01 * mm2Tom2}"/>
+<xacro:property name="Ankle_2_xz" value="${-2.2952550e+02 * mm2Tom2}"/>
+<xacro:property name="Ankle_2_yz" value="${-3.6337754e+01 * mm2Tom2}"/>
+<!-- Mass -->
+<xacro:property name="Ankle_2_mass" value="1.7656714e+00"/>
+<!-- Center of Mass -->
+<xacro:property name="Wheel_x" value="${0.0 * mmTom}"/>
+<xacro:property name="Wheel_y" value="${0.0 * mmTom}"/>
+<xacro:property name="Wheel_z" value="${-4.9165610e+01 * mmTom}"/>
+<!-- Inertia -->
+<xacro:property name="Wheel_xx" value="${2.8174054e+03 * mm2Tom2}"/>
+<xacro:property name="Wheel_yy" value="${2.8175648e+03 * mm2Tom2}"/>
+<xacro:property name="Wheel_zz" value="${4.1817162e+03 * mm2Tom2}"/>
+<xacro:property name="Wheel_xy" value="${0.0 * mm2Tom2}"/>
+<xacro:property name="Wheel_xz" value="${0.0 * mm2Tom2}"/>
+<xacro:property name="Wheel_yz" value="${0.0 * mm2Tom2}"/>
+<!-- Mass -->
+<xacro:property name="Wheel_mass" value="1.1116400e+00"/>  <!-- TODO CHECK THIS VALUE -->
 <!-- Center of Mass -->
 <xacro:property name="Torso_2_x" value=" -0.0194977940 "/>
