Commit message: updated kinematics and mass properties from latest cad data

File: centauro_urdf/urdf/parts/kinematics_properties.urdf.xacro (robot description, xacro)
@@ -28,42 +28,42 @@
 <xacro:property name="Neck_3_Oz" value=" 0.473262 "/>
 <!-- Origin -->
-<xacro:property name="Leg_1_Ox" value=" 0.250 "/>
-<xacro:property name="Leg_1_Oy" value=" -0.125 "/>
-<xacro:property name="Leg_1_Oz" value="-0.05660000 "/>
-<xacro:property name="Leg_1_roll" value=" 3.141592653589793 "/>
-<xacro:property name="Leg_1_pitch" value=" 0.0 "/>
-<xacro:property name="Leg_1_yaw" value=" -0.461416123228 "/>
+<xacro:property name="Leg_1_Ox" value="${250.000 * mmTom}"/>
+<xacro:property name="Leg_1_Oy" value="${-125.000 * mmTom}"/>
+<xacro:property name="Leg_1_Oz" value="${-56.6000 * mmTom}"/>
+<xacro:property name="Leg_1_roll" value="0.0"/>
+<xacro:property name="Leg_1_pitch" value="0.0"/>
+<xacro:property name="Leg_1_yaw" value="0.0"/>
 <!-- Origin -->
-<xacro:property name="Leg_2_Ox" value=" 0.000000 "/>
-<xacro:property name="Leg_2_Oy" value=" 0.000000 "/>
-<xacro:property name="Leg_2_Oz" value=" 0.0625 "/>
-<xacro:property name="Leg_2_roll" value=" 1.57079632679 "/>
-<xacro:property name="Leg_2_pitch" value=" 0.0 "/>
-<xacro:property name="Leg_2_yaw" value=" 2.68017653036 "/>
+<xacro:property name="Leg_2_Ox" value="0.0"/>
+<xacro:property name="Leg_2_Oy" value="${-114.600 * mmTom}"/>
+<xacro:property name="Leg_2_Oz" value="${-62.5000 * mmTom}"/>
+<xacro:property name="Leg_2_roll" value="${PI_2}"/>
+<xacro:property name="Leg_2_pitch" value="0.0"/>
+<xacro:property name="Leg_2_yaw" value="0.0"/>
 <!-- Origin -->
-<xacro:property name="Leg_3_Ox" value=" 0.000000 "/>
-<xacro:property name="Leg_3_Oy" value=" 0.3 "/>
-<xacro:property name="Leg_3_Oz" value=" -0.0036 "/>
-<xacro:property name="Leg_3_roll" value=" 3.14159265358979 "/>
-<xacro:property name="Leg_3_pitch" value=" 0.0 "/>
-<xacro:property name="Leg_3_yaw" value=" 1.5707963267948966 "/>
-<xacro:property name="Ankle_1_Ox" value=" 0.2 "/>
-<xacro:property name="Ankle_1_Oy" value=" 0.0 "/>
-<xacro:property name="Ankle_1_Oz" value=" -0.10015 "/>
-<xacro:property name="Ankle_1_roll" value=" 3.141592653589793 "/>
+<xacro:property name="Leg_3_Ox" value="0.0"/>
+<xacro:property name="Leg_3_Oy" value="${-300.000 * mmTom}"/>
+<xacro:property name="Leg_3_Oz" value="${-118.200 * mmTom}"/>
+<xacro:property name="Leg_3_roll" value="${PI}"/>
+<xacro:property name="Leg_3_pitch" value="0.0"/>
+<xacro:property name="Leg_3_yaw" value="0.0"/>
+<xacro:property name="Ankle_1_Ox" value="0.0"/>
+<xacro:property name="Ankle_1_Oy" value="${200.000 * mmTom}"/>
+<xacro:property name="Ankle_1_Oz" value="${-100.150 * mmTom}"/>
+<xacro:property name="Ankle_1_roll" value="${PI}"/>
 <xacro:property name="Ankle_1_pitch" value=" 0.0 "/>
 <xacro:property name="Ankle_1_yaw" value=" 0.0 "/>
-<xacro:property name="Ankle_2_Ox" value=" 0.0 "/>
-<xacro:property name="Ankle_2_Oy" value=" 0.0 "/>
-<xacro:property name="Ankle_2_Oz" value=" 0.0 "/>
-<xacro:property name="Ankle_2_roll" value=" 1.5707963267948966 "/>
-<xacro:property name="Ankle_2_pitch" value=" 0.0 "/>
-<xacro:property name="Ankle_2_yaw" value=" 1.5707963267948966 "/>
-<xacro:property name="Wheel_Ox" value=" 0.0 "/>
-<xacro:property name="Wheel_Oy" value=" 0.00085 "/>
-<xacro:property name="Wheel_Oz" value=" 0.237350 "/>
-<xacro:property name="Wheel_roll" value=" 1.5707963267948966 "/>
-<xacro:property name="Wheel_pitch" value=" 0.0 "/>
-<xacro:property name="Wheel_yaw" value=" 3.14159265359 "/>
+<xacro:property name="Ankle_2_Ox" value="${0.0 * mmTom}"/>
+<xacro:property name="Ankle_2_Oy" value="${-139.000 * mmTom}"/>
+<xacro:property name="Ankle_2_Oz" value="${0.850000 * mmTom}"/>
+<xacro:property name="Ankle_2_roll" value="${-PI_2}"/>
+<xacro:property name="Ankle_2_pitch" value="0.0"/>
+<xacro:property name="Ankle_2_yaw" value="'0.0'"/>
+<xacro:property name="Wheel_Ox" value="${0.0 * mmTom}"/>
+<xacro:property name="Wheel_Oy" value="${-52.3500 * mmTom}"/>
+<xacro:property name="Wheel_Oz" value="${-98.3500 * mmTom}"/>
+<xacro:property name="Wheel_roll" value="${PI_2}"/>
+<xacro:property name="Wheel_pitch" value="0.0"/>
+<xacro:property name="Wheel_yaw" value="0.0"/>
 <!-- Origin -->
 <xacro:property name="Torso_2_Ox" value=" 0.200 "/>

File: centauro_urdf/urdf/parts/legs.urdf.xacro (robot description, xacro)
@@ -2,11 +2,11 @@
 <robot xmlns:xacro="http://ros.org/wiki/xacro">
 <xacro:include filename="$(find centauro_urdf)/urdf/parts/centauro_leg.urdf.xacro" />
-<xacro:centauro_leg leg_num="1" origin_x="1" origin_y="-1">
+<xacro:centauro_leg leg_num="1" origin_x="1" origin_y="-1" mirror="-1">
 </xacro:centauro_leg>
-<xacro:centauro_leg leg_num="2" origin_x="1" origin_y="1">
+<xacro:centauro_leg leg_num="2" origin_x="1" origin_y="1" mirror="1">
 </xacro:centauro_leg>
-<xacro:centauro_leg leg_num="3" origin_x="-1" origin_y="-1">
+<xacro:centauro_leg leg_num="3" origin_x="-1" origin_y="-1" mirror="-1">
 </xacro:centauro_leg>
-<xacro:centauro_leg leg_num="4" origin_x="-1" origin_y="1">
+<xacro:centauro_leg leg_num="4" origin_x="-1" origin_y="1" mirror="1">
 </xacro:centauro_leg>
 </robot>

Commit message: fixed axis directions && centered wheel frame && linting

File: centauro_urdf/urdf/parts/centauro_leg.urdf.xacro (robot description, xacro)
@@ -28,18 +28,17 @@
 		<mass value="${Leg_2_mass}"/> <!-- org: 4.5 -->
 		<inertia ixx="${Leg_2_xx}" ixy="${Leg_2_xy}" ixz="${mirror*Leg_2_xz}" iyy="${Leg_2_yy}" iyz="${mirror*Leg_2_yz}" izz="${Leg_2_zz}"/>
-		<!-- <inertia ixx="0.01" ixy="0.01" ixz="0.01" iyy="0.01" iyz="0.01" izz="0.01"/> -->
-	</inertial>
-      <visual>
-         <origin xyz="0.0 0.0 0.0"  rpy="0.0 0.0 0.0"/>
-   <geometry>
-      <mesh filename="package://centauro_urdf/meshes/v2/hip-pitch.stl" scale="0.001 0.001 ${mirror*0.001}" />
-   </geometry>
-      </visual>
-      <collision>
-         <origin xyz="0.0 0.0 0.0"  rpy="0.0 0.0 0.0"/>
-   <geometry>
-      <mesh filename="package://centauro_urdf/meshes/simple/hip-pitch.stl" scale="0.001 ${0.001} 0.001" />
-   </geometry>
-      </collision>
+	</inertial>
+   <visual>
+      <origin xyz="0.0 0.0 0.0"  rpy="0.0 0.0 0.0"/>
+      <geometry>
+         <mesh filename="package://centauro_urdf/meshes/v2/hip-pitch.stl" scale="0.001 0.001 ${mirror*0.001}" />
+      </geometry>
+   </visual>
+   <collision>
+      <origin xyz="0.0 0.0 0.0"  rpy="0.0 0.0 0.0"/>
+      <geometry>
+         <mesh filename="package://centauro_urdf/meshes/simple/hip-pitch.stl" scale="0.001 ${0.001} 0.001" />
+      </geometry>
+   </collision>
 </link>
 <xacro:if value="${USE_STICKS}">
@@ -73,19 +72,18 @@
 		<mass value="${Leg_3_mass}"/>  <!-- org: 3.5, foot un modeled-->
 		<inertia ixx="${Leg_3_xx}" ixy="${Leg_3_xy}" ixz="${mirror*Leg_3_xz}" iyy="${Leg_3_yy}" iyz="${mirror*Leg_3_yz}" izz="${Leg_3_zz}"/>
-	<!--	<inertia ixx="0.01" ixy="0.01" ixz="0.01" iyy="0.01" iyz="0.01" izz="0.01"/>  -->
-	</inertial>
-      <visual>
-         <origin xyz="0.0 0.0 0.0"  rpy="0.0 0.0 0.0"/>
-   <geometry>
-      <mesh filename="package://centauro_urdf/meshes/v2/knee.stl" scale="0.001 0.001 ${mirror*0.001}" />
-   </geometry>
-         <material name="dark_grey"/>
-      </visual>
-      <collision>
-         <origin xyz="0.0 0.0 0.0"  rpy="0.0 0.0 0.0"/>
-   <geometry>
-      <mesh filename="package://centauro_urdf/meshes/simple/knee.stl" scale="0.001 ${0.001} 0.001" />
-   </geometry>
-      </collision>
+	</inertial>
+   <visual>
+      <origin xyz="0.0 0.0 0.0"  rpy="0.0 0.0 0.0"/>
+      <geometry>
+         <mesh filename="package://centauro_urdf/meshes/v2/knee.stl" scale="0.001 0.001 ${mirror*0.001}" />
+      </geometry>
+      <material name="dark_grey"/>
+   </visual>
+   <collision>
+      <origin xyz="0.0 0.0 0.0"  rpy="0.0 0.0 0.0"/>
+      <geometry>
+         <mesh filename="package://centauro_urdf/meshes/simple/knee.stl" scale="0.001 ${0.001} 0.001" />
+      </geometry>
+   </collision>
 </link>
 <link name="ankle1_${leg_num}">
@@ -94,18 +92,17 @@
 		<mass value="${Ankle_1_mass}"/>  <!-- org: 3.5, foot un modeled-->
 		<inertia ixx="${Ankle_1_xx}" ixy="${Ankle_1_xy}" ixz="${mirror*Ankle_1_xz}" iyy="${Ankle_1_yy}" iyz="${mirror*Ankle_1_yz}" izz="${Ankle_1_zz}"/>
-	<!--	<inertia ixx="0.01" ixy="0.01" ixz="0.01" iyy="0.01" iyz="0.01" izz="0.01"/>  -->
-	</inertial>
-      <visual>
-         <origin xyz="0.0 0.0 0.0"  rpy="0.0 0.0 0.0"/>
-   <geometry>
-      <mesh filename="package://centauro_urdf/meshes/v2/ankle-pitch.stl" scale="0.001 0.001 ${mirror*0.001}" />
-   </geometry>
-      </visual>
-      <collision>
-               <origin xyz="0.0 0.0 0.0"  rpy="0.0 0.0 0.0"/>
-   <geometry>
-      <mesh filename="package://centauro_urdf/meshes/simple/ankle-pitch.stl" scale="0.001 ${0.001} 0.001" />
-   </geometry>
-      </collision>
+	</inertial>
+   <visual>
+      <origin xyz="0.0 0.0 0.0"  rpy="0.0 0.0 0.0"/>
+      <geometry>
+         <mesh filename="package://centauro_urdf/meshes/v2/ankle-pitch.stl" scale="0.001 0.001 ${mirror*0.001}" />
+      </geometry>
+   </visual>
+   <collision>
+      <origin xyz="0.0 0.0 0.0"  rpy="0.0 0.0 0.0"/>
+      <geometry>
+         <mesh filename="package://centauro_urdf/meshes/simple/ankle-pitch.stl" scale="0.001 ${0.001} 0.001" />
+      </geometry>
+   </collision>
 </link>
 <link name="ankle2_${leg_num}">
@@ -115,53 +112,51 @@
 		<inertia ixx="${Ankle_2_xx}" ixy="${mirror*Ankle_2_xy}" ixz="${Ankle_2_xz}" iyy="${Ankle_2_yy}" iyz="${mirror*Ankle_2_yz}" izz="${Ankle_2_zz}"/>
 	</inertial>
-      <visual>
-         <origin xyz="0.0 0.0 0.0"  rpy="0.0 0.0 0.0"/>
-   <geometry>
-      <mesh filename="package://centauro_urdf/meshes/v2/ankle-yaw.stl" scale="0.001 ${origin_y*0.001} 0.001" />
-   </geometry>
-         <material name="dark_grey"/>
-      </visual>
-      <collision>
-         <origin xyz="0.0 0.0 0.0"  rpy="0.0 0.0 0.0"/>
-   <geometry>
-      <mesh filename="package://centauro_urdf/meshes/simple/ankle-yaw.stl" scale="0.001 ${0.001} 0.001" />
-   </geometry>
-      </collision>
-</link>
-<link name="wheel_${leg_num}">
+   <visual>
+      <origin xyz="0.0 0.0 0.0"  rpy="0.0 0.0 0.0"/>
+      <geometry>
+         <mesh filename="package://centauro_urdf/meshes/v2/ankle-yaw.stl" scale="0.001 ${origin_y*0.001} 0.001" />
+      </geometry>
+      <material name="dark_grey"/>
+   </visual>
+   <collision>
+      <origin xyz="0.0 0.0 0.0"  rpy="0.0 0.0 0.0"/>
+      <geometry>
+         <mesh filename="package://centauro_urdf/meshes/simple/ankle-yaw.stl" scale="0.001 ${0.001} 0.001" />
+      </geometry>
+   </collision>
+</link>
+<link name="wheel_cad_${leg_num}">
 	<inertial>
 		<origin xyz="${Wheel_x} ${Wheel_y} ${mirror*Wheel_z}"/>
-		<mass value="${Wheel_mass}"/>  <!-- org: 3.5, foot un modeled-->
+		<mass value="${Wheel_mass}"/>
 		<inertia ixx="${Wheel_xx}" ixy="${Wheel_xy}" ixz="${mirror*Wheel_xz}" iyy="${Wheel_yy}" iyz="${mirror*Wheel_yz}" izz="${Wheel_zz}"/>
 	</inertial>
-      <visual>
-         <origin xyz="0.0 0.0 0.0"  rpy="0.0 0.0 0.0"/>
-   <geometry>
-      <mesh filename="package://centauro_urdf/meshes/v2/wheel.stl" scale="0.001 0.001 ${mirror*0.001}" />
-   </geometry>
-         <material name="black"/>
-      </visual>
-      <!--collision>
-      	<origin xyz="0.0 0.0 0.0"  rpy="0.0 0.0 0.0"/>
-   		<geometry>
-      			<mesh filename="package://centauro_urdf/meshes/simple/wheel.stl" scale="0.001 ${0.001} 0.001" />
-   		</geometry>
-      </collision-->
+   <visual>
+      <origin xyz="0.0 0.0 0.0"  rpy="0.0 0.0 0.0"/>
+      <geometry>
+         <mesh filename="package://centauro_urdf/meshes/v2/wheel.stl" scale="0.001 0.001 ${mirror*0.001}" />
+      </geometry>
+      <material name="black"/>
+   </visual>
 	<collision>
 		<origin xyz="0 0 0" rpy="0 0 0"/>
 		<geometry>
 			<cylinder length="0.06" radius="0.078"/>
-      		</geometry>
+      </geometry>
 	</collision>
 </link>
 </xacro:unless>
 <!-- *****************************-->
-<link name="contact_${leg_num}">
-</link>
+<link name="contact_${leg_num}"/>
 <joint name="contact_joint_${leg_num}" type="fixed">
 	<parent link="ankle2_${leg_num}"/>
 	<child link="contact_${leg_num}"/>
-	<origin xyz="0 0 0.315" rpy="3.14159265 0 0"/>
-	<!--axis xyz="0 0 1" /-->
+	<origin xyz="0 0 -0.176" rpy="0 0 0"/>
+</joint>
+<link name="wheel_${leg_num}"/>
+<joint name="wheel_fixed_joint_${leg_num}" type="fixed">
+	<parent link="wheel_cad_${leg_num}"/>
+	<child link="wheel_${leg_num}"/>
+	<origin xyz="0 0 ${Wheel_z}" rpy="0 0 0"/>
 </joint>
 <!-- ******************************** -->
@@ -170,5 +165,5 @@
 	<child link="hip1_${leg_num}"/>
 	<origin xyz="${origin_x*Leg_1_Ox} ${origin_y*Leg_1_Oy} ${Leg_1_Oz}" rpy="${Leg_1_roll} ${Leg_1_pitch} ${Leg_1_yaw}"/>
-	<axis xyz="0 0 1"/>
+	<axis xyz="0 0 -1"/>
    <limit lower="${hip_yaw_lower[leg_num-1]}" upper="${hip_yaw_upper[leg_num-1]}" effort="${motor_A_effort}" velocity="${motor_A_velocity}"/> <!-- 200 Nm, 1 rad/s-->
 </joint>
@@ -177,5 +172,5 @@
 	<child link="hip2_${leg_num}"/>
 	<origin xyz="${Leg_2_Ox} ${mirror*Leg_2_Oy} ${Leg_2_Oz}" rpy="${Leg_2_roll} ${Leg_2_pitch} ${Leg_2_yaw}"/>
-	<axis xyz="0 0 1"/>
+	<axis xyz="0 0 ${mirror}"/>
    <limit lower="${hip_pitch_lower[leg_num-1]}" upper="${hip_pitch_upper[leg_num-1]}" effort="${motor_A_effort}" velocity="${motor_A_velocity}"/> <!-- 200 Nm, 1 rad/s-->
 </joint>
@@ -186,5 +181,5 @@
 	<origin xyz="${Leg_3_Ox} ${Leg_3_Oy} ${Leg_3_Oz}" rpy="${Leg_3_roll} ${Leg_3_pitch} ${Leg_3_yaw}"/>
 	<axis xyz="0 0 1"/>
-        <limit lower="${knee_pitch_lower[leg_num-1]}" upper="${knee_pitch_upper[leg_num-1]}" effort="${motor_A_effort}" velocity="${motor_A_velocity}"/> <!-- 200 Nm, 1 rad/s-->
+   <limit lower="${knee_pitch_lower[leg_num-1]}" upper="${knee_pitch_upper[leg_num-1]}" effort="${motor_A_effort}" velocity="${motor_A_velocity}"/> <!-- 200 Nm, 1 rad/s-->
 </joint>
 </xacro:if>
@@ -194,5 +189,5 @@
 	<child link="knee_${leg_num}"/>
 	<origin xyz="${Leg_3_Ox} ${Leg_3_Oy} ${mirror*Leg_3_Oz}" rpy="${Leg_3_roll} ${Leg_3_pitch} ${Leg_3_yaw}"/>
-	<axis xyz="0 0 1"/>
+	<axis xyz="0 0 ${mirror}"/>
    <limit lower="${knee_pitch_lower[leg_num-1]}" upper="${knee_pitch_upper[leg_num-1]}" effort="${motor_A_effort}" velocity="${motor_A_velocity}"/> <!-- 200 Nm, 1 rad/s-->
 </joint>
@@ -201,6 +196,6 @@
 	<child link="ankle1_${leg_num}"/>
 	<origin xyz="${Ankle_1_Ox} ${Ankle_1_Oy} ${mirror*Ankle_1_Oz}" rpy="${Ankle_1_roll} ${Ankle_1_pitch} ${Ankle_1_yaw}"/>
-	<axis xyz="0 0 1"/>
-        <limit lower="${ankle_pitch_lower[leg_num-1]}" upper="${ankle_pitch_upper[leg_num-1]}" effort="${motor_B_effort}" velocity="${motor_B_velocity}"/> <!-- 98 Nm, 1 rad/s-->
+	<axis xyz="0 0 ${mirror}"/>
+   <limit lower="${ankle_pitch_lower[leg_num-1]}" upper="${ankle_pitch_upper[leg_num-1]}" effort="${motor_B_effort}" velocity="${motor_B_velocity}"/> <!-- 98 Nm, 1 rad/s-->
 </joint>
 <joint name="ankle_yaw_${leg_num}" type="revolute">
@@ -208,13 +203,13 @@
 	<child link="ankle2_${leg_num}"/>
 	<origin xyz="${Ankle_2_Ox} ${Ankle_2_Oy} ${mirror*Ankle_2_Oz}" rpy="${Ankle_2_roll} ${Ankle_2_pitch} ${Ankle_2_yaw}"/>
-	<axis xyz="0 0 1"/>
-        <limit lower="${ankle_yaw_lower[leg_num-1]}" upper="${ankle_yaw_upper[leg_num-1]}" effort="${motor_C_effort}" velocity="${motor_C_velocity}"/>  <!-- 23 Nm, 1 rad/s-->
+	<axis xyz="0 0 -1"/>
+   <limit lower="${ankle_yaw_lower[leg_num-1]}" upper="${ankle_yaw_upper[leg_num-1]}" effort="${motor_C_effort}" velocity="${motor_C_velocity}"/>  <!-- 23 Nm, 1 rad/s-->
 </joint>
 <joint name="j_wheel_${leg_num}" type="continuous">
 	<parent link="ankle2_${leg_num}"/>
-	<child link="wheel_${leg_num}"/>
+	<child link="wheel_cad_${leg_num}"/>
 	<origin xyz="${Wheel_Ox} ${mirror*Wheel_Oy} ${Wheel_Oz}" rpy="${Wheel_roll} ${Wheel_pitch} ${Wheel_yaw}"/>
-	<axis xyz="0 0 1"/>
-        <limit  effort="${motor_C_effort}" velocity="${motor_C_velocity}"/>  <!-- 23 Nm, 1 rad/s-->
+	<axis xyz="0 0 ${mirror}"/>
+   <limit  effort="${motor_C_effort}" velocity="${motor_C_velocity}"/>  <!-- 23 Nm, 1 rad/s-->
 </joint>
 </xacro:unless>

Commit message: better wheel collision

File: centauro_urdf/urdf/parts/centauro_leg.urdf.xacro (robot description, xacro)
@@ -142,5 +142,5 @@
 		<origin xyz="0 0 0" rpy="0 0 0"/>
 		<geometry>
-			<cylinder length="0.06" radius="0.078"/>
+			<cylinder length="0.11" radius="0.078"/>
       </geometry>
 	</collision>

Commit message: parametric contact according to wheel radius and z position

File: centauro_urdf/urdf/parts/centauro_leg.urdf.xacro (robot description, xacro)
@@ -117,11 +117,20 @@
    </xacro:unless>
 </xacro:unless>
-<!-- *****************************-->
+<!-- *********** CONTACT FRAME ******************-->
 <link name="contact_${leg_num}"/>
-<joint name="contact_joint_${leg_num}" type="fixed">
-	<parent link="ankle2_${leg_num}"/>
-	<child link="contact_${leg_num}"/>
-	<origin xyz="0 0 -0.176" rpy="0 0 0"/>
-</joint>
+<xacro:if value="${USE_WHEEL_23}">
+	<joint name="contact_joint_${leg_num}" type="fixed">
+		<parent link="ankle2_${leg_num}"/>
+		<child link="contact_${leg_num}"/>
+		<origin xyz="0 0 ${Wheel23_Oz - Wheel23_radius}" rpy="0 0 0"/>
+	</joint>
+</xacro:if>
+<xacro:unless value="${USE_WHEEL_23}">
+	<joint name="contact_joint_${leg_num}" type="fixed">
+		<parent link="ankle2_${leg_num}"/>
+		<child link="contact_${leg_num}"/>
+		<origin xyz="0 0 ${Wheel_Oz - Wheel_radius}" rpy="0 0 0"/>
+	</joint>
+</xacro:unless>
 <!-- ******************************** -->
 <joint name="hip_yaw_${leg_num}" type="revolute">

File: centauro_urdf/urdf/parts/kinematics_properties.urdf.xacro (robot description, xacro)
@@ -66,4 +66,5 @@
 <xacro:property name="Wheel_pitch" value="0.0"/>
 <xacro:property name="Wheel_yaw" value="0.0"/>
+<xacro:property name="Wheel_radius" value="0.078"/>
 <xacro:property name="Wheel23_Ox" value="${0.0 * mmTom}"/>
 <xacro:property name="Wheel23_Oy" value="${0.0 * mmTom}"/>
@@ -72,4 +73,5 @@
 <xacro:property name="Wheel23_pitch" value="0.0"/>
 <xacro:property name="Wheel23_yaw" value="0.0"/>
+<xacro:property name="Wheel23_radius" value="0.124"/>
 <!-- Origin -->
 <xacro:property name="Torso_2_Ox" value=" 0.200 "/>
