Commit message: added neck dynamic parameters and meshes

File: centauro_urdf/urdf/parts/head.urdf.xacro (robot description, xacro)
@@ -3,7 +3,61 @@
 <!-- LINKS -->
 <!-- TODO: FINISH IMPLEMENTATION WITH CORRECT NUMBERS -->
-<link name="neck_1"/>
-<link name="neck_2"/>
-<link name="neck_3"/>
+<link name="neck_1">
+    <inertial>
+      <origin xyz="0.040479674 0.021377573 -0.014595112"/>
+      <mass value="0.33878686"/>
+      <inertia ixx="0.0003718568" ixy="-9.42983e-05" ixz="-2.80644e-05" iyy="0.0001886879" iyz="-1.54534e-05" izz="0.0005023443"/>
+    </inertial>
+    <visual>
+      <origin rpy="0.0 0.0 0.0" xyz="0.0 0 0.0"/>
+      <geometry>
+        <mesh filename="package://centauro_urdf/meshes/neck_yaw.stl" scale="0.001 0.001 0.001"/>
+      </geometry>
+    </visual>
+    <collision>
+      <origin rpy="0.0 0.0 0.0" xyz="0.0 0 0.0"/>
+      <geometry>
+        <mesh filename="package://centauro_urdf/meshes/simple/neck_yaw.stl" scale="0.001 0.001 0.001"/>
+      </geometry>
+    </collision>
+</link>
+<link name="neck_2">
+    <inertial>
+      <origin xyz="0.048466918 -0.059852318 -0.0085314894"/>
+      <mass value="0.78526942"/>
+      <inertia ixx="0.0004682345" ixy="-1.05438e-05" ixz="7.24398e-05" iyy="0.0002635246" iyz="1.6904e-06" izz="0.0003763351"/>
+    </inertial>
+    <visual>
+      <origin rpy="0.0 0.0 0.0" xyz="0.0 0 0.0"/>
+      <geometry>
+        <mesh filename="package://centauro_urdf/meshes/neck_pitch.stl" scale="0.001 0.001 0.001"/>
+      </geometry>
+    </visual>
+    <collision>
+      <origin rpy="0.0 0.0 0.0" xyz="0.0 0 0.0"/>
+      <geometry>
+        <mesh filename="package://centauro_urdf/meshes/simple/neck_pitch.stl" scale="0.001 0.001 0.001"/>
+      </geometry>
+    </collision>
+</link>
+<link name="neck_3">
+    <inertial>
+      <origin xyz="0.048466918 -0.059852318 -0.0085314894"/>
+      <mass value="0.78526942"/>
+      <inertia ixx="0.0004682345" ixy="-1.05438e-05" ixz="7.24398e-05" iyy="0.0002635246" iyz="1.6904e-06" izz="0.0003763351"/>
+    </inertial>
+    <visual>
+      <origin rpy="0.0 0.0 0.0" xyz="0.0 0 0.0"/>
+      <geometry>
+        <mesh filename="package://centauro_urdf/meshes/lidar.stl" scale="0.001 0.001 0.001"/>
+      </geometry>
+    </visual>
+    <collision>
+      <origin rpy="0.0 0.0 0.0" xyz="0.0 0 0.0"/>
+      <geometry>
+        <mesh filename="package://centauro_urdf/meshes/simple/lidar.stl" scale="0.001 0.001 0.001"/>
+      </geometry>
+    </collision>
+</link>
 <!--JOINTS -->
 <joint name="neck_yaw" type="revolute">

Commit message: added realsense

File: centauro_urdf/urdf/parts/head.urdf.xacro (robot description, xacro)
@@ -86,3 +86,27 @@
     <dynamics damping="0.2" friction="10.0"/>
 </joint>
+<xacro:if value="${ADD_INTEL_D435I}">
+        <xacro:include filename="$(find realsense_gazebo_description)/urdf/_d435i.urdf.xacro" />
+       <!-- <xacro:sensor_d435i parent="torso_2" name="d435i_camera" topics_ns="d435i_camera"
+                            enable_pointCloud="true" align_depth="true">
+            <origin xyz="0.13 0 0.03" rpy="0 0.25 0"/>
+        </xacro:sensor_d435i>-->
+        <xacro:sensor_d435i parent="neck_2" name="D435i_head_camera" topics_ns="D435i/D435i_head_camera"
+                      enable_pointCloud="true" align_depth="true"
+                      unite_imu_method="false"
+                      visualize="true"
+                      accel_fps="300"
+                      gyro_fps="300"
+                      depth_width="1280"
+                      depth_height="720"
+                      depth_fps="90"
+                      infra_width="1280"
+                      infra_height="720"
+                      infra_fps="90"
+                      color_width="1280"
+                      color_height="720"
+                      color_fps="30">
+            <origin xyz="0.219831 0 -0.0613293" rpy="0.0 0.5585052 0.0"/>
+        </xacro:sensor_d435i>
+    </xacro:if>
 </robot>

Commit message: temporary remedy for neck_yaw joint until urdf is updated with new head data

File: centauro_urdf/urdf/parts/head.urdf.xacro (robot description, xacro)
@@ -62,5 +62,5 @@
 </link>
 <!--JOINTS -->
-<joint name="neck_yaw" type="revolute">
+<joint name="neck_yaw" type="fixed">
     <parent link="torso_2"/>
     <origin xyz="0.0 0.0 0.2795"/>

Commit message: added D435_head_camera frames so xbot publish their tf always

File: centauro_urdf/urdf/parts/head.urdf.xacro (robot description, xacro)
@@ -85,9 +85,16 @@
     <dynamics friction="10.0"/>
   </joint>
+  <xacro:property name="d435_head_name" value="D435_head_camera" />
+  <xacro:property name="d435_head_parent_name" value="d435_head_motor" />
+  <xacro:property name="d435_head_origin">
+    <origin xyz="0.03015 0 -0.0125" rpy="0 0 0"/>
+  </xacro:property>
+  <xacro:property name="M_PI" value="3.1415926535897931"/>
   <xacro:if value="${ADD_D435I_HEAD}">
-    <xacro:include filename="$(find realsense_gazebo_description)/urdf/_d435i.urdf.xacro" />
-    <xacro:sensor_d435i parent="d435_head_motor"
-        name="D435_head_camera"
-        topics_ns="D435/D435_head_camera"
+<!--    <xacro:include filename="$(find realsense_gazebo_description)/urdf/_d435i.urdf.xacro" />-->
+    <xacro:include filename="$(find realsense2_description)/urdf/_d435i.urdf.xacro" />
+    <xacro:sensor_d435i parent="${d435_head_parent_name}"
+        name="${d435_head_name}"
+        topics_ns="D435/${d435_head_name}"
         enable_pointCloud="true"
         align_depth="true"
@@ -105,7 +112,51 @@
         color_height="720"
         color_fps="30">
-      <origin xyz="0.03015 0 -0.0125" rpy="0 0 0"/>
+        <xacro:insert_block name="d435_head_origin" />
     </xacro:sensor_d435i>
   </xacro:if>
+  <xacro:unless value="${ADD_D435I_HEAD}">
+    <!--  Copied from _d435.urdf.xacro    -->
+    <xacro:property name="d435_cam_width" value="0.090"/>
+    <xacro:property name="d435_cam_height" value="0.025"/>
+    <xacro:property name="d435_cam_depth" value="0.02505"/>
+    <xacro:property name="d435_cam_mount_from_center_offset" value="0.0149"/>
+    <xacro:property name="d435_cam_depth_px" value="${d435_cam_mount_from_center_offset}"/>
+    <xacro:property name="d435_cam_depth_py" value="0.0175"/>
+    <xacro:property name="d435_cam_depth_pz" value="${d435_cam_height/2}"/>
+    <!-- camera body, with origin at bottom screw mount -->
+    <joint name="${d435_head_name}_joint" type="fixed">
+      <xacro:insert_block name="d435_head_origin"/>
+      <parent link="${d435_head_parent_name}"/>
+      <child link="${d435_head_name}_bottom_screw_frame"/>
+    </joint>
+    <link name="${d435_head_name}_bottom_screw_frame"/>
+    <joint name="${d435_head_name}_link_joint" type="fixed">
+      <origin xyz="0 ${d435_cam_depth_py} ${d435_cam_depth_pz}" rpy="0 0 0"/>
+      <parent link="${d435_head_name}_bottom_screw_frame"/>
+      <child link="${d435_head_name}_link"/>
+    </joint>
+    <link name="${d435_head_name}_link">
+      <visual>
+      <origin xyz="${d435_cam_mount_from_center_offset} ${-d435_cam_depth_py} 0" rpy="${M_PI/2} 0 ${M_PI/2}"/>
+        <geometry>
+          <!-- <box size="${d435_cam_width} ${d435_cam_height} ${d435_cam_depth}"/> -->
+          <mesh filename="package://centauro_urdf/meshes/realsense/d435.dae"/>
+        </geometry>
+        <material name="${d435_head_name}_aluminum"/>
+      </visual>
+      <collision>
+        <origin xyz="0 ${-d435_cam_depth_py} 0" rpy="0 0 0"/>
+        <geometry>
+        <box size="${d435_cam_depth} ${d435_cam_width} ${d435_cam_height}"/>
+        </geometry>
+      </collision>
+      <inertial>
+        <!-- The following are not reliable values, and should not be used for modeling -->
+        <mass value="0.564"/>
+        <origin xyz="0 0 0"/>
+        <inertia ixx="0.003881243" ixy="0.0" ixz="0.0" iyy="0.000498940" iyz="0.0" izz="0.003879257"/>
+      </inertial>
+    </link>
+  </xacro:unless>
   <xacro:if value="${ADD_VELODYNE}">
     <xacro:include filename="$(find velodyne_description)/urdf/VLP-16.urdf.xacro"/>

Commit message: use PI variable from utils

File: centauro_urdf/urdf/parts/head.urdf.xacro (robot description, xacro)
@@ -90,5 +90,4 @@
     <origin xyz="0.03015 0 -0.0125" rpy="0 0 0"/>
   </xacro:property>
-  <xacro:property name="M_PI" value="3.1415926535897931"/>
   <xacro:if value="${ADD_D435I_HEAD}">
     <xacro:include filename="$(find realsense_gazebo_description)/urdf/_d435i.urdf.xacro" />
@@ -137,5 +136,5 @@
     <link name="${d435_head_name}_link">
       <visual>
-      <origin xyz="${d435_cam_mount_from_center_offset} ${-d435_cam_depth_py} 0" rpy="${M_PI/2} 0 ${M_PI/2}"/>
+      <origin xyz="${d435_cam_mount_from_center_offset} ${-d435_cam_depth_py} 0" rpy="${PI/2} 0 ${PI/2}"/>
         <geometry>
           <!-- <box size="${d435_cam_width} ${d435_cam_height} ${d435_cam_depth}"/> -->

Commit message: Update main head inertia (missing camera supports)

File: centauro_urdf/urdf/parts/head.urdf.xacro (robot description, xacro)
@@ -5,7 +5,7 @@
     <inertial>
       <origin xyz="0 0 0"/>
-      <mass value="0.33878686"/>
+      <mass value="2.146"/>
       <!-- MASS/INERTIA TO DO -->
-      <inertia ixx="0.0003718568" ixy="-9.42983e-05" ixz="-2.80644e-05" iyy="0.0001886879" iyz="-1.54534e-05" izz="0.0005023443"/>
+      <inertia ixx="${3.6754716e+04*mm2Tom2}" ixy="${-1.7440409e+02*mm2Tom2}" ixz="${-1.1571084e+03*mm2Tom2}" iyy="${3.7072505e+04*mm2Tom2}" iyz="${-1.4217709e+03*mm2Tom2}" izz="${3.5983886e+03*mm2Tom2}"/>
     </inertial>
     <visual>

Commit message: added calib frame

File: centauro_urdf/urdf/parts/head.urdf.xacro (robot description, xacro)
@@ -62,4 +62,10 @@
     </collision>
   </link>
+  <link name="d435_head_calib"/>
+  <joint name="d435_head_calib_joint" type="fixed">
+    <parent link="d435_head_motor"/>
+    <child link="d435_head_calib"/>
+    <!-- <origin xyz="1.06832322 0.03353594 0.1387841" rpy="-0.03851041 0.29866375 -0.06730427"/> -->
+  </joint>
   <!--JOINTS -->
   <joint name="neck_base" type="fixed">
@@ -86,5 +92,5 @@
   </joint>
   <xacro:property name="d435_head_name" value="D435_head_camera" />
-  <xacro:property name="d435_head_parent_name" value="d435_head_motor" />
+  <xacro:property name="d435_head_parent_name" value="d435_head_calib" />
   <xacro:property name="d435_head_origin">
     <origin xyz="0.03015 0 -0.0125" rpy="0 0 0"/>
