Commit message: armX_8 always to compliance with srdf file

File: centauro_urdf/urdf/parts/arms.urdf.xacro (robot description, xacro)
@@ -9,39 +9,115 @@
       <origin xyz="${Shoulder_1_Ox} ${-Shoulder_1_Oy} ${Shoulder_1_Oz}" rpy="${-Shoulder_1_roll} ${Shoulder_1_pitch} ${-Shoulder_1_yaw}" />
 </xacro:centauro_arm>
+<xacro:if value="${END_EFFECTOR_LEFT == 'none'}">
+	<xacro:property name="arm_num" value="1" />
+    <!-- add armX_8 link for compliance with srdf file -->
+	<joint name="j_none_${arm_num}_final" type="fixed">
+		  <parent link="arm${arm_num}_6"/>
+		  <child link="arm${arm_num}_8"/>
+	</joint>
+	<link name="arm${arm_num}_8">
+		<inertial>
+		  <mass value="0"/>
+		  <inertia ixx="0" ixy="0" ixz="0" iyy="0" iyz="0" izz="0"/>
+		</inertial>
+	</link>
+</xacro:if>
+<xacro:if value="${END_EFFECTOR_RIGHT == 'none'}">
+	<xacro:property name="arm_num" value="2" />
+    <!-- add armX_8 link for compliance with srdf file -->
+	<joint name="j_none_${arm_num}_final" type="fixed">
+		  <parent link="arm${arm_num}_6"/>
+		  <child link="arm${arm_num}_8"/>
+	</joint>
+	<link name="arm${arm_num}_8">
+		<inertial>
+		  <mass value="0"/>
+		  <inertia ixx="0" ixy="0" ixz="0" iyy="0" iyz="0" izz="0"/>
+		</inertial>
+	</link>
+</xacro:if>
 <xacro:if value="${END_EFFECTOR_LEFT == 'ball'}">
-      <xacro:include filename="$(find centauro_urdf)/urdf/parts/ball.urdf.xacro" />
-      <xacro:ball_end_effector arm_num="1"  parent_link="arm1_6">
-                  <origin xyz="0. -0.05 -0.105" rpy="0. 0. 0."/>
-      </xacro:ball_end_effector>
+	<xacro:include filename="$(find centauro_urdf)/urdf/parts/ball.urdf.xacro" />
+	<xacro:ball_end_effector arm_num="1"  parent_link="arm1_6">
+		      <origin xyz="0. -0.05 -0.105" rpy="0. 0. 0."/>
+	</xacro:ball_end_effector>
 </xacro:if>
 <xacro:if value="${END_EFFECTOR_RIGHT == 'ball'}">
-      <xacro:include filename="$(find centauro_urdf)/urdf/parts/ball.urdf.xacro" />
-      <xacro:ball_end_effector arm_num="2"  parent_link="arm2_6">
-                  <origin xyz="0. 0.05 -0.105" rpy="0. 0. 0."/>
-      </xacro:ball_end_effector>
+	<xacro:include filename="$(find centauro_urdf)/urdf/parts/ball.urdf.xacro" />
+	<xacro:ball_end_effector arm_num="2"  parent_link="arm2_6">
+	 <origin xyz="0. 0.05 -0.105" rpy="0. 0. 0."/>
+	</xacro:ball_end_effector>
 </xacro:if>
 <xacro:if value="${END_EFFECTOR_LEFT == 'dagana_fixed'}">
-	  <xacro:include filename="$(find dagana_urdf)/urdf/dagana_macro.urdf.xacro" />
-	  <xacro:dagana_gripper name="dagana_1" parent_link="arm1_6" joint_type="fixed">
-	    <origin xyz="0. -0.05 -0.08" rpy="0. ${PI} 0"/>
-	  </xacro:dagana_gripper>
+	<xacro:property name="arm_num" value="1" />
+	<xacro:include filename="$(find dagana_urdf)/urdf/dagana_macro.urdf.xacro" />
+	<xacro:dagana_gripper name="dagana_${arm_num}" parent_link="arm${arm_num}_6" joint_type="fixed">
+		<origin xyz="0. -0.05 -0.08" rpy="0. ${PI} 0"/>
+	</xacro:dagana_gripper>
+    <!-- add armX_8 link for compliance with srdf file -->
+	<joint name="j_dagana_${arm_num}_final" type="fixed">
+		  <parent link="dagana_${arm_num}_bottom_link"/>
+		  <child link="arm${arm_num}_8"/>
+	</joint>
+	<link name="arm${arm_num}_8">
+		<inertial>
+		  <mass value="0"/>
+		  <inertia ixx="0" ixy="0" ixz="0" iyy="0" iyz="0" izz="0"/>
+		</inertial>
+	</link>
 </xacro:if>
 <xacro:if value="${END_EFFECTOR_RIGHT == 'dagana_fixed'}">
-      <xacro:include filename="$(find dagana_urdf)/urdf/dagana_macro.urdf.xacro" />
-	  <xacro:dagana_gripper name="dagana_2" parent_link="arm2_6" joint_type="fixed">
-	    <origin xyz="0. 0.05 -0.08" rpy="0. ${PI} ${PI}"/>
-	  </xacro:dagana_gripper>
+	<xacro:property name="arm_num" value="2" />
+	<xacro:include filename="$(find dagana_urdf)/urdf/dagana_macro.urdf.xacro" />
+	<xacro:dagana_gripper name="dagana_${arm_num}" parent_link="arm${arm_num}_6" joint_type="fixed">
+		<origin xyz="0. 0.05 -0.08" rpy="0. ${PI} ${PI}"/>
+	</xacro:dagana_gripper>
+    <!-- add armX_8 link for compliance with srdf file -->
+	<joint name="j_dagana_${arm_num}_final" type="fixed">
+		  <parent link="dagana_${arm_num}_bottom_link"/>
+		  <child link="arm${arm_num}_8"/>
+	</joint>
+	<link name="arm${arm_num}_8">
+		<inertial>
+		  <mass value="0"/>
+		  <inertia ixx="0" ixy="0" ixz="0" iyy="0" iyz="0" izz="0"/>
+		</inertial>
+	</link>
 </xacro:if>
 <xacro:if value="${END_EFFECTOR_LEFT == 'dagana'}">
-	  <xacro:include filename="$(find dagana_urdf)/urdf/dagana_macro.urdf.xacro" />
-	  <xacro:dagana_gripper name="dagana_1" parent_link="arm1_6" joint_type="revolute">
-	    <origin xyz="0. -0.05 -0.08" rpy="0. ${PI} 0"/>
-	  </xacro:dagana_gripper>
+	<xacro:property name="arm_num" value="1" />
+	<xacro:include filename="$(find dagana_urdf)/urdf/dagana_macro.urdf.xacro" />
+	<xacro:dagana_gripper name="dagana_${arm_num}" parent_link="arm${arm_num}_6" joint_type="fixed">
+		<origin xyz="0. -0.05 -0.08" rpy="0. ${PI} 0"/>
+	</xacro:dagana_gripper>
+    <!-- add armX_8 link for compliance with srdf file -->
+	<joint name="j_dagana_${arm_num}_final" type="fixed">
+		  <parent link="dagana_${arm_num}_bottom_link"/>
+		  <child link="arm${arm_num}_8"/>
+	</joint>
+	<link name="arm${arm_num}_8">
+		<inertial>
+		  <mass value="0"/>
+		  <inertia ixx="0" ixy="0" ixz="0" iyy="0" iyz="0" izz="0"/>
+		</inertial>
+	</link>
 </xacro:if>
 <xacro:if value="${END_EFFECTOR_RIGHT == 'dagana'}">
-      <xacro:include filename="$(find dagana_urdf)/urdf/dagana_macro.urdf.xacro" />
-	  <xacro:dagana_gripper name="dagana_2" parent_link="arm2_6" joint_type="revolute">
-	    <origin xyz="0. 0.05 -0.08" rpy="0. ${PI} ${PI}"/>
-	  </xacro:dagana_gripper>
+	<xacro:property name="arm_num" value="2" />
+	<xacro:include filename="$(find dagana_urdf)/urdf/dagana_macro.urdf.xacro" />
+	<xacro:dagana_gripper name="dagana_${arm_num}" parent_link="arm${arm_num}_6" joint_type="fixed">
+		<origin xyz="0. 0.05 -0.08" rpy="0. ${PI} ${PI}"/>
+	</xacro:dagana_gripper>
+    <!-- add armX_8 link for compliance with srdf file -->
+	<joint name="j_dagana_${arm_num}_final" type="fixed">
+		  <parent link="dagana_${arm_num}_bottom_link"/>
+		  <child link="arm${arm_num}_8"/>
+	</joint>
+	<link name="arm${arm_num}_8">
+		<inertial>
+		  <mass value="0"/>
+		  <inertia ixx="0" ixy="0" ixz="0" iyy="0" iyz="0" izz="0"/>
+		</inertial>
+	</link>
 </xacro:if>
 </robot>

Commit message: dagana

File: centauro_urdf/urdf/parts/arms.urdf.xacro (robot description, xacro)
@@ -71,5 +71,5 @@
 	<xacro:include filename="$(find dagana_urdf)/urdf/dagana_macro.urdf.xacro" />
 	<xacro:dagana_gripper name="dagana_${arm_num}" parent_link="arm${arm_num}_6" joint_type="fixed">
-		<origin xyz="0. 0.05 -0.08" rpy="0. ${PI} ${PI}"/>
+		<origin xyz="0. 0.05 -0.08" rpy="0. ${PI} 0"/>
 	</xacro:dagana_gripper>
     <!-- add armX_8 link for compliance with srdf file -->

Commit message: dagana rotated correctly

File: centauro_urdf/urdf/parts/arms.urdf.xacro (robot description, xacro)
@@ -71,5 +71,5 @@
 	<xacro:include filename="$(find dagana_urdf)/urdf/dagana_macro.urdf.xacro" />
 	<xacro:dagana_gripper name="dagana_${arm_num}" parent_link="arm${arm_num}_6" joint_type="fixed">
-		<origin xyz="0. 0.05 -0.08" rpy="0. ${PI} ${PI}"/>
+		<origin xyz="0. 0.05 -0.08" rpy="0. ${PI} 0"/>
 	</xacro:dagana_gripper>
     <!-- add armX_8 link for compliance with srdf file -->
@@ -107,5 +107,5 @@
 	<xacro:include filename="$(find dagana_urdf)/urdf/dagana_macro.urdf.xacro" />
 	<xacro:dagana_gripper name="dagana_${arm_num}" parent_link="arm${arm_num}_6" joint_type="revolute">
-		<origin xyz="0. 0.05 -0.08" rpy="0. ${PI} ${PI}"/>
+		<origin xyz="0. 0.05 -0.08" rpy="0. ${PI} 0"/>
 	</xacro:dagana_gripper>
     <!-- add armX_8 link for compliance with srdf file -->
