Commit message: fixed duplicate param

File: centauro_urdf/urdf/parts/wheel23.urdf.xacro (robot description, xacro)
@@ -54,7 +54,10 @@
                 <origin xyz="0 0 0" rpy="0 0 0" />
                 <geometry>
+					<cylinder radius="${wheel23_radius}" length="${wheel23_depth}"/>
+				</geometry>
+                <!-- <geometry>
                     <mesh filename="${MESH_PATH}/v2/collision/mesh_wheel23.stl"
                         scale="0.001 0.001 ${mirror*0.001}" />
-                </geometry>
+                </geometry> -->
                 <material name="black" />
             </collision>

Commit message: added contact link

File: centauro_urdf/urdf/parts/wheel23.urdf.xacro (robot description, xacro)
@@ -58,10 +58,4 @@
                     </geometry>
                 </xacro:if>
-                <xacro:if value="${USE_WHEEL_23_SMALL_SPHERE_COLLISION}">
-                    <origin xyz="0 ${-(0.125-0.015)} 0" rpy="0 0 0" />
-                    <geometry>
-                        <sphere radius="0.015" />
-                    </geometry>
-                </xacro:if>
                 <xacro:unless value="${USE_WHEEL_23_SMALL_SPHERE_COLLISION or USE_WHEEL_23_SPHERE_COLLISION}">
                     <origin xyz="0 0 0" rpy="0 0 0" />
@@ -74,4 +68,31 @@
             </collision>
         </link>
+        <link name="wheel_contact_${leg_num}">
+            <inertial>
+                <origin xyz="0 0 0"/>
+                <mass value="0.001"/>
+                <inertia ixx="6.4e-7" ixy="0.0" ixz="0.0" iyy="6.4e-7" iyz="0.0" izz="6.4e-7"/>
+            </inertial>
+            <visual>
+                <origin xyz="0 0 0" rpy="0 0 0"/>
+                <geometry>
+                    <sphere radius="0.015"/>
+                </geometry>
+                <material name="white"/>
+            </visual>
+            <xacro:if value="${USE_WHEEL_23_SMALL_SPHERE_COLLISION}">
+                <collision name="wheel_contact_${leg_num}">
+                    <origin xyz="0 0 0" rpy="0 0 0"/>
+                    <geometry>
+                        <sphere radius="0.015"/>
+                    </geometry>
+                </collision>
+            </xacro:if>
+        </link>
+        <joint name="wheel_contact_${leg_num}_joint" type="fixed">
+            <parent link="wheel_${leg_num}"/>
+            <child link="wheel_contact_${leg_num}"/>
+            <origin xyz="0 ${-(0.125-0.015)} 0" rpy="0 0 0"/>
+        </joint>
     </xacro:macro>
     <!-- /macro arms -->

Commit message: Moved small sphere collision to contact link

File: centauro_urdf/urdf/parts/wheel23.urdf.xacro (robot description, xacro)
@@ -51,12 +51,15 @@
                 <material name="black" />
             </visual>
-            <collision>
-                <xacro:if value="${USE_WHEEL_23_SPHERE_COLLISION}">
+            <xacro:if value="${USE_WHEEL_23_SPHERE_COLLISION}">
+                <collision>
                     <origin xyz="0 0 0" rpy="0 0 0" />
                     <geometry>
                         <sphere radius="0.125"/>
                     </geometry>
-                </xacro:if>
-                <xacro:unless value="${USE_WHEEL_23_SMALL_SPHERE_COLLISION or USE_WHEEL_23_SPHERE_COLLISION}">
+                    <material name="black" />
+                </collision>
+            </xacro:if>
+            <xacro:unless value="${USE_WHEEL_23_SMALL_SPHERE_COLLISION or USE_WHEEL_23_SPHERE_COLLISION}">
+                <collision>
                     <origin xyz="0 0 0" rpy="0 0 0" />
                     <geometry>
@@ -64,7 +67,7 @@
                                 scale="0.001 0.001 ${mirror*0.001}" />
                     </geometry>
-                </xacro:unless>
-                <material name="black" />
-            </collision>
+                    <material name="black" />
+                </collision>
+            </xacro:unless>
         </link>
         <link name="wheel_contact_${leg_num}">

Commit message: wheel ellipsoid

File: centauro_urdf/urdf/parts/wheel23.urdf.xacro (robot description, xacro)
@@ -57,4 +57,11 @@
                         <sphere radius="0.125"/>
                     </geometry>
+                    <adarl>
+                        <!--
+                        Override collision geometry to an ellipsoid when using adarl
+                        This for example works for mujoco, which supports ellipsoids.
+                        -->
+                        <override type="ellipsoid" size="0.12 0.12 0.06"/>
+                    </adarl>
                     <material name="black" />
                 </collision>
@@ -88,5 +95,5 @@
                     <origin xyz="0 0 0" rpy="0 0 0"/>
                     <geometry>
-                        <sphere radius="0.015"/>
+                        <sphere radius="0.05"/>
                     </geometry>
                 </collision>
@@ -94,7 +101,10 @@
         </link>
         <joint name="wheel_contact_${leg_num}_joint" type="fixed">
-            <parent link="wheel_${leg_num}"/>
-            <child link="wheel_contact_${leg_num}"/>
-            <origin xyz="0 ${-(0.125-0.015)} 0" rpy="0 0 0"/>
+            <parent link="ankle2_${leg_num}" />
+            <child link="wheel_contact_${leg_num}" />
+            <origin xyz="${Wheel23_Ox} ${mirror*Wheel23_Oy} ${Wheel23_Oz-(0.125-0.015)}"
+                rpy="${Wheel23_roll} ${Wheel23_pitch} ${Wheel23_yaw}" />
+            <axis xyz="0 0 ${mirror}" />
+            <limit effort="${motor_C_effort}" velocity="${motor_C_velocity}" />  <!-- 23 Nm, 1 rad/s-->
         </joint>
     </xacro:macro>
