Commit message: updated capsule files

File: centauro_urdf/urdf/capsule/centauro_capsules.urdf (robot description, URDF)
Before this commit: robot centauro, 58 links, 57 joints
Links:
- link ankle1_1: mass 1.2380744 -> 1.4023368; geometry collision cylinder length=0.0492563156661 radius=0.0792379; collision sphere radius=0.0792379
- link ankle1_2: mass 1.2380744 -> 1.4023368; geometry collision cylinder length=0.0478840512856 radius=0.0781037; collision sphere radius=0.0781037
- link ankle1_3: mass 1.2380744 -> 1.4023368; geometry collision cylinder length=0.0492563156661 radius=0.0792379; collision sphere radius=0.0792379
- link ankle1_4: mass 1.2380744 -> 1.4023368; geometry collision cylinder length=0.0478840512856 radius=0.0781037; collision sphere radius=0.0781037
- link ankle2_1: mass 1.1565926 -> 1.7656714; geometry collision cylinder length=0.0737026312964 radius=0.0813545; collision sphere radius=0.0813545
- link ankle2_2: mass 1.1565926 -> 1.7656714; geometry collision cylinder length=0.0737026312964 radius=0.0813545; collision sphere radius=0.0813545
- link ankle2_3: mass 1.1565926 -> 1.7656714; geometry collision cylinder length=0.0737026312964 radius=0.0813545; collision sphere radius=0.0813545
- link ankle2_4: mass 1.1565926 -> 1.7656714; geometry collision cylinder length=0.0737026312964 radius=0.0813545; collision sphere radius=0.0813545
- link hip1_1: mass 1.9194403 -> 2.3349153; geometry collision cylinder length=0.030695458899 radius=0.0747223; collision sphere radius=0.0747223
- link hip1_2: mass 1.9194403 -> 2.3349153; geometry collision cylinder length=0.030695458899 radius=0.0747223; collision sphere radius=0.0747223
- link hip1_3: mass 1.9194403 -> 2.3349153; geometry collision cylinder length=0.030695458899 radius=0.0747223; collision sphere radius=0.0747223
- link hip1_4: mass 1.9194403 -> 2.3349153; geometry collision cylinder length=0.030695458899 radius=0.0747223; collision sphere radius=0.0747223
- link hip2_1: mass 2.7264471 -> 3.4572118; geometry collision cylinder length=0.291980452173 radius=0.0808941; collision sphere radius=0.0808941
- link hip2_2: mass 2.7264471 -> 3.4572118; geometry collision cylinder length=0.291980452173 radius=0.0808941; collision sphere radius=0.0808941
- link hip2_3: mass 2.7264471 -> 3.4572118; geometry collision cylinder length=0.291980452173 radius=0.0808941; collision sphere radius=0.0808941
- link hip2_4: mass 2.7264471 -> 3.4572118; geometry collision cylinder length=0.291980452173 radius=0.0808941; collision sphere radius=0.0808941
- link knee_1: mass 1.9356754 -> 2.1199315; geometry collision cylinder length=0.192750224606 radius=0.0664305; collision sphere radius=0.0664305
- link knee_2: mass 1.9356754 -> 2.1199315; geometry collision cylinder length=0.192750224606 radius=0.0664305; collision sphere radius=0.0664305
- link knee_3: mass 1.9356754 -> 2.1199315; geometry collision cylinder length=0.192750224606 radius=0.0664305; collision sphere radius=0.0664305
- link knee_4: mass 1.9356754 -> 2.1199315; geometry collision cylinder length=0.192750224606 radius=0.0664305; collision sphere radius=0.0664305
- link pelvis: mass 16.097574 -> 26.584529; geometry collision cylinder length=0.385941397914 radius=0.213204; collision sphere radius=0.213204
- link torso_2: mass 11.492689 -> 12.553731
- link wheel_1: mass 1.7289003 -> 1.11164; geometry collision cylinder length=0.11 radius=0.078; visual mesh filename=package://centauro_urdf/meshes/v2/wheel.stl scale=0.001 0.001 -0.001
- link wheel_2: mass 1.7289003 -> 1.11164; geometry collision cylinder length=0.11 radius=0.078; visual mesh filename=package://centauro_urdf/meshes/v2/wheel.stl scale=0.001 0.001 0.001
- link wheel_3: mass 1.7289003 -> 1.11164; geometry collision cylinder length=0.11 radius=0.078; visual mesh filename=package://centauro_urdf/meshes/v2/wheel.stl scale=0.001 0.001 -0.001
- link wheel_4: mass 1.7289003 -> 1.11164; geometry collision cylinder length=0.11 radius=0.078; visual mesh filename=package://centauro_urdf/meshes/v2/wheel.stl scale=0.001 0.001 0.001
Joints:
- joint ankle_pitch_1: axis 0.0 0.0 1.0 -> 0.0 0.0 -1.0; origin xyz=0.2 0.0 -0.10015 rpy=3.14159265359 0.0 0.0 -> xyz=0.0 0.2 0.10015 rpy=3.14159265359 0.0 0.0
- joint ankle_pitch_2: origin xyz=0.2 0.0 -0.10015 rpy=3.14159265359 0.0 0.0 -> xyz=0.0 0.2 -0.10015 rpy=3.14159265359 0.0 0.0
- joint ankle_pitch_3: axis 0.0 0.0 1.0 -> 0.0 0.0 -1.0; origin xyz=0.2 0.0 -0.10015 rpy=3.14159265359 0.0 0.0 -> xyz=0.0 0.2 0.10015 rpy=3.14159265359 0.0 0.0
- joint ankle_pitch_4: origin xyz=0.2 0.0 -0.10015 rpy=3.14159265359 0.0 0.0 -> xyz=0.0 0.2 -0.10015 rpy=3.14159265359 0.0 0.0
- joint ankle_yaw_1: axis 0.0 0.0 1.0 -> 0.0 0.0 -1.0; origin xyz=0.0 0.0 0.0 rpy=1.57079632679 0.0 1.57079632679 -> xyz=0.0 -0.139 -0.00085 rpy=-1.57079632679 0.0 0.0
- joint ankle_yaw_2: axis 0.0 0.0 1.0 -> 0.0 0.0 -1.0; origin xyz=0.0 0.0 0.0 rpy=1.57079632679 0.0 1.57079632679 -> xyz=0.0 -0.139 0.00085 rpy=-1.57079632679 0.0 0.0
- joint ankle_yaw_3: axis 0.0 0.0 1.0 -> 0.0 0.0 -1.0; origin xyz=0.0 0.0 0.0 rpy=1.57079632679 0.0 1.57079632679 -> xyz=0.0 -0.139 -0.00085 rpy=-1.57079632679 0.0 0.0
- joint ankle_yaw_4: axis 0.0 0.0 1.0 -> 0.0 0.0 -1.0; origin xyz=0.0 0.0 0.0 rpy=1.57079632679 0.0 1.57079632679 -> xyz=0.0 -0.139 0.00085 rpy=-1.57079632679 0.0 0.0
- joint contact_joint_1: origin xyz=0.0 0.0 0.315 rpy=3.14159265 0.0 0.0 -> xyz=0.0 0.0 -0.176 rpy=0.0 0.0 0.0
- joint contact_joint_2: origin xyz=0.0 0.0 0.315 rpy=3.14159265 0.0 0.0 -> xyz=0.0 0.0 -0.176 rpy=0.0 0.0 0.0
- joint contact_joint_3: origin xyz=0.0 0.0 0.315 rpy=3.14159265 0.0 0.0 -> xyz=0.0 0.0 -0.176 rpy=0.0 0.0 0.0
- joint contact_joint_4: origin xyz=0.0 0.0 0.315 rpy=3.14159265 0.0 0.0 -> xyz=0.0 0.0 -0.176 rpy=0.0 0.0 0.0
- joint hip_pitch_1: axis 0.0 0.0 1.0 -> 0.0 0.0 -1.0; origin xyz=0.0 0.0 0.0625 rpy=1.57079632679 0.0 0.46141612323 -> xyz=0.0 0.1146 -0.0625 rpy=1.57079632679 0.0 0.0
- joint hip_pitch_2: origin xyz=0.0 0.0 0.0625 rpy=1.57079632679 0.0 2.68017653036 -> xyz=0.0 -0.1146 -0.0625 rpy=1.57079632679 0.0 0.0
- joint hip_pitch_3: axis 0.0 0.0 1.0 -> 0.0 0.0 -1.0; origin xyz=0.0 0.0 0.0625 rpy=1.57079632679 0.0 2.68017653036 -> xyz=0.0 0.1146 -0.0625 rpy=1.57079632679 0.0 0.0
- joint hip_pitch_4: origin xyz=0.0 0.0 0.0625 rpy=1.57079632679 0.0 0.46141612323 -> xyz=0.0 -0.1146 -0.0625 rpy=1.57079632679 0.0 0.0
- joint hip_yaw_1: axis 0.0 0.0 1.0 -> 0.0 0.0 -1.0; origin xyz=0.25 0.125 -0.0566 rpy=3.14159265359 0.0 0.461416123228 -> xyz=0.25 0.125 -0.0566 rpy=0.0 0.0 0.0
- joint hip_yaw_2: axis 0.0 0.0 1.0 -> 0.0 0.0 -1.0; origin xyz=0.25 -0.125 -0.0566 rpy=3.14159265359 0.0 -0.461416123228 -> xyz=0.25 -0.125 -0.0566 rpy=0.0 0.0 0.0
- joint hip_yaw_3: axis 0.0 0.0 1.0 -> 0.0 0.0 -1.0; origin xyz=-0.25 0.125 -0.0566 rpy=3.14159265359 0.0 2.68017653036 -> xyz=-0.25 0.125 -0.0566 rpy=0.0 0.0 0.0
- joint hip_yaw_4: axis 0.0 0.0 1.0 -> 0.0 0.0 -1.0; origin xyz=-0.25 -0.125 -0.0566 rpy=3.14159265359 0.0 3.60300877682 -> xyz=-0.25 -0.125 -0.0566 rpy=0.0 0.0 0.0
- joint j_arm1_3: origin xyz=0.09015 0.0 -0.21815 -> xyz=0.09015 0.0 -0.21815 rpy=0 0 0
- joint j_arm1_4: origin xyz=0.045 0.05515 -0.074 -> xyz=0.045 0.05515 -0.074 rpy=0 0 0
- joint j_arm1_5: origin xyz=-0.015 -0.05515 -0.095 -> xyz=-0.015 -0.05515 -0.095 rpy=0 0 0
- joint j_arm1_6: origin xyz=0.0 0.049 -0.156 -> xyz=0.0 0.049 -0.156 rpy=0 0 0
- joint j_arm1_7: origin xyz=0.0 -0.049 -0.174 -> xyz=0.0 -0.049 -0.174 rpy=0 0 0
- joint j_arm2_3: origin xyz=0.09015 0.0 -0.21815 -> xyz=0.09015 0.0 -0.21815 rpy=0 0 0
- joint j_arm2_4: origin xyz=0.045 -0.05515 -0.074 -> xyz=0.045 -0.05515 -0.074 rpy=0 0 0
- joint j_arm2_5: origin xyz=-0.015 0.05515 -0.095 -> xyz=-0.015 0.05515 -0.095 rpy=0 0 0
- joint j_arm2_6: origin xyz=0.0 -0.049 -0.156 -> xyz=0.0 -0.049 -0.156 rpy=0 0 0
- joint j_arm2_7: origin xyz=0.0 0.049 -0.174 -> xyz=0.0 0.049 -0.174 rpy=0 0 0
- joint j_wheel_1: axis 0.0 0.0 1.0 -> 0.0 0.0 -1.0; limit effort=35.0 velocity=20.0 -> lower=0 upper=0 effort=35.0 velocity=20.0; origin xyz=0.0 0.00085 0.23735 rpy=1.57079632679 0.0 3.14159265359 -> xyz=0.0 -0.0 -0.09835 rpy=1.57079632679 0.0 0.0
- joint j_wheel_2: limit effort=35.0 velocity=20.0 -> lower=0 upper=0 effort=35.0 velocity=20.0; origin xyz=0.0 0.00085 0.23735 rpy=1.57079632679 0.0 3.14159265359 -> xyz=0.0 0.0 -0.09835 rpy=1.57079632679 0.0 0.0
- joint j_wheel_3: axis 0.0 0.0 1.0 -> 0.0 0.0 -1.0; limit effort=35.0 velocity=20.0 -> lower=0 upper=0 effort=35.0 velocity=20.0; origin xyz=0.0 0.00085 0.23735 rpy=1.57079632679 0.0 3.14159265359 -> xyz=0.0 -0.0 -0.09835 rpy=1.57079632679 0.0 0.0
- joint j_wheel_4: limit effort=35.0 velocity=20.0 -> lower=0 upper=0 effort=35.0 velocity=20.0; origin xyz=0.0 0.00085 0.23735 rpy=1.57079632679 0.0 3.14159265359 -> xyz=0.0 0.0 -0.09835 rpy=1.57079632679 0.0 0.0
- joint knee_pitch_1: axis 0.0 0.0 1.0 -> 0.0 0.0 -1.0; origin xyz=0.0 0.3 -0.0036 rpy=3.14159265359 0.0 1.57079632679 -> xyz=0.0 -0.3 0.1182 rpy=3.14159265359 0.0 0.0
- joint knee_pitch_2: origin xyz=0.0 0.3 -0.0036 rpy=3.14159265359 0.0 1.57079632679 -> xyz=0.0 -0.3 -0.1182 rpy=3.14159265359 0.0 0.0
- joint knee_pitch_3: axis 0.0 0.0 1.0 -> 0.0 0.0 -1.0; origin xyz=0.0 0.3 -0.0036 rpy=3.14159265359 0.0 1.57079632679 -> xyz=0.0 -0.3 0.1182 rpy=3.14159265359 0.0 0.0
- joint knee_pitch_4: origin xyz=0.0 0.3 -0.0036 rpy=3.14159265359 0.0 1.57079632679 -> xyz=0.0 -0.3 -0.1182 rpy=3.14159265359 0.0 0.0
- joint neck_pitch: origin xyz=0.054 0.0596 -0.0124975 -> xyz=0.054 0.0596 -0.0124975 rpy=0 0 0
- joint neck_velodyne: limit effort=35.0 velocity=5.7 -> lower=0 upper=0 effort=35.0 velocity=5.7
- joint neck_yaw: origin xyz=0.0 0.0 0.2795 -> xyz=0.0 0.0 0.2795 rpy=0 0 0
- joint torso_yaw: origin xyz=0.2 0.0 0.256 -> xyz=0.2 0.0 0.256 rpy=0 0 0

File: centauro_urdf/urdf/centauro_base.urdf.xacro (robot description, xacro)
@@ -25,5 +25,5 @@
          <origin xyz="0.0 0 0.0"  rpy="0.0 0.0 0.0"/>
         <geometry>
-         <mesh filename="package://centauro_urdf/meshes/simple/pelvis.stl" scale="0.001 0.001 0.001" />
+          <mesh filename="package://centauro_urdf/meshes/simple/pelvis.stl" scale="0.001 0.001 0.001" />
         </geometry>
       </collision>

Commit message: removed ball hand from capsules (for the rod plate case), setted zero mass of rod plate

File: centauro_urdf/urdf/capsule/centauro_capsules.urdf (robot description, URDF)
Before this commit: robot centauro, 58 links, 57 joints
Links:
- removed link arm1_8
- removed link arm2_8
- removed link ball1
- removed link ball1_tip
- removed link ball2
- removed link ball2_tip
Joints:
- removed joint j_arm1_8
- removed joint j_arm2_8
- removed joint j_ball1_fixed
- removed joint j_ball1_tip
- removed joint j_ball2_fixed
- removed joint j_ball2_tip

File: centauro_urdf/urdf/parts/rod_plate.urdf.xacro (robot description, xacro)
@@ -6,5 +6,6 @@
     <inertial>
       <origin xyz="${4.8407693e+01*mmTom} ${2.0035723e+01*mmTom} ${7.7533287e+01*mmTom}" rpy="0 0 0"/>
-      <mass value="3.45345"/>
+      <!--mass value="3.45345"/-->
+      <mass value="0.0"/>
       <inertia ixx="${2.3061092e+03*mm2Tom2}"  ixy="${2.9181758e-01*mm2Tom2}"  ixz="${-2.1246684e-01*mm2Tom2}" iyy="${2.3053155e+03*mm2Tom2}" iyz="${7.9290978e-01*mm2Tom2}" izz="${3.0675616e+03*mm2Tom2}" />
     </inertial>
@@ -24,4 +25,5 @@
 </link>
 <link name="rod_plate${arm_num}_tip"/>
+<!-- Parent link is arm*_7 -->
 <joint name="j_arm${arm_num}_8" type="fixed">
       <parent link="${parent_link}"/>
@@ -29,8 +31,9 @@
       <xacro:insert_block name="origin"/>
 </joint>
+<!-- <origin xyz="0 -0.174 -0.049" rpy="1.570796 0.0 0.0"/ -->
 <joint name="j_rod_plate${arm_num}_tip" type="fixed">
 	<parent link="rod_plate${arm_num}"/>
 	<child link="rod_plate${arm_num}_tip"/>
-	<origin xyz="0 -0.174 -0.049" rpy="0 0 0"/>
+	<origin xyz="0 0 -0.07" rpy="0 0 0"/>
 </joint>
 <!-- add armX_8 link for legacy reasons (same as ballX) -->
