Commit message: Add T265

File: centauro_urdf/urdf/_centauro_robot.urdf (robot description, URDF)
Before this commit: robot centauro, 70 links, 69 joints
Links:
- added link T265_camera_accel_frame
- added link T265_camera_accel_optical_frame
- added link T265_camera_fisheye1_optical_frame
- added link T265_camera_fisheye1_rgb_frame
- added link T265_camera_fisheye2_optical_frame
- added link T265_camera_fisheye2_rgb_frame
- added link T265_camera_gyro_frame
- added link T265_camera_gyro_optical_frame
- added link T265_camera_link
- added link T265_camera_pose_frame, mass 0.068024; collision mesh filename=package://realsense_gazebo_description/meshes/t265_simplifi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 scale=0.001 0.001 0.001; visual mesh filename=package://realsense_gazebo_description/meshes/t265_full.stl scale=0.001 0.001 0.001
Joints:
- added joint T265_camera_accel_joint: type fixed, parent T265_camera_link, child T265_camera_accel_frame, origin xyz=-0.0311 0 0.00655 rpy=0 3.14159265359 0
- added joint T265_camera_accel_optical_joint: type fixed, parent T265_camera_accel_frame, child T265_camera_accel_optical_frame, origin xyz=-0.0311 0 0.00655 rpy=0 3.14159265359 0
- added joint T265_camera_fisheye1_optical_joint: type fixed, parent T265_camera_fisheye1_rgb_frame, child T265_camera_fisheye1_optical_frame, origin xyz=0 0 0 rpy=-1.57079632679 0 -1.57079632679
- added joint T265_camera_fisheye1_rgb_joint: type fixed, parent T265_camera_link, child T265_camera_fisheye1_rgb_frame, origin xyz=-0.0411 0.0 0.0 rpy=0 1.57079632679 1.57079632679
- added joint T265_camera_fisheye2_optical_joint: type fixed, parent T265_camera_fisheye2_rgb_frame, child T265_camera_fisheye2_optical_frame, origin xyz=0 0 0 rpy=-1.57079632679 0 -1.57079632679
- added joint T265_camera_fisheye2_rgb_joint: type fixed, parent T265_camera_link, child T265_camera_fisheye2_rgb_frame, origin xyz=0.0229 0.0 0.0 rpy=0 1.57079632679 1.57079632679
- added joint T265_camera_gyro_joint: type fixed, parent T265_camera_link, child T265_camera_gyro_frame, origin xyz=-0.0311 0 0.00655 rpy=0 3.14159265359 0
- added joint T265_camera_gyro_optical_joint: type fixed, parent T265_camera_gyro_frame, child T265_camera_gyro_optical_frame, origin xyz=0 0 0 rpy=0 0 0
- added joint T265_camera_link_joint: type fixed, parent T265_camera_pose_frame, child T265_camera_link, origin xyz=0 0 0 rpy=1.57079632679 0 -1.57079632679
- added joint T265_camera_pose_joint: type fixed, parent torso_2, child T265_camera_pose_frame, origin xyz=0.125 0.0 0 rpy=0.0 0.25 0.0
- joint d435i_camera_joint: origin xyz=0.13 0 0.03 rpy=0 0.3 0 -> xyz=0.13 0 0.03 rpy=0 0.25 0

File: centauro_urdf/urdf/centauro.urdf (robot description, URDF)
Before this commit: robot centauro, 70 links, 69 joints
Links:
- added link T265_camera_accel_frame
- added link T265_camera_accel_optical_frame
- added link T265_camera_fisheye1_optical_frame
- added link T265_camera_fisheye1_rgb_frame
- added link T265_camera_fisheye2_optical_frame
- added link T265_camera_fisheye2_rgb_frame
- added link T265_camera_gyro_frame
- added link T265_camera_gyro_optical_frame
- added link T265_camera_link
- added link T265_camera_pose_frame, mass 0.068024; collision mesh filename=package://realsense_gazebo_description/meshes/t265_simplifi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 scale=0.001 0.001 0.001; visual mesh filename=package://realsense_gazebo_description/meshes/t265_full.stl scale=0.001 0.001 0.001
Joints:
- added joint T265_camera_accel_joint: type fixed, parent T265_camera_link, child T265_camera_accel_frame, origin xyz=-0.0311 0 0.00655 rpy=0 3.14159265359 0
- added joint T265_camera_accel_optical_joint: type fixed, parent T265_camera_accel_frame, child T265_camera_accel_optical_frame, origin xyz=-0.0311 0 0.00655 rpy=0 3.14159265359 0
- added joint T265_camera_fisheye1_optical_joint: type fixed, parent T265_camera_fisheye1_rgb_frame, child T265_camera_fisheye1_optical_frame, origin xyz=0 0 0 rpy=-1.57079632679 0 -1.57079632679
- added joint T265_camera_fisheye1_rgb_joint: type fixed, parent T265_camera_link, child T265_camera_fisheye1_rgb_frame, origin xyz=-0.0411 0.0 0.0 rpy=0 1.57079632679 1.57079632679
- added joint T265_camera_fisheye2_optical_joint: type fixed, parent T265_camera_fisheye2_rgb_frame, child T265_camera_fisheye2_optical_frame, origin xyz=0 0 0 rpy=-1.57079632679 0 -1.57079632679
- added joint T265_camera_fisheye2_rgb_joint: type fixed, parent T265_camera_link, child T265_camera_fisheye2_rgb_frame, origin xyz=0.0229 0.0 0.0 rpy=0 1.57079632679 1.57079632679
- added joint T265_camera_gyro_joint: type fixed, parent T265_camera_link, child T265_camera_gyro_frame, origin xyz=-0.0311 0 0.00655 rpy=0 3.14159265359 0
- added joint T265_camera_gyro_optical_joint: type fixed, parent T265_camera_gyro_frame, child T265_camera_gyro_optical_frame, origin xyz=0 0 0 rpy=0 0 0
- added joint T265_camera_link_joint: type fixed, parent T265_camera_pose_frame, child T265_camera_link, origin xyz=0 0 0 rpy=1.57079632679 0 -1.57079632679
- added joint T265_camera_pose_joint: type fixed, parent torso_2, child T265_camera_pose_frame, origin xyz=0.125 0.0 0 rpy=0.0 0.25 0.0
- joint d435i_camera_joint: origin xyz=0.13 0 0.03 rpy=0 0.3 0 -> xyz=0.13 0 0.03 rpy=0 0.25 0

File: centauro_urdf/urdf/centauro_base.urdf.xacro (robot description, xacro)
@@ -61,8 +61,16 @@
     <xacro:if value="${ADD_INTEL_D435I}">
         <xacro:include filename="$(find realsense_gazebo_description)/urdf/_d435i.urdf.xacro" />
-        <xacro:sensor_d435i parent="torso_2" name="d435i_camera" topics_ns="/d435i_camera"
+        <xacro:sensor_d435i parent="torso_2" name="d435i_camera" topics_ns="d435i_camera"
                             enable_pointCloud="true" align_depth="true">
-            <origin xyz="0.13 0 0.03" rpy="0 0.3 0"/>
+            <origin xyz="0.13 0 0.03" rpy="0 0.25 0"/>
         </xacro:sensor_d435i>
+    </xacro:if>
+    <xacro:if value="${ADD_INTEL_T265}">
+        <xacro:include filename="$(find realsense_gazebo_description)/urdf/_t265.urdf.xacro" />
+        <xacro:sensor_t265  parent="torso_2" name="T265_camera" topics_ns="T265_camera"
+                      xyz="0.125 0.0 0" rpy="0.0 0.25 0.0"
+                      unite_imu_method="false"> <!-- unite_imu_method can be false, copy or linear_interpolation -->
+            <origin xyz="0.125 0.0 0" rpy="0.0 0.25 0.0"/>
+        </xacro:sensor_t265>
     </xacro:if>
 </xacro:if>

File: centauro_urdf/urdf/centauro_config.urdf.xacro (robot description, xacro)
@@ -11,3 +11,4 @@
 <xacro:property name="ADD_VELODYNE" value="true" />
 <xacro:property name="ADD_INTEL_D435I" value="true" />
+<xacro:property name="ADD_INTEL_T265" value="true" />
 </robot>

Commit message: Adjust camera position

File: centauro_urdf/urdf/_centauro_robot.urdf (robot description, URDF)
Before this commit: robot centauro, 80 links, 79 joints
Joints:
- joint T265_camera_pose_joint: origin xyz=0.125 0.0 0 rpy=0.0 0.25 0.0 -> xyz=0.238 0 -0.035 rpy=0.0 0.349 0.0; parent torso_2 -> pelvis
- joint d435i_camera_joint: origin xyz=0.13 0 0.03 rpy=0 0.25 0 -> xyz=0.238 0 -0.035 rpy=0.0 0.349 0.0; parent torso_2 -> pelvis

File: centauro_urdf/urdf/centauro.urdf (robot description, URDF)
Before this commit: robot centauro, 80 links, 79 joints
Joints:
- joint T265_camera_pose_joint: origin xyz=0.125 0.0 0 rpy=0.0 0.25 0.0 -> xyz=0.238 0 -0.035 rpy=0.0 0.349 0.0; parent torso_2 -> pelvis
- joint d435i_camera_joint: origin xyz=0.13 0 0.03 rpy=0 0.25 0 -> xyz=0.238 0 -0.035 rpy=0.0 0.349 0.0; parent torso_2 -> pelvis

File: centauro_urdf/urdf/centauro_base.urdf.xacro (robot description, xacro)
@@ -61,15 +61,46 @@
     <xacro:if value="${ADD_INTEL_D435I}">
         <xacro:include filename="$(find realsense_gazebo_description)/urdf/_d435i.urdf.xacro" />
-        <xacro:sensor_d435i parent="torso_2" name="d435i_camera" topics_ns="d435i_camera"
+       <!-- <xacro:sensor_d435i parent="torso_2" name="d435i_camera" topics_ns="d435i_camera"
                             enable_pointCloud="true" align_depth="true">
             <origin xyz="0.13 0 0.03" rpy="0 0.25 0"/>
+        </xacro:sensor_d435i>-->
+        <xacro:sensor_d435i parent="pelvis" name="d435i_camera" topics_ns="d435i_camera"
+                      enable_pointCloud="true" align_depth="true"
+                      unite_imu_method="false">
+<!--
+                      accel_fps="250"
+                      gyro_fps="400"
+                      depth_width="1280"
+                      depth_height="720"
+                      depth_fps="30"
+                      infra_width="1280"
+                      infra_height="720"
+                      infra_fps="30"
+                      color_width="1280"
+                      color_height="720"
+                      color_fps="30"> -->
+            <origin xyz="0.238 0 -0.035" rpy="0.0 0.349 0.0"/>
         </xacro:sensor_d435i>
     </xacro:if>
     <xacro:if value="${ADD_INTEL_T265}">
         <xacro:include filename="$(find realsense_gazebo_description)/urdf/_t265.urdf.xacro" />
-        <xacro:sensor_t265  parent="torso_2" name="T265_camera" topics_ns="T265_camera"
+        <!-- unite_imu_method can be false, copy or linear_interpolation -->
+        <!--<xacro:sensor_t265  parent="torso_2" name="T265_camera" topics_ns="T265_camera"
                       xyz="0.125 0.0 0" rpy="0.0 0.25 0.0"
-                      unite_imu_method="false"> <!-- unite_imu_method can be false, copy or linear_interpolation -->
+                      unite_imu_method="false">
             <origin xyz="0.125 0.0 0" rpy="0.0 0.25 0.0"/>
+        </xacro:sensor_t265>-->
+        <xacro:sensor_t265  parent="pelvis" name="T265_camera" topics_ns="T265_camera" xyz="0.238 0 -0.035" rpy="0.0 0.349 0.0"  >
+                           <!--
+                      odom_xyz="0.0 0.0 0.25"
+                      odom_rpy="0.0 0.0 0.0"
+                      odom_fps="262"
+                      fisheye_width="848"
+                      fisheye_height="800"
+                      fisheye_fps="30"
+                      unite_imu_method="false"
+                      accel_fps="62.5"
+                      gyro_fps="200">-->
+            <origin xyz="0.238 0 -0.035" rpy="0.0 0.349 0.0" />
         </xacro:sensor_t265>
     </xacro:if>

Commit message: Changes related to parametrization of camera model

File: centauro_urdf/urdf/_centauro_robot.urdf (robot description, URDF)
Before this commit: robot centauro, 80 links, 79 joints
Joints:
- joint T265_camera_pose_joint: origin xyz=0.238 0 -0.035 rpy=0.0 0.349 0.0 -> xyz=0.24 0.01 -0.019 rpy=0.0 0.15 0.0
- joint d435i_camera_joint: origin xyz=0.238 0 -0.035 rpy=0.0 0.349 0.0 -> xyz=0.23 0 -0.061 rpy=0.0 0.28 0.0

File: centauro_urdf/urdf/centauro.urdf (robot description, URDF)
Before this commit: robot centauro, 80 links, 79 joints
Joints:
- joint T265_camera_pose_joint: origin xyz=0.238 0 -0.035 rpy=0.0 0.349 0.0 -> xyz=0.24 0.01 -0.019 rpy=0.0 0.15 0.0
- joint d435i_camera_joint: origin xyz=0.238 0 -0.035 rpy=0.0 0.349 0.0 -> xyz=0.23 0 -0.061 rpy=0.0 0.28 0.0

File: centauro_urdf/urdf/centauro_base.urdf.xacro (robot description, xacro)
@@ -66,19 +66,19 @@
         </xacro:sensor_d435i>-->
         <xacro:sensor_d435i parent="pelvis" name="d435i_camera" topics_ns="d435i_camera"
-                      enable_pointCloud="true" align_depth="true"
-                      unite_imu_method="false">
-<!--
-                      accel_fps="250"
-                      gyro_fps="400"
+                      enable_pointCloud="true" align_depth="false"
+                      unite_imu_method="false"
+                      visualize="true"
+                      accel_fps="300"
+                      gyro_fps="300"
                       depth_width="1280"
                       depth_height="720"
-                      depth_fps="30"
+                      depth_fps="90"
                       infra_width="1280"
                       infra_height="720"
-                      infra_fps="30"
+                      infra_fps="90"
                       color_width="1280"
                       color_height="720"
-                      color_fps="30"> -->
-            <origin xyz="0.238 0 -0.035" rpy="0.0 0.349 0.0"/>
+                      color_fps="30">
+            <origin xyz="0.23 0 -0.061" rpy="0.0 0.28 0.0"/>
         </xacro:sensor_d435i>
     </xacro:if>
@@ -91,6 +91,5 @@
             <origin xyz="0.125 0.0 0" rpy="0.0 0.25 0.0"/>
         </xacro:sensor_t265>-->
-        <xacro:sensor_t265  parent="pelvis" name="T265_camera" topics_ns="T265_camera" xyz="0.238 0 -0.035" rpy="0.0 0.349 0.0"  >
-                           <!--
+        <xacro:sensor_t265  parent="pelvis" name="T265_camera" topics_ns="T265_camera"
                       odom_xyz="0.0 0.0 0.25"
                       odom_rpy="0.0 0.0 0.0"
@@ -101,6 +100,6 @@
                       unite_imu_method="false"
                       accel_fps="62.5"
-                      gyro_fps="200">-->
-            <origin xyz="0.238 0 -0.035" rpy="0.0 0.349 0.0" />
+                      gyro_fps="200">
+            <origin xyz="0.24 0.01 -0.019" rpy="0.0 0.15 0.0" />
         </xacro:sensor_t265>
     </xacro:if>

Commit message: Update camera topic name

File: centauro_urdf/urdf/_centauro_robot.urdf (robot description, URDF)
Before this commit: robot centauro, 80 links, 79 joints
Links:
- removed link d435i_camera_accel_frame
- removed link d435i_camera_accel_optical_frame
- removed link d435i_camera_bottom_screw_frame
- removed link d435i_camera_color_frame
- removed link d435i_camera_color_optical_frame
- removed link d435i_camera_depth_frame
- removed link d435i_camera_depth_optical_frame
- removed link d435i_camera_gyro_frame
- removed link d435i_camera_gyro_optical_frame
- removed link d435i_camera_left_ir_frame
- removed link d435i_camera_left_ir_optical_frame
- removed link d435i_camera_link
- removed link d435i_camera_right_ir_frame
- removed link d435i_camera_right_ir_optical_frame
- added link D435i_camera_accel_frame
- added link D435i_camera_accel_optical_frame
- added link D435i_camera_bottom_screw_frame
- added link D435i_camera_color_frame
- added link D435i_camera_color_optical_frame
- added link D435i_camera_depth_frame
- added link D435i_camera_depth_optical_frame
- added link D435i_camera_gyro_frame
- added link D435i_camera_gyro_optical_frame
- added link D435i_camera_left_ir_frame
- added link D435i_camera_left_ir_optical_frame
- added link D435i_camera_link, mass 0.564; collision box size=0.02505 0.09 0.025; visual mesh filename=package://realsense2_description/meshes/d435.dae
- added link D435i_camera_right_ir_frame
- added link D435i_camera_right_ir_optical_frame
Joints:
- removed joint d435i_camera_accel_joint
- removed joint d435i_camera_accel_optical_joint
- removed joint d435i_camera_color_joint
- removed joint d435i_camera_color_optical_joint
- removed joint d435i_camera_depth_joint
- removed joint d435i_camera_depth_optical_joint
- removed joint d435i_camera_gyro_joint
- removed joint d435i_camera_gyro_optical_joint
- removed joint d435i_camera_joint
- removed joint d435i_camera_left_ir_joint
- removed joint d435i_camera_left_ir_optical_joint
- removed joint d435i_camera_link_joint
- removed joint d435i_camera_right_ir_joint
- removed joint d435i_camera_right_ir_optical_joint
- added joint D435i_camera_accel_joint: type fixed, parent D435i_camera_link, child D435i_camera_accel_frame, origin xyz=-0.00174 0.00552 0.0176 rpy=0 0 0
- added joint D435i_camera_accel_optical_joint: type fixed, parent D435i_camera_accel_frame, child D435i_camera_accel_optical_frame, origin xyz=0 0 0 rpy=-1.57079632679 0 -1.57079632679
- added joint D435i_camera_color_joint: type fixed, parent D435i_camera_depth_frame, child D435i_camera_color_frame, origin xyz=0 0.015 0 rpy=0 0 0
- added joint D435i_camera_color_optical_joint: type fixed, parent D435i_camera_color_frame, child D435i_camera_color_optical_frame, origin xyz=0 0 0 rpy=-1.57079632679 0 -1.57079632679
- added joint D435i_camera_depth_joint: type fixed, parent D435i_camera_link, child D435i_camera_depth_frame, origin xyz=0 0 0 rpy=0 0 0
- added joint D435i_camera_depth_optical_joint: type fixed, parent D435i_camera_depth_frame, child D435i_camera_depth_optical_frame, origin xyz=0 0 0 rpy=-1.57079632679 0 -1.57079632679
- added joint D435i_camera_gyro_joint: type fixed, parent D435i_camera_link, child D435i_camera_gyro_frame, origin xyz=-0.00174 0.00552 0.0176 rpy=0 0 0
- added joint D435i_camera_gyro_optical_joint: type fixed, parent D435i_camera_gyro_frame, child D435i_camera_gyro_optical_frame, origin xyz=0 0 0 rpy=-1.57079632679 0 -1.57079632679
- added joint D435i_camera_joint: type fixed, parent pelvis, child D435i_camera_bottom_screw_frame, origin xyz=0.23 0 -0.061 rpy=0.0 0.28 0.0
- added joint D435i_camera_left_ir_joint: type fixed, parent D435i_camera_depth_frame, child D435i_camera_left_ir_frame, origin xyz=0 0.0 0 rpy=0 0 0
- added joint D435i_camera_left_ir_optical_joint: type fixed, parent D435i_camera_left_ir_frame, child D435i_camera_left_ir_optical_frame, origin xyz=0 0 0 rpy=-1.57079632679 0 -1.57079632679
- added joint D435i_camera_link_joint: type fixed, parent D435i_camera_bottom_screw_frame, child D435i_camera_link, origin xyz=0 0.0175 0.0125 rpy=0 0 0
- added joint D435i_camera_right_ir_joint: type fixed, parent D435i_camera_depth_frame, child D435i_camera_right_ir_frame, origin xyz=0 -0.05 0 rpy=0 0 0
- added joint D435i_camera_right_ir_optical_joint: type fixed, parent D435i_camera_right_ir_frame, child D435i_camera_right_ir_optical_frame, origin xyz=0 0 0 rpy=-1.57079632679 0 -1.57079632679

File: centauro_urdf/urdf/centauro.urdf (robot description, URDF)
Before this commit: robot centauro, 80 links, 79 joints
Links:
- removed link d435i_camera_accel_frame
- removed link d435i_camera_accel_optical_frame
- removed link d435i_camera_bottom_screw_frame
- removed link d435i_camera_color_frame
- removed link d435i_camera_color_optical_frame
- removed link d435i_camera_depth_frame
- removed link d435i_camera_depth_optical_frame
- removed link d435i_camera_gyro_frame
- removed link d435i_camera_gyro_optical_frame
- removed link d435i_camera_left_ir_frame
- removed link d435i_camera_left_ir_optical_frame
- removed link d435i_camera_link
- removed link d435i_camera_right_ir_frame
- removed link d435i_camera_right_ir_optical_frame
- added link D435i_camera_accel_frame
- added link D435i_camera_accel_optical_frame
- added link D435i_camera_bottom_screw_frame
- added link D435i_camera_color_frame
- added link D435i_camera_color_optical_frame
- added link D435i_camera_depth_frame
- added link D435i_camera_depth_optical_frame
- added link D435i_camera_gyro_frame
- added link D435i_camera_gyro_optical_frame
- added link D435i_camera_left_ir_frame
- added link D435i_camera_left_ir_optical_frame
- added link D435i_camera_link, mass 0.564; collision box size=0.02505 0.09 0.025; visual mesh filename=package://realsense2_description/meshes/d435.dae
- added link D435i_camera_right_ir_frame
- added link D435i_camera_right_ir_optical_frame
Joints:
- removed joint d435i_camera_accel_joint
- removed joint d435i_camera_accel_optical_joint
- removed joint d435i_camera_color_joint
- removed joint d435i_camera_color_optical_joint
- removed joint d435i_camera_depth_joint
- removed joint d435i_camera_depth_optical_joint
- removed joint d435i_camera_gyro_joint
- removed joint d435i_camera_gyro_optical_joint
- removed joint d435i_camera_joint
- removed joint d435i_camera_left_ir_joint
- removed joint d435i_camera_left_ir_optical_joint
- removed joint d435i_camera_link_joint
- removed joint d435i_camera_right_ir_joint
- removed joint d435i_camera_right_ir_optical_joint
- added joint D435i_camera_accel_joint: type fixed, parent D435i_camera_link, child D435i_camera_accel_frame, origin xyz=-0.00174 0.00552 0.0176 rpy=0 0 0
- added joint D435i_camera_accel_optical_joint: type fixed, parent D435i_camera_accel_frame, child D435i_camera_accel_optical_frame, origin xyz=0 0 0 rpy=-1.57079632679 0 -1.57079632679
- added joint D435i_camera_color_joint: type fixed, parent D435i_camera_depth_frame, child D435i_camera_color_frame, origin xyz=0 0.015 0 rpy=0 0 0
- added joint D435i_camera_color_optical_joint: type fixed, parent D435i_camera_color_frame, child D435i_camera_color_optical_frame, origin xyz=0 0 0 rpy=-1.57079632679 0 -1.57079632679
- added joint D435i_camera_depth_joint: type fixed, parent D435i_camera_link, child D435i_camera_depth_frame, origin xyz=0 0 0 rpy=0 0 0
- added joint D435i_camera_depth_optical_joint: type fixed, parent D435i_camera_depth_frame, child D435i_camera_depth_optical_frame, origin xyz=0 0 0 rpy=-1.57079632679 0 -1.57079632679
- added joint D435i_camera_gyro_joint: type fixed, parent D435i_camera_link, child D435i_camera_gyro_frame, origin xyz=-0.00174 0.00552 0.0176 rpy=0 0 0
- added joint D435i_camera_gyro_optical_joint: type fixed, parent D435i_camera_gyro_frame, child D435i_camera_gyro_optical_frame, origin xyz=0 0 0 rpy=-1.57079632679 0 -1.57079632679
- added joint D435i_camera_joint: type fixed, parent pelvis, child D435i_camera_bottom_screw_frame, origin xyz=0.23 0 -0.061 rpy=0.0 0.28 0.0
- added joint D435i_camera_left_ir_joint: type fixed, parent D435i_camera_depth_frame, child D435i_camera_left_ir_frame, origin xyz=0 0.0 0 rpy=0 0 0
- added joint D435i_camera_left_ir_optical_joint: type fixed, parent D435i_camera_left_ir_frame, child D435i_camera_left_ir_optical_frame, origin xyz=0 0 0 rpy=-1.57079632679 0 -1.57079632679
- added joint D435i_camera_link_joint: type fixed, parent D435i_camera_bottom_screw_frame, child D435i_camera_link, origin xyz=0 0.0175 0.0125 rpy=0 0 0
- added joint D435i_camera_right_ir_joint: type fixed, parent D435i_camera_depth_frame, child D435i_camera_right_ir_frame, origin xyz=0 -0.05 0 rpy=0 0 0
- added joint D435i_camera_right_ir_optical_joint: type fixed, parent D435i_camera_right_ir_frame, child D435i_camera_right_ir_optical_frame, origin xyz=0 0 0 rpy=-1.57079632679 0 -1.57079632679

File: centauro_urdf/urdf/centauro_base.urdf.xacro (robot description, xacro)
@@ -65,5 +65,5 @@
             <origin xyz="0.13 0 0.03" rpy="0 0.25 0"/>
         </xacro:sensor_d435i>-->
-        <xacro:sensor_d435i parent="pelvis" name="d435i_camera" topics_ns="d435i_camera"
+        <xacro:sensor_d435i parent="pelvis" name="D435i_camera" topics_ns="D435i/D435i_camera"
                       enable_pointCloud="true" align_depth="false"
                       unite_imu_method="false"
@@ -91,5 +91,5 @@
             <origin xyz="0.125 0.0 0" rpy="0.0 0.25 0.0"/>
         </xacro:sensor_t265>-->
-        <xacro:sensor_t265  parent="pelvis" name="T265_camera" topics_ns="T265_camera"
+        <xacro:sensor_t265  parent="pelvis" name="T265_camera" topics_ns="T265/T265_camera"
                       odom_xyz="0.0 0.0 0.25"
                       odom_rpy="0.0 0.0 0.0"
