Commit message: Merge branch 'casannis-walking' into velodyne-realsense
# Conflicts:
#	centauro_config/configs/centauro_joint_map.yaml
#	centauro_gazebo/launch/centauro_world.launch
#	centauro_urdf/urdf/gazebo/centauro.gazebo.xacro

File: centauro_urdf/urdf/_centauro_robot.urdf (robot description, URDF)
Before this commit: robot centauro, 80 links, 79 joints
Links:
- added link contact_1
- added link contact_2
- added link contact_3
- added link contact_4
Joints:
- added joint contact_joint_1: type fixed, parent ankle2_1, child contact_1, origin xyz=0 0 0.315 rpy=3.14159265 0 0
- added joint contact_joint_2: type fixed, parent ankle2_2, child contact_2, origin xyz=0 0 0.315 rpy=3.14159265 0 0
- added joint contact_joint_3: type fixed, parent ankle2_3, child contact_3, origin xyz=0 0 0.315 rpy=3.14159265 0 0
- added joint contact_joint_4: type fixed, parent ankle2_4, child contact_4, origin xyz=0 0 0.315 rpy=3.14159265 0 0

File: centauro_urdf/urdf/centauro.urdf (robot description, URDF)
Before this commit: robot centauro, 80 links, 79 joints
Links:
- added link contact_1
- added link contact_2
- added link contact_3
- added link contact_4
Joints:
- added joint contact_joint_1: type fixed, parent ankle2_1, child contact_1, origin xyz=0 0 0.315 rpy=3.14159265 0 0
- added joint contact_joint_2: type fixed, parent ankle2_2, child contact_2, origin xyz=0 0 0.315 rpy=3.14159265 0 0
- added joint contact_joint_3: type fixed, parent ankle2_3, child contact_3, origin xyz=0 0 0.315 rpy=3.14159265 0 0
- added joint contact_joint_4: type fixed, parent ankle2_4, child contact_4, origin xyz=0 0 0.315 rpy=3.14159265 0 0

File: centauro_urdf/urdf/centauro_base.urdf.xacro (robot description, xacro)
@@ -42,5 +42,5 @@
 <xacro:if value="${ADD_UPPER_BODY}">
 	<xacro:include filename="$(find centauro_urdf)/urdf/parts/centauro_torso.urdf.xacro" />
-        <xacro:include filename="$(find centauro_urdf)/urdf/parts/arms.urdf.xacro" />
+    <xacro:include filename="$(find centauro_urdf)/urdf/parts/arms.urdf.xacro" />
 	<xacro:if value="${ADD_BALL_END_EFFECTOR}">
 		<xacro:include filename="$(find centauro_urdf)/urdf/parts/ball.urdf.xacro" />

File: centauro_urdf/urdf/centauro_config.urdf.xacro (robot description, xacro)
@@ -3,12 +3,18 @@
 <xacro:property name="model_name" value="centauro" />
 <xacro:property name="model_version" value="0.1" />
+<!-- command line arguments -->
+<xacro:arg name="add_legs" default="true"/>
+<xacro:arg name="add_upper_body" default="true"/>
+<xacro:arg name="add_velodyne" default="true"/>
+<xacro:arg name="add_realsense" default="true"/>
 <!-- ************SELECT PARTS*************-->
 <!-- *************************************-->
-<xacro:property name="ADD_LEGS" value="true" />
-<xacro:property name="ADD_UPPER_BODY" value="true" />
-<xacro:property name="ADD_BALL_END_EFFECTOR" value="true" />
-<xacro:property name="ADD_FLOATING_BASE" value="true" />
-<xacro:property name="ADD_VELODYNE" value="true" />
-<xacro:property name="ADD_INTEL_D435I" value="true" />
-<xacro:property name="ADD_INTEL_T265" value="true" />
+<xacro:property name="ADD_LEGS" value="$(arg add_legs)"/>
+<xacro:property name="ADD_UPPER_BODY" value="$(arg add_upper_body)"/>
+<xacro:property name="ADD_BALL_END_EFFECTOR" value="true"/>
+<xacro:property name="ADD_FLOATING_BASE" value="$(arg add_legs)"/>
+<xacro:property name="USE_STICKS" value="false"/>
+<xacro:property name="ADD_VELODYNE" value="$(arg add_velodyne)"/>
+<xacro:property name="ADD_INTEL_D435I" value="$(arg add_realsense)"/>
+<xacro:property name="ADD_INTEL_T265" value="$(arg add_realsense)"/>
 </robot>

File: centauro_urdf/urdf/centauro_robot.urdf.xacro (robot description, xacro)
@@ -12,4 +12,4 @@
   <xacro:include filename="$(find centauro_urdf)/urdf/gazebo/xbot.gazebo.xacro" />
   <xacro:include filename="$(find centauro_urdf)/urdf/gazebo/materials.gazebo.xacro" />
-<origin xyz="0.0 0.0 1.2" rpy="0 0 0" />
+  <origin xyz="0.0 0.0 1.2" rpy="0 0 0" />
 </robot>

File: centauro_urdf/urdf/config/centauro.urdf.xacro (robot description, xacro)
@@ -3,10 +3,14 @@
 <xacro:property name="model_name" value="centauro" />
 <xacro:property name="model_version" value="0.1" />
+<!-- command line arguments -->
+<xacro:arg name="add_legs" default="true"/>
+<xacro:arg name="add_upper_body" default="true"/>
 <!-- ************SELECT PARTS*************-->
 <!-- *************************************-->
-<xacro:property name="ADD_LEGS" value="true" />
-<xacro:property name="ADD_UPPER_BODY" value="true" />
+<xacro:property name="ADD_LEGS" value="$(arg add_legs)" />
+<xacro:property name="ADD_UPPER_BODY" value="$(arg add_upper_body)" />
 <xacro:property name="ADD_BALL_END_EFFECTOR" value="true" />
-<xacro:property name="ADD_FLOATING_BASE" value="true" />
+<xacro:property name="ADD_FLOATING_BASE" value="$(arg add_legs)" />
+<xacro:property name="USE_STICKS" value="false" />
 <xacro:property name="ADD_VELODYNE" value="true" />
 <xacro:property name="ADD_INTEL_D435I" value="true" />

File: centauro_urdf/urdf/gazebo/centauro.gazebo.xacro (robot description, xacro)
@@ -1,283 +1,303 @@
 <?xml version="1.0"?>
 <robot xmlns:xacro="http://ros.org/wiki/xacro">
-<xacro:if value="${ADD_LEGS}">
-<gazebo reference="wheel_1">
-    <material>Gazebo/Residential </material>
-    <collision>
-        <surface>
-            <friction>
-                <ode>
-                    <mu>0.5</mu>
-                    <mu2>0.5</mu2>
-                </ode>
-                <bullet>
-                    <friction>0.5</friction>
-                    <friction2>0.5</friction2>
-                </bullet>
-            </friction>
-            <contact>
-                <ode>
-                    <kp>2100000</kp>
-                    <kd>1</kd>
-                    <max_vel>100</max_vel>
-                </ode>
-                <bullet>
-                    <soft_cfm>0.007</soft_cfm>
-                    <soft_erp>0.25</soft_erp>
-                    <kp>1000000</kp>
-                    <kd>5</kd>
-                </bullet>
-            </contact>
-        </surface>
-    </collision>
-</gazebo>
-<gazebo reference="wheel_2">
-    <material>Gazebo/Residential</material>
-    <collision>
-        <surface>
-            <friction>
-                <ode>
-                    <mu>0.5</mu>
-                    <mu2>0.5</mu2>
-                </ode>
-                <bullet>
-                    <friction>0.5</friction>
-                    <friction2>0.5</friction2>
-                </bullet>
-            </friction>
-            <contact>
-                <ode>
-                    <kp>2100000</kp>
-                    <kd>1</kd>
-                    <max_vel>100</max_vel>
-                </ode>
-                <bullet>
-                    <soft_cfm>0.007</soft_cfm>
-                    <soft_erp>0.25</soft_erp>
-                    <kp>1000000</kp>
-                    <kd>5</kd>
-                </bullet>
-            </contact>
-        </surface>
-    </collision>
-</gazebo>
-<gazebo reference="wheel_3">
-    <material>Gazebo/Residential </material>
-    <collision>
-        <surface>
-            <friction>
-                <ode>
-                    <mu>0.5</mu>
-                    <mu2>0.5</mu2>
-                </ode>
-                <bullet>
-                    <friction>0.5</friction>
-                    <friction2>0.5</friction2>
-                </bullet>
-            </friction>
-            <contact>
-                <ode>
-                    <kp>2100000</kp>
-                    <kd>1</kd>
-                    <max_vel>100</max_vel>
-                </ode>
-                <bullet>
-                    <soft_cfm>0.007</soft_cfm>
-                    <soft_erp>0.25</soft_erp>
-                    <kp>1000000</kp>
-                    <kd>5</kd>
-                </bullet>
-            </contact>
-        </surface>
-    </collision>
-</gazebo>
-<gazebo reference="wheel_4">
-    <material>Gazebo/Residential</material>
-    <collision>
-        <surface>
-            <friction>
-                <ode>
-                    <mu>0.5</mu>
-                    <mu2>0.5</mu2>
-                </ode>
-                <bullet>
-                    <friction>0.5</friction>
-                    <friction2>0.5</friction2>
-                </bullet>
-            </friction>
-            <contact>
-                <ode>
-                    <kp>2100000</kp>
-                    <kd>1</kd>
-                    <max_vel>100</max_vel>
-                </ode>
-                <bullet>
-                    <soft_cfm>0.007</soft_cfm>
-                    <soft_erp>0.25</soft_erp>
-                    <kp>1000000</kp>
-                    <kd>5</kd>
-                </bullet>
-            </contact>
-        </surface>
-    </collision>
-</gazebo>
-<gazebo reference="hip_yaw_1">
-    <implicitSpringDamper>1</implicitSpringDamper>
-    <provideFeedback>true</provideFeedback>
-</gazebo>
-<gazebo reference="hip_pitch_1">
-    <implicitSpringDamper>1</implicitSpringDamper>
-    <provideFeedback>true</provideFeedback>
-</gazebo>
-<gazebo reference="knee_pitch_1">
-    <implicitSpringDamper>1</implicitSpringDamper>
-    <provideFeedback>true</provideFeedback>
-</gazebo>
-<gazebo reference="ankle_pitch_1">
-    <implicitSpringDamper>1</implicitSpringDamper>
-    <provideFeedback>true</provideFeedback>
-</gazebo>
-<gazebo reference="ankle_yaw_1">
-    <implicitSpringDamper>1</implicitSpringDamper>
-    <provideFeedback>true</provideFeedback>
-</gazebo>
-<gazebo reference="j_wheel_1">
-    <implicitSpringDamper>1</implicitSpringDamper>
-    <provideFeedback>true</provideFeedback>
-</gazebo>
-<gazebo reference="hip_yaw_2">
-    <implicitSpringDamper>1</implicitSpringDamper>
-    <provideFeedback>true</provideFeedback>
-</gazebo>
-<gazebo reference="hip_pitch_2">
-    <implicitSpringDamper>1</implicitSpringDamper>
-    <provideFeedback>true</provideFeedback>
-</gazebo>
-<gazebo reference="knee_pitch_2">
-    <implicitSpringDamper>1</implicitSpringDamper>
-    <provideFeedback>true</provideFeedback>
-</gazebo>
-<gazebo reference="ankle_pitch_2">
-    <implicitSpringDamper>1</implicitSpringDamper>
-    <provideFeedback>true</provideFeedback>
-</gazebo>
-<gazebo reference="ankle_yaw_2">
-    <implicitSpringDamper>1</implicitSpringDamper>
-    <provideFeedback>true</provideFeedback>
-</gazebo>
-<gazebo reference="j_wheel_2">
-    <implicitSpringDamper>1</implicitSpringDamper>
-    <provideFeedback>true</provideFeedback>
-</gazebo>
-<gazebo reference="hip_yaw_3">
-    <implicitSpringDamper>1</implicitSpringDamper>
-    <provideFeedback>true</provideFeedback>
-</gazebo>
-<gazebo reference="hip_pitch_3">
-    <implicitSpringDamper>1</implicitSpringDamper>
-    <provideFeedback>true</provideFeedback>
-</gazebo>
-<gazebo reference="knee_pitch_3">
-    <implicitSpringDamper>1</implicitSpringDamper>
-    <provideFeedback>true</provideFeedback>
-</gazebo>
-<gazebo reference="ankle_pitch_3">
-    <implicitSpringDamper>1</implicitSpringDamper>
-    <provideFeedback>true</provideFeedback>
-</gazebo>
-<gazebo reference="ankle_yaw_3">
-    <implicitSpringDamper>1</implicitSpringDamper>
-    <provideFeedback>true</provideFeedback>
-</gazebo>
-<gazebo reference="j_wheel_3">
-    <implicitSpringDamper>1</implicitSpringDamper>
-    <provideFeedback>true</provideFeedback>
-</gazebo>
-<gazebo reference="hip_yaw_4">
-    <implicitSpringDamper>1</implicitSpringDamper>
-    <provideFeedback>true</provideFeedback>
-</gazebo>
-<gazebo reference="hip_pitch_4">
-    <implicitSpringDamper>1</implicitSpringDamper>
-    <provideFeedback>true</provideFeedback>
-</gazebo>
-<gazebo reference="knee_pitch_4">
-    <implicitSpringDamper>1</implicitSpringDamper>
-    <provideFeedback>true</provideFeedback>
-</gazebo>
-<gazebo reference="ankle_pitch_4">
-    <implicitSpringDamper>1</implicitSpringDamper>
-    <provideFeedback>true</provideFeedback>
-</gazebo>
-<gazebo reference="ankle_yaw_4">
-    <implicitSpringDamper>1</implicitSpringDamper>
-    <provideFeedback>true</provideFeedback>
-</gazebo>
-<gazebo reference="j_wheel_4">
-    <implicitSpringDamper>1</implicitSpringDamper>
-    <provideFeedback>true</provideFeedback>
-</gazebo>
-</xacro:if>
-<xacro:if value="${ADD_UPPER_BODY}">
-<gazebo reference="torso_yaw">
-    <implicitSpringDamper>1</implicitSpringDamper>
-    <provideFeedback>true</provideFeedback>
-</gazebo>
-<gazebo reference="j_arm1_1">
-    <implicitSpringDamper>1</implicitSpringDamper>
-    <provideFeedback>true</provideFeedback>
-</gazebo>
-<gazebo reference="j_arm1_2">
-    <implicitSpringDamper>1</implicitSpringDamper>
-    <provideFeedback>true</provideFeedback>
-</gazebo>
-<gazebo reference="j_arm1_3">
-    <implicitSpringDamper>1</implicitSpringDamper>
-    <provideFeedback>true</provideFeedback>
-</gazebo>
-<gazebo reference="j_arm1_4">
-    <implicitSpringDamper>1</implicitSpringDamper>
-    <provideFeedback>true</provideFeedback>
-</gazebo>
-<gazebo reference="j_arm1_5">
-    <implicitSpringDamper>1</implicitSpringDamper>
-    <provideFeedback>true</provideFeedback>
-</gazebo>
-<gazebo reference="j_arm1_6">
-    <implicitSpringDamper>1</implicitSpringDamper>
-    <provideFeedback>true</provideFeedback>
-</gazebo>
-<gazebo reference="j_arm1_7">
-    <implicitSpringDamper>1</implicitSpringDamper>
-    <provideFeedback>true</provideFeedback>
-</gazebo>
-<gazebo reference="j_arm2_1">
-    <implicitSpringDamper>1</implicitSpringDamper>
-    <provideFeedback>true</provideFeedback>
-</gazebo>
-<gazebo reference="j_arm2_2">
-    <implicitSpringDamper>1</implicitSpringDamper>
-    <provideFeedback>true</provideFeedback>
-</gazebo>
-<gazebo reference="j_arm2_3">
-    <implicitSpringDamper>1</implicitSpringDamper>
-    <provideFeedback>true</provideFeedback>
-</gazebo>
-<gazebo reference="j_arm2_4">
-    <implicitSpringDamper>1</implicitSpringDamper>
-    <provideFeedback>true</provideFeedback>
-</gazebo>
-<gazebo reference="j_arm2_5">
-    <implicitSpringDamper>1</implicitSpringDamper>
-    <provideFeedback>true</provideFeedback>
-</gazebo>
-<gazebo reference="j_arm2_6">
-    <implicitSpringDamper>1</implicitSpringDamper>
-    <provideFeedback>true</provideFeedback>
-</gazebo>
-<gazebo reference="j_arm2_7">
-    <implicitSpringDamper>1</implicitSpringDamper>
-    <provideFeedback>true</provideFeedback>
-</gazebo>
-</xacro:if>
+    <xacro:if value="${ADD_LEGS}">
+        <gazebo reference="wheel_1">
+            <material>Gazebo/Residential </material>
+            <collision>
+                <surface>
+                    <friction>
+                        <!-- <torsional>
+                            <coefficient> 1.0 </coefficient>
+                            <use_patch_radius>true</use_patch_radius>
+                            <patch_radius>0.2</patch_radius>
+                        </torsional> -->
+                        <ode>
+                            <mu>1.0</mu>
+                            <mu2>1.0</mu2>
+                        </ode>
+                        <bullet>
+                            <friction>1.0</friction>
+                            <friction2>1.0</friction2>
+                        </bullet>
+                    </friction>
+                    <contact>
+                        <ode>
+                            <kp>2100000</kp>
+                            <kd>1</kd>
+                            <max_vel>100</max_vel>
+                        </ode>
+                        <bullet>
+                            <soft_cfm>0.007</soft_cfm>
+                            <soft_erp>0.25</soft_erp>
+                            <kp>1000000</kp>
+                            <kd>5</kd>
+                        </bullet>
+                    </contact>
+                </surface>
+            </collision>
+        </gazebo>
+        <gazebo reference="wheel_2">
+            <material>Gazebo/Residential</material>
+            <collision>
+                <surface>
+                    <friction>
+                        <!-- <torsional>
+                            <coefficient> 1.0 </coefficient>
+                            <use_patch_radius>true</use_patch_radius>
+                            <patch_radius>0.2</patch_radius>
+                        </torsional> -->
+                        <ode>
+                            <mu>1.0</mu>
+                            <mu2>1.0</mu2>
+                        </ode>
+                        <bullet>
+                            <friction>1.0</friction>
+                            <friction2>1.0</friction2>
+                        </bullet>
+                    </friction>
+                    <contact>
+                        <ode>
+                            <kp>2100000</kp>
+                            <kd>1</kd>
+                            <max_vel>100</max_vel>
+                        </ode>
+                        <bullet>
+                            <soft_cfm>0.007</soft_cfm>
+                            <soft_erp>0.25</soft_erp>
+                            <kp>1000000</kp>
+                            <kd>5</kd>
+                        </bullet>
+                    </contact>
+                </surface>
+            </collision>
+        </gazebo>
+        <gazebo reference="wheel_3">
+            <material>Gazebo/Residential </material>
+            <collision>
+                <surface>
+                    <friction>
+                        <!-- <torsional>
+                            <coefficient> 1.0 </coefficient>
+                            <use_patch_radius>true</use_patch_radius>
+                            <patch_radius>0.2</patch_radius>
+                        </torsional> -->
+                        <ode>
+                            <mu>1.0</mu>
+                            <mu2>1.0</mu2>
+                        </ode>
+                        <bullet>
+                            <friction>1.0</friction>
+                            <friction2>1.0</friction2>
+                        </bullet>
+                    </friction>
+                    <contact>
+                        <ode>
+                            <kp>2100000</kp>
+                            <kd>1</kd>
+                            <max_vel>100</max_vel>
+                        </ode>
+                        <bullet>
+                            <soft_cfm>0.007</soft_cfm>
+                            <soft_erp>0.25</soft_erp>
+                            <kp>1000000</kp>
+                            <kd>5</kd>
+                        </bullet>
+                    </contact>
+                </surface>
+            </collision>
+        </gazebo>
+        <gazebo reference="wheel_4">
+            <material>Gazebo/Residential</material>
+            <collision>
+                <surface>
+                    <friction>
+                        <!-- <torsional>
+                            <coefficient> 1.0 </coefficient>
+                            <use_patch_radius>true</use_patch_radius>
+                            <patch_radius>0.2</patch_radius>
+                        </torsional> -->
+                        <ode>
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
File: centauro_urdf/urdf/gazebo/xbot.gazebo.xacro (robot description, xacro)
@@ -2,5 +2,63 @@
 <robot xmlns:xacro="http://ros.org/wiki/xacro">
 <gazebo>
-    <plugin name="xbot_plugin_handler" filename="libGazeboXBotPlugin.so"/>
+    <plugin name="xbot2_link_state_sensor" filename="libxbot2_gz_link_state_sensor.so">
+        <links>
+            <link name="pelvis"/>
+            <link name="wheel_1"/>
+        </links>
+    </plugin>
+    <plugin name="xbot2_ft_driver" filename="libxbot2_gz_ft_server.so"/>
+    <plugin name="xbot2_imu_driver" filename="libxbot2_gz_imu_server.so"/>
+    <plugin name="xbot2_joint_driver" filename="libxbot2_gz_joint_server.so">
+        <pid>
+            <gain name="lowpwr_mot" p="50"  d="5"/>
+            <gain name="small_mot"  p="1000"  d="10"/>
+            <gain name="medium_mot" p="4000" d="40"/>
+            <gain name="big_mot"    p="8000" d="50"/>
+            <gain name="wheel_mot"  p="0" d="10"/>
+            <pid name="neck_yaw" profile="lowpwr_mot"/>
+            <pid name="neck_pitch" profile="lowpwr_mot"/>
+            <pid name="neck_velodyne" p="0"  d="20"/>
+            <pid name="j_arm1_1" profile="medium_mot"/>
+            <pid name="j_arm1_2" profile="medium_mot"/>
+            <pid name="j_arm1_3" profile="medium_mot"/>
+            <pid name="j_arm1_4" profile="medium_mot"/>
+            <pid name="j_arm1_5" profile="small_mot"/>
+            <pid name="j_arm1_6" profile="small_mot"/>
+            <pid name="j_arm1_7" profile="small_mot"/>
+            <pid name="j_arm2_1" profile="medium_mot"/>
+            <pid name="j_arm2_2" profile="medium_mot"/>
+            <pid name="j_arm2_3" profile="medium_mot"/>
+            <pid name="j_arm2_4" profile="medium_mot"/>
+            <pid name="j_arm2_5" profile="small_mot"/>
+            <pid name="j_arm2_6" profile="small_mot"/>
+            <pid name="j_arm2_7" profile="small_mot"/>
+            <pid name="torso_yaw" profile="big_mot"/>
+            <pid name="hip_yaw_1"     profile="big_mot"/>
+            <pid name="hip_pitch_1"   profile="big_mot"/>
+            <pid name="knee_pitch_1"  profile="big_mot"/>
+            <pid name="ankle_pitch_1" profile="medium_mot"/>
+            <pid name="ankle_yaw_1"   profile="medium_mot"/>
+            <pid name="j_wheel_1"     profile="wheel_mot"/>
+            <pid name="hip_yaw_2"     profile="big_mot"/>
+            <pid name="hip_pitch_2"   profile="big_mot"/>
+            <pid name="knee_pitch_2"  profile="big_mot"/>
+            <pid name="ankle_pitch_2" profile="medium_mot"/>
+            <pid name="ankle_yaw_2"   profile="medium_mot"/>
+            <pid name="j_wheel_2"     profile="wheel_mot"/>
+            <pid name="hip_yaw_3"     profile="big_mot"/>
+            <pid name="hip_pitch_3"   profile="big_mot"/>
+            <pid name="knee_pitch_3"  profile="big_mot"/>
+            <pid name="ankle_pitch_3" profile="medium_mot"/>
+            <pid name="ankle_yaw_3"   profile="medium_mot"/>
+            <pid name="j_wheel_3"     profile="wheel_mot"/>
+            <pid name="hip_yaw_4"     profile="big_mot"/>
+            <pid name="hip_pitch_4"   profile="big_mot"/>
+            <pid name="knee_pitch_4"  profile="big_mot"/>
+            <pid name="ankle_pitch_4" profile="medium_mot"/>
+            <pid name="ankle_yaw_4"   profile="medium_mot"/>
+            <pid name="j_wheel_4"     profile="wheel_mot"/>
+        </pid>
+    </plugin>
 </gazebo>
 </robot>
