Commit message: Merge branch 'casannis-walking' into velodyne-realsense
# Conflicts:
#	centauro_config/configs/centauro_joint_map.yaml
#	centauro_gazebo/launch/centauro_world.launch
#	centauro_urdf/urdf/gazebo/centauro.gazebo.xacro

File: centauro_urdf/urdf/parts/centauro_leg.urdf.xacro (robot description, xacro)
@@ -44,4 +44,29 @@
       </collision>
 </link>
+<xacro:if value="${USE_STICKS}">
+<link name="knee_${leg_num}">
+<inertial>
+	<mass value="${1.1927236}"/>
+    <origin xyz="${1.9572282e+02*mmTom} ${-1.4549221e+01*mmTom} ${-2.0785942e+01*mmTom}" rpy="0.0 0.0 0.0"/>
+	<!--origin xyz="${1.4549221e+01*mmTom} ${-2.0785942e+01*mmTom} ${-1.9572282e+02*mmTom}" rpy="0.0 0.0 0.0"/-->
+	<!--inertia ixx="${3.5313402e+04*mm2Tom2}"  ixy="${0.0*mm2Tom2}"  ixz="${1.1029574e-01*mm2Tom2}" iyy="${3.5530025e+04*mm2Tom2}" iyz="${-6.0307457e+02*mm2Tom2}" izz="${1.3302597e+03*mm2Tom2}" /-->
+    <inertia ixx="${1.3302597e+03*mm2Tom2}"  ixy="${6.0307457e+02*mm2Tom2}"  ixz="${0.0*mm2Tom2}" iyy="${3.5313402e+04*mm2Tom2}" iyz="${-1.1029574e-01*mm2Tom2}" izz="${3.5530025e+04*mm2Tom2}" />
+</inertial>
+<visual>
+      <origin xyz="0 0 0" rpy="${PI_2} 0 ${-PI_2}"/>
+      <material name="black"/>
+      <geometry name="${leg_num}_stick_visual">
+        <mesh filename="package://centauro_urdf/meshes/front_right_stick.stl" scale="${mmTom} ${mmTom} ${mmTom}"/>
+      </geometry>
+</visual>
+<collision>
+      <origin xyz="0 0 0" rpy="${PI_2} 0 ${-PI_2}"/>
+      <geometry name="${leg_num}_stick_collision">
+        <mesh filename="package://centauro_urdf/meshes/simple/front_right_stick.stl" scale="${mmTom} ${mmTom} ${mmTom}"/>
+      </geometry>
+</collision>
+</link>
+</xacro:if>
+<xacro:unless value="${USE_STICKS}">
 <link name="knee_${leg_num}">
 	<inertial>
@@ -131,4 +156,15 @@
 	</collision>
 </link>
+</xacro:unless>
+<!-- *****************************-->
+<link name="contact_${leg_num}">
+</link>
+<joint name="contact_joint_${leg_num}" type="fixed">
+	<parent link="ankle2_${leg_num}"/>
+	<child link="contact_${leg_num}"/>
+	<origin xyz="0 0 0.315" rpy="3.14159265 0 0"/>
+	<!--axis xyz="0 0 1" /-->
+</joint>
+<!-- ******************************** -->
 <joint name="hip_yaw_${leg_num}" type="revolute">
 	<parent link="pelvis"/>
@@ -145,4 +181,5 @@
         <limit lower="${hip_pitch_lower[leg_num-1]}" upper="${hip_pitch_upper[leg_num-1]}" effort="${motor_A_effort}" velocity="${motor_A_velocity}"/> <!-- 200 Nm, 1 rad/s-->
 </joint>
+<xacro:if  value="${USE_STICKS}">
 <joint name="knee_pitch_${leg_num}" type="revolute">
 	<parent link="hip2_${leg_num}"/>
@@ -152,4 +189,13 @@
         <limit lower="${knee_pitch_lower[leg_num-1]}" upper="${knee_pitch_upper[leg_num-1]}" effort="${motor_A_effort}" velocity="${motor_A_velocity}"/> <!-- 200 Nm, 1 rad/s-->
 </joint>
+</xacro:if>
+<xacro:unless value="${USE_STICKS}">
+<joint name="knee_pitch_${leg_num}" type="revolute">
+	<parent link="hip2_${leg_num}"/>
+	<child link="knee_${leg_num}"/>
+	<origin xyz="${Leg_3_Ox} ${Leg_3_Oy} ${Leg_3_Oz}" rpy="${Leg_3_roll} ${Leg_3_pitch} ${Leg_3_yaw}"/>
+	<axis xyz="0 0 1"/>
+        <limit lower="${knee_pitch_lower[leg_num-1]}" upper="${knee_pitch_upper[leg_num-1]}" effort="${motor_A_effort}" velocity="${motor_A_velocity}"/> <!-- 200 Nm, 1 rad/s-->
+</joint>
 <joint name="ankle_pitch_${leg_num}" type="revolute">
 	<parent link="knee_${leg_num}"/>
@@ -173,4 +219,5 @@
         <limit  effort="${motor_C_effort}" velocity="${motor_C_velocity}"/>  <!-- 23 Nm, 1 rad/s-->
 </joint>
+</xacro:unless>
 </xacro:macro>
 <!-- /macro legs -->

Commit message: Changes for xbot2

File: centauro_urdf/urdf/_centauro_robot.urdf (robot description, URDF)
Before this commit: robot centauro, 80 links, 79 joints
Links:
- removed link D435i_camera_accel_frame
- removed link D435i_camera_accel_optical_frame
- removed link D435i_camera_bottom_screw_frame
- removed link D435i_camera_color_frame
- removed link D435i_camera_color_optical_frame
- removed link D435i_camera_depth_frame
- removed link D435i_camera_depth_optical_frame
- removed link D435i_camera_gyro_frame
- removed link D435i_camera_gyro_optical_frame
- removed link D435i_camera_left_ir_frame
- removed link D435i_camera_left_ir_optical_frame
- removed link D435i_camera_link
- removed link D435i_camera_right_ir_frame
- removed link D435i_camera_right_ir_optical_frame
- added link contact_1
- added link contact_2
- added link contact_3
- added link contact_4
Joints:
- removed joint D435i_camera_accel_joint
- removed joint D435i_camera_accel_optical_joint
- removed joint D435i_camera_color_joint
- removed joint D435i_camera_color_optical_joint
- removed joint D435i_camera_depth_joint
- removed joint D435i_camera_depth_optical_joint
- removed joint D435i_camera_gyro_joint
- removed joint D435i_camera_gyro_optical_joint
- removed joint D435i_camera_joint
- removed joint D435i_camera_left_ir_joint
- removed joint D435i_camera_left_ir_optical_joint
- removed joint D435i_camera_link_joint
- removed joint D435i_camera_right_ir_joint
- removed joint D435i_camera_right_ir_optical_joint
- added joint contact_joint_1: type fixed, parent ankle2_1, child contact_1, origin xyz=0 0 0.315 rpy=3.14159265 0 0
- added joint contact_joint_2: type fixed, parent ankle2_2, child contact_2, origin xyz=0 0 0.315 rpy=3.14159265 0 0
- added joint contact_joint_3: type fixed, parent ankle2_3, child contact_3, origin xyz=0 0 0.315 rpy=3.14159265 0 0
- added joint contact_joint_4: type fixed, parent ankle2_4, child contact_4, origin xyz=0 0 0.315 rpy=3.14159265 0 0

File: centauro_urdf/urdf/centauro.urdf (robot description, URDF)
Before this commit: robot centauro, 80 links, 79 joints
Links:
- removed link D435i_camera_accel_frame
- removed link D435i_camera_accel_optical_frame
- removed link D435i_camera_bottom_screw_frame
- removed link D435i_camera_color_frame
- removed link D435i_camera_color_optical_frame
- removed link D435i_camera_depth_frame
- removed link D435i_camera_depth_optical_frame
- removed link D435i_camera_gyro_frame
- removed link D435i_camera_gyro_optical_frame
- removed link D435i_camera_left_ir_frame
- removed link D435i_camera_left_ir_optical_frame
- removed link D435i_camera_link
- removed link D435i_camera_right_ir_frame
- removed link D435i_camera_right_ir_optical_frame
- added link contact_1
- added link contact_2
- added link contact_3
- added link contact_4
Joints:
- removed joint D435i_camera_accel_joint
- removed joint D435i_camera_accel_optical_joint
- removed joint D435i_camera_color_joint
- removed joint D435i_camera_color_optical_joint
- removed joint D435i_camera_depth_joint
- removed joint D435i_camera_depth_optical_joint
- removed joint D435i_camera_gyro_joint
- removed joint D435i_camera_gyro_optical_joint
- removed joint D435i_camera_joint
- removed joint D435i_camera_left_ir_joint
- removed joint D435i_camera_left_ir_optical_joint
- removed joint D435i_camera_link_joint
- removed joint D435i_camera_right_ir_joint
- removed joint D435i_camera_right_ir_optical_joint
- added joint contact_joint_1: type fixed, parent ankle2_1, child contact_1, origin xyz=0 0 0.315 rpy=3.14159265 0 0
- added joint contact_joint_2: type fixed, parent ankle2_2, child contact_2, origin xyz=0 0 0.315 rpy=3.14159265 0 0
- added joint contact_joint_3: type fixed, parent ankle2_3, child contact_3, origin xyz=0 0 0.315 rpy=3.14159265 0 0
- added joint contact_joint_4: type fixed, parent ankle2_4, child contact_4, origin xyz=0 0 0.315 rpy=3.14159265 0 0

File: centauro_urdf/urdf/centauro.urdf.xacro (robot description, xacro)
@@ -8,16 +8,16 @@
 <!--xacro:include filename="$(find pholus_urdf)/urdf/control_frames.urdf.xacro"/-->
 <xacro:if value="${ADD_FLOATING_BASE}">
-<link name="world"/>
+  <link name="world"/>
   <joint name="reference" type="floating">
     <parent link="world"/>
     <child link="pelvis"/>
-</joint>
+  </joint>
 </xacro:if>
 <xacro:unless value="${ADD_FLOATING_BASE}">
-<link name="world"/>
+  <link name="world"/>
   <joint name="reference" type="fixed">
     <parent link="world"/>
     <child link="pelvis"/>
-</joint>
+  </joint>
 </xacro:unless>
 </robot>

File: centauro_urdf/urdf/centauro_base.urdf.xacro (robot description, xacro)
@@ -68,5 +68,5 @@
                       enable_pointCloud="true" align_depth="true"
                       unite_imu_method="false"
-                      visualize="true"
+                      visualize="false"
                       accel_fps="300"
                       gyro_fps="300"

File: centauro_urdf/urdf/centauro_config.urdf.xacro (robot description, xacro)
@@ -9,6 +9,7 @@
 <xacro:property name="ADD_BALL_END_EFFECTOR" value="true" />
 <xacro:property name="ADD_FLOATING_BASE" value="true" />
+<xacro:property name="USE_STICKS" value="false" />
 <xacro:property name="ADD_VELODYNE" value="true" />
-<xacro:property name="ADD_INTEL_D435I" value="true" />
+<xacro:property name="ADD_INTEL_D435I" value="false" />
 <xacro:property name="ADD_INTEL_T265" value="true" />
 </robot>

File: centauro_urdf/urdf/gazebo/xbot.gazebo.xacro (robot description, xacro)
@@ -2,5 +2,63 @@
 <robot xmlns:xacro="http://ros.org/wiki/xacro">
 <gazebo>
-    <plugin name="xbot_plugin_handler" filename="libGazeboXBotPlugin.so"/>
+    <plugin name="xbot2_link_state_sensor" filename="libxbot2_gz_link_state_sensor.so">
+        <links>
+            <link name="pelvis"/>
+            <link name="wheel_1"/>
+        </links>
+    </plugin>
+    <plugin name="xbot2_ft_driver" filename="libxbot2_gz_ft_server.so"/>
+    <plugin name="xbot2_imu_driver" filename="libxbot2_gz_imu_server.so"/>
+    <plugin name="xbot2_joint_driver" filename="libxbot2_gz_joint_server.so">
+        <pid>
+            <gain name="lowpwr_mot" p="50"  d="5"/>
+            <gain name="small_mot"  p="250"  d="5"/>
+            <gain name="medium_mot" p="1000" d="10"/>
+            <gain name="big_mot"    p="3000" d="10"/>
+            <gain name="wheel_mot"  p="0" d="10"/>
+            <pid name="neck_yaw" profile="lowpwr_mot"/>
+            <pid name="neck_pitch" profile="lowpwr_mot"/>
+            <pid name="neck_velodyne" p="0"  d="20"/>
+            <pid name="j_arm1_1" profile="medium_mot"/>
+            <pid name="j_arm1_2" profile="medium_mot"/>
+            <pid name="j_arm1_3" profile="medium_mot"/>
+            <pid name="j_arm1_4" profile="medium_mot"/>
+            <pid name="j_arm1_5" profile="small_mot"/>
+            <pid name="j_arm1_6" profile="small_mot"/>
+            <pid name="j_arm1_7" profile="small_mot"/>
+            <pid name="j_arm2_1" profile="medium_mot"/>
+            <pid name="j_arm2_2" profile="medium_mot"/>
+            <pid name="j_arm2_3" profile="medium_mot"/>
+            <pid name="j_arm2_4" profile="medium_mot"/>
+            <pid name="j_arm2_5" profile="small_mot"/>
+            <pid name="j_arm2_6" profile="small_mot"/>
+            <pid name="j_arm2_7" profile="small_mot"/>
+            <pid name="torso_yaw" profile="big_mot"/>
+            <pid name="hip_yaw_1"     profile="big_mot"/>
+            <pid name="hip_pitch_1"   profile="big_mot"/>
+            <pid name="knee_pitch_1"  profile="big_mot"/>
+            <pid name="ankle_pitch_1" profile="medium_mot"/>
+            <pid name="ankle_yaw_1"   profile="small_mot"/>
+            <pid name="j_wheel_1"     profile="wheel_mot"/>
+            <pid name="hip_yaw_2"     profile="big_mot"/>
+            <pid name="hip_pitch_2"   profile="big_mot"/>
+            <pid name="knee_pitch_2"  profile="big_mot"/>
+            <pid name="ankle_pitch_2" profile="medium_mot"/>
+            <pid name="ankle_yaw_2"   profile="small_mot"/>
+            <pid name="j_wheel_2"     profile="wheel_mot"/>
+            <pid name="hip_yaw_3"     profile="big_mot"/>
+            <pid name="hip_pitch_3"   profile="big_mot"/>
+            <pid name="knee_pitch_3"  profile="big_mot"/>
+            <pid name="ankle_pitch_3" profile="medium_mot"/>
+            <pid name="ankle_yaw_3"   profile="small_mot"/>
+            <pid name="j_wheel_3"     profile="wheel_mot"/>
+            <pid name="hip_yaw_4"     profile="big_mot"/>
+            <pid name="hip_pitch_4"   profile="big_mot"/>
+            <pid name="knee_pitch_4"  profile="big_mot"/>
+            <pid name="ankle_pitch_4" profile="medium_mot"/>
+            <pid name="ankle_yaw_4"   profile="small_mot"/>
+            <pid name="j_wheel_4"     profile="wheel_mot"/>
+        </pid>
+    </plugin>
 </gazebo>
 </robot>

Commit message: disable realsenses

File: centauro_urdf/urdf/_centauro_robot.urdf (robot description, URDF)
Before this commit: robot centauro, 84 links, 83 joints
Links:
- removed link D435i_camera_accel_frame
- removed link D435i_camera_accel_optical_frame
- removed link D435i_camera_bottom_screw_frame
- removed link D435i_camera_color_frame
- removed link D435i_camera_color_optical_frame
- removed link D435i_camera_depth_frame
- removed link D435i_camera_depth_optical_frame
- removed link D435i_camera_gyro_frame
- removed link D435i_camera_gyro_optical_frame
- removed link D435i_camera_left_ir_frame
- removed link D435i_camera_left_ir_optical_frame
- removed link D435i_camera_link
- removed link D435i_camera_right_ir_frame
- removed link D435i_camera_right_ir_optical_frame
- removed link T265_camera_accel_frame
- removed link T265_camera_accel_optical_frame
- removed link T265_camera_fisheye1_optical_frame
- removed link T265_camera_fisheye1_rgb_frame
- removed link T265_camera_fisheye2_optical_frame
- removed link T265_camera_fisheye2_rgb_frame
- removed link T265_camera_gyro_frame
- removed link T265_camera_gyro_optical_frame
- removed link T265_camera_link
- removed link T265_camera_pose_frame
Joints:
- removed joint D435i_camera_accel_joint
- removed joint D435i_camera_accel_optical_joint
- removed joint D435i_camera_color_joint
- removed joint D435i_camera_color_optical_joint
- removed joint D435i_camera_depth_joint
- removed joint D435i_camera_depth_optical_joint
- removed joint D435i_camera_gyro_joint
- removed joint D435i_camera_gyro_optical_joint
- removed joint D435i_camera_joint
- removed joint D435i_camera_left_ir_joint
- removed joint D435i_camera_left_ir_optical_joint
- removed joint D435i_camera_link_joint
- removed joint D435i_camera_right_ir_joint
- removed joint D435i_camera_right_ir_optical_joint
- removed joint T265_camera_accel_joint
- removed joint T265_camera_accel_optical_joint
- removed joint T265_camera_fisheye1_optical_joint
- removed joint T265_camera_fisheye1_rgb_joint
- removed joint T265_camera_fisheye2_optical_joint
- removed joint T265_camera_fisheye2_rgb_joint
- removed joint T265_camera_gyro_joint
- removed joint T265_camera_gyro_optical_joint
- removed joint T265_camera_link_joint
- removed joint T265_camera_pose_joint

File: centauro_urdf/urdf/centauro.urdf (robot description, URDF)
Before this commit: robot centauro, 84 links, 83 joints
Links:
- removed link D435i_camera_accel_frame
- removed link D435i_camera_accel_optical_frame
- removed link D435i_camera_bottom_screw_frame
- removed link D435i_camera_color_frame
- removed link D435i_camera_color_optical_frame
- removed link D435i_camera_depth_frame
- removed link D435i_camera_depth_optical_frame
- removed link D435i_camera_gyro_frame
- removed link D435i_camera_gyro_optical_frame
- removed link D435i_camera_left_ir_frame
- removed link D435i_camera_left_ir_optical_frame
- removed link D435i_camera_link
- removed link D435i_camera_right_ir_frame
- removed link D435i_camera_right_ir_optical_frame
- removed link T265_camera_accel_frame
- removed link T265_camera_accel_optical_frame
- removed link T265_camera_fisheye1_optical_frame
- removed link T265_camera_fisheye1_rgb_frame
- removed link T265_camera_fisheye2_optical_frame
- removed link T265_camera_fisheye2_rgb_frame
- removed link T265_camera_gyro_frame
- removed link T265_camera_gyro_optical_frame
- removed link T265_camera_link
- removed link T265_camera_pose_frame
Joints:
- removed joint D435i_camera_accel_joint
- removed joint D435i_camera_accel_optical_joint
- removed joint D435i_camera_color_joint
- removed joint D435i_camera_color_optical_joint
- removed joint D435i_camera_depth_joint
- removed joint D435i_camera_depth_optical_joint
- removed joint D435i_camera_gyro_joint
- removed joint D435i_camera_gyro_optical_joint
- removed joint D435i_camera_joint
- removed joint D435i_camera_left_ir_joint
- removed joint D435i_camera_left_ir_optical_joint
- removed joint D435i_camera_link_joint
- removed joint D435i_camera_right_ir_joint
- removed joint D435i_camera_right_ir_optical_joint
- removed joint T265_camera_accel_joint
- removed joint T265_camera_accel_optical_joint
- removed joint T265_camera_fisheye1_optical_joint
- removed joint T265_camera_fisheye1_rgb_joint
- removed joint T265_camera_fisheye2_optical_joint
- removed joint T265_camera_fisheye2_rgb_joint
- removed joint T265_camera_gyro_joint
- removed joint T265_camera_gyro_optical_joint
- removed joint T265_camera_link_joint
- removed joint T265_camera_pose_joint

File: centauro_urdf/urdf/centauro_config.urdf.xacro (robot description, xacro)
@@ -15,5 +15,5 @@
 <xacro:property name="USE_STICKS" value="false" />
 <xacro:property name="ADD_VELODYNE" value="true" />
-<xacro:property name="ADD_INTEL_D435I" value="true" />
-<xacro:property name="ADD_INTEL_T265" value="true" />
+<xacro:property name="ADD_INTEL_D435I" value="false" />
+<xacro:property name="ADD_INTEL_T265" value="false" />
 </robot>
