Commit message: set sensors to false

File: centauro_urdf/urdf/_centauro_robot.urdf (robot description, URDF)
Before this commit: robot centauro, 59 links, 58 joints
Links:
- removed link velodyne_calib
- removed link velodyne_calib_base_link
- added link d435_head_motor, mass 0.33878686; collision mesh filename=package://centauro_urdf/meshes/simple/neck-pitch_mesh.stl scale=0.001 0.001 0.001; visual mesh filename=package://centauro_urdf/meshes/neck-pitch_mesh.stl scale=0.001 0.001 0.001
Joints:
- removed joint velodyne_calib_base_mount_joint
- removed joint velodyne_calib_base_scan_joint
- added joint d435_head_joint: type revolute, parent neck_1, child d435_head_motor, origin xyz=0.06 0 0.1375 rpy=0 0 0, axis 0 1 0, limit lower=-1.1 upper=1.1 effort=35 velocity=5.7

File: centauro_urdf/urdf/centauro.urdf (robot description, URDF)
Before this commit: robot centauro, 59 links, 58 joints
Links:
- removed link velodyne_calib
- removed link velodyne_calib_base_link
- added link d435_head_motor, mass 0.33878686; collision mesh filename=package://centauro_urdf/meshes/simple/neck-pitch_mesh.stl scale=0.001 0.001 0.001; visual mesh filename=package://centauro_urdf/meshes/neck-pitch_mesh.stl scale=0.001 0.001 0.001
Joints:
- removed joint velodyne_calib_base_mount_joint
- removed joint velodyne_calib_base_scan_joint
- added joint d435_head_joint: type revolute, parent neck_1, child d435_head_motor, origin xyz=0.06 0 0.1375 rpy=0 0 0, axis 0 1 0, limit lower=-1.1 upper=1.1 effort=35 velocity=5.7

File: centauro_urdf/urdf/centauro_base.urdf.xacro (robot description, xacro)
@@ -59,32 +59,32 @@
         </xacro:VLP-16>
     </xacro:if>
+    <link name="d435_head_motor">
+        <inertial>
+        <origin xyz="0 0 0"/>
+        <mass value="0.33878686"/> <!-- MASS/INERTIA TO DO -->
+        <inertia ixx="0.0003718568" ixy="-9.42983e-05" ixz="-2.80644e-05" iyy="0.0001886879" iyz="-1.54534e-05" izz="0.0005023443"/>
+        </inertial>
+        <visual>
+        <origin rpy="0.0 0.0 0.0" xyz="0.0 0 0.0"/>
+        <geometry>
+            <mesh filename="package://centauro_urdf/meshes/neck-pitch_mesh.stl" scale="0.001 0.001 0.001"/>
+        </geometry>
+        </visual>
+        <collision>
+        <origin rpy="0.0 0.0 0.0" xyz="0.0 0 0.0"/>
+        <geometry>
+            <mesh filename="package://centauro_urdf/meshes/simple/neck-pitch_mesh.stl" scale="0.001 0.001 0.001"/>
+        </geometry>
+        </collision>
+    </link>
+    <joint name="d435_head_joint" type="revolute">
+        <parent link="neck_1"/>
+        <origin xyz="0.06 0 0.1375" rpy="0 0 0"/>
+        <child link="d435_head_motor"/>
+        <axis xyz="0 1 0"/>
+        <limit effort="35" lower="-1.1" upper="1.1" velocity="5.7"/>
+        <dynamics friction="10.0"/>
+    </joint>
     <xacro:if value="${ADD_D435_HEAD}">
-        <link name="d435_head_motor">
-            <inertial>
-            <origin xyz="0 0 0"/>
-            <mass value="0.33878686"/> <!-- MASS/INERTIA TO DO -->
-            <inertia ixx="0.0003718568" ixy="-9.42983e-05" ixz="-2.80644e-05" iyy="0.0001886879" iyz="-1.54534e-05" izz="0.0005023443"/>
-            </inertial>
-            <visual>
-            <origin rpy="0.0 0.0 0.0" xyz="0.0 0 0.0"/>
-            <geometry>
-                <mesh filename="package://centauro_urdf/meshes/neck-pitch_mesh.stl" scale="0.001 0.001 0.001"/>
-            </geometry>
-            </visual>
-            <collision>
-            <origin rpy="0.0 0.0 0.0" xyz="0.0 0 0.0"/>
-            <geometry>
-                <mesh filename="package://centauro_urdf/meshes/simple/neck-pitch_mesh.stl" scale="0.001 0.001 0.001"/>
-            </geometry>
-            </collision>
-        </link>
-        <joint name="d435_head_joint" type="revolute">
-            <parent link="neck_1"/>
-            <origin xyz="0.06 0 0.1375" rpy="0 0 0"/>
-            <child link="d435_head_motor"/>
-            <axis xyz="0 1 0"/>
-            <limit effort="35" lower="-1.1" upper="1.1" velocity="5.7"/>
-            <dynamics friction="10.0"/>
-        </joint>
         <xacro:include filename="$(find realsense_gazebo_description)/urdf/_d435i.urdf.xacro" />
         <xacro:sensor_d435i parent="d435_head_motor" name="D435_head_camera" topics_ns="D435/D435_head_camera"

File: centauro_urdf/urdf/centauro_config.urdf.xacro (robot description, xacro)
@@ -14,5 +14,5 @@
 <xacro:property name="ADD_VIRTUAL_FRAME" value="false" />
 <xacro:property name="USE_STICKS" value="false" />
-<xacro:property name="ADD_VELODYNE" value="true" />
+<xacro:property name="ADD_VELODYNE" value="false" />
 <xacro:property name="ADD_D435_HEAD" value="false" />
 <xacro:property name="ADD_INTEL_D435I" value="false" />

File: centauro_urdf/urdf/centauro_virtual_frame.urdf (robot description, URDF)
Before this commit: robot centauro, 75 links, 74 joints
Links:
- removed link T265_camera_accel_frame
- removed link T265_camera_accel_optical_frame
- removed link T265_camera_fisheye1_optical_frame
- removed link T265_camera_fisheye1_rgb_frame
- removed link T265_camera_fisheye2_optical_frame
- removed link T265_camera_fisheye2_rgb_frame
- removed link T265_camera_gyro_frame
- removed link T265_camera_gyro_optical_frame
- removed link T265_camera_link
- removed link T265_camera_pose_frame
- removed link velodyne_calib
- removed link velodyne_calib_base_link
- added link d435_head_motor, mass 0.33878686; collision mesh filename=package://centauro_urdf/meshes/simple/neck-pitch_mesh.stl scale=0.001 0.001 0.001; visual mesh filename=package://centauro_urdf/meshes/neck-pitch_mesh.stl scale=0.001 0.001 0.001
Joints:
- removed joint T265_camera_accel_joint
- removed joint T265_camera_accel_optical_joint
- removed joint T265_camera_fisheye1_optical_joint
- removed joint T265_camera_fisheye1_rgb_joint
- removed joint T265_camera_fisheye2_optical_joint
- removed joint T265_camera_fisheye2_rgb_joint
- removed joint T265_camera_gyro_joint
- removed joint T265_camera_gyro_optical_joint
- removed joint T265_camera_link_joint
- removed joint T265_camera_pose_joint
- removed joint velodyne_calib_base_mount_joint
- removed joint velodyne_calib_base_scan_joint
- added joint d435_head_joint: type revolute, parent neck_1, child d435_head_motor, origin xyz=0.06 0 0.1375 rpy=0 0 0, axis 0 1 0, limit lower=-1.1 upper=1.1 effort=35 velocity=5.7

File: centauro_urdf/urdf/centauro_virtual_frame_robot.urdf (robot description, URDF)
Before this commit: robot centauro, 75 links, 74 joints
Links:
- removed link T265_camera_accel_frame
- removed link T265_camera_accel_optical_frame
- removed link T265_camera_fisheye1_optical_frame
- removed link T265_camera_fisheye1_rgb_frame
- removed link T265_camera_fisheye2_optical_frame
- removed link T265_camera_fisheye2_rgb_frame
- removed link T265_camera_gyro_frame
- removed link T265_camera_gyro_optical_frame
- removed link T265_camera_link
- removed link T265_camera_pose_frame
- removed link velodyne_calib
- removed link velodyne_calib_base_link
- added link d435_head_motor, mass 0.33878686; collision mesh filename=package://centauro_urdf/meshes/simple/neck-pitch_mesh.stl scale=0.001 0.001 0.001; visual mesh filename=package://centauro_urdf/meshes/neck-pitch_mesh.stl scale=0.001 0.001 0.001
Joints:
- removed joint T265_camera_accel_joint
- removed joint T265_camera_accel_optical_joint
- removed joint T265_camera_fisheye1_optical_joint
- removed joint T265_camera_fisheye1_rgb_joint
- removed joint T265_camera_fisheye2_optical_joint
- removed joint T265_camera_fisheye2_rgb_joint
- removed joint T265_camera_gyro_joint
- removed joint T265_camera_gyro_optical_joint
- removed joint T265_camera_link_joint
- removed joint T265_camera_pose_joint
- removed joint velodyne_calib_base_mount_joint
- removed joint velodyne_calib_base_scan_joint
- added joint d435_head_joint: type revolute, parent neck_1, child d435_head_motor, origin xyz=0.06 0 0.1375 rpy=0 0 0, axis 0 1 0, limit lower=-1.1 upper=1.1 effort=35 velocity=5.7

File: centauro_urdf/urdf/config/centauro_virtual_frame.urdf.xacro (robot description, xacro)
@@ -14,7 +14,7 @@
 <xacro:property name="ADD_VIRTUAL_FRAME" value="true" />
 <xacro:property name="USE_STICKS" value="false" />
-<xacro:property name="ADD_VELODYNE" value="true" />
+<xacro:property name="ADD_VELODYNE" value="false" />
 <xacro:property name="ADD_D435_HEAD" value="false" />
 <xacro:property name="ADD_INTEL_D435I" value="false" />
-<xacro:property name="ADD_INTEL_T265" value="true" />
+<xacro:property name="ADD_INTEL_T265" value="false" />
 </robot>
