Commit message: bullet experiments

File: centauro_urdf/urdf/centauro_robot.urdf (robot description, URDF)
Before this commit: robot centauro, 58 links, 57 joints
Links:
- removed link world
- link ankle1_1: geometry collision mesh filename=package://centauro_urdf/meshes/v2/collision/ankle-pitch.stl scale=0.001 0.001 -0.001; visual mesh filename=package://centauro_urdf/meshes/v2/ankle-pitch.stl scale=0.001 0.001 -0.001
- link ankle1_2: geometry collision mesh filename=package://centauro_urdf/meshes/v2/collision/ankle-pitch.stl scale=0.001 0.001 0.001; visual mesh filename=package://centauro_urdf/meshes/v2/ankle-pitch.stl scale=0.001 0.001 0.001
- link ankle1_3: geometry collision mesh filename=package://centauro_urdf/meshes/v2/collision/ankle-pitch.stl scale=0.001 0.001 -0.001; visual mesh filename=package://centauro_urdf/meshes/v2/ankle-pitch.stl scale=0.001 0.001 -0.001
- link ankle1_4: geometry collision mesh filename=package://centauro_urdf/meshes/v2/collision/ankle-pitch.stl scale=0.001 0.001 0.001; visual mesh filename=package://centauro_urdf/meshes/v2/ankle-pitch.stl scale=0.001 0.001 0.001
- link ankle2_1: geometry collision mesh filename=package://centauro_urdf/meshes/v2/collision/ankle-yaw.stl scale=0.001 -0.001 0.001; visual mesh filename=package://centauro_urdf/meshes/v2/ankle-yaw.stl scale=0.001 -0.001 0.001
- link ankle2_2: geometry collision mesh filename=package://centauro_urdf/meshes/v2/collision/ankle-yaw.stl scale=0.001 0.001 0.001; visual mesh filename=package://centauro_urdf/meshes/v2/ankle-yaw.stl scale=0.001 0.001 0.001
- link ankle2_3: geometry collision mesh filename=package://centauro_urdf/meshes/v2/collision/ankle-yaw.stl scale=0.001 -0.001 0.001; visual mesh filename=package://centauro_urdf/meshes/v2/ankle-yaw.stl scale=0.001 -0.001 0.001
- link ankle2_4: geometry collision mesh filename=package://centauro_urdf/meshes/v2/collision/ankle-yaw.stl scale=0.001 0.001 0.001; visual mesh filename=package://centauro_urdf/meshes/v2/ankle-yaw.stl scale=0.001 0.001 0.001
- link arm1_1: geometry collision mesh filename=package://centauro_urdf/meshes/simple/ShoulderPitch.STL scale=0.001 -0.001 0.001; visual mesh filename=package://centauro_urdf/meshes/ShoulderPitch.STL scale=0.001 -0.001 0.001
- link arm1_2: geometry collision mesh filename=package://centauro_urdf/meshes/simple/ShoulderRoll.STL scale=0.001 -0.001 0.001; visual mesh filename=package://centauro_urdf/meshes/ShoulderRoll.STL scale=0.001 -0.001 0.001
- link arm1_3: geometry collision mesh filename=package://centauro_urdf/meshes/simple/ShoulderYaw.STL scale=0.001 -0.001 0.001; visual mesh filename=package://centauro_urdf/meshes/ShoulderYaw.STL scale=0.001 -0.001 0.001
- link arm1_4: geometry collision mesh filename=package://centauro_urdf/meshes/simple/Elbow.STL scale=0.001 -0.001 0.001; visual mesh filename=package://centauro_urdf/meshes/Elbow.STL scale=0.001 -0.001 0.001
- link arm1_5: geometry collision mesh filename=package://centauro_urdf/meshes/simple/Forearm.STL scale=0.001 -0.001 0.001; visual mesh filename=package://centauro_urdf/meshes/Forearm.STL scale=0.001 -0.001 0.001
- link arm1_6: geometry collision mesh filename=package://centauro_urdf/meshes/simple/ForearmPitch.STL scale=0.001 -0.001 0.001; visual mesh filename=package://centauro_urdf/meshes/ForearmPitch.STL scale=0.001 -0.001 0.001
- link arm1_7: geometry collision mesh filename=package://centauro_urdf/meshes/simple/ForearmYaw.STL scale=0.001 -0.001 0.001; visual mesh filename=package://centauro_urdf/meshes/ForearmYaw.STL scale=0.001 -0.001 0.001
- link arm2_1: geometry collision mesh filename=package://centauro_urdf/meshes/simple/ShoulderPitch.STL scale=0.001 0.001 0.001; visual mesh filename=package://centauro_urdf/meshes/ShoulderPitch.STL scale=0.001 0.001 0.001
- link arm2_2: geometry collision mesh filename=package://centauro_urdf/meshes/simple/ShoulderRoll.STL scale=0.001 0.001 0.001; visual mesh filename=package://centauro_urdf/meshes/ShoulderRoll.STL scale=0.001 0.001 0.001
- link arm2_3: geometry collision mesh filename=package://centauro_urdf/meshes/simple/ShoulderYaw.STL scale=0.001 0.001 0.001; visual mesh filename=package://centauro_urdf/meshes/ShoulderYaw.STL scale=0.001 0.001 0.001
- link arm2_4: geometry collision mesh filename=package://centauro_urdf/meshes/simple/Elbow.STL scale=0.001 0.001 0.001; visual mesh filename=package://centauro_urdf/meshes/Elbow.STL scale=0.001 0.001 0.001
- link arm2_5: geometry collision mesh filename=package://centauro_urdf/meshes/simple/Forearm.STL scale=0.001 0.001 0.001; visual mesh filename=package://centauro_urdf/meshes/Forearm.STL scale=0.001 0.001 0.001
- link arm2_6: geometry collision mesh filename=package://centauro_urdf/meshes/simple/ForearmPitch.STL scale=0.001 0.001 0.001; visual mesh filename=package://centauro_urdf/meshes/ForearmPitch.STL scale=0.001 0.001 0.001
- link arm2_7: geometry collision mesh filename=package://centauro_urdf/meshes/simple/ForearmYaw.STL scale=0.001 0.001 0.001; visual mesh filename=package://centauro_urdf/meshes/ForearmYaw.STL scale=0.001 0.001 0.001
- link ball1: geometry collision mesh filename=package://centauro_urdf/meshes/simple/BallHand.stl scale=0.001 0.001 0.001; visual mesh filename=package://centauro_urdf/meshes/BallHand.stl scale=0.001 0.001 0.001
- link ball2: geometry collision mesh filename=package://centauro_urdf/meshes/simple/BallHand.stl scale=0.001 0.001 0.001; visual mesh filename=package://centauro_urdf/meshes/BallHand.stl scale=0.001 0.001 0.001
- link hip1_1: geometry collision mesh filename=package://centauro_urdf/meshes/v2/collision/hip-yaw.stl scale=0.001 -0.001 0.001; visual mesh filename=package://centauro_urdf/meshes/v2/hip-yaw.stl scale=0.001 -0.001 0.001
- link hip1_2: geometry collision mesh filename=package://centauro_urdf/meshes/v2/collision/hip-yaw.stl scale=0.001 0.001 0.001; visual mesh filename=package://centauro_urdf/meshes/v2/hip-yaw.stl scale=0.001 0.001 0.001
- link hip1_3: geometry collision mesh filename=package://centauro_urdf/meshes/v2/collision/hip-yaw.stl scale=0.001 -0.001 0.001; visual mesh filename=package://centauro_urdf/meshes/v2/hip-yaw.stl scale=0.001 -0.001 0.001
- link hip1_4: geometry collision mesh filename=package://centauro_urdf/meshes/v2/collision/hip-yaw.stl scale=0.001 0.001 0.001; visual mesh filename=package://centauro_urdf/meshes/v2/hip-yaw.stl scale=0.001 0.001 0.001
- link hip2_1: geometry collision mesh filename=package://centauro_urdf/meshes/v2/collision/hip-pitch.stl scale=0.001 0.001 -0.001; visual mesh filename=package://centauro_urdf/meshes/v2/hip-pitch.stl scale=0.001 0.001 -0.001
- link hip2_2: geometry collision mesh filename=package://centauro_urdf/meshes/v2/collision/hip-pitch.stl scale=0.001 0.001 0.001; visual mesh filename=package://centauro_urdf/meshes/v2/hip-pitch.stl scale=0.001 0.001 0.001
- link hip2_3: geometry collision mesh filename=package://centauro_urdf/meshes/v2/collision/hip-pitch.stl scale=0.001 0.001 -0.001; visual mesh filename=package://centauro_urdf/meshes/v2/hip-pitch.stl scale=0.001 0.001 -0.001
- link hip2_4: geometry collision mesh filename=package://centauro_urdf/meshes/v2/collision/hip-pitch.stl scale=0.001 0.001 0.001; visual mesh filename=package://centauro_urdf/meshes/v2/hip-pitch.stl scale=0.001 0.001 0.001
- link knee_1: geometry collision mesh filename=package://centauro_urdf/meshes/v2/collision/knee.stl scale=0.001 0.001 -0.001; visual mesh filename=package://centauro_urdf/meshes/v2/knee.stl scale=0.001 0.001 -0.001
- link knee_2: geometry collision mesh filename=package://centauro_urdf/meshes/v2/collision/knee.stl scale=0.001 0.001 0.001; visual mesh filename=package://centauro_urdf/meshes/v2/knee.stl scale=0.001 0.001 0.001
- link knee_3: geometry collision mesh filename=package://centauro_urdf/meshes/v2/collision/knee.stl scale=0.001 0.001 -0.001; visual mesh filename=package://centauro_urdf/meshes/v2/knee.stl scale=0.001 0.001 -0.001
- link knee_4: geometry collision mesh filename=package://centauro_urdf/meshes/v2/collision/knee.stl scale=0.001 0.001 0.001; visual mesh filename=package://centauro_urdf/meshes/v2/knee.stl scale=0.001 0.001 0.001
- link neck_1: geometry collision mesh filename=package://centauro_urdf/meshes/simple/neck_yaw.stl scale=0.001 0.001 0.001; visual mesh filename=package://centauro_urdf/meshes/neck_yaw.stl scale=0.001 0.001 0.001
- link neck_2: geometry collision mesh filename=package://centauro_urdf/meshes/simple/neck_pitch.stl scale=0.001 0.001 0.001; visual mesh filename=package://centauro_urdf/meshes/neck_pitch.stl scale=0.001 0.001 0.001
- link neck_3: geometry collision mesh filename=package://centauro_urdf/meshes/simple/lidar.stl scale=0.001 0.001 0.001; visual mesh filename=package://centauro_urdf/meshes/lidar.stl scale=0.001 0.001 0.001
- link pelvis: geometry collision mesh filename=package://centauro_urdf/meshes/simple/pelvis.stl scale=0.001 0.001 0.001; visual mesh filename=package://centauro_urdf/meshes/v2/pelvis.stl scale=0.001 0.001 0.001
- link torso_2: geometry collision mesh filename=package://centauro_urdf/meshes/simple/link1.stl scale=0.001 0.001 0.001; visual mesh filename=package://centauro_urdf/meshes/link1.stl scale=0.001 0.001 0.001
- link wheel_1: geometry collision cylinder length=0.11 radius=0.078; visual mesh filename=package://centauro_urdf/meshes/v2/wheel.stl scale=0.001 0.001 -0.001
- link wheel_2: geometry collision cylinder length=0.11 radius=0.078; visual mesh filename=package://centauro_urdf/meshes/v2/wheel.stl scale=0.001 0.001 0.001
- link wheel_3: geometry collision cylinder length=0.11 radius=0.078; visual mesh filename=package://centauro_urdf/meshes/v2/wheel.stl scale=0.001 0.001 -0.001
- link wheel_4: geometry collision cylinder length=0.11 radius=0.078; visual mesh filename=package://centauro_urdf/meshes/v2/wheel.stl scale=0.001 0.001 0.001
Joints:
- removed joint reference

File: centauro_urdf/urdf/gazebo/xbot.gazebo.xacro (robot description, xacro)
@@ -17,7 +17,7 @@
             <gain name="big_mot"    p="8000" d="50"/>
             <gain name="wheel_mot"  p="0" d="10"/>
-            <pid name="neck_yaw" profile="lowpwr_mot"/>
-            <pid name="neck_pitch" profile="lowpwr_mot"/>
-            <pid name="neck_velodyne" p="0"  d="20"/>
+            <pid name="neck_yaw" p="5"  d="1"/>
+            <pid name="neck_pitch" p="5"  d="1"/>
+            <pid name="neck_velodyne" p="0"  d="10"/>
             <pid name="j_arm1_1" profile="medium_mot"/>
             <pid name="j_arm1_2" profile="medium_mot"/>
