Commit message: update centauro urdf with pinocchio capsules

File: centauro_urdf/urdf/centauro_pinocchio_capsule.urdf (robot description, URDF)
Before this commit: robot centauro, 98 links, 97 joints
Links:
- removed link arm1_7
- removed link arm2_7
- removed link ft_arm1
- removed link ft_arm2
- link ankle1_2: geometry collision cylinder length=0.04788405128558378 radius=0.0781037; visual mesh filename=package://centauro_urdf/meshes/v2/ankle-pitch.stl scale=0.001 0.001 0.001
- link ankle1_4: geometry collision cylinder length=0.04788405128558378 radius=0.0781037; visual mesh filename=package://centauro_urdf/meshes/v2/ankle-pitch.stl scale=0.001 0.001 0.001
- link arm1_5: geometry collision cylinder length=0.08434739747702645 radius=0.0804108; visual mesh filename=package://centauro_urdf/meshes/Forearm.STL scale=0.001 -0.001 0.001
- link arm1_6: geometry collision cylinder length=0.07750977987441161 radius=0.0474698; visual mesh filename=package://centauro_urdf/meshes/wrist_pitch_right.stl scale=0.001 -0.001 0.001
- link arm2_5: geometry collision cylinder length=0.08434739747702645 radius=0.0804108; visual mesh filename=package://centauro_urdf/meshes/Forearm.STL scale=0.001 0.001 0.001
- link arm2_6: geometry collision cylinder length=0.07750977987441161 radius=0.0474698; visual mesh filename=package://centauro_urdf/meshes/wrist_pitch_right.stl scale=0.001 0.001 0.001
- link knee_1: geometry collision cylinder length=0.1927502246061244 radius=0.0664305; visual mesh filename=package://centauro_urdf/meshes/v2/knee.stl scale=0.001 0.001 -0.001
- link knee_2: geometry collision cylinder length=0.1927502246061244 radius=0.0664305; visual mesh filename=package://centauro_urdf/meshes/v2/knee.stl scale=0.001 0.001 0.001
- link knee_3: geometry collision cylinder length=0.1927502246061244 radius=0.0664305; visual mesh filename=package://centauro_urdf/meshes/v2/knee.stl scale=0.001 0.001 -0.001
- link knee_4: geometry collision cylinder length=0.1927502246061244 radius=0.0664305; visual mesh filename=package://centauro_urdf/meshes/v2/knee.stl scale=0.001 0.001 0.001
Joints:
- removed joint j_arm1_7
- removed joint j_arm2_7
- removed joint j_ft_1
- removed joint j_ft_2
- joint j_arm1_8: origin xyz=0.0 0.0 0.0 rpy=0.0 0.0 0.0 -> xyz=0.0 -0.05 -0.105 rpy=0.0 0.0 0.0; parent arm1_7 -> arm1_6
- joint j_arm2_8: origin xyz=0.0 0.0 0.0 rpy=0.0 0.0 0.0 -> xyz=0.0 0.05 -0.105 rpy=0.0 0.0 0.0; parent arm2_7 -> arm2_6
