Commit message: upd generated

File: centauro_urdf/urdf/centauro_virtual_frame.urdf (robot description, URDF)
Before this commit: robot centauro, 64 links, 63 joints
Links:
- removed link arm1_7
- removed link arm2_7
- removed link ft_arm1
- removed link ft_arm2
- added link D435_head_camera_bottom_screw_frame
- added link D435_head_camera_link, mass 0.564; collision box size=0.02505 0.09 0.025; visual mesh filename=package://centauro_urdf/meshes/realsense/d435.dae
- added link D435i_camera_bottom_screw_frame
- added link D435i_camera_link, mass 0.564; collision box size=0.02505 0.09 0.025; visual mesh filename=package://centauro_urdf/meshes/realsense/d435.dae
- link arm1_6: geometry collision mesh filename=package://centauro_urdf/meshes/simple/wrist_pitch_right.stl scale=0.001 -0.001 0.001; visual mesh filename=package://centauro_urdf/meshes/wrist_pitch_right.stl scale=0.001 -0.001 0.001
- link arm2_6: geometry collision mesh filename=package://centauro_urdf/meshes/simple/wrist_pitch_right.stl scale=0.001 0.001 0.001; visual mesh filename=package://centauro_urdf/meshes/wrist_pitch_right.stl scale=0.001 0.001 0.001
Joints:
- removed joint j_arm1_7
- removed joint j_arm2_7
- removed joint j_ft_1
- removed joint j_ft_2
- added joint D435_head_camera_joint: type fixed, parent d435_head_motor, child D435_head_camera_bottom_screw_frame, origin xyz=0.03015 0 -0.0125 rpy=0 0 0
- added joint D435_head_camera_link_joint: type fixed, parent D435_head_camera_bottom_screw_frame, child D435_head_camera_link, origin xyz=0 0.0175 0.0125 rpy=0 0 0
- added joint D435i_camera_joint: type fixed, parent pelvis, child D435i_camera_bottom_screw_frame, origin xyz=0.27187 0 0.0215997 rpy=0 0.5251508 0
- added joint D435i_camera_link_joint: type fixed, parent D435i_camera_bottom_screw_frame, child D435i_camera_link, origin xyz=0 0.0175 0.0125 rpy=0 0 0
- joint j_arm1_8: origin xyz=0. 0. 0. rpy=0. 0. 0. -> xyz=0. -0.05 -0.105 rpy=0. 0. 0.; parent arm1_7 -> arm1_6
- joint j_arm2_8: origin xyz=0. 0. 0. rpy=0. 0. 0. -> xyz=0. 0.05 -0.105 rpy=0. 0. 0.; parent arm2_7 -> arm2_6

Commit message: virtual frame urdf includes cameras

File: centauro_urdf/urdf/centauro_virtual_frame.urdf (robot description, URDF)
Before this commit: robot centauro, 64 links, 63 joints
Links:
- added link D435_head_camera_accel_frame
- added link D435_head_camera_accel_optical_frame
- added link D435_head_camera_color_frame
- added link D435_head_camera_color_optical_frame
- added link D435_head_camera_depth_frame
- added link D435_head_camera_depth_optical_frame
- added link D435_head_camera_gyro_frame
- added link D435_head_camera_gyro_optical_frame
- added link D435_head_camera_left_ir_frame
- added link D435_head_camera_left_ir_optical_frame
- added link D435_head_camera_right_ir_frame
- added link D435_head_camera_right_ir_optical_frame
- added link D435i_camera_accel_frame
- added link D435i_camera_accel_optical_frame
- added link D435i_camera_color_frame
- added link D435i_camera_color_optical_frame
- added link D435i_camera_depth_frame
- added link D435i_camera_depth_optical_frame
- added link D435i_camera_gyro_frame
- added link D435i_camera_gyro_optical_frame
- added link D435i_camera_left_ir_frame
- added link D435i_camera_left_ir_optical_frame
- added link D435i_camera_right_ir_frame
- added link D435i_camera_right_ir_optical_frame
- added link T265_camera_accel_frame
- added link T265_camera_accel_optical_frame
- added link T265_camera_fisheye1_optical_frame
- added link T265_camera_fisheye1_rgb_frame
- added link T265_camera_fisheye2_optical_frame
- added link T265_camera_fisheye2_rgb_frame
- added link T265_camera_gyro_frame
- added link T265_camera_gyro_optical_frame
- added link T265_camera_link
- added link T265_camera_pose_frame, mass 0.068024; collision mesh filename=package://realsense_gazebo_description/meshes/t265_simplifi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 scale=0.001 0.001 0.001; visual mesh filename=package://realsense_gazebo_description/meshes/t265_full.stl scale=0.001 0.001 0.001
- added link velodyne_calib, mass 0.01; visual mesh filename=package://velodyne_description/meshes/VLP16_scan.dae
- added link velodyne_calib_base_link, mass 0.83; collision cylinder length=0.0717 radius=0.0516; visual mesh filename=package://velodyne_description/meshes/VLP16_base_1.dae
- link D435_head_camera_link: geometry collision box size=0.02505 0.09 0.025; visual mesh filename=package://realsense2_description/meshes/d435.dae
- link D435i_camera_link: geometry collision box size=0.02505 0.09 0.025; visual mesh filename=package://realsense2_description/meshes/d435.dae
Joints:
- added joint D435_head_camera_accel_joint: type fixed, parent D435_head_camera_link, child D435_head_camera_accel_frame, origin xyz=-0.00174 0.00552 0.0176 rpy=0 0 0
- added joint D435_head_camera_accel_optical_joint: type fixed, parent D435_head_camera_accel_frame, child D435_head_camera_accel_optical_frame, origin xyz=0 0 0 rpy=-1.5707963267948966 0 -1.5707963267948966
- added joint D435_head_camera_color_joint: type fixed, parent D435_head_camera_depth_frame, child D435_head_camera_color_frame, origin xyz=0 0.015 0 rpy=0 0 0
- added joint D435_head_camera_color_optical_joint: type fixed, parent D435_head_camera_color_frame, child D435_head_camera_color_optical_frame, origin xyz=0 0 0 rpy=-1.5707963267948966 0 -1.5707963267948966
- added joint D435_head_camera_depth_joint: type fixed, parent D435_head_camera_link, child D435_head_camera_depth_frame, origin xyz=0 0 0 rpy=0 0 0
- added joint D435_head_camera_depth_optical_joint: type fixed, parent D435_head_camera_depth_frame, child D435_head_camera_depth_optical_frame, origin xyz=0 0 0 rpy=-1.5707963267948966 0 -1.5707963267948966
- added joint D435_head_camera_gyro_joint: type fixed, parent D435_head_camera_link, child D435_head_camera_gyro_frame, origin xyz=-0.00174 0.00552 0.0176 rpy=0 0 0
- added joint D435_head_camera_gyro_optical_joint: type fixed, parent D435_head_camera_gyro_frame, child D435_head_camera_gyro_optical_frame, origin xyz=0 0 0 rpy=-1.5707963267948966 0 -1.5707963267948966
- added joint D435_head_camera_left_ir_joint: type fixed, parent D435_head_camera_depth_frame, child D435_head_camera_left_ir_frame, origin xyz=0 0.0 0 rpy=0 0 0
- added joint D435_head_camera_left_ir_optical_joint: type fixed, parent D435_head_camera_left_ir_frame, child D435_head_camera_left_ir_optical_frame, origin xyz=0 0 0 rpy=-1.5707963267948966 0 -1.5707963267948966
- added joint D435_head_camera_right_ir_joint: type fixed, parent D435_head_camera_depth_frame, child D435_head_camera_right_ir_frame, origin xyz=0 -0.05 0 rpy=0 0 0
- added joint D435_head_camera_right_ir_optical_joint: type fixed, parent D435_head_camera_right_ir_frame, child D435_head_camera_right_ir_optical_frame, origin xyz=0 0 0 rpy=-1.5707963267948966 0 -1.5707963267948966
- added joint D435i_camera_accel_joint: type fixed, parent D435i_camera_link, child D435i_camera_accel_frame, origin xyz=-0.00174 0.00552 0.0176 rpy=0 0 0
- added joint D435i_camera_accel_optical_joint: type fixed, parent D435i_camera_accel_frame, child D435i_camera_accel_optical_frame, origin xyz=0 0 0 rpy=-1.5707963267948966 0 -1.5707963267948966
- added joint D435i_camera_color_joint: type fixed, parent D435i_camera_depth_frame, child D435i_camera_color_frame, origin xyz=0 0.015 0 rpy=0 0 0
- added joint D435i_camera_color_optical_joint: type fixed, parent D435i_camera_color_frame, child D435i_camera_color_optical_frame, origin xyz=0 0 0 rpy=-1.5707963267948966 0 -1.5707963267948966
- added joint D435i_camera_depth_joint: type fixed, parent D435i_camera_link, child D435i_camera_depth_frame, origin xyz=0 0 0 rpy=0 0 0
- added joint D435i_camera_depth_optical_joint: type fixed, parent D435i_camera_depth_frame, child D435i_camera_depth_optical_frame, origin xyz=0 0 0 rpy=-1.5707963267948966 0 -1.5707963267948966
- added joint D435i_camera_gyro_joint: type fixed, parent D435i_camera_link, child D435i_camera_gyro_frame, origin xyz=-0.00174 0.00552 0.0176 rpy=0 0 0
- added joint D435i_camera_gyro_optical_joint: type fixed, parent D435i_camera_gyro_frame, child D435i_camera_gyro_optical_frame, origin xyz=0 0 0 rpy=-1.5707963267948966 0 -1.5707963267948966
- added joint D435i_camera_left_ir_joint: type fixed, parent D435i_camera_depth_frame, child D435i_camera_left_ir_frame, origin xyz=0 0.0 0 rpy=0 0 0
- added joint D435i_camera_left_ir_optical_joint: type fixed, parent D435i_camera_left_ir_frame, child D435i_camera_left_ir_optical_frame, origin xyz=0 0 0 rpy=-1.5707963267948966 0 -1.5707963267948966
- added joint D435i_camera_right_ir_joint: type fixed, parent D435i_camera_depth_frame, child D435i_camera_right_ir_frame, origin xyz=0 -0.05 0 rpy=0 0 0
- added joint D435i_camera_right_ir_optical_joint: type fixed, parent D435i_camera_right_ir_frame, child D435i_camera_right_ir_optical_frame, origin xyz=0 0 0 rpy=-1.5707963267948966 0 -1.5707963267948966
- added joint T265_camera_accel_joint: type fixed, parent T265_camera_link, child T265_camera_accel_frame, origin xyz=-0.0311 0 0.00655 rpy=0 3.141592653589793 0
- added joint T265_camera_accel_optical_joint: type fixed, parent T265_camera_accel_frame, child T265_camera_accel_optical_frame, origin xyz=-0.0311 0 0.00655 rpy=0 3.141592653589793 0
- added joint T265_camera_fisheye1_optical_joint: type fixed, parent T265_camera_fisheye1_rgb_frame, child T265_camera_fisheye1_optical_frame, origin xyz=0 0 0 rpy=-1.5707963267948966 0 -1.5707963267948966
- added joint T265_camera_fisheye1_rgb_joint: type fixed, parent T265_camera_link, child T265_camera_fisheye1_rgb_frame, origin xyz=-0.0411 0.0 0.0 rpy=0 1.5707963267948966 1.5707963267948966
- added joint T265_camera_fisheye2_optical_joint: type fixed, parent T265_camera_fisheye2_rgb_frame, child T265_camera_fisheye2_optical_frame, origin xyz=0 0 0 rpy=-1.5707963267948966 0 -1.5707963267948966
- added joint T265_camera_fisheye2_rgb_joint: type fixed, parent T265_camera_link, child T265_camera_fisheye2_rgb_frame, origin xyz=0.0229 0.0 0.0 rpy=0 1.5707963267948966 1.5707963267948966
- added joint T265_camera_gyro_joint: type fixed, parent T265_camera_link, child T265_camera_gyro_frame, origin xyz=-0.0311 0 0.00655 rpy=0 3.141592653589793 0
- added joint T265_camera_gyro_optical_joint: type fixed, parent T265_camera_gyro_frame, child T265_camera_gyro_optical_frame, origin xyz=0 0 0 rpy=0 0 0
- added joint T265_camera_link_joint: type fixed, parent T265_camera_pose_frame, child T265_camera_link, origin xyz=0 0 0 rpy=1.5707963267948966 0 -1.5707963267948966
- added joint T265_camera_pose_joint: type fixed, parent pelvis, child T265_camera_pose_frame, origin xyz=0.29245 0.00775 0.063 rpy=0 0 0
- added joint velodyne_calib_base_mount_joint: type fixed, parent velodyne_motor, child velodyne_calib_base_link, origin xyz=0 0 0 rpy=0 0 0
- added joint velodyne_calib_base_scan_joint: type fixed, parent velodyne_calib_base_link, child velodyne_calib, origin xyz=0 0 0.0377 rpy=0 0 0

File: centauro_urdf/urdf/config/centauro_virtual_frame.urdf.xacro (robot description, xacro)
@@ -14,7 +14,7 @@
     <xacro:property name="ADD_VIRTUAL_FRAME" value="true" />
     <xacro:property name="USE_STICKS" value="false" />
-    <xacro:property name="ADD_VELODYNE" value="false" />
-    <xacro:property name="ADD_D435I_HEAD" value="false" />
-    <xacro:property name="ADD_D435I_BASE" value="false" />
-    <xacro:property name="ADD_T265_BASE" value="false" />
+    <xacro:property name="ADD_VELODYNE" value="true" />
+    <xacro:property name="ADD_D435I_HEAD" value="true" />
+    <xacro:property name="ADD_D435I_BASE" value="true" />
+    <xacro:property name="ADD_T265_BASE" value="true" />
 </robot>

Commit message: fix virtual frame

File: centauro_urdf/urdf/centauro_virtual_frame.urdf (robot description, URDF)
Before this commit: robot centauro, 38 links, 37 joints
Links:
- added link D435_head_camera_bottom_screw_frame
- added link D435_head_camera_link, mass 0.564; collision box size=0.02505 0.09 0.025; visual mesh filename=package://centauro_urdf/meshes/realsense/d435.dae
- added link D435i_camera_bottom_screw_frame
- added link D435i_camera_link, mass 0.564; collision box size=0.02505 0.09 0.025; visual mesh filename=package://centauro_urdf/meshes/realsense/d435.dae
- added link arm1_1, mass 1.9628675; collision mesh filename=package://centauro_urdf/meshes/simple/ShoulderPitch.STL scale=0.001 -0.001 0.001; visual mesh filename=package://centauro_urdf/meshes/ShoulderPitch.STL scale=0.001 -0.001 0.001
- added link arm1_2, mass 1.8595811; collision mesh filename=package://centauro_urdf/meshes/simple/ShoulderRoll.STL scale=0.001 -0.001 0.001; visual mesh filename=package://centauro_urdf/meshes/ShoulderRoll.STL scale=0.001 -0.001 0.001
- added link arm1_3, mass 1.6678109; collision mesh filename=package://centauro_urdf/meshes/simple/ShoulderYaw.STL scale=0.001 -0.001 0.001; visual mesh filename=package://centauro_urdf/meshes/ShoulderYaw.STL scale=0.001 -0.001 0.001
- added link arm1_4, mass 1.3157289; collision mesh filename=package://centauro_urdf/meshes/simple/Elbow.STL scale=0.001 -0.001 0.001; visual mesh filename=package://centauro_urdf/meshes/Elbow.STL scale=0.001 -0.001 0.001
- added link arm1_5, mass 1.4908547; collision mesh filename=package://centauro_urdf/meshes/simple/Forearm.STL scale=0.001 -0.001 0.001; visual mesh filename=package://centauro_urdf/meshes/Forearm.STL scale=0.001 -0.001 0.001
- added link arm1_6, mass 1.1263612; collision mesh filename=package://centauro_urdf/meshes/simple/wrist_pitch_right.stl scale=0.001 -0.001 0.001; visual mesh filename=package://centauro_urdf/meshes/wrist_pitch_right.stl scale=0.001 -0.001 0.001
- added link arm1_8, mass 0
- added link arm2_1, mass 1.9628675; collision mesh filename=package://centauro_urdf/meshes/simple/ShoulderPitch.STL scale=0.001 0.001 0.001; visual mesh filename=package://centauro_urdf/meshes/ShoulderPitch.STL scale=0.001 0.001 0.001
- added link arm2_2, mass 1.8595811; collision mesh filename=package://centauro_urdf/meshes/simple/ShoulderRoll.STL scale=0.001 0.001 0.001; visual mesh filename=package://centauro_urdf/meshes/ShoulderRoll.STL scale=0.001 0.001 0.001
- added link arm2_3, mass 1.6678109; collision mesh filename=package://centauro_urdf/meshes/simple/ShoulderYaw.STL scale=0.001 0.001 0.001; visual mesh filename=package://centauro_urdf/meshes/ShoulderYaw.STL scale=0.001 0.001 0.001
- added link arm2_4, mass 1.3157289; collision mesh filename=package://centauro_urdf/meshes/simple/Elbow.STL scale=0.001 0.001 0.001; visual mesh filename=package://centauro_urdf/meshes/Elbow.STL scale=0.001 0.001 0.001
- added link arm2_5, mass 1.4908547; collision mesh filename=package://centauro_urdf/meshes/simple/Forearm.STL scale=0.001 0.001 0.001; visual mesh filename=package://centauro_urdf/meshes/Forearm.STL scale=0.001 0.001 0.001
- added link arm2_6, mass 1.1263612; collision mesh filename=package://centauro_urdf/meshes/simple/wrist_pitch_right.stl scale=0.001 0.001 0.001; visual mesh filename=package://centauro_urdf/meshes/wrist_pitch_right.stl scale=0.001 0.001 0.001
- added link arm2_8, mass 0
- added link ball1, mass 1.27; collision mesh filename=package://centauro_urdf/meshes/simple/BallHand.stl scale=0.001 0.001 0.001; visual mesh filename=package://centauro_urdf/meshes/BallHand.stl scale=0.001 0.001 0.001
- added link ball1_tip
- added link ball2, mass 1.27; collision mesh filename=package://centauro_urdf/meshes/simple/BallHand.stl scale=0.001 0.001 0.001; visual mesh filename=package://centauro_urdf/meshes/BallHand.stl scale=0.001 0.001 0.001
- added link ball2_tip
- added link d435_head_motor, mass 0.33878686; collision mesh filename=package://centauro_urdf/meshes/simple/neck-pitch_mesh.stl scale=0.001 0.001 0.001; visual mesh filename=package://centauro_urdf/meshes/neck-pitch_mesh.stl scale=0.001 0.001 0.001
- added link neck_1, mass 0.33878686; collision mesh filename=package://centauro_urdf/meshes/simple/head-base_mesh.stl scale=0.001 0.001 0.001; visual mesh filename=package://centauro_urdf/meshes/head-base_mesh.stl scale=0.001 0.001 0.001
- added link torso_2, mass 12.553731; collision mesh filename=package://centauro_urdf/meshes/simple/link1_no_head.stl scale=0.001 0.001 0.001; visual mesh filename=package://centauro_urdf/meshes/link1_no_head.stl scale=0.001 0.001 0.001
- added link velodyne_motor, mass 0.33878686; collision mesh filename=package://centauro_urdf/meshes/simple/lidar_mesh.stl scale=0.001 0.001 0.001; visual mesh filename=package://centauro_urdf/meshes/lidar_mesh.stl scale=0.001 0.001 0.001
Joints:
- added joint D435_head_camera_joint: type fixed, parent d435_head_motor, child D435_head_camera_bottom_screw_frame, origin xyz=0.03015 0 -0.0125 rpy=0 0 0
- added joint D435_head_camera_link_joint: type fixed, parent D435_head_camera_bottom_screw_frame, child D435_head_camera_link, origin xyz=0 0.0175 0.0125 rpy=0 0 0
- added joint D435i_camera_joint: type fixed, parent pelvis, child D435i_camera_bottom_screw_frame, origin xyz=0.272 0 0.084 rpy=0 0.54 0
- added joint D435i_camera_link_joint: type fixed, parent D435i_camera_bottom_screw_frame, child D435i_camera_link, origin xyz=0.053 0.0 -0.035 rpy=0 0.0050 -0.008
- added joint d435_head_joint: type revolute, parent neck_1, child d435_head_motor, origin xyz=0.06 0 0.1375 rpy=0 0 0, axis 0 -1 0, limit lower=-1.1 upper=1.1 effort=35 velocity=5.7
- added joint j_arm1_1: type revolute, parent torso_2, child arm1_1, origin xyz=0.0457475 0.169137 0.116626 rpy=0.174533 0.0 -0.5235988, axis 0 1 0, limit lower=-3.312 upper=1.615 effort=147.0 velocity=3.86
- added joint j_arm1_2: type revolute, parent arm1_1, child arm1_2, origin xyz=-0.09015 0.062 0.0 rpy=-0.1745327 0.0 0.0, axis 1 0 0, limit lower=0.02 upper=3.431 effort=147.0 velocity=3.86
- added joint j_arm1_3: type revolute, parent arm1_2, child arm1_3, origin xyz=0.09015 0.0 -0.21815, axis 0 0 1, limit lower=-2.552 upper=2.566 effort=147.0 velocity=6.06
- added joint j_arm1_4: type revolute, parent arm1_3, child arm1_4, origin xyz=0.045 0.05515 -0.074, axis 0 1 0, limit lower=-2.465 upper=0.28 effort=147.0 velocity=6.06
- added joint j_arm1_5: type revolute, parent arm1_4, child arm1_5, origin xyz=-0.015 -0.05515 -0.095, axis 0 0 1, limit lower=-2.569 upper=2.562 effort=55.0 velocity=11.72
- added joint j_arm1_6: type revolute, parent arm1_5, child arm1_6, origin xyz=0.0 0.049 -0.156, axis 0 1 0, limit lower=-1.529 upper=1.509 effort=55.0 velocity=11.72
- added joint j_arm1_8: type fixed, parent arm1_6, child ball1, origin xyz=0. -0.05 -0.105 rpy=0. 0. 0.
- added joint j_arm2_1: type revolute, parent torso_2, child arm2_1, origin xyz=0.0457475 -0.169137 0.116626 rpy=-0.174533 0.0 0.5235988, axis 0 1 0, limit lower=-3.3458 upper=1.6012 effort=147.0 velocity=3.86
- added joint j_arm2_2: type revolute, parent arm2_1, child arm2_2, origin xyz=-0.09015 -0.062 0.0 rpy=0.1745327 0.0 0.0, axis 1 0 0, limit lower=-3.4258 upper=-0.0138 effort=147.0 velocity=3.86
- added joint j_arm2_3: type revolute, parent arm2_2, child arm2_3, origin xyz=0.09015 0.0 -0.21815, axis 0 0 1, limit lower=-2.5614 upper=2.5606 effort=147.0 velocity=6.06
- added joint j_arm2_4: type revolute, parent arm2_3, child arm2_4, origin xyz=0.045 -0.05515 -0.074, axis 0 1 0, limit lower=-2.4794 upper=0.2886 effort=147.0 velocity=6.06
- added joint j_arm2_5: type revolute, parent arm2_4, child arm2_5, origin xyz=-0.015 0.05515 -0.095, axis 0 0 1, limit lower=-2.5394 upper=2.5546 effort=55.0 velocity=11.72
- added joint j_arm2_6: type revolute, parent arm2_5, child arm2_6, origin xyz=0.0 -0.049 -0.156, axis 0 1 0, limit lower=-1.5154 upper=1.5156 effort=55.0 velocity=11.72
- added joint j_arm2_8: type fixed, parent arm2_6, child ball2, origin xyz=0. 0.05 -0.105 rpy=0. 0. 0.
- added joint j_ball1_fixed: type fixed, parent ball1, child arm1_8
- added joint j_ball1_tip: type fixed, parent ball1, child ball1_tip, origin xyz=0 0 -0.07 rpy=0 0 0
- added joint j_ball2_fixed: type fixed, parent ball2, child arm2_8
- added joint j_ball2_tip: type fixed, parent ball2, child ball2_tip, origin xyz=0 0 -0.07 rpy=0 0 0
- added joint neck_base: type fixed, parent torso_2, child neck_1, origin xyz=0.0030637045 0.0061607221 0.158 rpy=0 0 0, axis 0 0 1
- added joint torso_yaw: type revolute, parent pelvis, child torso_2, origin xyz=0.2 0.0 0.256, axis 0 0 1, limit lower=-2.618 upper=2.618 effort=147 velocity=5.7
- added joint velodyne_joint: type revolute, parent neck_1, child velodyne_motor, origin xyz=0.0822724 0 0.242 rpy=0 0 0, axis 0 -1 0, limit lower=-1.1 upper=1.1 effort=35 velocity=5.7

File: centauro_urdf/urdf/config/centauro_virtual_frame.urdf.xacro (robot description, xacro)
@@ -6,5 +6,5 @@
     <!-- *************************************-->
     <xacro:property name="ADD_LEGS" value="true" />
-    <xacro:property name="ADD_UPPER_BODY" value="false" />
+    <xacro:property name="ADD_UPPER_BODY" value="true" />
     <xacro:property name="ADD_BALL_END_EFFECTOR" value="true" />
     <xacro:property name="ADD_FLOATING_BASE" value="true" />
