Commit message: upd generated

File: centauro_urdf/urdf/centauro_capsule.urdf (robot description, URDF)
Before this commit: robot centauro, 98 links, 97 joints
Links:
- link T265_camera_pose_frame: geometry collision cylinder length=0.102252855789 radius=0.0142751; collision sphere radius=0.0142751
- link ankle1_1: geometry collision cylinder length=0.0492563156661 radius=0.0792379; collision sphere radius=0.0792379
- link ankle1_2: geometry collision cylinder length=0.0478840512856 radius=0.0781037; collision sphere radius=0.0781037
- link ankle1_3: geometry collision cylinder length=0.0492563156661 radius=0.0792379; collision sphere radius=0.0792379
- link ankle1_4: geometry collision cylinder length=0.0478840512856 radius=0.0781037; collision sphere radius=0.0781037
- link ankle2_1: geometry collision cylinder length=0.0737026312964 radius=0.0813545; collision sphere radius=0.0813545
- link ankle2_2: geometry collision cylinder length=0.0737026312964 radius=0.0813545; collision sphere radius=0.0813545
- link ankle2_3: geometry collision cylinder length=0.0737026312964 radius=0.0813545; collision sphere radius=0.0813545
- link ankle2_4: geometry collision cylinder length=0.0737026312964 radius=0.0813545; collision sphere radius=0.0813545
- link arm1_1: geometry collision cylinder length=0.0373976849456 radius=0.0698859; collision sphere radius=0.0698859
- link arm1_2: geometry collision cylinder length=0.127992699814 radius=0.0700645; collision sphere radius=0.0700645
- link arm1_3: geometry collision cylinder length=0.0608225264434 radius=0.0896121; collision sphere radius=0.0896121
- link arm1_4: geometry collision cylinder length=0.0871341857294 radius=0.0600429; collision sphere radius=0.0600429
- link arm1_5: geometry collision cylinder length=0.084347397477 radius=0.0804108; collision sphere radius=0.0804108
- link arm1_6: geometry collision cylinder length=0.114251418714 radius=0.0583263; collision sphere radius=0.0583263
- link arm1_7: geometry collision cylinder length=0.00916730749359 radius=0.0207073; collision sphere radius=0.0207073
- link arm1_8: mass 0 -> 0.0
- link arm2_1: geometry collision cylinder length=0.0373976849456 radius=0.0698859; collision sphere radius=0.0698859
- link arm2_2: geometry collision cylinder length=0.127992699814 radius=0.0700645; collision sphere radius=0.0700645
- link arm2_3: geometry collision cylinder length=0.0608225264434 radius=0.0896121; collision sphere radius=0.0896121
- link arm2_4: geometry collision cylinder length=0.0871341857294 radius=0.0600429; collision sphere radius=0.0600429
- link arm2_5: geometry collision cylinder length=0.084347397477 radius=0.0804108; collision sphere radius=0.0804108
- link arm2_6: geometry collision cylinder length=0.114251418714 radius=0.0583263; collision sphere radius=0.0583263
- link arm2_7: geometry collision cylinder length=0.00916730749359 radius=0.0207073; collision sphere radius=0.0207073
- link arm2_8: mass 0 -> 0.0
- link ball1: geometry collision cylinder length=9.94007683594e-05 radius=0.0709883; collision sphere radius=0.0709883
- link ball2: geometry collision cylinder length=9.94007683594e-05 radius=0.0709883; collision sphere radius=0.0709883
- link d435_head_motor: geometry collision cylinder length=0.121344235484 radius=0.0261699; collision sphere radius=0.0261699
- link hip1_1: geometry collision cylinder length=0.030695458899 radius=0.0747223; collision sphere radius=0.0747223
- link hip1_2: geometry collision cylinder length=0.030695458899 radius=0.0747223; collision sphere radius=0.0747223
- link hip1_3: geometry collision cylinder length=0.030695458899 radius=0.0747223; collision sphere radius=0.0747223
- link hip1_4: geometry collision cylinder length=0.030695458899 radius=0.0747223; collision sphere radius=0.0747223
- link hip2_1: geometry collision cylinder length=0.291980452173 radius=0.0808941; collision sphere radius=0.0808941
- link hip2_2: geometry collision cylinder length=0.291980452173 radius=0.0808941; collision sphere radius=0.0808941
- link hip2_3: geometry collision cylinder length=0.291980452173 radius=0.0808941; collision sphere radius=0.0808941
- link hip2_4: geometry collision cylinder length=0.291980452173 radius=0.0808941; collision sphere radius=0.0808941
- link knee_1: geometry collision cylinder length=0.192750224606 radius=0.0664305; collision sphere radius=0.0664305
- link knee_2: geometry collision cylinder length=0.192750224606 radius=0.0664305; collision sphere radius=0.0664305
- link knee_3: geometry collision cylinder length=0.192750224606 radius=0.0664305; collision sphere radius=0.0664305
- link knee_4: geometry collision cylinder length=0.192750224606 radius=0.0664305; collision sphere radius=0.0664305
- link neck_1: geometry collision cylinder length=0.164540980255 radius=0.100414; collision sphere radius=0.100414
- link pelvis: geometry collision cylinder length=0.385941397914 radius=0.213204; collision sphere radius=0.213204
- link torso_2: geometry collision cylinder length=0.0954367599085 radius=0.158224; collision sphere radius=0.158224
- link velodyne_calib_base_link: geometry collision cylinder length=0.0717 radius=0.0516; collision sphere radius=0.0516
- link velodyne_motor: geometry collision cylinder length=0.0324631121345 radius=0.0544637; collision sphere radius=0.0544637
- link wheel_1: geometry collision cylinder length=0.11 radius=0.078; collision sphere radius=0.078
- link wheel_2: geometry collision cylinder length=0.11 radius=0.078; collision sphere radius=0.078
- link wheel_3: geometry collision cylinder length=0.11 radius=0.078; collision sphere radius=0.078
- link wheel_4: geometry collision cylinder length=0.11 radius=0.078; collision sphere radius=0.078
Joints:
- joint D435_head_camera_accel_joint: origin xyz=-0.00174 0.00552 0.0176 rpy=0 0 0 -> xyz=-0.00174 0.00552 0.0176 rpy=0.0 0.0 0.0
- joint D435_head_camera_accel_optical_joint: origin xyz=0 0 0 rpy=-1.57079632679 0 -1.57079632679 -> xyz=0.0 0.0 0.0 rpy=-1.57079632679 0.0 -1.57079632679
- joint D435_head_camera_color_joint: origin xyz=0 0.015 0 rpy=0 0 0 -> xyz=0.0 0.015 0.0 rpy=0.0 0.0 0.0
- joint D435_head_camera_color_optical_joint: origin xyz=0 0 0 rpy=-1.57079632679 0 -1.57079632679 -> xyz=0.0 0.0 0.0 rpy=-1.57079632679 0.0 -1.57079632679
- joint D435_head_camera_depth_joint: origin xyz=0 0 0 rpy=0 0 0 -> xyz=0.0 0.0 0.0 rpy=0.0 0.0 0.0
- joint D435_head_camera_depth_optical_joint: origin xyz=0 0 0 rpy=-1.57079632679 0 -1.57079632679 -> xyz=0.0 0.0 0.0 rpy=-1.57079632679 0.0 -1.57079632679
- joint D435_head_camera_gyro_joint: origin xyz=-0.00174 0.00552 0.0176 rpy=0 0 0 -> xyz=-0.00174 0.00552 0.0176 rpy=0.0 0.0 0.0
- joint D435_head_camera_gyro_optical_joint: origin xyz=0 0 0 rpy=-1.57079632679 0 -1.57079632679 -> xyz=0.0 0.0 0.0 rpy=-1.57079632679 0.0 -1.57079632679
- joint D435_head_camera_joint: origin xyz=0.03015 0 -0.0125 rpy=0 0 0 -> xyz=0.03015 0.0 -0.0125 rpy=0.0 0.0 0.0
- joint D435_head_camera_left_ir_joint: origin xyz=0 0.0 0 rpy=0 0 0 -> xyz=0.0 0.0 0.0 rpy=0.0 0.0 0.0
- joint D435_head_camera_left_ir_optical_joint: origin xyz=0 0 0 rpy=-1.57079632679 0 -1.57079632679 -> xyz=0.0 0.0 0.0 rpy=-1.57079632679 0.0 -1.57079632679
- joint D435_head_camera_link_joint: origin xyz=0 0.0175 0.0125 rpy=0 0 0 -> xyz=0.0 0.0175 0.0125 rpy=0.0 0.0 0.0
- joint D435_head_camera_right_ir_joint: origin xyz=0 -0.05 0 rpy=0 0 0 -> xyz=0.0 -0.05 0.0 rpy=0.0 0.0 0.0
- joint D435_head_camera_right_ir_optical_joint: origin xyz=0 0 0 rpy=-1.57079632679 0 -1.57079632679 -> xyz=0.0 0.0 0.0 rpy=-1.57079632679 0.0 -1.57079632679
- joint D435i_camera_accel_joint: origin xyz=-0.00174 0.00552 0.0176 rpy=0 0 0 -> xyz=-0.00174 0.00552 0.0176 rpy=0.0 0.0 0.0
- joint D435i_camera_accel_optical_joint: origin xyz=0 0 0 rpy=-1.57079632679 0 -1.57079632679 -> xyz=0.0 0.0 0.0 rpy=-1.57079632679 0.0 -1.57079632679
- joint D435i_camera_color_joint: origin xyz=0 0.015 0 rpy=0 0 0 -> xyz=0.0 0.015 0.0 rpy=0.0 0.0 0.0
- joint D435i_camera_color_optical_joint: origin xyz=0 0 0 rpy=-1.57079632679 0 -1.57079632679 -> xyz=0.0 0.0 0.0 rpy=-1.57079632679 0.0 -1.57079632679
- joint D435i_camera_depth_joint: origin xyz=0 0 0 rpy=0 0 0 -> xyz=0.0 0.0 0.0 rpy=0.0 0.0 0.0
- joint D435i_camera_depth_optical_joint: origin xyz=0 0 0 rpy=-1.57079632679 0 -1.57079632679 -> xyz=0.0 0.0 0.0 rpy=-1.57079632679 0.0 -1.57079632679
- joint D435i_camera_gyro_joint: origin xyz=-0.00174 0.00552 0.0176 rpy=0 0 0 -> xyz=-0.00174 0.00552 0.0176 rpy=0.0 0.0 0.0
- joint D435i_camera_gyro_optical_joint: origin xyz=0 0 0 rpy=-1.57079632679 0 -1.57079632679 -> xyz=0.0 0.0 0.0 rpy=-1.57079632679 0.0 -1.57079632679
- joint D435i_camera_joint: origin xyz=0.27187 0 0.0215997 rpy=0 0.5251508 0 -> xyz=0.27187 0.0 0.0215997 rpy=0.0 0.5251508 0.0
- joint D435i_camera_left_ir_joint: origin xyz=0 0.0 0 rpy=0 0 0 -> xyz=0.0 0.0 0.0 rpy=0.0 0.0 0.0
- joint D435i_camera_left_ir_optical_joint: origin xyz=0 0 0 rpy=-1.57079632679 0 -1.57079632679 -> xyz=0.0 0.0 0.0 rpy=-1.57079632679 0.0 -1.57079632679
- joint D435i_camera_link_joint: origin xyz=0 0.0175 0.0125 rpy=0 0 0 -> xyz=0.0 0.0175 0.0125 rpy=0.0 0.0 0.0
- joint D435i_camera_right_ir_joint: origin xyz=0 -0.05 0 rpy=0 0 0 -> xyz=0.0 -0.05 0.0 rpy=0.0 0.0 0.0
- joint D435i_camera_right_ir_optical_joint: origin xyz=0 0 0 rpy=-1.57079632679 0 -1.57079632679 -> xyz=0.0 0.0 0.0 rpy=-1.57079632679 0.0 -1.57079632679
- joint T265_camera_accel_joint: origin xyz=-0.0311 0 0.00655 rpy=0 3.14159265359 0 -> xyz=-0.0311 0.0 0.00655 rpy=0.0 3.14159265359 0.0
- joint T265_camera_accel_optical_joint: origin xyz=-0.0311 0 0.00655 rpy=0 3.14159265359 0 -> xyz=-0.0311 0.0 0.00655 rpy=0.0 3.14159265359 0.0
- joint T265_camera_fisheye1_optical_joint: origin xyz=0 0 0 rpy=-1.57079632679 0 -1.57079632679 -> xyz=0.0 0.0 0.0 rpy=-1.57079632679 0.0 -1.57079632679
- joint T265_camera_fisheye1_rgb_joint: origin xyz=-0.0411 0.0 0.0 rpy=0 1.57079632679 1.57079632679 -> xyz=-0.0411 0.0 0.0 rpy=0.0 1.57079632679 1.57079632679
- joint T265_camera_fisheye2_optical_joint: origin xyz=0 0 0 rpy=-1.57079632679 0 -1.57079632679 -> xyz=0.0 0.0 0.0 rpy=-1.57079632679 0.0 -1.57079632679
- joint T265_camera_fisheye2_rgb_joint: origin xyz=0.0229 0.0 0.0 rpy=0 1.57079632679 1.57079632679 -> xyz=0.0229 0.0 0.0 rpy=0.0 1.57079632679 1.57079632679
- joint T265_camera_gyro_joint: origin xyz=-0.0311 0 0.00655 rpy=0 3.14159265359 0 -> xyz=-0.0311 0.0 0.00655 rpy=0.0 3.14159265359 0.0
- joint T265_camera_gyro_optical_joint: origin xyz=0 0 0 rpy=0 0 0 -> xyz=0.0 0.0 0.0 rpy=0.0 0.0 0.0
- joint T265_camera_link_joint: origin xyz=0 0 0 rpy=1.57079632679 0 -1.57079632679 -> xyz=0.0 0.0 0.0 rpy=1.57079632679 0.0 -1.57079632679
- joint T265_camera_pose_joint: origin xyz=0.29245 0.00775 0.063 rpy=0 0 0 -> xyz=0.29245 0.00775 0.063 rpy=0.0 0.0 0.0
- joint ankle_pitch_1: axis 0 0 -1 -> 0.0 0.0 -1.0; limit lower=-2.4056 upper=2.3184 effort=147 velocity=8.1 -> lower=-2.4056 upper=2.3184 effort=147.0 velocity=8.1
- joint ankle_pitch_2: axis 0 0 1 -> 0.0 0.0 1.0; limit lower=-2.3266 upper=2.3914 effort=147 velocity=8.1 -> lower=-2.3266 upper=2.3914 effort=147.0 velocity=8.1
- joint ankle_pitch_3: axis 0 0 -1 -> 0.0 0.0 -1.0; limit lower=-2.4696 upper=2.4464 effort=147 velocity=8.1 -> lower=-2.4696 upper=2.4464 effort=147.0 velocity=8.1
- joint ankle_pitch_4: axis 0 0 1 -> 0.0 0.0 1.0; limit lower=-2.3426 upper=2.3934 effort=147 velocity=8.1 -> lower=-2.3426 upper=2.3934 effort=147.0 velocity=8.1
- joint ankle_yaw_1: axis 0 0 -1 -> 0.0 0.0 -1.0; limit lower=-2.5626 upper=2.5384 effort=35 velocity=20.0 -> lower=-2.5626 upper=2.5384 effort=35.0 velocity=20.0
- joint ankle_yaw_2: axis 0 0 -1 -> 0.0 0.0 -1.0; limit lower=-2.5546 upper=2.5484 effort=35 velocity=20.0 -> lower=-2.5546 upper=2.5484 effort=35.0 velocity=20.0
- joint ankle_yaw_3: axis 0 0 -1 -> 0.0 0.0 -1.0; limit lower=-2.5606 upper=2.5454 effort=35 velocity=20.0 -> lower=-2.5606 upper=2.5454 effort=35.0 velocity=20.0
- joint ankle_yaw_4: axis 0 0 -1 -> 0.0 0.0 -1.0; limit lower=-2.6046 upper=2.5514 effort=35 velocity=20.0 -> lower=-2.6046 upper=2.5514 effort=35.0 velocity=20.0
- joint base_joint: origin xyz=0 0 0 rpy=0 0 0 -> xyz=0.0 0.0 0.0 rpy=0.0 0.0 0.0
- joint contact_joint_1: origin xyz=0 0 -0.176 rpy=0 0 0 -> xyz=0.0 0.0 -0.176 rpy=0.0 0.0 0.0
- joint contact_joint_2: origin xyz=0 0 -0.176 rpy=0 0 0 -> xyz=0.0 0.0 -0.176 rpy=0.0 0.0 0.0
- joint contact_joint_3: origin xyz=0 0 -0.176 rpy=0 0 0 -> xyz=0.0 0.0 -0.176 rpy=0.0 0.0 0.0
- joint contact_joint_4: origin xyz=0 0 -0.176 rpy=0 0 0 -> xyz=0.0 0.0 -0.176 rpy=0.0 0.0 0.0
- joint d435_head_joint: axis 0 1 0 -> 0.0 1.0 0.0; limit lower=-1.1 upper=1.1 effort=35 velocity=5.7 -> lower=-1.1 upper=1.1 effort=35.0 velocity=5.7; origin xyz=0.06 0 0.1375 rpy=0 0 0 -> xyz=0.06 0.0 0.1375 rpy=0.0 0.0 0.0
- joint hip_pitch_1: axis 0 0 -1 -> 0.0 0.0 -1.0; limit lower=-2.0226 upper=2.02748 effort=304 velocity=8.8 -> lower=-2.0226 upper=2.02748 effort=304.0 velocity=8.8
- joint hip_pitch_2: axis 0 0 1 -> 0.0 0.0 1.0; limit lower=-2.0156 upper=2.0354 effort=304 velocity=8.8 -> lower=-2.0156 upper=2.0354 effort=304.0 velocity=8.8
- joint hip_pitch_3: axis 0 0 -1 -> 0.0 0.0 -1.0; limit lower=-2.0126 upper=2.0384 effort=304 velocity=8.8 -> lower=-2.0126 upper=2.0384 effort=304.0 velocity=8.8
- joint hip_pitch_4: axis 0 0 1 -> 0.0 0.0 1.0; limit lower=-2.0326 upper=2.0524 effort=304 velocity=8.8 -> lower=-2.0326 upper=2.0524 effort=304.0 velocity=8.8
- joint hip_yaw_1: axis 0 0 -1 -> 0.0 0.0 -1.0; limit lower=-2.03 upper=2.51 effort=304 velocity=8.8 -> lower=-2.03 upper=2.51 effort=304.0 velocity=8.8
- joint hip_yaw_2: axis 0 0 -1 -> 0.0 0.0 -1.0; limit lower=-2.51 upper=2.03 effort=304 velocity=8.8 -> lower=-2.51 upper=2.03 effort=304.0 velocity=8.8
- joint hip_yaw_3: axis 0 0 -1 -> 0.0 0.0 -1.0; limit lower=-2.51 upper=2.03 effort=304 velocity=8.8 -> lower=-2.51 upper=2.03 effort=304.0 velocity=8.8
- joint hip_yaw_4: axis 0 0 -1 -> 0.0 0.0 -1.0; limit lower=-2.03 upper=2.51 effort=304 velocity=8.8 -> lower=-2.03 upper=2.51 effort=304.0 velocity=8.8
- joint j_arm1_1: axis 0 1 0 -> 0.0 1.0 0.0
- joint j_arm1_2: axis 1 0 0 -> 1.0 0.0 0.0
- joint j_arm1_3: axis 0 0 1 -> 0.0 0.0 1.0; origin xyz=0.09015 0.0 -0.21815 -> xyz=0.09015 0.0 -0.21815 rpy=0 0 0
- joint j_arm1_4: axis 0 1 0 -> 0.0 1.0 0.0; origin xyz=0.045 0.05515 -0.074 -> xyz=0.045 0.05515 -0.074 rpy=0 0 0
- joint j_arm1_5: axis 0 0 1 -> 0.0 0.0 1.0; origin xyz=-0.015 -0.05515 -0.095 -> xyz=-0.015 -0.05515 -0.095 rpy=0 0 0
- joint j_arm1_6: axis 0 1 0 -> 0.0 1.0 0.0; origin xyz=0.0 0.049 -0.156 -> xyz=0.0 0.049 -0.156 rpy=0 0 0
- joint j_arm1_7: axis 0 0 1 -> 0.0 0.0 1.0; origin xyz=0.0 -0.049 -0.174 -> xyz=0.0 -0.049 -0.174 rpy=0 0 0
- joint j_arm1_8: origin xyz=0. 0. 0. rpy=0. 0. 0. -> xyz=0.0 0.0 0.0 rpy=0.0 0.0 0.0
- joint j_arm2_1: axis 0 1 0 -> 0.0 1.0 0.0
- joint j_arm2_2: axis 1 0 0 -> 1.0 0.0 0.0
- joint j_arm2_3: axis 0 0 1 -> 0.0 0.0 1.0; origin xyz=0.09015 0.0 -0.21815 -> xyz=0.09015 0.0 -0.21815 rpy=0 0 0
- joint j_arm2_4: axis 0 1 0 -> 0.0 1.0 0.0; origin xyz=0.045 -0.05515 -0.074 -> xyz=0.045 -0.05515 -0.074 rpy=0 0 0
- joint j_arm2_5: axis 0 0 1 -> 0.0 0.0 1.0; origin xyz=-0.015 0.05515 -0.095 -> xyz=-0.015 0.05515 -0.095 rpy=0 0 0
- joint j_arm2_6: axis 0 1 0 -> 0.0 1.0 0.0; origin xyz=0.0 -0.049 -0.156 -> xyz=0.0 -0.049 -0.156 rpy=0 0 0
- joint j_arm2_7: axis 0 0 1 -> 0.0 0.0 1.0; origin xyz=0.0 0.049 -0.174 -> xyz=0.0 0.049 -0.174 rpy=0 0 0
- joint j_arm2_8: origin xyz=0. 0. 0. rpy=0. 0. 0. -> xyz=0.0 0.0 0.0 rpy=0.0 0.0 0.0
- joint j_ball1_tip: origin xyz=0 0 -0.07 rpy=0 0 0 -> xyz=0.0 0.0 -0.07 rpy=0.0 0.0 0.0
- joint j_ball2_tip: origin xyz=0 0 -0.07 rpy=0 0 0 -> xyz=0.0 0.0 -0.07 rpy=0.0 0.0 0.0
- joint j_ft_1: axis 0 0 1 -> 0.0 0.0 1.0; limit lower=0.0 upper=0.0 effort=0 velocity=0 -> lower=0.0 upper=0.0 effort=0.0 velocity=0.0
- joint j_ft_2: axis 0 0 1 -> 0.0 0.0 1.0; limit lower=0.0 upper=0.0 effort=0 velocity=0 -> lower=0.0 upper=0.0 effort=0.0 velocity=0.0
- joint j_wheel_1: axis 0 0 -1 -> 0.0 0.0 -1.0; limit effort=35 velocity=20.0 -> lower=0 upper=0 effort=35.0 velocity=20.0
- joint j_wheel_2: axis 0 0 1 -> 0.0 0.0 1.0; limit effort=35 velocity=20.0 -> lower=0 upper=0 effort=35.0 velocity=20.0
- joint j_wheel_3: axis 0 0 -1 -> 0.0 0.0 -1.0; limit effort=35 velocity=20.0 -> lower=0 upper=0 effort=35.0 velocity=20.0
- joint j_wheel_4: axis 0 0 1 -> 0.0 0.0 1.0; limit effort=35 velocity=20.0 -> lower=0 upper=0 effort=35.0 velocity=20.0
- joint knee_pitch_1: axis 0 0 -1 -> 0.0 0.0 -1.0; limit lower=-2.4056 upper=2.3994 effort=304 velocity=8.8 -> lower=-2.4056 upper=2.3994 effort=304.0 velocity=8.8
- joint knee_pitch_2: axis 0 0 1 -> 0.0 0.0 1.0; limit lower=-2.4006 upper=2.4034 effort=304 velocity=8.8 -> lower=-2.4006 upper=2.4034 effort=304.0 velocity=8.8
- joint knee_pitch_3: axis 0 0 -1 -> 0.0 0.0 -1.0; limit lower=-2.4056 upper=2.4064 effort=304 velocity=8.8 -> lower=-2.4056 upper=2.4064 effort=304.0 velocity=8.8
- joint knee_pitch_4: axis 0 0 1 -> 0.0 0.0 1.0; limit lower=-2.4176 upper=2.3884 effort=304 velocity=8.8 -> lower=-2.4176 upper=2.3884 effort=304.0 velocity=8.8
- joint neck_base: axis 0 0 1 -> 0.0 0.0 1.0; origin xyz=0.0030637045 0.0061607221 0.224 rpy=0 0 0 -> xyz=0.0030637045 0.0061607221 0.224 rpy=0.0 0.0 0.0
- joint torso_yaw: axis 0 0 1 -> 0.0 0.0 1.0; limit lower=-2.618 upper=2.618 effort=147 velocity=5.7 -> lower=-2.618 upper=2.618 effort=147.0 velocity=5.7; origin xyz=0.2 0.0 0.256 -> xyz=0.2 0.0 0.256 rpy=0 0 0
- joint velodyne_calib_base_mount_joint: origin xyz=0 0 0 rpy=0 0 0 -> xyz=0.0 0.0 0.0 rpy=0.0 0.0 0.0
- joint velodyne_calib_base_scan_joint: origin xyz=0 0 0.0377 rpy=0 0 0 -> xyz=0.0 0.0 0.0377 rpy=0.0 0.0 0.0
- joint velodyne_joint: axis 0 1 0 -> 0.0 1.0 0.0; limit lower=-1.1 upper=1.1 effort=35 velocity=5.7 -> lower=-1.1 upper=1.1 effort=35.0 velocity=5.7; origin xyz=0.0825 0 0.243 rpy=0 0 0 -> xyz=0.0825 0.0 0.243 rpy=0.0 0.0 0.0

File: centauro_urdf/urdf/centauro_virtual_frame.urdf (robot description, URDF)
Before this commit: robot centauro, 90 links, 89 joints
Links:
- removed link D435i_camera_accel_frame
- removed link D435i_camera_accel_optical_frame
- removed link D435i_camera_bottom_screw_frame
- removed link D435i_camera_color_frame
- removed link D435i_camera_color_optical_frame
- removed link D435i_camera_depth_frame
- removed link D435i_camera_depth_optical_frame
- removed link D435i_camera_gyro_frame
- removed link D435i_camera_gyro_optical_frame
- removed link D435i_camera_left_ir_frame
- removed link D435i_camera_left_ir_optical_frame
- removed link D435i_camera_link
- removed link D435i_camera_right_ir_frame
- removed link D435i_camera_right_ir_optical_frame
- removed link T265_camera_accel_frame
- removed link T265_camera_accel_optical_frame
- removed link T265_camera_fisheye1_optical_frame
- removed link T265_camera_fisheye1_rgb_frame
- removed link T265_camera_fisheye2_optical_frame
- removed link T265_camera_fisheye2_rgb_frame
- removed link T265_camera_gyro_frame
- removed link T265_camera_gyro_optical_frame
- removed link T265_camera_link
- removed link T265_camera_pose_frame
- removed link neck_2
- removed link neck_3
- removed link velodyne_calib
- removed link velodyne_calib_base_link
- added link velodyne_motor, mass 0.33878686; collision mesh filename=package://centauro_urdf/meshes/simple/lidar_mesh.stl scale=0.001 0.001 0.001; visual mesh filename=package://centauro_urdf/meshes/lidar_mesh.stl scale=0.001 0.001 0.001
- link neck_1: geometry collision mesh filename=package://centauro_urdf/meshes/simple/head-base_mesh.stl scale=0.001 0.001 0.001; visual mesh filename=package://centauro_urdf/meshes/head-base_mesh.stl scale=0.001 0.001 0.001
- link torso_2: geometry collision mesh filename=package://centauro_urdf/meshes/simple/link1_no_head.stl scale=0.001 0.001 0.001; visual mesh filename=package://centauro_urdf/meshes/link1_no_head.stl scale=0.001 0.001 0.001
Joints:
- removed joint D435i_camera_accel_joint
- removed joint D435i_camera_accel_optical_joint
- removed joint D435i_camera_color_joint
- removed joint D435i_camera_color_optical_joint
- removed joint D435i_camera_depth_joint
- removed joint D435i_camera_depth_optical_joint
- removed joint D435i_camera_gyro_joint
- removed joint D435i_camera_gyro_optical_joint
- removed joint D435i_camera_joint
- removed joint D435i_camera_left_ir_joint
- removed joint D435i_camera_left_ir_optical_joint
- removed joint D435i_camera_link_joint
- removed joint D435i_camera_right_ir_joint
- removed joint D435i_camera_right_ir_optical_joint
- removed joint T265_camera_accel_joint
- removed joint T265_camera_accel_optical_joint
- removed joint T265_camera_fisheye1_optical_joint
- removed joint T265_camera_fisheye1_rgb_joint
- removed joint T265_camera_fisheye2_optical_joint
- removed joint T265_camera_fisheye2_rgb_joint
- removed joint T265_camera_gyro_joint
- removed joint T265_camera_gyro_optical_joint
- removed joint T265_camera_link_joint
- removed joint T265_camera_pose_joint
- removed joint neck_pitch
- removed joint neck_velodyne
- removed joint neck_yaw
- removed joint velodyne_calib_base_mount_joint
- removed joint velodyne_calib_base_scan_joint
- added joint neck_base: type fixed, parent torso_2, child neck_1, origin xyz=0.0030637045 0.0061607221 0.224 rpy=0 0 0, axis 0 0 1
- added joint velodyne_joint: type revolute, parent neck_1, child velodyne_motor, origin xyz=0.0825 0 0.243 rpy=0 0 0, axis 0 1 0, limit lower=-1.1 upper=1.1 effort=35 velocity=5.7
