Commit message: regenerate urdf/srdf (with all cameras true in xacro config file)

File: centauro_urdf/urdf/centauro_capsule.urdf (robot description, URDF)
Before this commit: robot centauro, 94 links, 93 joints
Links:
- link ankle1_2: geometry collision cylinder length=0.047884051265172006 radius=0.0781037; collision sphere radius=0.0781037
- link ankle1_4: geometry collision cylinder length=0.047884051265172006 radius=0.0781037; collision sphere radius=0.0781037
- link arm1_5: geometry collision cylinder length=0.08434739747702548 radius=0.0804108; collision sphere radius=0.0804108
- link arm2_5: geometry collision cylinder length=0.08434739747702548 radius=0.0804108; collision sphere radius=0.0804108
- link knee_1: geometry collision cylinder length=0.19275022460612404 radius=0.0664305; collision sphere radius=0.0664305
- link knee_2: geometry collision cylinder length=0.19275022460612404 radius=0.0664305; collision sphere radius=0.0664305
- link knee_3: geometry collision cylinder length=0.19275022460612404 radius=0.0664305; collision sphere radius=0.0664305
- link knee_4: geometry collision cylinder length=0.19275022460612404 radius=0.0664305; collision sphere radius=0.0664305
Joints:
- joint D435i_camera_joint: origin xyz=0.27187 0.0 0.0215997 rpy=0.0 0.5251508 0.0 -> xyz=0.272 0.0 0.084 rpy=0.0 0.54 0.0
- joint velodyne_calib_base_mount_joint: origin xyz=0.0 0.0 0.0 rpy=0.0 0.0 0.0 -> xyz=-0.01 0.02 0.06 rpy=0.025 0.019 0.0

File: centauro_urdf/urdf/centauro_virtual_frame.urdf (robot description, URDF)
Before this commit: robot centauro, 66 links, 65 joints
Joints:
- joint D435i_camera_joint: origin xyz=0.27187 0 0.0215997 rpy=0 0.5251508 0 -> xyz=0.272 0 0.084 rpy=0 0.54 0
- joint D435i_camera_link_joint: origin xyz=0 0.0175 0.0125 rpy=0 0 0 -> xyz=0.053 0.0 -0.035 rpy=0 0.0050 -0.008
- joint hip_yaw_1: origin xyz=0.25 0.125 -0.0566 rpy=0.0 0.0 0.0 -> xyz=0.25 0.125 -0.056600000000000004 rpy=0.0 0.0 0.0
- joint hip_yaw_2: origin xyz=0.25 -0.125 -0.0566 rpy=0.0 0.0 0.0 -> xyz=0.25 -0.125 -0.056600000000000004 rpy=0.0 0.0 0.0
- joint hip_yaw_3: origin xyz=-0.25 0.125 -0.0566 rpy=0.0 0.0 0.0 -> xyz=-0.25 0.125 -0.056600000000000004 rpy=0.0 0.0 0.0
- joint hip_yaw_4: origin xyz=-0.25 -0.125 -0.0566 rpy=0.0 0.0 0.0 -> xyz=-0.25 -0.125 -0.056600000000000004 rpy=0.0 0.0 0.0
- joint j_wheel_1: origin xyz=0.0 -0.0 -0.09835 rpy=1.57079632679 0.0 0.0 -> xyz=0.0 -0.0 -0.09834999999999999 rpy=1.57079632679 0.0 0.0
- joint j_wheel_2: origin xyz=0.0 0.0 -0.09835 rpy=1.57079632679 0.0 0.0 -> xyz=0.0 0.0 -0.09834999999999999 rpy=1.57079632679 0.0 0.0
- joint j_wheel_3: origin xyz=0.0 -0.0 -0.09835 rpy=1.57079632679 0.0 0.0 -> xyz=0.0 -0.0 -0.09834999999999999 rpy=1.57079632679 0.0 0.0
- joint j_wheel_4: origin xyz=0.0 0.0 -0.09835 rpy=1.57079632679 0.0 0.0 -> xyz=0.0 0.0 -0.09834999999999999 rpy=1.57079632679 0.0 0.0
- joint velodyne_calib_base_mount_joint: origin xyz=0 0 0 rpy=0 0 0 -> xyz=-0.01 0.02 0.06 rpy=0.025 0.019 0
