Commit message: ghost-limits for dagana to work on hw

File: centauro_urdf/urdf/centauro_dagana.urdf (robot description, URDF)
Before this commit: robot centauro, 95 links, 94 joints
Joints:
- joint dagana_2_claw_joint: limit lower=0 upper=1 effort=1000 velocity=2.0 -> lower=-3 upper=3 effort=1000 velocity=10.0

Commit message: correct min max position after ecat rearrangement by tory

File: centauro_urdf/urdf/centauro_dagana.urdf (robot description, URDF)
Before this commit: robot centauro, 95 links, 94 joints
Joints:
- joint dagana_2_claw_joint: limit lower=-3 upper=3 effort=1000 velocity=10.0 -> lower=0 upper=1.3 effort=1000 velocity=10.0

Commit message: update with 10 mm correction for bottom_screw frame

File: centauro_urdf/urdf/centauro_dagana.urdf (robot description, URDF)
Before this commit: robot centauro, 95 links, 94 joints
Joints:
- joint D435_head_camera_joint: origin xyz=0.0316 0 -0.01309 rpy=0 0.349065 0 -> xyz=0.0413 0 -0.016 rpy=0 0.349065 0
