Commit message: new branch for uncommited changes on embedded pc

File: centauro_urdf/urdf/centauro.urdf (robot description, URDF)
Before this commit: robot centauro, 60 links, 59 joints
Joints:
- joint neck_velodyne: origin xyz=0.055 0.0 0.473262 rpy=0 0 -1.828 -> xyz=0.055 0 0.473262 rpy=0 0 0.015
- joint velodyne_calib_base_mount_joint: origin xyz=0.032768 -0.01 0.048219 rpy=0 1.5709 -0.316519   -> xyz=0.032768 0 0.048219 rpy=0 1.5709 0
- joint velodyne_calib_base_scan_joint: origin xyz=0 0 0.0377 rpy=0 0 0 -> xyz=0 0 0 rpy=0 0 0

Commit message: adding perception frames to generated  urdf (unfortunately also plugins..)

File: centauro_urdf/urdf/centauro.urdf (robot description, URDF)
Before this commit: robot centauro, 58 links, 57 joints
Links:
- added link D435i_camera_accel_frame
- added link D435i_camera_accel_optical_frame
- added link D435i_camera_bottom_screw_frame
- added link D435i_camera_color_frame
- added link D435i_camera_color_optical_frame
- added link D435i_camera_depth_frame
- added link D435i_camera_depth_optical_frame
- added link D435i_camera_gyro_frame
- added link D435i_camera_gyro_optical_frame
- added link D435i_camera_left_ir_frame
- added link D435i_camera_left_ir_optical_frame
- added link D435i_camera_link, mass 0.564; collision box size=0.02505 0.09 0.025; visual mesh filename=package://realsense2_description/meshes/d435.dae
- added link D435i_camera_right_ir_frame
- added link D435i_camera_right_ir_optical_frame
- added link T265_camera_accel_frame
- added link T265_camera_accel_optical_frame
- added link T265_camera_fisheye1_optical_frame
- added link T265_camera_fisheye1_rgb_frame
- added link T265_camera_fisheye2_optical_frame
- added link T265_camera_fisheye2_rgb_frame
- added link T265_camera_gyro_frame
- added link T265_camera_gyro_optical_frame
- added link T265_camera_link
- added link T265_camera_pose_frame, mass 0.068024; collision mesh filename=package://realsense_gazebo_description/meshes/t265_simplifi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 scale=0.001 0.001 0.001; visual mesh filename=package://realsense_gazebo_description/meshes/t265_full.stl scale=0.001 0.001 0.001
- added link velodyne_calib, mass 0.01; visual mesh filename=package://velodyne_description/meshes/VLP16_scan.dae
- added link velodyne_calib_base_link, mass 0.83; collision cylinder length=0.0717 radius=0.0516; visual mesh filename=package://velodyne_description/meshes/VLP16_base_1.dae
Joints:
- added joint D435i_camera_accel_joint: type fixed, parent D435i_camera_link, child D435i_camera_accel_frame, origin xyz=-0.00174 0.00552 0.0176 rpy=0 0 0
- added joint D435i_camera_accel_optical_joint: type fixed, parent D435i_camera_accel_frame, child D435i_camera_accel_optical_frame, origin xyz=0 0 0 rpy=-1.57079632679 0 -1.57079632679
- added joint D435i_camera_color_joint: type fixed, parent D435i_camera_depth_frame, child D435i_camera_color_frame, origin xyz=0 0.015 0 rpy=0 0 0
- added joint D435i_camera_color_optical_joint: type fixed, parent D435i_camera_color_frame, child D435i_camera_color_optical_frame, origin xyz=0 0 0 rpy=-1.57079632679 0 -1.57079632679
- added joint D435i_camera_depth_joint: type fixed, parent D435i_camera_link, child D435i_camera_depth_frame, origin xyz=0 0 0 rpy=0 0 0
- added joint D435i_camera_depth_optical_joint: type fixed, parent D435i_camera_depth_frame, child D435i_camera_depth_optical_frame, origin xyz=0 0 0 rpy=-1.57079632679 0 -1.57079632679
- added joint D435i_camera_gyro_joint: type fixed, parent D435i_camera_link, child D435i_camera_gyro_frame, origin xyz=-0.00174 0.00552 0.0176 rpy=0 0 0
- added joint D435i_camera_gyro_optical_joint: type fixed, parent D435i_camera_gyro_frame, child D435i_camera_gyro_optical_frame, origin xyz=0 0 0 rpy=-1.57079632679 0 -1.57079632679
- added joint D435i_camera_joint: type fixed, parent pelvis, child D435i_camera_bottom_screw_frame, origin xyz=0.219831 0 -0.0613293 rpy=0.0 0.5585052 0.0
- added joint D435i_camera_left_ir_joint: type fixed, parent D435i_camera_depth_frame, child D435i_camera_left_ir_frame, origin xyz=0 0.0 0 rpy=0 0 0
- added joint D435i_camera_left_ir_optical_joint: type fixed, parent D435i_camera_left_ir_frame, child D435i_camera_left_ir_optical_frame, origin xyz=0 0 0 rpy=-1.57079632679 0 -1.57079632679
- added joint D435i_camera_link_joint: type fixed, parent D435i_camera_bottom_screw_frame, child D435i_camera_link, origin xyz=0 0.0175 0.0125 rpy=0 0 0
- added joint D435i_camera_right_ir_joint: type fixed, parent D435i_camera_depth_frame, child D435i_camera_right_ir_frame, origin xyz=0 -0.05 0 rpy=0 0 0
- added joint D435i_camera_right_ir_optical_joint: type fixed, parent D435i_camera_right_ir_frame, child D435i_camera_right_ir_optical_frame, origin xyz=0 0 0 rpy=-1.57079632679 0 -1.57079632679
- added joint T265_camera_accel_joint: type fixed, parent T265_camera_link, child T265_camera_accel_frame, origin xyz=-0.0311 0 0.00655 rpy=0 3.14159265359 0
- added joint T265_camera_accel_optical_joint: type fixed, parent T265_camera_accel_frame, child T265_camera_accel_optical_frame, origin xyz=-0.0311 0 0.00655 rpy=0 3.14159265359 0
- added joint T265_camera_fisheye1_optical_joint: type fixed, parent T265_camera_fisheye1_rgb_frame, child T265_camera_fisheye1_optical_frame, origin xyz=0 0 0 rpy=-1.57079632679 0 -1.57079632679
- added joint T265_camera_fisheye1_rgb_joint: type fixed, parent T265_camera_link, child T265_camera_fisheye1_rgb_frame, origin xyz=-0.0411 0.0 0.0 rpy=0 1.57079632679 1.57079632679
- added joint T265_camera_fisheye2_optical_joint: type fixed, parent T265_camera_fisheye2_rgb_frame, child T265_camera_fisheye2_optical_frame, origin xyz=0 0 0 rpy=-1.57079632679 0 -1.57079632679
- added joint T265_camera_fisheye2_rgb_joint: type fixed, parent T265_camera_link, child T265_camera_fisheye2_rgb_frame, origin xyz=0.0229 0.0 0.0 rpy=0 1.57079632679 1.57079632679
- added joint T265_camera_gyro_joint: type fixed, parent T265_camera_link, child T265_camera_gyro_frame, origin xyz=-0.0311 0 0.00655 rpy=0 3.14159265359 0
- added joint T265_camera_gyro_optical_joint: type fixed, parent T265_camera_gyro_frame, child T265_camera_gyro_optical_frame, origin xyz=0 0 0 rpy=0 0 0
- added joint T265_camera_link_joint: type fixed, parent T265_camera_pose_frame, child T265_camera_link, origin xyz=0 0 0 rpy=1.57079632679 0 -1.57079632679
- added joint T265_camera_pose_joint: type fixed, parent pelvis, child T265_camera_pose_frame, origin xyz=0.252619 0.00775 -0.0206926 rpy=0.0 0.2617993 0.0
- added joint velodyne_calib_base_mount_joint: type fixed, parent neck_3, child velodyne_calib_base_link, origin xyz=0.032768 -0.01 0.048219 rpy=0 1.5709 -0.316519  
- added joint velodyne_calib_base_scan_joint: type fixed, parent velodyne_calib_base_link, child velodyne_calib, origin xyz=0 0 0.0377 rpy=0 0 0

File: centauro_urdf/urdf/centauro_virtual_frame.urdf (robot description, URDF)
Before this commit: robot centauro, 64 links, 63 joints
Links:
- added link D435i_camera_accel_frame
- added link D435i_camera_accel_optical_frame
- added link D435i_camera_bottom_screw_frame
- added link D435i_camera_color_frame
- added link D435i_camera_color_optical_frame
- added link D435i_camera_depth_frame
- added link D435i_camera_depth_optical_frame
- added link D435i_camera_gyro_frame
- added link D435i_camera_gyro_optical_frame
- added link D435i_camera_left_ir_frame
- added link D435i_camera_left_ir_optical_frame
- added link D435i_camera_link, mass 0.564; collision box size=0.02505 0.09 0.025; visual mesh filename=package://realsense2_description/meshes/d435.dae
- added link D435i_camera_right_ir_frame
- added link D435i_camera_right_ir_optical_frame
- added link T265_camera_accel_frame
- added link T265_camera_accel_optical_frame
- added link T265_camera_fisheye1_optical_frame
- added link T265_camera_fisheye1_rgb_frame
- added link T265_camera_fisheye2_optical_frame
- added link T265_camera_fisheye2_rgb_frame
- added link T265_camera_gyro_frame
- added link T265_camera_gyro_optical_frame
- added link T265_camera_link
- added link T265_camera_pose_frame, mass 0.068024; collision mesh filename=package://realsense_gazebo_description/meshes/t265_simplifi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 scale=0.001 0.001 0.001; visual mesh filename=package://realsense_gazebo_description/meshes/t265_full.stl scale=0.001 0.001 0.001
- added link velodyne_calib, mass 0.01; visual mesh filename=package://velodyne_description/meshes/VLP16_scan.dae
- added link velodyne_calib_base_link, mass 0.83; collision cylinder length=0.0717 radius=0.0516; visual mesh filename=package://velodyne_description/meshes/VLP16_base_1.dae
Joints:
- added joint D435i_camera_accel_joint: type fixed, parent D435i_camera_link, child D435i_camera_accel_frame, origin xyz=-0.00174 0.00552 0.0176 rpy=0 0 0
- added joint D435i_camera_accel_optical_joint: type fixed, parent D435i_camera_accel_frame, child D435i_camera_accel_optical_frame, origin xyz=0 0 0 rpy=-1.57079632679 0 -1.57079632679
- added joint D435i_camera_color_joint: type fixed, parent D435i_camera_depth_frame, child D435i_camera_color_frame, origin xyz=0 0.015 0 rpy=0 0 0
- added joint D435i_camera_color_optical_joint: type fixed, parent D435i_camera_color_frame, child D435i_camera_color_optical_frame, origin xyz=0 0 0 rpy=-1.57079632679 0 -1.57079632679
- added joint D435i_camera_depth_joint: type fixed, parent D435i_camera_link, child D435i_camera_depth_frame, origin xyz=0 0 0 rpy=0 0 0
- added joint D435i_camera_depth_optical_joint: type fixed, parent D435i_camera_depth_frame, child D435i_camera_depth_optical_frame, origin xyz=0 0 0 rpy=-1.57079632679 0 -1.57079632679
- added joint D435i_camera_gyro_joint: type fixed, parent D435i_camera_link, child D435i_camera_gyro_frame, origin xyz=-0.00174 0.00552 0.0176 rpy=0 0 0
- added joint D435i_camera_gyro_optical_joint: type fixed, parent D435i_camera_gyro_frame, child D435i_camera_gyro_optical_frame, origin xyz=0 0 0 rpy=-1.57079632679 0 -1.57079632679
- added joint D435i_camera_joint: type fixed, parent pelvis, child D435i_camera_bottom_screw_frame, origin xyz=0.219831 0 -0.0613293 rpy=0.0 0.5585052 0.0
- added joint D435i_camera_left_ir_joint: type fixed, parent D435i_camera_depth_frame, child D435i_camera_left_ir_frame, origin xyz=0 0.0 0 rpy=0 0 0
- added joint D435i_camera_left_ir_optical_joint: type fixed, parent D435i_camera_left_ir_frame, child D435i_camera_left_ir_optical_frame, origin xyz=0 0 0 rpy=-1.57079632679 0 -1.57079632679
- added joint D435i_camera_link_joint: type fixed, parent D435i_camera_bottom_screw_frame, child D435i_camera_link, origin xyz=0 0.0175 0.0125 rpy=0 0 0
- added joint D435i_camera_right_ir_joint: type fixed, parent D435i_camera_depth_frame, child D435i_camera_right_ir_frame, origin xyz=0 -0.05 0 rpy=0 0 0
- added joint D435i_camera_right_ir_optical_joint: type fixed, parent D435i_camera_right_ir_frame, child D435i_camera_right_ir_optical_frame, origin xyz=0 0 0 rpy=-1.57079632679 0 -1.57079632679
- added joint T265_camera_accel_joint: type fixed, parent T265_camera_link, child T265_camera_accel_frame, origin xyz=-0.0311 0 0.00655 rpy=0 3.14159265359 0
- added joint T265_camera_accel_optical_joint: type fixed, parent T265_camera_accel_frame, child T265_camera_accel_optical_frame, origin xyz=-0.0311 0 0.00655 rpy=0 3.14159265359 0
- added joint T265_camera_fisheye1_optical_joint: type fixed, parent T265_camera_fisheye1_rgb_frame, child T265_camera_fisheye1_optical_frame, origin xyz=0 0 0 rpy=-1.57079632679 0 -1.57079632679
- added joint T265_camera_fisheye1_rgb_joint: type fixed, parent T265_camera_link, child T265_camera_fisheye1_rgb_frame, origin xyz=-0.0411 0.0 0.0 rpy=0 1.57079632679 1.57079632679
- added joint T265_camera_fisheye2_optical_joint: type fixed, parent T265_camera_fisheye2_rgb_frame, child T265_camera_fisheye2_optical_frame, origin xyz=0 0 0 rpy=-1.57079632679 0 -1.57079632679
- added joint T265_camera_fisheye2_rgb_joint: type fixed, parent T265_camera_link, child T265_camera_fisheye2_rgb_frame, origin xyz=0.0229 0.0 0.0 rpy=0 1.57079632679 1.57079632679
- added joint T265_camera_gyro_joint: type fixed, parent T265_camera_link, child T265_camera_gyro_frame, origin xyz=-0.0311 0 0.00655 rpy=0 3.14159265359 0
- added joint T265_camera_gyro_optical_joint: type fixed, parent T265_camera_gyro_frame, child T265_camera_gyro_optical_frame, origin xyz=0 0 0 rpy=0 0 0
- added joint T265_camera_link_joint: type fixed, parent T265_camera_pose_frame, child T265_camera_link, origin xyz=0 0 0 rpy=1.57079632679 0 -1.57079632679
- added joint T265_camera_pose_joint: type fixed, parent pelvis, child T265_camera_pose_frame, origin xyz=0.252619 0.00775 -0.0206926 rpy=0.0 0.2617993 0.0
- added joint velodyne_calib_base_mount_joint: type fixed, parent neck_3, child velodyne_calib_base_link, origin xyz=0.032768 -0.01 0.048219 rpy=0 1.5709 -0.316519  
- added joint velodyne_calib_base_scan_joint: type fixed, parent velodyne_calib_base_link, child velodyne_calib, origin xyz=0 0 0.0377 rpy=0 0 0

Commit message: tested new head configuration on real centauro

File: centauro_urdf/urdf/centauro.urdf (robot description, URDF)
Before this commit: robot centauro, 58 links, 57 joints
Joints:
- joint d435_head_joint: axis 0 1 0 -> 0 -1 0
- joint velodyne_joint: axis 0 1 0 -> 0 -1 0

Commit message: update generated files

File: centauro_urdf/urdf/centauro.urdf (robot description, URDF)
Before this commit: robot centauro, 98 links, 97 joints
Joints:
- joint d435_head_joint: axis 0 1 0 -> 0 -1 0
- joint neck_base: origin xyz=0.0030637045 0.0061607221 0.224 rpy=0 0 0 -> xyz=0.0030637045 0.0061607221 0.158 rpy=0 0 0
- joint velodyne_joint: axis 0 1 0 -> 0 -1 0; origin xyz=0.0825 0 0.243 rpy=0 0 0 -> xyz=0.0822724 0 0.242 rpy=0 0 0

File: centauro_urdf/urdf/centauro_capsule.urdf (robot description, URDF)
Before this commit: robot centauro, 98 links, 97 joints
Joints:
- joint d435_head_joint: axis 0.0 1.0 0.0 -> 0.0 -1.0 0.0
- joint neck_base: origin xyz=0.0030637045 0.0061607221 0.224 rpy=0.0 0.0 0.0 -> xyz=0.0030637045 0.0061607221 0.158 rpy=0.0 0.0 0.0
- joint velodyne_joint: axis 0.0 1.0 0.0 -> 0.0 -1.0 0.0; origin xyz=0.0825 0.0 0.243 rpy=0.0 0.0 0.0 -> xyz=0.0822724 0.0 0.242 rpy=0.0 0.0 0.0

File: centauro_urdf/urdf/centauro_virtual_frame.urdf (robot description, URDF)
Before this commit: robot centauro, 63 links, 62 joints
Links:
- added link d435_head_motor, mass 0.33878686; collision mesh filename=package://centauro_urdf/meshes/simple/neck-pitch_mesh.stl scale=0.001 0.001 0.001; visual mesh filename=package://centauro_urdf/meshes/neck-pitch_mesh.stl scale=0.001 0.001 0.001
Joints:
- added joint d435_head_joint: type revolute, parent neck_1, child d435_head_motor, origin xyz=0.06 0 0.1375 rpy=0 0 0, axis 0 -1 0, limit lower=-1.1 upper=1.1 effort=35 velocity=5.7
- joint neck_base: origin xyz=0.0030637045 0.0061607221 0.224 rpy=0 0 0 -> xyz=0.0030637045 0.0061607221 0.158 rpy=0 0 0
- joint velodyne_joint: axis 0 1 0 -> 0 -1 0; origin xyz=0.0825 0 0.243 rpy=0 0 0 -> xyz=0.0822724 0 0.242 rpy=0 0 0
