Commit message: it was time to define dark grey color

File: centauro_urdf/urdf/centauro.urdf (robot description, URDF)
Before this commit: robot centauro, 98 links, 97 joints
Joints:
- joint D435_head_camera_accel_optical_joint: origin xyz=0 0 0 rpy=-1.57079632679 0 -1.57079632679 -> xyz=0 0 0 rpy=-1.5707963267948966 0 -1.5707963267948966
- joint D435_head_camera_color_optical_joint: origin xyz=0 0 0 rpy=-1.57079632679 0 -1.57079632679 -> xyz=0 0 0 rpy=-1.5707963267948966 0 -1.5707963267948966
- joint D435_head_camera_depth_optical_joint: origin xyz=0 0 0 rpy=-1.57079632679 0 -1.57079632679 -> xyz=0 0 0 rpy=-1.5707963267948966 0 -1.5707963267948966
- joint D435_head_camera_gyro_optical_joint: origin xyz=0 0 0 rpy=-1.57079632679 0 -1.57079632679 -> xyz=0 0 0 rpy=-1.5707963267948966 0 -1.5707963267948966
- joint D435_head_camera_left_ir_optical_joint: origin xyz=0 0 0 rpy=-1.57079632679 0 -1.57079632679 -> xyz=0 0 0 rpy=-1.5707963267948966 0 -1.5707963267948966
- joint D435_head_camera_right_ir_optical_joint: origin xyz=0 0 0 rpy=-1.57079632679 0 -1.57079632679 -> xyz=0 0 0 rpy=-1.5707963267948966 0 -1.5707963267948966
- joint D435i_camera_accel_optical_joint: origin xyz=0 0 0 rpy=-1.57079632679 0 -1.57079632679 -> xyz=0 0 0 rpy=-1.5707963267948966 0 -1.5707963267948966
- joint D435i_camera_color_optical_joint: origin xyz=0 0 0 rpy=-1.57079632679 0 -1.57079632679 -> xyz=0 0 0 rpy=-1.5707963267948966 0 -1.5707963267948966
- joint D435i_camera_depth_optical_joint: origin xyz=0 0 0 rpy=-1.57079632679 0 -1.57079632679 -> xyz=0 0 0 rpy=-1.5707963267948966 0 -1.5707963267948966
- joint D435i_camera_gyro_optical_joint: origin xyz=0 0 0 rpy=-1.57079632679 0 -1.57079632679 -> xyz=0 0 0 rpy=-1.5707963267948966 0 -1.5707963267948966
- joint D435i_camera_left_ir_optical_joint: origin xyz=0 0 0 rpy=-1.57079632679 0 -1.57079632679 -> xyz=0 0 0 rpy=-1.5707963267948966 0 -1.5707963267948966
- joint D435i_camera_right_ir_optical_joint: origin xyz=0 0 0 rpy=-1.57079632679 0 -1.57079632679 -> xyz=0 0 0 rpy=-1.5707963267948966 0 -1.5707963267948966
- joint T265_camera_accel_joint: origin xyz=-0.0311 0 0.00655 rpy=0 3.14159265359 0 -> xyz=-0.0311 0 0.00655 rpy=0 3.141592653589793 0
- joint T265_camera_accel_optical_joint: origin xyz=-0.0311 0 0.00655 rpy=0 3.14159265359 0 -> xyz=-0.0311 0 0.00655 rpy=0 3.141592653589793 0
- joint T265_camera_fisheye1_optical_joint: origin xyz=0 0 0 rpy=-1.57079632679 0 -1.57079632679 -> xyz=0 0 0 rpy=-1.5707963267948966 0 -1.5707963267948966
- joint T265_camera_fisheye1_rgb_joint: origin xyz=-0.0411 0.0 0.0 rpy=0 1.57079632679 1.57079632679 -> xyz=-0.0411 0.0 0.0 rpy=0 1.5707963267948966 1.5707963267948966
- joint T265_camera_fisheye2_optical_joint: origin xyz=0 0 0 rpy=-1.57079632679 0 -1.57079632679 -> xyz=0 0 0 rpy=-1.5707963267948966 0 -1.5707963267948966
- joint T265_camera_fisheye2_rgb_joint: origin xyz=0.0229 0.0 0.0 rpy=0 1.57079632679 1.57079632679 -> xyz=0.0229 0.0 0.0 rpy=0 1.5707963267948966 1.5707963267948966
- joint T265_camera_gyro_joint: origin xyz=-0.0311 0 0.00655 rpy=0 3.14159265359 0 -> xyz=-0.0311 0 0.00655 rpy=0 3.141592653589793 0
- joint T265_camera_link_joint: origin xyz=0 0 0 rpy=1.57079632679 0 -1.57079632679 -> xyz=0 0 0 rpy=1.5707963267948966 0 -1.5707963267948966
- joint hip_yaw_1: origin xyz=0.25 0.125 -0.0566 rpy=0.0 0.0 0.0 -> xyz=0.25 0.125 -0.056600000000000004 rpy=0.0 0.0 0.0
- joint hip_yaw_2: origin xyz=0.25 -0.125 -0.0566 rpy=0.0 0.0 0.0 -> xyz=0.25 -0.125 -0.056600000000000004 rpy=0.0 0.0 0.0
- joint hip_yaw_3: origin xyz=-0.25 0.125 -0.0566 rpy=0.0 0.0 0.0 -> xyz=-0.25 0.125 -0.056600000000000004 rpy=0.0 0.0 0.0
- joint hip_yaw_4: origin xyz=-0.25 -0.125 -0.0566 rpy=0.0 0.0 0.0 -> xyz=-0.25 -0.125 -0.056600000000000004 rpy=0.0 0.0 0.0
- joint j_wheel_1: origin xyz=0.0 -0.0 -0.09835 rpy=1.57079632679 0.0 0.0 -> xyz=0.0 -0.0 -0.09834999999999999 rpy=1.57079632679 0.0 0.0
- joint j_wheel_2: origin xyz=0.0 0.0 -0.09835 rpy=1.57079632679 0.0 0.0 -> xyz=0.0 0.0 -0.09834999999999999 rpy=1.57079632679 0.0 0.0
- joint j_wheel_3: origin xyz=0.0 -0.0 -0.09835 rpy=1.57079632679 0.0 0.0 -> xyz=0.0 -0.0 -0.09834999999999999 rpy=1.57079632679 0.0 0.0
- joint j_wheel_4: origin xyz=0.0 0.0 -0.09835 rpy=1.57079632679 0.0 0.0 -> xyz=0.0 0.0 -0.09834999999999999 rpy=1.57079632679 0.0 0.0

File: centauro_urdf/urdf/centauro_capsule.urdf (robot description, URDF)
Before this commit: robot centauro, 98 links, 97 joints
Links:
- link T265_camera_pose_frame: geometry collision cylinder length=0.1022528557886848 radius=0.0142751; collision sphere radius=0.0142751
- link ankle1_1: geometry collision cylinder length=0.049256315666076876 radius=0.0792379; collision sphere radius=0.0792379
- link ankle1_2: geometry collision cylinder length=0.047884051265172006 radius=0.0781037; collision sphere radius=0.0781037
- link ankle1_3: geometry collision cylinder length=0.049256315666076876 radius=0.0792379; collision sphere radius=0.0792379
- link ankle1_4: geometry collision cylinder length=0.047884051265172006 radius=0.0781037; collision sphere radius=0.0781037
- link ankle2_1: geometry collision cylinder length=0.07370263129636398 radius=0.0813545; collision sphere radius=0.0813545
- link ankle2_2: geometry collision cylinder length=0.07370263129636398 radius=0.0813545; collision sphere radius=0.0813545
- link ankle2_3: geometry collision cylinder length=0.07370263129636398 radius=0.0813545; collision sphere radius=0.0813545
- link ankle2_4: geometry collision cylinder length=0.07370263129636398 radius=0.0813545; collision sphere radius=0.0813545
- link arm1_1: geometry collision cylinder length=0.03739768494560427 radius=0.0698859; collision sphere radius=0.0698859
- link arm1_2: geometry collision cylinder length=0.12799269981445732 radius=0.0700645; collision sphere radius=0.0700645
- link arm1_3: geometry collision cylinder length=0.06082252644344949 radius=0.0896121; collision sphere radius=0.0896121
- link arm1_4: geometry collision cylinder length=0.08713418572944408 radius=0.0600429; collision sphere radius=0.0600429
- link arm1_5: geometry collision cylinder length=0.08434739747702548 radius=0.0804108; collision sphere radius=0.0804108
- link arm1_6: geometry collision cylinder length=0.11425141871384588 radius=0.0583263; collision sphere radius=0.0583263
- link arm1_7: geometry collision cylinder length=0.009167307493588288 radius=0.0207073; collision sphere radius=0.0207073
- link arm2_1: geometry collision cylinder length=0.03739768494560427 radius=0.0698859; collision sphere radius=0.0698859
- link arm2_2: geometry collision cylinder length=0.12799269981445732 radius=0.0700645; collision sphere radius=0.0700645
- link arm2_3: geometry collision cylinder length=0.06082252644344949 radius=0.0896121; collision sphere radius=0.0896121
- link arm2_4: geometry collision cylinder length=0.08713418572944408 radius=0.0600429; collision sphere radius=0.0600429
- link arm2_5: geometry collision cylinder length=0.08434739747702548 radius=0.0804108; collision sphere radius=0.0804108
- link arm2_6: geometry collision cylinder length=0.11425141871384588 radius=0.0583263; collision sphere radius=0.0583263
- link arm2_7: geometry collision cylinder length=0.009167307493588288 radius=0.0207073; collision sphere radius=0.0207073
- link ball1: geometry collision cylinder length=9.940076835940455e-05 radius=0.0709883; collision sphere radius=0.0709883
- link ball2: geometry collision cylinder length=9.940076835940455e-05 radius=0.0709883; collision sphere radius=0.0709883
- link d435_head_motor: geometry collision cylinder length=0.12134423548428976 radius=0.0261699; collision sphere radius=0.0261699
- link hip1_1: geometry collision cylinder length=0.03069545889898954 radius=0.0747223; collision sphere radius=0.0747223
- link hip1_2: geometry collision cylinder length=0.03069545889898954 radius=0.0747223; collision sphere radius=0.0747223
- link hip1_3: geometry collision cylinder length=0.03069545889898954 radius=0.0747223; collision sphere radius=0.0747223
- link hip1_4: geometry collision cylinder length=0.03069545889898954 radius=0.0747223; collision sphere radius=0.0747223
- link hip2_1: geometry collision cylinder length=0.2919804521727749 radius=0.0808941; collision sphere radius=0.0808941
- link hip2_2: geometry collision cylinder length=0.2919804521727749 radius=0.0808941; collision sphere radius=0.0808941
- link hip2_3: geometry collision cylinder length=0.2919804521727749 radius=0.0808941; collision sphere radius=0.0808941
- link hip2_4: geometry collision cylinder length=0.2919804521727749 radius=0.0808941; collision sphere radius=0.0808941
- link knee_1: geometry collision cylinder length=0.19275022460612404 radius=0.0664305; collision sphere radius=0.0664305
- link knee_2: geometry collision cylinder length=0.19275022460612404 radius=0.0664305; collision sphere radius=0.0664305
- link knee_3: geometry collision cylinder length=0.19275022460612404 radius=0.0664305; collision sphere radius=0.0664305
- link knee_4: geometry collision cylinder length=0.19275022460612404 radius=0.0664305; collision sphere radius=0.0664305
- link neck_1: geometry collision cylinder length=0.16454098025546557 radius=0.100414; collision sphere radius=0.100414
- link pelvis: geometry collision cylinder length=0.38594139791384763 radius=0.213204; collision sphere radius=0.213204
- link torso_2: geometry collision cylinder length=0.09543675990850982 radius=0.158224; collision sphere radius=0.158224
- link velodyne_motor: geometry collision cylinder length=0.032463112134515464 radius=0.0544637; collision sphere radius=0.0544637
Joints:
- joint D435_head_camera_accel_optical_joint: origin xyz=0.0 0.0 0.0 rpy=-1.57079632679 0.0 -1.57079632679 -> xyz=0.0 0.0 0.0 rpy=-1.5707963267948966 0.0 -1.5707963267948966
- joint D435_head_camera_color_optical_joint: origin xyz=0.0 0.0 0.0 rpy=-1.57079632679 0.0 -1.57079632679 -> xyz=0.0 0.0 0.0 rpy=-1.5707963267948966 0.0 -1.5707963267948966
- joint D435_head_camera_depth_optical_joint: origin xyz=0.0 0.0 0.0 rpy=-1.57079632679 0.0 -1.57079632679 -> xyz=0.0 0.0 0.0 rpy=-1.5707963267948966 0.0 -1.5707963267948966
- joint D435_head_camera_gyro_optical_joint: origin xyz=0.0 0.0 0.0 rpy=-1.57079632679 0.0 -1.57079632679 -> xyz=0.0 0.0 0.0 rpy=-1.5707963267948966 0.0 -1.5707963267948966
- joint D435_head_camera_left_ir_optical_joint: origin xyz=0.0 0.0 0.0 rpy=-1.57079632679 0.0 -1.57079632679 -> xyz=0.0 0.0 0.0 rpy=-1.5707963267948966 0.0 -1.5707963267948966
- joint D435_head_camera_right_ir_optical_joint: origin xyz=0.0 0.0 0.0 rpy=-1.57079632679 0.0 -1.57079632679 -> xyz=0.0 0.0 0.0 rpy=-1.5707963267948966 0.0 -1.5707963267948966
- joint D435i_camera_accel_optical_joint: origin xyz=0.0 0.0 0.0 rpy=-1.57079632679 0.0 -1.57079632679 -> xyz=0.0 0.0 0.0 rpy=-1.5707963267948966 0.0 -1.5707963267948966
- joint D435i_camera_color_optical_joint: origin xyz=0.0 0.0 0.0 rpy=-1.57079632679 0.0 -1.57079632679 -> xyz=0.0 0.0 0.0 rpy=-1.5707963267948966 0.0 -1.5707963267948966
- joint D435i_camera_depth_optical_joint: origin xyz=0.0 0.0 0.0 rpy=-1.57079632679 0.0 -1.57079632679 -> xyz=0.0 0.0 0.0 rpy=-1.5707963267948966 0.0 -1.5707963267948966
- joint D435i_camera_gyro_optical_joint: origin xyz=0.0 0.0 0.0 rpy=-1.57079632679 0.0 -1.57079632679 -> xyz=0.0 0.0 0.0 rpy=-1.5707963267948966 0.0 -1.5707963267948966
- joint D435i_camera_left_ir_optical_joint: origin xyz=0.0 0.0 0.0 rpy=-1.57079632679 0.0 -1.57079632679 -> xyz=0.0 0.0 0.0 rpy=-1.5707963267948966 0.0 -1.5707963267948966
- joint D435i_camera_right_ir_optical_joint: origin xyz=0.0 0.0 0.0 rpy=-1.57079632679 0.0 -1.57079632679 -> xyz=0.0 0.0 0.0 rpy=-1.5707963267948966 0.0 -1.5707963267948966
- joint T265_camera_accel_joint: origin xyz=-0.0311 0.0 0.00655 rpy=0.0 3.14159265359 0.0 -> xyz=-0.0311 0.0 0.00655 rpy=0.0 3.141592653589793 0.0
- joint T265_camera_accel_optical_joint: origin xyz=-0.0311 0.0 0.00655 rpy=0.0 3.14159265359 0.0 -> xyz=-0.0311 0.0 0.00655 rpy=0.0 3.141592653589793 0.0
- joint T265_camera_fisheye1_optical_joint: origin xyz=0.0 0.0 0.0 rpy=-1.57079632679 0.0 -1.57079632679 -> xyz=0.0 0.0 0.0 rpy=-1.5707963267948966 0.0 -1.5707963267948966
- joint T265_camera_fisheye1_rgb_joint: origin xyz=-0.0411 0.0 0.0 rpy=0.0 1.57079632679 1.57079632679 -> xyz=-0.0411 0.0 0.0 rpy=0.0 1.5707963267948966 1.5707963267948966
- joint T265_camera_fisheye2_optical_joint: origin xyz=0.0 0.0 0.0 rpy=-1.57079632679 0.0 -1.57079632679 -> xyz=0.0 0.0 0.0 rpy=-1.5707963267948966 0.0 -1.5707963267948966
- joint T265_camera_fisheye2_rgb_joint: origin xyz=0.0229 0.0 0.0 rpy=0.0 1.57079632679 1.57079632679 -> xyz=0.0229 0.0 0.0 rpy=0.0 1.5707963267948966 1.5707963267948966
- joint T265_camera_gyro_joint: origin xyz=-0.0311 0.0 0.00655 rpy=0.0 3.14159265359 0.0 -> xyz=-0.0311 0.0 0.00655 rpy=0.0 3.141592653589793 0.0
- joint T265_camera_link_joint: origin xyz=0.0 0.0 0.0 rpy=1.57079632679 0.0 -1.57079632679 -> xyz=0.0 0.0 0.0 rpy=1.5707963267948966 0.0 -1.5707963267948966
- joint hip_yaw_1: origin xyz=0.25 0.125 -0.0566 rpy=0.0 0.0 0.0 -> xyz=0.25 0.125 -0.056600000000000004 rpy=0.0 0.0 0.0
- joint hip_yaw_2: origin xyz=0.25 -0.125 -0.0566 rpy=0.0 0.0 0.0 -> xyz=0.25 -0.125 -0.056600000000000004 rpy=0.0 0.0 0.0
- joint hip_yaw_3: origin xyz=-0.25 0.125 -0.0566 rpy=0.0 0.0 0.0 -> xyz=-0.25 0.125 -0.056600000000000004 rpy=0.0 0.0 0.0
- joint hip_yaw_4: origin xyz=-0.25 -0.125 -0.0566 rpy=0.0 0.0 0.0 -> xyz=-0.25 -0.125 -0.056600000000000004 rpy=0.0 0.0 0.0
- joint j_wheel_1: origin xyz=0.0 -0.0 -0.09835 rpy=1.57079632679 0.0 0.0 -> xyz=0.0 -0.0 -0.09834999999999999 rpy=1.57079632679 0.0 0.0
- joint j_wheel_2: origin xyz=0.0 0.0 -0.09835 rpy=1.57079632679 0.0 0.0 -> xyz=0.0 0.0 -0.09834999999999999 rpy=1.57079632679 0.0 0.0
- joint j_wheel_3: origin xyz=0.0 -0.0 -0.09835 rpy=1.57079632679 0.0 0.0 -> xyz=0.0 -0.0 -0.09834999999999999 rpy=1.57079632679 0.0 0.0
- joint j_wheel_4: origin xyz=0.0 0.0 -0.09835 rpy=1.57079632679 0.0 0.0 -> xyz=0.0 0.0 -0.09834999999999999 rpy=1.57079632679 0.0 0.0

File: centauro_urdf/urdf/centauro_virtual_frame.urdf (robot description, URDF)
Before this commit: robot centauro, 64 links, 63 joints
Joints:
- joint hip_yaw_1: origin xyz=0.25 0.125 -0.0566 rpy=0.0 0.0 0.0 -> xyz=0.25 0.125 -0.056600000000000004 rpy=0.0 0.0 0.0
- joint hip_yaw_2: origin xyz=0.25 -0.125 -0.0566 rpy=0.0 0.0 0.0 -> xyz=0.25 -0.125 -0.056600000000000004 rpy=0.0 0.0 0.0
- joint hip_yaw_3: origin xyz=-0.25 0.125 -0.0566 rpy=0.0 0.0 0.0 -> xyz=-0.25 0.125 -0.056600000000000004 rpy=0.0 0.0 0.0
- joint hip_yaw_4: origin xyz=-0.25 -0.125 -0.0566 rpy=0.0 0.0 0.0 -> xyz=-0.25 -0.125 -0.056600000000000004 rpy=0.0 0.0 0.0
- joint j_wheel_1: origin xyz=0.0 -0.0 -0.09835 rpy=1.57079632679 0.0 0.0 -> xyz=0.0 -0.0 -0.09834999999999999 rpy=1.57079632679 0.0 0.0
- joint j_wheel_2: origin xyz=0.0 0.0 -0.09835 rpy=1.57079632679 0.0 0.0 -> xyz=0.0 0.0 -0.09834999999999999 rpy=1.57079632679 0.0 0.0
- joint j_wheel_3: origin xyz=0.0 -0.0 -0.09835 rpy=1.57079632679 0.0 0.0 -> xyz=0.0 -0.0 -0.09834999999999999 rpy=1.57079632679 0.0 0.0
- joint j_wheel_4: origin xyz=0.0 0.0 -0.09835 rpy=1.57079632679 0.0 0.0 -> xyz=0.0 0.0 -0.09834999999999999 rpy=1.57079632679 0.0 0.0

File: centauro_urdf/urdf/utils.urdf.xacro (robot description, xacro)
@@ -15,3 +15,6 @@
     <color rgba="0.1 0.1 0.1 1"/>
 </material>
+<material name="dark_grey">
+    <color rgba="0.2 0.2 0.2 1"/>
+</material>
 </robot>

Commit message: with material

File: centauro_urdf/urdf/centauro.urdf (robot description, URDF)
Before this commit: robot centauro, 94 links, 93 joints
Joints:
- joint D435_head_camera_accel_optical_joint: origin xyz=0 0 0 rpy=-1.57079632679 0 -1.57079632679 -> xyz=0 0 0 rpy=-1.5707963267948966 0 -1.5707963267948966
- joint D435_head_camera_color_optical_joint: origin xyz=0 0 0 rpy=-1.57079632679 0 -1.57079632679 -> xyz=0 0 0 rpy=-1.5707963267948966 0 -1.5707963267948966
- joint D435_head_camera_depth_optical_joint: origin xyz=0 0 0 rpy=-1.57079632679 0 -1.57079632679 -> xyz=0 0 0 rpy=-1.5707963267948966 0 -1.5707963267948966
- joint D435_head_camera_gyro_optical_joint: origin xyz=0 0 0 rpy=-1.57079632679 0 -1.57079632679 -> xyz=0 0 0 rpy=-1.5707963267948966 0 -1.5707963267948966
- joint D435_head_camera_left_ir_optical_joint: origin xyz=0 0 0 rpy=-1.57079632679 0 -1.57079632679 -> xyz=0 0 0 rpy=-1.5707963267948966 0 -1.5707963267948966
- joint D435_head_camera_right_ir_optical_joint: origin xyz=0 0 0 rpy=-1.57079632679 0 -1.57079632679 -> xyz=0 0 0 rpy=-1.5707963267948966 0 -1.5707963267948966
- joint D435i_camera_accel_optical_joint: origin xyz=0 0 0 rpy=-1.57079632679 0 -1.57079632679 -> xyz=0 0 0 rpy=-1.5707963267948966 0 -1.5707963267948966
- joint D435i_camera_color_optical_joint: origin xyz=0 0 0 rpy=-1.57079632679 0 -1.57079632679 -> xyz=0 0 0 rpy=-1.5707963267948966 0 -1.5707963267948966
- joint D435i_camera_depth_optical_joint: origin xyz=0 0 0 rpy=-1.57079632679 0 -1.57079632679 -> xyz=0 0 0 rpy=-1.5707963267948966 0 -1.5707963267948966
- joint D435i_camera_gyro_optical_joint: origin xyz=0 0 0 rpy=-1.57079632679 0 -1.57079632679 -> xyz=0 0 0 rpy=-1.5707963267948966 0 -1.5707963267948966
- joint D435i_camera_left_ir_optical_joint: origin xyz=0 0 0 rpy=-1.57079632679 0 -1.57079632679 -> xyz=0 0 0 rpy=-1.5707963267948966 0 -1.5707963267948966
- joint D435i_camera_right_ir_optical_joint: origin xyz=0 0 0 rpy=-1.57079632679 0 -1.57079632679 -> xyz=0 0 0 rpy=-1.5707963267948966 0 -1.5707963267948966
- joint T265_camera_accel_joint: origin xyz=-0.0311 0 0.00655 rpy=0 3.14159265359 0 -> xyz=-0.0311 0 0.00655 rpy=0 3.141592653589793 0
- joint T265_camera_accel_optical_joint: origin xyz=-0.0311 0 0.00655 rpy=0 3.14159265359 0 -> xyz=-0.0311 0 0.00655 rpy=0 3.141592653589793 0
- joint T265_camera_fisheye1_optical_joint: origin xyz=0 0 0 rpy=-1.57079632679 0 -1.57079632679 -> xyz=0 0 0 rpy=-1.5707963267948966 0 -1.5707963267948966
- joint T265_camera_fisheye1_rgb_joint: origin xyz=-0.0411 0.0 0.0 rpy=0 1.57079632679 1.57079632679 -> xyz=-0.0411 0.0 0.0 rpy=0 1.5707963267948966 1.5707963267948966
- joint T265_camera_fisheye2_optical_joint: origin xyz=0 0 0 rpy=-1.57079632679 0 -1.57079632679 -> xyz=0 0 0 rpy=-1.5707963267948966 0 -1.5707963267948966
- joint T265_camera_fisheye2_rgb_joint: origin xyz=0.0229 0.0 0.0 rpy=0 1.57079632679 1.57079632679 -> xyz=0.0229 0.0 0.0 rpy=0 1.5707963267948966 1.5707963267948966
- joint T265_camera_gyro_joint: origin xyz=-0.0311 0 0.00655 rpy=0 3.14159265359 0 -> xyz=-0.0311 0 0.00655 rpy=0 3.141592653589793 0
- joint T265_camera_link_joint: origin xyz=0 0 0 rpy=1.57079632679 0 -1.57079632679 -> xyz=0 0 0 rpy=1.5707963267948966 0 -1.5707963267948966
- joint hip_yaw_1: origin xyz=0.25 0.125 -0.0566 rpy=0.0 0.0 0.0 -> xyz=0.25 0.125 -0.056600000000000004 rpy=0.0 0.0 0.0
- joint hip_yaw_2: origin xyz=0.25 -0.125 -0.0566 rpy=0.0 0.0 0.0 -> xyz=0.25 -0.125 -0.056600000000000004 rpy=0.0 0.0 0.0
- joint hip_yaw_3: origin xyz=-0.25 0.125 -0.0566 rpy=0.0 0.0 0.0 -> xyz=-0.25 0.125 -0.056600000000000004 rpy=0.0 0.0 0.0
- joint hip_yaw_4: origin xyz=-0.25 -0.125 -0.0566 rpy=0.0 0.0 0.0 -> xyz=-0.25 -0.125 -0.056600000000000004 rpy=0.0 0.0 0.0
- joint j_wheel_1: origin xyz=0.0 -0.0 -0.09835 rpy=1.57079632679 0.0 0.0 -> xyz=0.0 -0.0 -0.09834999999999999 rpy=1.57079632679 0.0 0.0
- joint j_wheel_2: origin xyz=0.0 0.0 -0.09835 rpy=1.57079632679 0.0 0.0 -> xyz=0.0 0.0 -0.09834999999999999 rpy=1.57079632679 0.0 0.0
- joint j_wheel_3: origin xyz=0.0 -0.0 -0.09835 rpy=1.57079632679 0.0 0.0 -> xyz=0.0 -0.0 -0.09834999999999999 rpy=1.57079632679 0.0 0.0
- joint j_wheel_4: origin xyz=0.0 0.0 -0.09835 rpy=1.57079632679 0.0 0.0 -> xyz=0.0 0.0 -0.09834999999999999 rpy=1.57079632679 0.0 0.0

File: centauro_urdf/urdf/centauro_virtual_frame.urdf (robot description, URDF)
Before this commit: robot centauro, 64 links, 63 joints
Links:
- removed link D435_head_camera_bottom_screw_frame
- removed link D435_head_camera_link
- removed link D435i_camera_bottom_screw_frame
- removed link D435i_camera_link
Joints:
- removed joint D435_head_camera_joint
- removed joint D435_head_camera_link_joint
- removed joint D435i_camera_joint
- removed joint D435i_camera_link_joint
- joint hip_yaw_1: origin xyz=0.25 0.125 -0.0566 rpy=0.0 0.0 0.0 -> xyz=0.25 0.125 -0.056600000000000004 rpy=0.0 0.0 0.0
- joint hip_yaw_2: origin xyz=0.25 -0.125 -0.0566 rpy=0.0 0.0 0.0 -> xyz=0.25 -0.125 -0.056600000000000004 rpy=0.0 0.0 0.0
- joint hip_yaw_3: origin xyz=-0.25 0.125 -0.0566 rpy=0.0 0.0 0.0 -> xyz=-0.25 0.125 -0.056600000000000004 rpy=0.0 0.0 0.0
- joint hip_yaw_4: origin xyz=-0.25 -0.125 -0.0566 rpy=0.0 0.0 0.0 -> xyz=-0.25 -0.125 -0.056600000000000004 rpy=0.0 0.0 0.0
- joint j_wheel_1: origin xyz=0.0 -0.0 -0.09835 rpy=1.57079632679 0.0 0.0 -> xyz=0.0 -0.0 -0.09834999999999999 rpy=1.57079632679 0.0 0.0
- joint j_wheel_2: origin xyz=0.0 0.0 -0.09835 rpy=1.57079632679 0.0 0.0 -> xyz=0.0 0.0 -0.09834999999999999 rpy=1.57079632679 0.0 0.0
- joint j_wheel_3: origin xyz=0.0 -0.0 -0.09835 rpy=1.57079632679 0.0 0.0 -> xyz=0.0 -0.0 -0.09834999999999999 rpy=1.57079632679 0.0 0.0
- joint j_wheel_4: origin xyz=0.0 0.0 -0.09835 rpy=1.57079632679 0.0 0.0 -> xyz=0.0 0.0 -0.09834999999999999 rpy=1.57079632679 0.0 0.0

File: centauro_urdf/urdf/utils.urdf.xacro (robot description, xacro)
@@ -12,6 +12,12 @@
     <color rgba="0.4 0.4 0.4 1"/>
 </material>
+<material name="grey">
+    <color rgba="0.7 0.7 0.7 1"/>
+</material>
 <material name="dark">
     <color rgba="0.1 0.1 0.1 1"/>
 </material>
+<material name="dark_grey">
+    <color rgba="0.6 0.6 0.6 1"/>
+</material>
 </robot>
