Commit message: rm cameras from urdf as tfs are published by camera manager

File: centauro_urdf/urdf/centauro.urdf (robot description, URDF)
Before this commit: robot centauro, 94 links, 93 joints
Links:
- removed link D435_head_camera_accel_frame
- removed link D435_head_camera_accel_optical_frame
- removed link D435_head_camera_color_frame
- removed link D435_head_camera_color_optical_frame
- removed link D435_head_camera_depth_frame
- removed link D435_head_camera_depth_optical_frame
- removed link D435_head_camera_gyro_frame
- removed link D435_head_camera_gyro_optical_frame
- removed link D435_head_camera_left_ir_frame
- removed link D435_head_camera_left_ir_optical_frame
- removed link D435_head_camera_right_ir_frame
- removed link D435_head_camera_right_ir_optical_frame
- removed link D435i_camera_accel_frame
- removed link D435i_camera_accel_optical_frame
- removed link D435i_camera_color_frame
- removed link D435i_camera_color_optical_frame
- removed link D435i_camera_depth_frame
- removed link D435i_camera_depth_optical_frame
- removed link D435i_camera_gyro_frame
- removed link D435i_camera_gyro_optical_frame
- removed link D435i_camera_left_ir_frame
- removed link D435i_camera_left_ir_optical_frame
- removed link D435i_camera_right_ir_frame
- removed link D435i_camera_right_ir_optical_frame
- removed link T265_camera_accel_frame
- removed link T265_camera_accel_optical_frame
- removed link T265_camera_fisheye1_optical_frame
- removed link T265_camera_fisheye1_rgb_frame
- removed link T265_camera_fisheye2_optical_frame
- removed link T265_camera_fisheye2_rgb_frame
- removed link T265_camera_gyro_frame
- removed link T265_camera_gyro_optical_frame
- removed link T265_camera_link
- removed link T265_camera_pose_frame
- link D435_head_camera_link: geometry collision box size=0.02505 0.09 0.025; visual mesh filename=package://centauro_urdf/meshes/realsense/d435.dae
- link D435i_camera_link: geometry collision box size=0.02505 0.09 0.025; visual mesh filename=package://centauro_urdf/meshes/realsense/d435.dae
Joints:
- removed joint D435_head_camera_accel_joint
- removed joint D435_head_camera_accel_optical_joint
- removed joint D435_head_camera_color_joint
- removed joint D435_head_camera_color_optical_joint
- removed joint D435_head_camera_depth_joint
- removed joint D435_head_camera_depth_optical_joint
- removed joint D435_head_camera_gyro_joint
- removed joint D435_head_camera_gyro_optical_joint
- removed joint D435_head_camera_left_ir_joint
- removed joint D435_head_camera_left_ir_optical_joint
- removed joint D435_head_camera_right_ir_joint
- removed joint D435_head_camera_right_ir_optical_joint
- removed joint D435i_camera_accel_joint
- removed joint D435i_camera_accel_optical_joint
- removed joint D435i_camera_color_joint
- removed joint D435i_camera_color_optical_joint
- removed joint D435i_camera_depth_joint
- removed joint D435i_camera_depth_optical_joint
- removed joint D435i_camera_gyro_joint
- removed joint D435i_camera_gyro_optical_joint
- removed joint D435i_camera_left_ir_joint
- removed joint D435i_camera_left_ir_optical_joint
- removed joint D435i_camera_right_ir_joint
- removed joint D435i_camera_right_ir_optical_joint
- removed joint T265_camera_accel_joint
- removed joint T265_camera_accel_optical_joint
- removed joint T265_camera_fisheye1_optical_joint
- removed joint T265_camera_fisheye1_rgb_joint
- removed joint T265_camera_fisheye2_optical_joint
- removed joint T265_camera_fisheye2_rgb_joint
- removed joint T265_camera_gyro_joint
- removed joint T265_camera_gyro_optical_joint
- removed joint T265_camera_link_joint
- removed joint T265_camera_pose_joint
- joint hip_yaw_1: origin xyz=0.25 0.125 -0.056600000000000004 rpy=0.0 0.0 0.0 -> xyz=0.25 0.125 -0.0566 rpy=0.0 0.0 0.0
- joint hip_yaw_2: origin xyz=0.25 -0.125 -0.056600000000000004 rpy=0.0 0.0 0.0 -> xyz=0.25 -0.125 -0.0566 rpy=0.0 0.0 0.0
- joint hip_yaw_3: origin xyz=-0.25 0.125 -0.056600000000000004 rpy=0.0 0.0 0.0 -> xyz=-0.25 0.125 -0.0566 rpy=0.0 0.0 0.0
- joint hip_yaw_4: origin xyz=-0.25 -0.125 -0.056600000000000004 rpy=0.0 0.0 0.0 -> xyz=-0.25 -0.125 -0.0566 rpy=0.0 0.0 0.0
- joint j_wheel_1: origin xyz=0.0 -0.0 -0.09834999999999999 rpy=1.57079632679 0.0 0.0 -> xyz=0.0 -0.0 -0.09835 rpy=1.57079632679 0.0 0.0
- joint j_wheel_2: origin xyz=0.0 0.0 -0.09834999999999999 rpy=1.57079632679 0.0 0.0 -> xyz=0.0 0.0 -0.09835 rpy=1.57079632679 0.0 0.0
- joint j_wheel_3: origin xyz=0.0 -0.0 -0.09834999999999999 rpy=1.57079632679 0.0 0.0 -> xyz=0.0 -0.0 -0.09835 rpy=1.57079632679 0.0 0.0
- joint j_wheel_4: origin xyz=0.0 0.0 -0.09834999999999999 rpy=1.57079632679 0.0 0.0 -> xyz=0.0 0.0 -0.09835 rpy=1.57079632679 0.0 0.0

File: centauro_urdf/urdf/centauro_virtual_frame.urdf (robot description, URDF)
Before this commit: robot centauro, 100 links, 99 joints
Links:
- removed link D435_head_camera_accel_frame
- removed link D435_head_camera_accel_optical_frame
- removed link D435_head_camera_color_frame
- removed link D435_head_camera_color_optical_frame
- removed link D435_head_camera_depth_frame
- removed link D435_head_camera_depth_optical_frame
- removed link D435_head_camera_gyro_frame
- removed link D435_head_camera_gyro_optical_frame
- removed link D435_head_camera_left_ir_frame
- removed link D435_head_camera_left_ir_optical_frame
- removed link D435_head_camera_right_ir_frame
- removed link D435_head_camera_right_ir_optical_frame
- removed link D435i_camera_accel_frame
- removed link D435i_camera_accel_optical_frame
- removed link D435i_camera_color_frame
- removed link D435i_camera_color_optical_frame
- removed link D435i_camera_depth_frame
- removed link D435i_camera_depth_optical_frame
- removed link D435i_camera_gyro_frame
- removed link D435i_camera_gyro_optical_frame
- removed link D435i_camera_left_ir_frame
- removed link D435i_camera_left_ir_optical_frame
- removed link D435i_camera_right_ir_frame
- removed link D435i_camera_right_ir_optical_frame
- removed link T265_camera_accel_frame
- removed link T265_camera_accel_optical_frame
- removed link T265_camera_fisheye1_optical_frame
- removed link T265_camera_fisheye1_rgb_frame
- removed link T265_camera_fisheye2_optical_frame
- removed link T265_camera_fisheye2_rgb_frame
- removed link T265_camera_gyro_frame
- removed link T265_camera_gyro_optical_frame
- removed link T265_camera_link
- removed link T265_camera_pose_frame
- link D435_head_camera_link: geometry collision box size=0.02505 0.09 0.025; visual mesh filename=package://centauro_urdf/meshes/realsense/d435.dae
- link D435i_camera_link: geometry collision box size=0.02505 0.09 0.025; visual mesh filename=package://centauro_urdf/meshes/realsense/d435.dae
Joints:
- removed joint D435_head_camera_accel_joint
- removed joint D435_head_camera_accel_optical_joint
- removed joint D435_head_camera_color_joint
- removed joint D435_head_camera_color_optical_joint
- removed joint D435_head_camera_depth_joint
- removed joint D435_head_camera_depth_optical_joint
- removed joint D435_head_camera_gyro_joint
- removed joint D435_head_camera_gyro_optical_joint
- removed joint D435_head_camera_left_ir_joint
- removed joint D435_head_camera_left_ir_optical_joint
- removed joint D435_head_camera_right_ir_joint
- removed joint D435_head_camera_right_ir_optical_joint
- removed joint D435i_camera_accel_joint
- removed joint D435i_camera_accel_optical_joint
- removed joint D435i_camera_color_joint
- removed joint D435i_camera_color_optical_joint
- removed joint D435i_camera_depth_joint
- removed joint D435i_camera_depth_optical_joint
- removed joint D435i_camera_gyro_joint
- removed joint D435i_camera_gyro_optical_joint
- removed joint D435i_camera_left_ir_joint
- removed joint D435i_camera_left_ir_optical_joint
- removed joint D435i_camera_right_ir_joint
- removed joint D435i_camera_right_ir_optical_joint
- removed joint T265_camera_accel_joint
- removed joint T265_camera_accel_optical_joint
- removed joint T265_camera_fisheye1_optical_joint
- removed joint T265_camera_fisheye1_rgb_joint
- removed joint T265_camera_fisheye2_optical_joint
- removed joint T265_camera_fisheye2_rgb_joint
- removed joint T265_camera_gyro_joint
- removed joint T265_camera_gyro_optical_joint
- removed joint T265_camera_link_joint
- removed joint T265_camera_pose_joint
- joint hip_yaw_1: origin xyz=0.25 0.125 -0.056600000000000004 rpy=0.0 0.0 0.0 -> xyz=0.25 0.125 -0.0566 rpy=0.0 0.0 0.0
- joint hip_yaw_2: origin xyz=0.25 -0.125 -0.056600000000000004 rpy=0.0 0.0 0.0 -> xyz=0.25 -0.125 -0.0566 rpy=0.0 0.0 0.0
- joint hip_yaw_3: origin xyz=-0.25 0.125 -0.056600000000000004 rpy=0.0 0.0 0.0 -> xyz=-0.25 0.125 -0.0566 rpy=0.0 0.0 0.0
- joint hip_yaw_4: origin xyz=-0.25 -0.125 -0.056600000000000004 rpy=0.0 0.0 0.0 -> xyz=-0.25 -0.125 -0.0566 rpy=0.0 0.0 0.0
- joint j_wheel_1: origin xyz=0.0 -0.0 -0.09834999999999999 rpy=1.57079632679 0.0 0.0 -> xyz=0.0 -0.0 -0.09835 rpy=1.57079632679 0.0 0.0
- joint j_wheel_2: origin xyz=0.0 0.0 -0.09834999999999999 rpy=1.57079632679 0.0 0.0 -> xyz=0.0 0.0 -0.09835 rpy=1.57079632679 0.0 0.0
- joint j_wheel_3: origin xyz=0.0 -0.0 -0.09834999999999999 rpy=1.57079632679 0.0 0.0 -> xyz=0.0 -0.0 -0.09835 rpy=1.57079632679 0.0 0.0
- joint j_wheel_4: origin xyz=0.0 0.0 -0.09834999999999999 rpy=1.57079632679 0.0 0.0 -> xyz=0.0 0.0 -0.09835 rpy=1.57079632679 0.0 0.0

File: centauro_urdf/urdf/config/centauro.urdf.xacro (robot description, xacro)
@@ -7,5 +7,5 @@
 <xacro:arg name="upper_body" default="true"/>
 <xacro:arg name="velodyne" default="true"/>
-<xacro:arg name="realsense" default="true"/>
+<xacro:arg name="realsense" default="false"/>
 <xacro:if value="$(arg realsense)">
 	<xacro:arg name="d435i_head" default="true"/>

File: centauro_urdf/urdf/config/centauro_virtual_frame.urdf.xacro (robot description, xacro)
@@ -15,6 +15,6 @@
     <xacro:property name="USE_STICKS" value="false" />
     <xacro:property name="ADD_VELODYNE" value="true" />
-    <xacro:property name="ADD_D435I_HEAD" value="true" />
-    <xacro:property name="ADD_D435I_BASE" value="true" />
-    <xacro:property name="ADD_T265_BASE" value="true" />
+    <xacro:property name="ADD_D435I_HEAD" value="false" />
+    <xacro:property name="ADD_D435I_BASE" value="false" />
+    <xacro:property name="ADD_T265_BASE" value="false" />
 </robot>
