Commit message: Try different sensors for new head

File: centauro_urdf/urdf/centauro.urdf (robot description, URDF)
Before this commit: robot centauro, 60 links, 59 joints
Links:
- added link D435i_camera_accel_frame
- added link D435i_camera_accel_optical_frame
- added link D435i_camera_color_frame
- added link D435i_camera_color_optical_frame
- added link D435i_camera_depth_frame
- added link D435i_camera_depth_optical_frame
- added link D435i_camera_gyro_frame
- added link D435i_camera_gyro_optical_frame
- added link D435i_camera_left_ir_frame
- added link D435i_camera_left_ir_optical_frame
- added link D435i_camera_right_ir_frame
- added link D435i_camera_right_ir_optical_frame
- added link T265_camera_accel_frame
- added link T265_camera_accel_optical_frame
- added link T265_camera_fisheye1_optical_frame
- added link T265_camera_fisheye1_rgb_frame
- added link T265_camera_fisheye2_optical_frame
- added link T265_camera_fisheye2_rgb_frame
- added link T265_camera_gyro_frame
- added link T265_camera_gyro_optical_frame
- added link T265_camera_link
- added link T265_camera_pose_frame, mass 0.068024; collision mesh filename=package://realsense_gazebo_description/meshes/t265_simplifi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 scale=0.001 0.001 0.001; visual mesh filename=package://realsense_gazebo_description/meshes/t265_full.stl scale=0.001 0.001 0.001
- added link zedx_front1_baro_link
- added link zedx_front1_camera_center, mass 0.16140; collision box size=0.094 0.030 0.037; visual box size=0.030 0.094 0.037
- added link zedx_front1_left_camera_frame
- added link zedx_front1_left_camera_optical_frame
- added link zedx_front1_mag_link
- added link zedx_front1_right_camera_frame
- added link zedx_front1_right_camera_optical_frame
- added link zedx_front1_temp_left_link
- added link zedx_front1_temp_right_link
- added link zedx_front2_baro_link
- added link zedx_front2_camera_center, mass 0.16140; collision box size=0.094 0.030 0.037; visual box size=0.030 0.094 0.037
- added link zedx_front2_left_camera_frame
- added link zedx_front2_left_camera_optical_frame
- added link zedx_front2_mag_link
- added link zedx_front2_right_camera_frame
- added link zedx_front2_right_camera_optical_frame
- added link zedx_front2_temp_left_link
- added link zedx_front2_temp_right_link
- link D435i_camera_link: geometry collision box size=0.02505 0.09 0.025; visual mesh filename=package://realsense2_description/meshes/d435.dae
- link velodyne_calib: geometry collision sphere radius=0; visual mesh filename=package://velodyne_description/meshes/VLP16_scan.dae
Joints:
- added joint D435i_camera_accel_joint: type fixed, parent D435i_camera_link, child D435i_camera_accel_frame, origin xyz=-0.00174 0.00552 0.0176 rpy=0 0 0
- added joint D435i_camera_accel_optical_joint: type fixed, parent D435i_camera_accel_frame, child D435i_camera_accel_optical_frame, origin xyz=0 0 0 rpy=-1.5707963267948966 0 -1.5707963267948966
- added joint D435i_camera_color_joint: type fixed, parent D435i_camera_depth_frame, child D435i_camera_color_frame, origin xyz=0 0.015 0 rpy=0 0 0
- added joint D435i_camera_color_optical_joint: type fixed, parent D435i_camera_color_frame, child D435i_camera_color_optical_frame, origin xyz=0 0 0 rpy=-1.5707963267948966 0 -1.5707963267948966
- added joint D435i_camera_depth_joint: type fixed, parent D435i_camera_link, child D435i_camera_depth_frame, origin xyz=0 0 0 rpy=0 0 0
- added joint D435i_camera_depth_optical_joint: type fixed, parent D435i_camera_depth_frame, child D435i_camera_depth_optical_frame, origin xyz=0 0 0 rpy=-1.5707963267948966 0 -1.5707963267948966
- added joint D435i_camera_gyro_joint: type fixed, parent D435i_camera_link, child D435i_camera_gyro_frame, origin xyz=-0.00174 0.00552 0.0176 rpy=0 0 0
- added joint D435i_camera_gyro_optical_joint: type fixed, parent D435i_camera_gyro_frame, child D435i_camera_gyro_optical_frame, origin xyz=0 0 0 rpy=-1.5707963267948966 0 -1.5707963267948966
- added joint D435i_camera_left_ir_joint: type fixed, parent D435i_camera_depth_frame, child D435i_camera_left_ir_frame, origin xyz=0 0.0 0 rpy=0 0 0
- added joint D435i_camera_left_ir_optical_joint: type fixed, parent D435i_camera_left_ir_frame, child D435i_camera_left_ir_optical_frame, origin xyz=0 0 0 rpy=-1.5707963267948966 0 -1.5707963267948966
- added joint D435i_camera_right_ir_joint: type fixed, parent D435i_camera_depth_frame, child D435i_camera_right_ir_frame, origin xyz=0 -0.05 0 rpy=0 0 0
- added joint D435i_camera_right_ir_optical_joint: type fixed, parent D435i_camera_right_ir_frame, child D435i_camera_right_ir_optical_frame, origin xyz=0 0 0 rpy=-1.5707963267948966 0 -1.5707963267948966
- added joint T265_camera_accel_joint: type fixed, parent T265_camera_link, child T265_camera_accel_frame, origin xyz=-0.0311 0 0.00655 rpy=0 3.141592653589793 0
- added joint T265_camera_accel_optical_joint: type fixed, parent T265_camera_accel_frame, child T265_camera_accel_optical_frame, origin xyz=-0.0311 0 0.00655 rpy=0 3.141592653589793 0
- added joint T265_camera_fisheye1_optical_joint: type fixed, parent T265_camera_fisheye1_rgb_frame, child T265_camera_fisheye1_optical_frame, origin xyz=0 0 0 rpy=-1.5707963267948966 0 -1.5707963267948966
- added joint T265_camera_fisheye1_rgb_joint: type fixed, parent T265_camera_link, child T265_camera_fisheye1_rgb_frame, origin xyz=-0.0411 0.0 0.0 rpy=0 1.5707963267948966 1.5707963267948966
- added joint T265_camera_fisheye2_optical_joint: type fixed, parent T265_camera_fisheye2_rgb_frame, child T265_camera_fisheye2_optical_frame, origin xyz=0 0 0 rpy=-1.5707963267948966 0 -1.5707963267948966
- added joint T265_camera_fisheye2_rgb_joint: type fixed, parent T265_camera_link, child T265_camera_fisheye2_rgb_frame, origin xyz=0.0229 0.0 0.0 rpy=0 1.5707963267948966 1.5707963267948966
- added joint T265_camera_gyro_joint: type fixed, parent T265_camera_link, child T265_camera_gyro_frame, origin xyz=-0.0311 0 0.00655 rpy=0 3.141592653589793 0
- added joint T265_camera_gyro_optical_joint: type fixed, parent T265_camera_gyro_frame, child T265_camera_gyro_optical_frame, origin xyz=0 0 0 rpy=0 0 0
- added joint T265_camera_link_joint: type fixed, parent T265_camera_pose_frame, child T265_camera_link, origin xyz=0 0 0 rpy=1.5707963267948966 0 -1.5707963267948966
- added joint T265_camera_pose_joint: type fixed, parent pelvis, child T265_camera_pose_frame, origin xyz=0.29245 0.00775 0.063 rpy=0 0 0
- added joint zedx_front1_baro_joint: type fixed, parent zedx_front1_camera_center, child zedx_front1_baro_link, origin xyz=0 0 0 rpy=0 0 0
- added joint zedx_front1_base_joint: type fixed, parent neck_1, child zedx_front1_camera_center, origin xyz=0.09 0.05 0.1375 rpy=-1.57 0 -0.5
- added joint zedx_front1_left_camera_joint: type fixed, parent zedx_front1_camera_center, child zedx_front1_left_camera_frame, origin xyz=0 0.025 0 rpy=0 0 0
- added joint zedx_front1_left_camera_optical_joint: type fixed, parent zedx_front1_left_camera_frame, child zedx_front1_left_camera_optical_frame, origin xyz=0 0 0 rpy=-1.5707963267948966 0.0 -1.5707963267948966
- added joint zedx_front1_mag_joint: type fixed, parent zedx_front1_camera_center, child zedx_front1_mag_link, origin xyz=0 0 0 rpy=0 0 0
- added joint zedx_front1_right_camera_joint: type fixed, parent zedx_front1_camera_center, child zedx_front1_right_camera_frame, origin xyz=0 -0.025 0 rpy=0 0 0
- added joint zedx_front1_right_camera_optical_joint: type fixed, parent zedx_front1_right_camera_frame, child zedx_front1_right_camera_optical_frame, origin xyz=0 0 0 rpy=-1.5707963267948966 0.0 -1.5707963267948966
- added joint zedx_front1_temp_left_joint: type fixed, parent zedx_front1_left_camera_frame, child zedx_front1_temp_left_link, origin xyz=0 0 0 rpy=0 0 0
- added joint zedx_front1_temp_right_joint: type fixed, parent zedx_front1_right_camera_frame, child zedx_front1_temp_right_link, origin xyz=0 0 0 rpy=0 0 0
- added joint zedx_front2_baro_joint: type fixed, parent zedx_front2_camera_center, child zedx_front2_baro_link, origin xyz=0 0 0 rpy=0 0 0
- added joint zedx_front2_base_joint: type fixed, parent neck_1, child zedx_front2_camera_center, origin xyz=0.09 -0.05 0.1375 rpy=-1.57 0 0.5
- added joint zedx_front2_left_camera_joint: type fixed, parent zedx_front2_camera_center, child zedx_front2_left_camera_frame, origin xyz=0 0.025 0 rpy=0 0 0
- added joint zedx_front2_left_camera_optical_joint: type fixed, parent zedx_front2_left_camera_frame, child zedx_front2_left_camera_optical_frame, origin xyz=0 0 0 rpy=-1.5707963267948966 0.0 -1.5707963267948966
- added joint zedx_front2_mag_joint: type fixed, parent zedx_front2_camera_center, child zedx_front2_mag_link, origin xyz=0 0 0 rpy=0 0 0
- added joint zedx_front2_right_camera_joint: type fixed, parent zedx_front2_camera_center, child zedx_front2_right_camera_frame, origin xyz=0 -0.025 0 rpy=0 0 0
- added joint zedx_front2_right_camera_optical_joint: type fixed, parent zedx_front2_right_camera_frame, child zedx_front2_right_camera_optical_frame, origin xyz=0 0 0 rpy=-1.5707963267948966 0.0 -1.5707963267948966
- added joint zedx_front2_temp_left_joint: type fixed, parent zedx_front2_left_camera_frame, child zedx_front2_temp_left_link, origin xyz=0 0 0 rpy=0 0 0
- added joint zedx_front2_temp_right_joint: type fixed, parent zedx_front2_right_camera_frame, child zedx_front2_temp_right_link, origin xyz=0 0 0 rpy=0 0 0
- joint D435i_camera_link_joint: origin xyz=0.053 0.0 -0.035 rpy=0 0.0050 -0.008 -> xyz=0 0.0175 0.0125 rpy=0 0 0
- joint hip_yaw_1: origin xyz=0.25 0.125 -0.0566 rpy=0.0 0.0 0.0 -> xyz=0.25 0.125 -0.056600000000000004 rpy=0.0 0.0 0.0
- joint hip_yaw_2: origin xyz=0.25 -0.125 -0.0566 rpy=0.0 0.0 0.0 -> xyz=0.25 -0.125 -0.056600000000000004 rpy=0.0 0.0 0.0
- joint hip_yaw_3: origin xyz=-0.25 0.125 -0.0566 rpy=0.0 0.0 0.0 -> xyz=-0.25 0.125 -0.056600000000000004 rpy=0.0 0.0 0.0
- joint hip_yaw_4: origin xyz=-0.25 -0.125 -0.0566 rpy=0.0 0.0 0.0 -> xyz=-0.25 -0.125 -0.056600000000000004 rpy=0.0 0.0 0.0
- joint j_wheel_1: origin xyz=0.0 -0.0 -0.09835 rpy=1.57079632679 0.0 0.0 -> xyz=0.0 -0.0 -0.09834999999999999 rpy=1.57079632679 0.0 0.0
- joint j_wheel_2: origin xyz=0.0 0.0 -0.09835 rpy=1.57079632679 0.0 0.0 -> xyz=0.0 0.0 -0.09834999999999999 rpy=1.57079632679 0.0 0.0
- joint j_wheel_3: origin xyz=0.0 -0.0 -0.09835 rpy=1.57079632679 0.0 0.0 -> xyz=0.0 -0.0 -0.09834999999999999 rpy=1.57079632679 0.0 0.0
- joint j_wheel_4: origin xyz=0.0 0.0 -0.09835 rpy=1.57079632679 0.0 0.0 -> xyz=0.0 0.0 -0.09834999999999999 rpy=1.57079632679 0.0 0.0

File: centauro_urdf/urdf/config/centauro.urdf.xacro (robot description, xacro)
@@ -7,7 +7,12 @@
 <xacro:arg name="upper_body" default="true"/>
 <xacro:arg name="velodyne" default="true"/>
-<xacro:arg name="realsense" default="false"/>
+<xacro:arg name="realsense" default="true"/>
+<xacro:arg name="eurobin_head" default="true"/>
+    <xacro:arg name="head_d455" default="false"/>
+    <xacro:arg name="head_d435" default="false"/>
+    <xacro:arg name="head_zed_x_mini" default="true"/>
+    <xacro:arg name="head_zed_mini" default="false"/>
 <xacro:if value="$(arg realsense)">
-	<xacro:arg name="d435i_head" default="true"/>
+        <xacro:arg name="d435i_head" default="false"/>
 	<xacro:arg name="d435i_base" default="true"/>
 	<xacro:arg name="t265_base" default="true"/>
@@ -31,3 +36,8 @@
 <xacro:property name="ADD_D435I_BASE" value="$(arg d435i_base)" />
 <xacro:property name="ADD_T265_BASE" value="$(arg t265_base)" />
+<xacro:property name="USE_EUROBIN_HEAD" value="$(arg eurobin_head)" />
+<xacro:property name="USE_HEAD_D455" value="$(arg head_d455)" />
+<xacro:property name="USE_HEAD_D435" value="$(arg head_d435)" />
+<xacro:property name="USE_HEAD_ZED_X_MINI" value="$(arg head_zed_x_mini)" />
+<xacro:property name="USE_HEAD_ZED_MINI" value="$(arg head_zed_mini)" />
 </robot>

File: centauro_urdf/urdf/gazebo/xbot.gazebo.xacro (robot description, xacro)
@@ -16,5 +16,5 @@
             <gain name="medium_mot" p="4000" d="40"/>
             <gain name="big_mot"    p="8000" d="50"/>
-            <gain name="wheel_mot"  p="0" d="10"/>
+            <gain name="wheel_mot"  p="20" d="5"/>
             <pid name="neck_yaw" profile="lowpwr_mot"/>
             <pid name="neck_pitch" profile="lowpwr_mot"/>

File: centauro_urdf/urdf/parts/head.urdf.xacro (robot description, xacro)
@@ -157,4 +157,126 @@
     </link>
   </xacro:unless>
+  <xacro:if value="${USE_EUROBIN_HEAD}">
+  <xacro:include filename="$(find centauro_urdf)/urdf/parts/zed_x_mini.urdf.xacro"/>
+  <xacro:include filename="$(find centauro_urdf)/urdf/parts/zed_mini.urdf.xacro"/>
+  <xacro:include filename="$(find realsense_gazebo_description)/urdf/_d435i.urdf.xacro"/>
+  <xacro:include filename="$(find realsense_gazebo_description)/urdf/_d455.urdf.xacro"/>
+    <xacro:if value="${USE_HEAD_ZED_MINI}">
+        <xacro:zed_mini
+            parent="neck_1"
+            name="zed_mini_front1">
+            <origin xyz="0.09 0.05 0.1375" rpy="-1.57 0 -0.5"/>
+        </xacro:zed_mini>
+        <xacro:zed_mini_gazebo
+                name="zed_mini_front1"/>
+        <xacro:zed_mini
+            parent="neck_1"
+            name="zed_mini_front2">
+        <origin xyz="0.09 -0.05 0.1375" rpy="-1.57 0 0.5"/>
+        </xacro:zed_mini>
+        <xacro:zed_mini_gazebo
+                name="zed_mini_front2"/>
+    </xacro:if>
+    <xacro:if value="${USE_HEAD_ZED_X_MINI}">
+        <xacro:zed_x_mini
+            parent="neck_1"
+            name="zedx_front1">
+            <origin xyz="0.09 0.05 0.1375" rpy="-1.57 0 -0.5"/>
+        </xacro:zed_x_mini>
+        <xacro:zed_x_mini_gazebo
+                name="zedx_front1"/>
+        <xacro:zed_x_mini
+            parent="neck_1"
+            name="zedx_front2">
+        <origin xyz="0.09 -0.05 0.1375" rpy="-1.57 0 0.5"/>
+        </xacro:zed_x_mini>
+        <xacro:zed_x_mini_gazebo
+                name="zedx_front2"/>
+      </xacro:if>
+    <xacro:if value="${USE_HEAD_D435}">
+        <xacro:sensor_d435i parent="neck_1"
+            name="d435_head_1"
+            topics_ns="d435_head_1"
+            enable_pointCloud="true"
+            align_depth="true"
+            unite_imu_method="false"
+            visualize="false"
+            accel_fps="300"
+            gyro_fps="300"
+            depth_width="1280"
+            depth_height="720"
+            depth_fps="90"
+            infra_width="1280"
+            infra_height="720"
+            infra_fps="90"
+            color_width="1280"
+            color_height="720"
+            color_fps="30">
+            <origin xyz="0.09 0.05 0.1375" rpy="-1.57 0 -0.5"/>
+        </xacro:sensor_d435i>
+        <xacro:sensor_d435i parent="neck_1"
+            name="d435_head_2"
+            topics_ns="d435_head_2"
+            enable_pointCloud="true"
+            align_depth="true"
+            unite_imu_method="false"
+            visualize="false"
+            accel_fps="300"
+            gyro_fps="300"
+            depth_width="1280"
+            depth_height="720"
+            depth_fps="90"
+            infra_width="1280"
+            infra_height="720"
+            infra_fps="90"
+            color_width="1280"
+            color_height="720"
+            color_fps="30">
+            <origin xyz="0.09 -0.05 0.1375" rpy="-1.57 0 0.5"/>
+        </xacro:sensor_d435i>
+    </xacro:if>
+    <xacro:if value="${USE_HEAD_D455}">
+        <xacro:sensor_d455 parent="neck_1"
+            name="d455_head_1"
+            topics_ns="d455_head_1"
+            enable_pointCloud="true"
+            align_depth="true"
+            unite_imu_method="false"
+            visualize="false"
+            accel_fps="300"
+            gyro_fps="300"
+            depth_width="1280"
+            depth_height="720"
+            depth_fps="90"
+            infra_width="1280"
+            infra_height="720"
+            infra_fps="90"
+            color_width="1280"
+            color_height="720"
+            color_fps="30">
+            <origin xyz="0.08 0.065 0.1375" rpy="-1.57 0 -0.52"/>
+        </xacro:sensor_d455>
+        <xacro:sensor_d455 parent="neck_1"
+            name="d455_head_2"
+            topics_ns="d455_head_2"
+            enable_pointCloud="true"
+            align_depth="true"
+            unite_imu_method="false"
+            visualize="false"
+            accel_fps="300"
+            gyro_fps="300"
+            depth_width="1280"
+            depth_height="720"
+            depth_fps="90"
+            infra_width="1280"
+            infra_height="720"
+            infra_fps="90"
+            color_width="1280"
+            color_height="720"
+            color_fps="30">
+            <origin xyz="0.08 -0.065 0.1375" rpy="-1.57 0 0.52"/>
+        </xacro:sensor_d455>
+    </xacro:if>
+  </xacro:if>
   <xacro:if value="${ADD_VELODYNE}">
     <xacro:include filename="$(find velodyne_description)/urdf/VLP-16.urdf.xacro"/>
