Commit message: generate urdf / srdf

File: centauro_urdf/urdf/centauro.urdf (robot description, URDF)
Before this commit: robot centauro, 60 links, 59 joints
Links:
- link ankle2_1: mass 1.7656714 -> 2.440929; geometry collision mesh filename=package://centauro_urdf/meshes/v2/collision/mesh_ankle-yaw_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 scale=0.001 -0.001 0.001; visual mesh filename=package://centauro_urdf/meshes/v2/mesh_ankle-yaw_wheel23.stl scale=0.001 -0.001 0.001
- link ankle2_2: mass 1.7656714 -> 2.440929; geometry collision mesh filename=package://centauro_urdf/meshes/v2/collision/mesh_ankle-yaw_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 scale=0.001 0.001 0.001; visual mesh filename=package://centauro_urdf/meshes/v2/mesh_ankle-yaw_wheel23.stl scale=0.001 0.001 0.001
- link ankle2_3: mass 1.7656714 -> 2.440929; geometry collision mesh filename=package://centauro_urdf/meshes/v2/collision/mesh_ankle-yaw_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 scale=0.001 -0.001 0.001; visual mesh filename=package://centauro_urdf/meshes/v2/mesh_ankle-yaw_wheel23.stl scale=0.001 -0.001 0.001
- link ankle2_4: mass 1.7656714 -> 2.440929; geometry collision mesh filename=package://centauro_urdf/meshes/v2/collision/mesh_ankle-yaw_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 scale=0.001 0.001 0.001; visual mesh filename=package://centauro_urdf/meshes/v2/mesh_ankle-yaw_wheel23.stl scale=0.001 0.001 0.001
- link velodyne_calib: geometry collision sphere radius=0; visual mesh filename=package://velodyne_description/meshes/VLP16_scan.dae
- link wheel_1: mass 1.11164 -> 1.8569388; geometry collision mesh filename=package://centauro_urdf/meshes/v2/collision/mesh_wheel23.stl scale=0.001 0.001 -0.001; visual mesh filename=package://centauro_urdf/meshes/v2/mesh_wheel23.stl scale=0.001 0.001 -0.001
- link wheel_2: mass 1.11164 -> 1.8569388; geometry collision mesh filename=package://centauro_urdf/meshes/v2/collision/mesh_wheel23.stl scale=0.001 0.001 0.001; visual mesh filename=package://centauro_urdf/meshes/v2/mesh_wheel23.stl scale=0.001 0.001 0.001
- link wheel_3: mass 1.11164 -> 1.8569388; geometry collision mesh filename=package://centauro_urdf/meshes/v2/collision/mesh_wheel23.stl scale=0.001 0.001 -0.001; visual mesh filename=package://centauro_urdf/meshes/v2/mesh_wheel23.stl scale=0.001 0.001 -0.001
- link wheel_4: mass 1.11164 -> 1.8569388; geometry collision mesh filename=package://centauro_urdf/meshes/v2/collision/mesh_wheel23.stl scale=0.001 0.001 0.001; visual mesh filename=package://centauro_urdf/meshes/v2/mesh_wheel23.stl scale=0.001 0.001 0.001
Joints:
- joint hip_yaw_1: origin xyz=0.25 0.125 -0.0566 rpy=0.0 0.0 0.0 -> xyz=0.25 0.125 -0.056600000000000004 rpy=0.0 0.0 0.0
- joint hip_yaw_2: origin xyz=0.25 -0.125 -0.0566 rpy=0.0 0.0 0.0 -> xyz=0.25 -0.125 -0.056600000000000004 rpy=0.0 0.0 0.0
- joint hip_yaw_3: origin xyz=-0.25 0.125 -0.0566 rpy=0.0 0.0 0.0 -> xyz=-0.25 0.125 -0.056600000000000004 rpy=0.0 0.0 0.0
- joint hip_yaw_4: origin xyz=-0.25 -0.125 -0.0566 rpy=0.0 0.0 0.0 -> xyz=-0.25 -0.125 -0.056600000000000004 rpy=0.0 0.0 0.0
- joint j_wheel_1: origin xyz=0.0 -0.0 -0.09835 rpy=1.57079632679 0.0 0.0 -> xyz=0.0 -0.0 -0.14435 rpy=1.57079632679 0.0 0.0
- joint j_wheel_2: origin xyz=0.0 0.0 -0.09835 rpy=1.57079632679 0.0 0.0 -> xyz=0.0 0.0 -0.14435 rpy=1.57079632679 0.0 0.0
- joint j_wheel_3: origin xyz=0.0 -0.0 -0.09835 rpy=1.57079632679 0.0 0.0 -> xyz=0.0 -0.0 -0.14435 rpy=1.57079632679 0.0 0.0
- joint j_wheel_4: origin xyz=0.0 0.0 -0.09835 rpy=1.57079632679 0.0 0.0 -> xyz=0.0 0.0 -0.14435 rpy=1.57079632679 0.0 0.0

File: centauro_urdf/urdf/centauro_capsule.urdf (robot description, URDF)
Before this commit: robot centauro, 94 links, 93 joints
Links:
- removed link D435_head_camera_accel_frame
- removed link D435_head_camera_accel_optical_frame
- removed link D435_head_camera_color_frame
- removed link D435_head_camera_color_optical_frame
- removed link D435_head_camera_depth_frame
- removed link D435_head_camera_depth_optical_frame
- removed link D435_head_camera_gyro_frame
- removed link D435_head_camera_gyro_optical_frame
- removed link D435_head_camera_left_ir_frame
- removed link D435_head_camera_left_ir_optical_frame
- removed link D435_head_camera_right_ir_frame
- removed link D435_head_camera_right_ir_optical_frame
- removed link D435i_camera_accel_frame
- removed link D435i_camera_accel_optical_frame
- removed link D435i_camera_color_frame
- removed link D435i_camera_color_optical_frame
- removed link D435i_camera_depth_frame
- removed link D435i_camera_depth_optical_frame
- removed link D435i_camera_gyro_frame
- removed link D435i_camera_gyro_optical_frame
- removed link D435i_camera_left_ir_frame
- removed link D435i_camera_left_ir_optical_frame
- removed link D435i_camera_right_ir_frame
- removed link D435i_camera_right_ir_optical_frame
- removed link T265_camera_accel_frame
- removed link T265_camera_accel_optical_frame
- removed link T265_camera_fisheye1_optical_frame
- removed link T265_camera_fisheye1_rgb_frame
- removed link T265_camera_fisheye2_optical_frame
- removed link T265_camera_fisheye2_rgb_frame
- removed link T265_camera_gyro_frame
- removed link T265_camera_gyro_optical_frame
- removed link T265_camera_link
- removed link T265_camera_pose_frame
- link D435_head_camera_link: geometry collision box size=0.02505 0.09 0.025; visual mesh filename=package://centauro_urdf/meshes/realsense/d435.dae
- link D435i_camera_link: geometry collision box size=0.02505 0.09 0.025; visual mesh filename=package://centauro_urdf/meshes/realsense/d435.dae
- link ankle1_2: geometry collision cylinder length=0.047884051265172006 radius=0.0781037; collision sphere radius=0.0781037
- link ankle1_4: geometry collision cylinder length=0.047884051265172006 radius=0.0781037; collision sphere radius=0.0781037
- link ankle2_1: mass 1.7656714 -> 2.440929; geometry collision cylinder length=0.13078435048455633 radius=0.08586; collision sphere radius=0.08586
- link ankle2_2: mass 1.7656714 -> 2.440929; geometry collision cylinder length=0.13078435048455633 radius=0.08586; collision sphere radius=0.08586
- link ankle2_3: mass 1.7656714 -> 2.440929; geometry collision cylinder length=0.13078435048455633 radius=0.08586; collision sphere radius=0.08586
- link ankle2_4: mass 1.7656714 -> 2.440929; geometry collision cylinder length=0.13078435048455633 radius=0.08586; collision sphere radius=0.08586
- link arm1_5: geometry collision cylinder length=0.08434739747702548 radius=0.0804108; collision sphere radius=0.0804108
- link arm2_5: geometry collision cylinder length=0.08434739747702548 radius=0.0804108; collision sphere radius=0.0804108
- link knee_1: geometry collision cylinder length=0.19275022460612404 radius=0.0664305; collision sphere radius=0.0664305
- link knee_2: geometry collision cylinder length=0.19275022460612404 radius=0.0664305; collision sphere radius=0.0664305
- link knee_3: geometry collision cylinder length=0.19275022460612404 radius=0.0664305; collision sphere radius=0.0664305
- link knee_4: geometry collision cylinder length=0.19275022460612404 radius=0.0664305; collision sphere radius=0.0664305
- link velodyne_calib: geometry collision sphere radius=0.0; visual mesh filename=package://velodyne_description/meshes/VLP16_scan.dae
- link wheel_1: mass 1.11164 -> 1.8569388; geometry collision cylinder length=0.0004424382093719415 radius=0.119659; collision sphere radius=0.119659
- link wheel_2: mass 1.11164 -> 1.8569388; geometry collision cylinder length=0.0004424382093719415 radius=0.119659; collision sphere radius=0.119659
- link wheel_3: mass 1.11164 -> 1.8569388; geometry collision cylinder length=0.0004424382093719415 radius=0.119659; collision sphere radius=0.119659
- link wheel_4: mass 1.11164 -> 1.8569388; geometry collision cylinder length=0.0004424382093719415 radius=0.119659; collision sphere radius=0.119659
Joints:
- removed joint D435_head_camera_accel_joint
- removed joint D435_head_camera_accel_optical_joint
- removed joint D435_head_camera_color_joint
- removed joint D435_head_camera_color_optical_joint
- removed joint D435_head_camera_depth_joint
- removed joint D435_head_camera_depth_optical_joint
- removed joint D435_head_camera_gyro_joint
- removed joint D435_head_camera_gyro_optical_joint
- removed joint D435_head_camera_left_ir_joint
- removed joint D435_head_camera_left_ir_optical_joint
- removed joint D435_head_camera_right_ir_joint
- removed joint D435_head_camera_right_ir_optical_joint
- removed joint D435i_camera_accel_joint
- removed joint D435i_camera_accel_optical_joint
- removed joint D435i_camera_color_joint
- removed joint D435i_camera_color_optical_joint
- removed joint D435i_camera_depth_joint
- removed joint D435i_camera_depth_optical_joint
- removed joint D435i_camera_gyro_joint
- removed joint D435i_camera_gyro_optical_joint
- removed joint D435i_camera_left_ir_joint
- removed joint D435i_camera_left_ir_optical_joint
- removed joint D435i_camera_right_ir_joint
- removed joint D435i_camera_right_ir_optical_joint
- removed joint T265_camera_accel_joint
- removed joint T265_camera_accel_optical_joint
- removed joint T265_camera_fisheye1_optical_joint
- removed joint T265_camera_fisheye1_rgb_joint
- removed joint T265_camera_fisheye2_optical_joint
- removed joint T265_camera_fisheye2_rgb_joint
- removed joint T265_camera_gyro_joint
- removed joint T265_camera_gyro_optical_joint
- removed joint T265_camera_link_joint
- removed joint T265_camera_pose_joint
- joint D435i_camera_joint: origin xyz=0.27187 0.0 0.0215997 rpy=0.0 0.5251508 0.0 -> xyz=0.272 0.0 0.084 rpy=0.0 0.54 0.0
- joint D435i_camera_link_joint: origin xyz=0.0 0.0175 0.0125 rpy=0.0 0.0 0.0 -> xyz=0.053 0.0 -0.035 rpy=0.0 0.005 -0.008
- joint j_wheel_1: origin xyz=0.0 -0.0 -0.09834999999999999 rpy=1.57079632679 0.0 0.0 -> xyz=0.0 -0.0 -0.14435 rpy=1.57079632679 0.0 0.0
- joint j_wheel_2: origin xyz=0.0 0.0 -0.09834999999999999 rpy=1.57079632679 0.0 0.0 -> xyz=0.0 0.0 -0.14435 rpy=1.57079632679 0.0 0.0
- joint j_wheel_3: origin xyz=0.0 -0.0 -0.09834999999999999 rpy=1.57079632679 0.0 0.0 -> xyz=0.0 -0.0 -0.14435 rpy=1.57079632679 0.0 0.0
- joint j_wheel_4: origin xyz=0.0 0.0 -0.09834999999999999 rpy=1.57079632679 0.0 0.0 -> xyz=0.0 0.0 -0.14435 rpy=1.57079632679 0.0 0.0
- joint velodyne_calib_base_mount_joint: origin xyz=0.0 0.0 0.0 rpy=0.0 0.0 0.0 -> xyz=-0.01 0.02 0.06 rpy=0.025 0.019 0.0

File: centauro_urdf/urdf/centauro_virtual_frame.urdf (robot description, URDF)
Before this commit: robot centauro, 66 links, 65 joints
Links:
- removed link D435_head_camera_bottom_screw_frame
- removed link D435_head_camera_link
- removed link D435i_camera_bottom_screw_frame
- removed link D435i_camera_link
- removed link arm1_1
- removed link arm1_2
- removed link arm1_3
- removed link arm1_4
- removed link arm1_5
- removed link arm1_6
- removed link arm1_8
- removed link arm2_1
- removed link arm2_2
- removed link arm2_3
- removed link arm2_4
- removed link arm2_5
- removed link arm2_6
- removed link arm2_8
- removed link ball1
- removed link ball1_tip
- removed link ball2
- removed link ball2_tip
- removed link d435_head_motor
- removed link neck_1
- removed link torso_2
- removed link velodyne_calib
- removed link velodyne_calib_base_link
- removed link velodyne_motor
- link ankle2_1: mass 1.7656714 -> 2.440929; geometry collision mesh filename=package://centauro_urdf/meshes/v2/collision/mesh_ankle-yaw_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 scale=0.001 -0.001 0.001; visual mesh filename=package://centauro_urdf/meshes/v2/mesh_ankle-yaw_wheel23.stl scale=0.001 -0.001 0.001
- link ankle2_2: mass 1.7656714 -> 2.440929; geometry collision mesh filename=package://centauro_urdf/meshes/v2/collision/mesh_ankle-yaw_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 scale=0.001 0.001 0.001; visual mesh filename=package://centauro_urdf/meshes/v2/mesh_ankle-yaw_wheel23.stl scale=0.001 0.001 0.001
- link ankle2_3: mass 1.7656714 -> 2.440929; geometry collision mesh filename=package://centauro_urdf/meshes/v2/collision/mesh_ankle-yaw_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 scale=0.001 -0.001 0.001; visual mesh filename=package://centauro_urdf/meshes/v2/mesh_ankle-yaw_wheel23.stl scale=0.001 -0.001 0.001
- link ankle2_4: mass 1.7656714 -> 2.440929; geometry collision mesh filename=package://centauro_urdf/meshes/v2/collision/mesh_ankle-yaw_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 scale=0.001 0.001 0.001; visual mesh filename=package://centauro_urdf/meshes/v2/mesh_ankle-yaw_wheel23.stl scale=0.001 0.001 0.001
- link wheel_1: mass 1.11164 -> 1.8569388; geometry collision mesh filename=package://centauro_urdf/meshes/v2/collision/mesh_wheel23.stl scale=0.001 0.001 -0.001; visual mesh filename=package://centauro_urdf/meshes/v2/mesh_wheel23.stl scale=0.001 0.001 -0.001
- link wheel_2: mass 1.11164 -> 1.8569388; geometry collision mesh filename=package://centauro_urdf/meshes/v2/collision/mesh_wheel23.stl scale=0.001 0.001 0.001; visual mesh filename=package://centauro_urdf/meshes/v2/mesh_wheel23.stl scale=0.001 0.001 0.001
- link wheel_3: mass 1.11164 -> 1.8569388; geometry collision mesh filename=package://centauro_urdf/meshes/v2/collision/mesh_wheel23.stl scale=0.001 0.001 -0.001; visual mesh filename=package://centauro_urdf/meshes/v2/mesh_wheel23.stl scale=0.001 0.001 -0.001
- link wheel_4: mass 1.11164 -> 1.8569388; geometry collision mesh filename=package://centauro_urdf/meshes/v2/collision/mesh_wheel23.stl scale=0.001 0.001 0.001; visual mesh filename=package://centauro_urdf/meshes/v2/mesh_wheel23.stl scale=0.001 0.001 0.001
Joints:
- removed joint D435_head_camera_joint
- removed joint D435_head_camera_link_joint
- removed joint D435i_camera_joint
- removed joint D435i_camera_link_joint
- removed joint d435_head_joint
- removed joint j_arm1_1
- removed joint j_arm1_2
- removed joint j_arm1_3
- removed joint j_arm1_4
- removed joint j_arm1_5
- removed joint j_arm1_6
- removed joint j_arm1_8
- removed joint j_arm2_1
- removed joint j_arm2_2
- removed joint j_arm2_3
- removed joint j_arm2_4
- removed joint j_arm2_5
- removed joint j_arm2_6
- removed joint j_arm2_8
- removed joint j_ball1_fixed
- removed joint j_ball1_tip
- removed joint j_ball2_fixed
- removed joint j_ball2_tip
- removed joint neck_base
- removed joint torso_yaw
- removed joint velodyne_calib_base_mount_joint
- removed joint velodyne_calib_base_scan_joint
- removed joint velodyne_joint
- joint hip_yaw_1: origin xyz=0.25 0.125 -0.0566 rpy=0.0 0.0 0.0 -> xyz=0.25 0.125 -0.056600000000000004 rpy=0.0 0.0 0.0
- joint hip_yaw_2: origin xyz=0.25 -0.125 -0.0566 rpy=0.0 0.0 0.0 -> xyz=0.25 -0.125 -0.056600000000000004 rpy=0.0 0.0 0.0
- joint hip_yaw_3: origin xyz=-0.25 0.125 -0.0566 rpy=0.0 0.0 0.0 -> xyz=-0.25 0.125 -0.056600000000000004 rpy=0.0 0.0 0.0
- joint hip_yaw_4: origin xyz=-0.25 -0.125 -0.0566 rpy=0.0 0.0 0.0 -> xyz=-0.25 -0.125 -0.056600000000000004 rpy=0.0 0.0 0.0
- joint j_wheel_1: origin xyz=0.0 -0.0 -0.09835 rpy=1.57079632679 0.0 0.0 -> xyz=0.0 -0.0 -0.14435 rpy=1.57079632679 0.0 0.0
- joint j_wheel_2: origin xyz=0.0 0.0 -0.09835 rpy=1.57079632679 0.0 0.0 -> xyz=0.0 0.0 -0.14435 rpy=1.57079632679 0.0 0.0
- joint j_wheel_3: origin xyz=0.0 -0.0 -0.09835 rpy=1.57079632679 0.0 0.0 -> xyz=0.0 -0.0 -0.14435 rpy=1.57079632679 0.0 0.0
- joint j_wheel_4: origin xyz=0.0 0.0 -0.09835 rpy=1.57079632679 0.0 0.0 -> xyz=0.0 0.0 -0.14435 rpy=1.57079632679 0.0 0.0

File: centauro_urdf/urdf/config/centauro_virtual_frame.urdf.xacro (robot description, xacro)
@@ -3,16 +3,14 @@
     <xacro:property name="model_name" value="centauro" />
     <xacro:property name="model_version" value="0.1" />
-    <!-- command line arguments -->
-    <xacro:arg name="add_legs" default="true"/>
-    <xacro:arg name="add_upper_body" default="true"/>
     <!-- ************SELECT PARTS*************-->
     <!-- *************************************-->
-    <xacro:property name="ADD_LEGS" value="$(arg add_legs)" />
-    <xacro:property name="ADD_UPPER_BODY" value="$(arg add_upper_body)" />
+    <xacro:property name="ADD_LEGS" value="true" />
+    <xacro:property name="ADD_UPPER_BODY" value="false" />
     <xacro:property name="ADD_BALL_END_EFFECTOR" value="true" />
-    <xacro:property name="ADD_FLOATING_BASE" value="$(arg add_legs)" />
+    <xacro:property name="ADD_FLOATING_BASE" value="true" />
     <xacro:property name="ADD_VIRTUAL_FRAME" value="true" />
     <xacro:property name="USE_STICKS" value="false" />
-    <xacro:property name="ADD_VELODYNE" value="true" />
+    <xacro:property name="USE_WHEEL_23" value="true" />
+    <xacro:property name="ADD_VELODYNE" value="false" />
     <xacro:property name="ADD_D435I_HEAD" value="false" />
     <xacro:property name="ADD_D435I_BASE" value="false" />
