Commit message: merge big_wheels into ioannis-devel and regenerate urdf/srdf

File: centauro_urdf/urdf/centauro.urdf (robot description, URDF)
Before this commit: robot centauro, 94 links, 93 joints
Links:
- link ankle2_1: mass 1.7656714 -> 2.440929; geometry collision mesh filename=package://centauro_urdf/meshes/v2/collision/mesh_ankle-yaw_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 scale=0.001 -0.001 0.001; visual mesh filename=package://centauro_urdf/meshes/v2/mesh_ankle-yaw_wheel23.stl scale=0.001 -0.001 0.001
- link ankle2_2: mass 1.7656714 -> 2.440929; geometry collision mesh filename=package://centauro_urdf/meshes/v2/collision/mesh_ankle-yaw_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 scale=0.001 0.001 0.001; visual mesh filename=package://centauro_urdf/meshes/v2/mesh_ankle-yaw_wheel23.stl scale=0.001 0.001 0.001
- link ankle2_3: mass 1.7656714 -> 2.440929; geometry collision mesh filename=package://centauro_urdf/meshes/v2/collision/mesh_ankle-yaw_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 scale=0.001 -0.001 0.001; visual mesh filename=package://centauro_urdf/meshes/v2/mesh_ankle-yaw_wheel23.stl scale=0.001 -0.001 0.001
- link ankle2_4: mass 1.7656714 -> 2.440929; geometry collision mesh filename=package://centauro_urdf/meshes/v2/collision/mesh_ankle-yaw_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 scale=0.001 0.001 0.001; visual mesh filename=package://centauro_urdf/meshes/v2/mesh_ankle-yaw_wheel23.stl scale=0.001 0.001 0.001
- link wheel_1: mass 1.11164 -> 1.8569388; geometry collision mesh filename=package://centauro_urdf/meshes/v2/collision/mesh_wheel23.stl scale=0.001 0.001 -0.001; visual mesh filename=package://centauro_urdf/meshes/v2/mesh_wheel23.stl scale=0.001 0.001 -0.001
- link wheel_2: mass 1.11164 -> 1.8569388; geometry collision mesh filename=package://centauro_urdf/meshes/v2/collision/mesh_wheel23.stl scale=0.001 0.001 0.001; visual mesh filename=package://centauro_urdf/meshes/v2/mesh_wheel23.stl scale=0.001 0.001 0.001
- link wheel_3: mass 1.11164 -> 1.8569388; geometry collision mesh filename=package://centauro_urdf/meshes/v2/collision/mesh_wheel23.stl scale=0.001 0.001 -0.001; visual mesh filename=package://centauro_urdf/meshes/v2/mesh_wheel23.stl scale=0.001 0.001 -0.001
- link wheel_4: mass 1.11164 -> 1.8569388; geometry collision mesh filename=package://centauro_urdf/meshes/v2/collision/mesh_wheel23.stl scale=0.001 0.001 0.001; visual mesh filename=package://centauro_urdf/meshes/v2/mesh_wheel23.stl scale=0.001 0.001 0.001
Joints:
- joint contact_joint_1: origin xyz=0 0 -0.176 rpy=0 0 0 -> xyz=0 0 -0.26835 rpy=0 0 0
- joint contact_joint_2: origin xyz=0 0 -0.176 rpy=0 0 0 -> xyz=0 0 -0.26835 rpy=0 0 0
- joint contact_joint_3: origin xyz=0 0 -0.176 rpy=0 0 0 -> xyz=0 0 -0.26835 rpy=0 0 0
- joint contact_joint_4: origin xyz=0 0 -0.176 rpy=0 0 0 -> xyz=0 0 -0.26835 rpy=0 0 0
- joint j_wheel_1: origin xyz=0.0 -0.0 -0.09834999999999999 rpy=1.57079632679 0.0 0.0 -> xyz=0.0 -0.0 -0.14435 rpy=1.57079632679 0.0 0.0
- joint j_wheel_2: origin xyz=0.0 0.0 -0.09834999999999999 rpy=1.57079632679 0.0 0.0 -> xyz=0.0 0.0 -0.14435 rpy=1.57079632679 0.0 0.0
- joint j_wheel_3: origin xyz=0.0 -0.0 -0.09834999999999999 rpy=1.57079632679 0.0 0.0 -> xyz=0.0 -0.0 -0.14435 rpy=1.57079632679 0.0 0.0
- joint j_wheel_4: origin xyz=0.0 0.0 -0.09834999999999999 rpy=1.57079632679 0.0 0.0 -> xyz=0.0 0.0 -0.14435 rpy=1.57079632679 0.0 0.0

File: centauro_urdf/urdf/centauro_capsule.urdf (robot description, URDF)
Before this commit: robot centauro, 94 links, 93 joints
Links:
- link ankle2_1: mass 1.7656714 -> 2.440929; geometry collision cylinder length=0.13078435048455633 radius=0.08586; collision sphere radius=0.08586
- link ankle2_2: mass 1.7656714 -> 2.440929; geometry collision cylinder length=0.13078435048455633 radius=0.08586; collision sphere radius=0.08586
- link ankle2_3: mass 1.7656714 -> 2.440929; geometry collision cylinder length=0.13078435048455633 radius=0.08586; collision sphere radius=0.08586
- link ankle2_4: mass 1.7656714 -> 2.440929; geometry collision cylinder length=0.13078435048455633 radius=0.08586; collision sphere radius=0.08586
- link wheel_1: mass 1.11164 -> 1.8569388; geometry collision cylinder length=0.0004424382093719415 radius=0.119659; collision sphere radius=0.119659
- link wheel_2: mass 1.11164 -> 1.8569388; geometry collision cylinder length=0.0004424382093719415 radius=0.119659; collision sphere radius=0.119659
- link wheel_3: mass 1.11164 -> 1.8569388; geometry collision cylinder length=0.0004424382093719415 radius=0.119659; collision sphere radius=0.119659
- link wheel_4: mass 1.11164 -> 1.8569388; geometry collision cylinder length=0.0004424382093719415 radius=0.119659; collision sphere radius=0.119659
Joints:
- joint contact_joint_1: origin xyz=0.0 0.0 -0.176 rpy=0.0 0.0 0.0 -> xyz=0.0 0.0 -0.26835 rpy=0.0 0.0 0.0
- joint contact_joint_2: origin xyz=0.0 0.0 -0.176 rpy=0.0 0.0 0.0 -> xyz=0.0 0.0 -0.26835 rpy=0.0 0.0 0.0
- joint contact_joint_3: origin xyz=0.0 0.0 -0.176 rpy=0.0 0.0 0.0 -> xyz=0.0 0.0 -0.26835 rpy=0.0 0.0 0.0
- joint contact_joint_4: origin xyz=0.0 0.0 -0.176 rpy=0.0 0.0 0.0 -> xyz=0.0 0.0 -0.26835 rpy=0.0 0.0 0.0
- joint j_wheel_1: origin xyz=0.0 -0.0 -0.09834999999999999 rpy=1.57079632679 0.0 0.0 -> xyz=0.0 -0.0 -0.14435 rpy=1.57079632679 0.0 0.0
- joint j_wheel_2: origin xyz=0.0 0.0 -0.09834999999999999 rpy=1.57079632679 0.0 0.0 -> xyz=0.0 0.0 -0.14435 rpy=1.57079632679 0.0 0.0
- joint j_wheel_3: origin xyz=0.0 -0.0 -0.09834999999999999 rpy=1.57079632679 0.0 0.0 -> xyz=0.0 -0.0 -0.14435 rpy=1.57079632679 0.0 0.0
- joint j_wheel_4: origin xyz=0.0 0.0 -0.09834999999999999 rpy=1.57079632679 0.0 0.0 -> xyz=0.0 0.0 -0.14435 rpy=1.57079632679 0.0 0.0

File: centauro_urdf/urdf/centauro_dagana_fixed.urdf (robot description, URDF)
Before this commit: robot centauro, 95 links, 94 joints
Links:
- link ankle2_1: mass 1.7656714 -> 2.440929; geometry collision mesh filename=package://centauro_urdf/meshes/v2/collision/mesh_ankle-yaw_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 scale=0.001 -0.001 0.001; visual mesh filename=package://centauro_urdf/meshes/v2/mesh_ankle-yaw_wheel23.stl scale=0.001 -0.001 0.001
- link ankle2_2: mass 1.7656714 -> 2.440929; geometry collision mesh filename=package://centauro_urdf/meshes/v2/collision/mesh_ankle-yaw_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 scale=0.001 0.001 0.001; visual mesh filename=package://centauro_urdf/meshes/v2/mesh_ankle-yaw_wheel23.stl scale=0.001 0.001 0.001
- link ankle2_3: mass 1.7656714 -> 2.440929; geometry collision mesh filename=package://centauro_urdf/meshes/v2/collision/mesh_ankle-yaw_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 scale=0.001 -0.001 0.001; visual mesh filename=package://centauro_urdf/meshes/v2/mesh_ankle-yaw_wheel23.stl scale=0.001 -0.001 0.001
- link ankle2_4: mass 1.7656714 -> 2.440929; geometry collision mesh filename=package://centauro_urdf/meshes/v2/collision/mesh_ankle-yaw_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 scale=0.001 0.001 0.001; visual mesh filename=package://centauro_urdf/meshes/v2/mesh_ankle-yaw_wheel23.stl scale=0.001 0.001 0.001
- link wheel_1: mass 1.11164 -> 1.8569388; geometry collision mesh filename=package://centauro_urdf/meshes/v2/collision/mesh_wheel23.stl scale=0.001 0.001 -0.001; visual mesh filename=package://centauro_urdf/meshes/v2/mesh_wheel23.stl scale=0.001 0.001 -0.001
- link wheel_2: mass 1.11164 -> 1.8569388; geometry collision mesh filename=package://centauro_urdf/meshes/v2/collision/mesh_wheel23.stl scale=0.001 0.001 0.001; visual mesh filename=package://centauro_urdf/meshes/v2/mesh_wheel23.stl scale=0.001 0.001 0.001
- link wheel_3: mass 1.11164 -> 1.8569388; geometry collision mesh filename=package://centauro_urdf/meshes/v2/collision/mesh_wheel23.stl scale=0.001 0.001 -0.001; visual mesh filename=package://centauro_urdf/meshes/v2/mesh_wheel23.stl scale=0.001 0.001 -0.001
- link wheel_4: mass 1.11164 -> 1.8569388; geometry collision mesh filename=package://centauro_urdf/meshes/v2/collision/mesh_wheel23.stl scale=0.001 0.001 0.001; visual mesh filename=package://centauro_urdf/meshes/v2/mesh_wheel23.stl scale=0.001 0.001 0.001
Joints:
- joint contact_joint_1: origin xyz=0 0 -0.176 rpy=0 0 0 -> xyz=0 0 -0.26835 rpy=0 0 0
- joint contact_joint_2: origin xyz=0 0 -0.176 rpy=0 0 0 -> xyz=0 0 -0.26835 rpy=0 0 0
- joint contact_joint_3: origin xyz=0 0 -0.176 rpy=0 0 0 -> xyz=0 0 -0.26835 rpy=0 0 0
- joint contact_joint_4: origin xyz=0 0 -0.176 rpy=0 0 0 -> xyz=0 0 -0.26835 rpy=0 0 0
- joint dagana_2_mount_joint: origin xyz=0. 0.05 -0.08 rpy=0. 3.14159265359 3.14159265359 -> xyz=0. 0.05 -0.08 rpy=0. 3.14159265359 0
- joint j_wheel_1: origin xyz=0.0 -0.0 -0.09834999999999999 rpy=1.57079632679 0.0 0.0 -> xyz=0.0 -0.0 -0.14435 rpy=1.57079632679 0.0 0.0
- joint j_wheel_2: origin xyz=0.0 0.0 -0.09834999999999999 rpy=1.57079632679 0.0 0.0 -> xyz=0.0 0.0 -0.14435 rpy=1.57079632679 0.0 0.0
- joint j_wheel_3: origin xyz=0.0 -0.0 -0.09834999999999999 rpy=1.57079632679 0.0 0.0 -> xyz=0.0 -0.0 -0.14435 rpy=1.57079632679 0.0 0.0
- joint j_wheel_4: origin xyz=0.0 0.0 -0.09834999999999999 rpy=1.57079632679 0.0 0.0 -> xyz=0.0 0.0 -0.14435 rpy=1.57079632679 0.0 0.0

File: centauro_urdf/urdf/centauro_virtual_frame.urdf (robot description, URDF)
Before this commit: robot centauro, 66 links, 65 joints
Links:
- removed link velodyne_calib
- removed link velodyne_calib_base_link
- link ankle2_1: mass 1.7656714 -> 2.440929; geometry collision mesh filename=package://centauro_urdf/meshes/v2/collision/mesh_ankle-yaw_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 scale=0.001 -0.001 0.001; visual mesh filename=package://centauro_urdf/meshes/v2/mesh_ankle-yaw_wheel23.stl scale=0.001 -0.001 0.001
- link ankle2_2: mass 1.7656714 -> 2.440929; geometry collision mesh filename=package://centauro_urdf/meshes/v2/collision/mesh_ankle-yaw_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 scale=0.001 0.001 0.001; visual mesh filename=package://centauro_urdf/meshes/v2/mesh_ankle-yaw_wheel23.stl scale=0.001 0.001 0.001
- link ankle2_3: mass 1.7656714 -> 2.440929; geometry collision mesh filename=package://centauro_urdf/meshes/v2/collision/mesh_ankle-yaw_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 scale=0.001 -0.001 0.001; visual mesh filename=package://centauro_urdf/meshes/v2/mesh_ankle-yaw_wheel23.stl scale=0.001 -0.001 0.001
- link ankle2_4: mass 1.7656714 -> 2.440929; geometry collision mesh filename=package://centauro_urdf/meshes/v2/collision/mesh_ankle-yaw_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 scale=0.001 0.001 0.001; visual mesh filename=package://centauro_urdf/meshes/v2/mesh_ankle-yaw_wheel23.stl scale=0.001 0.001 0.001
- link wheel_1: mass 1.11164 -> 1.8569388; geometry collision mesh filename=package://centauro_urdf/meshes/v2/collision/mesh_wheel23.stl scale=0.001 0.001 -0.001; visual mesh filename=package://centauro_urdf/meshes/v2/mesh_wheel23.stl scale=0.001 0.001 -0.001
- link wheel_2: mass 1.11164 -> 1.8569388; geometry collision mesh filename=package://centauro_urdf/meshes/v2/collision/mesh_wheel23.stl scale=0.001 0.001 0.001; visual mesh filename=package://centauro_urdf/meshes/v2/mesh_wheel23.stl scale=0.001 0.001 0.001
- link wheel_3: mass 1.11164 -> 1.8569388; geometry collision mesh filename=package://centauro_urdf/meshes/v2/collision/mesh_wheel23.stl scale=0.001 0.001 -0.001; visual mesh filename=package://centauro_urdf/meshes/v2/mesh_wheel23.stl scale=0.001 0.001 -0.001
- link wheel_4: mass 1.11164 -> 1.8569388; geometry collision mesh filename=package://centauro_urdf/meshes/v2/collision/mesh_wheel23.stl scale=0.001 0.001 0.001; visual mesh filename=package://centauro_urdf/meshes/v2/mesh_wheel23.stl scale=0.001 0.001 0.001
Joints:
- removed joint velodyne_calib_base_mount_joint
- removed joint velodyne_calib_base_scan_joint
- joint contact_joint_1: origin xyz=0 0 -0.176 rpy=0 0 0 -> xyz=0 0 -0.26835 rpy=0 0 0
- joint contact_joint_2: origin xyz=0 0 -0.176 rpy=0 0 0 -> xyz=0 0 -0.26835 rpy=0 0 0
- joint contact_joint_3: origin xyz=0 0 -0.176 rpy=0 0 0 -> xyz=0 0 -0.26835 rpy=0 0 0
- joint contact_joint_4: origin xyz=0 0 -0.176 rpy=0 0 0 -> xyz=0 0 -0.26835 rpy=0 0 0
- joint j_wheel_1: origin xyz=0.0 -0.0 -0.09834999999999999 rpy=1.57079632679 0.0 0.0 -> xyz=0.0 -0.0 -0.14435 rpy=1.57079632679 0.0 0.0
- joint j_wheel_2: origin xyz=0.0 0.0 -0.09834999999999999 rpy=1.57079632679 0.0 0.0 -> xyz=0.0 0.0 -0.14435 rpy=1.57079632679 0.0 0.0
- joint j_wheel_3: origin xyz=0.0 -0.0 -0.09834999999999999 rpy=1.57079632679 0.0 0.0 -> xyz=0.0 -0.0 -0.14435 rpy=1.57079632679 0.0 0.0
- joint j_wheel_4: origin xyz=0.0 0.0 -0.09834999999999999 rpy=1.57079632679 0.0 0.0 -> xyz=0.0 0.0 -0.14435 rpy=1.57079632679 0.0 0.0

File: centauro_urdf/urdf/config/centauro.urdf.xacro (robot description, xacro)
@@ -5,4 +5,5 @@
 <!-- command line arguments -->
 <xacro:arg name="legs" default="true"/>
+<xacro:arg name="big_wheel" default="true"/>
 <xacro:arg name="upper_body" default="true"/>
 <xacro:arg name="velodyne" default="true"/>
@@ -40,4 +41,5 @@
 <xacro:property name="ADD_VIRTUAL_FRAME" value="$(arg virtual_frame)" />
 <xacro:property name="USE_STICKS" value="false" />
+<xacro:property name="USE_WHEEL_23" value="$(arg big_wheel)" />
 <xacro:property name="ADD_VELODYNE" value="$(arg velodyne)" />
 <xacro:property name="ADD_D435I_HEAD" value="$(arg d435i_head)" />

File: centauro_urdf/urdf/config/centauro_virtual_frame.urdf.xacro (robot description, xacro)
@@ -23,5 +23,8 @@
     <xacro:property name="ADD_VIRTUAL_FRAME" value="true" />
     <xacro:property name="USE_STICKS" value="false" />
-    <xacro:property name="ADD_VELODYNE" value="true" />
+    <xacro:property name="USE_WHEEL_23" value="true" />
+    <xacro:property name="END_EFFECTOR_LEFT" value="ball" />
+    <xacro:property name="END_EFFECTOR_RIGHT" value="ball" />
+    <xacro:property name="ADD_VELODYNE" value="false" />
     <xacro:property name="ADD_D435I_HEAD" value="false" />
     <xacro:property name="ADD_D435I_BASE" value="false" />
