Commit message: merge big_wheels into ioannis-devel and regenerate urdf/srdf

File: centauro_urdf/urdf/parts/centauro_leg.urdf.xacro (robot description, xacro)
@@ -1,4 +1,6 @@
 <?xml version="1.0"?>
 <robot xmlns:xacro="http://ros.org/wiki/xacro">
+<xacro:include filename="$(find centauro_urdf)/urdf/parts/wheel.urdf.xacro"/>
+<xacro:include filename="$(find centauro_urdf)/urdf/parts/wheel23.urdf.xacro"/>
 <!-- macro legs -->
 <xacro:macro name="centauro_leg" params="leg_num origin_x origin_y mirror">
@@ -43,115 +45,92 @@
 </link>
 <xacro:if value="${USE_STICKS}">
-<link name="knee_${leg_num}">
-<inertial>
-	<mass value="${1.1927236}"/>
-    <origin xyz="${1.9572282e+02*mmTom} ${-1.4549221e+01*mmTom} ${-2.0785942e+01*mmTom}" rpy="0.0 0.0 0.0"/>
-	<!--origin xyz="${1.4549221e+01*mmTom} ${-2.0785942e+01*mmTom} ${-1.9572282e+02*mmTom}" rpy="0.0 0.0 0.0"/-->
-	<!--inertia ixx="${3.5313402e+04*mm2Tom2}"  ixy="${0.0*mm2Tom2}"  ixz="${1.1029574e-01*mm2Tom2}" iyy="${3.5530025e+04*mm2Tom2}" iyz="${-6.0307457e+02*mm2Tom2}" izz="${1.3302597e+03*mm2Tom2}" /-->
-    <inertia ixx="${1.3302597e+03*mm2Tom2}"  ixy="${6.0307457e+02*mm2Tom2}"  ixz="${0.0*mm2Tom2}" iyy="${3.5313402e+04*mm2Tom2}" iyz="${-1.1029574e-01*mm2Tom2}" izz="${3.5530025e+04*mm2Tom2}" />
-</inertial>
-<visual>
-      <origin xyz="0 0 0" rpy="${PI_2} 0 ${-PI_2}"/>
-      <material name="black"/>
-      <geometry name="${leg_num}_stick_visual">
-        <mesh filename="package://centauro_urdf/meshes/front_right_stick.stl" scale="${mmTom} ${mmTom} ${mmTom}"/>
-      </geometry>
-</visual>
-<collision>
-      <origin xyz="0 0 0" rpy="${PI_2} 0 ${-PI_2}"/>
-      <geometry name="${leg_num}_stick_collision">
-        <mesh filename="package://centauro_urdf/meshes/simple/front_right_stick.stl" scale="${mmTom} ${mmTom} ${mmTom}"/>
-      </geometry>
-</collision>
-</link>
+   <link name="knee_${leg_num}">
+   <inertial>
+      <mass value="${1.1927236}"/>
+      <origin xyz="${1.9572282e+02*mmTom} ${-1.4549221e+01*mmTom} ${-2.0785942e+01*mmTom}" rpy="0.0 0.0 0.0"/>
+      <!--origin xyz="${1.4549221e+01*mmTom} ${-2.0785942e+01*mmTom} ${-1.9572282e+02*mmTom}" rpy="0.0 0.0 0.0"/-->
+      <!--inertia ixx="${3.5313402e+04*mm2Tom2}"  ixy="${0.0*mm2Tom2}"  ixz="${1.1029574e-01*mm2Tom2}" iyy="${3.5530025e+04*mm2Tom2}" iyz="${-6.0307457e+02*mm2Tom2}" izz="${1.3302597e+03*mm2Tom2}" /-->
+      <inertia ixx="${1.3302597e+03*mm2Tom2}"  ixy="${6.0307457e+02*mm2Tom2}"  ixz="${0.0*mm2Tom2}" iyy="${3.5313402e+04*mm2Tom2}" iyz="${-1.1029574e-01*mm2Tom2}" izz="${3.5530025e+04*mm2Tom2}" />
+   </inertial>
+   <visual>
+         <origin xyz="0 0 0" rpy="${PI_2} 0 ${-PI_2}"/>
+         <material name="black"/>
+         <geometry name="${leg_num}_stick_visual">
+         <mesh filename="package://centauro_urdf/meshes/front_right_stick.stl" scale="${mmTom} ${mmTom} ${mmTom}"/>
+         </geometry>
+   </visual>
+   <collision>
+         <origin xyz="0 0 0" rpy="${PI_2} 0 ${-PI_2}"/>
+         <geometry name="${leg_num}_stick_collision">
+         <mesh filename="package://centauro_urdf/meshes/simple/front_right_stick.stl" scale="${mmTom} ${mmTom} ${mmTom}"/>
+         </geometry>
+   </collision>
+   </link>
 </xacro:if>
 <xacro:unless value="${USE_STICKS}">
-<link name="knee_${leg_num}">
-	<inertial>
-		<origin xyz="${Leg_3_x} ${Leg_3_y} ${mirror*Leg_3_z}"/>
-		<mass value="${Leg_3_mass}"/>  <!-- org: 3.5, foot un modeled-->
-		<inertia ixx="${Leg_3_xx}" ixy="${Leg_3_xy}" ixz="${mirror*Leg_3_xz}" iyy="${Leg_3_yy}" iyz="${mirror*Leg_3_yz}" izz="${Leg_3_zz}"/>
-	</inertial>
-   <visual>
-      <origin xyz="0.0 0.0 0.0"  rpy="0.0 0.0 0.0"/>
-      <geometry>
-         <mesh filename="package://centauro_urdf/meshes/v2/knee.stl" scale="0.001 0.001 ${mirror*0.001}" />
-      </geometry>
-      <material name="dark_grey"/>
-   </visual>
-   <collision>
-      <origin xyz="0.0 0.0 0.0"  rpy="0.0 0.0 0.0"/>
-      <geometry>
-         <mesh filename="package://centauro_urdf/meshes/v2/collision/knee.stl" scale="0.001 0.001 ${mirror*0.001}" />
-      </geometry>
-   </collision>
-</link>
-<link name="ankle1_${leg_num}">
-	<inertial>
-		<origin xyz="${Ankle_1_x} ${Ankle_1_y} ${mirror*Ankle_1_z}"/>
-		<mass value="${Ankle_1_mass}"/>  <!-- org: 3.5, foot un modeled-->
-		<inertia ixx="${Ankle_1_xx}" ixy="${Ankle_1_xy}" ixz="${mirror*Ankle_1_xz}" iyy="${Ankle_1_yy}" iyz="${mirror*Ankle_1_yz}" izz="${Ankle_1_zz}"/>
-	</inertial>
-   <visual>
-      <origin xyz="0.0 0.0 0.0"  rpy="0.0 0.0 0.0"/>
-      <geometry>
-         <mesh filename="package://centauro_urdf/meshes/v2/ankle-pitch.stl" scale="0.001 0.001 ${mirror*0.001}" />
-      </geometry>
-   </visual>
-   <collision>
-      <origin xyz="0.0 0.0 0.0"  rpy="0.0 0.0 0.0"/>
-      <geometry>
-         <mesh filename="package://centauro_urdf/meshes/v2/collision/ankle-pitch.stl" scale="0.001 0.001 ${mirror*0.001}" />
-      </geometry>
-   </collision>
-</link>
-<link name="ankle2_${leg_num}">
-	<inertial>
-		<origin xyz="${Ankle_2_x} ${mirror*Ankle_2_y} ${Ankle_2_z}"/>
-		<mass value="${Ankle_2_mass}"/>  <!-- org: 3.5, foot un modeled-->
-		<inertia ixx="${Ankle_2_xx}" ixy="${mirror*Ankle_2_xy}" ixz="${Ankle_2_xz}" iyy="${Ankle_2_yy}" iyz="${mirror*Ankle_2_yz}" izz="${Ankle_2_zz}"/>
-	</inertial>
-   <visual>
-      <origin xyz="0.0 0.0 0.0"  rpy="0.0 0.0 0.0"/>
-      <geometry>
-         <mesh filename="package://centauro_urdf/meshes/v2/ankle-yaw.stl" scale="0.001 ${mirror*0.001} 0.001" />
-      </geometry>
-      <material name="dark_grey"/>
-   </visual>
-   <collision>
-      <origin xyz="0.0 0.0 0.0"  rpy="0.0 0.0 0.0"/>
-      <geometry>
-         <mesh filename="package://centauro_urdf/meshes/v2/collision/ankle-yaw.stl" scale="0.001 ${mirror*0.001} 0.001" />
-      </geometry>
-   </collision>
-</link>
-<link name="wheel_${leg_num}">
-	<inertial>
-		<origin xyz="${Wheel_x} ${Wheel_y} ${mirror*Wheel_z}"/>
-		<mass value="${Wheel_mass}"/>
-		<inertia ixx="${Wheel_xx}" ixy="${Wheel_xy}" ixz="${mirror*Wheel_xz}" iyy="${Wheel_yy}" iyz="${mirror*Wheel_yz}" izz="${Wheel_zz}"/>
-	</inertial>
-   <visual>
-      <origin xyz="0.0 0.0 0.0"  rpy="0.0 0.0 0.0"/>
-      <geometry>
-         <mesh filename="package://centauro_urdf/meshes/v2/wheel.stl" scale="0.001 0.001 ${mirror*0.001}" />
-      </geometry>
-      <material name="black"/>
-   </visual>
-	<collision>
-		<origin xyz="0 0 0" rpy="0 0 0"/>
-		<geometry>
-			<cylinder length="0.11" radius="0.078"/>
-      </geometry>
-	</collision>
-</link>
+   <link name="knee_${leg_num}">
+      <inertial>
+         <origin xyz="${Leg_3_x} ${Leg_3_y} ${mirror*Leg_3_z}"/>
+         <mass value="${Leg_3_mass}"/>  <!-- org: 3.5, foot un modeled-->
+         <inertia ixx="${Leg_3_xx}" ixy="${Leg_3_xy}" ixz="${mirror*Leg_3_xz}" iyy="${Leg_3_yy}" iyz="${mirror*Leg_3_yz}" izz="${Leg_3_zz}"/>
+      </inertial>
+      <visual>
+         <origin xyz="0.0 0.0 0.0"  rpy="0.0 0.0 0.0"/>
+         <geometry>
+            <mesh filename="package://centauro_urdf/meshes/v2/knee.stl" scale="0.001 0.001 ${mirror*0.001}" />
+         </geometry>
+         <material name="dark_grey"/>
+      </visual>
+      <collision>
+         <origin xyz="0.0 0.0 0.0"  rpy="0.0 0.0 0.0"/>
+         <geometry>
+            <mesh filename="package://centauro_urdf/meshes/v2/collision/knee.stl" scale="0.001 0.001 ${mirror*0.001}" />
+         </geometry>
+      </collision>
+   </link>
+   <link name="ankle1_${leg_num}">
+      <inertial>
+         <origin xyz="${Ankle_1_x} ${Ankle_1_y} ${mirror*Ankle_1_z}"/>
+         <mass value="${Ankle_1_mass}"/>  <!-- org: 3.5, foot un modeled-->
+         <inertia ixx="${Ankle_1_xx}" ixy="${Ankle_1_xy}" ixz="${mirror*Ankle_1_xz}" iyy="${Ankle_1_yy}" iyz="${mirror*Ankle_1_yz}" izz="${Ankle_1_zz}"/>
+      </inertial>
+      <visual>
+         <origin xyz="0.0 0.0 0.0"  rpy="0.0 0.0 0.0"/>
+         <geometry>
+            <mesh filename="package://centauro_urdf/meshes/v2/ankle-pitch.stl" scale="0.001 0.001 ${mirror*0.001}" />
+         </geometry>
+      </visual>
+      <collision>
+         <origin xyz="0.0 0.0 0.0"  rpy="0.0 0.0 0.0"/>
+         <geometry>
+            <mesh filename="package://centauro_urdf/meshes/v2/collision/ankle-pitch.stl" scale="0.001 0.001 ${mirror*0.001}" />
+         </geometry>
+      </collision>
+   </link>
+   <!-- New centauro wheel -->
+   <xacro:if value="${USE_WHEEL_23}">
+      <xacro:centauro_wheel23 leg_num="${leg_num}" mirror="${mirror}"/>
+   </xacro:if>
+   <!-- Old centauro wheel -->
+   <xacro:unless value="${USE_WHEEL_23}">
+      <xacro:centauro_wheel leg_num="${leg_num}" mirror="${mirror}"/>
+   </xacro:unless>
 </xacro:unless>
-<!-- *****************************-->
+<!-- *********** CONTACT FRAME ******************-->
 <link name="contact_${leg_num}"/>
-<joint name="contact_joint_${leg_num}" type="fixed">
-	<parent link="ankle2_${leg_num}"/>
-	<child link="contact_${leg_num}"/>
-	<origin xyz="0 0 -0.176" rpy="0 0 0"/>
-</joint>
+<xacro:if value="${USE_WHEEL_23}">
+	<joint name="contact_joint_${leg_num}" type="fixed">
+		<parent link="ankle2_${leg_num}"/>
+		<child link="contact_${leg_num}"/>
+		<origin xyz="0 0 ${Wheel23_Oz - Wheel23_radius}" rpy="0 0 0"/>
+	</joint>
+</xacro:if>
+<xacro:unless value="${USE_WHEEL_23}">
+	<joint name="contact_joint_${leg_num}" type="fixed">
+		<parent link="ankle2_${leg_num}"/>
+		<child link="contact_${leg_num}"/>
+		<origin xyz="0 0 ${Wheel_Oz - Wheel_radius}" rpy="0 0 0"/>
+	</joint>
+</xacro:unless>
 <!-- ******************************** -->
 <joint name="hip_yaw_${leg_num}" type="revolute">
@@ -170,41 +149,34 @@
 </joint>
 <xacro:if  value="${USE_STICKS}">
-<joint name="knee_pitch_${leg_num}" type="revolute">
-	<parent link="hip2_${leg_num}"/>
-	<child link="knee_${leg_num}"/>
-	<origin xyz="${Leg_3_Ox} ${Leg_3_Oy} ${Leg_3_Oz}" rpy="${Leg_3_roll} ${Leg_3_pitch} ${Leg_3_yaw}"/>
-	<axis xyz="0 0 1"/>
-   <limit lower="${knee_pitch_lower[leg_num-1]}" upper="${knee_pitch_upper[leg_num-1]}" effort="${motor_A_effort}" velocity="${motor_A_velocity}"/> <!-- 200 Nm, 1 rad/s-->
-</joint>
+   <joint name="knee_pitch_${leg_num}" type="revolute">
+      <parent link="hip2_${leg_num}"/>
+      <child link="knee_${leg_num}"/>
+      <origin xyz="${Leg_3_Ox} ${Leg_3_Oy} ${Leg_3_Oz}" rpy="${Leg_3_roll} ${Leg_3_pitch} ${Leg_3_yaw}"/>
+      <axis xyz="0 0 1"/>
+      <limit lower="${knee_pitch_lower[leg_num-1]}" upper="${knee_pitch_upper[leg_num-1]}" effort="${motor_A_effort}" velocity="${motor_A_velocity}"/> <!-- 200 Nm, 1 rad/s-->
+   </joint>
 </xacro:if>
 <xacro:unless value="${USE_STICKS}">
-<joint name="knee_pitch_${leg_num}" type="revolute">
-	<parent link="hip2_${leg_num}"/>
-	<child link="knee_${leg_num}"/>
-	<origin xyz="${Leg_3_Ox} ${Leg_3_Oy} ${mirror*Leg_3_Oz}" rpy="${Leg_3_roll} ${Leg_3_pitch} ${Leg_3_yaw}"/>
-	<axis xyz="0 0 ${mirror}"/>
-   <limit lower="${knee_pitch_lower[leg_num-1]}" upper="${knee_pitch_upper[leg_num-1]}" effort="${motor_A_effort}" velocity="${motor_A_velocity}"/> <!-- 200 Nm, 1 rad/s-->
-</joint>
-<joint name="ankle_pitch_${leg_num}" type="revolute">
-	<parent link="knee_${leg_num}"/>
-	<child link="ankle1_${leg_num}"/>
-	<origin xyz="${Ankle_1_Ox} ${Ankle_1_Oy} ${mirror*Ankle_1_Oz}" rpy="${Ankle_1_roll} ${Ankle_1_pitch} ${Ankle_1_yaw}"/>
-	<axis xyz="0 0 ${mirror}"/>
-   <limit lower="${ankle_pitch_lower[leg_num-1]}" upper="${ankle_pitch_upper[leg_num-1]}" effort="${motor_B_effort}" velocity="${motor_B_velocity}"/> <!-- 98 Nm, 1 rad/s-->
-</joint>
-<joint name="ankle_yaw_${leg_num}" type="revolute">
-	<parent link="ankle1_${leg_num}"/>
-	<child link="ankle2_${leg_num}"/>
-	<origin xyz="${Ankle_2_Ox} ${Ankle_2_Oy} ${mirror*Ankle_2_Oz}" rpy="${Ankle_2_roll} ${Ankle_2_pitch} ${Ankle_2_yaw}"/>
-	<axis xyz="0 0 -1"/>
-   <limit lower="${ankle_yaw_lower[leg_num-1]}" upper="${ankle_yaw_upper[leg_num-1]}" effort="${motor_C_effort}" velocity="${motor_C_velocity}"/>  <!-- 23 Nm, 1 rad/s-->
-</joint>
-<joint name="j_wheel_${leg_num}" type="continuous">
-	<parent link="ankle2_${leg_num}"/>
-	<child link="wheel_${leg_num}"/>
-	<origin xyz="${Wheel_Ox} ${mirror*Wheel_Oy} ${Wheel_Oz}" rpy="${Wheel_roll} ${Wheel_pitch} ${Wheel_yaw}"/>
-	<axis xyz="0 0 ${mirror}"/>
-   <limit  effort="${motor_C_effort}" velocity="${motor_C_velocity}"/>  <!-- 23 Nm, 1 rad/s-->
-</joint>
+   <joint name="knee_pitch_${leg_num}" type="revolute">
+      <parent link="hip2_${leg_num}"/>
+      <child link="knee_${leg_num}"/>
+      <origin xyz="${Leg_3_Ox} ${Leg_3_Oy} ${mirror*Leg_3_Oz}" rpy="${Leg_3_roll} ${Leg_3_pitch} ${Leg_3_yaw}"/>
+      <axis xyz="0 0 ${mirror}"/>
+      <limit lower="${knee_pitch_lower[leg_num-1]}" upper="${knee_pitch_upper[leg_num-1]}" effort="${motor_A_effort}" velocity="${motor_A_velocity}"/> <!-- 200 Nm, 1 rad/s-->
+   </joint>
+   <joint name="ankle_pitch_${leg_num}" type="revolute">
+      <parent link="knee_${leg_num}"/>
+      <child link="ankle1_${leg_num}"/>
+      <origin xyz="${Ankle_1_Ox} ${Ankle_1_Oy} ${mirror*Ankle_1_Oz}" rpy="${Ankle_1_roll} ${Ankle_1_pitch} ${Ankle_1_yaw}"/>
+      <axis xyz="0 0 ${mirror}"/>
+      <limit lower="${ankle_pitch_lower[leg_num-1]}" upper="${ankle_pitch_upper[leg_num-1]}" effort="${motor_B_effort}" velocity="${motor_B_velocity}"/> <!-- 98 Nm, 1 rad/s-->
+   </joint>
+   <joint name="ankle_yaw_${leg_num}" type="revolute">
+      <parent link="ankle1_${leg_num}"/>
+      <child link="ankle2_${leg_num}"/>
+      <origin xyz="${Ankle_2_Ox} ${Ankle_2_Oy} ${mirror*Ankle_2_Oz}" rpy="${Ankle_2_roll} ${Ankle_2_pitch} ${Ankle_2_yaw}"/>
+      <axis xyz="0 0 -1"/>
+      <limit lower="${ankle_yaw_lower[leg_num-1]}" upper="${ankle_yaw_upper[leg_num-1]}" effort="${motor_C_effort}" velocity="${motor_C_velocity}"/>  <!-- 23 Nm, 1 rad/s-->
+   </joint>
 </xacro:unless>
 </xacro:macro>

File: centauro_urdf/urdf/parts/kinematics_properties.urdf.xacro (robot description, xacro)
@@ -66,4 +66,12 @@
 <xacro:property name="Wheel_pitch" value="0.0"/>
 <xacro:property name="Wheel_yaw" value="0.0"/>
+<xacro:property name="Wheel_radius" value="0.078"/>
+<xacro:property name="Wheel23_Ox" value="${0.0 * mmTom}"/>
+<xacro:property name="Wheel23_Oy" value="${0.0 * mmTom}"/>
+<xacro:property name="Wheel23_Oz" value="${-144.350 * mmTom}"/>
+<xacro:property name="Wheel23_roll" value="${PI_2}"/>
+<xacro:property name="Wheel23_pitch" value="0.0"/>
+<xacro:property name="Wheel23_yaw" value="0.0"/>
+<xacro:property name="Wheel23_radius" value="0.124"/>
 <!-- Origin -->
 <xacro:property name="Torso_2_Ox" value=" 0.200 "/>

Commit message: upd generated

File: centauro_urdf/urdf/centauro.urdf (robot description, URDF)
Before this commit: robot centauro, 60 links, 59 joints
Links:
- added link D435_head_camera_accel_frame
- added link D435_head_camera_accel_optical_frame
- added link D435_head_camera_color_frame
- added link D435_head_camera_color_optical_frame
- added link D435_head_camera_depth_frame
- added link D435_head_camera_depth_optical_frame
- added link D435_head_camera_gyro_frame
- added link D435_head_camera_gyro_optical_frame
- added link D435_head_camera_left_ir_frame
- added link D435_head_camera_left_ir_optical_frame
- added link D435_head_camera_right_ir_frame
- added link D435_head_camera_right_ir_optical_frame
- added link D435i_camera_accel_frame
- added link D435i_camera_accel_optical_frame
- added link D435i_camera_color_frame
- added link D435i_camera_color_optical_frame
- added link D435i_camera_depth_frame
- added link D435i_camera_depth_optical_frame
- added link D435i_camera_gyro_frame
- added link D435i_camera_gyro_optical_frame
- added link D435i_camera_left_ir_frame
- added link D435i_camera_left_ir_optical_frame
- added link D435i_camera_right_ir_frame
- added link D435i_camera_right_ir_optical_frame
- added link T265_camera_accel_frame
- added link T265_camera_accel_optical_frame
- added link T265_camera_fisheye1_optical_frame
- added link T265_camera_fisheye1_rgb_frame
- added link T265_camera_fisheye2_optical_frame
- added link T265_camera_fisheye2_rgb_frame
- added link T265_camera_gyro_frame
- added link T265_camera_gyro_optical_frame
- added link T265_camera_link
- added link T265_camera_pose_frame, mass 0.068024; collision mesh filename=package://realsense_gazebo_description/meshes/t265_simplifi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 scale=0.001 0.001 0.001; visual mesh filename=package://realsense_gazebo_description/meshes/t265_full.stl scale=0.001 0.001 0.001
- link D435_head_camera_link: geometry collision box size=0.02505 0.09 0.025; visual mesh filename=package://realsense2_description/meshes/d435.dae
- link D435i_camera_link: geometry collision box size=0.02505 0.09 0.025; visual mesh filename=package://realsense2_description/meshes/d435.dae
Joints:
- added joint D435_head_camera_accel_joint: type fixed, parent D435_head_camera_link, child D435_head_camera_accel_frame, origin xyz=-0.00174 0.00552 0.0176 rpy=0 0 0
- added joint D435_head_camera_accel_optical_joint: type fixed, parent D435_head_camera_accel_frame, child D435_head_camera_accel_optical_frame, origin xyz=0 0 0 rpy=-1.5707963267948966 0 -1.5707963267948966
- added joint D435_head_camera_color_joint: type fixed, parent D435_head_camera_depth_frame, child D435_head_camera_color_frame, origin xyz=0 0.015 0 rpy=0 0 0
- added joint D435_head_camera_color_optical_joint: type fixed, parent D435_head_camera_color_frame, child D435_head_camera_color_optical_frame, origin xyz=0 0 0 rpy=-1.5707963267948966 0 -1.5707963267948966
- added joint D435_head_camera_depth_joint: type fixed, parent D435_head_camera_link, child D435_head_camera_depth_frame, origin xyz=0 0 0 rpy=0 0 0
- added joint D435_head_camera_depth_optical_joint: type fixed, parent D435_head_camera_depth_frame, child D435_head_camera_depth_optical_frame, origin xyz=0 0 0 rpy=-1.5707963267948966 0 -1.5707963267948966
- added joint D435_head_camera_gyro_joint: type fixed, parent D435_head_camera_link, child D435_head_camera_gyro_frame, origin xyz=-0.00174 0.00552 0.0176 rpy=0 0 0
- added joint D435_head_camera_gyro_optical_joint: type fixed, parent D435_head_camera_gyro_frame, child D435_head_camera_gyro_optical_frame, origin xyz=0 0 0 rpy=-1.5707963267948966 0 -1.5707963267948966
- added joint D435_head_camera_left_ir_joint: type fixed, parent D435_head_camera_depth_frame, child D435_head_camera_left_ir_frame, origin xyz=0 0.0 0 rpy=0 0 0
- added joint D435_head_camera_left_ir_optical_joint: type fixed, parent D435_head_camera_left_ir_frame, child D435_head_camera_left_ir_optical_frame, origin xyz=0 0 0 rpy=-1.5707963267948966 0 -1.5707963267948966
- added joint D435_head_camera_right_ir_joint: type fixed, parent D435_head_camera_depth_frame, child D435_head_camera_right_ir_frame, origin xyz=0 -0.05 0 rpy=0 0 0
- added joint D435_head_camera_right_ir_optical_joint: type fixed, parent D435_head_camera_right_ir_frame, child D435_head_camera_right_ir_optical_frame, origin xyz=0 0 0 rpy=-1.5707963267948966 0 -1.5707963267948966
- added joint D435i_camera_accel_joint: type fixed, parent D435i_camera_link, child D435i_camera_accel_frame, origin xyz=-0.00174 0.00552 0.0176 rpy=0 0 0
- added joint D435i_camera_accel_optical_joint: type fixed, parent D435i_camera_accel_frame, child D435i_camera_accel_optical_frame, origin xyz=0 0 0 rpy=-1.5707963267948966 0 -1.5707963267948966
- added joint D435i_camera_color_joint: type fixed, parent D435i_camera_depth_frame, child D435i_camera_color_frame, origin xyz=0 0.015 0 rpy=0 0 0
- added joint D435i_camera_color_optical_joint: type fixed, parent D435i_camera_color_frame, child D435i_camera_color_optical_frame, origin xyz=0 0 0 rpy=-1.5707963267948966 0 -1.5707963267948966
- added joint D435i_camera_depth_joint: type fixed, parent D435i_camera_link, child D435i_camera_depth_frame, origin xyz=0 0 0 rpy=0 0 0
- added joint D435i_camera_depth_optical_joint: type fixed, parent D435i_camera_depth_frame, child D435i_camera_depth_optical_frame, origin xyz=0 0 0 rpy=-1.5707963267948966 0 -1.5707963267948966
- added joint D435i_camera_gyro_joint: type fixed, parent D435i_camera_link, child D435i_camera_gyro_frame, origin xyz=-0.00174 0.00552 0.0176 rpy=0 0 0
- added joint D435i_camera_gyro_optical_joint: type fixed, parent D435i_camera_gyro_frame, child D435i_camera_gyro_optical_frame, origin xyz=0 0 0 rpy=-1.5707963267948966 0 -1.5707963267948966
- added joint D435i_camera_left_ir_joint: type fixed, parent D435i_camera_depth_frame, child D435i_camera_left_ir_frame, origin xyz=0 0.0 0 rpy=0 0 0
- added joint D435i_camera_left_ir_optical_joint: type fixed, parent D435i_camera_left_ir_frame, child D435i_camera_left_ir_optical_frame, origin xyz=0 0 0 rpy=-1.5707963267948966 0 -1.5707963267948966
- added joint D435i_camera_right_ir_joint: type fixed, parent D435i_camera_depth_frame, child D435i_camera_right_ir_frame, origin xyz=0 -0.05 0 rpy=0 0 0
- added joint D435i_camera_right_ir_optical_joint: type fixed, parent D435i_camera_right_ir_frame, child D435i_camera_right_ir_optical_frame, origin xyz=0 0 0 rpy=-1.5707963267948966 0 -1.5707963267948966
- added joint T265_camera_accel_joint: type fixed, parent T265_camera_link, child T265_camera_accel_frame, origin xyz=-0.0311 0 0.00655 rpy=0 3.141592653589793 0
- added joint T265_camera_accel_optical_joint: type fixed, parent T265_camera_accel_frame, child T265_camera_accel_optical_frame, origin xyz=-0.0311 0 0.00655 rpy=0 3.141592653589793 0
- added joint T265_camera_fisheye1_optical_joint: type fixed, parent T265_camera_fisheye1_rgb_frame, child T265_camera_fisheye1_optical_frame, origin xyz=0 0 0 rpy=-1.5707963267948966 0 -1.5707963267948966
- added joint T265_camera_fisheye1_rgb_joint: type fixed, parent T265_camera_link, child T265_camera_fisheye1_rgb_frame, origin xyz=-0.0411 0.0 0.0 rpy=0 1.5707963267948966 1.5707963267948966
- added joint T265_camera_fisheye2_optical_joint: type fixed, parent T265_camera_fisheye2_rgb_frame, child T265_camera_fisheye2_optical_frame, origin xyz=0 0 0 rpy=-1.5707963267948966 0 -1.5707963267948966
- added joint T265_camera_fisheye2_rgb_joint: type fixed, parent T265_camera_link, child T265_camera_fisheye2_rgb_frame, origin xyz=0.0229 0.0 0.0 rpy=0 1.5707963267948966 1.5707963267948966
- added joint T265_camera_gyro_joint: type fixed, parent T265_camera_link, child T265_camera_gyro_frame, origin xyz=-0.0311 0 0.00655 rpy=0 3.141592653589793 0
- added joint T265_camera_gyro_optical_joint: type fixed, parent T265_camera_gyro_frame, child T265_camera_gyro_optical_frame, origin xyz=0 0 0 rpy=0 0 0
- added joint T265_camera_link_joint: type fixed, parent T265_camera_pose_frame, child T265_camera_link, origin xyz=0 0 0 rpy=1.5707963267948966 0 -1.5707963267948966
- added joint T265_camera_pose_joint: type fixed, parent pelvis, child T265_camera_pose_frame, origin xyz=0.29245 0.00775 0.063 rpy=0 0 0
- joint D435i_camera_link_joint: origin xyz=0.053 0.0 -0.035 rpy=0 0.0050 -0.008 -> xyz=0 0.0175 0.0125 rpy=0 0 0
