Commit message: upd generated

File: centauro_urdf/urdf/centauro.urdf (robot description, URDF)
Before this commit: robot centauro, 94 links, 93 joints
Joints:
- joint contact_joint_1: origin xyz=0 0 -0.176 rpy=0 0 0 -> xyz=0 0 -0.26835 rpy=0 0 0
- joint contact_joint_2: origin xyz=0 0 -0.176 rpy=0 0 0 -> xyz=0 0 -0.26835 rpy=0 0 0
- joint contact_joint_3: origin xyz=0 0 -0.176 rpy=0 0 0 -> xyz=0 0 -0.26835 rpy=0 0 0
- joint contact_joint_4: origin xyz=0 0 -0.176 rpy=0 0 0 -> xyz=0 0 -0.26835 rpy=0 0 0

Commit message: hack: generated defaults to dagana (todo: improve this mess)

File: centauro_urdf/urdf/centauro.urdf (robot description, URDF)
Before this commit: robot centauro, 94 links, 93 joints
Links:
- removed link ball2
- removed link ball2_tip
- added link dagana_2_bottom_link, mass 4.6117745e-01; collision mesh filename=package://dagana_urdf/meshes/dg0002-ch.stl scale=0.001 0.001 0.001; visual mesh filename=package://dagana_urdf/meshes/dg0002.stl scale=0.001 0.001 0.001
- added link dagana_2_tcp
- added link dagana_2_top_link, mass 1.7432400; collision mesh filename=package://dagana_urdf/meshes/dg0001-ch.stl scale=0.001 0.001 0.001; visual mesh filename=package://dagana_urdf/meshes/dg0001-simplified.stl scale=0.001 0.001 0.001
Joints:
- removed joint j_arm2_8
- removed joint j_ball2_fixed
- removed joint j_ball2_tip
- added joint dagana_2_claw_joint: type revolute, parent dagana_2_top_link, child dagana_2_bottom_link, origin xyz=0.0 -0.028 0.05025 rpy=1.57079632679 0 3.14159265359, axis -1 0 0, limit lower=0 upper=1 effort=1000 velocity=2.0
- added joint dagana_2_mount_joint: type fixed, parent arm2_6, child dagana_2_top_link, origin xyz=0. 0.05 -0.08 rpy=0. 3.14159265359 0
- added joint dagana_2_tcp_joint: type fixed, parent dagana_2_top_link, child dagana_2_tcp, origin xyz=0 -0.05 0.15 rpy=0 0 0
- added joint j_dagana_2_final: type fixed, parent dagana_2_bottom_link, child arm2_8

File: centauro_urdf/urdf/centauro_capsule.urdf (robot description, URDF)
Before this commit: robot centauro, 60 links, 59 joints
Links:
- removed link ball2
- removed link ball2_tip
- added link D435_head_camera_accel_frame
- added link D435_head_camera_accel_optical_frame
- added link D435_head_camera_color_frame
- added link D435_head_camera_color_optical_frame
- added link D435_head_camera_depth_frame
- added link D435_head_camera_depth_optical_frame
- added link D435_head_camera_gyro_frame
- added link D435_head_camera_gyro_optical_frame
- added link D435_head_camera_left_ir_frame
- added link D435_head_camera_left_ir_optical_frame
- added link D435_head_camera_right_ir_frame
- added link D435_head_camera_right_ir_optical_frame
- added link D435i_camera_accel_frame
- added link D435i_camera_accel_optical_frame
- added link D435i_camera_color_frame
- added link D435i_camera_color_optical_frame
- added link D435i_camera_depth_frame
- added link D435i_camera_depth_optical_frame
- added link D435i_camera_gyro_frame
- added link D435i_camera_gyro_optical_frame
- added link D435i_camera_left_ir_frame
- added link D435i_camera_left_ir_optical_frame
- added link D435i_camera_right_ir_frame
- added link D435i_camera_right_ir_optical_frame
- added link T265_camera_accel_frame
- added link T265_camera_accel_optical_frame
- added link T265_camera_fisheye1_optical_frame
- added link T265_camera_fisheye1_rgb_frame
- added link T265_camera_fisheye2_optical_frame
- added link T265_camera_fisheye2_rgb_frame
- added link T265_camera_gyro_frame
- added link T265_camera_gyro_optical_frame
- added link T265_camera_link
- added link T265_camera_pose_frame, mass 0.068024; collision cylinder length=0.1022528557886848 radius=0.0142751; collision sphere radius=0.0142751
- added link dagana_2_bottom_link, mass 0.46117745; collision cylinder length=0.11781363498578913 radius=0.0618624; collision sphere radius=0.0618624
- added link dagana_2_tcp
- added link dagana_2_top_link, mass 1.74324; collision cylinder length=0.10212404260993166 radius=0.0760764; collision sphere radius=0.0760764
- link D435_head_camera_link: geometry collision box size=0.02505 0.09 0.025; visual mesh filename=package://realsense2_description/meshes/d435.dae
- link D435i_camera_link: geometry collision box size=0.02505 0.09 0.025; visual mesh filename=package://realsense2_description/meshes/d435.dae
Joints:
- removed joint j_arm2_8
- removed joint j_ball2_fixed
- removed joint j_ball2_tip
- added joint D435_head_camera_accel_joint: type fixed, parent D435_head_camera_link, child D435_head_camera_accel_frame, origin xyz=-0.00174 0.00552 0.0176 rpy=0.0 0.0 0.0
- added joint D435_head_camera_accel_optical_joint: type fixed, parent D435_head_camera_accel_frame, child D435_head_camera_accel_optical_frame, origin xyz=0.0 0.0 0.0 rpy=-1.5707963267948966 0.0 -1.5707963267948966
- added joint D435_head_camera_color_joint: type fixed, parent D435_head_camera_depth_frame, child D435_head_camera_color_frame, origin xyz=0.0 0.015 0.0 rpy=0.0 0.0 0.0
- added joint D435_head_camera_color_optical_joint: type fixed, parent D435_head_camera_color_frame, child D435_head_camera_color_optical_frame, origin xyz=0.0 0.0 0.0 rpy=-1.5707963267948966 0.0 -1.5707963267948966
- added joint D435_head_camera_depth_joint: type fixed, parent D435_head_camera_link, child D435_head_camera_depth_frame, origin xyz=0.0 0.0 0.0 rpy=0.0 0.0 0.0
- added joint D435_head_camera_depth_optical_joint: type fixed, parent D435_head_camera_depth_frame, child D435_head_camera_depth_optical_frame, origin xyz=0.0 0.0 0.0 rpy=-1.5707963267948966 0.0 -1.5707963267948966
- added joint D435_head_camera_gyro_joint: type fixed, parent D435_head_camera_link, child D435_head_camera_gyro_frame, origin xyz=-0.00174 0.00552 0.0176 rpy=0.0 0.0 0.0
- added joint D435_head_camera_gyro_optical_joint: type fixed, parent D435_head_camera_gyro_frame, child D435_head_camera_gyro_optical_frame, origin xyz=0.0 0.0 0.0 rpy=-1.5707963267948966 0.0 -1.5707963267948966
- added joint D435_head_camera_left_ir_joint: type fixed, parent D435_head_camera_depth_frame, child D435_head_camera_left_ir_frame, origin xyz=0.0 0.0 0.0 rpy=0.0 0.0 0.0
- added joint D435_head_camera_left_ir_optical_joint: type fixed, parent D435_head_camera_left_ir_frame, child D435_head_camera_left_ir_optical_frame, origin xyz=0.0 0.0 0.0 rpy=-1.5707963267948966 0.0 -1.5707963267948966
- added joint D435_head_camera_right_ir_joint: type fixed, parent D435_head_camera_depth_frame, child D435_head_camera_right_ir_frame, origin xyz=0.0 -0.05 0.0 rpy=0.0 0.0 0.0
- added joint D435_head_camera_right_ir_optical_joint: type fixed, parent D435_head_camera_right_ir_frame, child D435_head_camera_right_ir_optical_frame, origin xyz=0.0 0.0 0.0 rpy=-1.5707963267948966 0.0 -1.5707963267948966
- added joint D435i_camera_accel_joint: type fixed, parent D435i_camera_link, child D435i_camera_accel_frame, origin xyz=-0.00174 0.00552 0.0176 rpy=0.0 0.0 0.0
- added joint D435i_camera_accel_optical_joint: type fixed, parent D435i_camera_accel_frame, child D435i_camera_accel_optical_frame, origin xyz=0.0 0.0 0.0 rpy=-1.5707963267948966 0.0 -1.5707963267948966
- added joint D435i_camera_color_joint: type fixed, parent D435i_camera_depth_frame, child D435i_camera_color_frame, origin xyz=0.0 0.015 0.0 rpy=0.0 0.0 0.0
- added joint D435i_camera_color_optical_joint: type fixed, parent D435i_camera_color_frame, child D435i_camera_color_optical_frame, origin xyz=0.0 0.0 0.0 rpy=-1.5707963267948966 0.0 -1.5707963267948966
- added joint D435i_camera_depth_joint: type fixed, parent D435i_camera_link, child D435i_camera_depth_frame, origin xyz=0.0 0.0 0.0 rpy=0.0 0.0 0.0
- added joint D435i_camera_depth_optical_joint: type fixed, parent D435i_camera_depth_frame, child D435i_camera_depth_optical_frame, origin xyz=0.0 0.0 0.0 rpy=-1.5707963267948966 0.0 -1.5707963267948966
- added joint D435i_camera_gyro_joint: type fixed, parent D435i_camera_link, child D435i_camera_gyro_frame, origin xyz=-0.00174 0.00552 0.0176 rpy=0.0 0.0 0.0
- added joint D435i_camera_gyro_optical_joint: type fixed, parent D435i_camera_gyro_frame, child D435i_camera_gyro_optical_frame, origin xyz=0.0 0.0 0.0 rpy=-1.5707963267948966 0.0 -1.5707963267948966
- added joint D435i_camera_left_ir_joint: type fixed, parent D435i_camera_depth_frame, child D435i_camera_left_ir_frame, origin xyz=0.0 0.0 0.0 rpy=0.0 0.0 0.0
- added joint D435i_camera_left_ir_optical_joint: type fixed, parent D435i_camera_left_ir_frame, child D435i_camera_left_ir_optical_frame, origin xyz=0.0 0.0 0.0 rpy=-1.5707963267948966 0.0 -1.5707963267948966
- added joint D435i_camera_right_ir_joint: type fixed, parent D435i_camera_depth_frame, child D435i_camera_right_ir_frame, origin xyz=0.0 -0.05 0.0 rpy=0.0 0.0 0.0
- added joint D435i_camera_right_ir_optical_joint: type fixed, parent D435i_camera_right_ir_frame, child D435i_camera_right_ir_optical_frame, origin xyz=0.0 0.0 0.0 rpy=-1.5707963267948966 0.0 -1.5707963267948966
- added joint T265_camera_accel_joint: type fixed, parent T265_camera_link, child T265_camera_accel_frame, origin xyz=-0.0311 0.0 0.00655 rpy=0.0 3.141592653589793 0.0
- added joint T265_camera_accel_optical_joint: type fixed, parent T265_camera_accel_frame, child T265_camera_accel_optical_frame, origin xyz=-0.0311 0.0 0.00655 rpy=0.0 3.141592653589793 0.0
- added joint T265_camera_fisheye1_optical_joint: type fixed, parent T265_camera_fisheye1_rgb_frame, child T265_camera_fisheye1_optical_frame, origin xyz=0.0 0.0 0.0 rpy=-1.5707963267948966 0.0 -1.5707963267948966
- added joint T265_camera_fisheye1_rgb_joint: type fixed, parent T265_camera_link, child T265_camera_fisheye1_rgb_frame, origin xyz=-0.0411 0.0 0.0 rpy=0.0 1.5707963267948966 1.5707963267948966
- added joint T265_camera_fisheye2_optical_joint: type fixed, parent T265_camera_fisheye2_rgb_frame, child T265_camera_fisheye2_optical_frame, origin xyz=0.0 0.0 0.0 rpy=-1.5707963267948966 0.0 -1.5707963267948966
- added joint T265_camera_fisheye2_rgb_joint: type fixed, parent T265_camera_link, child T265_camera_fisheye2_rgb_frame, origin xyz=0.0229 0.0 0.0 rpy=0.0 1.5707963267948966 1.5707963267948966
- added joint T265_camera_gyro_joint: type fixed, parent T265_camera_link, child T265_camera_gyro_frame, origin xyz=-0.0311 0.0 0.00655 rpy=0.0 3.141592653589793 0.0
- added joint T265_camera_gyro_optical_joint: type fixed, parent T265_camera_gyro_frame, child T265_camera_gyro_optical_frame, origin xyz=0.0 0.0 0.0 rpy=0.0 0.0 0.0
- added joint T265_camera_link_joint: type fixed, parent T265_camera_pose_frame, child T265_camera_link, origin xyz=0.0 0.0 0.0 rpy=1.5707963267948966 0.0 -1.5707963267948966
- added joint T265_camera_pose_joint: type fixed, parent pelvis, child T265_camera_pose_frame, origin xyz=0.29245 0.00775 0.063 rpy=0.0 0.0 0.0
- added joint dagana_2_claw_joint: type revolute, parent dagana_2_top_link, child dagana_2_bottom_link, origin xyz=0.0 -0.028 0.05025 rpy=1.57079632679 0.0 3.14159265359, axis -1.0 0.0 0.0, limit lower=0.0 upper=1.0 effort=1000.0 velocity=2.0
- added joint dagana_2_mount_joint: type fixed, parent arm2_6, child dagana_2_top_link, origin xyz=0.0 0.05 -0.08 rpy=0.0 3.14159265359 0.0
- added joint dagana_2_tcp_joint: type fixed, parent dagana_2_top_link, child dagana_2_tcp, origin xyz=0.0 -0.05 0.15 rpy=0.0 0.0 0.0
- added joint j_dagana_2_final: type fixed, parent dagana_2_bottom_link, child arm2_8
- joint D435i_camera_link_joint: origin xyz=0.053 0.0 -0.035 rpy=0.0 0.005 -0.008 -> xyz=0.0 0.0175 0.0125 rpy=0.0 0.0 0.0
- joint contact_joint_1: origin xyz=0.0 0.0 -0.176 rpy=0.0 0.0 0.0 -> xyz=0.0 0.0 -0.26835 rpy=0.0 0.0 0.0
- joint contact_joint_2: origin xyz=0.0 0.0 -0.176 rpy=0.0 0.0 0.0 -> xyz=0.0 0.0 -0.26835 rpy=0.0 0.0 0.0
- joint contact_joint_3: origin xyz=0.0 0.0 -0.176 rpy=0.0 0.0 0.0 -> xyz=0.0 0.0 -0.26835 rpy=0.0 0.0 0.0
- joint contact_joint_4: origin xyz=0.0 0.0 -0.176 rpy=0.0 0.0 0.0 -> xyz=0.0 0.0 -0.26835 rpy=0.0 0.0 0.0

Commit message: Merge remote-tracking branch 'origin/big_wheels_v2.10' into ioannis-devel-v2.10 joint gripper adapter is not found from xbot
# Conflicts:
#	centauro_config/hal/centauro_gz.yaml
#	centauro_srdf/srdf/centauro.srdf
#	centauro_srdf/srdf/centauro_capsule.srdf
#	centauro_srdf/srdf/centauro_virtual_frame.srdf
#	centauro_urdf/urdf/centauro.urdf
#	centauro_urdf/urdf/centauro_capsule.urdf
#	centauro_urdf/urdf/centauro_virtual_frame.urdf
#	centauro_urdf/urdf/config/centauro.urdf.xacro
#	centauro_urdf/urdf/config/centauro_virtual_frame.urdf.xacro

File: centauro_urdf/urdf/centauro.urdf (robot description, URDF)
Before this commit: robot centauro, 94 links, 93 joints
Links:
- removed link ball2
- removed link ball2_tip
- added link dagana_2_bottom_link, mass 4.6117745e-01; collision mesh filename=package://dagana_urdf/meshes/dg0002-ch.stl scale=0.001 0.001 0.001; visual mesh filename=package://dagana_urdf/meshes/dg0002.stl scale=0.001 0.001 0.001
- added link dagana_2_tcp
- added link dagana_2_top_link, mass 1.27; collision mesh filename=package://dagana_urdf/meshes/dg0001-ch.stl scale=0.001 0.001 0.001; visual mesh filename=package://dagana_urdf/meshes/dg0001-simplified.stl scale=0.001 0.001 0.001
- link velodyne_calib: geometry collision sphere radius=0; visual mesh filename=package://velodyne_description/meshes/VLP16_scan.dae
Joints:
- removed joint j_arm2_8
- removed joint j_ball2_fixed
- removed joint j_ball2_tip
- added joint dagana_2_claw_joint: type revolute, parent dagana_2_top_link, child dagana_2_bottom_link, origin xyz=0.0 -0.028 0.05025 rpy=1.57079632679 0 3.14159265359, axis -1 0 0, limit lower=0 upper=1 effort=1000 velocity=2.0
- added joint dagana_2_mount_joint: type fixed, parent arm2_6, child dagana_2_top_link, origin xyz=0. 0.05 -0.08 rpy=0. 3.14159265359 0
- added joint dagana_2_tcp_joint: type fixed, parent dagana_2_top_link, child dagana_2_tcp, origin xyz=0 -0.05 0.15 rpy=0 0 0
- added joint j_dagana_2_final: type fixed, parent dagana_2_bottom_link, child arm2_8

File: centauro_urdf/urdf/centauro_capsule.urdf (robot description, URDF)
Before this commit: robot centauro, 94 links, 93 joints
Links:
- removed link ball2
- removed link ball2_tip
- added link dagana_2_bottom_link, mass 0.46117745; collision cylinder length=0.11781363498578913 radius=0.0618624; collision sphere radius=0.0618624
- added link dagana_2_tcp
- added link dagana_2_top_link, mass 1.74324; collision cylinder length=0.10212404260993166 radius=0.0760764; collision sphere radius=0.0760764
- link velodyne_calib: geometry collision sphere radius=0.0; visual mesh filename=package://velodyne_description/meshes/VLP16_scan.dae
Joints:
- removed joint j_arm2_8
- removed joint j_ball2_fixed
- removed joint j_ball2_tip
- added joint dagana_2_claw_joint: type revolute, parent dagana_2_top_link, child dagana_2_bottom_link, origin xyz=0.0 -0.028 0.05025 rpy=1.57079632679 0.0 3.14159265359, axis -1.0 0.0 0.0, limit lower=0.0 upper=1.0 effort=1000.0 velocity=2.0
- added joint dagana_2_mount_joint: type fixed, parent arm2_6, child dagana_2_top_link, origin xyz=0.0 0.05 -0.08 rpy=0.0 3.14159265359 0.0
- added joint dagana_2_tcp_joint: type fixed, parent dagana_2_top_link, child dagana_2_tcp, origin xyz=0.0 -0.05 0.15 rpy=0.0 0.0 0.0
- added joint j_dagana_2_final: type fixed, parent dagana_2_bottom_link, child arm2_8

Commit message: head camera mounted on a 20 deg angle

File: centauro_urdf/urdf/centauro.urdf (robot description, URDF)
Before this commit: robot centauro, 95 links, 94 joints
Joints:
- joint D435_head_camera_joint: origin xyz=0.03015 0 -0.0125 rpy=0 0 0 -> xyz=0.0316 0 -0.01309 rpy=0 0.349065 0

File: centauro_urdf/urdf/centauro_dagana.urdf (robot description, URDF)
Before this commit: robot centauro, 95 links, 94 joints
Joints:
- joint D435_head_camera_joint: origin xyz=0.03015 0 -0.0125 rpy=0 0 0 -> xyz=0.0316 0 -0.01309 rpy=0 0.349065 0

File: centauro_urdf/urdf/parts/head.urdf.xacro (robot description, xacro)
@@ -88,5 +88,5 @@
   <xacro:property name="d435_head_parent_name" value="d435_head_motor" />
   <xacro:property name="d435_head_origin">
-    <origin xyz="0.03015 0 -0.0125" rpy="0 0 0"/>
+    <origin xyz="0.0316 0 -0.01309" rpy="0 0.349065 0"/>
   </xacro:property>
   <xacro:if value="${ADD_D435I_HEAD}">

Commit message: ros2 wip

File: centauro_urdf/urdf/centauro.urdf (robot description, URDF)
Before this commit: robot centauro, 95 links, 94 joints
Links:
- link T265_camera_pose_frame: geometry collision mesh filename=package://realsense2_description/meshes/t265_simplified.stl scale=0.001 0.001 0.001; visual mesh filename=package://realsense2_description/meshes/t265_full.stl scale=0.001 0.001 0.001

File: centauro_urdf/urdf/centauro_base.urdf.xacro (robot description, xacro)
@@ -50,5 +50,5 @@
         </xacro:property>
         <xacro:if value="${ADD_D435I_BASE}">
-            <xacro:include filename="$(find realsense_gazebo_description)/urdf/_d435i.urdf.xacro" />
+            <xacro:include filename="$(find realsense2_description)/urdf/_d435i.urdf.xacro" />
             <xacro:sensor_d435i parent="${d435_base_parent_name}"
                 name="${d435_base_name}"
@@ -117,5 +117,5 @@
         </xacro:unless>
         <xacro:if value="${ADD_T265_BASE}">
-            <xacro:include filename="$(find realsense_gazebo_description)/urdf/_t265.urdf.xacro" />
+            <xacro:include filename="$(find realsense2_description)/urdf/_t265.urdf.xacro" />
             <xacro:sensor_t265 parent="pelvis" name="T265_camera" topics_ns="T265/T265_camera"
                 odom_xyz="0.0 0.0 0.25"

File: centauro_urdf/urdf/centauro_capsule.urdf (robot description, URDF)
Before this commit: robot centauro, 95 links, 94 joints
Links:
- link T265_camera_pose_frame: geometry collision cylinder length=0.1022528557886848 radius=0.0142751; collision sphere radius=0.0142751

File: centauro_urdf/urdf/centauro_mjc_test.urdf (robot description, URDF)
Before this commit: robot centauro, 97 links, 96 joints
Links:
- link T265_camera_pose_frame: geometry collision mesh filename=package://realsense2_description/meshes/t265_simplified.stl scale=0.001 0.001 0.001; visual mesh filename=package://realsense2_description/meshes/t265_full.stl scale=0.001 0.001 0.001

File: centauro_urdf/urdf/parts/head.urdf.xacro (robot description, xacro)
@@ -91,5 +91,5 @@
   </xacro:property>
   <xacro:if value="${ADD_D435I_HEAD}">
-    <xacro:include filename="$(find realsense_gazebo_description)/urdf/_d435i.urdf.xacro" />
+    <xacro:include filename="$(find realsense2_description)/urdf/_d435i.urdf.xacro" />
     <xacro:sensor_d435i parent="${d435_head_parent_name}"
         name="${d435_head_name}"

Commit message: now using a cut mesh to avoid collision between pelvis and simulation issues

File: centauro_urdf/urdf/centauro.urdf (robot description, URDF)
Before this commit: robot centauro, 95 links, 94 joints
Links:
- link pelvis: geometry collision mesh filename=package://centauro_urdf/meshes/simple/pelvis_reduced.stl scale=0.001 0.001 0.001; visual mesh filename=package://centauro_urdf/meshes/v2/pelvis.stl scale=0.001 0.001 0.001

File: centauro_urdf/urdf/centauro_base.urdf.xacro (robot description, xacro)
@@ -27,5 +27,5 @@
             <origin xyz="0.0 0 0.0" rpy="0.0 0.0 0.0" />
             <geometry>
-                <mesh filename="${MESH_PATH}/simple/pelvis.stl" scale="0.001 0.001 0.001" />
+                <mesh filename="${MESH_PATH}/simple/pelvis_reduced.stl" scale="0.001 0.001 0.001" />
             </geometry>
         </collision>

File: centauro_urdf/urdf/centauro_virtual_frame.urdf (robot description, URDF)
Before this commit: robot centauro, 64 links, 63 joints
Links:
- link pelvis: geometry collision mesh filename=${MESH_PATH}/simple/pelvis_reduced.stl scale=0.001 0.001 0.001; visual mesh filename=${MESH_PATH}/v2/pelvis.stl scale=0.001 0.001 0.001

Commit message: now using pelvis coll mesh without self collisions

File: centauro_urdf/urdf/centauro.urdf (robot description, URDF)
Before this commit: robot centauro, 95 links, 94 joints
Links:
- link pelvis: geometry collision mesh filename=package://centauro_urdf/meshes/simple/pelvis_reduced.stl scale=0.001 0.001 0.001; visual mesh filename=package://centauro_urdf/meshes/v2/pelvis.stl scale=0.001 0.001 0.001

File: centauro_urdf/urdf/centauro_base.urdf.xacro (robot description, xacro)
@@ -30,5 +30,5 @@
             <origin xyz="0.0 0 0.0" rpy="0.0 0.0 0.0" />
             <geometry>
-                <mesh filename="${MESH_PATH}/simple/pelvis.stl" scale="0.001 0.001 0.001" />
+                <mesh filename="${MESH_PATH}/simple/pelvis_reduced.stl" scale="0.001 0.001 0.001" />
             </geometry>
         </collision>
