Commit message: bad trials to save somewhere

File: centauro_urdf/urdf/centauro_upper_dagana.urdf (robot description, URDF)
Before this commit: robot centauro, 54 links, 53 joints
Links:
- removed link D435_head_camera_accel_frame
- removed link D435_head_camera_accel_optical_frame
- removed link D435_head_camera_color_frame
- removed link D435_head_camera_color_optical_frame
- removed link D435_head_camera_depth_frame
- removed link D435_head_camera_depth_optical_frame
- removed link D435_head_camera_gyro_frame
- removed link D435_head_camera_gyro_optical_frame
- removed link D435_head_camera_left_ir_frame
- removed link D435_head_camera_left_ir_optical_frame
- removed link D435_head_camera_right_ir_frame
- removed link D435_head_camera_right_ir_optical_frame
- removed link D435i_camera_accel_frame
- removed link D435i_camera_accel_optical_frame
- removed link D435i_camera_color_frame
- removed link D435i_camera_color_optical_frame
- removed link D435i_camera_depth_frame
- removed link D435i_camera_depth_optical_frame
- removed link D435i_camera_gyro_frame
- removed link D435i_camera_gyro_optical_frame
- removed link D435i_camera_left_ir_frame
- removed link D435i_camera_left_ir_optical_frame
- removed link D435i_camera_right_ir_frame
- removed link D435i_camera_right_ir_optical_frame
- added link velodyne_motor, mass 0.33878686; collision mesh filename=package://centauro_urdf/meshes/simple/lidar_mesh.stl scale=0.001 0.001 0.001; visual mesh filename=package://centauro_urdf/meshes/lidar_mesh.stl scale=0.001 0.001 0.001
- link D435_head_camera_link: geometry collision box size=0.02505 0.09 0.025; visual box size=0.09 0.025 0.02505
- link D435i_camera_link: geometry collision box size=0.02505 0.09 0.025; visual box size=0.09 0.025 0.02505
- link d435_head_motor: geometry collision mesh filename=package://centauro_urdf/meshes/simple/neck-pitch_mesh.stl scale=0.001 0.001 0.001; visual mesh filename=package://centauro_urdf/meshes/neck-pitch_mesh.stl scale=0.001 0.001 0.001
- link dagana_1_bottom_link: geometry collision mesh filename=package://dagana_urdf/meshes/dg0002-ch.stl scale=0.001 0.001 0.001; visual mesh filename=package://dagana_urdf/meshes/dg0002.stl scale=0.001 0.001 0.001
- link dagana_1_top_link: geometry collision mesh filename=package://dagana_urdf/meshes/dg0001-simplified_v2.stl scale=0.001 0.001 0.001; visual mesh filename=package://dagana_urdf/meshes/dg0001-simplified.stl scale=0.001 0.001 0.001
- link dagana_2_bottom_link: geometry collision mesh filename=package://dagana_urdf/meshes/dg0002-ch.stl scale=0.001 0.001 0.001; visual mesh filename=package://dagana_urdf/meshes/dg0002.stl scale=0.001 0.001 0.001
- link dagana_2_top_link: geometry collision mesh filename=package://dagana_urdf/meshes/dg0001-simplified_v2.stl scale=0.001 0.001 0.001; visual mesh filename=package://dagana_urdf/meshes/dg0001-simplified.stl scale=0.001 0.001 0.001
- link neck_1: geometry collision mesh filename=package://centauro_urdf/meshes/simple/head-base_mesh.stl scale=0.001 0.001 0.001; visual mesh filename=package://centauro_urdf/meshes/head-base_mesh.stl scale=0.001 0.001 0.001
- link pelvis: mass 18.845851 -> 26.584529
Joints:
- removed joint D435_head_camera_accel_joint
- removed joint D435_head_camera_accel_optical_joint
- removed joint D435_head_camera_color_joint
- removed joint D435_head_camera_color_optical_joint
- removed joint D435_head_camera_depth_joint
- removed joint D435_head_camera_depth_optical_joint
- removed joint D435_head_camera_gyro_joint
- removed joint D435_head_camera_gyro_optical_joint
- removed joint D435_head_camera_left_ir_joint
- removed joint D435_head_camera_left_ir_optical_joint
- removed joint D435_head_camera_right_ir_joint
- removed joint D435_head_camera_right_ir_optical_joint
- removed joint D435i_camera_accel_joint
- removed joint D435i_camera_accel_optical_joint
- removed joint D435i_camera_color_joint
- removed joint D435i_camera_color_optical_joint
- removed joint D435i_camera_depth_joint
- removed joint D435i_camera_depth_optical_joint
- removed joint D435i_camera_gyro_joint
- removed joint D435i_camera_gyro_optical_joint
- removed joint D435i_camera_left_ir_joint
- removed joint D435i_camera_left_ir_optical_joint
- removed joint D435i_camera_right_ir_joint
- removed joint D435i_camera_right_ir_optical_joint
- added joint velodyne_joint: type revolute, parent neck_1, child velodyne_motor, origin xyz=0.0822724 0 0.242 rpy=0 0 0, axis 0 -1 0, limit lower=-1.1 upper=1.1 effort=35 velocity=5.7

File: centauro_urdf/urdf/config/centauro.urdf.xacro (robot description, xacro)
@@ -4,11 +4,11 @@
 <xacro:property name="model_version" value="0.1" />
 <!-- command line arguments -->
-<xacro:arg name="legs" default="true"/>
+<xacro:arg name="legs" default="false"/>
 <xacro:arg name="big_wheel" default="true"/>
 <xacro:arg name="upper_body" default="true"/>
-<xacro:arg name="velodyne" default="true"/>
+<xacro:arg name="velodyne" default="false"/>
 <xacro:arg name="realsense" default="true"/>
-<xacro:arg name="end_effector_left" default="ball"/>
-<xacro:arg name="end_effector_right" default="ball"/>
+<xacro:arg name="end_effector_left" default="dagana"/>
+<xacro:arg name="end_effector_right" default="dagana"/>
 <xacro:if value="$(arg realsense)">
 	<xacro:arg name="d435i_head" default="true"/>
@@ -21,5 +21,5 @@
 	<xacro:arg name="t265_base" default="false"/>
 </xacro:unless>
-<xacro:arg name="floating_joint" default="true"/>
+<xacro:arg name="floating_joint" default="false"/>
 <xacro:arg name="virtual_frame" default="false"/> <!-- For cartesio model must be set to true-->
 <xacro:arg name="end_effector_left" default="$(arg end_effector_left)"/> <!-- none, ball, dagana_fixed, dagana -->
