Commit message: added floating/fixed base

File: centauro_urdf/urdf/centauro.urdf.xacro (robot description, xacro)
@@ -7,9 +7,9 @@
 <!-- ************ Control frames ************ -->
 <!--xacro:include filename="$(find pholus_urdf)/urdf/control_frames.urdf.xacro"/-->
-<!--xacro:if value="${ADD_FLOATING_BASE}">
+<xacro:if value="${ADD_FLOATING_BASE}">
 <link name="world"/>
   <joint name="reference" type="floating">
     <parent link="world"/>
-    <child link="base_link"/>
+    <child link="pelvis"/>
 </joint>
 </xacro:if>
@@ -18,6 +18,6 @@
   <joint name="reference" type="fixed">
     <parent link="world"/>
-    <child link="base_link"/>
+    <child link="pelvis"/>
 </joint>
-</xacro:unless-->
+</xacro:unless>
 </robot>

File: centauro_urdf/urdf/centauro_base.urdf.xacro (robot description, xacro)
@@ -36,6 +36,6 @@
     </joint>
 <joint name="base_joint" type="fixed">
-    <parent link="base_link"/>
-    <child link="pelvis"/>
+    <parent link="pelvis"/>
+    <child link="base_link"/>
     <origin xyz="0 0 0" rpy="0 0 0" />
 </joint>

Commit message: simulation of single leg

File: centauro_urdf/urdf/centauro.urdf.xacro (robot description, xacro)
@@ -7,17 +7,9 @@
 <!-- ************ Control frames ************ -->
 <!--xacro:include filename="$(find pholus_urdf)/urdf/control_frames.urdf.xacro"/-->
-<xacro:if value="${ADD_FLOATING_BASE}">
 <link name="world"/>
-  <joint name="reference" type="floating">
+<joint name="reference" type="fixed">
     <parent link="world"/>
-    <child link="pelvis"/>
+    <child link="base_link"/>
+    <origin rpy="0 0 0" xyz="0 0 ${c/2.}"/>
 </joint>
-</xacro:if>
-<xacro:unless value="${ADD_FLOATING_BASE}">
-<link name="world"/>
-  <joint name="reference" type="fixed">
-    <parent link="world"/>
-    <child link="pelvis"/>
-</joint>
-</xacro:unless>
 </robot>

File: centauro_urdf/urdf/centauro_base.urdf.xacro (robot description, xacro)
@@ -9,51 +9,49 @@
 <xacro:include filename="$(find centauro_urdf)/urdf/parts/inertial_properties.urdf.xacro" />
 <xacro:include filename="$(find centauro_urdf)/urdf/parts/limits.urdf.xacro" />
-<link name="base_link"/>
+<xacro:property name="a" value="0.1"/> <!-- along x -->
+<xacro:property name="b" value="0.1"/> <!-- along y -->
+<xacro:property name="c" value="1.5"/> <!-- along z -->
+<link name="base_link">
+    <visual>
+      <geometry>
+        <box size="${a} ${b} ${c}"/>
+      </geometry>
+    </visual>
+    <collision>
+      <geometry>
+        <box size="${a} ${b} ${c}"/>
+      </geometry>
+    </collision>
+</link>
+<xacro:property name="r" value="0.1"/> <!-- along x -->
+<xacro:property name="h" value="0.1"/> <!-- along y -->
+<xacro:property name="m" value="1.0"/>
 <link name="pelvis">
-      <inertial>
-         <origin xyz="${Pelvis_x} ${Pelvis_y} ${Pelvis_z}"/>
-         <mass value="${Pelvis_mass}"/>
-         <inertia ixx="${Pelvis_xx}" ixy="${Pelvis_xy}" ixz="${Pelvis_xz}" iyy="${Pelvis_yy}" iyz="${Pelvis_yz}" izz="${Pelvis_zz}"/>
-      </inertial>
-      <visual>
-        <origin xyz="0.0 0 0.0"  rpy="0.0 0.0 0.0"/>
-        <geometry>
-         <mesh filename="package://centauro_urdf/meshes/pelvis.stl" scale="0.001 0.001 0.001" />
-        </geometry>
-      </visual>
-      <collision>
-         <origin xyz="0.0 0 0.0"  rpy="0.0 0.0 0.0"/>
-        <geometry>
-         <mesh filename="package://centauro_urdf/meshes/simple/pelvis.stl" scale="0.001 0.001 0.001" />
-        </geometry>
-      </collision>
-   </link>
-    <link name="imu_link"/>
-    <joint name="imu_joint" type="fixed">
-        <parent link="pelvis"/>
-        <origin xyz="${Imu_Ox} ${Imu_Oy} ${Imu_Oz}" rpy="${Imu_raw} ${Imu_pitch} ${Imu_yaw}"/>
-        <child link="imu_link"/>
-    </joint>
-<joint name="base_joint" type="fixed">
-    <parent link="pelvis"/>
-    <child link="base_link"/>
-    <origin xyz="0 0 0" rpy="0 0 0" />
+    <inertial>
+      <mass value="${m}"/>
+      <inertia ixx="${(m/48)*(6*r*r + 4*h*h)}" ixy="0.0" ixz="0.0" iyy="${(m/48)*(6*r*r + 4*h*h)}" iyz="0.0" izz="${m*h*h/4.}"/>
+    </inertial>
+    <visual>
+      <geometry>
+        <cylinder length="${h}" radius="${r}"/>
+      </geometry>
+    </visual>
+    <visual>
+      <geometry>
+        <cylinder length="${h}" radius="${r}"/>
+      </geometry>
+    </visual>
+</link>
+<joint name="passive_joint" type="prismatic">
+    <parent link="base_link"/>
+    <child link="pelvis"/>
+    <origin xyz="${r+0.05} 0. ${c/2. + h/2.}"/>
+    <axis xyz="0 0 1"/>
+    <limit effort="1000.0" lower="${-c}" upper="0." velocity="100."/>
 </joint>
-<xacro:if value="${ADD_UPPER_BODY}">
-	<xacro:include filename="$(find centauro_urdf)/urdf/parts/centauro_torso.urdf.xacro" />
-    <xacro:include filename="$(find centauro_urdf)/urdf/parts/arms.urdf.xacro" />
-	<xacro:if value="${ADD_BALL_END_EFFECTOR}">
-		<xacro:include filename="$(find centauro_urdf)/urdf/parts/ball.urdf.xacro" />
-		<xacro:ball_end_effector arm_num="1"  parent_link="arm1_7">
-      			<origin xyz="0. 0. 0." rpy="0. 0. 0."/>
-   		</xacro:ball_end_effector>
-		<xacro:ball_end_effector arm_num="2"  parent_link="arm2_7">
-      			<origin xyz="0. 0. 0." rpy="0. 0. 0."/>
-   		</xacro:ball_end_effector>
-	</xacro:if>
-	<xacro:include filename="$(find centauro_urdf)/urdf/parts/head.urdf.xacro" />
-</xacro:if>
-<xacro:if value="${ADD_LEGS}">
+<xacro:include filename="$(find centauro_urdf)/urdf/parts/centauro_leg.urdf.xacro" />
+<xacro:centauro_leg leg_num="1" origin_x="0" origin_y="0" />
+<!-- <xacro:if value="${ADD_LEGS}">
 	<xacro:include filename="$(find centauro_urdf)/urdf/parts/legs.urdf.xacro" />
-</xacro:if>
+</xacro:if> -->
 </robot>

File: centauro_urdf/urdf/centauro_robot.urdf.xacro (robot description, xacro)
@@ -7,7 +7,5 @@
   -->
   <xacro:include filename="$(find centauro_urdf)/urdf/centauro.urdf.xacro" />
-  <xacro:include filename="$(find centauro_urdf)/urdf/gazebo/centauro.gazebo.xacro" />
-  <!--xacro:include filename="$(find cogimon_urdf)/urdf/gazebo/force_torque.gazebo.xacro" /-->
-  <xacro:include filename="$(find centauro_urdf)/urdf/gazebo/imu.gazebo.xacro" />
+  <!-- <xacro:include filename="$(find centauro_urdf)/urdf/gazebo/centauro.gazebo.xacro" /> -->
   <xacro:include filename="$(find centauro_urdf)/urdf/gazebo/xbot.gazebo.xacro" />
   <xacro:include filename="$(find centauro_urdf)/urdf/gazebo/materials.gazebo.xacro" />

File: centauro_urdf/urdf/config/centauro.urdf.xacro (robot description, xacro)
@@ -12,4 +12,4 @@
 <xacro:property name="ADD_BALL_END_EFFECTOR" value="true" />
 <xacro:property name="ADD_FLOATING_BASE" value="$(arg add_legs)" />
-<xacro:property name="USE_STICKS" value="false" />
+<xacro:property name="USE_STICKS" value="true" />
 </robot>

File: centauro_urdf/urdf/parts/centauro_leg.urdf.xacro (robot description, xacro)
@@ -157,10 +157,10 @@
 </link>
 </xacro:unless>
-<joint name="hip_yaw_${leg_num}" type="revolute">
+<joint name="hip_yaw_${leg_num}" type="fixed">
 	<parent link="pelvis"/>
 	<child link="hip1_${leg_num}"/>
-	<origin xyz="${origin_x*Leg_1_Ox} ${origin_y*Leg_1_Oy} ${Leg_1_Oz}" rpy="${Leg_1_roll} ${Leg_1_pitch} ${PI/2-origin_x*PI/2+origin_x*origin_y*Leg_1_yaw}"/>
-	<axis xyz="0 0 1"/>
-        <limit lower="${hip_yaw_lower[leg_num-1]}" upper="${hip_yaw_upper[leg_num-1]}" effort="${motor_A_effort}" velocity="${motor_A_velocity}"/> <!-- 200 Nm, 1 rad/s-->
+	<origin xyz="${origin_x*Leg_1_Ox} ${origin_y*Leg_1_Oy} ${Leg_1_Oz}" rpy="${Leg_1_roll} ${Leg_1_pitch} ${-origin_x*PI/2+origin_x*origin_y*Leg_1_yaw}"/>
+	<!-- axis xyz="0 0 1"/>
+        <limit lower="${hip_yaw_lower[leg_num-1]}" upper="${hip_yaw_upper[leg_num-1]}" effort="${motor_A_effort}" velocity="${motor_A_velocity}"/--> <!-- 200 Nm, 1 rad/s-->
 </joint>
 <joint name="hip_pitch_${leg_num}" type="revolute">
