Commit message: fixed wrong mesh path in case of use with RViz
Signed-off-by: Andrea Patrizi <andreapatrizi1b6e6@gmail.com>

File: centauro_urdf/urdf/centauro.urdf.xacro (robot description, xacro)
@@ -5,4 +5,16 @@
 <xacro:arg name="centauro_root" default="$(find centauro_urdf)" />
 <xacro:property name="CENTAURO_ROOT" value="$(arg centauro_root)" />
+<!-- setting use_abs_mesh_paths should be kept to false
+for use with tools like RViz, which does not accept plain
+abolute paths for mesh paths-->
+<xacro:arg name="use_abs_mesh_paths" default="false" />
+<xacro:property name="USE_ABS_MESH_PATHS" value="$(arg use_abs_mesh_paths)" />
+<xacro:if value="${USE_ABS_MESH_PATHS}">
+  <xacro:property name="MESH_PATH" value="${CENTAURO_ROOT}/meshes" />
+</xacro:if>
+<xacro:unless value="${USE_ABS_MESH_PATHS}">
+  <xacro:property name="MESH_PATH" value="package://centauro_urdf/meshes" />
+</xacro:unless>
+<!-- configuration -->
 <xacro:arg name="config" default="${CENTAURO_ROOT}/urdf/config/centauro.urdf.xacro"/>
 <!-- ************ MODEL CONFIGURATION ************ -->
@@ -34,5 +46,5 @@
   <joint name="reference" type="floating">
     <parent link="world"/>
-    <child link="pelvis"/>
+    <child link="base_link"/>
 </joint>
 </xacro:if>

File: centauro_urdf/urdf/centauro_base.urdf.xacro (robot description, xacro)
@@ -24,5 +24,5 @@
             <origin xyz="0.0 0 0.0" rpy="0.0 0.0 0.0" />
             <geometry>
-                <mesh filename="${CENTAURO_ROOT}/meshes/v2/pelvis.stl" scale="0.001 0.001 0.001" />
+                <mesh filename="${MESH_PATH}/v2/pelvis.stl" scale="0.001 0.001 0.001" />
             </geometry>
         </visual>
@@ -30,5 +30,5 @@
             <origin xyz="0.0 0 0.0" rpy="0.0 0.0 0.0" />
             <geometry>
-                <mesh filename="${CENTAURO_ROOT}/meshes/simple/pelvis.stl" scale="0.001 0.001 0.001" />
+                <mesh filename="${MESH_PATH}/simple/pelvis.stl" scale="0.001 0.001 0.001" />
             </geometry>
         </collision>
@@ -98,5 +98,5 @@
                     <geometry>
                         <!-- <box size="${d435_cam_width} ${d435_cam_height} ${d435_cam_depth}"/> -->
-                        <mesh filename="${CENTAURO_ROOT}/meshes/realsense/d435.dae" />
+                        <mesh filename="${MESH_PATH}/realsense/d435.dae" />
                     </geometry>
                     <material name="${d435_base_name}_aluminum" />

File: centauro_urdf/urdf/centauro_robot.urdf.xacro (robot description, xacro)
@@ -10,4 +10,15 @@
   <xacro:arg name="centauro_root" default="$(find centauro_urdf)" />
   <xacro:property name="CENTAURO_ROOT" value="$(arg centauro_root)" />
+  <!-- setting use_abs_mesh_paths should be kept to false
+  for use with tools like RViz, which does not accept plain
+  abolute paths for mesh paths-->
+  <xacro:arg name="use_abs_mesh_paths" default="false" />
+  <xacro:property name="USE_ABS_MESH_PATHS" value="$(arg use_abs_mesh_paths)" />
+  <xacro:if value="${USE_ABS_MESH_PATHS}">
+    <xacro:property name="MESH_PATH" value="${CENTAURO_ROOT}/meshes" />
+  </xacro:if>
+  <xacro:unless value="${USE_ABS_MESH_PATHS}">
+    <xacro:property name="MESH_PATH" value="package://centauro_urdf/meshes" />
+  </xacro:unless>
   <xacro:include filename="${CENTAURO_ROOT}/urdf/centauro.urdf.xacro" />
   <xacro:include filename="${CENTAURO_ROOT}/urdf/gazebo/centauro.gazebo.xacro" />
@@ -18,5 +29,5 @@
       <joint name="reference" type="fixed">
       <parent link="world"/>
-      <child link="pelvis"/>
+      <child link="base_link"/>
     </joint>
   </xacro:unless>

File: centauro_urdf/urdf/centauro_virtual_frame.urdf (robot description, URDF)
Before this commit: robot centauro, 64 links, 63 joints
Links:
- link D435_head_camera_link: geometry collision box size=0.02505 0.09 0.025; visual mesh filename=${MESH_PATH}/realsense/d435.dae
- link D435i_camera_link: geometry collision box size=0.02505 0.09 0.025; visual mesh filename=${MESH_PATH}/realsense/d435.dae
- link ankle1_1: geometry collision mesh filename=${MESH_PATH}/v2/collision/ankle-pitch.stl scale=0.001 0.001 -0.001; visual mesh filename=${MESH_PATH}/v2/ankle-pitch.stl scale=0.001 0.001 -0.001
- link ankle1_2: geometry collision mesh filename=${MESH_PATH}/v2/collision/ankle-pitch.stl scale=0.001 0.001 0.001; visual mesh filename=${MESH_PATH}/v2/ankle-pitch.stl scale=0.001 0.001 0.001
- link ankle1_3: geometry collision mesh filename=${MESH_PATH}/v2/collision/ankle-pitch.stl scale=0.001 0.001 -0.001; visual mesh filename=${MESH_PATH}/v2/ankle-pitch.stl scale=0.001 0.001 -0.001
- link ankle1_4: geometry collision mesh filename=${MESH_PATH}/v2/collision/ankle-pitch.stl scale=0.001 0.001 0.001; visual mesh filename=${MESH_PATH}/v2/ankle-pitch.stl scale=0.001 0.001 0.001
- link ankle2_1: geometry collision mesh filename=${MESH_PATH}/v2/collision/mesh_ankle-yaw_wheel23.stl scale=0.001 -0.001 0.001; visual mesh filename=${MESH_PATH}/v2/mesh_ankle-yaw_wheel23.stl scale=0.001 -0.001 0.001
- link ankle2_2: geometry collision mesh filename=${MESH_PATH}/v2/collision/mesh_ankle-yaw_wheel23.stl scale=0.001 0.001 0.001; visual mesh filename=${MESH_PATH}/v2/mesh_ankle-yaw_wheel23.stl scale=0.001 0.001 0.001
- link ankle2_3: geometry collision mesh filename=${MESH_PATH}/v2/collision/mesh_ankle-yaw_wheel23.stl scale=0.001 -0.001 0.001; visual mesh filename=${MESH_PATH}/v2/mesh_ankle-yaw_wheel23.stl scale=0.001 -0.001 0.001
- link ankle2_4: geometry collision mesh filename=${MESH_PATH}/v2/collision/mesh_ankle-yaw_wheel23.stl scale=0.001 0.001 0.001; visual mesh filename=${MESH_PATH}/v2/mesh_ankle-yaw_wheel23.stl scale=0.001 0.001 0.001
- link arm1_1: geometry collision mesh filename=${MESH_PATH}/simple/ShoulderPitch.STL scale=0.001 -0.001 0.001; visual mesh filename=${MESH_PATH}/ShoulderPitch.STL scale=0.001 -0.001 0.001
- link arm1_2: geometry collision mesh filename=${MESH_PATH}/simple/ShoulderRoll.STL scale=0.001 -0.001 0.001; visual mesh filename=${MESH_PATH}/ShoulderRoll.STL scale=0.001 -0.001 0.001
- link arm1_3: geometry collision mesh filename=${MESH_PATH}/simple/ShoulderYaw.STL scale=0.001 -0.001 0.001; visual mesh filename=${MESH_PATH}/ShoulderYaw.STL scale=0.001 -0.001 0.001
- link arm1_4: geometry collision mesh filename=${MESH_PATH}/simple/Elbow.STL scale=0.001 -0.001 0.001; visual mesh filename=${MESH_PATH}/Elbow.STL scale=0.001 -0.001 0.001
- link arm1_5: geometry collision mesh filename=${MESH_PATH}/simple/Forearm.STL scale=0.001 -0.001 0.001; visual mesh filename=${MESH_PATH}/Forearm.STL scale=0.001 -0.001 0.001
- link arm1_6: geometry collision mesh filename=${MESH_PATH}/simple/wrist_pitch_right.stl scale=0.001 -0.001 0.001; visual mesh filename=${MESH_PATH}/wrist_pitch_right.stl scale=0.001 -0.001 0.001
- link arm2_1: geometry collision mesh filename=${MESH_PATH}/simple/ShoulderPitch.STL scale=0.001 0.001 0.001; visual mesh filename=${MESH_PATH}/ShoulderPitch.STL scale=0.001 0.001 0.001
- link arm2_2: geometry collision mesh filename=${MESH_PATH}/simple/ShoulderRoll.STL scale=0.001 0.001 0.001; visual mesh filename=${MESH_PATH}/ShoulderRoll.STL scale=0.001 0.001 0.001
- link arm2_3: geometry collision mesh filename=${MESH_PATH}/simple/ShoulderYaw.STL scale=0.001 0.001 0.001; visual mesh filename=${MESH_PATH}/ShoulderYaw.STL scale=0.001 0.001 0.001
- link arm2_4: geometry collision mesh filename=${MESH_PATH}/simple/Elbow.STL scale=0.001 0.001 0.001; visual mesh filename=${MESH_PATH}/Elbow.STL scale=0.001 0.001 0.001
- link arm2_5: geometry collision mesh filename=${MESH_PATH}/simple/Forearm.STL scale=0.001 0.001 0.001; visual mesh filename=${MESH_PATH}/Forearm.STL scale=0.001 0.001 0.001
- link arm2_6: geometry collision mesh filename=${MESH_PATH}/simple/wrist_pitch_right.stl scale=0.001 0.001 0.001; visual mesh filename=${MESH_PATH}/wrist_pitch_right.stl scale=0.001 0.001 0.001
- link ball1: geometry collision mesh filename=${MESH_PATH}/simple/BallHand.stl scale=0.001 0.001 0.001; visual mesh filename=${MESH_PATH}/BallHand.stl scale=0.001 0.001 0.001
- link ball2: geometry collision mesh filename=${MESH_PATH}/simple/BallHand.stl scale=0.001 0.001 0.001; visual mesh filename=${MESH_PATH}/BallHand.stl scale=0.001 0.001 0.001
- link d435_head_motor: geometry collision mesh filename=${MESH_PATH}/simple/neck-pitch_mesh.stl scale=0.001 0.001 0.001; visual mesh filename=${MESH_PATH}/neck-pitch_mesh.stl scale=0.001 0.001 0.001
- link hip1_1: geometry collision mesh filename=${MESH_PATH}/v2/collision/hip-yaw.stl scale=0.001 -0.001 0.001; visual mesh filename=${MESH_PATH}/v2/hip-yaw.stl scale=0.001 -0.001 0.001
- link hip1_2: geometry collision mesh filename=${MESH_PATH}/v2/collision/hip-yaw.stl scale=0.001 0.001 0.001; visual mesh filename=${MESH_PATH}/v2/hip-yaw.stl scale=0.001 0.001 0.001
- link hip1_3: geometry collision mesh filename=${MESH_PATH}/v2/collision/hip-yaw.stl scale=0.001 -0.001 0.001; visual mesh filename=${MESH_PATH}/v2/hip-yaw.stl scale=0.001 -0.001 0.001
- link hip1_4: geometry collision mesh filename=${MESH_PATH}/v2/collision/hip-yaw.stl scale=0.001 0.001 0.001; visual mesh filename=${MESH_PATH}/v2/hip-yaw.stl scale=0.001 0.001 0.001
- link hip2_1: geometry collision mesh filename=${MESH_PATH}/v2/collision/hip-pitch.stl scale=0.001 0.001 -0.001; visual mesh filename=${MESH_PATH}/v2/hip-pitch.stl scale=0.001 0.001 -0.001
- link hip2_2: geometry collision mesh filename=${MESH_PATH}/v2/collision/hip-pitch.stl scale=0.001 0.001 0.001; visual mesh filename=${MESH_PATH}/v2/hip-pitch.stl scale=0.001 0.001 0.001
- link hip2_3: geometry collision mesh filename=${MESH_PATH}/v2/collision/hip-pitch.stl scale=0.001 0.001 -0.001; visual mesh filename=${MESH_PATH}/v2/hip-pitch.stl scale=0.001 0.001 -0.001
- link hip2_4: geometry collision mesh filename=${MESH_PATH}/v2/collision/hip-pitch.stl scale=0.001 0.001 0.001; visual mesh filename=${MESH_PATH}/v2/hip-pitch.stl scale=0.001 0.001 0.001
- link knee_1: geometry collision mesh filename=${MESH_PATH}/v2/collision/knee.stl scale=0.001 0.001 -0.001; visual mesh filename=${MESH_PATH}/v2/knee.stl scale=0.001 0.001 -0.001
- link knee_2: geometry collision mesh filename=${MESH_PATH}/v2/collision/knee.stl scale=0.001 0.001 0.001; visual mesh filename=${MESH_PATH}/v2/knee.stl scale=0.001 0.001 0.001
- link knee_3: geometry collision mesh filename=${MESH_PATH}/v2/collision/knee.stl scale=0.001 0.001 -0.001; visual mesh filename=${MESH_PATH}/v2/knee.stl scale=0.001 0.001 -0.001
- link knee_4: geometry collision mesh filename=${MESH_PATH}/v2/collision/knee.stl scale=0.001 0.001 0.001; visual mesh filename=${MESH_PATH}/v2/knee.stl scale=0.001 0.001 0.001
- link neck_1: geometry collision mesh filename=${MESH_PATH}/simple/head-base_mesh.stl scale=0.001 0.001 0.001; visual mesh filename=${MESH_PATH}/head-base_mesh.stl scale=0.001 0.001 0.001
- link pelvis: geometry collision mesh filename=${MESH_PATH}/simple/pelvis.stl scale=0.001 0.001 0.001; visual mesh filename=${MESH_PATH}/v2/pelvis.stl scale=0.001 0.001 0.001
- link torso_2: geometry collision mesh filename=${MESH_PATH}/simple/link1_no_head.stl scale=0.001 0.001 0.001; visual mesh filename=${MESH_PATH}/link1_no_head.stl scale=0.001 0.001 0.001
- link velodyne_motor: geometry collision mesh filename=${MESH_PATH}/simple/lidar_mesh.stl scale=0.001 0.001 0.001; visual mesh filename=${MESH_PATH}/lidar_mesh.stl scale=0.001 0.001 0.001
- link wheel_1: geometry collision mesh filename=${MESH_PATH}/v2/collision/mesh_wheel23.stl scale=0.001 0.001 -0.001; visual mesh filename=${MESH_PATH}/v2/mesh_wheel23.stl scale=0.001 0.001 -0.001
- link wheel_2: geometry collision mesh filename=${MESH_PATH}/v2/collision/mesh_wheel23.stl scale=0.001 0.001 0.001; visual mesh filename=${MESH_PATH}/v2/mesh_wheel23.stl scale=0.001 0.001 0.001
- link wheel_3: geometry collision mesh filename=${MESH_PATH}/v2/collision/mesh_wheel23.stl scale=0.001 0.001 -0.001; visual mesh filename=${MESH_PATH}/v2/mesh_wheel23.stl scale=0.001 0.001 -0.001
- link wheel_4: geometry collision mesh filename=${MESH_PATH}/v2/collision/mesh_wheel23.stl scale=0.001 0.001 0.001; visual mesh filename=${MESH_PATH}/v2/mesh_wheel23.stl scale=0.001 0.001 0.001

File: centauro_urdf/urdf/centauro_virtual_frame_capsule.urdf (robot description, URDF)
Before this commit: robot centauro, 64 links, 63 joints
Links:
- link D435_head_camera_link: geometry collision box size=0.02505 0.09 0.025; visual mesh filename=${MESH_PATH}/realsense/d435.dae
- link D435i_camera_link: geometry collision box size=0.02505 0.09 0.025; visual mesh filename=${MESH_PATH}/realsense/d435.dae
- link ankle1_1: geometry collision cylinder length=0.049256315666076876 radius=0.0792379; collision sphere radius=0.0792379
- link ankle1_2: geometry collision cylinder length=0.04788405128558378 radius=0.0781037; collision sphere radius=0.0781037
- link ankle1_3: geometry collision cylinder length=0.049256315666076876 radius=0.0792379; collision sphere radius=0.0792379
- link ankle1_4: geometry collision cylinder length=0.04788405128558378 radius=0.0781037; collision sphere radius=0.0781037
- link ankle2_1: geometry collision cylinder length=0.07370263129636398 radius=0.0813545; collision sphere radius=0.0813545
- link ankle2_2: geometry collision cylinder length=0.07370263129636398 radius=0.0813545; collision sphere radius=0.0813545
- link ankle2_3: geometry collision cylinder length=0.07370263129636398 radius=0.0813545; collision sphere radius=0.0813545
- link ankle2_4: geometry collision cylinder length=0.07370263129636398 radius=0.0813545; collision sphere radius=0.0813545
- link arm1_1: geometry collision cylinder length=0.03739768494560427 radius=0.0698859; collision sphere radius=0.0698859
- link arm1_2: geometry collision cylinder length=0.12799269981445732 radius=0.0700645; collision sphere radius=0.0700645
- link arm1_3: geometry collision cylinder length=0.06082252644344949 radius=0.0896121; collision sphere radius=0.0896121
- link arm1_4: geometry collision cylinder length=0.08713418572944408 radius=0.0600429; collision sphere radius=0.0600429
- link arm1_5: geometry collision cylinder length=0.08434739747702645 radius=0.0804108; collision sphere radius=0.0804108
- link arm1_6: geometry collision cylinder length=0.07750977987441161 radius=0.0474698; collision sphere radius=0.0474698
- link arm2_1: geometry collision cylinder length=0.03739768494560427 radius=0.0698859; collision sphere radius=0.0698859
- link arm2_2: geometry collision cylinder length=0.12799269981445732 radius=0.0700645; collision sphere radius=0.0700645
- link arm2_3: geometry collision cylinder length=0.06082252644344949 radius=0.0896121; collision sphere radius=0.0896121
- link arm2_4: geometry collision cylinder length=0.08713418572944408 radius=0.0600429; collision sphere radius=0.0600429
- link arm2_5: geometry collision cylinder length=0.08434739747702645 radius=0.0804108; collision sphere radius=0.0804108
- link arm2_6: geometry collision cylinder length=0.07750977987441161 radius=0.0474698; collision sphere radius=0.0474698
- link ball1: geometry collision cylinder length=9.940076835940455e-05 radius=0.0709883; collision sphere radius=0.0709883
- link ball2: geometry collision cylinder length=9.940076835940455e-05 radius=0.0709883; collision sphere radius=0.0709883
- link d435_head_motor: geometry collision cylinder length=0.12134423548428976 radius=0.0261699; collision sphere radius=0.0261699
- link hip1_1: geometry collision cylinder length=0.03069545889898954 radius=0.0747223; collision sphere radius=0.0747223
- link hip1_2: geometry collision cylinder length=0.03069545889898954 radius=0.0747223; collision sphere radius=0.0747223
- link hip1_3: geometry collision cylinder length=0.03069545889898954 radius=0.0747223; collision sphere radius=0.0747223
- link hip1_4: geometry collision cylinder length=0.03069545889898954 radius=0.0747223; collision sphere radius=0.0747223
- link hip2_1: geometry collision cylinder length=0.2919804521727749 radius=0.0808941; collision sphere radius=0.0808941
- link hip2_2: geometry collision cylinder length=0.2919804521727749 radius=0.0808941; collision sphere radius=0.0808941
- link hip2_3: geometry collision cylinder length=0.2919804521727749 radius=0.0808941; collision sphere radius=0.0808941
- link hip2_4: geometry collision cylinder length=0.2919804521727749 radius=0.0808941; collision sphere radius=0.0808941
- link knee_1: geometry collision cylinder length=0.1927502246061244 radius=0.0664305; collision sphere radius=0.0664305
- link knee_2: geometry collision cylinder length=0.1927502246061244 radius=0.0664305; collision sphere radius=0.0664305
- link knee_3: geometry collision cylinder length=0.1927502246061244 radius=0.0664305; collision sphere radius=0.0664305
- link knee_4: geometry collision cylinder length=0.1927502246061244 radius=0.0664305; collision sphere radius=0.0664305
- link neck_1: geometry collision cylinder length=0.16454098025546557 radius=0.100414; collision sphere radius=0.100414
- link pelvis: geometry collision cylinder length=0.38594139791384763 radius=0.213204; collision sphere radius=0.213204
- link torso_2: geometry collision cylinder length=0.09543675990850982 radius=0.158224; collision sphere radius=0.158224
- link velodyne_motor: geometry collision cylinder length=0.032463112134515464 radius=0.0544637; collision sphere radius=0.0544637
- link wheel_1: geometry collision cylinder length=0.11 radius=0.078; collision sphere radius=0.078
- link wheel_2: geometry collision cylinder length=0.11 radius=0.078; collision sphere radius=0.078
- link wheel_3: geometry collision cylinder length=0.11 radius=0.078; collision sphere radius=0.078
- link wheel_4: geometry collision cylinder length=0.11 radius=0.078; collision sphere radius=0.078

File: centauro_urdf/urdf/parts/ball.urdf.xacro (robot description, xacro)
@@ -11,5 +11,5 @@
       <origin xyz="0.0 0.0 0.0" rpy="0.0 0.0 0.0"/>
       <geometry name="ball${arm_num}_visual">
-        <mesh filename="${CENTAURO_ROOT}/meshes/BallHand.stl" scale="0.001 0.001 0.001" />
+        <mesh filename="${MESH_PATH}/BallHand.stl" scale="0.001 0.001 0.001" />
       </geometry>
       <material name="dark_grey"/>
@@ -18,5 +18,5 @@
       <origin xyz="0.0 0.0 0.0" rpy="0.0 0.0 0.0"/>
       <geometry name="ball${arm_num}_collision">
-        <mesh filename="${CENTAURO_ROOT}/meshes/simple/BallHand.stl" scale="0.001 0.001 0.001" />
+        <mesh filename="${MESH_PATH}/simple/BallHand.stl" scale="0.001 0.001 0.001" />
       </geometry>
    </collision>
