Commit message: fixed wrong mesh path in case of use with RViz
Signed-off-by: Andrea Patrizi <andreapatrizi1b6e6@gmail.com>

File: centauro_urdf/urdf/parts/centauro_arm.urdf.xacro (robot description, xacro)
@@ -14,5 +14,5 @@
    <origin xyz="0.0 0.0 0.0"  rpy="0.0 0.0 0.0"/>
    <geometry>
-      <mesh filename="${CENTAURO_ROOT}/meshes/ShoulderPitch.STL" scale="0.001 ${-rot*0.001} 0.001" />
+      <mesh filename="${MESH_PATH}/ShoulderPitch.STL" scale="0.001 ${-rot*0.001} 0.001" />
    </geometry>
          <material name="dark_grey"/>
@@ -21,5 +21,5 @@
    <origin xyz="0.0 0.0 0.0"  rpy="0.0 0.0 0.0"/>
    <geometry>
-      <mesh filename="${CENTAURO_ROOT}/meshes/simple/ShoulderPitch.STL" scale="0.001 ${-rot*0.001} 0.001" />
+      <mesh filename="${MESH_PATH}/simple/ShoulderPitch.STL" scale="0.001 ${-rot*0.001} 0.001" />
    </geometry>
       </collision>
@@ -36,11 +36,11 @@
          <origin xyz="0.0 0.0 0.0"  rpy="0.0 0.0 0.0"/>
    <geometry>
-      <mesh filename="${CENTAURO_ROOT}/meshes/ShoulderRoll.STL" scale="0.001 ${-rot*0.001} 0.001" />
-   </geometry>
-      </visual>
-      <collision>
-         <origin xyz="0.0 0.0 0.0"  rpy="0.0 0.0 0.0"/>
-   <geometry>
-      <mesh filename="${CENTAURO_ROOT}/meshes/simple/ShoulderRoll.STL" scale="0.001 ${-rot*0.001} 0.001" />
+      <mesh filename="${MESH_PATH}/ShoulderRoll.STL" scale="0.001 ${-rot*0.001} 0.001" />
+   </geometry>
+      </visual>
+      <collision>
+         <origin xyz="0.0 0.0 0.0"  rpy="0.0 0.0 0.0"/>
+   <geometry>
+      <mesh filename="${MESH_PATH}/simple/ShoulderRoll.STL" scale="0.001 ${-rot*0.001} 0.001" />
    </geometry>
       </collision>
@@ -57,12 +57,12 @@
          <origin xyz="0.0 0.0 0.0"  rpy="0.0 0.0 0.0"/>
    <geometry>
-      <mesh filename="${CENTAURO_ROOT}/meshes/ShoulderYaw.STL" scale="0.001 ${-rot*0.001} 0.001" />
-   </geometry>
-         <material name="dark_grey"/>
-      </visual>
-      <collision>
-         <origin xyz="0.0 0.0 0.0"  rpy="0.0 0.0 0.0"/>
-   <geometry>
-      <mesh filename="${CENTAURO_ROOT}/meshes/simple/ShoulderYaw.STL" scale="0.001 ${-rot*0.001} 0.001" />
+      <mesh filename="${MESH_PATH}/ShoulderYaw.STL" scale="0.001 ${-rot*0.001} 0.001" />
+   </geometry>
+         <material name="dark_grey"/>
+      </visual>
+      <collision>
+         <origin xyz="0.0 0.0 0.0"  rpy="0.0 0.0 0.0"/>
+   <geometry>
+      <mesh filename="${MESH_PATH}/simple/ShoulderYaw.STL" scale="0.001 ${-rot*0.001} 0.001" />
    </geometry>
       </collision>
@@ -79,11 +79,11 @@
          <origin xyz="0.0 0.0 0.0"  rpy="0.0 0.0 0.0"/>
    <geometry>
-      <mesh filename="${CENTAURO_ROOT}/meshes/Elbow.STL" scale="0.001 ${-rot*0.001} 0.001" />
-   </geometry>
-      </visual>
-      <collision>
-         <origin xyz="0.0 0.0 0.0"  rpy="0.0 0.0 0.0"/>
-   <geometry>
-      <mesh filename="${CENTAURO_ROOT}/meshes/simple/Elbow.STL" scale="0.001 ${-rot*0.001} 0.001" />
+      <mesh filename="${MESH_PATH}/Elbow.STL" scale="0.001 ${-rot*0.001} 0.001" />
+   </geometry>
+      </visual>
+      <collision>
+         <origin xyz="0.0 0.0 0.0"  rpy="0.0 0.0 0.0"/>
+   <geometry>
+      <mesh filename="${MESH_PATH}/simple/Elbow.STL" scale="0.001 ${-rot*0.001} 0.001" />
    </geometry>
       </collision>
@@ -100,12 +100,12 @@
          <origin xyz="0.0 0.0 0.0"  rpy="0.0 0.0 0.0"/>
    <geometry>
-      <mesh filename="${CENTAURO_ROOT}/meshes/Forearm.STL" scale="0.001 ${-rot*0.001} 0.001" />
-   </geometry>
-         <material name="dark_grey"/>
-      </visual>
-      <collision>
-         <origin xyz="0.0 0.0 0.0"  rpy="0.0 0.0 0.0"/>
-   <geometry>
-      <mesh filename="${CENTAURO_ROOT}/meshes/simple/Forearm.STL" scale="0.001 ${-rot*0.001} 0.001" />
+      <mesh filename="${MESH_PATH}/Forearm.STL" scale="0.001 ${-rot*0.001} 0.001" />
+   </geometry>
+         <material name="dark_grey"/>
+      </visual>
+      <collision>
+         <origin xyz="0.0 0.0 0.0"  rpy="0.0 0.0 0.0"/>
+   <geometry>
+      <mesh filename="${MESH_PATH}/simple/Forearm.STL" scale="0.001 ${-rot*0.001} 0.001" />
    </geometry>
       </collision>
@@ -122,11 +122,11 @@
          <origin xyz="0.0 0.0 0.0"  rpy="0.0 0.0 0.0"/>
    <geometry>
-      <mesh filename="${CENTAURO_ROOT}/meshes/wrist_pitch_right.stl" scale="0.001 ${-rot*0.001} 0.001" />
-   </geometry>
-      </visual>
-      <collision>
-         <origin xyz="0.0 0.0 0.0"  rpy="0.0 0.0 0.0"/>
-   <geometry>
-      <mesh filename="${CENTAURO_ROOT}/meshes/simple/wrist_pitch_right.stl" scale="0.001 ${-rot*0.001} 0.001" />
+      <mesh filename="${MESH_PATH}/wrist_pitch_right.stl" scale="0.001 ${-rot*0.001} 0.001" />
+   </geometry>
+      </visual>
+      <collision>
+         <origin xyz="0.0 0.0 0.0"  rpy="0.0 0.0 0.0"/>
+   <geometry>
+      <mesh filename="${MESH_PATH}/simple/wrist_pitch_right.stl" scale="0.001 ${-rot*0.001} 0.001" />
    </geometry>
       </collision>
@@ -142,12 +142,12 @@
          <origin xyz="0.0 0.0 0.0"  rpy="0.0 0.0 0.0"/>
    <geometry>
-      <mesh filename="${CENTAURO_ROOT}/meshes/ForearmYaw.STL" scale="0.001 ${-rot*0.001} 0.001" />
-   </geometry>
-         <material name="dark_grey"/>
-      </visual>
-      <collision>
-         <origin xyz="0.0 0.0 0.0"  rpy="0.0 0.0 0.0"/>
-   <geometry>
-      <mesh filename="${CENTAURO_ROOT}/meshes/simple/ForearmYaw.STL" scale="0.001 ${-rot*0.001} 0.001" />
+      <mesh filename="${MESH_PATH}/ForearmYaw.STL" scale="0.001 ${-rot*0.001} 0.001" />
+   </geometry>
+         <material name="dark_grey"/>
+      </visual>
+      <collision>
+         <origin xyz="0.0 0.0 0.0"  rpy="0.0 0.0 0.0"/>
+   <geometry>
+      <mesh filename="${MESH_PATH}/simple/ForearmYaw.STL" scale="0.001 ${-rot*0.001} 0.001" />
    </geometry>
       </collision>
@@ -238,5 +238,5 @@
          <origin xyz="0.0 0.0 0.0"  rpy="${PI} 0.0 0.0"/>
    <geometry>
-      <mesh filename="${CENTAURO_ROOT}/meshes/Wrist.STL" scale="0.001 ${-rot*0.001} 0.001" />
+      <mesh filename="${MESH_PATH}/Wrist.STL" scale="0.001 ${-rot*0.001} 0.001" />
    </geometry>
       </visual-->
@@ -244,5 +244,5 @@
          <origin xyz="0.0 0.0 0.0"  rpy="${PI} 0.0 0.0"/>
    <geometry>
-      <mesh filename="${CENTAURO_ROOT}/meshes/simple/Wrist.STL" scale="0.001 ${-rot*0.001} 0.001" />
+      <mesh filename="${MESH_PATH}/simple/Wrist.STL" scale="0.001 ${-rot*0.001} 0.001" />
    </geometry>
       </collision-->

File: centauro_urdf/urdf/parts/centauro_leg.urdf.xacro (robot description, xacro)
@@ -14,5 +14,5 @@
       <origin xyz="0.0 0.0 0.0"  rpy="0.0 0.0 0.0"/>
       <geometry>
-         <mesh filename="${CENTAURO_ROOT}/meshes/v2/hip-yaw.stl" scale="0.001 ${mirror*0.001} 0.001" />
+         <mesh filename="${MESH_PATH}/v2/hip-yaw.stl" scale="0.001 ${mirror*0.001} 0.001" />
       </geometry>
       <material name="dark_grey"/>
@@ -21,5 +21,5 @@
       <origin xyz="0.0 0.0 0.0"  rpy="0.0 0.0 0.0"/>
       <geometry>
-         <mesh filename="${CENTAURO_ROOT}/meshes/v2/collision/hip-yaw.stl" scale="0.001 ${mirror*0.001} 0.001" />
+         <mesh filename="${MESH_PATH}/v2/collision/hip-yaw.stl" scale="0.001 ${mirror*0.001} 0.001" />
       </geometry>
    </collision>
@@ -34,5 +34,5 @@
       <origin xyz="0.0 0.0 0.0"  rpy="0.0 0.0 0.0"/>
       <geometry>
-         <mesh filename="${CENTAURO_ROOT}/meshes/v2/hip-pitch.stl" scale="0.001 0.001 ${mirror*0.001}" />
+         <mesh filename="${MESH_PATH}/v2/hip-pitch.stl" scale="0.001 0.001 ${mirror*0.001}" />
       </geometry>
    </visual>
@@ -40,5 +40,5 @@
       <origin xyz="0.0 0.0 0.0"  rpy="0.0 0.0 0.0"/>
       <geometry>
-         <mesh filename="${CENTAURO_ROOT}/meshes/v2/collision/hip-pitch.stl" scale="0.001 0.001 ${mirror*0.001}" />
+         <mesh filename="${MESH_PATH}/v2/collision/hip-pitch.stl" scale="0.001 0.001 ${mirror*0.001}" />
       </geometry>
    </collision>
@@ -57,5 +57,5 @@
          <material name="black"/>
          <geometry name="${leg_num}_stick_visual">
-         <mesh filename="${CENTAURO_ROOT}/meshes/front_right_stick.stl" scale="${mmTom} ${mmTom} ${mmTom}"/>
+         <mesh filename="${MESH_PATH}/front_right_stick.stl" scale="${mmTom} ${mmTom} ${mmTom}"/>
          </geometry>
    </visual>
@@ -63,5 +63,5 @@
          <origin xyz="0 0 0" rpy="${PI_2} 0 ${-PI_2}"/>
          <geometry name="${leg_num}_stick_collision">
-         <mesh filename="${CENTAURO_ROOT}/meshes/simple/front_right_stick.stl" scale="${mmTom} ${mmTom} ${mmTom}"/>
+         <mesh filename="${MESH_PATH}/simple/front_right_stick.stl" scale="${mmTom} ${mmTom} ${mmTom}"/>
          </geometry>
    </collision>
@@ -78,5 +78,5 @@
          <origin xyz="0.0 0.0 0.0"  rpy="0.0 0.0 0.0"/>
          <geometry>
-            <mesh filename="${CENTAURO_ROOT}/meshes/v2/knee.stl" scale="0.001 0.001 ${mirror*0.001}" />
+            <mesh filename="${MESH_PATH}/v2/knee.stl" scale="0.001 0.001 ${mirror*0.001}" />
          </geometry>
          <material name="dark_grey"/>
@@ -85,5 +85,5 @@
          <origin xyz="0.0 0.0 0.0"  rpy="0.0 0.0 0.0"/>
          <geometry>
-            <mesh filename="${CENTAURO_ROOT}/meshes/v2/collision/knee.stl" scale="0.001 0.001 ${mirror*0.001}" />
+            <mesh filename="${MESH_PATH}/v2/collision/knee.stl" scale="0.001 0.001 ${mirror*0.001}" />
          </geometry>
       </collision>
@@ -98,5 +98,5 @@
          <origin xyz="0.0 0.0 0.0"  rpy="0.0 0.0 0.0"/>
          <geometry>
-            <mesh filename="${CENTAURO_ROOT}/meshes/v2/ankle-pitch.stl" scale="0.001 0.001 ${mirror*0.001}" />
+            <mesh filename="${MESH_PATH}/v2/ankle-pitch.stl" scale="0.001 0.001 ${mirror*0.001}" />
          </geometry>
       </visual>
@@ -104,5 +104,5 @@
          <origin xyz="0.0 0.0 0.0"  rpy="0.0 0.0 0.0"/>
          <geometry>
-            <mesh filename="${CENTAURO_ROOT}/meshes/v2/collision/ankle-pitch.stl" scale="0.001 0.001 ${mirror*0.001}" />
+            <mesh filename="${MESH_PATH}/v2/collision/ankle-pitch.stl" scale="0.001 0.001 ${mirror*0.001}" />
          </geometry>
       </collision>

File: centauro_urdf/urdf/parts/centauro_torso.urdf.xacro (robot description, xacro)
@@ -11,5 +11,5 @@
           <origin xyz="0.0 0 0.0"  rpy="0.0 0.0 0.0"/>
    	  <geometry>
-      	  <mesh filename="${CENTAURO_ROOT}/meshes/link1_no_head.stl" scale="0.001 0.001 0.001" />
+      	  <mesh filename="${MESH_PATH}/link1_no_head.stl" scale="0.001 0.001 0.001" />
    	  </geometry>
 	</visual>
@@ -17,5 +17,5 @@
           <origin xyz="0.0 0 0.0"  rpy="0.0 0.0 0.0"/>
    	  <geometry>
-      	  <mesh filename="${CENTAURO_ROOT}/meshes/simple/link1_no_head.stl" scale="0.001 0.001 0.001" />
+      	  <mesh filename="${MESH_PATH}/simple/link1_no_head.stl" scale="0.001 0.001 0.001" />
    	  </geometry>
 	</collision>

File: centauro_urdf/urdf/parts/head.urdf.xacro (robot description, xacro)
@@ -12,5 +12,5 @@
       <origin rpy="0.0 0.0 0.0" xyz="0.0 0 0.0"/>
       <geometry>
-        <mesh filename="${CENTAURO_ROOT}/meshes/head-base_mesh.stl" scale="0.001 0.001 0.001"/>
+        <mesh filename="${MESH_PATH}/head-base_mesh.stl" scale="0.001 0.001 0.001"/>
       </geometry>
     </visual>
@@ -18,5 +18,5 @@
       <origin rpy="0.0 0.0 0.0" xyz="0.0 0 0.0"/>
       <geometry>
-        <mesh filename="${CENTAURO_ROOT}/meshes/simple/head-base_mesh.stl" scale="0.001 0.001 0.001"/>
+        <mesh filename="${MESH_PATH}/simple/head-base_mesh.stl" scale="0.001 0.001 0.001"/>
       </geometry>
     </collision>
@@ -32,5 +32,5 @@
       <origin rpy="0.0 0.0 0.0" xyz="0.0 0 0.0"/>
       <geometry>
-        <mesh filename="${CENTAURO_ROOT}/meshes/lidar_mesh.stl" scale="0.001 0.001 0.001"/>
+        <mesh filename="${MESH_PATH}/lidar_mesh.stl" scale="0.001 0.001 0.001"/>
       </geometry>
     </visual>
@@ -38,5 +38,5 @@
       <origin rpy="0.0 0.0 0.0" xyz="0.0 0 0.0"/>
       <geometry>
-        <mesh filename="${CENTAURO_ROOT}/meshes/simple/lidar_mesh.stl" scale="0.001 0.001 0.001"/>
+        <mesh filename="${MESH_PATH}/simple/lidar_mesh.stl" scale="0.001 0.001 0.001"/>
       </geometry>
     </collision>
@@ -52,5 +52,5 @@
       <origin rpy="0.0 0.0 0.0" xyz="0.0 0 0.0"/>
       <geometry>
-        <mesh filename="${CENTAURO_ROOT}/meshes/neck-pitch_mesh.stl" scale="0.001 0.001 0.001"/>
+        <mesh filename="${MESH_PATH}/neck-pitch_mesh.stl" scale="0.001 0.001 0.001"/>
       </geometry>
     </visual>
@@ -58,5 +58,5 @@
       <origin rpy="0.0 0.0 0.0" xyz="0.0 0 0.0"/>
       <geometry>
-        <mesh filename="${CENTAURO_ROOT}/meshes/simple/neck-pitch_mesh.stl" scale="0.001 0.001 0.001"/>
+        <mesh filename="${MESH_PATH}/simple/neck-pitch_mesh.stl" scale="0.001 0.001 0.001"/>
       </geometry>
     </collision>
@@ -139,5 +139,5 @@
         <geometry>
           <!-- <box size="${d435_cam_width} ${d435_cam_height} ${d435_cam_depth}"/> -->
-          <mesh filename="${CENTAURO_ROOT}/meshes/realsense/d435.dae"/>
+          <mesh filename="${MESH_PATH}/realsense/d435.dae"/>
         </geometry>
         <material name="${d435_head_name}_aluminum"/>

File: centauro_urdf/urdf/parts/wheel23.urdf.xacro (robot description, xacro)
@@ -13,5 +13,5 @@
                 <origin xyz="0.0 0.0 0.0" rpy="0.0 0.0 0.0" />
                 <geometry>
-                    <mesh filename="${CENTAURO_ROOT}/meshes/v2/mesh_ankle-yaw_wheel23.stl"
+                    <mesh filename="${MESH_PATH}/v2/mesh_ankle-yaw_wheel23.stl"
                         scale="0.001 ${mirror*0.001} 0.001" />
                 </geometry>
@@ -22,5 +22,5 @@
                 <geometry>
                     <mesh
-                        filename="${CENTAURO_ROOT}/meshes/v2/collision/mesh_ankle-yaw_wheel23.stl"
+                        filename="${MESH_PATH}/v2/collision/mesh_ankle-yaw_wheel23.stl"
                         scale="0.001 ${mirror*0.001} 0.001" />
                 </geometry>
@@ -46,5 +46,5 @@
                 <origin xyz="0.0 0.0 0.0" rpy="0.0 0.0 0.0" />
                 <geometry>
-                    <mesh filename="${CENTAURO_ROOT}/meshes/v2/mesh_wheel23.stl"
+                    <mesh filename="${MESH_PATH}/v2/mesh_wheel23.stl"
                         scale="0.001 0.001 ${mirror*0.001}" />
                 </geometry>
@@ -54,5 +54,5 @@
                 <origin xyz="0 0 0" rpy="0 0 0" />
                 <geometry>
-                    <mesh filename="${CENTAURO_ROOT}/meshes/v2/collision/mesh_wheel23.stl"
+                    <mesh filename="${MESH_PATH}/v2/collision/mesh_wheel23.stl"
                         scale="0.001 0.001 ${mirror*0.001}" />
                 </geometry>

Commit message: added flag to allow use with abs paths and rviz

File: centauro_urdf/urdf/centauro.urdf.xacro (robot description, xacro)
@@ -9,10 +9,17 @@
 abolute paths for mesh paths-->
 <xacro:arg name="use_abs_mesh_paths" default="false" />
+<xacro:arg name="use_local_filesys_for_meshes" default="false" />
 <xacro:property name="USE_ABS_MESH_PATHS" value="$(arg use_abs_mesh_paths)" />
+  <xacro:property name="USE_LOCAL_FILESYS_FOR_MESHES" value="$(arg use_local_filesys_for_meshes)" />
 <xacro:if value="${USE_ABS_MESH_PATHS}">
-  <xacro:property name="MESH_PATH" value="${CENTAURO_ROOT}/meshes" />
+    <xacro:if value="${USE_LOCAL_FILESYS_FOR_MESHES}">
+    <xacro:property name="MESH_PATH" value="file://${CENTAURO_ROOT}/meshes" />
+    </xacro:if>
+    <xacro:unless value="${USE_ABS_MESH_PATHS}">
+    <xacro:property name="MESH_PATH" value="${CENTAURO_ROOT}/meshes" />
+    </xacro:unless>
 </xacro:if>
 <xacro:unless value="${USE_ABS_MESH_PATHS}">
-  <xacro:property name="MESH_PATH" value="package://centauro_urdf/meshes" />
+    <xacro:property name="MESH_PATH" value="package://centauro_urdf/meshes" />
 </xacro:unless>
 <!-- configuration -->

Commit message: Signed-off-by: Andrea Patrizi <andreapatrizi1b6e6@gmail.com>

File: centauro_urdf/urdf/centauro.urdf.xacro (robot description, xacro)
@@ -16,5 +16,5 @@
     <xacro:property name="MESH_PATH" value="file://${CENTAURO_ROOT}/meshes" />
     </xacro:if>
-    <xacro:unless value="${USE_ABS_MESH_PATHS}">
+    <xacro:unless value="${USE_LOCAL_FILESYS_FOR_MESHES}">
     <xacro:property name="MESH_PATH" value="${CENTAURO_ROOT}/meshes" />
     </xacro:unless>
@@ -23,4 +23,7 @@
     <xacro:property name="MESH_PATH" value="package://centauro_urdf/meshes" />
 </xacro:unless>
+<xacro:macro name="example_macro">
+  <example_element message="${MESH_PATH}" />
+</xacro:macro>
 <!-- configuration -->
 <xacro:arg name="config" default="${CENTAURO_ROOT}/urdf/config/centauro.urdf.xacro"/>

Commit message: dont add the floating joint !

File: centauro_urdf/urdf/centauro.urdf.xacro (robot description, xacro)
@@ -7,13 +7,4 @@
 <xacro:include filename="$(find centauro_urdf)/urdf/centauro_base.urdf.xacro"/>
 <!-- ************ Control frames ************ -->
-<xacro:if value="${ADD_FLOATING_BASE}">
-<xacro:if value="${ADD_LEGS}">
-<link name="world"/>
-  <joint name="reference" type="floating">
-    <parent link="world"/>
-    <child link="pelvis"/>
-</joint>
-</xacro:if>
-</xacro:if>
 <xacro:if value="${ADD_VIRTUAL_FRAME}">
   <xacro:include filename="$(find centauro_urdf)/urdf/parts/virtual_frame.urdf.xacro"/>

Commit message: conditional add floatning base

File: centauro_urdf/urdf/centauro.urdf.xacro (robot description, xacro)
@@ -4,4 +4,11 @@
 <!-- ************ MODEL CONFIGURATION ************ -->
 <xacro:include filename="$(arg config)"/>
+<xacro:if value="${ADD_FLOATING_BASE}">
+  <link name="world"/>
+  <joint name="reference" type="floating">
+    <parent link="world"/>
+    <child link="pelvis"/>
+  </joint>
+</xacro:if>
 <!-- ************ Pholus plain model ************ -->
 <xacro:include filename="$(find centauro_urdf)/urdf/centauro_base.urdf.xacro"/>
