Commit message: added lower body

File: centauro_urdf/urdf/centauro_base.urdf.xacro (robot description, xacro)
@@ -6,24 +6,33 @@
 -->
 <xacro:include filename="$(find centauro_urdf)/urdf/utils.urdf.xacro" />
+<xacro:include filename="$(find centauro_urdf)/urdf/parts/kinematics_properties.urdf.xacro" />
+<xacro:include filename="$(find centauro_urdf)/urdf/parts/inertial_properties.urdf.xacro" />
+<xacro:include filename="$(find centauro_urdf)/urdf/parts/limits.urdf.xacro" />
 <link name="base_link"/>
 <link name="pelvis">
-    <inertial>
-      <origin xyz="0.0013890071 -0.0015989148 0.063101012"/>
-      <mass value="16.097574"/>
-      <inertia ixx="0.23912627" ixy="-0.0050541269" ixz="-0.019746055" iyy="0.71430078" iyz="0.0002131204" izz="0.81870448"/>
-    </inertial>
-    <visual>
-      <origin rpy="0.0 0.0 0.0" xyz="0.0 0 0.0"/>
-      <geometry>
-        <mesh filename="package://centauro_urdf/meshes/pelvis.stl" scale="0.001 0.001 0.001"/>
-      </geometry>
-    </visual>
-    <collision>
-      <origin rpy="0.0 0.0 0.0" xyz="0.0 0 0.0"/>
-      <geometry>
-        <mesh filename="package://centauro_urdf/meshes/simple/pelvis.stl" scale="0.001 0.001 0.001"/>
-      </geometry>
-    </collision>
-</link>
+      <inertial>
+         <origin xyz="${Pelvis_x} ${Pelvis_y} ${Pelvis_z}"/>
+         <mass value="${Pelvis_mass}"/>
+         <inertia ixx="${Pelvis_xx}" ixy="${Pelvis_xy}" ixz="${Pelvis_xz}" iyy="${Pelvis_yy}" iyz="${Pelvis_yz}" izz="${Pelvis_zz}"/>
+      </inertial>
+      <visual>
+        <origin xyz="0.0 0 0.0"  rpy="0.0 0.0 0.0"/>
+        <geometry>
+         <mesh filename="package://centauro_urdf/meshes/pelvis.stl" scale="0.001 0.001 0.001" />
+        </geometry>
+      </visual>
+      <collision>
+         <origin xyz="0.0 0 0.0"  rpy="0.0 0.0 0.0"/>
+        <geometry>
+         <mesh filename="package://centauro_urdf/meshes/simple/pelvis.stl" scale="0.001 0.001 0.001" />
+        </geometry>
+      </collision>
+   </link>
+    <link name="imu_link"/>
+    <joint name="imu_joint" type="fixed">
+        <parent link="pelvis"/>
+        <origin xyz="${Imu_Ox} ${Imu_Oy} ${Imu_Oz}" rpy="${Imu_raw} ${Imu_pitch} ${Imu_yaw}"/>
+        <child link="imu_link"/>
+    </joint>
 <joint name="base_joint" type="fixed">
     <parent link="base_link"/>
@@ -36,6 +45,6 @@
 	<xacro:include filename="$(find pholus_urdf)/urdf/parts/head.urdf.xacro" />
 </xacro:if-->
-<!--xacro:if value="${ADD_LEGS}">
-	<xacro:include filename="$(find pholus_urdf)/urdf/parts/legs.urdf.xacro" />
-</xacro:if-->
+<xacro:if value="${ADD_LEGS}">
+	<xacro:include filename="$(find centauro_urdf)/urdf/parts/legs.urdf.xacro" />
+</xacro:if>
 </robot>

File: centauro_urdf/urdf/parts/legs.urdf.xacro (robot description, xacro)
@@ -1,8 +1,12 @@
 <?xml version="1.0"?>
 <robot xmlns:xacro="http://ros.org/wiki/xacro">
-<xacro:include filename="$(find pholus_urdf)/urdf/parts/leg_macro.urdf.xacro" />
-<xacro:leg prefix="fr"  x="${250*mmTom}"  y="${-125*mmTom}" z="${-56.6*mmTom}" mirror_link="1"/>
-<xacro:leg prefix="fl"  x="${250*mmTom}"  y="${125*mmTom}"  z="${-56.6*mmTom}" mirror_link="-1"/>
-<xacro:leg prefix="hr"  x="${-250*mmTom}" y="${-125*mmTom}" z="${-56.6*mmTom}" mirror_link="1"/>
-<xacro:leg prefix="hl"  x="${-250*mmTom}" y="${125*mmTom}"  z="${-56.6*mmTom}" mirror_link="-1"/>
+<xacro:include filename="$(find centauro_urdf)/urdf/parts/centauro_leg.urdf.xacro" />
+<xacro:centauro_leg leg_num="1" origin_x="1" origin_y="-1">
+</xacro:centauro_leg>
+<xacro:centauro_leg leg_num="2" origin_x="1" origin_y="1">
+</xacro:centauro_leg>
+<xacro:centauro_leg leg_num="3" origin_x="-1" origin_y="-1">
+</xacro:centauro_leg>
+<xacro:centauro_leg leg_num="4" origin_x="-1" origin_y="1">
+</xacro:centauro_leg>
 </robot>

Commit message: added arms

File: centauro_urdf/urdf/centauro_base.urdf.xacro (robot description, xacro)
@@ -42,5 +42,5 @@
 <xacro:if value="${ADD_UPPER_BODY}">
 	<xacro:include filename="$(find centauro_urdf)/urdf/parts/centauro_torso.urdf.xacro" />
-        <!--xacro:include filename="$(find pholus_urdf)/urdf/parts/arms.urdf.xacro" /-->
+        <xacro:include filename="$(find centauro_urdf)/urdf/parts/arms.urdf.xacro" />
 	<!--xacro:include filename="$(find pholus_urdf)/urdf/parts/head.urdf.xacro" /-->
 </xacro:if>

File: centauro_urdf/urdf/parts/arms.urdf.xacro (robot description, xacro)
@@ -1,9 +1,11 @@
 <?xml version="1.0"?>
 <robot xmlns:xacro="http://ros.org/wiki/xacro">
-<xacro:include filename="$(find pholus_urdf)/urdf/parts/arm_macro.urdf.xacro" />
-<xacro:include filename="$(find pholus_urdf)/urdf/parts/heri_hand_macro.urdf.xacro" />
-<xacro:arm prefix="r"  mirror_link="1"/>
-<xacro:heri_hand prefix="r"  mirror_link="1" ft_sensor_roll="0.0" ft_sensor_pitch="0.0" ft_sensor_yaw="0.0"/>
-<xacro:arm prefix="l"  mirror_link="-1"/>
-<xacro:heri_hand prefix="l"  mirror_link="-1" ft_sensor_roll="0.0" ft_sensor_pitch="0.0" ft_sensor_yaw="0.0"/>
+<xacro:include filename="$(find centauro_urdf)/urdf/parts/centauro_arm.urdf.xacro" />
+<!-- arms -->
+<xacro:centauro_arm arm_num="1"  rot="1"  parent="torso_2">
+      <origin xyz="${Shoulder_1_Ox} ${Shoulder_1_Oy} ${Shoulder_1_Oz}" rpy="${Shoulder_1_roll} ${Shoulder_1_pitch} ${Shoulder_1_yaw}"/>
+   </xacro:centauro_arm>
+<xacro:centauro_arm arm_num="2" rot="-1"  parent="torso_2">
+      <origin xyz="${Shoulder_1_Ox} ${-Shoulder_1_Oy} ${Shoulder_1_Oz}" rpy="${-Shoulder_1_roll} ${Shoulder_1_pitch} ${-Shoulder_1_yaw}" />
+</xacro:centauro_arm>
 </robot>

Commit message: Added meshes of ball end effectors. Added ball end-effectors to model. Commented out visulaization and collision of ft_joints.

File: centauro_urdf/urdf/centauro_base.urdf.xacro (robot description, xacro)
@@ -43,4 +43,13 @@
 	<xacro:include filename="$(find centauro_urdf)/urdf/parts/centauro_torso.urdf.xacro" />
         <xacro:include filename="$(find centauro_urdf)/urdf/parts/arms.urdf.xacro" />
+	<xacro:if value="${ADD_BALL_END_EFFECTOR}">
+		<xacro:include filename="$(find centauro_urdf)/urdf/parts/ball.urdf.xacro" />
+		<xacro:ball_end_effector arm_num="1"  parent_link="arm1_7">
+      			<origin xyz="0. 0. 0." rpy="0. 0. 0."/>
+   		</xacro:ball_end_effector>
+		<xacro:ball_end_effector arm_num="2"  parent_link="arm2_7">
+      			<origin xyz="0. 0. 0." rpy="0. 0. 0."/>
+   		</xacro:ball_end_effector>
+	</xacro:if>
 	<!--xacro:include filename="$(find pholus_urdf)/urdf/parts/head.urdf.xacro" /-->
 </xacro:if>

File: centauro_urdf/urdf/config/centauro.urdf.xacro (robot description, xacro)
@@ -7,4 +7,5 @@
 <xacro:property name="ADD_LEGS" value="true" />
 <xacro:property name="ADD_UPPER_BODY" value="true" />
+<xacro:property name="ADD_BALL_END_EFFECTOR" value="true" />
 <xacro:property name="ADD_FLOATING_BASE" value="true" />
 </robot>

File: centauro_urdf/urdf/parts/centauro_arm.urdf.xacro (robot description, xacro)
@@ -235,16 +235,16 @@
          <inertia ixx="${Ft_arm_xx}" ixy="${rot*Ft_arm_xy}" ixz="${Ft_arm_xz}" iyy="${Ft_arm_yy}" iyz="${rot*Ft_arm_yz}" izz="${Ft_arm_zz}"/>
       </inertial>
-      <visual>
+      <!--visual>
          <origin xyz="0.0 0.0 0.0"  rpy="${PI} 0.0 0.0"/>
    <geometry>
       <mesh filename="package://centauro_urdf/meshes/Wrist.STL" scale="0.001 ${-rot*0.001} 0.001" />
    </geometry>
-      </visual>
-      <collision>
+      </visual-->
+      <!--collision>
          <origin xyz="0.0 0.0 0.0"  rpy="${PI} 0.0 0.0"/>
    <geometry>
       <mesh filename="package://centauro_urdf/meshes/simple/Wrist.STL" scale="0.001 ${-rot*0.001} 0.001" />
    </geometry>
-      </collision>
+      </collision-->
    </link>
 </xacro:macro>

Commit message: added legs:=false and arms:=false option in launch file

File: centauro_urdf/urdf/centauro_base.urdf.xacro (robot description, xacro)
@@ -42,5 +42,5 @@
 <xacro:if value="${ADD_UPPER_BODY}">
 	<xacro:include filename="$(find centauro_urdf)/urdf/parts/centauro_torso.urdf.xacro" />
-        <xacro:include filename="$(find centauro_urdf)/urdf/parts/arms.urdf.xacro" />
+    <xacro:include filename="$(find centauro_urdf)/urdf/parts/arms.urdf.xacro" />
 	<xacro:if value="${ADD_BALL_END_EFFECTOR}">
 		<xacro:include filename="$(find centauro_urdf)/urdf/parts/ball.urdf.xacro" />

File: centauro_urdf/urdf/config/centauro.urdf.xacro (robot description, xacro)
@@ -3,9 +3,12 @@
 <xacro:property name="model_name" value="centauro" />
 <xacro:property name="model_version" value="0.1" />
+<!-- command line arguments -->
+<xacro:arg name="add_legs" default="true"/>
+<xacro:arg name="add_upper_body" default="true"/>
 <!-- ************SELECT PARTS*************-->
 <!-- *************************************-->
-<xacro:property name="ADD_LEGS" value="true" />
-<xacro:property name="ADD_UPPER_BODY" value="true" />
+<xacro:property name="ADD_LEGS" value="$(arg add_legs)" />
+<xacro:property name="ADD_UPPER_BODY" value="$(arg add_upper_body)" />
 <xacro:property name="ADD_BALL_END_EFFECTOR" value="true" />
-<xacro:property name="ADD_FLOATING_BASE" value="true" />
+<xacro:property name="ADD_FLOATING_BASE" value="$(arg add_legs)" />
 </robot>

Commit message: centered wheel frame

File: centauro_urdf/urdf/centauro_base.urdf.xacro (robot description, xacro)
@@ -19,5 +19,5 @@
         <origin xyz="0.0 0 0.0"  rpy="0.0 0.0 0.0"/>
         <geometry>
-         <mesh filename="package://centauro_urdf/meshes/pelvis.stl" scale="0.001 0.001 0.001" />
+         <mesh filename="package://centauro_urdf/meshes/v2/pelvis.stl" scale="0.001 0.001 0.001" />
         </geometry>
       </visual>

File: centauro_urdf/urdf/parts/centauro_leg.urdf.xacro (robot description, xacro)
@@ -17,7 +17,7 @@
    </visual>
    <collision>
-      <origin xyz="0.0 0.0 0.0"  rpy="0.0 0.0 ${origin_x*origin_y*(Leg_1_yaw-PI/2)-Leg_1_yaw+PI/2}"/>
-      <geometry>
-         <mesh filename="package://centauro_urdf/meshes/simple/hip-yaw.stl" scale="0.001 ${0.001} 0.001" />
+      <origin xyz="0.0 0.0 0.0"  rpy="0.0 0.0 0.0"/>
+      <geometry>
+         <mesh filename="package://centauro_urdf/meshes/v2/collision/hip-yaw.stl" scale="0.001 ${mirror*0.001} 0.001" />
       </geometry>
    </collision>
@@ -38,5 +38,5 @@
       <origin xyz="0.0 0.0 0.0"  rpy="0.0 0.0 0.0"/>
       <geometry>
-         <mesh filename="package://centauro_urdf/meshes/simple/hip-pitch.stl" scale="0.001 ${0.001} 0.001" />
+         <mesh filename="package://centauro_urdf/meshes/v2/collision/hip-pitch.stl" scale="0.001 0.001 ${mirror*0.001}" />
       </geometry>
    </collision>
@@ -83,5 +83,5 @@
       <origin xyz="0.0 0.0 0.0"  rpy="0.0 0.0 0.0"/>
       <geometry>
-         <mesh filename="package://centauro_urdf/meshes/simple/knee.stl" scale="0.001 ${0.001} 0.001" />
+         <mesh filename="package://centauro_urdf/meshes/v2/collision/knee.stl" scale="0.001 0.001 ${mirror*0.001}" />
       </geometry>
    </collision>
@@ -102,5 +102,5 @@
       <origin xyz="0.0 0.0 0.0"  rpy="0.0 0.0 0.0"/>
       <geometry>
-         <mesh filename="package://centauro_urdf/meshes/simple/ankle-pitch.stl" scale="0.001 ${0.001} 0.001" />
+         <mesh filename="package://centauro_urdf/meshes/v2/collision/ankle-pitch.stl" scale="0.001 0.001 ${mirror*0.001}" />
       </geometry>
    </collision>
@@ -115,5 +115,5 @@
       <origin xyz="0.0 0.0 0.0"  rpy="0.0 0.0 0.0"/>
       <geometry>
-         <mesh filename="package://centauro_urdf/meshes/v2/ankle-yaw.stl" scale="0.001 ${origin_y*0.001} 0.001" />
+         <mesh filename="package://centauro_urdf/meshes/v2/ankle-yaw.stl" scale="0.001 ${mirror*0.001} 0.001" />
       </geometry>
       <material name="dark_grey"/>
@@ -122,9 +122,9 @@
       <origin xyz="0.0 0.0 0.0"  rpy="0.0 0.0 0.0"/>
       <geometry>
-         <mesh filename="package://centauro_urdf/meshes/simple/ankle-yaw.stl" scale="0.001 ${0.001} 0.001" />
-      </geometry>
-   </collision>
-</link>
-<link name="wheel_cad_${leg_num}">
+         <mesh filename="package://centauro_urdf/meshes/v2/collision/ankle-yaw.stl" scale="0.001 ${mirror*0.001} 0.001" />
+      </geometry>
+   </collision>
+</link>
+<link name="wheel_${leg_num}">
 	<inertial>
 		<origin xyz="${Wheel_x} ${Wheel_y} ${mirror*Wheel_z}"/>
@@ -154,10 +154,4 @@
 	<origin xyz="0 0 -0.176" rpy="0 0 0"/>
 </joint>
-<link name="wheel_${leg_num}"/>
-<joint name="wheel_fixed_joint_${leg_num}" type="fixed">
-	<parent link="wheel_cad_${leg_num}"/>
-	<child link="wheel_${leg_num}"/>
-	<origin xyz="0 0 ${Wheel_z}" rpy="0 0 0"/>
-</joint>
 <!-- ******************************** -->
 <joint name="hip_yaw_${leg_num}" type="revolute">
@@ -208,5 +202,5 @@
 <joint name="j_wheel_${leg_num}" type="continuous">
 	<parent link="ankle2_${leg_num}"/>
-	<child link="wheel_cad_${leg_num}"/>
+	<child link="wheel_${leg_num}"/>
 	<origin xyz="${Wheel_Ox} ${mirror*Wheel_Oy} ${Wheel_Oz}" rpy="${Wheel_roll} ${Wheel_pitch} ${Wheel_yaw}"/>
 	<axis xyz="0 0 ${mirror}"/>

File: centauro_urdf/urdf/parts/inertial_properties.urdf.xacro (robot description, xacro)
@@ -11,16 +11,16 @@
 <xacro:property name="wheel_weight" value=" 2.000000 "/>
 <!-- Center of Mass -->
-<xacro:property name="Pelvis_x" value=" 0.0013890071 "/>
-<xacro:property name="Pelvis_y" value=" -0.0015989148 "/>
-<xacro:property name="Pelvis_z" value=" 0.0631010120 "/>
-<!-- Inertia -->
-<xacro:property name="Pelvis_xx" value=" 0.2391262700 "/>
-<xacro:property name="Pelvis_yy" value=" 0.7143007800 "/>
-<xacro:property name="Pelvis_zz" value=" 0.8187044800 "/>
-<xacro:property name="Pelvis_xy" value=" -0.0050541269 "/>
-<xacro:property name="Pelvis_xz" value=" -0.0197460550 "/>
-<xacro:property name="Pelvis_yz" value=" 0.0002131204 "/>
-<!-- Mass -->
-<xacro:property name="Pelvis_mass" value=" 16.0975740000 "/>
+<xacro:property name="Pelvis_x" value="${-1.6320207e+00 * mmTom}"/>
+<xacro:property name="Pelvis_y" value="${2.6534004e+00 * mmTom}"/>
+<xacro:property name="Pelvis_z" value="${7.9167428e+01 * mmTom}"/>
+<!-- Inertia -->
+<xacro:property name="Pelvis_xx" value="${3.9195477e+05 * mm2Tom2}"/>
+<xacro:property name="Pelvis_yy" value="${1.0000709e+06 * mm2Tom2}"/>
+<xacro:property name="Pelvis_zz" value="${1.0679989e+06 * mm2Tom2}"/>
+<xacro:property name="Pelvis_xy" value="${2.4781259e+04 * mm2Tom2}"/>
+<xacro:property name="Pelvis_xz" value="${1.7108607e+04 * mm2Tom2}"/>
+<xacro:property name="Pelvis_yz" value="${5.2627106e+03 * mm2Tom2}"/>
+<!-- Mass -->
+<xacro:property name="Pelvis_mass" value="2.6584529e+01"/>
 <!-- Center of Mass -->
 <xacro:property name="Leg_1_x" value="${3.5958550e-01 * mmTom}"/>
@@ -91,5 +91,5 @@
 <xacro:property name="Wheel_x" value="${0.0 * mmTom}"/>
 <xacro:property name="Wheel_y" value="${0.0 * mmTom}"/>
-<xacro:property name="Wheel_z" value="${-4.9165610e+01 * mmTom}"/>
+<xacro:property name="Wheel_z" value="${3.1155904e+00 * mmTom}"/>
 <!-- Inertia -->
 <xacro:property name="Wheel_xx" value="${2.8174054e+03 * mm2Tom2}"/>
@@ -113,5 +113,5 @@
 <xacro:property name="Torso_2_yz" value=" -0.00004657 "/>
 <!-- Mass -->
-<xacro:property name="Torso_2_mass" value=" 11.4926890000 "/>
+<xacro:property name="Torso_2_mass" value="1.2553731e+01"/>
 <!-- Center of Mass -->
 <xacro:property name="Neck_1_x" value=" 0.0404796740 "/>

File: centauro_urdf/urdf/parts/kinematics_properties.urdf.xacro (robot description, xacro)
@@ -61,5 +61,5 @@
 <xacro:property name="Ankle_2_yaw" value="'0.0'"/>
 <xacro:property name="Wheel_Ox" value="${0.0 * mmTom}"/>
-<xacro:property name="Wheel_Oy" value="${-52.3500 * mmTom}"/>
+<xacro:property name="Wheel_Oy" value="${0.0 * mmTom}"/>
 <xacro:property name="Wheel_Oz" value="${-98.3500 * mmTom}"/>
 <xacro:property name="Wheel_roll" value="${PI_2}"/>

Commit message: added everything needed for rod_plates, need to correct the properties in xacro

File: centauro_urdf/urdf/centauro_base.urdf.xacro (robot description, xacro)
@@ -52,4 +52,13 @@
    		</xacro:ball_end_effector>
 	</xacro:if>
+	<xacro:if value="${ADD_ROD_PLATE_END_EFFECTOR}">
+		<xacro:include filename="parts/rod_plate.urdf.xacro" />
+		<xacro:rod_plate_end_effector arm_num="1"  parent_link="arm1_7">
+      			<origin xyz="0. 0. 0." rpy="0. 0. 0."/>
+   		</xacro:rod_plate_end_effector>
+		<xacro:rod_plate_end_effector arm_num="2"  parent_link="arm2_7">
+      			<origin xyz="0. 0. 0." rpy="0. 0. 0."/>
+   		</xacro:rod_plate_end_effector>
+	</xacro:if>
 	<xacro:include filename="parts/head.urdf.xacro" />
 </xacro:if>

File: centauro_urdf/urdf/config/centauro.urdf.xacro (robot description, xacro)
@@ -10,5 +10,6 @@
 <xacro:property name="ADD_LEGS" value="$(arg add_legs)" />
 <xacro:property name="ADD_UPPER_BODY" value="$(arg add_upper_body)" />
-<xacro:property name="ADD_BALL_END_EFFECTOR" value="true" />
+<xacro:property name="ADD_BALL_END_EFFECTOR" value="false" />
+<xacro:property name="ADD_ROD_PLATE_END_EFFECTOR" value="true" />
 <xacro:property name="ADD_FLOATING_BASE" value="$(arg add_legs)" />
 <xacro:property name="ADD_VIRTUAL_FRAME" value="false" />

File: centauro_urdf/urdf/config/centauro_virtual_frame.urdf.xacro (robot description, xacro)
@@ -10,5 +10,6 @@
 <xacro:property name="ADD_LEGS" value="$(arg add_legs)" />
 <xacro:property name="ADD_UPPER_BODY" value="$(arg add_upper_body)" />
-<xacro:property name="ADD_BALL_END_EFFECTOR" value="true" />
+<xacro:property name="ADD_BALL_END_EFFECTOR" value="false" />
+<xacro:property name="ADD_ROD_PLATE_END_EFFECTOR" value="true" />
 <xacro:property name="ADD_FLOATING_BASE" value="$(arg add_legs)" />
 <xacro:property name="ADD_VIRTUAL_FRAME" value="true" />

File: centauro_urdf/urdf/gazebo/materials.gazebo.xacro (robot description, xacro)
@@ -67,4 +67,12 @@
 </gazebo>
 </xacro:if>
+<xacro:if value="${ADD_ROD_PLATE_END_EFFECTOR}">
+<gazebo reference="rod_plate1">
+	<material>Gazebo/BlackTransparent</material>
+</gazebo>
+<gazebo reference="rod_plate2">
+	<material>Gazebo/BlackTransparent</material>
+</gazebo>
+</xacro:if>
 </xacro:if>
 </robot>

Commit message: option for different mass at each rod plate (currently both zero)

File: centauro_urdf/urdf/centauro_base.urdf.xacro (robot description, xacro)
@@ -54,8 +54,8 @@
 	<xacro:if value="${ADD_ROD_PLATE_END_EFFECTOR}">
 		<xacro:include filename="parts/rod_plate.urdf.xacro" />
-		<xacro:rod_plate_end_effector arm_num="1"  parent_link="arm1_7">
+		<xacro:rod_plate_end_effector arm_num="1"  parent_link="arm1_7" rod_mass="0.0">
       			<origin xyz="0. 0. 0." rpy="0. 0. 0."/>
    		</xacro:rod_plate_end_effector>
-		<xacro:rod_plate_end_effector arm_num="2"  parent_link="arm2_7">
+		<xacro:rod_plate_end_effector arm_num="2"  parent_link="arm2_7" rod_mass="0.0">
       			<origin xyz="0. 0. 0." rpy="0. 0. 0."/>
    		</xacro:rod_plate_end_effector>

File: centauro_urdf/urdf/parts/rod_plate.urdf.xacro (robot description, xacro)
@@ -2,10 +2,10 @@
 <robot xmlns:xacro="http://ros.org/wiki/xacro">
 <!-- This is an attempt to model rod plate, the file is based on the ball hand -->
-<xacro:macro name="rod_plate_end_effector" params="arm_num parent_link *origin">
+<xacro:macro name="rod_plate_end_effector" params="arm_num parent_link rod_mass *origin">
 <link name="rod_plate${arm_num}">
     <inertial>
       <origin xyz="${4.8407693e+01*mmTom} ${2.0035723e+01*mmTom} ${7.7533287e+01*mmTom}" rpy="0 0 0"/>
       <!--mass value="3.45345"/-->
-      <mass value="0.0"/>
+      <mass value="${rod_mass}"/>
       <inertia ixx="${2.3061092e+03*mm2Tom2}"  ixy="${2.9181758e-01*mm2Tom2}"  ixz="${-2.1246684e-01*mm2Tom2}" iyy="${2.3053155e+03*mm2Tom2}" iyz="${7.9290978e-01*mm2Tom2}" izz="${3.0675616e+03*mm2Tom2}" />
     </inertial>

Commit message: option for different ball masses

File: centauro_urdf/urdf/centauro_base.urdf.xacro (robot description, xacro)
@@ -45,8 +45,8 @@
 	<xacro:if value="${ADD_BALL_END_EFFECTOR}">
 		<xacro:include filename="parts/ball.urdf.xacro" />
-		<xacro:ball_end_effector arm_num="1"  parent_link="arm1_7">
+		<xacro:ball_end_effector arm_num="1"  parent_link="arm1_7" ball_mass="1.27">
       			<origin xyz="0. 0. 0." rpy="0. 0. 0."/>
    		</xacro:ball_end_effector>
-		<xacro:ball_end_effector arm_num="2"  parent_link="arm2_7">
+		<xacro:ball_end_effector arm_num="2"  parent_link="arm2_7" ball_mass="1.27">
       			<origin xyz="0. 0. 0." rpy="0. 0. 0."/>
    		</xacro:ball_end_effector>

File: centauro_urdf/urdf/parts/ball.urdf.xacro (robot description, xacro)
@@ -1,9 +1,9 @@
 <?xml version="1.0"?>
 <robot xmlns:xacro="http://ros.org/wiki/xacro">
-<xacro:macro name="ball_end_effector" params="arm_num parent_link *origin">
+<xacro:macro name="ball_end_effector" params="arm_num parent_link ball_mass *origin">
 <link name="ball${arm_num}">
     <inertial>
       <origin xyz="${-1.0072498e-02*mmTom} ${3.7590658e-02*mmTom} ${1.9772332e+01*mmTom}" rpy="0 0 0"/>
-      <mass value="1.27"/>
+      <mass value="${ball_mass}"/>
       <inertia ixx="${2.3061092e+03*mm2Tom2}"  ixy="${2.9181758e-01*mm2Tom2}"  ixz="${-2.1246684e-01*mm2Tom2}" iyy="${2.3053155e+03*mm2Tom2}" iyz="${7.9290978e-01*mm2Tom2}" izz="${3.0675616e+03*mm2Tom2}" />
     </inertial>
