Commit message: fixed rod plates properties and frames (missing correect transform for the tip)

File: centauro_urdf/urdf/centauro_base.urdf.xacro (robot description, xacro)
@@ -54,8 +54,8 @@
 	<xacro:if value="${ADD_ROD_PLATE_END_EFFECTOR}">
 		<xacro:include filename="parts/rod_plate.urdf.xacro" />
-		<xacro:rod_plate_end_effector arm_num="1"  parent_link="arm1_7" rod_mass="0.01">
+		<xacro:rod_plate_end_effector arm_num="1" rot="1" parent_link="arm1_7" rod_mass="0.01">
       			<origin xyz="0. 0. 0." rpy="0. 0. 0."/>
    		</xacro:rod_plate_end_effector>
-		<xacro:rod_plate_end_effector arm_num="2"  parent_link="arm2_7" rod_mass="0.01">
+		<xacro:rod_plate_end_effector arm_num="2" rot="-1"  parent_link="arm2_7" rod_mass="0.01">
       			<origin xyz="0. 0. 0." rpy="0. 0. 0."/>
    		</xacro:rod_plate_end_effector>

File: centauro_urdf/urdf/parts/rod_plate.urdf.xacro (robot description, xacro)
@@ -2,27 +2,28 @@
 <robot xmlns:xacro="http://ros.org/wiki/xacro">
 <!-- This is an attempt to model rod plate, the file is based on the ball hand -->
-<xacro:macro name="rod_plate_end_effector" params="arm_num parent_link rod_mass *origin">
+<xacro:macro name="rod_plate_end_effector" params="arm_num rot parent_link rod_mass *origin">
 <link name="rod_plate${arm_num}">
     <inertial>
-      <origin xyz="${4.8407693e+01*mmTom} ${2.0035723e+01*mmTom} ${7.7533287e+01*mmTom}" rpy="0 0 0"/>
+      <origin xyz="${4.8407693e+01*mmTom} ${rot*2.0035723e+01*mmTom} ${7.7533287e+01*mmTom}" rpy="0 0 0"/>
       <!--mass value="3.45345"/-->
       <mass value="${rod_mass}"/>
-      <inertia ixx="${2.3061092e+03*mm2Tom2}"  ixy="${2.9181758e-01*mm2Tom2}"  ixz="${-2.1246684e-01*mm2Tom2}" iyy="${2.3053155e+03*mm2Tom2}" iyz="${7.9290978e-01*mm2Tom2}" izz="${3.0675616e+03*mm2Tom2}" />
+      <inertia ixx="${1.1323020e+04*mm2Tom2}"  ixy="${-6.7302376e+02*rot*mm2Tom2}"  ixz="${-2.8429136e+03*mm2Tom2}" iyy="${1.2661574e+04*mm2Tom2}" iyz="${-1.1815269e+03*rot*mm2Tom2}" izz="${8.4787328e+03*mm2Tom2}" />
     </inertial>
     <visual>
-      <origin xyz="0.0 0.0 0.0" rpy="3.14 0.0 0.0"/>
+      <origin xyz="0.0 0.0 0.0" rpy="3.1415 0.0 0.0"/>
       <geometry name="rod_plate${arm_num}_visual">
-        <mesh filename="package://centauro_urdf/meshes/simple/RodPlate.stl" scale="0.001 0.001 0.001" />
+        <mesh filename="package://centauro_urdf/meshes/simple/RodPlate.stl" scale="0.001 ${-rot*0.001} 0.001" />
       </geometry>
       <material name="grey"/>
    </visual>
    <collision>
-      <origin xyz="0.0 0.0 0.0" rpy="0.0 0.0 0.0"/>
+      <origin xyz="0.0 0.0 0.0" rpy="3.1415 0.0 0.0"/>
       <geometry name="rod_plate${arm_num}_collision">
-        <mesh filename="package://centauro_urdf/meshes/simple/RodPlate.stl" scale="0.001 0.001 0.001" />
+        <mesh filename="package://centauro_urdf/meshes/simple/RodPlate.stl" scale="0.001 ${-rot*0.001} 0.001" />
       </geometry>
    </collision>
 </link>
 <link name="rod_plate${arm_num}_tip"/>
+<!-- <origin xyz="0 -0.174 -0.049" rpy="1.570796 0.0 0.0"/ -->
 <!-- Parent link is arm*_7 -->
 <joint name="j_arm${arm_num}_8" type="fixed">
@@ -31,9 +32,9 @@
       <xacro:insert_block name="origin"/>
 </joint>
-<!-- <origin xyz="0 -0.174 -0.049" rpy="1.570796 0.0 0.0"/ -->
+<!-- tip frame is not perfectly correct, need to receive tf from cad -->
 <joint name="j_rod_plate${arm_num}_tip" type="fixed">
 	<parent link="rod_plate${arm_num}"/>
 	<child link="rod_plate${arm_num}_tip"/>
-	<origin xyz="0 0 -0.07" rpy="0 0 0"/>
+	<origin xyz="0.06 0.0 -0.16" rpy="0.0 0.0 ${rot*0.349066}"/>
 </joint>
 <!-- add armX_8 link for legacy reasons (same as ballX) -->

Commit message: frames also for pelvis d435

File: centauro_urdf/urdf/centauro_base.urdf.xacro (robot description, xacro)
@@ -44,7 +44,14 @@
     <xacro:include filename="$(find centauro_urdf)/urdf/parts/arms.urdf.xacro" />
 	<xacro:include filename="$(find centauro_urdf)/urdf/parts/head.urdf.xacro" />
+    <xacro:property name="d435_base_name" value="D435i_camera" />
+    <xacro:property name="d435_base_parent_name" value="pelvis" />
+    <xacro:property name="d435_base_origin">
+        <origin xyz="0.27187 0 0.0215997" rpy="0 0.5251508 0"/>
+    </xacro:property>
     <xacro:if value="${ADD_D435I_BASE}">
         <xacro:include filename="$(find realsense_gazebo_description)/urdf/_d435i.urdf.xacro" />
-        <xacro:sensor_d435i parent="pelvis" name="D435i_camera" topics_ns="D435i/D435i_camera"
+        <xacro:sensor_d435i parent="${d435_base_parent_name}"
+                      name="${d435_base_name}"
+                      topics_ns="${d435_base_name}"
                       enable_pointCloud="true" align_depth="true"
                       unite_imu_method="false"
@@ -61,7 +68,51 @@
                       color_height="720"
                       color_fps="30">
-            <origin xyz="0.27187 0 0.0215997" rpy="0 0.5251508 0"/>
+            <xacro:insert_block name="d435_base_origin" />
         </xacro:sensor_d435i>
     </xacro:if>
+    <xacro:unless value="${ADD_D435I_BASE}">
+        <!--  Copied from _d435.urdf.xacro    -->
+        <xacro:property name="d435_cam_width" value="0.090"/>
+        <xacro:property name="d435_cam_height" value="0.025"/>
+        <xacro:property name="d435_cam_depth" value="0.02505"/>
+        <xacro:property name="d435_cam_mount_from_center_offset" value="0.0149"/>
+        <xacro:property name="d435_cam_depth_px" value="${d435_cam_mount_from_center_offset}"/>
+        <xacro:property name="d435_cam_depth_py" value="0.0175"/>
+        <xacro:property name="d435_cam_depth_pz" value="${d435_cam_height/2}"/>
+        <!-- camera body, with origin at bottom screw mount -->
+        <joint name="${d435_base_name}_joint" type="fixed">
+        <xacro:insert_block name="d435_base_origin"/>
+        <parent link="${d435_base_parent_name}"/>
+        <child link="${d435_base_name}_bottom_screw_frame"/>
+        </joint>
+        <link name="${d435_base_name}_bottom_screw_frame"/>
+        <joint name="${d435_base_name}_link_joint" type="fixed">
+        <origin xyz="0 ${d435_cam_depth_py} ${d435_cam_depth_pz}" rpy="0 0 0"/>
+        <parent link="${d435_base_name}_bottom_screw_frame"/>
+        <child link="${d435_base_name}_link"/>
+        </joint>
+        <link name="${d435_base_name}_link">
+        <visual>
+        <origin xyz="${d435_cam_mount_from_center_offset} ${-d435_cam_depth_py} 0" rpy="${PI/2} 0 ${PI/2}"/>
+            <geometry>
+            <!-- <box size="${d435_cam_width} ${d435_cam_height} ${d435_cam_depth}"/> -->
+            <mesh filename="package://centauro_urdf/meshes/realsense/d435.dae"/>
+            </geometry>
+            <material name="${d435_base_name}_aluminum"/>
+        </visual>
+        <collision>
+            <origin xyz="0 ${-d435_cam_depth_py} 0" rpy="0 0 0"/>
+            <geometry>
+            <box size="${d435_cam_depth} ${d435_cam_width} ${d435_cam_height}"/>
+            </geometry>
+        </collision>
+        <inertial>
+            <!-- The following are not reliable values, and should not be used for modeling -->
+            <mass value="0.564"/>
+            <origin xyz="0 0 0"/>
+            <inertia ixx="0.003881243" ixy="0.0" ixz="0.0" iyy="0.000498940" iyz="0.0" izz="0.003879257"/>
+        </inertial>
+        </link>
+    </xacro:unless>
     <xacro:if value="${ADD_T265_BASE}">
         <xacro:include filename="$(find realsense_gazebo_description)/urdf/_t265.urdf.xacro" />

Commit message: Signed-off-by: Andrea Patrizi <andreapatrizi1b6e6@gmail.com>

File: centauro_urdf/urdf/centauro_base.urdf.xacro (robot description, xacro)
@@ -10,4 +10,9 @@
     <xacro:include filename="${CENTAURO_ROOT}/urdf/parts/limits.urdf.xacro" />
     <link name="base_link" />
+    <joint name="base_joint" type="fixed">
+        <parent link="base_link" />
+        <child link="pelvis" />
+        <origin xyz="0 0 0" rpy="0 0 0" />
+    </joint>
     <link name="pelvis">
         <inertial>
@@ -34,9 +39,4 @@
         <origin xyz="${Imu_Ox} ${Imu_Oy} ${Imu_Oz}" rpy="${Imu_raw} ${Imu_pitch} ${Imu_yaw}" />
         <child link="imu_link" />
-    </joint>
-    <joint name="base_joint" type="fixed">
-        <parent link="pelvis" />
-        <child link="base_link" />
-        <origin xyz="0 0 0" rpy="0 0 0" />
     </joint>
     <xacro:if value="${ADD_UPPER_BODY}">

File: centauro_urdf/urdf/parts/wheel23.urdf.xacro (robot description, xacro)
@@ -13,5 +13,5 @@
                 <origin xyz="0.0 0.0 0.0" rpy="0.0 0.0 0.0" />
                 <geometry>
-                    <mesh filename="package://centauro_urdf/meshes/v2/mesh_ankle-yaw_wheel23.stl"
+                    <mesh filename="${CENTAURO_ROOT}/meshes/v2/mesh_ankle-yaw_wheel23.stl"
                         scale="0.001 ${mirror*0.001} 0.001" />
                 </geometry>
@@ -22,5 +22,5 @@
                 <geometry>
                     <mesh
-                        filename="package://centauro_urdf/meshes/v2/collision/mesh_ankle-yaw_wheel23.stl"
+                        filename="${CENTAURO_ROOT}/meshes/v2/collision/mesh_ankle-yaw_wheel23.stl"
                         scale="0.001 ${mirror*0.001} 0.001" />
                 </geometry>
@@ -46,5 +46,5 @@
                 <origin xyz="0.0 0.0 0.0" rpy="0.0 0.0 0.0" />
                 <geometry>
-                    <mesh filename="package://centauro_urdf/meshes/v2/mesh_wheel23.stl"
+                    <mesh filename="${CENTAURO_ROOT}/meshes/v2/mesh_wheel23.stl"
                         scale="0.001 0.001 ${mirror*0.001}" />
                 </geometry>
@@ -54,5 +54,5 @@
                 <origin xyz="0 0 0" rpy="0 0 0" />
                 <geometry>
-                    <mesh filename="package://centauro_urdf/meshes/v2/collision/mesh_wheel23.stl"
+                    <mesh filename="${CENTAURO_ROOT}/meshes/v2/collision/mesh_wheel23.stl"
                         scale="0.001 0.001 ${mirror*0.001}" />
                 </geometry>

Commit message: argument to add or remove the battery from the model

File: centauro_urdf/urdf/centauro_base.urdf.xacro (robot description, xacro)
@@ -3,5 +3,4 @@
     <!--
   ROS urdf definition of the CENTAURO humanoid robot by Istituto Italiano di Tecnologia
-  Author: Enrico Mingo Hoffman
 -->
     <xacro:include filename="$(find centauro_urdf)/urdf/utils.urdf.xacro" />
@@ -11,9 +10,18 @@
     <link name="base_link" />
     <link name="pelvis">
-        <inertial>
-            <origin xyz="${Pelvis_x} ${Pelvis_y} ${Pelvis_z}" />
-            <mass value="${Pelvis_mass}" />
-            <inertia ixx="${Pelvis_xx}" ixy="${Pelvis_xy}" ixz="${Pelvis_xz}" iyy="${Pelvis_yy}" iyz="${Pelvis_yz}" izz="${Pelvis_zz}" />
-        </inertial>
+		<xacro:if value="${ADD_BATTERY}">
+		    <inertial>
+		        <origin xyz="${Pelvis_x} ${Pelvis_y} ${Pelvis_z}" />
+		        <mass value="${Pelvis_mass}" />
+		        <inertia ixx="${Pelvis_xx}" ixy="${Pelvis_xy}" ixz="${Pelvis_xz}" iyy="${Pelvis_yy}" iyz="${Pelvis_yz}" izz="${Pelvis_zz}" />
+		    </inertial>
+		</xacro:if>
+		<xacro:unless value="${ADD_BATTERY}">
+			<inertial>
+		        <origin xyz="${PelvisNoBattery_x} ${PelvisNoBattery_y} ${PelvisNoBattery_z}" />
+		        <mass value="${PelvisNoBattery_mass}" />
+		        <inertia ixx="${PelvisNoBattery_xx}" ixy="${PelvisNoBattery_xy}" ixz="${PelvisNoBattery_xz}" iyy="${PelvisNoBattery_yy}" iyz="${PelvisNoBattery_yz}" izz="${PelvisNoBattery_zz}" />
+		    </inertial>
+		</xacro:unless>
         <visual>
             <origin xyz="0.0 0 0.0" rpy="0.0 0.0 0.0" />

File: centauro_urdf/urdf/config/centauro.urdf.xacro (robot description, xacro)
@@ -11,4 +11,5 @@
 <xacro:arg name="end_effector_left" default="ball"/>
 <xacro:arg name="end_effector_right" default="ball"/>
+<xacro:arg name="battery" default="false"/>
 <xacro:if value="$(arg realsense)">
 	<xacro:arg name="d435i_head" default="true"/>
@@ -27,4 +28,5 @@
 <!-- ************SELECT PARTS*************-->
 <!-- *************************************-->
+<xacro:property name="ADD_BATTERY" value="$(arg battery)"/>
 <xacro:property name="ADD_LEGS" value="$(arg legs)" />
 <xacro:property name="ADD_UPPER_BODY" value="$(arg upper_body)" />

File: centauro_urdf/urdf/parts/inertial_properties.urdf.xacro (robot description, xacro)
@@ -14,4 +14,7 @@
 <xacro:property name="Pelvis_y" value="${2.6534004e+00 * mmTom}"/>
 <xacro:property name="Pelvis_z" value="${7.9167428e+01 * mmTom}"/>
+<xacro:property name="PelvisNoBattery_x" value="${1.0310423e+01 * mmTom}"/>
+<xacro:property name="PelvisNoBattery_y" value="${3.4907373e+00 * mmTom}"/>
+<xacro:property name="PelvisNoBattery_z" value="${5.7233845e+01 * mmTom}"/>
 <!-- Inertia -->
 <xacro:property name="Pelvis_xx" value="${3.9195477e+05 * mm2Tom2}"/>
@@ -21,6 +24,13 @@
 <xacro:property name="Pelvis_xz" value="${1.7108607e+04 * mm2Tom2}"/>
 <xacro:property name="Pelvis_yz" value="${5.2627106e+03 * mm2Tom2}"/>
+<xacro:property name="PelvisNoBattery_xx" value="${8.7627533e+05 * mm2Tom2}"/>
+<xacro:property name="PelvisNoBattery_yy" value="${1.6329655e+06 * mm2Tom2}"/>
+<xacro:property name="PelvisNoBattery_zz" value="${1.9611303e+06  * mm2Tom2}"/>
+<xacro:property name="PelvisNoBattery_xy" value="${2.2209997e+04 * mm2Tom2}"/>
+<xacro:property name="PelvisNoBattery_xz" value="${-6.1989843e+03 * mm2Tom2}"/>
+<xacro:property name="PelvisNoBattery_yz" value="${4.5514872e+03 * mm2Tom2}"/>
 <!-- Mass -->
 <xacro:property name="Pelvis_mass" value="2.6584529e+01"/>
+<xacro:property name="PelvisNoBattery_mass" value="1.8845851e+01"/>
 <!-- Center of Mass -->
 <xacro:property name="Leg_1_x" value="${3.5958550e-01 * mmTom}"/>

Commit message: removed ": " from all files to avoid misterious bug when passing URDF as argument of ros2 run --ros-args (parses as YAML)

File: centauro_urdf/urdf/centauro_base.urdf.xacro (robot description, xacro)
@@ -1,8 +1,5 @@
 <?xml version="1.0"?>
 <robot xmlns:xacro="http://ros.org/wiki/xacro" name="centauro">
-    <!--
-  ROS urdf definition of the CENTAURO humanoid robot by Istituto Italiano di Tecnologia
-  Author: Enrico Mingo Hoffman
--->
+    <!-- ROS urdf definition of the CENTAURO humanoid robot by Istituto Italiano di Tecnologia. Author Enrico Mingo Hoffman-->
     <xacro:include filename="${CENTAURO_ROOT}/urdf/utils.urdf.xacro" />
     <xacro:include filename="${CENTAURO_ROOT}/urdf/parts/kinematics_properties.urdf.xacro" />

File: centauro_urdf/urdf/centauro_robot.urdf.xacro (robot description, xacro)
@@ -3,5 +3,5 @@
   <!--
   ROS urdf definition of the PHOLUS humanoid robot by Istituto Italiano di Tecnologia
-  Author: Enrico Mingo
+  Author Enrico Mingo
   This file groups files to use CENTAURO in GAZEBO
   -->

File: centauro_urdf/urdf/parts/centauro_leg.urdf.xacro (robot description, xacro)
@@ -8,5 +8,5 @@
 	<inertial>
 		<origin xyz="${Leg_1_x} ${mirror*Leg_1_y} ${Leg_1_z}" />
-		<mass value="${Leg_1_mass}"/> <!-- org: 2 -->
+		<mass value="${Leg_1_mass}"/> <!-- org 2 -->
 		<inertia ixx="${Leg_1_xx}" ixy="${mirror*Leg_1_xy}" ixz="${Leg_1_xz}" iyy="${Leg_1_yy}" iyz="${mirror*Leg_1_yz}" izz="${Leg_1_zz}"/>
 	</inertial>
@@ -28,5 +28,5 @@
 	<inertial>
 		<origin xyz="${Leg_2_x} ${Leg_2_y} ${mirror*Leg_2_z}"/>
-		<mass value="${Leg_2_mass}"/> <!-- org: 4.5 -->
+		<mass value="${Leg_2_mass}"/> <!-- org 4.5 -->
 		<inertia ixx="${Leg_2_xx}" ixy="${Leg_2_xy}" ixz="${mirror*Leg_2_xz}" iyy="${Leg_2_yy}" iyz="${mirror*Leg_2_yz}" izz="${Leg_2_zz}"/>
 	</inertial>
@@ -72,5 +72,5 @@
       <inertial>
          <origin xyz="${Leg_3_x} ${Leg_3_y} ${mirror*Leg_3_z}"/>
-         <mass value="${Leg_3_mass}"/>  <!-- org: 3.5, foot un modeled-->
+         <mass value="${Leg_3_mass}"/>  <!-- org 3.5, foot un modeled-->
          <inertia ixx="${Leg_3_xx}" ixy="${Leg_3_xy}" ixz="${mirror*Leg_3_xz}" iyy="${Leg_3_yy}" iyz="${mirror*Leg_3_yz}" izz="${Leg_3_zz}"/>
       </inertial>
@@ -92,5 +92,5 @@
       <inertial>
          <origin xyz="${Ankle_1_x} ${Ankle_1_y} ${mirror*Ankle_1_z}"/>
-         <mass value="${Ankle_1_mass}"/>  <!-- org: 3.5, foot un modeled-->
+         <mass value="${Ankle_1_mass}"/>  <!-- org 3.5, foot un modeled-->
          <inertia ixx="${Ankle_1_xx}" ixy="${Ankle_1_xy}" ixz="${mirror*Ankle_1_xz}" iyy="${Ankle_1_yy}" iyz="${mirror*Ankle_1_yz}" izz="${Ankle_1_zz}"/>
       </inertial>

File: centauro_urdf/urdf/parts/inertial_properties.urdf.xacro (robot description, xacro)
@@ -88,5 +88,5 @@
 <!-- Mass -->
 <xacro:property name="Ankle_2_mass" value="1.7656714e+00"/>
-<!-- Note: the "23" suffix denotes the new bigger-size wheel -->
+<!-- Note that the "23" suffix denotes the new bigger-size wheel -->
 <!-- Center of Mass -->
 <xacro:property name="Ankle23_2_x" value="${1.8512273e-01 * mmTom}"/>

File: centauro_urdf/urdf/parts/wheel.urdf.xacro (robot description, xacro)
@@ -6,5 +6,5 @@
         <inertial>
         <origin xyz="${Ankle_2_x} ${mirror*Ankle_2_y} ${Ankle_2_z}"/>
-        <mass value="${Ankle_2_mass}"/>  <!-- org: 3.5, foot un modeled-->
+        <mass value="${Ankle_2_mass}"/>  <!-- org 3.5, foot un modeled-->
         <inertia ixx="${Ankle_2_xx}" ixy="${mirror*Ankle_2_xy}" ixz="${Ankle_2_xz}" iyy="${Ankle_2_yy}" iyz="${mirror*Ankle_2_yz}" izz="${Ankle_2_zz}"/>
         </inertial>

File: centauro_urdf/urdf/parts/wheel23.urdf.xacro (robot description, xacro)
@@ -6,5 +6,5 @@
             <inertial>
                 <origin xyz="${Ankle23_2_x} ${mirror*Ankle23_2_y} ${Ankle23_2_z}" />
-                <mass value="${Ankle23_2_mass}" />  <!-- org: 3.5, foot un modeled-->
+                <mass value="${Ankle23_2_mass}" />  <!-- org 3.5, foot un modeled-->
                 <inertia ixx="${Ankle23_2_xx}" ixy="${mirror*Ankle23_2_xy}" ixz="${Ankle23_2_xz}"
                     iyy="${Ankle23_2_yy}" iyz="${mirror*Ankle23_2_yz}" izz="${Ankle23_2_zz}" />

Commit message: added option to use/remove battery (adapted pelvis inertias)

File: centauro_urdf/urdf/centauro_base.urdf.xacro (robot description, xacro)
@@ -12,23 +12,46 @@
         <origin xyz="0 0 0" rpy="0 0 0" />
     </joint>
-    <link name="pelvis">
-        <inertial>
-            <origin xyz="${Pelvis_x} ${Pelvis_y} ${Pelvis_z}" />
-            <mass value="${Pelvis_mass}" />
-            <inertia ixx="${Pelvis_xx}" ixy="${Pelvis_xy}" ixz="${Pelvis_xz}" iyy="${Pelvis_yy}" iyz="${Pelvis_yz}" izz="${Pelvis_zz}" />
-        </inertial>
-        <visual>
-            <origin xyz="0.0 0 0.0" rpy="0.0 0.0 0.0" />
-            <geometry>
-                <mesh filename="${MESH_PATH}/v2/pelvis.stl" scale="0.001 0.001 0.001" />
-            </geometry>
-        </visual>
-        <collision>
-            <origin xyz="0.0 0 0.0" rpy="0.0 0.0 0.0" />
-            <geometry>
-                <mesh filename="${MESH_PATH}/simple/pelvis_reduced.stl" scale="0.001 0.001 0.001" />
-            </geometry>
-        </collision>
-    </link>
+    <xacro:if value="${WITH_BATTERY}">
+        <link name="pelvis">
+            <inertial>
+                <origin xyz="${Pelvis_x} ${Pelvis_y} ${Pelvis_z}" />
+                <mass value="${Pelvis_mass}" />
+                <inertia ixx="${Pelvis_xx}" ixy="${Pelvis_xy}" ixz="${Pelvis_xz}" iyy="${Pelvis_yy}" iyz="${Pelvis_yz}" izz="${Pelvis_zz}" />
+            </inertial>
+            <visual>
+                <origin xyz="0.0 0 0.0" rpy="0.0 0.0 0.0" />
+                <geometry>
+                    <mesh filename="${MESH_PATH}/v2/pelvis.stl" scale="0.001 0.001 0.001" />
+                </geometry>
+            </visual>
+            <collision>
+                <origin xyz="0.0 0 0.0" rpy="0.0 0.0 0.0" />
+                <geometry>
+                    <mesh filename="${MESH_PATH}/simple/pelvis_reduced.stl" scale="0.001 0.001 0.001" />
+                </geometry>
+            </collision>
+        </link>
+    </xacro:if>
+    <xacro:unless value="WITH_BATTERY">
+        <link name="pelvis">
+            <inertial>
+                <origin xyz="${PelvisNoBatt_x} ${PelvisNoBatt_y} ${PelvisNoBatt_z}" />
+                <mass value="${PelvisNoBatt_mass}" />
+                <inertia ixx="${PelvisNoBatt_xx}" ixy="${PelvisNoBatt_xy}" ixz="${PelvisNoBatt_xz}" iyy="${PelvisNoBatt_yy}" iyz="${PelvisNoBatt_yz}" izz="${PelvisNoBatt_zz}" />
+            </inertial>
+            <visual>
+                <origin xyz="0.0 0 0.0" rpy="0.0 0.0 0.0" />
+                <geometry>
+                    <mesh filename="${MESH_PATH}/v2/pelvis.stl" scale="0.001 0.001 0.001" />
+                </geometry>
+            </visual>
+            <collision>
+                <origin xyz="0.0 0 0.0" rpy="0.0 0.0 0.0" />
+                <geometry>
+                    <mesh filename="${MESH_PATH}/simple/pelvis_reduced.stl" scale="0.001 0.001 0.001" />
+                </geometry>
+            </collision>
+        </link>
+    </xacro:unless>
     <link name="imu_link" />
     <joint name="imu_joint" type="fixed">

File: centauro_urdf/urdf/config/centauro.urdf.xacro (robot description, xacro)
@@ -9,4 +9,5 @@
 <xacro:arg name="big_wheel" default="true"/>
 <xacro:arg name="upper_body" default="true"/>
+<xacro:arg name="battery" default="true"/>
 <xacro:arg name="velodyne" default="false"/>
 <xacro:arg name="realsense" default="false"/>
@@ -31,4 +32,5 @@
 <xacro:property name="ADD_LEGS" value="$(arg legs)" />
 <xacro:property name="ADD_UPPER_BODY" value="$(arg upper_body)" />
+<xacro:property name="WITH_BATTERY" value="$(arg battery)" />
 <xacro:property name="END_EFFECTOR_LEFT" value="$(arg end_effector_left)" />
 <xacro:property name="END_EFFECTOR_RIGHT" value="$(arg end_effector_right)" />

File: centauro_urdf/urdf/parts/inertial_properties.urdf.xacro (robot description, xacro)
@@ -14,4 +14,7 @@
 <xacro:property name="Pelvis_y" value="${2.6534004e+00 * mmTom}"/>
 <xacro:property name="Pelvis_z" value="${7.9167428e+01 * mmTom}"/>
+<xacro:property name="PelvisNoBatt_x" value="${1.0310423e+01 * mmTom}"/>
+<xacro:property name="PelvisNoBatt_y" value="${3.4907373e+00 * mmTom}"/>
+<xacro:property name="PelvisNoBatt_z" value="${5.7233845+01 * mmTom}"/>
 <!-- Inertia -->
 <xacro:property name="Pelvis_xx" value="${3.9195477e+05 * mm2Tom2}"/>
@@ -21,6 +24,13 @@
 <xacro:property name="Pelvis_xz" value="${1.7108607e+04 * mm2Tom2}"/>
 <xacro:property name="Pelvis_yz" value="${5.2627106e+03 * mm2Tom2}"/>
+<xacro:property name="PelvisNoBatt_xx" value="${8.7627533e+05 * mm2Tom2}"/>
+<xacro:property name="PelvisNoBatt_yy" value="${1.6329655e+06 * mm2Tom2}"/>
+<xacro:property name="PelvisNoBatt_zz" value="${1.9611303e+06 * mm2Tom2}"/>
+<xacro:property name="PelvisNoBatt_xy" value="${2.2209997e+04 * mm2Tom2}"/>
+<xacro:property name="PelvisNoBatt_xz" value="${-6.1989843e+03 * mm2Tom2}"/>
+<xacro:property name="PelvisNoBatt_yz" value="${4.5514872+03 * mm2Tom2}"/>
 <!-- Mass -->
 <xacro:property name="Pelvis_mass" value="2.6584529e+01"/>
+<xacro:property name="PelvisNoBatt_mass" value="1.8845851e+01"/>
 <!-- Center of Mass -->
 <xacro:property name="Leg_1_x" value="${3.5958550e-01 * mmTom}"/>
