Commit message: added option to use/remove battery (adapted pelvis inertias)

File: centauro_urdf/urdf/centauro_base.urdf.xacro (robot description, xacro)
@@ -1,8 +1,5 @@
 <?xml version="1.0"?>
 <robot xmlns:xacro="http://ros.org/wiki/xacro" name="centauro">
-    <!--
-  ROS urdf definition of the CENTAURO humanoid robot by Istituto Italiano di Tecnologia
-  Author: Enrico Mingo Hoffman
--->
+    <!-- ROS urdf definition of the CENTAURO humanoid robot by Istituto Italiano di Tecnologia. Author Enrico Mingo Hoffman-->
     <xacro:include filename="${ROOT}/urdf/utils.urdf.xacro" />
     <xacro:include filename="${ROOT}/urdf/parts/kinematics_properties.urdf.xacro" />
@@ -15,23 +12,46 @@
         <origin xyz="0 0 0" rpy="0 0 0" />
     </joint>
-    <link name="pelvis">
-        <inertial>
-            <origin xyz="${Pelvis_x} ${Pelvis_y} ${Pelvis_z}" />
-            <mass value="${Pelvis_mass}" />
-            <inertia ixx="${Pelvis_xx}" ixy="${Pelvis_xy}" ixz="${Pelvis_xz}" iyy="${Pelvis_yy}" iyz="${Pelvis_yz}" izz="${Pelvis_zz}" />
-        </inertial>
-        <visual>
-            <origin xyz="0.0 0 0.0" rpy="0.0 0.0 0.0" />
-            <geometry>
-                <mesh filename="${MESH_PATH}/v2/pelvis.stl" scale="0.001 0.001 0.001" />
-            </geometry>
-        </visual>
-        <collision>
-            <origin xyz="0.0 0 0.0" rpy="0.0 0.0 0.0" />
-            <geometry>
-                <mesh filename="${MESH_PATH}/simple/pelvis_reduced.stl" scale="0.001 0.001 0.001" />
-            </geometry>
-        </collision>
-    </link>
+    <xacro:if value="${WITH_BATTERY}">
+        <link name="pelvis">
+            <inertial>
+                <origin xyz="${Pelvis_x} ${Pelvis_y} ${Pelvis_z}" />
+                <mass value="${Pelvis_mass}" />
+                <inertia ixx="${Pelvis_xx}" ixy="${Pelvis_xy}" ixz="${Pelvis_xz}" iyy="${Pelvis_yy}" iyz="${Pelvis_yz}" izz="${Pelvis_zz}" />
+            </inertial>
+            <visual>
+                <origin xyz="0.0 0 0.0" rpy="0.0 0.0 0.0" />
+                <geometry>
+                    <mesh filename="${MESH_PATH}/v2/pelvis.stl" scale="0.001 0.001 0.001" />
+                </geometry>
+            </visual>
+            <collision>
+                <origin xyz="0.0 0 0.0" rpy="0.0 0.0 0.0" />
+                <geometry>
+                    <mesh filename="${MESH_PATH}/simple/pelvis_reduced.stl" scale="0.001 0.001 0.001" />
+                </geometry>
+            </collision>
+        </link>
+    </xacro:if>
+    <xacro:unless value="WITH_BATTERY">
+        <link name="pelvis">
+            <inertial>
+                <origin xyz="${PelvisNoBatt_x} ${PelvisNoBatt_y} ${PelvisNoBatt_z}" />
+                <mass value="${PelvisNoBatt_mass}" />
+                <inertia ixx="${PelvisNoBatt_xx}" ixy="${PelvisNoBatt_xy}" ixz="${PelvisNoBatt_xz}" iyy="${PelvisNoBatt_yy}" iyz="${PelvisNoBatt_yz}" izz="${PelvisNoBatt_zz}" />
+            </inertial>
+            <visual>
+                <origin xyz="0.0 0 0.0" rpy="0.0 0.0 0.0" />
+                <geometry>
+                    <mesh filename="${MESH_PATH}/v2/pelvis.stl" scale="0.001 0.001 0.001" />
+                </geometry>
+            </visual>
+            <collision>
+                <origin xyz="0.0 0 0.0" rpy="0.0 0.0 0.0" />
+                <geometry>
+                    <mesh filename="${MESH_PATH}/simple/pelvis_reduced.stl" scale="0.001 0.001 0.001" />
+                </geometry>
+            </collision>
+        </link>
+    </xacro:unless>
     <link name="imu_link" />
     <joint name="imu_joint" type="fixed">

File: centauro_urdf/urdf/parts/inertial_properties.urdf.xacro (robot description, xacro)
@@ -14,4 +14,7 @@
 <xacro:property name="Pelvis_y" value="${2.6534004e+00 * mmTom}"/>
 <xacro:property name="Pelvis_z" value="${7.9167428e+01 * mmTom}"/>
+<xacro:property name="PelvisNoBatt_x" value="${1.0310423e+01 * mmTom}"/>
+<xacro:property name="PelvisNoBatt_y" value="${3.4907373e+00 * mmTom}"/>
+<xacro:property name="PelvisNoBatt_z" value="${5.7233845+01 * mmTom}"/>
 <!-- Inertia -->
 <xacro:property name="Pelvis_xx" value="${3.9195477e+05 * mm2Tom2}"/>
@@ -21,6 +24,13 @@
 <xacro:property name="Pelvis_xz" value="${1.7108607e+04 * mm2Tom2}"/>
 <xacro:property name="Pelvis_yz" value="${5.2627106e+03 * mm2Tom2}"/>
+<xacro:property name="PelvisNoBatt_xx" value="${8.7627533e+05 * mm2Tom2}"/>
+<xacro:property name="PelvisNoBatt_yy" value="${1.6329655e+06 * mm2Tom2}"/>
+<xacro:property name="PelvisNoBatt_zz" value="${1.9611303e+06 * mm2Tom2}"/>
+<xacro:property name="PelvisNoBatt_xy" value="${2.2209997e+04 * mm2Tom2}"/>
+<xacro:property name="PelvisNoBatt_xz" value="${-6.1989843e+03 * mm2Tom2}"/>
+<xacro:property name="PelvisNoBatt_yz" value="${4.5514872+03 * mm2Tom2}"/>
 <!-- Mass -->
 <xacro:property name="Pelvis_mass" value="2.6584529e+01"/>
+<xacro:property name="PelvisNoBatt_mass" value="1.8845851e+01"/>
 <!-- Center of Mass -->
 <xacro:property name="Leg_1_x" value="${3.5958550e-01 * mmTom}"/>
@@ -88,5 +98,5 @@
 <!-- Mass -->
 <xacro:property name="Ankle_2_mass" value="1.7656714e+00"/>
-<!-- Note: the "23" suffix denotes the new bigger-size wheel -->
+<!-- Note that the "23" suffix denotes the new bigger-size wheel -->
 <!-- Center of Mass -->
 <xacro:property name="Ankle23_2_x" value="${1.8512273e-01 * mmTom}"/>

Commit message: optional floating joint, realsense mesh to box, wheel mesh to sphere

File: centauro_urdf/urdf/centauro_base.urdf.xacro (robot description, xacro)
@@ -29,4 +29,11 @@
         </collision>
     </link>
+    <xacro:if value="${ADD_FLOATING_BASE}">
+        <link name="world"/>
+        <joint name="floating_joint" type="floating">
+            <parent link="world" />
+            <child link="pelvis" />
+        </joint>
+    </xacro:if>
     <link name="imu_link" />
     <joint name="imu_joint" type="fixed">
@@ -82,6 +89,6 @@
                     <origin xyz="${d435_cam_mount_from_center_offset} ${-d435_cam_depth_py} 0" rpy="${PI/2} 0 ${PI/2}" />
                     <geometry>
-                        <!-- <box size="${d435_cam_width} ${d435_cam_height} ${d435_cam_depth}"/> -->
-                        <mesh filename="package://centauro_urdf/meshes/realsense/d435.dae" />
+                        <box size="${d435_cam_width} ${d435_cam_height} ${d435_cam_depth}"/>
+                        <!-- <mesh filename="package://centauro_urdf/meshes/realsense/d435.dae" /> -->
                     </geometry>
                     <material name="${d435_base_name}_aluminum" />

File: centauro_urdf/urdf/config/centauro.urdf.xacro (robot description, xacro)
@@ -21,5 +21,5 @@
 	<xacro:arg name="t265_base" default="false"/>
 </xacro:unless>
-<xacro:arg name="floating_joint" default="true"/>
+<xacro:arg name="floating_joint" default="false"/>
 <xacro:arg name="virtual_frame" default="false"/> <!-- For cartesio model must be set to true-->
 <xacro:arg name="end_effector_left" default="$(arg end_effector_left)"/> <!-- none, ball, dagana_fixed, dagana -->

File: centauro_urdf/urdf/parts/head.urdf.xacro (robot description, xacro)
@@ -123,6 +123,6 @@
       <origin xyz="${d435_cam_mount_from_center_offset} ${-d435_cam_depth_py} 0" rpy="${PI/2} 0 ${PI/2}"/>
         <geometry>
-          <!-- <box size="${d435_cam_width} ${d435_cam_height} ${d435_cam_depth}"/> -->
-          <mesh filename="package://centauro_urdf/meshes/realsense/d435.dae"/>
+          <box size="${d435_cam_width} ${d435_cam_height} ${d435_cam_depth}"/>
+          <!-- <mesh filename="package://centauro_urdf/meshes/realsense/d435.dae"/> -->
         </geometry>
         <material name="${d435_head_name}_aluminum"/>

File: centauro_urdf/urdf/parts/wheel23.urdf.xacro (robot description, xacro)
@@ -54,6 +54,7 @@
                 <origin xyz="0 0 0" rpy="0 0 0" />
                 <geometry>
-                    <mesh filename="package://centauro_urdf/meshes/v2/collision/mesh_wheel23.stl"
-                        scale="0.001 0.001 ${mirror*0.001}" />
+                    <sphere radius="0.125"/>
+                    <!-- <mesh filename="package://centauro_urdf/meshes/v2/collision/mesh_wheel23.stl"
+                        scale="0.001 0.001 ${mirror*0.001}" /> -->
                 </geometry>
                 <material name="black" />

Commit message: ros2 compat mujoco

File: centauro_urdf/urdf/centauro_base.urdf.xacro (robot description, xacro)
@@ -82,6 +82,6 @@
                     <origin xyz="${d435_cam_mount_from_center_offset} ${-d435_cam_depth_py} 0" rpy="${PI/2} 0 ${PI/2}" />
                     <geometry>
-                        <!-- <box size="${d435_cam_width} ${d435_cam_height} ${d435_cam_depth}"/> -->
-                        <mesh filename="package://centauro_urdf/meshes/realsense/d435.dae" />
+                        <box size="${d435_cam_width} ${d435_cam_height} ${d435_cam_depth}"/>
+                        <!-- <mesh filename="package://centauro_urdf/meshes/realsense/d435.dae" /> -->
                     </geometry>
                     <material name="${d435_base_name}_aluminum" />

Commit message: converted depth .dae to .stl for compatibility with mujoco

File: centauro_urdf/urdf/centauro_base.urdf.xacro (robot description, xacro)
@@ -118,5 +118,5 @@
                     <geometry>
                         <!-- <box size="${d435_cam_width} ${d435_cam_height} ${d435_cam_depth}"/> -->
-                        <mesh filename="${MESH_PATH}/realsense/d435.dae" />
+                        <mesh filename="${MESH_PATH}/realsense/d435.stl" />
                     </geometry>
                     <material name="${d435_base_name}_aluminum" />

Commit message: added fixed_base_joint option

File: centauro_urdf/urdf/centauro_base.urdf.xacro (robot description, xacro)
@@ -34,4 +34,12 @@
             <parent link="world" />
             <child link="pelvis" />
+        </joint>
+    </xacro:if>
+    <xacro:if value="${ADD_FIXED_BASE}">
+        <link name="world"/>
+        <joint name="fixed_joint" type="fixed">
+            <parent link="world" />
+            <child link="pelvis" />
+            <origin xyz="0 0 0.85" rpy="0 0 0" />
         </joint>
     </xacro:if>

File: centauro_urdf/urdf/config/centauro.urdf.xacro (robot description, xacro)
@@ -23,4 +23,5 @@
 </xacro:unless>
 <xacro:arg name="floating_joint" default="false"/>
+<xacro:arg name="fixed_base_joint" default="false"/>
 <xacro:arg name="virtual_frame" default="false"/> <!-- For cartesio model must be set to true-->
 <xacro:arg name="end_effector_left" default="$(arg end_effector_left)"/> <!-- none, ball, dagana_fixed, dagana -->
@@ -37,4 +38,5 @@
 <xacro:property name="DAGANA_STANDALONE_PLUGIN" value="true" />
 <xacro:property name="ADD_FLOATING_BASE" value="$(arg floating_joint)" />
+<xacro:property name="ADD_FIXED_BASE" value="$(arg fixed_base_joint)" />
 <xacro:property name="ADD_VIRTUAL_FRAME" value="$(arg virtual_frame)" />
 <xacro:property name="USE_STICKS" value="false" />

Commit message: add floating joint if required

File: centauro_urdf/urdf/centauro_base.urdf.xacro (robot description, xacro)
@@ -35,4 +35,11 @@
         <child link="imu_link" />
     </joint>
+    <xacro:if value="${ADD_FLOATING_BASE}">
+        <link name="world"/>
+        <joint name="reference" type="floating">
+            <parent link="world"/>
+            <child link="pelvis"/>
+        </joint>
+    </xacro:if>
     <joint name="base_joint" type="fixed">
         <parent link="pelvis" />

Commit message: Added optinal pelvis twist joint

File: centauro_urdf/urdf/centauro_base.urdf.xacro (robot description, xacro)
@@ -55,4 +55,20 @@
         <origin xyz="0 0 0" rpy="0 0 0" />
     </joint>
+    <xacro:if value="${ADD_PELVIS_TWIST}">
+        <link name="twisting_pelvis" >
+            <inertial>
+                <origin xyz="0 0 0" />
+                <mass value="1" />
+                <inertia ixx="${1*1/6*0.2*0.2}" ixy="0" ixz="0" iyy="${1*1/6*0.2*0.2}" iyz="0" izz="${1*1/6*0.2*0.2}" />
+            </inertial>
+        </link>
+        <joint name="twisting_pelvis_joint" type="revolute">
+            <parent link="pelvis" />
+            <child link="twisting_pelvis" />
+            <origin xyz="0 0 0" rpy="0 0 0" />
+            <axis xyz="1 0 0" />
+            <limit effort="10000" velocity="100" lower="-0.15" upper="0.15" />
+        </joint>
+    </xacro:if>
     <xacro:if value="${ADD_UPPER_BODY}">
         <xacro:include filename="$(find centauro_urdf)/urdf/parts/centauro_torso.urdf.xacro" />

File: centauro_urdf/urdf/config/centauro.urdf.xacro (robot description, xacro)
@@ -8,4 +8,5 @@
 <xacro:arg name="sphere_or_ellipsoid_wheel_collision" default="false"/>
 <xacro:arg name="small_sphere_wheel_collision" default="false"/>
+<xacro:arg name="add_twisting_pelvis" default="false"/>
 <xacro:arg name="upper_body" default="true"/>
 <xacro:arg name="velodyne" default="true"/>
@@ -39,4 +40,5 @@
 <xacro:property name="ADD_LEGS" value="$(arg legs)" />
 <xacro:property name="ADD_UPPER_BODY" value="$(arg upper_body)" />
+<xacro:property name="ADD_PELVIS_TWIST" value="$(arg add_twisting_pelvis)" />
 <xacro:property name="END_EFFECTOR_LEFT" value="$(arg end_effector_left)" />
 <xacro:property name="END_EFFECTOR_RIGHT" value="$(arg end_effector_right)" />

File: centauro_urdf/urdf/parts/centauro_leg.urdf.xacro (robot description, xacro)
@@ -4,5 +4,5 @@
 <xacro:include filename="$(find centauro_urdf)/urdf/parts/wheel23.urdf.xacro"/>
 <!-- macro legs -->
-<xacro:macro name="centauro_leg" params="leg_num origin_x origin_y mirror">
+<xacro:macro name="centauro_leg" params="leg_num origin_x origin_y mirror attach_link">
 <link name="hip1_${leg_num}">
 	<inertial>
@@ -135,5 +135,5 @@
 <!-- ******************************** -->
 <joint name="hip_yaw_${leg_num}" type="revolute">
-	<parent link="pelvis"/>
+	<parent link="${attach_link}"/>
 	<child link="hip1_${leg_num}"/>
 	<origin xyz="${origin_x*Leg_1_Ox} ${origin_y*Leg_1_Oy} ${Leg_1_Oz}" rpy="${Leg_1_roll} ${Leg_1_pitch} ${Leg_1_yaw}"/>

File: centauro_urdf/urdf/parts/legs.urdf.xacro (robot description, xacro)
@@ -2,11 +2,19 @@
 <robot xmlns:xacro="http://ros.org/wiki/xacro">
 <xacro:include filename="$(find centauro_urdf)/urdf/parts/centauro_leg.urdf.xacro" />
-<xacro:centauro_leg leg_num="1" origin_x="1" origin_y="-1" mirror="-1">
+<xacro:centauro_leg leg_num="1" origin_x="1" origin_y="-1" mirror="-1" attach_link="pelvis">
 </xacro:centauro_leg>
-<xacro:centauro_leg leg_num="2" origin_x="1" origin_y="1" mirror="1">
+<xacro:centauro_leg leg_num="2" origin_x="1" origin_y="1" mirror="1" attach_link="pelvis">
 </xacro:centauro_leg>
-<xacro:centauro_leg leg_num="3" origin_x="-1" origin_y="-1" mirror="-1">
-</xacro:centauro_leg>
-<xacro:centauro_leg leg_num="4" origin_x="-1" origin_y="1" mirror="1">
-</xacro:centauro_leg>
+<xacro:unless value="${ADD_PELVIS_TWIST}">
+    <xacro:centauro_leg leg_num="3" origin_x="-1" origin_y="-1" mirror="-1" attach_link="pelvis">
+    </xacro:centauro_leg>
+    <xacro:centauro_leg leg_num="4" origin_x="-1" origin_y="1" mirror="1" attach_link="pelvis">
+    </xacro:centauro_leg>
+</xacro:unless>
+<xacro:if value="${ADD_PELVIS_TWIST}">
+    <xacro:centauro_leg leg_num="3" origin_x="-1" origin_y="-1" mirror="-1" attach_link="twisting_pelvis">
+    </xacro:centauro_leg>
+    <xacro:centauro_leg leg_num="4" origin_x="-1" origin_y="1" mirror="1" attach_link="twisting_pelvis">
+    </xacro:centauro_leg>
+</xacro:if>
 </robot>
