Commit message: wheel custom physics from mkamedula's centauro-simulator

File: centauro_urdf/urdf/gazebo/centauro.gazebo.xacro (robot description, xacro)
@@ -3,38 +3,122 @@
 <xacro:if value="${ADD_LEGS}">
 <gazebo reference="wheel_1">
-	<kp>1000000.0</kp>
-	<kd>100.0</kd>
-	<mu1>1.0</mu1>
-	<mu2>1.0</mu2>
-	<!--fdir1>1 0 0</fdir1-->
-	<maxVel>1.0</maxVel>
-	<minDepth>0.00</minDepth>
+    <material>Gazebo/Residential </material>
+    <collision>
+        <surface>
+            <friction>
+                <ode>
+                    <mu>0.5</mu>
+                    <mu2>0.5</mu2>
+                </ode>
+                <bullet>
+                    <friction>0.5</friction>
+                    <friction2>0.5</friction2>
+                </bullet>
+            </friction>
+            <contact>
+                <ode>
+                    <kp>2100000</kp>
+                    <kd>1</kd>
+                    <max_vel>100</max_vel>
+                </ode>
+                <bullet>
+                    <soft_cfm>0.007</soft_cfm>
+                    <soft_erp>0.25</soft_erp>
+                    <kp>1000000</kp>
+                    <kd>5</kd>
+                </bullet>
+            </contact>
+        </surface>
+    </collision>
 </gazebo>
 <gazebo reference="wheel_2">
-	<kp>1000000.0</kp>
-	<kd>100.0</kd>
-	<mu1>1.0</mu1>
-	<mu2>1.0</mu2>
-	<!--fdir1>1 0 0</fdir1-->
-	<maxVel>1.0</maxVel>
-	<minDepth>0.00</minDepth>
+    <material>Gazebo/Residential</material>
+    <collision>
+        <surface>
+            <friction>
+                <ode>
+                    <mu>0.5</mu>
+                    <mu2>0.5</mu2>
+                </ode>
+                <bullet>
+                    <friction>0.5</friction>
+                    <friction2>0.5</friction2>
+                </bullet>
+            </friction>
+            <contact>
+                <ode>
+                    <kp>2100000</kp>
+                    <kd>1</kd>
+                    <max_vel>100</max_vel>
+                </ode>
+                <bullet>
+                    <soft_cfm>0.007</soft_cfm>
+                    <soft_erp>0.25</soft_erp>
+                    <kp>1000000</kp>
+                    <kd>5</kd>
+                </bullet>
+            </contact>
+        </surface>
+    </collision>
 </gazebo>
 <gazebo reference="wheel_3">
-	<kp>1000000.0</kp>
-	<kd>100.0</kd>
-	<mu1>1.0</mu1>
-	<mu2>1.0</mu2>
-	<!--fdir1>1 0 0</fdir1-->
-	<maxVel>1.0</maxVel>
-	<minDepth>0.00</minDepth>
+    <material>Gazebo/Residential </material>
+    <collision>
+        <surface>
+            <friction>
+                <ode>
+                    <mu>0.5</mu>
+                    <mu2>0.5</mu2>
+                </ode>
+                <bullet>
+                    <friction>0.5</friction>
+                    <friction2>0.5</friction2>
+                </bullet>
+            </friction>
+            <contact>
+                <ode>
+                    <kp>2100000</kp>
+                    <kd>1</kd>
+                    <max_vel>100</max_vel>
+                </ode>
+                <bullet>
+                    <soft_cfm>0.007</soft_cfm>
+                    <soft_erp>0.25</soft_erp>
+                    <kp>1000000</kp>
+                    <kd>5</kd>
+                </bullet>
+            </contact>
+        </surface>
+    </collision>
 </gazebo>
 <gazebo reference="wheel_4">
-	<kp>1000000.0</kp>
-	<kd>100.0</kd>
-	<mu1>1.0</mu1>
-	<mu2>1.0</mu2>
-	<!--fdir1>1 0 0</fdir1-->
-	<maxVel>1.0</maxVel>
-	<minDepth>0.00</minDepth>
+    <material>Gazebo/Residential</material>
+    <collision>
+        <surface>
+            <friction>
+                <ode>
+                    <mu>0.5</mu>
+                    <mu2>0.5</mu2>
+                </ode>
+                <bullet>
+                    <friction>0.5</friction>
+                    <friction2>0.5</friction2>
+                </bullet>
+            </friction>
+            <contact>
+                <ode>
+                    <kp>2100000</kp>
+                    <kd>1</kd>
+                    <max_vel>100</max_vel>
+                </ode>
+                <bullet>
+                    <soft_cfm>0.007</soft_cfm>
+                    <soft_erp>0.25</soft_erp>
+                    <kp>1000000</kp>
+                    <kd>5</kd>
+                </bullet>
+            </contact>
+        </surface>
+    </collision>
 </gazebo>
 <gazebo reference="hip_yaw_1">

Commit message: Adjust gains and friction values wheels

File: centauro_urdf/urdf/gazebo/centauro.gazebo.xacro (robot description, xacro)
@@ -3,38 +3,122 @@
 <xacro:if value="${ADD_LEGS}">
 <gazebo reference="wheel_1">
-	<kp>1000000.0</kp>
-	<kd>100.0</kd>
-	<mu1>1.0</mu1>
-	<mu2>1.0</mu2>
-	<fdir1>1 0 0</fdir1>
-	<maxVel>1.0</maxVel>
-	<minDepth>0.00</minDepth>
+    <material>Gazebo/Residential </material>
+    <collision>
+        <surface>
+            <friction>
+                <ode>
+                    <mu>0.5</mu>
+                    <mu2>0.5</mu2>
+                </ode>
+                <bullet>
+                    <friction>0.5</friction>
+                    <friction2>0.5</friction2>
+                </bullet>
+            </friction>
+            <contact>
+                <ode>
+                    <kp>2100000</kp>
+                    <kd>1</kd>
+                    <max_vel>100</max_vel>
+                </ode>
+                <bullet>
+                    <soft_cfm>0.007</soft_cfm>
+                    <soft_erp>0.25</soft_erp>
+                    <kp>1000000</kp>
+                    <kd>5</kd>
+                </bullet>
+            </contact>
+        </surface>
+    </collision>
 </gazebo>
 <gazebo reference="wheel_2">
-	<kp>1000000.0</kp>
-	<kd>100.0</kd>
-	<mu1>1.0</mu1>
-	<mu2>1.0</mu2>
-	<fdir1>1 0 0</fdir1>
-	<maxVel>1.0</maxVel>
-	<minDepth>0.00</minDepth>
+    <material>Gazebo/Residential</material>
+    <collision>
+        <surface>
+            <friction>
+                <ode>
+                    <mu>0.5</mu>
+                    <mu2>0.5</mu2>
+                </ode>
+                <bullet>
+                    <friction>0.5</friction>
+                    <friction2>0.5</friction2>
+                </bullet>
+            </friction>
+            <contact>
+                <ode>
+                    <kp>2100000</kp>
+                    <kd>1</kd>
+                    <max_vel>100</max_vel>
+                </ode>
+                <bullet>
+                    <soft_cfm>0.007</soft_cfm>
+                    <soft_erp>0.25</soft_erp>
+                    <kp>1000000</kp>
+                    <kd>5</kd>
+                </bullet>
+            </contact>
+        </surface>
+    </collision>
 </gazebo>
 <gazebo reference="wheel_3">
-	<kp>1000000.0</kp>
-	<kd>100.0</kd>
-	<mu1>1.0</mu1>
-	<mu2>1.0</mu2>
-	<fdir1>1 0 0</fdir1>
-	<maxVel>1.0</maxVel>
-	<minDepth>0.00</minDepth>
+    <material>Gazebo/Residential </material>
+    <collision>
+        <surface>
+            <friction>
+                <ode>
+                    <mu>0.5</mu>
+                    <mu2>0.5</mu2>
+                </ode>
+                <bullet>
+                    <friction>0.5</friction>
+                    <friction2>0.5</friction2>
+                </bullet>
+            </friction>
+            <contact>
+                <ode>
+                    <kp>2100000</kp>
+                    <kd>1</kd>
+                    <max_vel>100</max_vel>
+                </ode>
+                <bullet>
+                    <soft_cfm>0.007</soft_cfm>
+                    <soft_erp>0.25</soft_erp>
+                    <kp>1000000</kp>
+                    <kd>5</kd>
+                </bullet>
+            </contact>
+        </surface>
+    </collision>
 </gazebo>
 <gazebo reference="wheel_4">
-	<kp>1000000.0</kp>
-	<kd>100.0</kd>
-	<mu1>1.0</mu1>
-	<mu2>1.0</mu2>
-	<fdir1>1 0 0</fdir1>
-	<maxVel>1.0</maxVel>
-	<minDepth>0.00</minDepth>
+    <material>Gazebo/Residential</material>
+    <collision>
+        <surface>
+            <friction>
+                <ode>
+                    <mu>0.5</mu>
+                    <mu2>0.5</mu2>
+                </ode>
+                <bullet>
+                    <friction>0.5</friction>
+                    <friction2>0.5</friction2>
+                </bullet>
+            </friction>
+            <contact>
+                <ode>
+                    <kp>2100000</kp>
+                    <kd>1</kd>
+                    <max_vel>100</max_vel>
+                </ode>
+                <bullet>
+                    <soft_cfm>0.007</soft_cfm>
+                    <soft_erp>0.25</soft_erp>
+                    <kp>1000000</kp>
+                    <kd>5</kd>
+                </bullet>
+            </contact>
+        </surface>
+    </collision>
 </gazebo>
 <gazebo reference="hip_yaw_1">

Commit message: increase wheels friction coeff to 0.9

File: centauro_urdf/urdf/gazebo/centauro.gazebo.xacro (robot description, xacro)
@@ -1,4 +1,5 @@
 <?xml version="1.0"?>
 <robot xmlns:xacro="http://ros.org/wiki/xacro">
+<xacro:property name="friction_coeff" value="0.9" />
 <xacro:if value="${ADD_LEGS}">
 <gazebo reference="wheel_1">
@@ -8,10 +9,10 @@
             <friction>
                 <ode>
-                    <mu>0.5</mu>
-                    <mu2>0.5</mu2>
-                </ode>
-                <bullet>
-                    <friction>0.5</friction>
-                    <friction2>0.5</friction2>
+                    <mu>${friction_coeff}</mu>
+                    <mu2>${friction_coeff}</mu2>
+                </ode>
+                <bullet>
+                    <friction>${friction_coeff}</friction>
+                    <friction2>${friction_coeff}</friction2>
                 </bullet>
             </friction>
@@ -38,10 +39,10 @@
             <friction>
                 <ode>
-                    <mu>0.5</mu>
-                    <mu2>0.5</mu2>
-                </ode>
-                <bullet>
-                    <friction>0.5</friction>
-                    <friction2>0.5</friction2>
+                    <mu>${friction_coeff}</mu>
+                    <mu2>${friction_coeff}</mu2>
+                </ode>
+                <bullet>
+                    <friction>${friction_coeff}</friction>
+                    <friction2>${friction_coeff}</friction2>
                 </bullet>
             </friction>
@@ -68,10 +69,10 @@
             <friction>
                 <ode>
-                    <mu>0.5</mu>
-                    <mu2>0.5</mu2>
-                </ode>
-                <bullet>
-                    <friction>0.5</friction>
-                    <friction2>0.5</friction2>
+                    <mu>${friction_coeff}</mu>
+                    <mu2>${friction_coeff}</mu2>
+                </ode>
+                <bullet>
+                    <friction>${friction_coeff}</friction>
+                    <friction2>${friction_coeff}</friction2>
                 </bullet>
             </friction>
@@ -98,10 +99,10 @@
             <friction>
                 <ode>
-                    <mu>0.5</mu>
-                    <mu2>0.5</mu2>
-                </ode>
-                <bullet>
-                    <friction>0.5</friction>
-                    <friction2>0.5</friction2>
+                    <mu>${friction_coeff}</mu>
+                    <mu2>${friction_coeff}</mu2>
+                </ode>
+                <bullet>
+                    <friction>${friction_coeff}</friction>
+                    <friction2>${friction_coeff}</friction2>
                 </bullet>
             </friction>

Commit message: add gazebo collision properties for ball EEs to stabilize contacts (for now same as wheels)

File: centauro_urdf/urdf/gazebo/centauro.gazebo.xacro (robot description, xacro)
@@ -267,4 +267,75 @@
     </xacro:if>
     <xacro:if value="${ADD_UPPER_BODY}">
+    	<!-- add tags similar with wheels so that arm ball EE can have stable contacts -->
+        <gazebo reference="ball1">
+            <material>Gazebo/Residential</material>
+            <collision>
+                <surface>
+                    <friction>
+                        <!-- <torsional>
+                            <coefficient> 1.0 </coefficient>
+                            <use_patch_radius>true</use_patch_radius>
+                            <patch_radius>0.2</patch_radius>
+                        </torsional> -->
+                        <ode>
+                            <mu>1.0</mu>
+                            <mu2>1.0</mu2>
+                        </ode>
+                        <bullet>
+                            <friction>1.0</friction>
+                            <friction2>1.0</friction2>
+                        </bullet>
+                    </friction>
+                    <contact>
+                        <ode>
+                            <kp>2100000</kp>
+                            <kd>1</kd>
+                            <max_vel>100</max_vel>
+                        </ode>
+                        <bullet>
+                            <soft_cfm>0.007</soft_cfm>
+                            <soft_erp>0.25</soft_erp>
+                            <kp>1000000</kp>
+                            <kd>5</kd>
+                        </bullet>
+                    </contact>
+                </surface>
+            </collision>
+        </gazebo>
+        <gazebo reference="ball2">
+            <material>Gazebo/Residential</material>
+            <collision>
+                <surface>
+                    <friction>
+                        <!-- <torsional>
+                            <coefficient> 1.0 </coefficient>
+                            <use_patch_radius>true</use_patch_radius>
+                            <patch_radius>0.2</patch_radius>
+                        </torsional> -->
+                        <ode>
+                            <mu>1.0</mu>
+                            <mu2>1.0</mu2>
+                        </ode>
+                        <bullet>
+                            <friction>1.0</friction>
+                            <friction2>1.0</friction2>
+                        </bullet>
+                    </friction>
+                    <contact>
+                        <ode>
+                            <kp>2100000</kp>
+                            <kd>1</kd>
+                            <max_vel>100</max_vel>
+                        </ode>
+                        <bullet>
+                            <soft_cfm>0.007</soft_cfm>
+                            <soft_erp>0.25</soft_erp>
+                            <kp>1000000</kp>
+                            <kd>5</kd>
+                        </bullet>
+                    </contact>
+                </surface>
+            </collision>
+        </gazebo>
         <gazebo reference="torso_yaw">
             <implicitSpringDamper>1</implicitSpringDamper>

Commit message: delete color overwriting

File: centauro_urdf/urdf/gazebo/centauro.gazebo.xacro (robot description, xacro)
@@ -30,5 +30,4 @@
         </gazebo>
         <gazebo reference="wheel_1">
-            <material>Gazebo/Residential </material>
             <collision>
                 <surface>
@@ -65,5 +64,4 @@
         </gazebo>
         <gazebo reference="wheel_2">
-            <material>Gazebo/Residential</material>
             <collision>
                 <surface>
@@ -100,5 +98,4 @@
         </gazebo>
         <gazebo reference="wheel_3">
-            <material>Gazebo/Residential </material>
             <collision>
                 <surface>
@@ -135,5 +132,4 @@
         </gazebo>
         <gazebo reference="wheel_4">
-            <material>Gazebo/Residential</material>
             <collision>
                 <surface>
@@ -269,5 +265,4 @@
     	<!-- add tags similar with wheels so that arm ball EE can have stable contacts -->
         <gazebo reference="ball1">
-            <material>Gazebo/Residential</material>
             <collision>
                 <surface>
@@ -304,5 +299,4 @@
         </gazebo>
         <gazebo reference="ball2">
-            <material>Gazebo/Residential</material>
             <collision>
                 <surface>
