Commit message: colours

File: centauro_urdf/urdf/gazebo/materials.gazebo.xacro (robot description, xacro)
@@ -69,8 +69,8 @@
 <xacro:if value="${ADD_ROD_PLATE_END_EFFECTOR}">
 <gazebo reference="rod_plate1">
-	<material>Gazebo/BlackTransparent</material>
+	<material>Gazebo/GreenTransparent</material>
 </gazebo>
 <gazebo reference="rod_plate2">
-	<material>Gazebo/BlackTransparent</material>
+	<material>Gazebo/RedTransparent</material>
 </gazebo>
 </xacro:if>

Commit message: change materials

File: centauro_urdf/urdf/gazebo/materials.gazebo.xacro (robot description, xacro)
@@ -69,8 +69,8 @@
 <xacro:if value="${ADD_ROD_PLATE_END_EFFECTOR}">
 <gazebo reference="rod_plate1">
-	<material>Gazebo/GreenTransparent</material>
+	<material>Gazebo/BlueTransparent</material>
 </gazebo>
 <gazebo reference="rod_plate2">
-	<material>Gazebo/RedTransparent</material>
+	<material>Gazebo/GreenTransparent</material>
 </gazebo>
 </xacro:if>

Commit message: Green color ball ee that consist payload

File: centauro_urdf/urdf/gazebo/materials.gazebo.xacro (robot description, xacro)
@@ -61,8 +61,8 @@
 <xacro:if value="${ADD_BALL_END_EFFECTOR}">
 <gazebo reference="ball1">
-	<material>Gazebo/BlackTransparent</material>
+	<material>Gazebo/GreenTransparent</material>
 </gazebo>
 <gazebo reference="ball2">
-	<material>Gazebo/BlackTransparent</material>
+	<material>Gazebo/GreenTransparent</material>
 </gazebo>
 </xacro:if>

Commit message: xacro if with or

File: centauro_urdf/urdf/gazebo/materials.gazebo.xacro (robot description, xacro)
@@ -69,5 +69,5 @@
 	</gazebo>
 </xacro:if>
-<xacro:if value="${END_EFFECTOR_LEFT == 'dagana_fixed'}">
+<xacro:if value="${END_EFFECTOR_LEFT == 'dagana_fixed' or END_EFFECTOR_LEFT == 'dagana'}">
 	<gazebo reference="dagana_1_top_link">
 		<material>Gazebo/BlackTransparent</material>
@@ -77,21 +77,5 @@
 	</gazebo>
 </xacro:if>
-<xacro:if value="${END_EFFECTOR_RIGHT == 'dagana_fixed'}">
-	<gazebo reference="dagana_2_top_link">
-		<material>Gazebo/BlackTransparent</material>
-	</gazebo>
-	<gazebo reference="dagana_2_bottom_link">
-		<material>Gazebo/BlackTransparent</material>
-	</gazebo>
-</xacro:if>
-<xacro:if value="${END_EFFECTOR_LEFT == 'dagana'}">
-	<gazebo reference="dagana_1_top_link">
-		<material>Gazebo/BlackTransparent</material>
-	</gazebo>
-	<gazebo reference="dagana_1_bottom_link">
-		<material>Gazebo/BlackTransparent</material>
-	</gazebo>
-</xacro:if>
-<xacro:if value="${END_EFFECTOR_RIGHT == 'dagana'}">
+<xacro:if value="${END_EFFECTOR_RIGHT == 'dagana_fixed' or END_EFFECTOR_RIGHT == 'dagana'}">
 	<gazebo reference="dagana_2_top_link">
 		<material>Gazebo/BlackTransparent</material>

Commit message: orange centauro with ligher grey

File: centauro_urdf/urdf/gazebo/materials.gazebo.xacro (robot description, xacro)
@@ -3,47 +3,47 @@
 <xacro:macro name="centauro_leg_materials" params="leg_num">
 <gazebo reference="hip1_${leg_num}">
-	<material>Gazebo/LightBlueLaser</material>
+	<material>Gazebo/Orange</material>
 </gazebo>
 <gazebo reference="hip2_${leg_num}">
-	<material>Gazebo/BlackTransparent</material>
+	<material>Gazebo/DarkGrey</material>
 </gazebo>
 <gazebo reference="knee_${leg_num}">
-	<material>Gazebo/LightBlueLaser</material>
+	<material>Gazebo/Orange</material>
 </gazebo>
 <gazebo reference="ankle1_${leg_num}">
-	<material>Gazebo/LightBlueLaser</material>
+	<material>Gazebo/Orange</material>
 </gazebo>
 <gazebo reference="ankle2_${leg_num}">
-	<material>Gazebo/LightBlueLaser</material>
+	<material>Gazebo/Orange</material>
 </gazebo>
 <gazebo reference="wheel_${leg_num}">
-	<material>Gazebo/BlackTransparent</material>
+	<material>Gazebo/DarkGrey</material>
 </gazebo>
 </xacro:macro>
 <xacro:macro name="centauro_arm_materials" params="arm_num">
 <gazebo reference="arm${arm_num}_1">
-	<material>Gazebo/BlackTransparent</material>
+	<material>Gazebo/DarkGrey</material>
 </gazebo>
 <gazebo reference="arm${arm_num}_2">
-	<material>Gazebo/LightBlueLaser</material>
+	<material>Gazebo/Orange</material>
 </gazebo>
 <gazebo reference="arm${arm_num}_3">
-	<material>Gazebo/LightBlueLaser</material>
+	<material>Gazebo/Orange</material>
 </gazebo>
 <gazebo reference="arm${arm_num}_4">
-	<material>Gazebo/LightBlueLaser</material>
+	<material>Gazebo/Orange</material>
 </gazebo>
 <gazebo reference="arm${arm_num}_5">
-	<material>Gazebo/BlackTransparent</material>
+	<material>Gazebo/DarkGrey</material>
 </gazebo>
 <gazebo reference="arm${arm_num}_6">
-	<material>Gazebo/LightBlueLaser</material>
+	<material>Gazebo/Orange</material>
 </gazebo>
 <gazebo reference="arm${arm_num}_7">
-	<material>Gazebo/LightBlueLaser</material>
+	<material>Gazebo/Orange</material>
 </gazebo>
 </xacro:macro>
 <gazebo reference="pelvis">
-	<material>Gazebo/LightBlueLaser</material>
+	<material>Gazebo/Orange</material>
 </gazebo>
 <xacro:if value="${ADD_LEGS}">
@@ -55,5 +55,5 @@
 <xacro:if value="${ADD_UPPER_BODY}">
 <gazebo reference="torso_2">
-	<material>Gazebo/BlackTransparent</material>
+	<material>Gazebo/DarkGrey</material>
 </gazebo>
 <xacro:centauro_arm_materials arm_num="1"/>
@@ -61,26 +61,26 @@
 <xacro:if value="${END_EFFECTOR_LEFT == 'ball'}">
 	<gazebo reference="ball1">
-		<material>Gazebo/BlackTransparent</material>
+		<material>Gazebo/DarkGrey</material>
 	</gazebo>
 </xacro:if>
 <xacro:if value="${END_EFFECTOR_RIGHT == 'ball'}">
 	<gazebo reference="ball2">
-		<material>Gazebo/BlackTransparent</material>
+		<material>Gazebo/DarkGrey</material>
 	</gazebo>
 </xacro:if>
 <xacro:if value="${END_EFFECTOR_LEFT == 'dagana_fixed' or END_EFFECTOR_LEFT == 'dagana'}">
 	<gazebo reference="dagana_1_top_link">
-		<material>Gazebo/BlackTransparent</material>
+		<material>Gazebo/DarkGrey</material>
 	</gazebo>
 	<gazebo reference="dagana_1_bottom_link">
-		<material>Gazebo/BlackTransparent</material>
+		<material>Gazebo/DarkGrey</material>
 	</gazebo>
 </xacro:if>
 <xacro:if value="${END_EFFECTOR_RIGHT == 'dagana_fixed' or END_EFFECTOR_RIGHT == 'dagana'}">
 	<gazebo reference="dagana_2_top_link">
-		<material>Gazebo/BlackTransparent</material>
+		<material>Gazebo/DarkGrey</material>
 	</gazebo>
 	<gazebo reference="dagana_2_bottom_link">
-		<material>Gazebo/BlackTransparent</material>
+		<material>Gazebo/DarkGrey</material>
 	</gazebo>
 </xacro:if>
