Commit message: added xbot2 link state sensor

File: centauro_urdf/urdf/gazebo/xbot.gazebo.xacro (robot description, xacro)
@@ -2,4 +2,10 @@
 <robot xmlns:xacro="http://ros.org/wiki/xacro">
 <gazebo>
+    <plugin name="xbot2_link_state_sensor" filename="libxbot2_gz_link_state_sensor.so">
+        <links>
+            <link name="pelvis"/>
+            <link name="wheel_1"/>
+        </links>
+    </plugin>
     <plugin name="xbot2_joint_driver" filename="libxbot2_gz_joint_server.so">
         <pid>

Commit message: gripper adapter for dagana control

File: centauro_urdf/urdf/gazebo/xbot.gazebo.xacro (robot description, xacro)
@@ -10,26 +10,5 @@
     <plugin name="xbot2_ft_driver" filename="libxbot2_gz_ft_server.so"/>
     <plugin name="xbot2_imu_driver" filename="libxbot2_gz_imu_server.so"/>
-    <xacro:if value="${END_EFFECTOR_RIGHT == 'dagana'}">
-    <xacro:if value="${DAGANA_STANDALONE_PLUGIN}">
-        <plugin filename="libdagana_gazebo_DaganaPlugin.so" name="dagana_plugin">
-            <gripperName>dagana_2</gripperName>
-            <jointName>dagana_2_claw_joint</jointName>
-            <rate>100</rate>
-            <p>1</p>
-            <i>0.1</i>
-            <d>0.01</d>
-            <cmdMax>1000</cmdMax>
-            <cmdMin>-1000</cmdMin>
-        </plugin>
-    </xacro:if>
-    </xacro:if>
     <plugin name="xbot2_joint_driver" filename="libxbot2_gz_joint_server.so">
-        <xacro:if value="${END_EFFECTOR_RIGHT == 'dagana'}">
-        <xacro:if value="${DAGANA_STANDALONE_PLUGIN}">
-        <ignore_joints>
-            <joint name="dagana_2_claw_joint" />
-        </ignore_joints>
-        </xacro:if>
-        </xacro:if>
         <pid>
             <gain name="lowpwr_mot" p="50"  d="5"/>
@@ -38,4 +17,5 @@
             <gain name="big_mot"    p="8000" d="50"/>
             <gain name="wheel_mot"  p="0" d="10"/>
+            <gain name="dagana_mot"  p="10" d="0.5"/>
             <pid name="neck_yaw" profile="lowpwr_mot"/>
             <pid name="neck_pitch" profile="lowpwr_mot"/>
@@ -47,5 +27,5 @@
             <pid name="j_arm1_5" profile="small_mot"/>
             <pid name="j_arm1_6" profile="small_mot"/>
-            <pid name="j_arm1_7" profile="small_mot"/>
+            <pid name="dagana_1_claw_joint" profile="dagana_mot"/>
             <pid name="j_arm2_1" profile="medium_mot"/>
             <pid name="j_arm2_2" profile="medium_mot"/>
@@ -54,5 +34,5 @@
             <pid name="j_arm2_5" profile="small_mot"/>
             <pid name="j_arm2_6" profile="small_mot"/>
-            <pid name="j_arm2_7" profile="small_mot"/>
+            <pid name="dagana_2_claw_joint" profile="dagana_mot"/>
             <pid name="torso_yaw" profile="big_mot"/>
             <pid name="hip_yaw_1"     profile="big_mot"/>

Commit message: wip camera :(

File: centauro_urdf/urdf/gazebo/xbot.gazebo.xacro (robot description, xacro)
@@ -5,5 +5,4 @@
         <links>
             <link name="pelvis"/>
-            <link name="wheel_1"/>
         </links>
     </plugin>

File: centauro_urdf/urdf/parts/head.urdf.xacro (robot description, xacro)
@@ -90,5 +90,5 @@
     <origin xyz="0.03015 0 -0.0125" rpy="0 0 0"/>
   </xacro:property>
-  <xacro:if value="${ADD_D435I_HEAD}">
+  <!-- <xacro:if value="${ADD_D435I_HEAD}">
     <xacro:include filename="$(find realsense_gazebo_description)/urdf/_d435i.urdf.xacro" />
     <xacro:sensor_d435i parent="${d435_head_parent_name}"
@@ -111,6 +111,6 @@
         <xacro:insert_block name="d435_head_origin" />
     </xacro:sensor_d435i>
-  </xacro:if>
-  <xacro:unless value="${ADD_D435I_HEAD}">
+  </xacro:if> -->
+  <!-- <xacro:unless value="${ADD_D435I_HEAD}"> -->
     <!--  Copied from _d435.urdf.xacro    -->
     <xacro:property name="d435_cam_width" value="0.090"/>
@@ -155,5 +155,5 @@
       </inertial>
     </link>
-  </xacro:unless>
+  <!-- </xacro:unless> -->
   <xacro:if value="${ADD_VELODYNE}">
     <xacro:include filename="$(find velodyne_description)/urdf/VLP-16.urdf.xacro"/>
