Commit message: new end effectors also for config of virtual frame and gazebo materials files

File: centauro_urdf/urdf/config/centauro_virtual_frame.urdf.xacro (robot description, xacro)
@@ -6,9 +6,12 @@
     <xacro:arg name="add_legs" default="true"/>
     <xacro:arg name="add_upper_body" default="true"/>
+    <xacro:arg name="end_effector_left" default="ball"/> <!-- none, ball, dagana_fixed, dagana -->
+	<xacro:arg name="end_effector_right" default="ball"/> <!-- none, ball, dagana_fixed, dagana -->
     <!-- ************SELECT PARTS*************-->
     <!-- *************************************-->
     <xacro:property name="ADD_LEGS" value="$(arg add_legs)" />
     <xacro:property name="ADD_UPPER_BODY" value="$(arg add_upper_body)" />
-    <xacro:property name="ADD_BALL_END_EFFECTOR" value="true" />
+	<xacro:property name="END_EFFECTOR_LEFT" value="$(arg end_effector_left)" />
+	<xacro:property name="END_EFFECTOR_RIGHT" value="$(arg end_effector_right)" />
     <xacro:property name="ADD_FLOATING_BASE" value="$(arg add_legs)" />
     <xacro:property name="ADD_VIRTUAL_FRAME" value="true" />

File: centauro_urdf/urdf/gazebo/materials.gazebo.xacro (robot description, xacro)
@@ -59,11 +59,45 @@
 <xacro:centauro_arm_materials arm_num="1"/>
 <xacro:centauro_arm_materials arm_num="2"/>
-<xacro:if value="${ADD_BALL_END_EFFECTOR}">
-<gazebo reference="ball1">
-	<material>Gazebo/BlackTransparent</material>
-</gazebo>
-<gazebo reference="ball2">
-	<material>Gazebo/BlackTransparent</material>
-</gazebo>
+<xacro:if value="${END_EFFECTOR_LEFT == 'ball'}">
+	<gazebo reference="ball1">
+		<material>Gazebo/BlackTransparent</material>
+	</gazebo>
+</xacro:if>
+<xacro:if value="${END_EFFECTOR_RIGHT == 'ball'}">
+	<gazebo reference="ball2">
+		<material>Gazebo/BlackTransparent</material>
+	</gazebo>
+</xacro:if>
+<xacro:if value="${END_EFFECTOR_LEFT == 'dagana_fixed'}">
+	<gazebo reference="dagana_1_top_link">
+		<material>Gazebo/BlackTransparent</material>
+	</gazebo>
+	<gazebo reference="dagana_1_bottom_link">
+		<material>Gazebo/BlackTransparent</material>
+	</gazebo>
+</xacro:if>
+<xacro:if value="${END_EFFECTOR_RIGHT == 'dagana_fixed'}">
+	<gazebo reference="dagana_2_top_link">
+		<material>Gazebo/BlackTransparent</material>
+	</gazebo>
+	<gazebo reference="dagana_2_bottom_link">
+		<material>Gazebo/BlackTransparent</material>
+	</gazebo>
+</xacro:if>
+<xacro:if value="${END_EFFECTOR_LEFT == 'dagana'}">
+	<gazebo reference="dagana_1_top_link">
+		<material>Gazebo/BlackTransparent</material>
+	</gazebo>
+	<gazebo reference="dagana_1_bottom_link">
+		<material>Gazebo/BlackTransparent</material>
+	</gazebo>
+</xacro:if>
+<xacro:if value="${END_EFFECTOR_RIGHT == 'dagana'}">
+	<gazebo reference="dagana_2_top_link">
+		<material>Gazebo/BlackTransparent</material>
+	</gazebo>
+	<gazebo reference="dagana_2_bottom_link">
+		<material>Gazebo/BlackTransparent</material>
+	</gazebo>
 </xacro:if>
 </xacro:if>

Commit message: add ft_sensor xacro propery at config file of virtual_frame related xacro

File: centauro_urdf/urdf/config/centauro_virtual_frame.urdf.xacro (robot description, xacro)
@@ -7,15 +7,17 @@
     <xacro:arg name="add_upper_body" default="true"/>
     <xacro:arg name="end_effector_left" default="ball"/> <!-- none, ball, dagana_fixed, dagana -->
-	<xacro:arg name="end_effector_right" default="ball"/> <!-- none, ball, dagana_fixed, dagana -->
+    <xacro:arg name="end_effector_right" default="ball"/> <!-- none, ball, dagana_fixed, dagana -->
+    <xacro:arg name="ft_sensors" default="false"/>
     <!-- ************SELECT PARTS*************-->
     <!-- *************************************-->
     <xacro:property name="ADD_LEGS" value="$(arg add_legs)" />
     <xacro:property name="ADD_UPPER_BODY" value="$(arg add_upper_body)" />
-	<xacro:property name="END_EFFECTOR_LEFT" value="$(arg end_effector_left)" />
-	<xacro:property name="END_EFFECTOR_RIGHT" value="$(arg end_effector_right)" />
+    <xacro:property name="END_EFFECTOR_LEFT" value="$(arg end_effector_left)" />
+    <xacro:property name="END_EFFECTOR_RIGHT" value="$(arg end_effector_right)" />
     <!-- HACK to add standalone dagana plugin and ignore the dagana joint in the libxbot2_gz_joint_server -->
     <!-- This property is used in the gazebo/xbot.gazebo.xacro file -->
     <!-- In future, xbot will be able to ignore end-effectors in the hal and this should not be neccesary anymore -->
     <xacro:property name="DAGANA_STANDALONE_PLUGIN" value="true" />
+    <xacro:property name="FORCE_TORQUE_SENSORS" value="$(arg ft_sensors)" />
     <xacro:property name="ADD_FLOATING_BASE" value="$(arg add_legs)" />
     <xacro:property name="ADD_VIRTUAL_FRAME" value="true" />
