Commit message: added stick-legs

File: centauro_urdf/urdf/config/centauro.urdf.xacro (robot description, xacro)
@@ -12,3 +12,4 @@
 <xacro:property name="ADD_BALL_END_EFFECTOR" value="true" />
 <xacro:property name="ADD_FLOATING_BASE" value="$(arg add_legs)" />
+<xacro:property name="USE_STICKS" value="false" />
 </robot>

File: centauro_urdf/urdf/parts/centauro_leg.urdf.xacro (robot description, xacro)
@@ -44,4 +44,29 @@
       </collision>
 </link>
+<xacro:if value="${USE_STICKS}">
+<link name="knee_${leg_num}">
+<inertial>
+	<mass value="${1.1927236}"/>
+    <origin xyz="${1.9572282e+02*mmTom} ${-1.4549221e+01*mmTom} ${-2.0785942e+01*mmTom}" rpy="0.0 0.0 0.0"/>
+	<!--origin xyz="${1.4549221e+01*mmTom} ${-2.0785942e+01*mmTom} ${-1.9572282e+02*mmTom}" rpy="0.0 0.0 0.0"/-->
+	<!--inertia ixx="${3.5313402e+04*mm2Tom2}"  ixy="${0.0*mm2Tom2}"  ixz="${1.1029574e-01*mm2Tom2}" iyy="${3.5530025e+04*mm2Tom2}" iyz="${-6.0307457e+02*mm2Tom2}" izz="${1.3302597e+03*mm2Tom2}" /-->
+    <inertia ixx="${1.3302597e+03*mm2Tom2}"  ixy="${6.0307457e+02*mm2Tom2}"  ixz="${0.0*mm2Tom2}" iyy="${3.5313402e+04*mm2Tom2}" iyz="${-1.1029574e-01*mm2Tom2}" izz="${3.5530025e+04*mm2Tom2}" />
+</inertial>
+<visual>
+      <origin xyz="0 0 0" rpy="${PI_2} 0 ${-PI_2}"/>
+      <material name="black"/>
+      <geometry name="${leg_num}_stick_visual">
+        <mesh filename="package://centauro_urdf/meshes/front_right_stick.stl" scale="${mmTom} ${mmTom} ${mmTom}"/>
+      </geometry>
+</visual>
+<collision>
+      <origin xyz="0 0 0" rpy="${PI_2} 0 ${-PI_2}"/>
+      <geometry name="${leg_num}_stick_collision">
+        <mesh filename="package://centauro_urdf/meshes/simple/front_right_stick.stl" scale="${mmTom} ${mmTom} ${mmTom}"/>
+      </geometry>
+</collision>
+</link>
+</xacro:if>
+<xacro:unless value="${USE_STICKS}">
 <link name="knee_${leg_num}">
 	<inertial>
@@ -131,4 +156,5 @@
 	</collision>
 </link>
+</xacro:unless>
 <joint name="hip_yaw_${leg_num}" type="revolute">
 	<parent link="pelvis"/>
@@ -145,4 +171,5 @@
         <limit lower="${hip_pitch_lower[leg_num-1]}" upper="${hip_pitch_upper[leg_num-1]}" effort="${motor_A_effort}" velocity="${motor_A_velocity}"/> <!-- 200 Nm, 1 rad/s-->
 </joint>
+<xacro:if  value="${USE_STICKS}">
 <joint name="knee_pitch_${leg_num}" type="revolute">
 	<parent link="hip2_${leg_num}"/>
@@ -152,4 +179,13 @@
         <limit lower="${knee_pitch_lower[leg_num-1]}" upper="${knee_pitch_upper[leg_num-1]}" effort="${motor_A_effort}" velocity="${motor_A_velocity}"/> <!-- 200 Nm, 1 rad/s-->
 </joint>
+</xacro:if>
+<xacro:unless value="${USE_STICKS}">
+<joint name="knee_pitch_${leg_num}" type="revolute">
+	<parent link="hip2_${leg_num}"/>
+	<child link="knee_${leg_num}"/>
+	<origin xyz="${Leg_3_Ox} ${Leg_3_Oy} ${Leg_3_Oz}" rpy="${Leg_3_roll} ${Leg_3_pitch} ${Leg_3_yaw}"/>
+	<axis xyz="0 0 1"/>
+        <limit lower="${knee_pitch_lower[leg_num-1]}" upper="${knee_pitch_upper[leg_num-1]}" effort="${motor_A_effort}" velocity="${motor_A_velocity}"/> <!-- 200 Nm, 1 rad/s-->
+</joint>
 <joint name="ankle_pitch_${leg_num}" type="revolute">
 	<parent link="knee_${leg_num}"/>
@@ -173,4 +209,5 @@
         <limit  effort="${motor_C_effort}" velocity="${motor_C_velocity}"/>  <!-- 23 Nm, 1 rad/s-->
 </joint>
+</xacro:unless>
 </xacro:macro>
 <!-- /macro legs -->

Commit message: do not include D435i cam

File: centauro_urdf/urdf/config/centauro.urdf.xacro (robot description, xacro)
@@ -14,5 +14,5 @@
 <xacro:property name="USE_STICKS" value="false" />
 <xacro:property name="ADD_VELODYNE" value="true" />
-<xacro:property name="ADD_INTEL_D435I" value="true" />
+<xacro:property name="ADD_INTEL_D435I" value="false" />
 <xacro:property name="ADD_INTEL_T265" value="true" />
 </robot>

Commit message: ball hands and not rod plates currently

File: centauro_urdf/urdf/config/centauro.urdf.xacro (robot description, xacro)
@@ -10,6 +10,6 @@
 <xacro:property name="ADD_LEGS" value="$(arg add_legs)" />
 <xacro:property name="ADD_UPPER_BODY" value="$(arg add_upper_body)" />
-<xacro:property name="ADD_BALL_END_EFFECTOR" value="false" />
-<xacro:property name="ADD_ROD_PLATE_END_EFFECTOR" value="true" />
+<xacro:property name="ADD_BALL_END_EFFECTOR" value="true" />
+<xacro:property name="ADD_ROD_PLATE_END_EFFECTOR" value="false" />
 <xacro:property name="ADD_FLOATING_BASE" value="$(arg add_legs)" />
 <xacro:property name="ADD_VIRTUAL_FRAME" value="false" />

Commit message: add sensors to generated urdf

File: centauro_urdf/urdf/config/centauro.urdf.xacro (robot description, xacro)
@@ -6,6 +6,6 @@
 <xacro:arg name="legs" default="true"/>
 <xacro:arg name="upper_body" default="true"/>
-<xacro:arg name="velodyne" default="false"/>
-<xacro:arg name="realsense" default="false"/>
+<xacro:arg name="velodyne" default="true"/>
+<xacro:arg name="realsense" default="true"/>
 <xacro:arg name="floating_joint" default="true"/>
 <!-- ************SELECT PARTS*************-->

File: centauro_urdf/urdf/config/centauro_virtual_frame.urdf.xacro (robot description, xacro)
@@ -14,6 +14,6 @@
 <xacro:property name="ADD_VIRTUAL_FRAME" value="true" />
 <xacro:property name="USE_STICKS" value="false" />
-<xacro:property name="ADD_VELODYNE" value="false" />
-<xacro:property name="ADD_INTEL_D435I" value="false" />
-<xacro:property name="ADD_INTEL_T265" value="false" />
+<xacro:property name="ADD_VELODYNE" value="true" />
+<xacro:property name="ADD_INTEL_D435I" value="true" />
+<xacro:property name="ADD_INTEL_T265" value="true" />
 </robot>

Commit message: separate options for realsense cameras

File: centauro_urdf/urdf/config/centauro.urdf.xacro (robot description, xacro)
@@ -8,4 +8,14 @@
 <xacro:arg name="velodyne" default="true"/>
 <xacro:arg name="realsense" default="true"/>
+<xacro:if value="$(arg realsense)">
+	<xacro:arg name="d435i_head" default="true"/>
+	<xacro:arg name="d435i_base" default="true"/>
+	<xacro:arg name="t265_base" default="true"/>
+</xacro:if>
+<xacro:unless value="$(arg realsense)">
+	<xacro:arg name="d435i_head" default="false"/>
+	<xacro:arg name="d435i_base" default="false"/>
+	<xacro:arg name="t265_base" default="false"/>
+</xacro:unless>
 <xacro:arg name="floating_joint" default="true"/>
 <!-- ************SELECT PARTS*************-->
@@ -18,6 +28,6 @@
 <xacro:property name="USE_STICKS" value="false" />
 <xacro:property name="ADD_VELODYNE" value="$(arg velodyne)" />
-<xacro:property name="ADD_D435I_HEAD" value="$(arg realsense)" />
-<xacro:property name="ADD_D435I_BASE" value="$(arg realsense)" />
-<xacro:property name="ADD_T265_BASE" value="$(arg realsense)" />
+<xacro:property name="ADD_D435I_HEAD" value="$(arg d435i_head)" />
+<xacro:property name="ADD_D435I_BASE" value="$(arg d435i_base)" />
+<xacro:property name="ADD_T265_BASE" value="$(arg t265_base)" />
 </robot>

Commit message: handling of different end-effectors for left and right arm separately

File: centauro_urdf/urdf/config/centauro.urdf.xacro (robot description, xacro)
@@ -19,9 +19,12 @@
 </xacro:unless>
 <xacro:arg name="floating_joint" default="true"/>
+<xacro:arg name="end_effector_left" default="ball"/> <!-- none, ball, dagana_fixed, dagana -->
+<xacro:arg name="end_effector_right" default="ball"/> <!-- none, ball, dagana_fixed, dagana -->
 <!-- ************SELECT PARTS*************-->
 <!-- *************************************-->
 <xacro:property name="ADD_LEGS" value="$(arg legs)" />
 <xacro:property name="ADD_UPPER_BODY" value="$(arg upper_body)" />
-<xacro:property name="ADD_BALL_END_EFFECTOR" value="true" />
+<xacro:property name="END_EFFECTOR_LEFT" value="$(arg end_effector_left)" />
+<xacro:property name="END_EFFECTOR_RIGHT" value="$(arg end_effector_right)" />
 <xacro:property name="ADD_FLOATING_BASE" value="$(arg floating_joint)" />
 <xacro:property name="ADD_VIRTUAL_FRAME" value="false" />

File: centauro_urdf/urdf/parts/arms.urdf.xacro (robot description, xacro)
@@ -9,12 +9,39 @@
       <origin xyz="${Shoulder_1_Ox} ${-Shoulder_1_Oy} ${Shoulder_1_Oz}" rpy="${-Shoulder_1_roll} ${Shoulder_1_pitch} ${-Shoulder_1_yaw}" />
 </xacro:centauro_arm>
-<xacro:if value="${ADD_BALL_END_EFFECTOR}">
+<xacro:if value="${END_EFFECTOR_LEFT == 'ball'}">
       <xacro:include filename="$(find centauro_urdf)/urdf/parts/ball.urdf.xacro" />
       <xacro:ball_end_effector arm_num="1"  parent_link="arm1_6">
                   <origin xyz="0. -0.05 -0.105" rpy="0. 0. 0."/>
       </xacro:ball_end_effector>
+</xacro:if>
+<xacro:if value="${END_EFFECTOR_RIGHT == 'ball'}">
+      <xacro:include filename="$(find centauro_urdf)/urdf/parts/ball.urdf.xacro" />
       <xacro:ball_end_effector arm_num="2"  parent_link="arm2_6">
                   <origin xyz="0. 0.05 -0.105" rpy="0. 0. 0."/>
       </xacro:ball_end_effector>
 </xacro:if>
+<xacro:if value="${END_EFFECTOR_LEFT == 'dagana_fixed'}">
+	  <xacro:include filename="$(find dagana_urdf)/urdf/dagana_macro.urdf.xacro" />
+	  <xacro:dagana_gripper name="dagana_1" parent_link="arm1_6" joint_type="fixed">
+	    <origin xyz="0. -0.05 -0.08" rpy="0. ${PI} 0"/>
+	  </xacro:dagana_gripper>
+</xacro:if>
+<xacro:if value="${END_EFFECTOR_RIGHT == 'dagana_fixed'}">
+      <xacro:include filename="$(find dagana_urdf)/urdf/dagana_macro.urdf.xacro" />
+	  <xacro:dagana_gripper name="dagana_2" parent_link="arm2_6" joint_type="fixed">
+	    <origin xyz="0. 0.05 -0.08" rpy="0. ${PI} ${PI}"/>
+	  </xacro:dagana_gripper>
+</xacro:if>
+<xacro:if value="${END_EFFECTOR_LEFT == 'dagana'}">
+	  <xacro:include filename="$(find dagana_urdf)/urdf/dagana_macro.urdf.xacro" />
+	  <xacro:dagana_gripper name="dagana_1" parent_link="arm1_6" joint_type="revolute">
+	    <origin xyz="0. -0.05 -0.08" rpy="0. ${PI} 0"/>
+	  </xacro:dagana_gripper>
+</xacro:if>
+<xacro:if value="${END_EFFECTOR_RIGHT == 'dagana'}">
+      <xacro:include filename="$(find dagana_urdf)/urdf/dagana_macro.urdf.xacro" />
+	  <xacro:dagana_gripper name="dagana_2" parent_link="arm2_6" joint_type="revolute">
+	    <origin xyz="0. 0.05 -0.08" rpy="0. ${PI} ${PI}"/>
+	  </xacro:dagana_gripper>
+</xacro:if>
 </robot>

Commit message: optional virtual frame in main config (default is same behaviour as before)

File: centauro_urdf/urdf/config/centauro.urdf.xacro (robot description, xacro)
@@ -19,4 +19,5 @@
 </xacro:unless>
 <xacro:arg name="floating_joint" default="true"/>
+<xacro:arg name="virtual_frame" default="false"/> <!-- For cartesio model must be set to true-->
 <xacro:arg name="end_effector_left" default="ball"/> <!-- none, ball, dagana_fixed, dagana -->
 <xacro:arg name="end_effector_right" default="ball"/> <!-- none, ball, dagana_fixed, dagana -->
@@ -28,5 +29,5 @@
 <xacro:property name="END_EFFECTOR_RIGHT" value="$(arg end_effector_right)" />
 <xacro:property name="ADD_FLOATING_BASE" value="$(arg floating_joint)" />
-<xacro:property name="ADD_VIRTUAL_FRAME" value="false" />
+<xacro:property name="ADD_VIRTUAL_FRAME" value="$(arg virtual_frame)" />
 <xacro:property name="USE_STICKS" value="false" />
 <xacro:property name="ADD_VELODYNE" value="$(arg velodyne)" />

Commit message: dagana standalone plugin for gazebo and ignoring dagana in xbot_gz_server plugin

File: centauro_urdf/urdf/config/centauro.urdf.xacro (robot description, xacro)
@@ -28,4 +28,8 @@
 <xacro:property name="END_EFFECTOR_LEFT" value="$(arg end_effector_left)" />
 <xacro:property name="END_EFFECTOR_RIGHT" value="$(arg end_effector_right)" />
+<!-- HACK to add standalone dagana plugin and ignore the dagana joint in the libxbot2_gz_joint_server -->
+<!-- This property is used in the gazebo/xbot.gazebo.xacro file -->
+<!-- In future, xbot will be able to ignore end-effectors in the hal and this should not be neccesary anymore -->
+<xacro:property name="DAGANA_STANDALONE_PLUGIN" value="true" />
 <xacro:property name="ADD_FLOATING_BASE" value="$(arg floating_joint)" />
 <xacro:property name="ADD_VIRTUAL_FRAME" value="$(arg virtual_frame)" />

File: centauro_urdf/urdf/config/centauro_virtual_frame.urdf.xacro (robot description, xacro)
@@ -14,4 +14,8 @@
 	<xacro:property name="END_EFFECTOR_LEFT" value="$(arg end_effector_left)" />
 	<xacro:property name="END_EFFECTOR_RIGHT" value="$(arg end_effector_right)" />
+    <!-- HACK to add standalone dagana plugin and ignore the dagana joint in the libxbot2_gz_joint_server -->
+    <!-- This property is used in the gazebo/xbot.gazebo.xacro file -->
+    <!-- In future, xbot will be able to ignore end-effectors in the hal and this should not be neccesary anymore -->
+    <xacro:property name="DAGANA_STANDALONE_PLUGIN" value="true" />
     <xacro:property name="ADD_FLOATING_BASE" value="$(arg add_legs)" />
     <xacro:property name="ADD_VIRTUAL_FRAME" value="true" />

File: centauro_urdf/urdf/gazebo/xbot.gazebo.xacro (robot description, xacro)
@@ -10,5 +10,26 @@
     <plugin name="xbot2_ft_driver" filename="libxbot2_gz_ft_server.so"/>
     <plugin name="xbot2_imu_driver" filename="libxbot2_gz_imu_server.so"/>
+    <xacro:if value="${END_EFFECTOR_RIGHT == 'dagana'}">
+    <xacro:if value="${DAGANA_STANDALONE_PLUGIN}">
+        <plugin filename="libdagana_gazebo_DaganaPlugin.so" name="dagana_plugin">
+            <gripperName>dagana_2</gripperName>
+            <jointName>dagana_2_claw_joint</jointName>
+            <rate>100</rate>
+            <p>1</p>
+            <i>0.1</i>
+            <d>0.01</d>
+            <cmdMax>1000</cmdMax>
+            <cmdMin>-1000</cmdMin>
+        </plugin>
+    </xacro:if>
+    </xacro:if>
     <plugin name="xbot2_joint_driver" filename="libxbot2_gz_joint_server.so">
+        <xacro:if value="${END_EFFECTOR_RIGHT == 'dagana'}">
+        <xacro:if value="${DAGANA_STANDALONE_PLUGIN}">
+        <ignore_joints>
+            <joint name="dagana_2_claw_joint" />
+        </ignore_joints>
+        </xacro:if>
+        </xacro:if>
         <pid>
             <gain name="lowpwr_mot" p="50"  d="5"/>
