Commit message: integrate big wheels

File: centauro_urdf/urdf/config/centauro.urdf.xacro (robot description, xacro)
@@ -5,4 +5,5 @@
 <!-- command line arguments -->
 <xacro:arg name="legs" default="true"/>
+<xacro:arg name="big_wheel" default="true"/>
 <xacro:arg name="upper_body" default="true"/>
 <xacro:arg name="velodyne" default="true"/>
@@ -27,4 +28,5 @@
 <xacro:property name="ADD_VIRTUAL_FRAME" value="false" />
 <xacro:property name="USE_STICKS" value="false" />
+<xacro:property name="USE_WHEEL_23" value="$(arg big_wheel)" />
 <xacro:property name="ADD_VELODYNE" value="$(arg velodyne)" />
 <xacro:property name="ADD_D435I_HEAD" value="$(arg d435i_head)" />

File: centauro_urdf/urdf/parts/centauro_leg.urdf.xacro (robot description, xacro)
@@ -1,4 +1,6 @@
 <?xml version="1.0"?>
 <robot xmlns:xacro="http://ros.org/wiki/xacro">
+<xacro:include filename="$(find centauro_urdf)/urdf/parts/wheel.urdf.xacro"/>
+<xacro:include filename="$(find centauro_urdf)/urdf/parts/wheel23.urdf.xacro"/>
 <!-- macro legs -->
 <xacro:macro name="centauro_leg" params="leg_num origin_x origin_y mirror">
@@ -43,107 +45,75 @@
 </link>
 <xacro:if value="${USE_STICKS}">
-<link name="knee_${leg_num}">
-<inertial>
-	<mass value="${1.1927236}"/>
-    <origin xyz="${1.9572282e+02*mmTom} ${-1.4549221e+01*mmTom} ${-2.0785942e+01*mmTom}" rpy="0.0 0.0 0.0"/>
-	<!--origin xyz="${1.4549221e+01*mmTom} ${-2.0785942e+01*mmTom} ${-1.9572282e+02*mmTom}" rpy="0.0 0.0 0.0"/-->
-	<!--inertia ixx="${3.5313402e+04*mm2Tom2}"  ixy="${0.0*mm2Tom2}"  ixz="${1.1029574e-01*mm2Tom2}" iyy="${3.5530025e+04*mm2Tom2}" iyz="${-6.0307457e+02*mm2Tom2}" izz="${1.3302597e+03*mm2Tom2}" /-->
-    <inertia ixx="${1.3302597e+03*mm2Tom2}"  ixy="${6.0307457e+02*mm2Tom2}"  ixz="${0.0*mm2Tom2}" iyy="${3.5313402e+04*mm2Tom2}" iyz="${-1.1029574e-01*mm2Tom2}" izz="${3.5530025e+04*mm2Tom2}" />
-</inertial>
-<visual>
-      <origin xyz="0 0 0" rpy="${PI_2} 0 ${-PI_2}"/>
-      <material name="black"/>
-      <geometry name="${leg_num}_stick_visual">
-        <mesh filename="package://centauro_urdf/meshes/front_right_stick.stl" scale="${mmTom} ${mmTom} ${mmTom}"/>
-      </geometry>
-</visual>
-<collision>
-      <origin xyz="0 0 0" rpy="${PI_2} 0 ${-PI_2}"/>
-      <geometry name="${leg_num}_stick_collision">
-        <mesh filename="package://centauro_urdf/meshes/simple/front_right_stick.stl" scale="${mmTom} ${mmTom} ${mmTom}"/>
-      </geometry>
-</collision>
-</link>
+   <link name="knee_${leg_num}">
+   <inertial>
+      <mass value="${1.1927236}"/>
+      <origin xyz="${1.9572282e+02*mmTom} ${-1.4549221e+01*mmTom} ${-2.0785942e+01*mmTom}" rpy="0.0 0.0 0.0"/>
+      <!--origin xyz="${1.4549221e+01*mmTom} ${-2.0785942e+01*mmTom} ${-1.9572282e+02*mmTom}" rpy="0.0 0.0 0.0"/-->
+      <!--inertia ixx="${3.5313402e+04*mm2Tom2}"  ixy="${0.0*mm2Tom2}"  ixz="${1.1029574e-01*mm2Tom2}" iyy="${3.5530025e+04*mm2Tom2}" iyz="${-6.0307457e+02*mm2Tom2}" izz="${1.3302597e+03*mm2Tom2}" /-->
+      <inertia ixx="${1.3302597e+03*mm2Tom2}"  ixy="${6.0307457e+02*mm2Tom2}"  ixz="${0.0*mm2Tom2}" iyy="${3.5313402e+04*mm2Tom2}" iyz="${-1.1029574e-01*mm2Tom2}" izz="${3.5530025e+04*mm2Tom2}" />
+   </inertial>
+   <visual>
+         <origin xyz="0 0 0" rpy="${PI_2} 0 ${-PI_2}"/>
+         <material name="black"/>
+         <geometry name="${leg_num}_stick_visual">
+         <mesh filename="package://centauro_urdf/meshes/front_right_stick.stl" scale="${mmTom} ${mmTom} ${mmTom}"/>
+         </geometry>
+   </visual>
+   <collision>
+         <origin xyz="0 0 0" rpy="${PI_2} 0 ${-PI_2}"/>
+         <geometry name="${leg_num}_stick_collision">
+         <mesh filename="package://centauro_urdf/meshes/simple/front_right_stick.stl" scale="${mmTom} ${mmTom} ${mmTom}"/>
+         </geometry>
+   </collision>
+   </link>
 </xacro:if>
 <xacro:unless value="${USE_STICKS}">
-<link name="knee_${leg_num}">
-	<inertial>
-		<origin xyz="${Leg_3_x} ${Leg_3_y} ${mirror*Leg_3_z}"/>
-		<mass value="${Leg_3_mass}"/>  <!-- org: 3.5, foot un modeled-->
-		<inertia ixx="${Leg_3_xx}" ixy="${Leg_3_xy}" ixz="${mirror*Leg_3_xz}" iyy="${Leg_3_yy}" iyz="${mirror*Leg_3_yz}" izz="${Leg_3_zz}"/>
-	</inertial>
-   <visual>
-      <origin xyz="0.0 0.0 0.0"  rpy="0.0 0.0 0.0"/>
-      <geometry>
-         <mesh filename="package://centauro_urdf/meshes/v2/knee.stl" scale="0.001 0.001 ${mirror*0.001}" />
-      </geometry>
-      <material name="dark_grey"/>
-   </visual>
-   <collision>
-      <origin xyz="0.0 0.0 0.0"  rpy="0.0 0.0 0.0"/>
-      <geometry>
-         <mesh filename="package://centauro_urdf/meshes/v2/collision/knee.stl" scale="0.001 0.001 ${mirror*0.001}" />
-      </geometry>
-   </collision>
-</link>
-<link name="ankle1_${leg_num}">
-	<inertial>
-		<origin xyz="${Ankle_1_x} ${Ankle_1_y} ${mirror*Ankle_1_z}"/>
-		<mass value="${Ankle_1_mass}"/>  <!-- org: 3.5, foot un modeled-->
-		<inertia ixx="${Ankle_1_xx}" ixy="${Ankle_1_xy}" ixz="${mirror*Ankle_1_xz}" iyy="${Ankle_1_yy}" iyz="${mirror*Ankle_1_yz}" izz="${Ankle_1_zz}"/>
-	</inertial>
-   <visual>
-      <origin xyz="0.0 0.0 0.0"  rpy="0.0 0.0 0.0"/>
-      <geometry>
-         <mesh filename="package://centauro_urdf/meshes/v2/ankle-pitch.stl" scale="0.001 0.001 ${mirror*0.001}" />
-      </geometry>
-   </visual>
-   <collision>
-      <origin xyz="0.0 0.0 0.0"  rpy="0.0 0.0 0.0"/>
-      <geometry>
-         <mesh filename="package://centauro_urdf/meshes/v2/collision/ankle-pitch.stl" scale="0.001 0.001 ${mirror*0.001}" />
-      </geometry>
-   </collision>
-</link>
-<link name="ankle2_${leg_num}">
-	<inertial>
-		<origin xyz="${Ankle_2_x} ${mirror*Ankle_2_y} ${Ankle_2_z}"/>
-		<mass value="${Ankle_2_mass}"/>  <!-- org: 3.5, foot un modeled-->
-		<inertia ixx="${Ankle_2_xx}" ixy="${mirror*Ankle_2_xy}" ixz="${Ankle_2_xz}" iyy="${Ankle_2_yy}" iyz="${mirror*Ankle_2_yz}" izz="${Ankle_2_zz}"/>
-	</inertial>
-   <visual>
-      <origin xyz="0.0 0.0 0.0"  rpy="0.0 0.0 0.0"/>
-      <geometry>
-         <mesh filename="package://centauro_urdf/meshes/v2/ankle-yaw.stl" scale="0.001 ${mirror*0.001} 0.001" />
-      </geometry>
-      <material name="dark_grey"/>
-   </visual>
-   <collision>
-      <origin xyz="0.0 0.0 0.0"  rpy="0.0 0.0 0.0"/>
-      <geometry>
-         <mesh filename="package://centauro_urdf/meshes/v2/collision/ankle-yaw.stl" scale="0.001 ${mirror*0.001} 0.001" />
-      </geometry>
-   </collision>
-</link>
-<link name="wheel_${leg_num}">
-	<inertial>
-		<origin xyz="${Wheel_x} ${Wheel_y} ${mirror*Wheel_z}"/>
-		<mass value="${Wheel_mass}"/>
-		<inertia ixx="${Wheel_xx}" ixy="${Wheel_xy}" ixz="${mirror*Wheel_xz}" iyy="${Wheel_yy}" iyz="${mirror*Wheel_yz}" izz="${Wheel_zz}"/>
-	</inertial>
-   <visual>
-      <origin xyz="0.0 0.0 0.0"  rpy="0.0 0.0 0.0"/>
-      <geometry>
-         <mesh filename="package://centauro_urdf/meshes/v2/wheel.stl" scale="0.001 0.001 ${mirror*0.001}" />
-      </geometry>
-      <material name="black"/>
-   </visual>
-	<collision>
-		<origin xyz="0 0 0" rpy="0 0 0"/>
-		<geometry>
-			<cylinder length="0.11" radius="0.078"/>
-      </geometry>
-	</collision>
-</link>
+   <link name="knee_${leg_num}">
+      <inertial>
+         <origin xyz="${Leg_3_x} ${Leg_3_y} ${mirror*Leg_3_z}"/>
+         <mass value="${Leg_3_mass}"/>  <!-- org: 3.5, foot un modeled-->
+         <inertia ixx="${Leg_3_xx}" ixy="${Leg_3_xy}" ixz="${mirror*Leg_3_xz}" iyy="${Leg_3_yy}" iyz="${mirror*Leg_3_yz}" izz="${Leg_3_zz}"/>
+      </inertial>
+      <visual>
+         <origin xyz="0.0 0.0 0.0"  rpy="0.0 0.0 0.0"/>
+         <geometry>
+            <mesh filename="package://centauro_urdf/meshes/v2/knee.stl" scale="0.001 0.001 ${mirror*0.001}" />
+         </geometry>
+         <material name="dark_grey"/>
+      </visual>
+      <collision>
+         <origin xyz="0.0 0.0 0.0"  rpy="0.0 0.0 0.0"/>
+         <geometry>
+            <mesh filename="package://centauro_urdf/meshes/v2/collision/knee.stl" scale="0.001 0.001 ${mirror*0.001}" />
+         </geometry>
+      </collision>
+   </link>
+   <link name="ankle1_${leg_num}">
+      <inertial>
+         <origin xyz="${Ankle_1_x} ${Ankle_1_y} ${mirror*Ankle_1_z}"/>
+         <mass value="${Ankle_1_mass}"/>  <!-- org: 3.5, foot un modeled-->
+         <inertia ixx="${Ankle_1_xx}" ixy="${Ankle_1_xy}" ixz="${mirror*Ankle_1_xz}" iyy="${Ankle_1_yy}" iyz="${mirror*Ankle_1_yz}" izz="${Ankle_1_zz}"/>
+      </inertial>
+      <visual>
+         <origin xyz="0.0 0.0 0.0"  rpy="0.0 0.0 0.0"/>
+         <geometry>
+            <mesh filename="package://centauro_urdf/meshes/v2/ankle-pitch.stl" scale="0.001 0.001 ${mirror*0.001}" />
+         </geometry>
+      </visual>
+      <collision>
+         <origin xyz="0.0 0.0 0.0"  rpy="0.0 0.0 0.0"/>
+         <geometry>
+            <mesh filename="package://centauro_urdf/meshes/v2/collision/ankle-pitch.stl" scale="0.001 0.001 ${mirror*0.001}" />
+         </geometry>
+      </collision>
+   </link>
+   <!-- New centauro wheel -->
+   <xacro:if value="${USE_WHEEL_23}">
+      <xacro:centauro_wheel23 leg_num="${leg_num}" mirror="${mirror}"/>
+   </xacro:if>
+   <!-- Old centauro wheel -->
+   <xacro:unless value="${USE_WHEEL_23}">
+      <xacro:centauro_wheel leg_num="${leg_num}" mirror="${mirror}"/>
+   </xacro:unless>
 </xacro:unless>
 <!-- *****************************-->
@@ -170,41 +140,34 @@
 </joint>
 <xacro:if  value="${USE_STICKS}">
-<joint name="knee_pitch_${leg_num}" type="revolute">
-	<parent link="hip2_${leg_num}"/>
-	<child link="knee_${leg_num}"/>
-	<origin xyz="${Leg_3_Ox} ${Leg_3_Oy} ${Leg_3_Oz}" rpy="${Leg_3_roll} ${Leg_3_pitch} ${Leg_3_yaw}"/>
-	<axis xyz="0 0 1"/>
-   <limit lower="${knee_pitch_lower[leg_num-1]}" upper="${knee_pitch_upper[leg_num-1]}" effort="${motor_A_effort}" velocity="${motor_A_velocity}"/> <!-- 200 Nm, 1 rad/s-->
-</joint>
+   <joint name="knee_pitch_${leg_num}" type="revolute">
+      <parent link="hip2_${leg_num}"/>
+      <child link="knee_${leg_num}"/>
+      <origin xyz="${Leg_3_Ox} ${Leg_3_Oy} ${Leg_3_Oz}" rpy="${Leg_3_roll} ${Leg_3_pitch} ${Leg_3_yaw}"/>
+      <axis xyz="0 0 1"/>
+      <limit lower="${knee_pitch_lower[leg_num-1]}" upper="${knee_pitch_upper[leg_num-1]}" effort="${motor_A_effort}" velocity="${motor_A_velocity}"/> <!-- 200 Nm, 1 rad/s-->
+   </joint>
 </xacro:if>
 <xacro:unless value="${USE_STICKS}">
-<joint name="knee_pitch_${leg_num}" type="revolute">
-	<parent link="hip2_${leg_num}"/>
-	<child link="knee_${leg_num}"/>
-	<origin xyz="${Leg_3_Ox} ${Leg_3_Oy} ${mirror*Leg_3_Oz}" rpy="${Leg_3_roll} ${Leg_3_pitch} ${Leg_3_yaw}"/>
-	<axis xyz="0 0 ${mirror}"/>
-   <limit lower="${knee_pitch_lower[leg_num-1]}" upper="${knee_pitch_upper[leg_num-1]}" effort="${motor_A_effort}" velocity="${motor_A_velocity}"/> <!-- 200 Nm, 1 rad/s-->
-</joint>
-<joint name="ankle_pitch_${leg_num}" type="revolute">
-	<parent link="knee_${leg_num}"/>
-	<child link="ankle1_${leg_num}"/>
-	<origin xyz="${Ankle_1_Ox} ${Ankle_1_Oy} ${mirror*Ankle_1_Oz}" rpy="${Ankle_1_roll} ${Ankle_1_pitch} ${Ankle_1_yaw}"/>
-	<axis xyz="0 0 ${mirror}"/>
-   <limit lower="${ankle_pitch_lower[leg_num-1]}" upper="${ankle_pitch_upper[leg_num-1]}" effort="${motor_B_effort}" velocity="${motor_B_velocity}"/> <!-- 98 Nm, 1 rad/s-->
-</joint>
-<joint name="ankle_yaw_${leg_num}" type="revolute">
-	<parent link="ankle1_${leg_num}"/>
-	<child link="ankle2_${leg_num}"/>
-	<origin xyz="${Ankle_2_Ox} ${Ankle_2_Oy} ${mirror*Ankle_2_Oz}" rpy="${Ankle_2_roll} ${Ankle_2_pitch} ${Ankle_2_yaw}"/>
-	<axis xyz="0 0 -1"/>
-   <limit lower="${ankle_yaw_lower[leg_num-1]}" upper="${ankle_yaw_upper[leg_num-1]}" effort="${motor_C_effort}" velocity="${motor_C_velocity}"/>  <!-- 23 Nm, 1 rad/s-->
-</joint>
-<joint name="j_wheel_${leg_num}" type="continuous">
-	<parent link="ankle2_${leg_num}"/>
-	<child link="wheel_${leg_num}"/>
-	<origin xyz="${Wheel_Ox} ${mirror*Wheel_Oy} ${Wheel_Oz}" rpy="${Wheel_roll} ${Wheel_pitch} ${Wheel_yaw}"/>
-	<axis xyz="0 0 ${mirror}"/>
-   <limit  effort="${motor_C_effort}" velocity="${motor_C_velocity}"/>  <!-- 23 Nm, 1 rad/s-->
-</joint>
+   <joint name="knee_pitch_${leg_num}" type="revolute">
+      <parent link="hip2_${leg_num}"/>
+      <child link="knee_${leg_num}"/>
+      <origin xyz="${Leg_3_Ox} ${Leg_3_Oy} ${mirror*Leg_3_Oz}" rpy="${Leg_3_roll} ${Leg_3_pitch} ${Leg_3_yaw}"/>
+      <axis xyz="0 0 ${mirror}"/>
+      <limit lower="${knee_pitch_lower[leg_num-1]}" upper="${knee_pitch_upper[leg_num-1]}" effort="${motor_A_effort}" velocity="${motor_A_velocity}"/> <!-- 200 Nm, 1 rad/s-->
+   </joint>
+   <joint name="ankle_pitch_${leg_num}" type="revolute">
+      <parent link="knee_${leg_num}"/>
+      <child link="ankle1_${leg_num}"/>
+      <origin xyz="${Ankle_1_Ox} ${Ankle_1_Oy} ${mirror*Ankle_1_Oz}" rpy="${Ankle_1_roll} ${Ankle_1_pitch} ${Ankle_1_yaw}"/>
+      <axis xyz="0 0 ${mirror}"/>
+      <limit lower="${ankle_pitch_lower[leg_num-1]}" upper="${ankle_pitch_upper[leg_num-1]}" effort="${motor_B_effort}" velocity="${motor_B_velocity}"/> <!-- 98 Nm, 1 rad/s-->
+   </joint>
+   <joint name="ankle_yaw_${leg_num}" type="revolute">
+      <parent link="ankle1_${leg_num}"/>
+      <child link="ankle2_${leg_num}"/>
+      <origin xyz="${Ankle_2_Ox} ${Ankle_2_Oy} ${mirror*Ankle_2_Oz}" rpy="${Ankle_2_roll} ${Ankle_2_pitch} ${Ankle_2_yaw}"/>
+      <axis xyz="0 0 -1"/>
+      <limit lower="${ankle_yaw_lower[leg_num-1]}" upper="${ankle_yaw_upper[leg_num-1]}" effort="${motor_C_effort}" velocity="${motor_C_velocity}"/>  <!-- 23 Nm, 1 rad/s-->
+   </joint>
 </xacro:unless>
 </xacro:macro>

File: centauro_urdf/urdf/parts/inertial_properties.urdf.xacro (robot description, xacro)
@@ -88,4 +88,18 @@
 <!-- Mass -->
 <xacro:property name="Ankle_2_mass" value="1.7656714e+00"/>
+<!-- Note: the "23" suffix denotes the new bigger-size wheel -->
+<!-- Center of Mass -->
+<xacro:property name="Ankle23_2_x" value="${1.8512273e-01 * mmTom}"/>
+<xacro:property name="Ankle23_2_y" value="${-1.7369405e+00 * mmTom}"/>
+<xacro:property name="Ankle23_2_z" value="${-9.1340683e+01 * mmTom}"/>
+<!-- Inertia -->
+<xacro:property name="Ankle23_2_xx" value="${1.7711499e+04 * mm2Tom2}"/>
+<xacro:property name="Ankle23_2_yy" value="${1.4263485e+04 * mm2Tom2}"/>
+<xacro:property name="Ankle23_2_zz" value="${8.0747557e+03 * mm2Tom2}"/>
+<xacro:property name="Ankle23_2_xy" value="${-1.0713141e+01 * mm2Tom2}"/>
+<xacro:property name="Ankle23_2_xz" value="${-2.2094697e+01 * mm2Tom2}"/>
+<xacro:property name="Ankle23_2_yz" value="${-3.3426702e+02 * mm2Tom2}"/>
+<!-- Mass -->
+<xacro:property name="Ankle23_2_mass" value="2.4409290e+00"/>
 <!-- Center of Mass -->
 <xacro:property name="Wheel_x" value="${0.0 * mmTom}"/>
@@ -100,5 +114,18 @@
 <xacro:property name="Wheel_yz" value="${0.0 * mm2Tom2}"/>
 <!-- Mass -->
-<xacro:property name="Wheel_mass" value="1.1116400e+00"/>  <!-- TODO CHECK THIS VALUE -->
+<xacro:property name="Wheel_mass" value="1.1116400e+00"/>
+<!-- Center of Mass -->
+<xacro:property name="Wheel23_x" value="${0.0 * mmTom}"/>
+<xacro:property name="Wheel23_y" value="${0.0 * mmTom}"/>
+<xacro:property name="Wheel23_z" value="${-1.5403767e-01 * mmTom}"/>
+<!-- Inertia -->
+<xacro:property name="Wheel23_xx" value="${8.6373591e+03 * mm2Tom2}"/>
+<xacro:property name="Wheel23_yy" value="${8.6373644e+03 * mm2Tom2}"/>
+<xacro:property name="Wheel23_zz" value="${1.6376551e+04 * mm2Tom2}"/>
+<xacro:property name="Wheel23_xy" value="${0.0 * mm2Tom2}"/>
+<xacro:property name="Wheel23_xz" value="${0.0 * mm2Tom2}"/>
+<xacro:property name="Wheel23_yz" value="${0.0 * mm2Tom2}"/>
+<!-- Mass -->
+<xacro:property name="Wheel23_mass" value="1.8569388e+00"/>
 <!-- Center of Mass -->
 <xacro:property name="Torso_2_x" value=" -0.0194977940 "/>

File: centauro_urdf/urdf/parts/kinematics_properties.urdf.xacro (robot description, xacro)
@@ -66,4 +66,10 @@
 <xacro:property name="Wheel_pitch" value="0.0"/>
 <xacro:property name="Wheel_yaw" value="0.0"/>
+<xacro:property name="Wheel23_Ox" value="${0.0 * mmTom}"/>
+<xacro:property name="Wheel23_Oy" value="${0.0 * mmTom}"/>
+<xacro:property name="Wheel23_Oz" value="${-144.350 * mmTom}"/>
+<xacro:property name="Wheel23_roll" value="${PI_2}"/>
+<xacro:property name="Wheel23_pitch" value="0.0"/>
+<xacro:property name="Wheel23_yaw" value="0.0"/>
 <!-- Origin -->
 <xacro:property name="Torso_2_Ox" value=" 0.200 "/>

Commit message: rm useless flag for dagana old standalone plugin

File: centauro_urdf/urdf/config/centauro.urdf.xacro (robot description, xacro)
@@ -31,8 +31,4 @@
 <xacro:property name="END_EFFECTOR_LEFT" value="$(arg end_effector_left)" />
 <xacro:property name="END_EFFECTOR_RIGHT" value="$(arg end_effector_right)" />
-<!-- HACK to add standalone dagana plugin and ignore the dagana joint in the libxbot2_gz_joint_server -->
-<!-- This property is used in the gazebo/xbot.gazebo.xacro file -->
-<!-- In future, xbot will be able to ignore end-effectors in the hal and this should not be neccesary anymore -->
-<xacro:property name="DAGANA_STANDALONE_PLUGIN" value="true" />
 <xacro:property name="ADD_FLOATING_BASE" value="$(arg floating_joint)" />
 <xacro:property name="ADD_VIRTUAL_FRAME" value="$(arg virtual_frame)" />

Commit message: fixed duplicate param name

File: centauro_urdf/urdf/config/centauro.urdf.xacro (robot description, xacro)
@@ -3,4 +3,6 @@
 <xacro:property name="model_name" value="centauro" />
 <xacro:property name="model_version" value="0.1" />
+<xacro:property name="wheel23_radius" value="0.124"/>
+<xacro:property name="wheel23_depth" value="0.03"/>
 <!-- command line arguments -->
 <xacro:arg name="legs" default="true"/>

File: centauro_urdf/urdf/parts/wheel23.urdf.xacro (robot description, xacro)
@@ -54,7 +54,10 @@
                 <origin xyz="0 0 0" rpy="0 0 0" />
                 <geometry>
+					<cylinder radius="${wheel23_radius}" length="${wheel23_depth}"/>
+				</geometry>
+                <!-- <geometry>
                     <mesh filename="${MESH_PATH}/v2/collision/mesh_wheel23.stl"
                         scale="0.001 0.001 ${mirror*0.001}" />
-                </geometry>
+                </geometry> -->
                 <material name="black" />
             </collision>

Commit message: optional wheel sphere collision

File: centauro_urdf/urdf/config/centauro.urdf.xacro (robot description, xacro)
@@ -6,4 +6,5 @@
 <xacro:arg name="legs" default="true"/>
 <xacro:arg name="big_wheel" default="true"/>
+<xacro:arg name="sphere_wheel_collision" default="false"/>
 <xacro:arg name="upper_body" default="true"/>
 <xacro:arg name="velodyne" default="true"/>
@@ -39,4 +40,5 @@
 <xacro:property name="USE_STICKS" value="false" />
 <xacro:property name="USE_WHEEL_23" value="$(arg big_wheel)" />
+<xacro:property name="USE_WHEEL_23_SPHERE_COLLISION" value="$(arg sphere_wheel_collision)" />
 <xacro:property name="ADD_VELODYNE" value="$(arg velodyne)" />
 <xacro:property name="ADD_D435I_HEAD" value="$(arg d435i_head)" />

File: centauro_urdf/urdf/parts/wheel23.urdf.xacro (robot description, xacro)
@@ -54,7 +54,11 @@
                 <origin xyz="0 0 0" rpy="0 0 0" />
                 <geometry>
+                <xacro:if value="${USE_WHEEL_23_SPHERE_COLLISION}">
                     <sphere radius="0.125"/>
-                    <!-- <mesh filename="package://centauro_urdf/meshes/v2/collision/mesh_wheel23.stl"
-                        scale="0.001 0.001 ${mirror*0.001}" /> -->
+                </xacro:if>
+                <xacro:unless value="${USE_WHEEL_23_SPHERE_COLLISION}">
+                    <mesh filename="package://centauro_urdf/meshes/v2/collision/mesh_wheel23.stl"
+                        scale="0.001 0.001 ${mirror*0.001}" />
+                </xacro:unless>
                 </geometry>
                 <material name="black" />

Commit message: dagana standalone plugin not necessary anymore since a while

File: centauro_urdf/urdf/config/centauro.urdf.xacro (robot description, xacro)
@@ -33,8 +33,4 @@
 <xacro:property name="END_EFFECTOR_LEFT" value="$(arg end_effector_left)" />
 <xacro:property name="END_EFFECTOR_RIGHT" value="$(arg end_effector_right)" />
-<!-- HACK to add standalone dagana plugin and ignore the dagana joint in the libxbot2_gz_joint_server -->
-<!-- This property is used in the gazebo/xbot.gazebo.xacro file -->
-<!-- In future, xbot will be able to ignore end-effectors in the hal and this should not be neccesary anymore -->
-<xacro:property name="DAGANA_STANDALONE_PLUGIN" value="true" />
 <xacro:property name="ADD_FLOATING_BASE" value="$(arg floating_joint)" />
 <xacro:property name="ADD_VIRTUAL_FRAME" value="$(arg virtual_frame)" />
