Commit message: optional resolution for gazebo d435 head camera

File: centauro_urdf/urdf/config/centauro.urdf.xacro (robot description, xacro)
@@ -22,4 +22,11 @@
 	<xacro:arg name="t265_base" default="false"/>
 </xacro:unless>
+<xacro:arg name="d435i_head_color_width" default="1280"/>
+<xacro:arg name="d435i_head_color_height" default="720"/>
+<xacro:arg name="d435i_head_color_fps" default="30"/>
+<xacro:arg name="d435i_head_depth_width" default="1280"/>
+<xacro:arg name="d435i_head_depth_height" default="720"/>
+<xacro:arg name="d435i_head_depth_fps" default="90"/>
+<xacro:arg name="d435i_head_enable_pointcloud" default="true"/>
 <xacro:arg name="floating_joint" default="true"/>
 <xacro:arg name="virtual_frame" default="false"/> <!-- For cartesio model must be set to true-->
@@ -39,4 +46,11 @@
 <xacro:property name="ADD_VELODYNE" value="$(arg velodyne)" />
 <xacro:property name="ADD_D435I_HEAD" value="$(arg d435i_head)" />
+<xacro:property name="D435I_HEAD_COLOR_WIDTH" value="$(arg d435i_head_color_width)" />
+<xacro:property name="D435I_HEAD_COLOR_HEIGHT" value="$(arg d435i_head_color_height)" />
+<xacro:property name="D435I_HEAD_COLOR_FPS" value="$(arg d435i_head_color_height)" />
+<xacro:property name="D435I_HEAD_DEPTH_WIDTH" value="$(arg d435i_head_depth_width)" />
+<xacro:property name="D435I_HEAD_DEPTH_HEIGHT" value="$(arg d435i_head_depth_height)" />
+<xacro:property name="D435I_HEAD_DEPTH_FPS" value="$(arg d435i_head_depth_height)" />
+<xacro:property name="D435I_HEAD_ENABLE_POINTCLOUD" value="$(arg d435i_head_enable_pointcloud)" />
 <xacro:property name="ADD_D435I_BASE" value="$(arg d435i_base)" />
 <xacro:property name="ADD_T265_BASE" value="$(arg t265_base)" />

File: centauro_urdf/urdf/config/centauro_virtual_frame.urdf.xacro (robot description, xacro)
@@ -18,3 +18,10 @@
     <xacro:property name="ADD_D435I_BASE" value="false" />
     <xacro:property name="ADD_T265_BASE" value="false" />
+    <xacro:property name="D435I_HEAD_COLOR_WIDTH" value="1280" />
+    <xacro:property name="D435I_HEAD_COLOR_HEIGHT" value="720"/>
+    <xacro:property name="D435I_HEAD_COLOR_FPS" value="30" />
+    <xacro:property name="D435I_HEAD_DEPTH_WIDTH" value="1280" />
+    <xacro:property name="D435I_HEAD_DEPTH_HEIGHT" value="720" />
+    <xacro:property name="D435I_HEAD_DEPTH_FPS" value="90" />
+    <xacro:property name="D435I_HEAD_ENABLE_POINTCLOUD" value="true" />
 </robot>

File: centauro_urdf/urdf/parts/head.urdf.xacro (robot description, xacro)
@@ -95,5 +95,5 @@
         name="${d435_head_name}"
         topics_ns="${d435_head_name}"
-        enable_pointCloud="true"
+        enable_pointCloud="${D435I_HEAD_ENABLE_POINTCLOUD}"
         align_depth="true"
         unite_imu_method="false"
@@ -101,13 +101,13 @@
         accel_fps="300"
         gyro_fps="300"
-        depth_width="1280"
-        depth_height="720"
-        depth_fps="90"
+        depth_width="${D435I_HEAD_DEPTH_WIDTH}"
+        depth_height="${D435I_HEAD_DEPTH_HEIGHT}"
+        depth_fps="${D435I_HEAD_DEPTH_FPS}"
         infra_width="1280"
         infra_height="720"
         infra_fps="90"
-        color_width="1280"
-        color_height="720"
-        color_fps="30">
+        color_width="${D435I_HEAD_COLOR_WIDTH}"
+        color_height="${D435I_HEAD_COLOR_HEIGHT}"
+        color_fps="${D435I_HEAD_COLOR_FPS}">
         <xacro:insert_block name="d435_head_origin" />
     </xacro:sensor_d435i>

Commit message: optional resolution for gazebo d435 head camera

File: centauro_urdf/urdf/config/centauro.urdf.xacro (robot description, xacro)
@@ -21,4 +21,11 @@
 	<xacro:arg name="t265_base" default="false"/>
 </xacro:unless>
+<xacro:arg name="d435i_head_color_width" default="1280"/>
+<xacro:arg name="d435i_head_color_height" default="720"/>
+<xacro:arg name="d435i_head_color_fps" default="30"/>
+<xacro:arg name="d435i_head_depth_width" default="1280"/>
+<xacro:arg name="d435i_head_depth_height" default="720"/>
+<xacro:arg name="d435i_head_depth_fps" default="90"/>
+<xacro:arg name="d435i_head_enable_pointcloud" default="true"/>
 <xacro:arg name="floating_joint" default="true"/>
 <xacro:arg name="virtual_frame" default="false"/> <!-- For cartesio model must be set to true-->
@@ -37,4 +44,11 @@
 <xacro:property name="ADD_VELODYNE" value="$(arg velodyne)" />
 <xacro:property name="ADD_D435I_HEAD" value="$(arg d435i_head)" />
+<xacro:property name="D435I_HEAD_COLOR_WIDTH" value="$(arg d435i_head_color_width)" />
+<xacro:property name="D435I_HEAD_COLOR_HEIGHT" value="$(arg d435i_head_color_height)" />
+<xacro:property name="D435I_HEAD_COLOR_FPS" value="$(arg d435i_head_color_height)" />
+<xacro:property name="D435I_HEAD_DEPTH_WIDTH" value="$(arg d435i_head_depth_width)" />
+<xacro:property name="D435I_HEAD_DEPTH_HEIGHT" value="$(arg d435i_head_depth_height)" />
+<xacro:property name="D435I_HEAD_DEPTH_FPS" value="$(arg d435i_head_depth_height)" />
+<xacro:property name="D435I_HEAD_ENABLE_POINTCLOUD" value="$(arg d435i_head_enable_pointcloud)" />
 <xacro:property name="ADD_D435I_BASE" value="$(arg d435i_base)" />
 <xacro:property name="ADD_T265_BASE" value="$(arg t265_base)" />

File: centauro_urdf/urdf/parts/head.urdf.xacro (robot description, xacro)
@@ -94,5 +94,20 @@
     <xacro:sensor_d435i parent="${d435_head_parent_name}"
         name="${d435_head_name}"
-        use_nominal_extrinsics="true">
+        topics_ns="${d435_head_name}"
+        enable_pointCloud="${D435I_HEAD_ENABLE_POINTCLOUD}"
+        align_depth="true"
+        unite_imu_method="false"
+        visualize="false"
+        accel_fps="300"
+        gyro_fps="300"
+        depth_width="${D435I_HEAD_DEPTH_WIDTH}"
+        depth_height="${D435I_HEAD_DEPTH_HEIGHT}"
+        depth_fps="${D435I_HEAD_DEPTH_FPS}"
+        infra_width="1280"
+        infra_height="720"
+        infra_fps="90"
+        color_width="${D435I_HEAD_COLOR_WIDTH}"
+        color_height="${D435I_HEAD_COLOR_HEIGHT}"
+        color_fps="${D435I_HEAD_COLOR_FPS}">
         <xacro:insert_block name="d435_head_origin" />
     </xacro:sensor_d435i>

Commit message: added small sphere contacts

File: centauro_urdf/urdf/config/centauro.urdf.xacro (robot description, xacro)
@@ -7,4 +7,5 @@
 <xacro:arg name="big_wheel" default="true"/>
 <xacro:arg name="sphere_wheel_collision" default="false"/>
+<xacro:arg name="small_sphere_wheel_collision" default="false"/>
 <xacro:arg name="upper_body" default="true"/>
 <xacro:arg name="velodyne" default="true"/>
@@ -43,4 +44,5 @@
 <xacro:property name="USE_WHEEL_23" value="$(arg big_wheel)" />
 <xacro:property name="USE_WHEEL_23_SPHERE_COLLISION" value="$(arg sphere_wheel_collision)" />
+<xacro:property name="USE_WHEEL_23_SMALL_SPHERE_COLLISION" value="$(arg small_sphere_wheel_collision)" />
 <xacro:property name="ADD_VELODYNE" value="$(arg velodyne)" />
 <xacro:property name="ADD_D435I_HEAD" value="$(arg d435i_head)" />

File: centauro_urdf/urdf/parts/wheel23.urdf.xacro (robot description, xacro)
@@ -52,14 +52,23 @@
             </visual>
             <collision>
-                <origin xyz="0 0 0" rpy="0 0 0" />
-                <geometry>
                 <xacro:if value="${USE_WHEEL_23_SPHERE_COLLISION}">
-                    <sphere radius="0.125"/>
+                    <origin xyz="0 0 0" rpy="0 0 0" />
+                    <geometry>
+                        <sphere radius="0.125"/>
+                    </geometry>
                 </xacro:if>
-                <xacro:unless value="${USE_WHEEL_23_SPHERE_COLLISION}">
-                    <mesh filename="package://centauro_urdf/meshes/v2/collision/mesh_wheel23.stl"
-                        scale="0.001 0.001 ${mirror*0.001}" />
+                <xacro:if value="${USE_WHEEL_23_SMALL_SPHERE_COLLISION}">
+                    <origin xyz="0 ${-(0.125-0.015)} 0" rpy="0 0 0" />
+                    <geometry>
+                        <sphere radius="0.015" />
+                    </geometry>
+                </xacro:if>
+                <xacro:unless value="${USE_WHEEL_23_SMALL_SPHERE_COLLISION or USE_WHEEL_23_SPHERE_COLLISION}">
+                    <origin xyz="0 0 0" rpy="0 0 0" />
+                    <geometry>
+                        <mesh   filename="package://centauro_urdf/meshes/v2/collision/mesh_wheel23.stl"
+                                scale="0.001 0.001 ${mirror*0.001}" />
+                    </geometry>
                 </xacro:unless>
-                </geometry>
                 <material name="black" />
             </collision>

Commit message: optional configs for head camera instrinsic

File: centauro_urdf/urdf/config/centauro.urdf.xacro (robot description, xacro)
@@ -25,7 +25,17 @@
 <xacro:arg name="d435i_head_color_height" default="720"/>
 <xacro:arg name="d435i_head_color_fps" default="30"/>
+<xacro:arg name="d435i_head_color_fx" default="909.7210083007812"/>
+<xacro:arg name="d435i_head_color_fy" default="909.655029296875"/>
+<xacro:arg name="d435i_head_color_cx" default="649.3759155273438"/>
+<xacro:arg name="d435i_head_color_cy" default="381.8260498046875"/>
 <xacro:arg name="d435i_head_depth_width" default="1280"/>
 <xacro:arg name="d435i_head_depth_height" default="720"/>
-<xacro:arg name="d435i_head_depth_fps" default="90"/>
+<xacro:arg name="d435i_head_depth_fps" default="30"/>
+<xacro:arg name="d435i_head_depth_fx" default="650.98046875"/>
+<xacro:arg name="d435i_head_depth_fy" default="650.98046875"/>
+<xacro:arg name="d435i_head_depth_cx" default="639.7286987304688"/>
+<xacro:arg name="d435i_head_depth_cy" default="361.9244384765625"/>
+<xacro:arg name="d435i_head_clip_distance" default="10"/>
+<xacro:arg name="d435i_head_clip_distance_min" default="0.280"/>
 <xacro:arg name="d435i_head_enable_pointcloud" default="true"/>
 <xacro:arg name="floating_joint" default="true"/>
@@ -48,8 +58,18 @@
 <xacro:property name="D435I_HEAD_COLOR_WIDTH" value="$(arg d435i_head_color_width)" />
 <xacro:property name="D435I_HEAD_COLOR_HEIGHT" value="$(arg d435i_head_color_height)" />
-<xacro:property name="D435I_HEAD_COLOR_FPS" value="$(arg d435i_head_color_height)" />
+<xacro:property name="D435I_HEAD_COLOR_FPS" value="$(arg d435i_head_color_fps)" />
+<xacro:property name="D435I_HEAD_COLOR_FX" value="$(arg d435i_head_color_fx)" />
+<xacro:property name="D435I_HEAD_COLOR_FY" value="$(arg d435i_head_color_fy)" />
+<xacro:property name="D435I_HEAD_COLOR_CX" value="$(arg d435i_head_color_cx)" />
+<xacro:property name="D435I_HEAD_COLOR_CY" value="$(arg d435i_head_color_cy)" />
 <xacro:property name="D435I_HEAD_DEPTH_WIDTH" value="$(arg d435i_head_depth_width)" />
 <xacro:property name="D435I_HEAD_DEPTH_HEIGHT" value="$(arg d435i_head_depth_height)" />
-<xacro:property name="D435I_HEAD_DEPTH_FPS" value="$(arg d435i_head_depth_height)" />
+<xacro:property name="D435I_HEAD_DEPTH_FPS" value="$(arg d435i_head_depth_fps)" />
+<xacro:property name="D435I_HEAD_DEPTH_FX" value="$(arg d435i_head_depth_fx)" />
+<xacro:property name="D435I_HEAD_DEPTH_FY" value="$(arg d435i_head_depth_fy)" />
+<xacro:property name="D435I_HEAD_DEPTH_CX" value="$(arg d435i_head_depth_cx)" />
+<xacro:property name="D435I_HEAD_DEPTH_CY" value="$(arg d435i_head_depth_cy)" />
+<xacro:property name="D435I_HEAD_CLIP_DISTANCE" value="$(arg d435i_head_clip_distance)" />
+<xacro:property name="D435I_HEAD_CLIP_DISTANCE_MIN" value="$(arg d435i_head_clip_distance_min)" />
 <xacro:property name="D435I_HEAD_ENABLE_POINTCLOUD" value="$(arg d435i_head_enable_pointcloud)" />
 <xacro:property name="ADD_D435I_BASE" value="$(arg d435i_base)" />

File: centauro_urdf/urdf/parts/head.urdf.xacro (robot description, xacro)
@@ -104,4 +104,10 @@
         depth_height="${D435I_HEAD_DEPTH_HEIGHT}"
         depth_fps="${D435I_HEAD_DEPTH_FPS}"
+        depth_fx="${D435I_HEAD_DEPTH_FX}"
+        depth_fy="${D435I_HEAD_DEPTH_FY}"
+        depth_cx="${D435I_HEAD_DEPTH_CX}"
+        depth_cy="${D435I_HEAD_DEPTH_CY}"
+        clip_distance="${D435I_HEAD_CLIP_DISTANCE}"
+        clip_distance_min="${D435I_HEAD_CLIP_DISTANCE_MIN}"
         infra_width="1280"
         infra_height="720"
@@ -109,5 +115,10 @@
         color_width="${D435I_HEAD_COLOR_WIDTH}"
         color_height="${D435I_HEAD_COLOR_HEIGHT}"
-        color_fps="${D435I_HEAD_COLOR_FPS}">
+        color_fps="${D435I_HEAD_COLOR_FPS}"
+        color_fx="${D435I_HEAD_COLOR_FX}"
+        color_fy="${D435I_HEAD_COLOR_FY}"
+        color_cx="${D435I_HEAD_COLOR_CX}"
+        color_cy="${D435I_HEAD_COLOR_CY}"
+        >
         <xacro:insert_block name="d435_head_origin" />
     </xacro:sensor_d435i>

Commit message: Update lighting and collision properties in URDF and XML configurations, changed bigsphere/ellipsoid arg

File: centauro_urdf/urdf/config/centauro.urdf.xacro (robot description, xacro)
@@ -6,5 +6,5 @@
 <xacro:arg name="legs" default="true"/>
 <xacro:arg name="big_wheel" default="true"/>
-<xacro:arg name="sphere_wheel_collision" default="false"/>
+<xacro:arg name="sphere_or_ellipsoid_wheel_collision" default="false"/>
 <xacro:arg name="small_sphere_wheel_collision" default="false"/>
 <xacro:arg name="upper_body" default="true"/>
@@ -46,5 +46,5 @@
 <xacro:property name="USE_STICKS" value="false" />
 <xacro:property name="USE_WHEEL_23" value="$(arg big_wheel)" />
-<xacro:property name="USE_WHEEL_23_SPHERE_COLLISION" value="$(arg sphere_wheel_collision)" />
+<xacro:property name="USE_WHEEL_23_SPHERE_OR_ELLIPSOID_COLLISION" value="$(arg sphere_or_ellipsoid_wheel_collision)" />
 <xacro:property name="USE_WHEEL_23_SMALL_SPHERE_COLLISION" value="$(arg small_sphere_wheel_collision)" />
 <xacro:property name="ADD_VELODYNE" value="$(arg velodyne)" />

File: centauro_urdf/urdf/parts/wheel23.urdf.xacro (robot description, xacro)
@@ -51,9 +51,9 @@
                 <material name="black" />
             </visual>
-            <xacro:if value="${USE_WHEEL_23_SPHERE_COLLISION}">
+            <xacro:if value="${USE_WHEEL_23_SPHERE_OR_ELLIPSOID_COLLISION}">
                 <collision>
                     <origin xyz="0 0 0" rpy="0 0 0" />
                     <geometry>
-                        <sphere radius="0.125"/>
+                        <sphere radius="0.12"/>
                     </geometry>
                     <adarl>
@@ -67,5 +67,5 @@
                 </collision>
             </xacro:if>
-            <xacro:unless value="${USE_WHEEL_23_SMALL_SPHERE_COLLISION or USE_WHEEL_23_SPHERE_COLLISION}">
+            <xacro:unless value="${USE_WHEEL_23_SMALL_SPHERE_COLLISION or USE_WHEEL_23_SPHERE_OR_ELLIPSOID_COLLISION}">
                 <collision>
                     <origin xyz="0 0 0" rpy="0 0 0" />
