Commit message: added homing

File: centauro_srdf/srdf/centauro.srdf.xacro (robot description, xacro)
@@ -47,4 +47,44 @@
 </xacro:if>
 </group>
+<!-- Homing posture -->
+<group_state name="home" group="chains">
+	<joint name="hip_yaw_1" value="-0.746874"/>
+	<joint name="hip_pitch_1" value="-1.25409"/>
+	<joint name="knee_pitch_1" value="-1.55576"/>
+	<joint name="ankle_pitch_1" value="-0.301666"/>
+	<joint name="ankle_yaw_1" value="0.746874"/>
+	<joint name="hip_yaw_2" value="0.746874"/>
+	<joint name="hip_pitch_2" value="1.25409"/>
+	<joint name="knee_pitch_2" value="1.55576"/>
+	<joint name="ankle_pitch_2" value="0.301666"/>
+	<joint name="ankle_yaw_2" value="-0.746874"/>
+	<joint name="hip_yaw_3" value="0.746874"/>
+	<joint name="hip_pitch_3" value="1.25409"/>
+	<joint name="knee_pitch_3" value="1.55576"/>
+	<joint name="ankle_pitch_3" value="0.301667"/>
+	<joint name="ankle_yaw_3" value="-0.746874"/>
+	<joint name="hip_yaw_4" value="-0.746874"/>
+	<joint name="hip_pitch_4" value="-1.25409"/>
+	<joint name="knee_pitch_4" value="-1.55576"/>
+	<joint name="ankle_pitch_4" value="-0.301667"/>
+	<joint name="ankle_yaw_4" value="0.746874"/>
+	<joint name="torso_yaw" value="3.56617e-13"/>
+	<joint name="neck_yaw" value="1.22719e-16"/>
+	<joint name="neck_pitch" value="0.45"/>
+	<joint name="j_arm1_1" value="0.520149"/>
+	<joint name="j_arm1_2" value="0.320865"/>
+	<joint name="j_arm1_3" value="0.274669"/>
+	<joint name="j_arm1_4" value="-2.23604"/>
+	<joint name="j_arm1_5" value="0.0500815"/>
+	<joint name="j_arm1_6" value="-0.781461"/>
+	<joint name="j_arm1_7" value="-0.0567608"/>
+	<joint name="j_arm2_1" value="0.520149"/>
+	<joint name="j_arm2_2" value="-0.320865"/>
+	<joint name="j_arm2_3" value="-0.274669"/>
+	<joint name="j_arm2_4" value="-2.23604"/>
+	<joint name="j_arm2_5" value="-0.0500815"/>
+	<joint name="j_arm2_6" value="-0.781461"/>
+	<joint name="j_arm2_7" value="0.0567608"/>
+   </group_state>
 <!--DISABLE COLLISIONS: By default it is assumed that any link of the robot could potentially come into collision with any other link in the robot. This tag disables collision checking between a specified pair of links. -->
     <disable_collisions link1="ankle1_1" link2="ankle2_1" reason="Adjacent" />

Commit message: Added imu

File: centauro_srdf/srdf/centauro.srdf.xacro (robot description, xacro)
@@ -9,4 +9,7 @@
         <link name="pelvis"/>
     </group>
+<group name="imu_sensors">
+     <link name="imu_link"/>
+</group>
 <xacro:if value="${ADD_LEGS}">
     <group name="front_left_leg">

File: centauro_urdf/urdf/centauro_robot.urdf.xacro (robot description, xacro)
@@ -8,6 +8,6 @@
   <xacro:include filename="$(find centauro_urdf)/urdf/centauro.urdf.xacro" />
   <xacro:include filename="$(find centauro_urdf)/urdf/gazebo/centauro.gazebo.xacro" />
-  <!--xacro:include filename="$(find cogimon_urdf)/urdf/gazebo/force_torque.gazebo.xacro" />
-  <xacro:include filename="$(find cogimon_urdf)/urdf/gazebo/imu.gazebo.xacro" /-->
+  <!--xacro:include filename="$(find cogimon_urdf)/urdf/gazebo/force_torque.gazebo.xacro" /-->
+  <xacro:include filename="$(find centauro_urdf)/urdf/gazebo/imu.gazebo.xacro" />
   <xacro:include filename="$(find centauro_urdf)/urdf/gazebo/xbot.gazebo.xacro" />
   <xacro:include filename="$(find centauro_urdf)/urdf/gazebo/materials.gazebo.xacro" />

Commit message: commented neck joints

File: centauro_srdf/srdf/centauro.srdf.xacro (robot description, xacro)
@@ -73,6 +73,6 @@
 	<joint name="ankle_yaw_4" value="0.746874"/>
 	<joint name="torso_yaw" value="3.56617e-13"/>
-	<joint name="neck_yaw" value="1.22719e-16"/>
-	<joint name="neck_pitch" value="0.45"/>
+	<!--joint name="neck_yaw" value="1.22719e-16"/>
+	<joint name="neck_pitch" value="0.45"/-->
 	<joint name="j_arm1_1" value="0.520149"/>
 	<joint name="j_arm1_2" value="0.320865"/>

Commit message: Started implementation of neck

File: centauro_srdf/srdf/centauro.srdf.xacro (robot description, xacro)
@@ -36,4 +36,10 @@
         <chain base_link="pelvis" tip_link="torso_2" />
     </group>
+    <group name="velodyne">
+    	<chain base_link="torso_2" tip_link="neck_3" />
+    </group>
+    <group name="neck">
+    	<chain base_link="torso_2" tip_link="neck_2" />
+    </group>
 </xacro:if>
 <group name="chains"> <!--THIS HAS TO BE THE LAST GROUP IN THE FILE -->
@@ -48,4 +54,6 @@
         <group name="right_arm" />
         <group name="torso" />
+        <group name="velodyne" />
+        <group name="neck" />
 </xacro:if>
 </group>
@@ -73,6 +81,6 @@
 	<joint name="ankle_yaw_4" value="0.746874"/>
 	<joint name="torso_yaw" value="3.56617e-13"/>
-	<!--joint name="neck_yaw" value="1.22719e-16"/>
-	<joint name="neck_pitch" value="0.45"/-->
+	<joint name="neck_yaw" value="0."/>
+	<joint name="neck_pitch" value="0.2"/>
 	<joint name="j_arm1_1" value="0.520149"/>
 	<joint name="j_arm1_2" value="0.320865"/>

File: centauro_urdf/urdf/centauro_base.urdf.xacro (robot description, xacro)
@@ -52,5 +52,5 @@
    		</xacro:ball_end_effector>
 	</xacro:if>
-	<!--xacro:include filename="$(find pholus_urdf)/urdf/parts/head.urdf.xacro" /-->
+	<xacro:include filename="$(find centauro_urdf)/urdf/parts/head.urdf.xacro" />
 </xacro:if>
 <xacro:if value="${ADD_LEGS}">

File: centauro_urdf/urdf/parts/head.urdf.xacro (robot description, xacro)
@@ -2,60 +2,33 @@
 <robot xmlns:xacro="http://ros.org/wiki/xacro">
 <!-- LINKS -->
-<link name="tof_camera">
-<inertial>
-	<mass value="1.3821576"/>
-	<origin xyz="${4.7324138e+01*mmTom} ${3.1235337*mmTom} ${-3.1691096e+01*mmTom}" rpy="0.0 0.0 0.0"/>
-	<inertia ixx="${3.2284354e+03*mm2Tom2}"  ixy="${6.9551181e+01*mm2Tom2}"  ixz="${-1.2721217e+02*mm2Tom2}" iyy="${2.2420795e+03*mm2Tom2}" iyz="${-1.3961831e+02*mm2Tom2}" izz="${1.8844809e+03*mm2Tom2}" />
-</inertial>
-<visual>
-      <origin xyz="0 0 0" rpy="0 0 0"/>
-      <material name="black"/>
-      <geometry name="tof_camera_visual">
-        <mesh filename="package://pholus_urdf/meshes/tof_camera.stl" scale="${mmTom} ${mmTom} ${mmTom}"/>
-      </geometry>
-</visual>
-<collision>
-      <origin xyz="0 0 0" rpy="0 0 0"/>
-      <geometry name="tof_camera_collision">
-        <mesh filename="package://pholus_urdf/meshes/simple/tof_camera.stl" scale="${mmTom} ${mmTom} ${mmTom}"/>
-      </geometry>
-</collision>
-</link>
-<link name="lidar">
-<inertial>
-	<mass value="8.7087474e-01"/>
-	<origin xyz="${6.0475783e-02*mmTom} ${-8.1621602e-03*mmTom} ${-7.2175098*mmTom}" rpy="0.0 0.0 0.0"/>
-	<inertia ixx="${1.1279642e+02*mm2Tom2}"  ixy="${-3.2830282e-04*mm2Tom2}"  ixz="${-3.9329952e-01*mm2Tom2}" iyy="${6.6830231e+01*mm2Tom2}" iyz="${5.1251186e-02*mm2Tom2}" izz="${1.7248379e+02*mm2Tom2}" />
-</inertial>
-<visual>
-      <origin xyz="0 0 0" rpy="0 0 0"/>
-      <material name="black"/>
-      <geometry name="tof_camera_visual">
-        <mesh filename="package://pholus_urdf/meshes/lidar.stl" scale="${mmTom} ${mmTom} ${mmTom}"/>
-      </geometry>
-</visual>
-<collision>
-      <origin xyz="0 0 0" rpy="0 0 0"/>
-      <geometry name="tof_camera_collision">
-        <mesh filename="package://pholus_urdf/meshes/simple/lidar.stl" scale="${mmTom} ${mmTom} ${mmTom}"/>
-      </geometry>
-</collision>
-</link>
-<!-- JOINTS -->
-<joint name="tof_camera_joint" type="revolute">
-    <parent link="torso"/>
-    <child link="tof_camera"/>
+<!-- TODO: FINISH IMPLEMENTATION WITH CORRECT NUMBERS -->
+<link name="neck_1"/>
+<link name="neck_2"/>
+<link name="neck_3"/>
+<!--JOINTS -->
+<joint name="neck_yaw" type="revolute">
+    <parent link="torso_2"/>
+    <origin xyz="0.0 0.0 0.2795"/>
+    <child link="neck_1"/>
+    <axis xyz="0 0 1"/>
+    <limit effort="35" lower="-0.78539816" upper="0.78539816" velocity="5.7"/>
+    <dynamics friction="10.0"/>
+</joint>
+<joint name="neck_pitch" type="revolute">
+    <parent link="neck_1"/>
+    <origin xyz="0.054 0.0596 -0.0124975"/>
+    <child link="neck_2"/>
     <axis xyz="0 1 0"/>
-    <limit velocity="11.72" effort="${5*torque_scale}" lower="-0.25" upper="0.7" /> <!-- TORQUE AND VELOCITY LIMITS ARE WRONG! -->
-    <dynamics friction="0" damping="0.03"/>
-    <origin xyz="${60*mmTom} 0 ${285.5*mmTom}" rpy="0 0 0" />
+    <limit effort="35" lower="-0.34906585" upper="0.78539816" velocity="5.7"/>
+    <dynamics friction="10.0"/>
 </joint>
-<joint name="lidar_joint" type="revolute">
-    <parent link="torso"/>
-    <child link="lidar"/>
-    <axis xyz="0 1 0"/>
-    <limit velocity="11.72" effort="${5*torque_scale}" lower="-1.57" upper="1.57" />  <!-- TORQUE AND VELOCITY LIMITS ARE WRONG! -->
-    <dynamics friction="0" damping="0.03"/>
-    <origin xyz="${82.27*mmTom} 0 ${399.5*mmTom}" rpy="0 0 0" />
+<joint name="neck_velodyne" type="continuous">
+    <parent link="torso_2"/>
+    <origin xyz="0.055 0.0 0.473262" rpy="0 0 -1.828"/>
+    <!--origin xyz="0.055 0.0 0.473262" rpy="0 0 -1.311481"/-->
+    <child link="neck_3"/>
+    <axis xyz="0 0 1"/>
+    <limit effort="35" velocity="5.7"/>
+    <dynamics damping="0.2" friction="10.0"/>
 </joint>
 </robot>

Commit message: upper-body joints set to "fixed" + update joint transforms

File: centauro_srdf/srdf/centauro.srdf.xacro (robot description, xacro)
@@ -26,5 +26,5 @@
     </group>
 </xacro:if>
-<xacro:if value="${ADD_UPPER_BODY}">
+<!--xacro:if value="${ADD_UPPER_BODY}">
     <group name="left_arm">
         <chain base_link="torso_2" tip_link="arm1_7" />
@@ -42,5 +42,5 @@
     	<chain base_link="torso_2" tip_link="neck_2" />
     </group>
-</xacro:if>
+</xacro:if-->
 <group name="chains"> <!--THIS HAS TO BE THE LAST GROUP IN THE FILE -->
 <xacro:if value="${ADD_LEGS}">
@@ -50,5 +50,5 @@
         <group name="rear_left_leg" />
 </xacro:if>
-<xacro:if value="${ADD_UPPER_BODY}">
+<!--xacro:if value="${ADD_UPPER_BODY}">
 	<group name="left_arm" />
         <group name="right_arm" />
@@ -56,5 +56,5 @@
         <group name="velodyne" />
         <group name="neck" />
-</xacro:if>
+</xacro:if-->
 </group>
 <!-- Homing posture -->
@@ -81,5 +81,5 @@
 	<joint name="ankle_yaw_4" value="0.746874"/>
 	<joint name="torso_yaw" value="3.56617e-13"/>
-	<joint name="neck_yaw" value="0."/>
+	<!--joint name="neck_yaw" value="0."/>
 	<joint name="neck_pitch" value="0.2"/>
 	<joint name="j_arm1_1" value="0.520149"/>
@@ -96,5 +96,5 @@
 	<joint name="j_arm2_5" value="-0.0500815"/>
 	<joint name="j_arm2_6" value="-0.781461"/>
-	<joint name="j_arm2_7" value="0.0567608"/>
+	<joint name="j_arm2_7" value="0.0567608"/-->
    </group_state>
 <!--DISABLE COLLISIONS: By default it is assumed that any link of the robot could potentially come into collision with any other link in the robot. This tag disables collision checking between a specified pair of links. -->
@@ -128,5 +128,5 @@
     <disable_collisions link1="ankle2_4" link2="knee_4" reason="Never" />
     <disable_collisions link1="ankle2_4" link2="wheel_4" reason="Adjacent" />
-    <disable_collisions link1="arm1_1" link2="arm1_2" reason="Adjacent" />
+    <!--disable_collisions link1="arm1_1" link2="arm1_2" reason="Adjacent" />
     <disable_collisions link1="arm1_1" link2="arm1_3" reason="Never" />
     <disable_collisions link1="arm1_1" link2="arm1_4" reason="Never" />
@@ -247,5 +247,5 @@
     <disable_collisions link1="arm2_6" link2="arm2_7" reason="Adjacent" />
     <disable_collisions link1="arm2_6" link2="ft_arm2" reason="Never" />
-    <disable_collisions link1="arm2_7" link2="ft_arm2" reason="Adjacent" />
+    <disable_collisions link1="arm2_7" link2="ft_arm2" reason="Adjacent" /-->
     <disable_collisions link1="hip1_1" link2="hip1_2" reason="Never" />
     <disable_collisions link1="hip1_1" link2="hip1_3" reason="Never" />
@@ -256,5 +256,5 @@
     <disable_collisions link1="hip1_1" link2="knee_1" reason="Never" />
     <disable_collisions link1="hip1_1" link2="pelvis" reason="Adjacent" />
-    <disable_collisions link1="hip1_1" link2="torso_2" reason="Never" />
+    <!--disable_collisions link1="hip1_1" link2="torso_2" reason="Never" /-->
     <disable_collisions link1="hip1_2" link2="hip1_3" reason="Never" />
     <disable_collisions link1="hip1_2" link2="hip1_4" reason="Never" />
@@ -263,5 +263,5 @@
     <disable_collisions link1="hip1_2" link2="hip2_4" reason="Never" />
     <disable_collisions link1="hip1_2" link2="knee_2" reason="Never" />
-    <disable_collisions link1="hip1_2" link2="pelvis" reason="Adjacent" />
+    <!--disable_collisions link1="hip1_2" link2="pelvis" reason="Adjacent" /-->
     <disable_collisions link1="hip1_2" link2="torso_2" reason="Never" />
     <disable_collisions link1="hip1_3" link2="hip1_4" reason="Never" />
@@ -271,5 +271,5 @@
     <disable_collisions link1="hip1_3" link2="knee_3" reason="Never" />
     <disable_collisions link1="hip1_3" link2="pelvis" reason="Adjacent" />
-    <disable_collisions link1="hip1_3" link2="torso_2" reason="Never" />
+    <!--disable_collisions link1="hip1_3" link2="torso_2" reason="Never" /-->
     <disable_collisions link1="hip1_4" link2="hip2_1" reason="Never" />
     <disable_collisions link1="hip1_4" link2="hip2_2" reason="Never" />
@@ -277,17 +277,17 @@
     <disable_collisions link1="hip1_4" link2="knee_4" reason="Never" />
     <disable_collisions link1="hip1_4" link2="pelvis" reason="Adjacent" />
-    <disable_collisions link1="hip1_4" link2="torso_2" reason="Never" />
+    <!--disable_collisions link1="hip1_4" link2="torso_2" reason="Never" /-->
     <disable_collisions link1="hip2_1" link2="knee_1" reason="Adjacent" />
-    <disable_collisions link1="hip2_1" link2="torso_2" reason="Never" />
+    <!--disable_collisions link1="hip2_1" link2="torso_2" reason="Never" /-->
     <disable_collisions link1="hip2_2" link2="knee_2" reason="Adjacent" />
-    <disable_collisions link1="hip2_2" link2="torso_2" reason="Never" />
+    <!--disable_collisions link1="hip2_2" link2="torso_2" reason="Never" /-->
     <disable_collisions link1="hip2_3" link2="knee_3" reason="Adjacent" />
-    <disable_collisions link1="hip2_3" link2="torso_2" reason="Never" />
+    <!--disable_collisions link1="hip2_3" link2="torso_2" reason="Never" /-->
     <disable_collisions link1="hip2_4" link2="knee_4" reason="Adjacent" />
-    <disable_collisions link1="hip2_4" link2="torso_2" reason="Never" />
+    <!--disable_collisions link1="hip2_4" link2="torso_2" reason="Never" /-->
     <disable_collisions link1="knee_1" link2="wheel_1" reason="Never" />
     <disable_collisions link1="knee_2" link2="wheel_2" reason="Never" />
     <disable_collisions link1="knee_3" link2="wheel_3" reason="Never" />
     <disable_collisions link1="knee_4" link2="wheel_4" reason="Never" />
-    <disable_collisions link1="pelvis" link2="torso_2" reason="Adjacent" />
+    <!--disable_collisions link1="pelvis" link2="torso_2" reason="Adjacent" /-->
 </robot>

File: centauro_urdf/urdf/parts/centauro_arm.urdf.xacro (robot description, xacro)
@@ -156,8 +156,10 @@
 <!-- JOINTS -->
 <!-- shoulder yaw -->
-   <joint name="j_arm${arm_num}_1" type="revolute">
+   <joint name="j_arm${arm_num}_1" type="fixed">
       <parent link="${parent}"/>
       <child link="arm${arm_num}_1"/>
-      <xacro:insert_block name="origin"/>
+      <!--xacro:insert_block name="origin"/-->
+      <origin xyz="${Shoulder_1_Ox} ${rot*Shoulder_1_Oy} ${Shoulder_1_Oz}" rpy="0.0 0.520149 0.0"/>
+      <!--origin xyz="${Shoulder_1_Ox} ${rot*Shoulder_1_Oy} ${Shoulder_1_Oz}" rpy="0.0 1.520149 0.0"/-->
       <axis xyz="0 1 0"/>
       <limit lower="${j_arm_1_lower[arm_num-1]}" upper="${j_arm_1_upper[arm_num-1]}" effort="${j_arm_1_torque[arm_num-1]}" velocity="${j_arm_1_velocity[arm_num-1]}"/>
@@ -165,26 +167,27 @@
 <!-- /shoulder yaw -->
 <!-- shoulder roll -->
-   <joint name="j_arm${arm_num}_2" type="revolute">
+   <joint name="j_arm${arm_num}_2" type="fixed">
       <parent link="arm${arm_num}_1"/>
       <child link="arm${arm_num}_2"/>
-      <origin xyz="${Shoulder_2_Ox} ${rot*Shoulder_2_Oy} ${Shoulder_2_Oz}" rpy="${rot*Shoulder_2_roll} ${Shoulder_2_pitch} ${Shoulder_2_yaw}"/>
-      <axis xyz="1 0 0"/>
+      <!--origin xyz="${Shoulder_2_Ox} ${rot*Shoulder_2_Oy} ${Shoulder_2_Oz}" rpy="${rot*Shoulder_2_roll} ${Shoulder_2_pitch} ${Shoulder_2_yaw}"/-->
+      <origin xyz="${Shoulder_2_Ox} ${rot*Shoulder_2_Oy} ${Shoulder_2_Oz}" rpy="${rot*0.320865} 0.0 0.0"/>
+      <axis xyz="1 0 0" />
       <limit lower="${j_arm_2_lower[arm_num-1]}" upper="${j_arm_2_upper[arm_num-1]}" effort="${j_arm_2_torque[arm_num-1]}" velocity="${j_arm_2_velocity[arm_num-1]}"/>
    </joint>
 <!-- /shoulder roll -->
 <!-- shoulder pitch-->
-   <joint name="j_arm${arm_num}_3" type="revolute">
+   <joint name="j_arm${arm_num}_3" type="fixed">
       <parent link="arm${arm_num}_2"/>
       <child link="arm${arm_num}_3"/>
-      <origin xyz="${Shoulder_3_Ox} ${Shoulder_3_Oy} ${Shoulder_3_Oz}"/>
-      <axis xyz="0 0 1"/>
+      <origin xyz="${Shoulder_3_Ox} ${Shoulder_3_Oy} ${Shoulder_3_Oz}" rpy="0.0 0.0 ${rot*0.274669}"/>
+      <axis xyz="0 0 1" />
       <limit lower="${j_arm_3_lower[arm_num-1]}" upper="${j_arm_3_upper[arm_num-1]}" effort="${j_arm_3_torque[arm_num-1]}" velocity="${j_arm_3_velocity[arm_num-1]}"/>
    </joint>
 <!-- /shoulder pitch -->
 <!-- elbow yaw -->
-   <joint name="j_arm${arm_num}_4" type="revolute">
+   <joint name="j_arm${arm_num}_4" type="fixed">
       <parent link="arm${arm_num}_3"/>
       <child link="arm${arm_num}_4"/>
-      <origin xyz="${Elbow_1_Ox} ${rot*Elbow_1_Oy} ${Elbow_1_Oz}"/>
+      <origin xyz="${Elbow_1_Ox} ${rot*Elbow_1_Oy} ${Elbow_1_Oz}" rpy="0.0 -2.23604 0.0"/>
       <axis xyz="0 1 0"/>
       <limit lower="${j_arm_4_lower[arm_num-1]}" upper="${j_arm_4_upper[arm_num-1]}" effort="${j_arm_4_torque[arm_num-1]}" velocity="${j_arm_4_velocity[arm_num-1]}"/>
@@ -192,8 +195,8 @@
 <!-- /elbow yaw -->
 <!-- elbow pitch-->
-   <joint name="j_arm${arm_num}_5" type="revolute">
+   <joint name="j_arm${arm_num}_5" type="fixed">
       <parent link="arm${arm_num}_4"/>
       <child link="arm${arm_num}_5"/>
-      <origin xyz="${Wrist_1_Ox} ${rot*Wrist_1_Oy} ${Wrist_1_Oz}"/>
+      <origin xyz="${Wrist_1_Ox} ${rot*Wrist_1_Oy} ${Wrist_1_Oz}" rpy="0.0 0.0 ${rot*0.0500815}"/>
       <axis xyz="0 0 1"/>
       <limit lower="${j_arm_5_lower[arm_num-1]}" upper="${j_arm_5_upper[arm_num-1]}" effort="${j_arm_5_torque[arm_num-1]}" velocity="${j_arm_5_velocity[arm_num-1]}"/>
@@ -201,8 +204,8 @@
 <!-- /elbow pitch-->
 <!-- wrist yaw-->
-   <joint name="j_arm${arm_num}_6" type="revolute">
+   <joint name="j_arm${arm_num}_6" type="fixed">
       <parent link="arm${arm_num}_5"/>
       <child link="arm${arm_num}_6"/>
-      <origin xyz="${Wrist_2_Ox} ${rot*Wrist_2_Oy} ${Wrist_2_Oz}"/>
+      <origin xyz="${Wrist_2_Ox} ${rot*Wrist_2_Oy} ${Wrist_2_Oz}" rpy="0.0 -0.781461 0.0"/>
       <axis xyz="0 1 0"/>
       <limit lower="${j_arm_6_lower[arm_num-1]}" upper="${j_arm_6_upper[arm_num-1]}" effort="${j_arm_6_torque[arm_num-1]}" velocity="${j_arm_6_velocity[arm_num-1]}"/>
@@ -210,8 +213,8 @@
 <!-- /wrist yaw-->
 <!-- wrist pitch-->
-   <joint name="j_arm${arm_num}_7" type="revolute">
+   <joint name="j_arm${arm_num}_7" type="fixed">
       <parent link="arm${arm_num}_6"/>
       <child link="arm${arm_num}_7"/>
-      <origin xyz="${Wrist_3_Ox} ${rot*Wrist_3_Oy} ${Wrist_3_Oz}"/>
+      <origin xyz="${Wrist_3_Ox} ${rot*Wrist_3_Oy} ${Wrist_3_Oz}" rpy="0.0 0.0 ${-rot*0.0500815}"/>
       <axis xyz="0 0 1"/>
       <limit lower="${j_arm_7_lower[arm_num-1]}" upper="${j_arm_7_upper[arm_num-1]}" effort="${j_arm_7_torque[arm_num-1]}" velocity="${j_arm_7_velocity[arm_num-1]}"/>

File: centauro_urdf/urdf/parts/centauro_torso.urdf.xacro (robot description, xacro)
@@ -23,5 +23,5 @@
 <!-- /torso links -->
 <!-- torso joints -->
-<joint name="torso_yaw" type="revolute">
+<joint name="torso_yaw" type="fixed">
    <parent link="pelvis"/>
    <origin xyz="${Torso_2_Ox} ${Torso_2_Oy} ${Torso_2_Oz}"/>

File: centauro_urdf/urdf/parts/head.urdf.xacro (robot description, xacro)
@@ -61,5 +61,5 @@
 </link>
 <!--JOINTS -->
-<joint name="neck_yaw" type="revolute">
+<joint name="neck_yaw" type="fixed">
     <parent link="torso_2"/>
     <origin xyz="0.0 0.0 0.2795"/>
@@ -69,5 +69,5 @@
     <dynamics friction="10.0"/>
 </joint>
-<joint name="neck_pitch" type="revolute">
+<joint name="neck_pitch" type="fixed">
     <parent link="neck_1"/>
     <origin xyz="0.054 0.0596 -0.0124975"/>
@@ -77,5 +77,5 @@
     <dynamics friction="10.0"/>
 </joint>
-<joint name="neck_velodyne" type="continuous">
+<joint name="neck_velodyne" type="fixed">
     <parent link="torso_2"/>
     <origin xyz="0.055 0.0 0.473262" rpy="0 0 -1.828"/>
