Commit message: Adding Velodyne to the model

File: centauro_srdf/srdf/centauro.srdf.xacro (robot description, xacro)
@@ -43,18 +43,26 @@
     </group>
 </xacro:if>
+<xacro:if value="${ADD_INTEL_D435I}">
+    <group name="sensor_d435i">
+        <chain base_link="base_camera_link" tip_link="camera_gyro_optical_frame" />
+    </group>
+</xacro:if>
 <group name="chains"> <!--THIS HAS TO BE THE LAST GROUP IN THE FILE -->
-<xacro:if value="${ADD_LEGS}">
-	<group name="front_left_leg" />
+    <xacro:if value="${ADD_LEGS}">
+        <group name="front_left_leg" />
         <group name="front_right_leg" />
         <group name="rear_right_leg" />
         <group name="rear_left_leg" />
-</xacro:if>
-<xacro:if value="${ADD_UPPER_BODY}">
-	<group name="left_arm" />
+    </xacro:if>
+    <xacro:if value="${ADD_UPPER_BODY}">
+        <group name="left_arm" />
         <group name="right_arm" />
         <group name="torso" />
         <group name="velodyne" />
         <group name="neck" />
-</xacro:if>
+    </xacro:if>
+    <xacro:if value="${ADD_INTEL_D435I}">
+        <group name="sensor_d435i" />
+    </xacro:if>
 </group>
 <!-- Homing posture -->

File: centauro_urdf/urdf/centauro_base.urdf.xacro (robot description, xacro)
@@ -29,10 +29,10 @@
       </collision>
    </link>
-    <link name="imu_link"/>
-    <joint name="imu_joint" type="fixed">
-        <parent link="pelvis"/>
-        <origin xyz="${Imu_Ox} ${Imu_Oy} ${Imu_Oz}" rpy="${Imu_raw} ${Imu_pitch} ${Imu_yaw}"/>
-        <child link="imu_link"/>
-    </joint>
+<link name="imu_link"/>
+<joint name="imu_joint" type="fixed">
+    <parent link="pelvis"/>
+    <origin xyz="${Imu_Ox} ${Imu_Oy} ${Imu_Oz}" rpy="${Imu_raw} ${Imu_pitch} ${Imu_yaw}"/>
+    <child link="imu_link"/>
+</joint>
 <joint name="base_joint" type="fixed">
     <parent link="pelvis"/>
@@ -57,3 +57,20 @@
 	<xacro:include filename="$(find centauro_urdf)/urdf/parts/legs.urdf.xacro" />
 </xacro:if>
+<xacro:if value="${ADD_VELODYNE}">
+  <xacro:include filename="$(find velodyne_description)/urdf/VLP-16.urdf.xacro"/>
+</xacro:if>
+<xacro:if value="${ADD_INTEL_D435I}">
+    <xacro:arg name="use_nominal_extrinsics" default="false" />
+	<xacro:include filename="$(find centauro_urdf)/urdf/parts/d435i.urdf.xacro" />
+    <link name="base_camera_link" />
+    <joint name="d435i_joint" type="fixed">
+        <parent link="torso_2"/>
+        <origin xyz="0.14 0 0.03" rpy="0 0.3 0"/>
+        <child link="base_camera_link"/>
+    </joint>
+    <xacro:sensor_d435i parent="base_camera_link" name="camera" topics_ns="camera"
+                        enable_pointCloud="true" align_depth="true">
+        <origin xyz="0 0 0" rpy="0 0 0"/>
+    </xacro:sensor_d435i>
+</xacro:if>
 </robot>

File: centauro_urdf/urdf/centauro_robot.urdf.xacro (robot description, xacro)
@@ -8,4 +8,8 @@
   <xacro:include filename="$(find centauro_urdf)/urdf/centauro.urdf.xacro" />
   <xacro:include filename="$(find centauro_urdf)/urdf/gazebo/centauro.gazebo.xacro" />
+  <xacro:if value="${ADD_INTEL_D435I}">
+    <xacro:include filename="$(find centauro_urdf)/urdf/gazebo/d435i.gazebo.xacro" parent="base_camera_link" name="camera" topics_ns="camera"
+                        enable_pointCloud="true" align_depth="true"/>
+  </xacro:if>
   <!--xacro:include filename="$(find cogimon_urdf)/urdf/gazebo/force_torque.gazebo.xacro" /-->
   <xacro:include filename="$(find centauro_urdf)/urdf/gazebo/imu.gazebo.xacro" />

File: centauro_urdf/urdf/gazebo/centauro.gazebo.xacro (robot description, xacro)
@@ -197,3 +197,9 @@
 </gazebo>
 </xacro:if>
+<!-- SENSORS -->
+<xacro:if value="${ADD_VELODYNE}">
+    <VLP-16 parent="neck_3" name="velodyne_calib" topic="/velodyne_points" hz="10" samples="440">
+        <origin xyz="0.032768 -0.01 0.048219" rpy="0 1.5709 -0.316519  " />
+    </VLP-16>
+</xacro:if>
 </robot>

File: centauro_urdf/urdf/parts/head.urdf.xacro (robot description, xacro)
@@ -60,4 +60,12 @@
     </collision>
 </link>
+<!--
+<link name="velodyne_mount">
+	<inertial>
+		<origin xyz="${Dummy_x} ${Dummy_y} ${Dummy_z}"/>
+		<mass value="${Dummy_mass}"/>
+                <inertia ixx="${Dummy_xx}" ixy="${Dummy_xy}" ixz="${Dummy_xz}" iyy="${Dummy_yy}" iyz="${Dummy_yz}" izz="${Dummy_zz}"/>
+        </inertial>
+</link> -->
 <!--JOINTS -->
 <joint name="neck_yaw" type="revolute">
@@ -86,3 +94,10 @@
     <dynamics damping="0.2" friction="10.0"/>
 </joint>
+<!--
+<joint name="j_velodyne" type="fixed">
+   <parent link="neck_3"/>
+   <origin xyz="${Velodyne_Ox} ${Velodyne_Oy} ${Velodyne_Oz}" rpy="${Velodyne_roll} ${Velodyne_pitch} ${Velodyne_yaw}"/>
+   <child link="velodyne_mount"/>
+</joint>
+-->
 </robot>

Commit message: Parameteric velodyne + D435i

File: centauro_srdf/srdf/centauro.srdf.xacro (robot description, xacro)
@@ -36,14 +36,16 @@
         <chain base_link="pelvis" tip_link="torso_2" />
     </group>
+    <group name="neck">
+    	<chain base_link="torso_2" tip_link="neck_2" />
+    </group>
+</xacro:if>
+<xacro:if value="${ADD_VELODYNE}">
     <group name="velodyne">
     	<chain base_link="torso_2" tip_link="neck_3" />
     </group>
-    <group name="neck">
-    	<chain base_link="torso_2" tip_link="neck_2" />
-    </group>
 </xacro:if>
 <xacro:if value="${ADD_INTEL_D435I}">
-    <group name="sensor_d435i">
-        <chain base_link="base_camera_link" tip_link="camera_gyro_optical_frame" />
+    <group name="intel_d435i">
+        <chain base_link="torso_2" tip_link="d435i_base_torso" />
     </group>
 </xacro:if>
@@ -59,9 +61,11 @@
         <group name="right_arm" />
         <group name="torso" />
-        <group name="velodyne" />
         <group name="neck" />
     </xacro:if>
+    <xacro:if value="${ADD_VELODYNE}">
+        <group name="velodyne">
+    </xacro:if>
     <xacro:if value="${ADD_INTEL_D435I}">
-        <group name="sensor_d435i" />
+        <group name="intel_d435i">
     </xacro:if>
 </group>

File: centauro_urdf/urdf/centauro_base.urdf.xacro (robot description, xacro)
@@ -53,24 +53,14 @@
 	</xacro:if>
 	<xacro:include filename="$(find centauro_urdf)/urdf/parts/head.urdf.xacro" />
+    <xacro:if value="${ADD_VELODYNE}">
+        <xacro:include filename="$(find velodyne_description)/urdf/VLP-16.urdf.xacro"/>
+    </xacro:if>
+    <xacro:if value="${ADD_INTEL_D435I}">
+        <xacro:include filename="$(find centauro_urdf)/urdf/parts/intel_d435i_frames.urdf.xacro" />
+        <xacro:include filename="$(find realsense_gazebo_description)/urdf/_d435i.urdf.xacro" />
+    </xacro:if>
 </xacro:if>
 <xacro:if value="${ADD_LEGS}">
 	<xacro:include filename="$(find centauro_urdf)/urdf/parts/legs.urdf.xacro" />
 </xacro:if>
-<xacro:if value="${ADD_VELODYNE}">
-  <xacro:include filename="$(find velodyne_description)/urdf/VLP-16.urdf.xacro"/>
-</xacro:if>
-<xacro:if value="${ADD_INTEL_D435I}">
-    <xacro:arg name="use_nominal_extrinsics" default="false" />
-	<xacro:include filename="$(find centauro_urdf)/urdf/parts/d435i.urdf.xacro" />
-    <link name="base_camera_link" />
-    <joint name="d435i_joint" type="fixed">
-        <parent link="torso_2"/>
-        <origin xyz="0.14 0 0.03" rpy="0 0.3 0"/>
-        <child link="base_camera_link"/>
-    </joint>
-    <xacro:sensor_d435i parent="base_camera_link" name="camera" topics_ns="camera"
-                        enable_pointCloud="true" align_depth="true">
-        <origin xyz="0 0 0" rpy="0 0 0"/>
-    </xacro:sensor_d435i>
-</xacro:if>
 </robot>

File: centauro_urdf/urdf/centauro_config.urdf.xacro (robot description, xacro)
@@ -9,5 +9,5 @@
 <xacro:property name="ADD_BALL_END_EFFECTOR" value="true" />
 <xacro:property name="ADD_FLOATING_BASE" value="true" />
-<xacro:property name="ADD_VELODYNE" value="true" />
-<xacro:property name="ADD_INTEL_D435I" value="false" />
+<xacro:property name="ADD_VELODYNE" value="$(arg VELODYNE)" />
+<xacro:property name="ADD_INTEL_D435I" value="$(arg INTEL_D435I)" />
 </robot>

File: centauro_urdf/urdf/centauro_robot.urdf.xacro (robot description, xacro)
@@ -8,8 +8,4 @@
   <xacro:include filename="$(find centauro_urdf)/urdf/centauro.urdf.xacro" />
   <xacro:include filename="$(find centauro_urdf)/urdf/gazebo/centauro.gazebo.xacro" />
-  <xacro:if value="${ADD_INTEL_D435I}">
-    <xacro:include filename="$(find centauro_urdf)/urdf/gazebo/d435i.gazebo.xacro" parent="base_camera_link" name="camera" topics_ns="camera"
-                        enable_pointCloud="true" align_depth="true"/>
-  </xacro:if>
   <!--xacro:include filename="$(find cogimon_urdf)/urdf/gazebo/force_torque.gazebo.xacro" /-->
   <xacro:include filename="$(find centauro_urdf)/urdf/gazebo/imu.gazebo.xacro" />

File: centauro_urdf/urdf/config/centauro.urdf.xacro (robot description, xacro)
@@ -9,3 +9,5 @@
 <xacro:property name="ADD_BALL_END_EFFECTOR" value="true" />
 <xacro:property name="ADD_FLOATING_BASE" value="true" />
+<xacro:property name="ADD_VELODYNE" value="false" />
+<xacro:property name="ADD_INTEL_D435I" value="true" />
 </robot>

File: centauro_urdf/urdf/gazebo/centauro.gazebo.xacro (robot description, xacro)
@@ -196,5 +196,4 @@
     <provideFeedback>true</provideFeedback>
 </gazebo>
-</xacro:if>
 <!-- SENSORS -->
 <xacro:if value="${ADD_VELODYNE}">
@@ -203,3 +202,10 @@
     </VLP-16>
 </xacro:if>
+<xacro:if value="${ADD_INTEL_D435I}">
+    <xacro:sensor_d435i parent="d435i_base_torso" name="d453i_camera" topics_ns="/d453i_camera"
+                        enable_pointCloud="true" align_depth="true">
+        <origin xyz="0.13 0 0.03" rpy="0 0.3 0"/>
+    </xacro:sensor_d435i>
+</xacro:if>
+</xacro:if>
 </robot>

File: centauro_urdf/urdf/parts/head.urdf.xacro (robot description, xacro)
@@ -41,4 +41,5 @@
     </collision>
 </link>
+<!-- LINKS -->
 <link name="neck_3">
     <inertial>
@@ -60,12 +61,4 @@
     </collision>
 </link>
-<!--
-<link name="velodyne_mount">
-	<inertial>
-		<origin xyz="${Dummy_x} ${Dummy_y} ${Dummy_z}"/>
-		<mass value="${Dummy_mass}"/>
-                <inertia ixx="${Dummy_xx}" ixy="${Dummy_xy}" ixz="${Dummy_xz}" iyy="${Dummy_yy}" iyz="${Dummy_yz}" izz="${Dummy_zz}"/>
-        </inertial>
-</link> -->
 <!--JOINTS -->
 <joint name="neck_yaw" type="revolute">
@@ -94,10 +87,3 @@
     <dynamics damping="0.2" friction="10.0"/>
 </joint>
-<!--
-<joint name="j_velodyne" type="fixed">
-   <parent link="neck_3"/>
-   <origin xyz="${Velodyne_Ox} ${Velodyne_Oy} ${Velodyne_Oz}" rpy="${Velodyne_roll} ${Velodyne_pitch} ${Velodyne_yaw}"/>
-   <child link="velodyne_mount"/>
-</joint>
--->
 </robot>

Commit message: Adjust Velodyne orientation

File: centauro_srdf/srdf/centauro.srdf.xacro (robot description, xacro)
@@ -64,8 +64,8 @@
     </xacro:if>
     <xacro:if value="${ADD_VELODYNE}">
-        <group name="velodyne">
+        <group name="velodyne"/>
     </xacro:if>
     <xacro:if value="${ADD_INTEL_D435I}">
-        <group name="intel_d435i">
+        <group name="intel_d435i"/>
     </xacro:if>
 </group>

File: centauro_urdf/urdf/config/centauro.urdf.xacro (robot description, xacro)
@@ -10,4 +10,4 @@
 <xacro:property name="ADD_FLOATING_BASE" value="true" />
 <xacro:property name="ADD_VELODYNE" value="false" />
-<xacro:property name="ADD_INTEL_D435I" value="true" />
+<xacro:property name="ADD_INTEL_D435I" value="false" />
 </robot>

File: centauro_urdf/urdf/parts/head.urdf.xacro (robot description, xacro)
@@ -80,6 +80,5 @@
 <joint name="neck_velodyne" type="continuous">
     <parent link="torso_2"/>
-    <origin xyz="0.055 0.0 0.473262" rpy="0 0 -1.828"/>
-    <!--origin xyz="0.055 0.0 0.473262" rpy="0 0 -1.311481"/-->
+    <origin xyz="0.055 0.0 0.473262" rpy="0 0 0"/>
     <child link="neck_3"/>
     <axis xyz="0 0 1"/>

Commit message: Add D435i sensor

File: centauro_srdf/srdf/centauro.srdf.xacro (robot description, xacro)
@@ -43,9 +43,4 @@
     <group name="velodyne">
     	<chain base_link="torso_2" tip_link="neck_3" />
-    </group>
-</xacro:if>
-<xacro:if value="${ADD_INTEL_D435I}">
-    <group name="intel_d435i">
-        <chain base_link="torso_2" tip_link="d435i_base_torso" />
     </group>
 </xacro:if>
@@ -65,7 +60,4 @@
     <xacro:if value="${ADD_VELODYNE}">
         <group name="velodyne"/>
-    </xacro:if>
-    <xacro:if value="${ADD_INTEL_D435I}">
-        <group name="intel_d435i"/>
     </xacro:if>
 </group>

File: centauro_urdf/urdf/centauro_base.urdf.xacro (robot description, xacro)
@@ -55,8 +55,14 @@
     <xacro:if value="${ADD_VELODYNE}">
         <xacro:include filename="$(find velodyne_description)/urdf/VLP-16.urdf.xacro"/>
+        <xacro:VLP-16 parent="neck_3" name="velodyne_calib" topic="/velodyne_points" hz="10" samples="440">
+            <origin xyz="0.032768 -0.01 0.048219" rpy="0 1.5709 -0.316519  " />
+        </xacro:VLP-16>
     </xacro:if>
     <xacro:if value="${ADD_INTEL_D435I}">
-        <xacro:include filename="$(find centauro_urdf)/urdf/parts/intel_d435i_frames.urdf.xacro" />
         <xacro:include filename="$(find realsense_gazebo_description)/urdf/_d435i.urdf.xacro" />
+        <xacro:sensor_d435i parent="torso_2" name="d435i_camera" topics_ns="/d435i_camera"
+                            enable_pointCloud="true" align_depth="true">
+            <origin xyz="0.13 0 0.03" rpy="0 0.3 0"/>
+        </xacro:sensor_d435i>
     </xacro:if>
 </xacro:if>

File: centauro_urdf/urdf/centauro_config.urdf.xacro (robot description, xacro)
@@ -9,5 +9,5 @@
 <xacro:property name="ADD_BALL_END_EFFECTOR" value="true" />
 <xacro:property name="ADD_FLOATING_BASE" value="true" />
-<xacro:property name="ADD_VELODYNE" value="$(arg VELODYNE)" />
-<xacro:property name="ADD_INTEL_D435I" value="$(arg INTEL_D435I)" />
+<xacro:property name="ADD_VELODYNE" value="true" />
+<xacro:property name="ADD_INTEL_D435I" value="true" />
 </robot>

File: centauro_urdf/urdf/config/centauro.urdf.xacro (robot description, xacro)
@@ -9,5 +9,5 @@
 <xacro:property name="ADD_BALL_END_EFFECTOR" value="true" />
 <xacro:property name="ADD_FLOATING_BASE" value="true" />
-<xacro:property name="ADD_VELODYNE" value="false" />
-<xacro:property name="ADD_INTEL_D435I" value="false" />
+<xacro:property name="ADD_VELODYNE" value="true" />
+<xacro:property name="ADD_INTEL_D435I" value="true" />
 </robot>

File: centauro_urdf/urdf/gazebo/centauro.gazebo.xacro (robot description, xacro)
@@ -196,16 +196,4 @@
     <provideFeedback>true</provideFeedback>
 </gazebo>
-<!-- SENSORS -->
-<xacro:if value="${ADD_VELODYNE}">
-    <VLP-16 parent="neck_3" name="velodyne_calib" topic="/velodyne_points" hz="10" samples="440">
-        <origin xyz="0.032768 -0.01 0.048219" rpy="0 1.5709 -0.316519  " />
-    </VLP-16>
-</xacro:if>
-<xacro:if value="${ADD_INTEL_D435I}">
-    <xacro:sensor_d435i parent="d435i_base_torso" name="d453i_camera" topics_ns="/d453i_camera"
-                        enable_pointCloud="true" align_depth="true">
-        <origin xyz="0.13 0 0.03" rpy="0 0.3 0"/>
-    </xacro:sensor_d435i>
-</xacro:if>
 </xacro:if>
 </robot>
