Commit message: adding virtual frame model

File: centauro_srdf/srdf/centauro.srdf.xacro (robot description, xacro)
@@ -9,94 +9,102 @@
         <link name="pelvis"/>
     </group>
-<group name="imu_sensors">
-     <link name="imu_link"/>
-</group>
-<xacro:if value="${ADD_LEGS}">
-    <group name="front_left_leg">
-        <chain base_link="pelvis" tip_link="wheel_1" />
+    <group name="imu_sensors">
+        <link name="imu_link"/>
     </group>
-    <group name="front_right_leg">
-        <chain base_link="pelvis" tip_link="wheel_2" />
+    <xacro:if value="${ADD_LEGS}">
+        <group name="front_left_leg">
+            <chain base_link="pelvis" tip_link="wheel_1" />
+        </group>
+        <group name="front_right_leg">
+            <chain base_link="pelvis" tip_link="wheel_2" />
+        </group>
+        <group name="rear_right_leg">
+            <chain base_link="pelvis" tip_link="wheel_4" />
+        </group>
+        <group name="rear_left_leg">
+            <chain base_link="pelvis" tip_link="wheel_3" />
+        </group>
+    </xacro:if>
+    <xacro:if value="${ADD_UPPER_BODY}">
+        <group name="left_arm">
+            <chain base_link="torso_2" tip_link="arm1_7" />
+        </group>
+        <group name="right_arm">
+            <chain base_link="torso_2" tip_link="arm2_7" />
+        </group>
+        <group name="torso">
+            <chain base_link="pelvis" tip_link="torso_2" />
+        </group>
+        <group name="velodyne">
+            <chain base_link="torso_2" tip_link="neck_3" />
+        </group>
+        <group name="neck">
+            <chain base_link="torso_2" tip_link="neck_2" />
+        </group>
+    </xacro:if>
+    <xacro:if value="${ADD_VIRTUAL_FRAME}">
+        <group name="car_frame_chain">
+            <chain base_link="pelvis" tip_link="car_frame"/>
+        </group>
+    </xacro:if>
+    <group name="chains">        <!--THIS HAS TO BE THE LAST GROUP IN THE FILE -->
+        <xacro:if value="${ADD_LEGS}">
+            <group name="front_left_leg" />
+            <group name="front_right_leg" />
+            <group name="rear_right_leg" />
+            <group name="rear_left_leg" />
+        </xacro:if>
+        <xacro:if value="${ADD_UPPER_BODY}">
+            <group name="left_arm" />
+            <group name="right_arm" />
+            <group name="torso" />
+            <group name="velodyne" />
+            <group name="neck" />
+        </xacro:if>
+        <xacro:if value="${ADD_VIRTUAL_FRAME}">
+            <group name="car_frame_chain"/>
+        </xacro:if>
     </group>
-    <group name="rear_right_leg">
-        <chain base_link="pelvis" tip_link="wheel_4" />
-    </group>
-    <group name="rear_left_leg">
-        <chain base_link="pelvis" tip_link="wheel_3" />
-    </group>
-</xacro:if>
-<xacro:if value="${ADD_UPPER_BODY}">
-    <group name="left_arm">
-        <chain base_link="torso_2" tip_link="arm1_7" />
-    </group>
-    <group name="right_arm">
-        <chain base_link="torso_2" tip_link="arm2_7" />
-    </group>
-    <group name="torso">
-        <chain base_link="pelvis" tip_link="torso_2" />
-    </group>
-    <group name="velodyne">
-    	<chain base_link="torso_2" tip_link="neck_3" />
-    </group>
-    <group name="neck">
-    	<chain base_link="torso_2" tip_link="neck_2" />
-    </group>
-</xacro:if>
-<group name="chains"> <!--THIS HAS TO BE THE LAST GROUP IN THE FILE -->
-<xacro:if value="${ADD_LEGS}">
-	<group name="front_left_leg" />
-        <group name="front_right_leg" />
-        <group name="rear_right_leg" />
-        <group name="rear_left_leg" />
-</xacro:if>
-<xacro:if value="${ADD_UPPER_BODY}">
-	<group name="left_arm" />
-        <group name="right_arm" />
-        <group name="torso" />
-        <group name="velodyne" />
-        <group name="neck" />
-</xacro:if>
-</group>
-<!-- Homing posture -->
-<group_state name="home" group="chains">
-	<joint name="hip_yaw_1" value="-0.746874"/>
-	<joint name="hip_pitch_1" value="-1.25409"/>
-	<joint name="knee_pitch_1" value="-1.55576"/>
-	<joint name="ankle_pitch_1" value="-0.301666"/>
-	<joint name="ankle_yaw_1" value="0.746874"/>
-	<joint name="hip_yaw_2" value="0.746874"/>
-	<joint name="hip_pitch_2" value="1.25409"/>
-	<joint name="knee_pitch_2" value="1.55576"/>
-	<joint name="ankle_pitch_2" value="0.301666"/>
-	<joint name="ankle_yaw_2" value="-0.746874"/>
-	<joint name="hip_yaw_3" value="0.746874"/>
-	<joint name="hip_pitch_3" value="1.25409"/>
-	<joint name="knee_pitch_3" value="1.55576"/>
-	<joint name="ankle_pitch_3" value="0.301667"/>
-	<joint name="ankle_yaw_3" value="-0.746874"/>
-	<joint name="hip_yaw_4" value="-0.746874"/>
-	<joint name="hip_pitch_4" value="-1.25409"/>
-	<joint name="knee_pitch_4" value="-1.55576"/>
-	<joint name="ankle_pitch_4" value="-0.301667"/>
-	<joint name="ankle_yaw_4" value="0.746874"/>
-	<joint name="torso_yaw" value="3.56617e-13"/>
-	<joint name="neck_yaw" value="0."/>
-	<joint name="neck_pitch" value="0.2"/>
-	<joint name="j_arm1_1" value="0.520149"/>
-	<joint name="j_arm1_2" value="0.320865"/>
-	<joint name="j_arm1_3" value="0.274669"/>
-	<joint name="j_arm1_4" value="-2.23604"/>
-	<joint name="j_arm1_5" value="0.0500815"/>
-	<joint name="j_arm1_6" value="-0.781461"/>
-	<joint name="j_arm1_7" value="-0.0567608"/>
-	<joint name="j_arm2_1" value="0.520149"/>
-	<joint name="j_arm2_2" value="-0.320865"/>
-	<joint name="j_arm2_3" value="-0.274669"/>
-	<joint name="j_arm2_4" value="-2.23604"/>
-	<joint name="j_arm2_5" value="-0.0500815"/>
-	<joint name="j_arm2_6" value="-0.781461"/>
-	<joint name="j_arm2_7" value="0.0567608"/>
-   </group_state>
-<!--DISABLE COLLISIONS: By default it is assumed that any link of the robot could potentially come into collision with any other link in the robot. This tag disables collision checking between a specified pair of links. -->
+    <!-- Homing posture -->
+    <group_state name="home" group="chains">
+        <joint name="hip_yaw_1" value="-0.746874"/>
+        <joint name="hip_pitch_1" value="-1.25409"/>
+        <joint name="knee_pitch_1" value="-1.55576"/>
+        <joint name="ankle_pitch_1" value="-0.301666"/>
+        <joint name="ankle_yaw_1" value="0.746874"/>
+        <joint name="hip_yaw_2" value="0.746874"/>
+        <joint name="hip_pitch_2" value="1.25409"/>
+        <joint name="knee_pitch_2" value="1.55576"/>
+        <joint name="ankle_pitch_2" value="0.301666"/>
+        <joint name="ankle_yaw_2" value="-0.746874"/>
+        <joint name="hip_yaw_3" value="0.746874"/>
+        <joint name="hip_pitch_3" value="1.25409"/>
+        <joint name="knee_pitch_3" value="1.55576"/>
+        <joint name="ankle_pitch_3" value="0.301667"/>
+        <joint name="ankle_yaw_3" value="-0.746874"/>
+        <joint name="hip_yaw_4" value="-0.746874"/>
+        <joint name="hip_pitch_4" value="-1.25409"/>
+        <joint name="knee_pitch_4" value="-1.55576"/>
+        <joint name="ankle_pitch_4" value="-0.301667"/>
+        <joint name="ankle_yaw_4" value="0.746874"/>
+        <joint name="torso_yaw" value="3.56617e-13"/>
+        <joint name="neck_yaw" value="0."/>
+        <joint name="neck_pitch" value="0.2"/>
+        <joint name="j_arm1_1" value="0.520149"/>
+        <joint name="j_arm1_2" value="0.320865"/>
+        <joint name="j_arm1_3" value="0.274669"/>
+        <joint name="j_arm1_4" value="-2.23604"/>
+        <joint name="j_arm1_5" value="0.0500815"/>
+        <joint name="j_arm1_6" value="-0.781461"/>
+        <joint name="j_arm1_7" value="-0.0567608"/>
+        <joint name="j_arm2_1" value="0.520149"/>
+        <joint name="j_arm2_2" value="-0.320865"/>
+        <joint name="j_arm2_3" value="-0.274669"/>
+        <joint name="j_arm2_4" value="-2.23604"/>
+        <joint name="j_arm2_5" value="-0.0500815"/>
+        <joint name="j_arm2_6" value="-0.781461"/>
+        <joint name="j_arm2_7" value="0.0567608"/>
+    </group_state>
+    <!--DISABLE COLLISIONS: By default it is assumed that any link of the robot could potentially come into collision with any other link in the robot. This tag disables collision checking between a specified pair of links. -->
     <disable_collisions link1="ankle1_1" link2="ankle2_1" reason="Adjacent" />
     <disable_collisions link1="ankle1_1" link2="hip1_1" reason="Never" />

File: centauro_urdf/urdf/centauro.urdf.xacro (robot description, xacro)
@@ -21,3 +21,6 @@
 </joint>
 </xacro:unless>
+<xacro:if value="${ADD_VIRTUAL_FRAME}">
+  <xacro:include filename="$(find centauro_urdf)/urdf/parts/virtual_frame.urdf.xacro"/>
+</xacro:if>
 </robot>

File: centauro_urdf/urdf/config/centauro_virtual_frame.urdf.xacro (robot description, xacro)
@@ -12,5 +12,5 @@
 <xacro:property name="ADD_BALL_END_EFFECTOR" value="true" />
 <xacro:property name="ADD_FLOATING_BASE" value="$(arg add_legs)" />
-<xacro:property name="ADD_VIRTUAL_FRAME" value="false" />
+<xacro:property name="ADD_VIRTUAL_FRAME" value="true" />
 <xacro:property name="USE_STICKS" value="false" />
 </robot>
