Commit message: cmake-based generation && avoid to clutter src folder

File: centauro_srdf/srdf/centauro.srdf.xacro (robot description, xacro)
@@ -5,5 +5,7 @@
 -->
 <robot xmlns:xacro="http://ros.org/wiki/xacro" name="centauro">
-    <xacro:include filename="$(find centauro_urdf)/urdf/centauro_config.urdf.xacro" />
+    <!-- ************ MODEL CONFIGURATION ************ -->
+    <xacro:arg name="config" default="$(find centauro_urdf)/urdf/config/centauro.urdf.xacro"/>
+    <xacro:include filename="$(arg config)"/>
     <group name="base">
         <link name="pelvis"/>

File: centauro_urdf/urdf/centauro.urdf (robot description, URDF)
Before this commit: robot centauro, 84 links, 83 joints
Links:
- removed link D435i_camera_accel_frame
- removed link D435i_camera_accel_optical_frame
- removed link D435i_camera_bottom_screw_frame
- removed link D435i_camera_color_frame
- removed link D435i_camera_color_optical_frame
- removed link D435i_camera_depth_frame
- removed link D435i_camera_depth_optical_frame
- removed link D435i_camera_gyro_frame
- removed link D435i_camera_gyro_optical_frame
- removed link D435i_camera_left_ir_frame
- removed link D435i_camera_left_ir_optical_frame
- removed link D435i_camera_link
- removed link D435i_camera_right_ir_frame
- removed link D435i_camera_right_ir_optical_frame
- removed link T265_camera_accel_frame
- removed link T265_camera_accel_optical_frame
- removed link T265_camera_fisheye1_optical_frame
- removed link T265_camera_fisheye1_rgb_frame
- removed link T265_camera_fisheye2_optical_frame
- removed link T265_camera_fisheye2_rgb_frame
- removed link T265_camera_gyro_frame
- removed link T265_camera_gyro_optical_frame
- removed link T265_camera_link
- removed link T265_camera_pose_frame
- removed link velodyne_calib
- removed link velodyne_calib_base_link
- link ankle1_1: mass 1.2380744 -> 1.4023368; geometry collision mesh filename=package://centauro_urdf/meshes/v2/collision/ankle-pitch.stl scale=0.001 0.001 -0.001; visual mesh filename=package://centauro_urdf/meshes/v2/ankle-pitch.stl scale=0.001 0.001 -0.001
- link ankle1_2: mass 1.2380744 -> 1.4023368; geometry collision mesh filename=package://centauro_urdf/meshes/v2/collision/ankle-pitch.stl scale=0.001 0.001 0.001; visual mesh filename=package://centauro_urdf/meshes/v2/ankle-pitch.stl scale=0.001 0.001 0.001
- link ankle1_3: mass 1.2380744 -> 1.4023368; geometry collision mesh filename=package://centauro_urdf/meshes/v2/collision/ankle-pitch.stl scale=0.001 0.001 -0.001; visual mesh filename=package://centauro_urdf/meshes/v2/ankle-pitch.stl scale=0.001 0.001 -0.001
- link ankle1_4: mass 1.2380744 -> 1.4023368; geometry collision mesh filename=package://centauro_urdf/meshes/v2/collision/ankle-pitch.stl scale=0.001 0.001 0.001; visual mesh filename=package://centauro_urdf/meshes/v2/ankle-pitch.stl scale=0.001 0.001 0.001
- link ankle2_1: mass 1.1565926 -> 1.7656714; geometry collision mesh filename=package://centauro_urdf/meshes/v2/collision/ankle-yaw.stl scale=0.001 -0.001 0.001; visual mesh filename=package://centauro_urdf/meshes/v2/ankle-yaw.stl scale=0.001 -0.001 0.001
- link ankle2_2: mass 1.1565926 -> 1.7656714; geometry collision mesh filename=package://centauro_urdf/meshes/v2/collision/ankle-yaw.stl scale=0.001 0.001 0.001; visual mesh filename=package://centauro_urdf/meshes/v2/ankle-yaw.stl scale=0.001 0.001 0.001
- link ankle2_3: mass 1.1565926 -> 1.7656714; geometry collision mesh filename=package://centauro_urdf/meshes/v2/collision/ankle-yaw.stl scale=0.001 -0.001 0.001; visual mesh filename=package://centauro_urdf/meshes/v2/ankle-yaw.stl scale=0.001 -0.001 0.001
- link ankle2_4: mass 1.1565926 -> 1.7656714; geometry collision mesh filename=package://centauro_urdf/meshes/v2/collision/ankle-yaw.stl scale=0.001 0.001 0.001; visual mesh filename=package://centauro_urdf/meshes/v2/ankle-yaw.stl scale=0.001 0.001 0.001
- link hip1_1: mass 1.9194403 -> 2.3349153; geometry collision mesh filename=package://centauro_urdf/meshes/v2/collision/hip-yaw.stl scale=0.001 -0.001 0.001; visual mesh filename=package://centauro_urdf/meshes/v2/hip-yaw.stl scale=0.001 -0.001 0.001
- link hip1_2: mass 1.9194403 -> 2.3349153; geometry collision mesh filename=package://centauro_urdf/meshes/v2/collision/hip-yaw.stl scale=0.001 0.001 0.001; visual mesh filename=package://centauro_urdf/meshes/v2/hip-yaw.stl scale=0.001 0.001 0.001
- link hip1_3: mass 1.9194403 -> 2.3349153; geometry collision mesh filename=package://centauro_urdf/meshes/v2/collision/hip-yaw.stl scale=0.001 -0.001 0.001; visual mesh filename=package://centauro_urdf/meshes/v2/hip-yaw.stl scale=0.001 -0.001 0.001
- link hip1_4: mass 1.9194403 -> 2.3349153; geometry collision mesh filename=package://centauro_urdf/meshes/v2/collision/hip-yaw.stl scale=0.001 0.001 0.001; visual mesh filename=package://centauro_urdf/meshes/v2/hip-yaw.stl scale=0.001 0.001 0.001
- link hip2_1: mass 2.7264471 -> 3.4572118; geometry collision mesh filename=package://centauro_urdf/meshes/v2/collision/hip-pitch.stl scale=0.001 0.001 -0.001; visual mesh filename=package://centauro_urdf/meshes/v2/hip-pitch.stl scale=0.001 0.001 -0.001
- link hip2_2: mass 2.7264471 -> 3.4572118; geometry collision mesh filename=package://centauro_urdf/meshes/v2/collision/hip-pitch.stl scale=0.001 0.001 0.001; visual mesh filename=package://centauro_urdf/meshes/v2/hip-pitch.stl scale=0.001 0.001 0.001
- link hip2_3: mass 2.7264471 -> 3.4572118; geometry collision mesh filename=package://centauro_urdf/meshes/v2/collision/hip-pitch.stl scale=0.001 0.001 -0.001; visual mesh filename=package://centauro_urdf/meshes/v2/hip-pitch.stl scale=0.001 0.001 -0.001
- link hip2_4: mass 2.7264471 -> 3.4572118; geometry collision mesh filename=package://centauro_urdf/meshes/v2/collision/hip-pitch.stl scale=0.001 0.001 0.001; visual mesh filename=package://centauro_urdf/meshes/v2/hip-pitch.stl scale=0.001 0.001 0.001
- link knee_1: mass 1.9356754 -> 2.1199315; geometry collision mesh filename=package://centauro_urdf/meshes/v2/collision/knee.stl scale=0.001 0.001 -0.001; visual mesh filename=package://centauro_urdf/meshes/v2/knee.stl scale=0.001 0.001 -0.001
- link knee_2: mass 1.9356754 -> 2.1199315; geometry collision mesh filename=package://centauro_urdf/meshes/v2/collision/knee.stl scale=0.001 0.001 0.001; visual mesh filename=package://centauro_urdf/meshes/v2/knee.stl scale=0.001 0.001 0.001
- link knee_3: mass 1.9356754 -> 2.1199315; geometry collision mesh filename=package://centauro_urdf/meshes/v2/collision/knee.stl scale=0.001 0.001 -0.001; visual mesh filename=package://centauro_urdf/meshes/v2/knee.stl scale=0.001 0.001 -0.001
- link knee_4: mass 1.9356754 -> 2.1199315; geometry collision mesh filename=package://centauro_urdf/meshes/v2/collision/knee.stl scale=0.001 0.001 0.001; visual mesh filename=package://centauro_urdf/meshes/v2/knee.stl scale=0.001 0.001 0.001
- link pelvis: mass 16.097574 -> 26.584529; geometry collision mesh filename=package://centauro_urdf/meshes/simple/pelvis.stl scale=0.001 0.001 0.001; visual mesh filename=package://centauro_urdf/meshes/v2/pelvis.stl scale=0.001 0.001 0.001
- link torso_2: mass 11.492689 -> 12.553731
- link wheel_1: mass 1.7289003 -> 1.11164; geometry collision cylinder length=0.11 radius=0.078; visual mesh filename=package://centauro_urdf/meshes/v2/wheel.stl scale=0.001 0.001 -0.001
- link wheel_2: mass 1.7289003 -> 1.11164; geometry collision cylinder length=0.11 radius=0.078; visual mesh filename=package://centauro_urdf/meshes/v2/wheel.stl scale=0.001 0.001 0.001
- link wheel_3: mass 1.7289003 -> 1.11164; geometry collision cylinder length=0.11 radius=0.078; visual mesh filename=package://centauro_urdf/meshes/v2/wheel.stl scale=0.001 0.001 -0.001
- link wheel_4: mass 1.7289003 -> 1.11164; geometry collision cylinder length=0.11 radius=0.078; visual mesh filename=package://centauro_urdf/meshes/v2/wheel.stl scale=0.001 0.001 0.001
Joints:
- removed joint D435i_camera_accel_joint
- removed joint D435i_camera_accel_optical_joint
- removed joint D435i_camera_color_joint
- removed joint D435i_camera_color_optical_joint
- removed joint D435i_camera_depth_joint
- removed joint D435i_camera_depth_optical_joint
- removed joint D435i_camera_gyro_joint
- removed joint D435i_camera_gyro_optical_joint
- removed joint D435i_camera_joint
- removed joint D435i_camera_left_ir_joint
- removed joint D435i_camera_left_ir_optical_joint
- removed joint D435i_camera_link_joint
- removed joint D435i_camera_right_ir_joint
- removed joint D435i_camera_right_ir_optical_joint
- removed joint T265_camera_accel_joint
- removed joint T265_camera_accel_optical_joint
- removed joint T265_camera_fisheye1_optical_joint
- removed joint T265_camera_fisheye1_rgb_joint
- removed joint T265_camera_fisheye2_optical_joint
- removed joint T265_camera_fisheye2_rgb_joint
- removed joint T265_camera_gyro_joint
- removed joint T265_camera_gyro_optical_joint
- removed joint T265_camera_link_joint
- removed joint T265_camera_pose_joint
- removed joint velodyne_calib_base_mount_joint
- removed joint velodyne_calib_base_scan_joint
- joint ankle_pitch_1: axis 0 0 1 -> 0 0 -1; origin xyz=0.2 0.0 -0.10015 rpy=3.14159265359 0.0 0.0 -> xyz=0.0 0.2 0.10015 rpy=3.14159265359 0.0 0.0
- joint ankle_pitch_2: origin xyz=0.2 0.0 -0.10015 rpy=3.14159265359 0.0 0.0 -> xyz=0.0 0.2 -0.10015 rpy=3.14159265359 0.0 0.0
- joint ankle_pitch_3: axis 0 0 1 -> 0 0 -1; origin xyz=0.2 0.0 -0.10015 rpy=3.14159265359 0.0 0.0 -> xyz=0.0 0.2 0.10015 rpy=3.14159265359 0.0 0.0
- joint ankle_pitch_4: origin xyz=0.2 0.0 -0.10015 rpy=3.14159265359 0.0 0.0 -> xyz=0.0 0.2 -0.10015 rpy=3.14159265359 0.0 0.0
- joint ankle_yaw_1: axis 0 0 1 -> 0 0 -1; origin xyz=0.0 0.0 0.0 rpy=1.57079632679 0.0 1.57079632679 -> xyz=0.0 -0.139 -0.00085 rpy=-1.57079632679 0.0 0.0
- joint ankle_yaw_2: axis 0 0 1 -> 0 0 -1; origin xyz=0.0 0.0 0.0 rpy=1.57079632679 0.0 1.57079632679 -> xyz=0.0 -0.139 0.00085 rpy=-1.57079632679 0.0 0.0
- joint ankle_yaw_3: axis 0 0 1 -> 0 0 -1; origin xyz=0.0 0.0 0.0 rpy=1.57079632679 0.0 1.57079632679 -> xyz=0.0 -0.139 -0.00085 rpy=-1.57079632679 0.0 0.0
- joint ankle_yaw_4: axis 0 0 1 -> 0 0 -1; origin xyz=0.0 0.0 0.0 rpy=1.57079632679 0.0 1.57079632679 -> xyz=0.0 -0.139 0.00085 rpy=-1.57079632679 0.0 0.0
- joint contact_joint_1: origin xyz=0 0 0.315 rpy=3.14159265 0 0 -> xyz=0 0 -0.176 rpy=0 0 0
- joint contact_joint_2: origin xyz=0 0 0.315 rpy=3.14159265 0 0 -> xyz=0 0 -0.176 rpy=0 0 0
- joint contact_joint_3: origin xyz=0 0 0.315 rpy=3.14159265 0 0 -> xyz=0 0 -0.176 rpy=0 0 0
- joint contact_joint_4: origin xyz=0 0 0.315 rpy=3.14159265 0 0 -> xyz=0 0 -0.176 rpy=0 0 0
- joint hip_pitch_1: axis 0 0 1 -> 0 0 -1; origin xyz=0.0 0.0 0.0625 rpy=1.57079632679 0.0 0.46141612323 -> xyz=0.0 0.1146 -0.0625 rpy=1.57079632679 0.0 0.0
- joint hip_pitch_2: origin xyz=0.0 0.0 0.0625 rpy=1.57079632679 0.0 2.68017653036 -> xyz=0.0 -0.1146 -0.0625 rpy=1.57079632679 0.0 0.0
- joint hip_pitch_3: axis 0 0 1 -> 0 0 -1; origin xyz=0.0 0.0 0.0625 rpy=1.57079632679 0.0 2.68017653036 -> xyz=0.0 0.1146 -0.0625 rpy=1.57079632679 0.0 0.0
- joint hip_pitch_4: origin xyz=0.0 0.0 0.0625 rpy=1.57079632679 0.0 0.46141612323 -> xyz=0.0 -0.1146 -0.0625 rpy=1.57079632679 0.0 0.0
- joint hip_yaw_1: axis 0 0 1 -> 0 0 -1; origin xyz=0.25 0.125 -0.0566 rpy=3.14159265359 0.0 0.461416123228 -> xyz=0.25 0.125 -0.0566 rpy=0.0 0.0 0.0
- joint hip_yaw_2: axis 0 0 1 -> 0 0 -1; origin xyz=0.25 -0.125 -0.0566 rpy=3.14159265359 0.0 -0.461416123228 -> xyz=0.25 -0.125 -0.0566 rpy=0.0 0.0 0.0
- joint hip_yaw_3: axis 0 0 1 -> 0 0 -1; origin xyz=-0.25 0.125 -0.0566 rpy=3.14159265359 0.0 2.68017653036 -> xyz=-0.25 0.125 -0.0566 rpy=0.0 0.0 0.0
- joint hip_yaw_4: axis 0 0 1 -> 0 0 -1; origin xyz=-0.25 -0.125 -0.0566 rpy=3.14159265359 0.0 3.60300877682 -> xyz=-0.25 -0.125 -0.0566 rpy=0.0 0.0 0.0
- joint j_wheel_1: axis 0 0 1 -> 0 0 -1; origin xyz=0.0 0.00085 0.23735 rpy=1.57079632679 0.0 3.14159265359 -> xyz=0.0 -0.0 -0.09835 rpy=1.57079632679 0.0 0.0
- joint j_wheel_2: origin xyz=0.0 0.00085 0.23735 rpy=1.57079632679 0.0 3.14159265359 -> xyz=0.0 0.0 -0.09835 rpy=1.57079632679 0.0 0.0
- joint j_wheel_3: axis 0 0 1 -> 0 0 -1; origin xyz=0.0 0.00085 0.23735 rpy=1.57079632679 0.0 3.14159265359 -> xyz=0.0 -0.0 -0.09835 rpy=1.57079632679 0.0 0.0
- joint j_wheel_4: origin xyz=0.0 0.00085 0.23735 rpy=1.57079632679 0.0 3.14159265359 -> xyz=0.0 0.0 -0.09835 rpy=1.57079632679 0.0 0.0
- joint knee_pitch_1: axis 0 0 1 -> 0 0 -1; origin xyz=0.0 0.3 -0.0036 rpy=3.14159265359 0.0 1.57079632679 -> xyz=0.0 -0.3 0.1182 rpy=3.14159265359 0.0 0.0
- joint knee_pitch_2: origin xyz=0.0 0.3 -0.0036 rpy=3.14159265359 0.0 1.57079632679 -> xyz=0.0 -0.3 -0.1182 rpy=3.14159265359 0.0 0.0
- joint knee_pitch_3: axis 0 0 1 -> 0 0 -1; origin xyz=0.0 0.3 -0.0036 rpy=3.14159265359 0.0 1.57079632679 -> xyz=0.0 -0.3 0.1182 rpy=3.14159265359 0.0 0.0
- joint knee_pitch_4: origin xyz=0.0 0.3 -0.0036 rpy=3.14159265359 0.0 1.57079632679 -> xyz=0.0 -0.3 -0.1182 rpy=3.14159265359 0.0 0.0

File: centauro_urdf/urdf/centauro.urdf.xacro (robot description, xacro)
@@ -1,6 +1,7 @@
 <?xml version="1.0"?>
 <robot xmlns:xacro="http://ros.org/wiki/xacro" name="centauro">
+<xacro:arg name="config" default="$(find centauro_urdf)/urdf/config/centauro.urdf.xacro"/>
 <!-- ************ MODEL CONFIGURATION ************ -->
-<xacro:include filename="$(find centauro_urdf)/urdf/centauro_config.urdf.xacro" />
+<xacro:include filename="$(arg config)"/>
 <!-- ************ Pholus plain model ************ -->
 <xacro:include filename="$(find centauro_urdf)/urdf/centauro_base.urdf.xacro"/>
@@ -8,4 +9,5 @@
 <!--xacro:include filename="$(find pholus_urdf)/urdf/control_frames.urdf.xacro"/-->
 <xacro:if value="${ADD_FLOATING_BASE}">
+<xacro:if value="${ADD_LEGS}">
 <link name="world"/>
   <joint name="reference" type="floating">
@@ -14,11 +16,5 @@
 </joint>
 </xacro:if>
-<xacro:unless value="${ADD_FLOATING_BASE}">
-<link name="world"/>
-  <joint name="reference" type="fixed">
-    <parent link="world"/>
-    <child link="pelvis"/>
-</joint>
-</xacro:unless>
+</xacro:if>
 <xacro:if value="${ADD_VIRTUAL_FRAME}">
   <xacro:include filename="$(find centauro_urdf)/urdf/parts/virtual_frame.urdf.xacro"/>

File: centauro_urdf/urdf/centauro_robot.urdf.xacro (robot description, xacro)
@@ -12,4 +12,11 @@
   <xacro:include filename="$(find centauro_urdf)/urdf/gazebo/xbot.gazebo.xacro" />
   <xacro:include filename="$(find centauro_urdf)/urdf/gazebo/materials.gazebo.xacro" />
+  <xacro:unless value="${ADD_LEGS}">
+    <link name="world"/>
+      <joint name="reference" type="fixed">
+      <parent link="world"/>
+      <child link="pelvis"/>
+    </joint>
+  </xacro:unless>
   <origin xyz="0.0 0.0 1.2" rpy="0 0 0" />
 </robot>

File: centauro_urdf/urdf/config/centauro.urdf.xacro (robot description, xacro)
@@ -4,16 +4,19 @@
 <xacro:property name="model_version" value="0.1" />
 <!-- command line arguments -->
-<xacro:arg name="add_legs" default="true"/>
-<xacro:arg name="add_upper_body" default="true"/>
+<xacro:arg name="legs" default="true"/>
+<xacro:arg name="upper_body" default="true"/>
+<xacro:arg name="velodyne" default="false"/>
+<xacro:arg name="realsense" default="false"/>
+<xacro:arg name="floating_joint" default="true"/>
 <!-- ************SELECT PARTS*************-->
 <!-- *************************************-->
-<xacro:property name="ADD_LEGS" value="true" />
-<xacro:property name="ADD_UPPER_BODY" value="true" />
+<xacro:property name="ADD_LEGS" value="$(arg legs)" />
+<xacro:property name="ADD_UPPER_BODY" value="$(arg upper_body)" />
 <xacro:property name="ADD_BALL_END_EFFECTOR" value="true" />
-<xacro:property name="ADD_FLOATING_BASE" value="$(arg add_legs)" />
+<xacro:property name="ADD_FLOATING_BASE" value="$(arg floating_joint)" />
 <xacro:property name="ADD_VIRTUAL_FRAME" value="false" />
 <xacro:property name="USE_STICKS" value="false" />
-<xacro:property name="ADD_VELODYNE" value="true" />
-<xacro:property name="ADD_INTEL_D435I" value="true" />
-<xacro:property name="ADD_INTEL_T265" value="true" />
+<xacro:property name="ADD_VELODYNE" value="$(arg velodyne)" />
+<xacro:property name="ADD_INTEL_D435I" value="$(arg realsense)" />
+<xacro:property name="ADD_INTEL_T265" value="$(arg realsense)" />
 </robot>

File: centauro_urdf/urdf/config/centauro_virtual_frame.urdf.xacro (robot description, xacro)
@@ -14,3 +14,6 @@
 <xacro:property name="ADD_VIRTUAL_FRAME" value="true" />
 <xacro:property name="USE_STICKS" value="false" />
+<xacro:property name="ADD_VELODYNE" value="false" />
+<xacro:property name="ADD_INTEL_D435I" value="false" />
+<xacro:property name="ADD_INTEL_T265" value="false" />
 </robot>

Commit message: generates robot_description, robot_description_gz, robot_description_semantic. can handle fixed base case

File: centauro_srdf/srdf/centauro.srdf.xacro (robot description, xacro)
@@ -59,8 +59,8 @@
         <xacro:if value="${ADD_UPPER_BODY}">
             <group name="left_arm" />
-            <group name="right_arm" />
+            <!--group name="right_arm" />
             <group name="torso" />
             <group name="velodyne" />
-            <group name="neck" />
+            <group name="neck" /-->
         </xacro:if>
         <xacro:if value="${ADD_VIRTUAL_FRAME}">

File: centauro_urdf/urdf/centauro.urdf.xacro (robot description, xacro)
@@ -17,4 +17,11 @@
 </xacro:if>
 </xacro:if>
+<xacro:unless value="${ADD_LEGS}">
+<link name="world"/>
+  <joint name="reference" type="fixed">
+    <parent link="world"/>
+    <child link="pelvis"/>
+</joint>
+</xacro:unless>
 <xacro:if value="${ADD_VIRTUAL_FRAME}">
   <xacro:include filename="$(find centauro_urdf)/urdf/parts/virtual_frame.urdf.xacro"/>
