Commit message: srdf takes into account xacro args

File: centauro_srdf/srdf/centauro.srdf.xacro (robot description, xacro)
@@ -52,8 +52,8 @@
     <group name="chains">        <!--THIS HAS TO BE THE LAST GROUP IN THE FILE -->
         <xacro:if value="${ADD_LEGS}">
-            <group name="front_left_leg" />
+            <!--group name="front_left_leg" />
             <group name="front_right_leg" />
             <group name="rear_right_leg" />
-            <group name="rear_left_leg" />
+            <group name="rear_left_leg" /-->
         </xacro:if>
         <xacro:if value="${ADD_UPPER_BODY}">
@@ -70,80 +70,296 @@
     <!-- Homing posture -->
     <group_state name="home" group="chains">
-        <joint name="hip_yaw_1" value="-0.746874"/>
-        <joint name="hip_pitch_1" value="-1.25409"/>
-        <joint name="knee_pitch_1" value="-1.55576"/>
-        <joint name="ankle_pitch_1" value="-0.301666"/>
-        <joint name="ankle_yaw_1" value="0.746874"/>
-        <joint name="hip_yaw_2" value="0.746874"/>
-        <joint name="hip_pitch_2" value="1.25409"/>
-        <joint name="knee_pitch_2" value="1.55576"/>
-        <joint name="ankle_pitch_2" value="0.301666"/>
-        <joint name="ankle_yaw_2" value="-0.746874"/>
-        <joint name="hip_yaw_3" value="0.746874"/>
-        <joint name="hip_pitch_3" value="1.25409"/>
-        <joint name="knee_pitch_3" value="1.55576"/>
-        <joint name="ankle_pitch_3" value="0.301667"/>
-        <joint name="ankle_yaw_3" value="-0.746874"/>
-        <joint name="hip_yaw_4" value="-0.746874"/>
-        <joint name="hip_pitch_4" value="-1.25409"/>
-        <joint name="knee_pitch_4" value="-1.55576"/>
-        <joint name="ankle_pitch_4" value="-0.301667"/>
-        <joint name="ankle_yaw_4" value="0.746874"/>
-        <joint name="torso_yaw" value="3.56617e-13"/>
-        <joint name="neck_yaw" value="0."/>
-        <joint name="neck_pitch" value="0.2"/>
-        <joint name="j_arm1_1" value="0.520149"/>
-        <joint name="j_arm1_2" value="0.320865"/>
-        <joint name="j_arm1_3" value="0.274669"/>
-        <joint name="j_arm1_4" value="-2.23604"/>
-        <joint name="j_arm1_5" value="0.0500815"/>
-        <joint name="j_arm1_6" value="-0.781461"/>
-        <joint name="j_arm1_7" value="-0.0567608"/>
-        <joint name="j_arm2_1" value="0.520149"/>
-        <joint name="j_arm2_2" value="-0.320865"/>
-        <joint name="j_arm2_3" value="-0.274669"/>
-        <joint name="j_arm2_4" value="-2.23604"/>
-        <joint name="j_arm2_5" value="-0.0500815"/>
-        <joint name="j_arm2_6" value="-0.781461"/>
-        <joint name="j_arm2_7" value="0.0567608"/>
+	<xacro:if value="${ADD_LEGS}">
+            <joint name="hip_yaw_1" value="-0.746874"/>
+            <joint name="hip_pitch_1" value="-1.25409"/>
+            <joint name="knee_pitch_1" value="-1.55576"/>
+            <joint name="ankle_pitch_1" value="-0.301666"/>
+            <joint name="ankle_yaw_1" value="0.746874"/>
+            <joint name="hip_yaw_2" value="0.746874"/>
+            <joint name="hip_pitch_2" value="1.25409"/>
+            <joint name="knee_pitch_2" value="1.55576"/>
+            <joint name="ankle_pitch_2" value="0.301666"/>
+            <joint name="ankle_yaw_2" value="-0.746874"/>
+            <joint name="hip_yaw_3" value="0.746874"/>
+            <joint name="hip_pitch_3" value="1.25409"/>
+            <joint name="knee_pitch_3" value="1.55576"/>
+            <joint name="ankle_pitch_3" value="0.301667"/>
+            <joint name="ankle_yaw_3" value="-0.746874"/>
+            <joint name="hip_yaw_4" value="-0.746874"/>
+            <joint name="hip_pitch_4" value="-1.25409"/>
+            <joint name="knee_pitch_4" value="-1.55576"/>
+            <joint name="ankle_pitch_4" value="-0.301667"/>
+            <joint name="ankle_yaw_4" value="0.746874"/>
+	</xacro:if>
+	<xacro:if value="${ADD_UPPER_BODY}">
+            <joint name="torso_yaw" value="3.56617e-13"/>
+            <joint name="neck_yaw" value="0."/>
+            <joint name="neck_pitch" value="0.2"/>
+            <joint name="j_arm1_1" value="0.520149"/>
+            <joint name="j_arm1_2" value="0.320865"/>
+            <joint name="j_arm1_3" value="0.274669"/>
+            <joint name="j_arm1_4" value="-2.23604"/>
+            <joint name="j_arm1_5" value="0.0500815"/>
+            <joint name="j_arm1_6" value="-0.781461"/>
+            <joint name="j_arm1_7" value="-0.0567608"/>
+            <joint name="j_arm2_1" value="0.520149"/>
+            <joint name="j_arm2_2" value="-0.320865"/>
+            <joint name="j_arm2_3" value="-0.274669"/>
+            <joint name="j_arm2_4" value="-2.23604"/>
+            <joint name="j_arm2_5" value="-0.0500815"/>
+            <joint name="j_arm2_6" value="-0.781461"/>
+            <joint name="j_arm2_7" value="0.0567608"/>
+	</xacro:if>
     </group_state>
     <!--DISABLE COLLISIONS: By default it is assumed that any link of the robot could potentially come into collision with any other link in the robot. This tag disables collision checking between a specified pair of links. -->
-    <disable_collisions link1="ankle1_1" link2="ankle2_1" reason="Adjacent" />
-    <disable_collisions link1="ankle1_1" link2="hip1_1" reason="Never" />
-    <disable_collisions link1="ankle1_1" link2="knee_1" reason="Adjacent" />
-    <disable_collisions link1="ankle1_1" link2="wheel_1" reason="Never" />
-    <disable_collisions link1="ankle1_2" link2="ankle2_2" reason="Adjacent" />
-    <disable_collisions link1="ankle1_2" link2="arm1_1" reason="Never" />
-    <disable_collisions link1="ankle1_2" link2="arm2_1" reason="Never" />
-    <disable_collisions link1="ankle1_2" link2="hip1_2" reason="Never" />
-    <disable_collisions link1="ankle1_2" link2="knee_2" reason="Adjacent" />
-    <disable_collisions link1="ankle1_2" link2="wheel_2" reason="Never" />
-    <disable_collisions link1="ankle1_3" link2="ankle2_3" reason="Adjacent" />
-    <disable_collisions link1="ankle1_3" link2="arm1_1" reason="Never" />
-    <disable_collisions link1="ankle1_3" link2="arm2_1" reason="Never" />
-    <disable_collisions link1="ankle1_3" link2="hip1_3" reason="Never" />
-    <disable_collisions link1="ankle1_3" link2="knee_3" reason="Adjacent" />
-    <disable_collisions link1="ankle1_3" link2="wheel_3" reason="Never" />
-    <disable_collisions link1="ankle1_4" link2="ankle2_4" reason="Adjacent" />
-    <disable_collisions link1="ankle1_4" link2="arm1_1" reason="Never" />
-    <disable_collisions link1="ankle1_4" link2="arm2_1" reason="Never" />
-    <disable_collisions link1="ankle1_4" link2="hip1_4" reason="Never" />
-    <disable_collisions link1="ankle1_4" link2="knee_4" reason="Adjacent" />
-    <disable_collisions link1="ankle1_4" link2="wheel_4" reason="Never" />
-    <disable_collisions link1="ankle2_1" link2="knee_1" reason="Never" />
-    <disable_collisions link1="ankle2_1" link2="wheel_1" reason="Adjacent" />
-    <disable_collisions link1="ankle2_2" link2="knee_2" reason="Never" />
-    <disable_collisions link1="ankle2_2" link2="wheel_2" reason="Adjacent" />
-    <disable_collisions link1="ankle2_3" link2="wheel_3" reason="Adjacent" />
-    <disable_collisions link1="ankle2_4" link2="knee_4" reason="Never" />
-    <disable_collisions link1="ankle2_4" link2="wheel_4" reason="Adjacent" />
+<xacro:if value="${ADD_UPPER_BODY}">
+    <disable_collisions link1="arm1_1" link2="torso_2" reason="Adjacent" />
+    <disable_collisions link1="arm1_1" link2="pelvis" reason="Never" />
     <disable_collisions link1="arm1_1" link2="arm1_2" reason="Adjacent" />
     <disable_collisions link1="arm1_1" link2="arm1_3" reason="Never" />
     <disable_collisions link1="arm1_1" link2="arm1_4" reason="Never" />
     <disable_collisions link1="arm1_1" link2="arm1_5" reason="Never" />
+    <disable_collisions link1="arm1_1" link2="arm1_7" reason="Never" />
     <disable_collisions link1="arm1_1" link2="arm2_1" reason="Never" />
     <disable_collisions link1="arm1_1" link2="arm2_2" reason="Never" />
     <disable_collisions link1="arm1_1" link2="arm2_3" reason="Never" />
     <disable_collisions link1="arm1_1" link2="arm2_4" reason="Never" />
+    <disable_collisions link1="arm1_2" link2="arm1_3" reason="Adjacent" />
+    <disable_collisions link1="arm1_2" link2="arm1_4" reason="Never" />
+    <disable_collisions link1="arm1_2" link2="arm2_1" reason="Never" />
+    <disable_collisions link1="arm1_2" link2="arm2_2" reason="Never" />
+    <disable_collisions link1="arm1_2" link2="arm2_3" reason="Never" />
+    <disable_collisions link1="arm1_2" link2="arm2_4" reason="Never" />
+    <disable_collisions link1="arm1_3" link2="arm1_4" reason="Adjacent" />
+    <disable_collisions link1="arm1_3" link2="arm1_6" reason="Never" />
+    <disable_collisions link1="arm1_3" link2="arm1_7" reason="Never" />
+    <disable_collisions link1="arm1_3" link2="arm2_1" reason="Never" />
+    <disable_collisions link1="arm1_3" link2="arm2_2" reason="Never" />
+    <disable_collisions link1="arm1_3" link2="ball1" reason="Never" />
+    <disable_collisions link1="arm1_4" link2="arm1_5" reason="Adjacent" />
+    <disable_collisions link1="arm1_4" link2="arm1_6" reason="Never" />
+    <disable_collisions link1="arm1_4" link2="arm1_7" reason="Never" />
+    <disable_collisions link1="arm1_4" link2="arm2_1" reason="Never" />
+    <disable_collisions link1="arm1_4" link2="arm2_2" reason="Never" />
+    <disable_collisions link1="arm1_4" link2="ball1" reason="Never" />
+    <disable_collisions link1="arm1_5" link2="arm1_6" reason="Adjacent" />
+    <disable_collisions link1="arm1_5" link2="arm1_7" reason="Never" />
+    <disable_collisions link1="arm1_5" link2="ball1" reason="Never" />
+    <disable_collisions link1="arm1_6" link2="arm1_7" reason="Adjacent" />
+    <disable_collisions link1="arm1_6" link2="ball1" reason="Default" />
+    <disable_collisions link1="arm1_7" link2="ball1" reason="Adjacent" />
+    <disable_collisions link1="arm2_1" link2="pelvis" reason="Never" />
+    <disable_collisions link1="arm2_1" link2="torso_2" reason="Adjacent" />
+    <disable_collisions link1="arm2_1" link2="arm2_2" reason="Adjacent" />
+    <disable_collisions link1="arm2_1" link2="arm2_3" reason="Never" />
+    <disable_collisions link1="arm2_1" link2="arm2_4" reason="Never" />
+    <disable_collisions link1="arm2_1" link2="arm2_5" reason="Never" />
+    <disable_collisions link1="arm2_1" link2="arm2_7" reason="Never" />
+    <disable_collisions link1="arm2_2" link2="arm2_3" reason="Adjacent" />
+    <disable_collisions link1="arm2_2" link2="arm2_4" reason="Never" />
+    <disable_collisions link1="arm2_3" link2="arm2_4" reason="Adjacent" />
+    <disable_collisions link1="arm2_3" link2="arm2_6" reason="Never" />
+    <disable_collisions link1="arm2_3" link2="arm2_7" reason="Never" />
+    <disable_collisions link1="arm2_3" link2="ball2" reason="Never" />
+    <disable_collisions link1="arm2_4" link2="arm2_5" reason="Adjacent" />
+    <disable_collisions link1="arm2_4" link2="arm2_6" reason="Never" />
+    <disable_collisions link1="arm2_4" link2="arm2_7" reason="Never" />
+    <disable_collisions link1="arm2_4" link2="ball2" reason="Never" />
+    <disable_collisions link1="arm2_5" link2="arm2_6" reason="Adjacent" />
+    <disable_collisions link1="arm2_5" link2="arm2_7" reason="Never" />
+    <disable_collisions link1="arm2_5" link2="ball2" reason="Never" />
+    <disable_collisions link1="arm2_6" link2="arm2_7" reason="Adjacent" />
+    <disable_collisions link1="arm2_6" link2="ball2" reason="Default" />
+    <disable_collisions link1="arm2_7" link2="ball2" reason="Adjacent" />
+    <disable_collisions link1="arm1_1" link2="neck_1" reason="Never" />
+    <disable_collisions link1="arm1_1" link2="neck_2" reason="Never" />
+    <disable_collisions link1="arm1_1" link2="neck_3" reason="Never" />
+    <disable_collisions link1="arm1_2" link2="neck_1" reason="Never" />
+    <disable_collisions link1="arm1_2" link2="neck_2" reason="Never" />
+    <disable_collisions link1="arm1_2" link2="neck_3" reason="Never" />
+    <disable_collisions link1="arm1_3" link2="neck_1" reason="Never" />
+    <disable_collisions link1="arm1_3" link2="neck_3" reason="Never" />
+    <disable_collisions link1="arm2_1" link2="neck_1" reason="Never" />
+    <disable_collisions link1="arm2_1" link2="neck_2" reason="Never" />
+    <disable_collisions link1="arm2_1" link2="neck_3" reason="Never" />
+    <disable_collisions link1="arm2_2" link2="neck_1" reason="Never" />
+    <disable_collisions link1="arm2_2" link2="neck_2" reason="Never" />
+    <disable_collisions link1="arm2_2" link2="neck_3" reason="Never" />
+    <disable_collisions link1="arm2_3" link2="neck_1" reason="Never" />
+    <disable_collisions link1="arm2_3" link2="neck_3" reason="Never" />
+    <disable_collisions link1="neck_1" link2="neck_2" reason="Adjacent" />
+    <disable_collisions link1="neck_1" link2="neck_3" reason="Never" />
+    <disable_collisions link1="neck_2" link2="neck_3" reason="Never" />
+    <disable_collisions link1="neck_3" link2="torso_2" reason="Adjacent" />
+    <disable_collisions link1="neck_1" link2="torso_2" reason="Adjacent" />
+    <disable_collisions link1="neck_1" link2="pelvis" reason="Never" />
+    <disable_collisions link1="neck_2" link2="pelvis" reason="Never" />
+    <disable_collisions link1="neck_3" link2="pelvis" reason="Never" />
+    <disable_collisions link1="pelvis" link2="torso_2" reason="Adjacent" />
+    <xacro:if value="${ADD_INTEL_D435I}">
+    <disable_collisions link1="D435i_camera_link" link2="D435i_head_camera_link" reason="Never" />
+    <disable_collisions link1="D435i_camera_link" link2="pelvis" reason="Adjacent" />
+    <disable_collisions link1="D435i_head_camera_link" link2="pelvis" reason="Never" />
+    <disable_collisions link1="D435i_camera_link" link2="arm1_1" reason="Never" />
+    <disable_collisions link1="D435i_camera_link" link2="arm1_2" reason="Never" />
+    <disable_collisions link1="D435i_camera_link" link2="arm1_3" reason="Never" />
+    <disable_collisions link1="D435i_camera_link" link2="arm1_4" reason="Never" />
+    <disable_collisions link1="D435i_camera_link" link2="arm2_1" reason="Never" />
+    <disable_collisions link1="D435i_camera_link" link2="arm2_2" reason="Never" />
+    <disable_collisions link1="D435i_camera_link" link2="arm2_3" reason="Never" />
+    <disable_collisions link1="D435i_camera_link" link2="arm2_4" reason="Never" />
+    <disable_collisions link1="D435i_camera_link" link2="neck_1" reason="Never" />
+    <disable_collisions link1="D435i_camera_link" link2="neck_2" reason="Never" />
+    <disable_collisions link1="D435i_camera_link" link2="neck_3" reason="Never" />
+    <disable_collisions link1="D435i_camera_link" link2="torso_2" reason="Never" />
+    <disable_collisions link1="D435i_head_camera_link" link2="arm1_1" reason="Never" />
+    <disable_collisions link1="D435i_head_camera_link" link2="arm2_1" reason="Never" />
+    <disable_collisions link1="D435i_head_camera_link" link2="neck_1" reason="Never" />
+    <disable_collisions link1="D435i_head_camera_link" link2="neck_2" reason="Adjacent" />
+    <disable_collisions link1="D435i_head_camera_link" link2="neck_3" reason="Never" />
+    <xacro:if value="${ADD_INTEL_T265}">
+    <disable_collisions link1="D435i_camera_link" link2="T265_camera_pose_frame" reason="Never" />
+    <disable_collisions link1="D435i_head_camera_link" link2="T265_camera_pose_frame" reason="Never" />
+    </xacro:if>
+    <xacro:if value="${ADD_VELODYNE}">
+    <disable_collisions link1="D435i_camera_link" link2="velodyne_calib" reason="Never" />
+    <disable_collisions link1="D435i_camera_link" link2="velodyne_calib_base_link" reason="Never" />
+    <disable_collisions link1="D435i_head_camera_link" link2="velodyne_calib" reason="Never" />
+    <disable_collisions link1="D435i_head_camera_link" link2="velodyne_calib_base_link" reason="Never" />
+    </xacro:if>
+    <xacro:if value="${ADD_LEGS}">
+    <disable_collisions link1="D435i_camera_link" link2="hip1_1" reason="Never" />
+    <disable_collisions link1="D435i_camera_link" link2="hip1_2" reason="Never" />
+    <disable_collisions link1="D435i_camera_link" link2="hip1_3" reason="Never" />
+    <disable_collisions link1="D435i_camera_link" link2="hip1_4" reason="Never" />
+    <disable_collisions link1="D435i_camera_link" link2="hip2_3" reason="Never" />
+    <disable_collisions link1="D435i_camera_link" link2="hip2_4" reason="Never" />
+    <disable_collisions link1="D435i_head_camera_link" link2="ankle1_1" reason="Never" />
+    <disable_collisions link1="D435i_head_camera_link" link2="ankle1_2" reason="Never" />
+    <disable_collisions link1="D435i_head_camera_link" link2="ankle1_3" reason="Never" />
+    <disable_collisions link1="D435i_head_camera_link" link2="ankle1_4" reason="Never" />
+    <disable_collisions link1="D435i_head_camera_link" link2="ankle2_3" reason="Never" />
+    <disable_collisions link1="D435i_head_camera_link" link2="hip1_1" reason="Never" />
+    <disable_collisions link1="D435i_head_camera_link" link2="hip1_2" reason="Never" />
+    <disable_collisions link1="D435i_head_camera_link" link2="hip1_3" reason="Never" />
+    <disable_collisions link1="D435i_head_camera_link" link2="hip1_4" reason="Never" />
+    <disable_collisions link1="D435i_head_camera_link" link2="hip2_1" reason="Never" />
+    <disable_collisions link1="D435i_head_camera_link" link2="hip2_2" reason="Never" />
+    <disable_collisions link1="D435i_head_camera_link" link2="hip2_3" reason="Never" />
+    <disable_collisions link1="D435i_head_camera_link" link2="hip2_4" reason="Never" />
+    <disable_collisions link1="D435i_head_camera_link" link2="knee_1" reason="Never" />
+    <disable_collisions link1="D435i_head_camera_link" link2="knee_2" reason="Never" />
+    <disable_collisions link1="D435i_head_camera_link" link2="knee_3" reason="Never" />
+    <disable_collisions link1="D435i_head_camera_link" link2="knee_4" reason="Never" />
+    <disable_collisions link1="D435i_head_camera_link" link2="wheel_3" reason="Never" />
+    </xacro:if>
+    </xacro:if>
+    <xacro:if value="${ADD_INTEL_T265}">
+    <disable_collisions link1="T265_camera_pose_frame" link2="pelvis" reason="Adjacent" />
+    <disable_collisions link1="T265_camera_pose_frame" link2="arm1_1" reason="Never" />
+    <disable_collisions link1="T265_camera_pose_frame" link2="arm1_2" reason="Never" />
+    <disable_collisions link1="T265_camera_pose_frame" link2="arm1_3" reason="Never" />
+    <disable_collisions link1="T265_camera_pose_frame" link2="arm1_4" reason="Never" />
+    <disable_collisions link1="T265_camera_pose_frame" link2="arm2_1" reason="Never" />
+    <disable_collisions link1="T265_camera_pose_frame" link2="arm2_2" reason="Never" />
+    <disable_collisions link1="T265_camera_pose_frame" link2="arm2_3" reason="Never" />
+    <disable_collisions link1="T265_camera_pose_frame" link2="arm2_4" reason="Never" />
+    <disable_collisions link1="T265_camera_pose_frame" link2="neck_1" reason="Never" />
+    <disable_collisions link1="T265_camera_pose_frame" link2="neck_2" reason="Never" />
+    <disable_collisions link1="T265_camera_pose_frame" link2="neck_3" reason="Never" />
+    <disable_collisions link1="T265_camera_pose_frame" link2="torso_2" reason="Never" />
+    <xacro:if value="${ADD_VELODYNE}">
+    <disable_collisions link1="T265_camera_pose_frame" link2="velodyne_calib" reason="Never" />
+    <disable_collisions link1="T265_camera_pose_frame" link2="velodyne_calib_base_link" reason="Never" />
+    </xacro:if>
+    <xacro:if value="${ADD_LEGS}">
+    <disable_collisions link1="T265_camera_pose_frame" link2="hip1_1" reason="Never" />
+    <disable_collisions link1="T265_camera_pose_frame" link2="hip1_2" reason="Never" />
+    <disable_collisions link1="T265_camera_pose_frame" link2="hip1_3" reason="Never" />
+    <disable_collisions link1="T265_camera_pose_frame" link2="hip1_4" reason="Never" />
+    <disable_collisions link1="T265_camera_pose_frame" link2="hip2_3" reason="Never" />
+    <disable_collisions link1="T265_camera_pose_frame" link2="hip2_4" reason="Never" />
+    </xacro:if>
+    </xacro:if>
+    <xacro:if value="${ADD_VELODYNE}">
+    <disable_collisions link1="pelvis" link2="velodyne_calib" reason="Never" />
+    <disable_collisions link1="pelvis" link2="velodyne_calib_base_link" reason="Never" />
+    <disable_collisions link1="velodyne_calib" link2="velodyne_calib_base_link" reason="Adjacent" />
+    <disable_collisions link1="arm1_1" link2="velodyne_calib" reason="Never" />
+    <disable_collisions link1="arm1_1" link2="velodyne_calib_base_link" reason="Never" />
+    <disable_collisions link1="arm1_2" link2="velodyne_calib" reason="Never" />
+    <disable_collisions link1="arm1_2" link2="velodyne_calib_base_link" reason="Never" />
+    <disable_collisions link1="arm1_3" link2="velodyne_calib" reason="Never" />
+    <disable_collisions link1="arm1_3" link2="velodyne_calib_base_link" reason="Never" />
+    <disable_collisions link1="arm2_1" link2="velodyne_calib" reason="Never" />
+    <disable_collisions link1="arm2_1" link2="velodyne_calib_base_link" reason="Never" />
+    <disable_collisions link1="arm2_2" link2="velodyne_calib" reason="Never" />
+    <disable_collisions link1="arm2_2" link2="velodyne_calib_base_link" reason="Never" />
+    <disable_collisions link1="arm2_3" link2="velodyne_calib" reason="Never" />
+    <disable_collisions link1="arm2_3" link2="velodyne_calib_base_link" reason="Never" />
+    <disable_collisions link1="neck_1" link2="velodyne_calib" reason="Never" />
+    <disable_collisions link1="neck_1" link2="velodyne_calib_base_link" reason="Never" />
+    <disable_collisions link1="neck_2" link2="velodyne_calib" reason="Never" />
+    <disable_collisions link1="neck_2" link2="velodyne_calib_base_link" reason="Never" />
+    <disable_collisions link1="neck_3" link2="velodyne_calib" reason="Never" />
+    <disable_collisions link1="neck_3" link2="velodyne_calib_base_link" reason="Adjacent" />
+    <disable_collisions link1="torso_2" link2="velodyne_calib" reason="Never" />
+    <disable_collisions link1="torso_2" link2="velodyne_calib_base_link" reason="Never" />
+    <xacro:if value="${ADD_LEGS}">
+    <disable_collisions link1="ankle1_1" link2="velodyne_calib" reason="Never" />
+    <disable_collisions link1="ankle1_1" link2="velodyne_calib_base_link" reason="Never" />
+    <disable_collisions link1="ankle1_2" link2="velodyne_calib" reason="Never" />
+    <disable_collisions link1="ankle1_2" link2="velodyne_calib_base_link" reason="Never" />
+    <disable_collisions link1="ankle1_3" link2="velodyne_calib" reason="Never" />
+    <disable_collisions link1="ankle1_3" link2="velodyne_calib_base_link" reason="Never" />
+    <disable_collisions link1="ankle1_4" link2="velodyne_calib" reason="Never" />
+    <disable_collisions link1="ankle1_4" link2="velodyne_calib_base_link" reason="Never" />
+    <disable_collisions link1="ankle2_1" link2="velodyne_calib" reason="Never" />
+    <disable_collisions link1="ankle2_1" link2="velodyne_calib_base_link" reason="Never" />
+    <disable_collisions link1="ankle2_2" link2="velodyne_calib" reason="Never" />
+    <disable_collisions link1="ankle2_2" link2="velodyne_calib_base_link" reason="Never" />
+    <disable_collisions link1="ankle2_3" link2="velodyne_calib" reason="Never" />
+    <disable_collisions link1="ankle2_3" link2="velodyne_calib_base_link" reason="Never" />
+    <disable_collisions link1="ankle2_4" link2="velodyne_calib" reason="Never" />
+    <disable_collisions link1="ankle2_4" link2="velodyne_calib_base_link" reason="Never" />
+    <disable_collisions link1="hip1_1" link2="velodyne_calib" reason="Never" />
+    <disable_collisions link1="hip1_1" link2="velodyne_calib_base_link" reason="Never" />
+    <disable_collisions link1="hip1_2" link2="velodyne_calib" reason="Never" />
+    <disable_collisions link1="hip1_2" link2="velodyne_calib_base_link" reason="Never" />
+    <disable_collisions link1="hip1_3" link2="velodyne_calib" reason="Never" />
+    <disable_collisions link1="hip1_3" link2="velodyne_calib_base_link" reason="Never" />
+    <disable_collisions link1="hip1_4" link2="velodyne_calib" reason="Never" />
+    <disable_collisions link1="hip1_4" link2="velodyne_calib_base_link" reason="Never" />
+    <disable_collisions link1="hip2_1" link2="velodyne_calib" reason="Never" />
+    <disable_collisions link1="hip2_1" link2="velodyne_calib_base_link" reason="Never" />
+    <disable_collisions link1="hip2_2" link2="velodyne_calib" reason="Never" />
+    <disable_collisions link1="hip2_2" link2="velodyne_calib_base_link" reason="Never" />
+    <disable_collisions link1="hip2_3" link2="velodyne_calib" reason="Never" />
+    <disable_collisions link1="hip2_3" link2="velodyne_calib_base_link" reason="Never" />
+    <disable_collisions link1="hip2_4" link2="velodyne_calib" reason="Never" />
+    <disable_collisions link1="hip2_4" link2="velodyne_calib_base_link" reason="Never" />
+    <disable_collisions link1="knee_1" link2="velodyne_calib" reason="Never" />
+    <disable_collisions link1="knee_1" link2="velodyne_calib_base_link" reason="Never" />
+    <disable_collisions link1="knee_2" link2="velodyne_calib" reason="Never" />
+    <disable_collisions link1="knee_2" link2="velodyne_calib_base_link" reason="Never" />
+    <disable_collisions link1="knee_3" link2="velodyne_calib" reason="Never" />
+    <disable_collisions link1="knee_3" link2="velodyne_calib_base_link" reason="Never" />
+    <disable_collisions link1="knee_4" link2="velodyne_calib" reason="Never" />
+    <disable_collisions link1="knee_4" link2="velodyne_calib_base_link" reason="Never" />
+    <disable_collisions link1="velodyne_calib" link2="wheel_1" reason="Never" />
+    <disable_collisions link1="velodyne_calib" link2="wheel_2" reason="Never" />
+    <disable_collisions link1="velodyne_calib" link2="wheel_3" reason="Never" />
+    <disable_collisions link1="velodyne_calib" link2="wheel_4" reason="Never" />
+    <disable_collisions link1="velodyne_calib_base_link" link2="wheel_1" reason="Never" />
+    <disable_collisions link1="velodyne_calib_base_link" link2="wheel_2" reason="Never" />
+    <disable_collisions link1="velodyne_calib_base_link" link2="wheel_3" reason="Never" />
+    <disable_collisions link1="velodyne_calib_base_link" link2="wheel_4" reason="Never" />
+    </xacro:if>
+    </xacro:if>
+    <xacro:if value="${ADD_LEGS}">
+    <disable_collisions link1="ankle1_2" link2="arm1_1" reason="Never" />
+    <disable_collisions link1="ankle1_2" link2="arm2_1" reason="Never" />
+    <disable_collisions link1="ankle1_3" link2="arm2_1" reason="Never" />
+    <disable_collisions link1="ankle1_4" link2="arm1_1" reason="Never" />
     <disable_collisions link1="arm1_1" link2="hip1_1" reason="Never" />
     <disable_collisions link1="arm1_1" link2="hip1_2" reason="Never" />
@@ -158,13 +374,4 @@
     <disable_collisions link1="arm1_1" link2="knee_3" reason="Never" />
     <disable_collisions link1="arm1_1" link2="knee_4" reason="Never" />
-    <disable_collisions link1="arm1_1" link2="pelvis" reason="Never" />
-    <disable_collisions link1="arm1_1" link2="torso_2" reason="Adjacent" />
-    <disable_collisions link1="arm1_2" link2="arm1_3" reason="Adjacent" />
-    <disable_collisions link1="arm1_2" link2="arm1_4" reason="Never" />
-    <disable_collisions link1="arm1_2" link2="arm1_7" reason="Never" />
-    <disable_collisions link1="arm1_2" link2="arm2_1" reason="Never" />
-    <disable_collisions link1="arm1_2" link2="arm2_2" reason="Never" />
-    <disable_collisions link1="arm1_2" link2="arm2_3" reason="Never" />
-    <disable_collisions link1="arm1_2" link2="arm2_4" reason="Never" />
     <disable_collisions link1="arm1_2" link2="hip1_1" reason="Never" />
     <disable_collisions link1="arm1_2" link2="hip1_2" reason="Never" />
@@ -175,39 +382,15 @@
     <disable_collisions link1="arm1_2" link2="hip2_3" reason="Never" />
     <disable_collisions link1="arm1_2" link2="hip2_4" reason="Never" />
-    <disable_collisions link1="arm1_2" link2="knee_1" reason="Never" />
-    <disable_collisions link1="arm1_2" link2="knee_4" reason="Never" />
-    <disable_collisions link1="arm1_3" link2="arm1_4" reason="Adjacent" />
-    <disable_collisions link1="arm1_3" link2="arm1_6" reason="Never" />
-    <disable_collisions link1="arm1_3" link2="arm1_7" reason="Never" />
-    <disable_collisions link1="arm1_3" link2="arm2_1" reason="Never" />
-    <disable_collisions link1="arm1_3" link2="arm2_2" reason="Never" />
-    <disable_collisions link1="arm1_3" link2="ft_arm1" reason="Never" />
+    <disable_collisions link1="arm1_2" link2="knee_2" reason="Never" />
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