Commit message: srdf takes into account xacro args

File: centauro_urdf/urdf/centauro.urdf.xacro (robot description, xacro)
@@ -17,5 +17,5 @@
 </xacro:if>
 </xacro:if>
-<xacro:unless value="${ADD_LEGS}">
+<xacro:unless value="${ADD_FLOATING_BASE}">
 <link name="world"/>
   <joint name="reference" type="fixed">

File: centauro_urdf/urdf/parts/head.urdf.xacro (robot description, xacro)
@@ -34,10 +34,10 @@
       </geometry>
     </visual>
-    <collision>
+    <!--collision>
       <origin rpy="0.0 0.0 0.0" xyz="0.0 0 0.0"/>
       <geometry>
         <mesh filename="package://centauro_urdf/meshes/simple/neck_pitch.stl" scale="0.001 0.001 0.001"/>
       </geometry>
-    </collision>
+    </collision-->
 </link>
 <!-- LINKS -->
@@ -107,5 +107,5 @@
                       color_height="720"
                       color_fps="30">
-            <origin xyz="0.219831 0 -0.0613293" rpy="0.0 0.5585052 0.0"/>
+            <origin xyz="0.11 -0.05 0.0" rpy="0.0 0.0 0.0"/>
         </xacro:sensor_d435i>
     </xacro:if>
