Commit message: Change sensor location. Missing: inertia/mass and joint_map for head d435. Velodyne to correct

File: centauro_srdf/srdf/centauro.srdf.xacro (robot description, xacro)
@@ -35,13 +35,18 @@
     <group name="torso">
         <chain base_link="pelvis" tip_link="torso_2" />
-    </group>
+    </group><!--
     <group name="neck">
     	<chain base_link="torso_2" tip_link="neck_2" />
-    </group>
-</xacro:if>
-<xacro:if value="${ADD_VELODYNE}">
-    <group name="velodyne">
-    	<chain base_link="torso_2" tip_link="neck_3" />
-    </group>
+    </group>-->
+    <xacro:if value="${ADD_VELODYNE}">
+        <group name="velodyne">
+            <chain base_link="torso_2" tip_link="velodyne_motor" />
+        </group>
+    </xacro:if>
+    <xacro:if value="${ADD_D435_HEAD}">
+        <group name="d435_head">
+            <chain base_link="torso_2" tip_link="d435_head_motor" />
+        </group>
+    </xacro:if>
 </xacro:if>
 <xacro:if value="${ADD_VIRTUAL_FRAME}">
@@ -61,8 +66,10 @@
         <group name="right_arm" />
         <group name="torso" />
-        <group name="neck" />
-    </xacro:if>
-    <xacro:if value="${ADD_VELODYNE}">
-        <group name="velodyne"/>
+        <xacro:if value="${ADD_VELODYNE}">
+            <group name="velodyne"/>
+        </xacro:if>
+        <xacro:if value="${ADD_D435_HEAD}">
+            <group name="d435_head"/>
+        </xacro:if>
     </xacro:if>
     <xacro:if value="${ADD_VIRTUAL_FRAME}">
@@ -93,6 +100,6 @@
 	<joint name="ankle_yaw_4" value="0.746874"/>
 	<joint name="torso_yaw" value="3.56617e-13"/>
-	<joint name="neck_yaw" value="0."/>
-	<joint name="neck_pitch" value="0.2"/>
+	<joint name="velodyne_joint" value="0"/>
+	<joint name="d435_head_joint" value="0"/>
 	<joint name="j_arm1_1" value="0.520149"/>
 	<joint name="j_arm1_2" value="0.320865"/>

File: centauro_urdf/urdf/_centauro_robot.urdf (robot description, URDF)
Before this commit: robot centauro, 60 links, 59 joints
Links:
- removed link neck_2
- removed link neck_3
- added link D435_head_camera_accel_frame
- added link D435_head_camera_accel_optical_frame
- added link D435_head_camera_bottom_screw_frame
- added link D435_head_camera_color_frame
- added link D435_head_camera_color_optical_frame
- added link D435_head_camera_depth_frame
- added link D435_head_camera_depth_optical_frame
- added link D435_head_camera_gyro_frame
- added link D435_head_camera_gyro_optical_frame
- added link D435_head_camera_left_ir_frame
- added link D435_head_camera_left_ir_optical_frame
- added link D435_head_camera_link, mass 0.564; collision box size=0.02505 0.09 0.025; visual mesh filename=package://realsense2_description/meshes/d435.dae
- added link D435_head_camera_right_ir_frame
- added link D435_head_camera_right_ir_optical_frame
- added link D435i_camera_accel_frame
- added link D435i_camera_accel_optical_frame
- added link D435i_camera_bottom_screw_frame
- added link D435i_camera_color_frame
- added link D435i_camera_color_optical_frame
- added link D435i_camera_depth_frame
- added link D435i_camera_depth_optical_frame
- added link D435i_camera_gyro_frame
- added link D435i_camera_gyro_optical_frame
- added link D435i_camera_left_ir_frame
- added link D435i_camera_left_ir_optical_frame
- added link D435i_camera_link, mass 0.564; collision box size=0.02505 0.09 0.025; visual mesh filename=package://realsense2_description/meshes/d435.dae
- added link D435i_camera_right_ir_frame
- added link D435i_camera_right_ir_optical_frame
- added link T265_camera_accel_frame
- added link T265_camera_accel_optical_frame
- added link T265_camera_fisheye1_optical_frame
- added link T265_camera_fisheye1_rgb_frame
- added link T265_camera_fisheye2_optical_frame
- added link T265_camera_fisheye2_rgb_frame
- added link T265_camera_gyro_frame
- added link T265_camera_gyro_optical_frame
- added link T265_camera_link
- added link T265_camera_pose_frame, mass 0.068024; collision mesh filename=package://realsense_gazebo_description/meshes/t265_simplifi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 scale=0.001 0.001 0.001; visual mesh filename=package://realsense_gazebo_description/meshes/t265_full.stl scale=0.001 0.001 0.001
- added link d435_head_motor, mass 0.33878686; collision mesh filename=package://centauro_urdf/meshes/simple/neck-pitch_mesh.stl scale=0.001 0.001 0.001; visual mesh filename=package://centauro_urdf/meshes/neck-pitch_mesh.stl scale=0.001 0.001 0.001
- added link velodyne_motor, mass 0.33878686; collision mesh filename=package://centauro_urdf/meshes/simple/lidar_mesh.stl scale=0.001 0.001 0.001; visual mesh filename=package://centauro_urdf/meshes/lidar_mesh.stl scale=0.001 0.001 0.001
- link neck_1: geometry collision mesh filename=package://centauro_urdf/meshes/simple/head-base_mesh.stl scale=0.001 0.001 0.001; visual mesh filename=package://centauro_urdf/meshes/head-base_mesh.stl scale=0.001 0.001 0.001
- link torso_2: geometry collision mesh filename=package://centauro_urdf/meshes/simple/link1_no_head.stl scale=0.001 0.001 0.001; visual mesh filename=package://centauro_urdf/meshes/link1_no_head.stl scale=0.001 0.001 0.001
Joints:
- removed joint neck_pitch
- removed joint neck_velodyne
- removed joint neck_yaw
- added joint D435_head_camera_accel_joint: type fixed, parent D435_head_camera_link, child D435_head_camera_accel_frame, origin xyz=-0.00174 0.00552 0.0176 rpy=0 0 0
- added joint D435_head_camera_accel_optical_joint: type fixed, parent D435_head_camera_accel_frame, child D435_head_camera_accel_optical_frame, origin xyz=0 0 0 rpy=-1.57079632679 0 -1.57079632679
- added joint D435_head_camera_color_joint: type fixed, parent D435_head_camera_depth_frame, child D435_head_camera_color_frame, origin xyz=0 0.015 0 rpy=0 0 0
- added joint D435_head_camera_color_optical_joint: type fixed, parent D435_head_camera_color_frame, child D435_head_camera_color_optical_frame, origin xyz=0 0 0 rpy=-1.57079632679 0 -1.57079632679
- added joint D435_head_camera_depth_joint: type fixed, parent D435_head_camera_link, child D435_head_camera_depth_frame, origin xyz=0 0 0 rpy=0 0 0
- added joint D435_head_camera_depth_optical_joint: type fixed, parent D435_head_camera_depth_frame, child D435_head_camera_depth_optical_frame, origin xyz=0 0 0 rpy=-1.57079632679 0 -1.57079632679
- added joint D435_head_camera_gyro_joint: type fixed, parent D435_head_camera_link, child D435_head_camera_gyro_frame, origin xyz=-0.00174 0.00552 0.0176 rpy=0 0 0
- added joint D435_head_camera_gyro_optical_joint: type fixed, parent D435_head_camera_gyro_frame, child D435_head_camera_gyro_optical_frame, origin xyz=0 0 0 rpy=-1.57079632679 0 -1.57079632679
- added joint D435_head_camera_joint: type fixed, parent d435_head_motor, child D435_head_camera_bottom_screw_frame, origin xyz=0.03015 0 -0.0125 rpy=0 0 0
- added joint D435_head_camera_left_ir_joint: type fixed, parent D435_head_camera_depth_frame, child D435_head_camera_left_ir_frame, origin xyz=0 0.0 0 rpy=0 0 0
- added joint D435_head_camera_left_ir_optical_joint: type fixed, parent D435_head_camera_left_ir_frame, child D435_head_camera_left_ir_optical_frame, origin xyz=0 0 0 rpy=-1.57079632679 0 -1.57079632679
- added joint D435_head_camera_link_joint: type fixed, parent D435_head_camera_bottom_screw_frame, child D435_head_camera_link, origin xyz=0 0.0175 0.0125 rpy=0 0 0
- added joint D435_head_camera_right_ir_joint: type fixed, parent D435_head_camera_depth_frame, child D435_head_camera_right_ir_frame, origin xyz=0 -0.05 0 rpy=0 0 0
- added joint D435_head_camera_right_ir_optical_joint: type fixed, parent D435_head_camera_right_ir_frame, child D435_head_camera_right_ir_optical_frame, origin xyz=0 0 0 rpy=-1.57079632679 0 -1.57079632679
- added joint D435i_camera_accel_joint: type fixed, parent D435i_camera_link, child D435i_camera_accel_frame, origin xyz=-0.00174 0.00552 0.0176 rpy=0 0 0
- added joint D435i_camera_accel_optical_joint: type fixed, parent D435i_camera_accel_frame, child D435i_camera_accel_optical_frame, origin xyz=0 0 0 rpy=-1.57079632679 0 -1.57079632679
- added joint D435i_camera_color_joint: type fixed, parent D435i_camera_depth_frame, child D435i_camera_color_frame, origin xyz=0 0.015 0 rpy=0 0 0
- added joint D435i_camera_color_optical_joint: type fixed, parent D435i_camera_color_frame, child D435i_camera_color_optical_frame, origin xyz=0 0 0 rpy=-1.57079632679 0 -1.57079632679
- added joint D435i_camera_depth_joint: type fixed, parent D435i_camera_link, child D435i_camera_depth_frame, origin xyz=0 0 0 rpy=0 0 0
- added joint D435i_camera_depth_optical_joint: type fixed, parent D435i_camera_depth_frame, child D435i_camera_depth_optical_frame, origin xyz=0 0 0 rpy=-1.57079632679 0 -1.57079632679
- added joint D435i_camera_gyro_joint: type fixed, parent D435i_camera_link, child D435i_camera_gyro_frame, origin xyz=-0.00174 0.00552 0.0176 rpy=0 0 0
- added joint D435i_camera_gyro_optical_joint: type fixed, parent D435i_camera_gyro_frame, child D435i_camera_gyro_optical_frame, origin xyz=0 0 0 rpy=-1.57079632679 0 -1.57079632679
- added joint D435i_camera_joint: type fixed, parent pelvis, child D435i_camera_bottom_screw_frame, origin xyz=0.27187 0 0.0215997 rpy=0 0.5251508 0
- added joint D435i_camera_left_ir_joint: type fixed, parent D435i_camera_depth_frame, child D435i_camera_left_ir_frame, origin xyz=0 0.0 0 rpy=0 0 0
- added joint D435i_camera_left_ir_optical_joint: type fixed, parent D435i_camera_left_ir_frame, child D435i_camera_left_ir_optical_frame, origin xyz=0 0 0 rpy=-1.57079632679 0 -1.57079632679
- added joint D435i_camera_link_joint: type fixed, parent D435i_camera_bottom_screw_frame, child D435i_camera_link, origin xyz=0 0.0175 0.0125 rpy=0 0 0
- added joint D435i_camera_right_ir_joint: type fixed, parent D435i_camera_depth_frame, child D435i_camera_right_ir_frame, origin xyz=0 -0.05 0 rpy=0 0 0
- added joint D435i_camera_right_ir_optical_joint: type fixed, parent D435i_camera_right_ir_frame, child D435i_camera_right_ir_optical_frame, origin xyz=0 0 0 rpy=-1.57079632679 0 -1.57079632679
- added joint T265_camera_accel_joint: type fixed, parent T265_camera_link, child T265_camera_accel_frame, origin xyz=-0.0311 0 0.00655 rpy=0 3.14159265359 0
- added joint T265_camera_accel_optical_joint: type fixed, parent T265_camera_accel_frame, child T265_camera_accel_optical_frame, origin xyz=-0.0311 0 0.00655 rpy=0 3.14159265359 0
- added joint T265_camera_fisheye1_optical_joint: type fixed, parent T265_camera_fisheye1_rgb_frame, child T265_camera_fisheye1_optical_frame, origin xyz=0 0 0 rpy=-1.57079632679 0 -1.57079632679
- added joint T265_camera_fisheye1_rgb_joint: type fixed, parent T265_camera_link, child T265_camera_fisheye1_rgb_frame, origin xyz=-0.0411 0.0 0.0 rpy=0 1.57079632679 1.57079632679
- added joint T265_camera_fisheye2_optical_joint: type fixed, parent T265_camera_fisheye2_rgb_frame, child T265_camera_fisheye2_optical_frame, origin xyz=0 0 0 rpy=-1.57079632679 0 -1.57079632679
- added joint T265_camera_fisheye2_rgb_joint: type fixed, parent T265_camera_link, child T265_camera_fisheye2_rgb_frame, origin xyz=0.0229 0.0 0.0 rpy=0 1.57079632679 1.57079632679
- added joint T265_camera_gyro_joint: type fixed, parent T265_camera_link, child T265_camera_gyro_frame, origin xyz=-0.0311 0 0.00655 rpy=0 3.14159265359 0
- added joint T265_camera_gyro_optical_joint: type fixed, parent T265_camera_gyro_frame, child T265_camera_gyro_optical_frame, origin xyz=0 0 0 rpy=0 0 0
- added joint T265_camera_link_joint: type fixed, parent T265_camera_pose_frame, child T265_camera_link, origin xyz=0 0 0 rpy=1.57079632679 0 -1.57079632679
- added joint T265_camera_pose_joint: type fixed, parent pelvis, child T265_camera_pose_frame, origin xyz=0.29245 0.00775 0.063 rpy=0 0 0
- added joint d435_head_joint: type revolute, parent neck_1, child d435_head_motor, origin xyz=0.06 0 0.1375 rpy=0 0 0, axis 0 1 0, limit lower=-1.1 upper=1.1 effort=35 velocity=5.7
- added joint neck_base: type fixed, parent torso_2, child neck_1, origin xyz=0.0030637045 0.0061607221 0.224 rpy=0 0 0, axis 0 0 1
- added joint velodyne_joint: type revolute, parent neck_1, child velodyne_motor, origin xyz=0.0825 0 0.243 rpy=0 0 0, axis 0 1 0, limit lower=-1.1 upper=1.1 effort=35 velocity=5.7
- joint velodyne_calib_base_mount_joint: origin xyz=0.032768 -0.01 0.048219 rpy=0 1.5709 -0.316519   -> xyz=0 0 0 rpy=0 0 0; parent neck_3 -> velodyne_motor

File: centauro_urdf/urdf/centauro.urdf (robot description, URDF)
Before this commit: robot centauro, 60 links, 59 joints
Links:
- removed link neck_2
- removed link neck_3
- added link D435_head_camera_accel_frame
- added link D435_head_camera_accel_optical_frame
- added link D435_head_camera_bottom_screw_frame
- added link D435_head_camera_color_frame
- added link D435_head_camera_color_optical_frame
- added link D435_head_camera_depth_frame
- added link D435_head_camera_depth_optical_frame
- added link D435_head_camera_gyro_frame
- added link D435_head_camera_gyro_optical_frame
- added link D435_head_camera_left_ir_frame
- added link D435_head_camera_left_ir_optical_frame
- added link D435_head_camera_link, mass 0.564; collision box size=0.02505 0.09 0.025; visual mesh filename=package://realsense2_description/meshes/d435.dae
- added link D435_head_camera_right_ir_frame
- added link D435_head_camera_right_ir_optical_frame
- added link D435i_camera_accel_frame
- added link D435i_camera_accel_optical_frame
- added link D435i_camera_bottom_screw_frame
- added link D435i_camera_color_frame
- added link D435i_camera_color_optical_frame
- added link D435i_camera_depth_frame
- added link D435i_camera_depth_optical_frame
- added link D435i_camera_gyro_frame
- added link D435i_camera_gyro_optical_frame
- added link D435i_camera_left_ir_frame
- added link D435i_camera_left_ir_optical_frame
- added link D435i_camera_link, mass 0.564; collision box size=0.02505 0.09 0.025; visual mesh filename=package://realsense2_description/meshes/d435.dae
- added link D435i_camera_right_ir_frame
- added link D435i_camera_right_ir_optical_frame
- added link T265_camera_accel_frame
- added link T265_camera_accel_optical_frame
- added link T265_camera_fisheye1_optical_frame
- added link T265_camera_fisheye1_rgb_frame
- added link T265_camera_fisheye2_optical_frame
- added link T265_camera_fisheye2_rgb_frame
- added link T265_camera_gyro_frame
- added link T265_camera_gyro_optical_frame
- added link T265_camera_link
- added link T265_camera_pose_frame, mass 0.068024; collision mesh filename=package://realsense_gazebo_description/meshes/t265_simplifi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 scale=0.001 0.001 0.001; visual mesh filename=package://realsense_gazebo_description/meshes/t265_full.stl scale=0.001 0.001 0.001
- added link d435_head_motor, mass 0.33878686; collision mesh filename=package://centauro_urdf/meshes/simple/neck-pitch_mesh.stl scale=0.001 0.001 0.001; visual mesh filename=package://centauro_urdf/meshes/neck-pitch_mesh.stl scale=0.001 0.001 0.001
- added link velodyne_motor, mass 0.33878686; collision mesh filename=package://centauro_urdf/meshes/simple/lidar_mesh.stl scale=0.001 0.001 0.001; visual mesh filename=package://centauro_urdf/meshes/lidar_mesh.stl scale=0.001 0.001 0.001
- link neck_1: geometry collision mesh filename=package://centauro_urdf/meshes/simple/head-base_mesh.stl scale=0.001 0.001 0.001; visual mesh filename=package://centauro_urdf/meshes/head-base_mesh.stl scale=0.001 0.001 0.001
- link torso_2: geometry collision mesh filename=package://centauro_urdf/meshes/simple/link1_no_head.stl scale=0.001 0.001 0.001; visual mesh filename=package://centauro_urdf/meshes/link1_no_head.stl scale=0.001 0.001 0.001
Joints:
- removed joint neck_pitch
- removed joint neck_velodyne
- removed joint neck_yaw
- added joint D435_head_camera_accel_joint: type fixed, parent D435_head_camera_link, child D435_head_camera_accel_frame, origin xyz=-0.00174 0.00552 0.0176 rpy=0 0 0
- added joint D435_head_camera_accel_optical_joint: type fixed, parent D435_head_camera_accel_frame, child D435_head_camera_accel_optical_frame, origin xyz=0 0 0 rpy=-1.57079632679 0 -1.57079632679
- added joint D435_head_camera_color_joint: type fixed, parent D435_head_camera_depth_frame, child D435_head_camera_color_frame, origin xyz=0 0.015 0 rpy=0 0 0
- added joint D435_head_camera_color_optical_joint: type fixed, parent D435_head_camera_color_frame, child D435_head_camera_color_optical_frame, origin xyz=0 0 0 rpy=-1.57079632679 0 -1.57079632679
- added joint D435_head_camera_depth_joint: type fixed, parent D435_head_camera_link, child D435_head_camera_depth_frame, origin xyz=0 0 0 rpy=0 0 0
- added joint D435_head_camera_depth_optical_joint: type fixed, parent D435_head_camera_depth_frame, child D435_head_camera_depth_optical_frame, origin xyz=0 0 0 rpy=-1.57079632679 0 -1.57079632679
- added joint D435_head_camera_gyro_joint: type fixed, parent D435_head_camera_link, child D435_head_camera_gyro_frame, origin xyz=-0.00174 0.00552 0.0176 rpy=0 0 0
- added joint D435_head_camera_gyro_optical_joint: type fixed, parent D435_head_camera_gyro_frame, child D435_head_camera_gyro_optical_frame, origin xyz=0 0 0 rpy=-1.57079632679 0 -1.57079632679
- added joint D435_head_camera_joint: type fixed, parent d435_head_motor, child D435_head_camera_bottom_screw_frame, origin xyz=0.03015 0 -0.0125 rpy=0 0 0
- added joint D435_head_camera_left_ir_joint: type fixed, parent D435_head_camera_depth_frame, child D435_head_camera_left_ir_frame, origin xyz=0 0.0 0 rpy=0 0 0
- added joint D435_head_camera_left_ir_optical_joint: type fixed, parent D435_head_camera_left_ir_frame, child D435_head_camera_left_ir_optical_frame, origin xyz=0 0 0 rpy=-1.57079632679 0 -1.57079632679
- added joint D435_head_camera_link_joint: type fixed, parent D435_head_camera_bottom_screw_frame, child D435_head_camera_link, origin xyz=0 0.0175 0.0125 rpy=0 0 0
- added joint D435_head_camera_right_ir_joint: type fixed, parent D435_head_camera_depth_frame, child D435_head_camera_right_ir_frame, origin xyz=0 -0.05 0 rpy=0 0 0
- added joint D435_head_camera_right_ir_optical_joint: type fixed, parent D435_head_camera_right_ir_frame, child D435_head_camera_right_ir_optical_frame, origin xyz=0 0 0 rpy=-1.57079632679 0 -1.57079632679
- added joint D435i_camera_accel_joint: type fixed, parent D435i_camera_link, child D435i_camera_accel_frame, origin xyz=-0.00174 0.00552 0.0176 rpy=0 0 0
- added joint D435i_camera_accel_optical_joint: type fixed, parent D435i_camera_accel_frame, child D435i_camera_accel_optical_frame, origin xyz=0 0 0 rpy=-1.57079632679 0 -1.57079632679
- added joint D435i_camera_color_joint: type fixed, parent D435i_camera_depth_frame, child D435i_camera_color_frame, origin xyz=0 0.015 0 rpy=0 0 0
- added joint D435i_camera_color_optical_joint: type fixed, parent D435i_camera_color_frame, child D435i_camera_color_optical_frame, origin xyz=0 0 0 rpy=-1.57079632679 0 -1.57079632679
- added joint D435i_camera_depth_joint: type fixed, parent D435i_camera_link, child D435i_camera_depth_frame, origin xyz=0 0 0 rpy=0 0 0
- added joint D435i_camera_depth_optical_joint: type fixed, parent D435i_camera_depth_frame, child D435i_camera_depth_optical_frame, origin xyz=0 0 0 rpy=-1.57079632679 0 -1.57079632679
- added joint D435i_camera_gyro_joint: type fixed, parent D435i_camera_link, child D435i_camera_gyro_frame, origin xyz=-0.00174 0.00552 0.0176 rpy=0 0 0
- added joint D435i_camera_gyro_optical_joint: type fixed, parent D435i_camera_gyro_frame, child D435i_camera_gyro_optical_frame, origin xyz=0 0 0 rpy=-1.57079632679 0 -1.57079632679
- added joint D435i_camera_joint: type fixed, parent pelvis, child D435i_camera_bottom_screw_frame, origin xyz=0.27187 0 0.0215997 rpy=0 0.5251508 0
- added joint D435i_camera_left_ir_joint: type fixed, parent D435i_camera_depth_frame, child D435i_camera_left_ir_frame, origin xyz=0 0.0 0 rpy=0 0 0
- added joint D435i_camera_left_ir_optical_joint: type fixed, parent D435i_camera_left_ir_frame, child D435i_camera_left_ir_optical_frame, origin xyz=0 0 0 rpy=-1.57079632679 0 -1.57079632679
- added joint D435i_camera_link_joint: type fixed, parent D435i_camera_bottom_screw_frame, child D435i_camera_link, origin xyz=0 0.0175 0.0125 rpy=0 0 0
- added joint D435i_camera_right_ir_joint: type fixed, parent D435i_camera_depth_frame, child D435i_camera_right_ir_frame, origin xyz=0 -0.05 0 rpy=0 0 0
- added joint D435i_camera_right_ir_optical_joint: type fixed, parent D435i_camera_right_ir_frame, child D435i_camera_right_ir_optical_frame, origin xyz=0 0 0 rpy=-1.57079632679 0 -1.57079632679
- added joint T265_camera_accel_joint: type fixed, parent T265_camera_link, child T265_camera_accel_frame, origin xyz=-0.0311 0 0.00655 rpy=0 3.14159265359 0
- added joint T265_camera_accel_optical_joint: type fixed, parent T265_camera_accel_frame, child T265_camera_accel_optical_frame, origin xyz=-0.0311 0 0.00655 rpy=0 3.14159265359 0
- added joint T265_camera_fisheye1_optical_joint: type fixed, parent T265_camera_fisheye1_rgb_frame, child T265_camera_fisheye1_optical_frame, origin xyz=0 0 0 rpy=-1.57079632679 0 -1.57079632679
- added joint T265_camera_fisheye1_rgb_joint: type fixed, parent T265_camera_link, child T265_camera_fisheye1_rgb_frame, origin xyz=-0.0411 0.0 0.0 rpy=0 1.57079632679 1.57079632679
- added joint T265_camera_fisheye2_optical_joint: type fixed, parent T265_camera_fisheye2_rgb_frame, child T265_camera_fisheye2_optical_frame, origin xyz=0 0 0 rpy=-1.57079632679 0 -1.57079632679
- added joint T265_camera_fisheye2_rgb_joint: type fixed, parent T265_camera_link, child T265_camera_fisheye2_rgb_frame, origin xyz=0.0229 0.0 0.0 rpy=0 1.57079632679 1.57079632679
- added joint T265_camera_gyro_joint: type fixed, parent T265_camera_link, child T265_camera_gyro_frame, origin xyz=-0.0311 0 0.00655 rpy=0 3.14159265359 0
- added joint T265_camera_gyro_optical_joint: type fixed, parent T265_camera_gyro_frame, child T265_camera_gyro_optical_frame, origin xyz=0 0 0 rpy=0 0 0
- added joint T265_camera_link_joint: type fixed, parent T265_camera_pose_frame, child T265_camera_link, origin xyz=0 0 0 rpy=1.57079632679 0 -1.57079632679
- added joint T265_camera_pose_joint: type fixed, parent pelvis, child T265_camera_pose_frame, origin xyz=0.29245 0.00775 0.063 rpy=0 0 0
- added joint d435_head_joint: type revolute, parent neck_1, child d435_head_motor, origin xyz=0.06 0 0.1375 rpy=0 0 0, axis 0 1 0, limit lower=-1.1 upper=1.1 effort=35 velocity=5.7
- added joint neck_base: type fixed, parent torso_2, child neck_1, origin xyz=0.0030637045 0.0061607221 0.224 rpy=0 0 0, axis 0 0 1
- added joint velodyne_joint: type revolute, parent neck_1, child velodyne_motor, origin xyz=0.0825 0 0.243 rpy=0 0 0, axis 0 1 0, limit lower=-1.1 upper=1.1 effort=35 velocity=5.7
- joint velodyne_calib_base_mount_joint: origin xyz=0.032768 -0.01 0.048219 rpy=0 1.5709 -0.316519   -> xyz=0 0 0 rpy=0 0 0; parent neck_3 -> velodyne_motor
