Commit message: Change sensor location. Missing: inertia/mass and joint_map for head d435. Velodyne to correct

File: centauro_urdf/urdf/centauro_base.urdf.xacro (robot description, xacro)
@@ -55,7 +55,54 @@
     <xacro:if value="${ADD_VELODYNE}">
         <xacro:include filename="$(find velodyne_description)/urdf/VLP-16.urdf.xacro"/>
-        <xacro:VLP-16 parent="neck_3" name="velodyne_calib" topic="/velodyne_points" hz="10" samples="440">
-            <origin xyz="0.032768 -0.01 0.048219" rpy="0 1.5709 -0.316519  " />
+        <xacro:VLP-16 parent="velodyne_motor" name="velodyne_calib" topic="/velodyne_points" hz="10" samples="440">
+            <origin xyz="0 0 0" rpy="0 0 0" />
         </xacro:VLP-16>
+    </xacro:if>
+    <xacro:if value="${ADD_D435_HEAD}">
+        <link name="d435_head_motor">
+            <inertial>
+            <origin xyz="0 0 0"/>
+            <mass value="0.33878686"/> <!-- MASS/INERTIA TO DO -->
+            <inertia ixx="0.0003718568" ixy="-9.42983e-05" ixz="-2.80644e-05" iyy="0.0001886879" iyz="-1.54534e-05" izz="0.0005023443"/>
+            </inertial>
+            <visual>
+            <origin rpy="0.0 0.0 0.0" xyz="0.0 0 0.0"/>
+            <geometry>
+                <mesh filename="package://centauro_urdf/meshes/neck-pitch_mesh.stl" scale="0.001 0.001 0.001"/>
+            </geometry>
+            </visual>
+            <collision>
+            <origin rpy="0.0 0.0 0.0" xyz="0.0 0 0.0"/>
+            <geometry>
+                <mesh filename="package://centauro_urdf/meshes/simple/neck-pitch_mesh.stl" scale="0.001 0.001 0.001"/>
+            </geometry>
+            </collision>
+        </link>
+        <joint name="d435_head_joint" type="revolute">
+            <parent link="neck_1"/>
+            <origin xyz="0.06 0 0.1375" rpy="0 0 0"/>
+            <child link="d435_head_motor"/>
+            <axis xyz="0 1 0"/>
+            <limit effort="35" lower="-1.1" upper="1.1" velocity="5.7"/>
+            <dynamics friction="10.0"/>
+        </joint>
+        <xacro:include filename="$(find realsense_gazebo_description)/urdf/_d435i.urdf.xacro" />
+        <xacro:sensor_d435i parent="d435_head_motor" name="D435_head_camera" topics_ns="D435/D435_head_camera"
+                      enable_pointCloud="true" align_depth="true"
+                      unite_imu_method="false"
+                      visualize="false"
+                      accel_fps="300"
+                      gyro_fps="300"
+                      depth_width="1280"
+                      depth_height="720"
+                      depth_fps="90"
+                      infra_width="1280"
+                      infra_height="720"
+                      infra_fps="90"
+                      color_width="1280"
+                      color_height="720"
+                      color_fps="30">
+            <origin xyz="0.03015 0 -0.0125" rpy="0 0 0"/>
+        </xacro:sensor_d435i>
     </xacro:if>
     <xacro:if value="${ADD_INTEL_D435I}">
@@ -80,5 +127,5 @@
                       color_height="720"
                       color_fps="30">
-            <origin xyz="0.219831 0 -0.0613293" rpy="0.0 0.5585052 0.0"/>
+            <origin xyz="0.27187 0 0.0215997" rpy="0 0.5251508 0"/>
         </xacro:sensor_d435i>
     </xacro:if>
@@ -101,5 +148,5 @@
                       accel_fps="62.5"
                       gyro_fps="200">
-            <origin xyz="0.252619 0.00775 -0.0206926" rpy="0.0 0.2617993 0.0" />
+            <origin xyz="0.29245 0.00775 0.063" rpy="0 0 0" />
         </xacro:sensor_t265>
     </xacro:if>

File: centauro_urdf/urdf/centauro_config.urdf.xacro (robot description, xacro)
@@ -15,5 +15,6 @@
 <xacro:property name="USE_STICKS" value="false" />
 <xacro:property name="ADD_VELODYNE" value="true" />
-<xacro:property name="ADD_INTEL_D435I" value="false" />
-<xacro:property name="ADD_INTEL_T265" value="false" />
+<xacro:property name="ADD_D435_HEAD" value="true" />
+<xacro:property name="ADD_INTEL_D435I" value="true" />
+<xacro:property name="ADD_INTEL_T265" value="true" />
 </robot>

File: centauro_urdf/urdf/centauro_virtual_frame.urdf (robot description, URDF)
Before this commit: robot centauro, 76 links, 75 joints
Links:
- removed link neck_2
- removed link neck_3
- added link velodyne_motor, mass 0.33878686; collision mesh filename=package://centauro_urdf/meshes/simple/lidar_mesh.stl scale=0.001 0.001 0.001; visual mesh filename=package://centauro_urdf/meshes/lidar_mesh.stl scale=0.001 0.001 0.001
- link neck_1: geometry collision mesh filename=package://centauro_urdf/meshes/simple/head-base_mesh.stl scale=0.001 0.001 0.001; visual mesh filename=package://centauro_urdf/meshes/head-base_mesh.stl scale=0.001 0.001 0.001
- link torso_2: geometry collision mesh filename=package://centauro_urdf/meshes/simple/link1_no_head.stl scale=0.001 0.001 0.001; visual mesh filename=package://centauro_urdf/meshes/link1_no_head.stl scale=0.001 0.001 0.001
Joints:
- removed joint neck_pitch
- removed joint neck_velodyne
- removed joint neck_yaw
- added joint neck_base: type fixed, parent torso_2, child neck_1, origin xyz=0.0030637045 0.0061607221 0.224 rpy=0 0 0, axis 0 0 1
- added joint velodyne_joint: type revolute, parent neck_1, child velodyne_motor, origin xyz=0.0825 0 0.243 rpy=0 0 0, axis 0 1 0, limit lower=-1.1 upper=1.1 effort=35 velocity=5.7
- joint T265_camera_pose_joint: origin xyz=0.252619 0.00775 -0.0206926 rpy=0.0 0.2617993 0.0 -> xyz=0.29245 0.00775 0.063 rpy=0 0 0
- joint velodyne_calib_base_mount_joint: origin xyz=0.032768 -0.01 0.048219 rpy=0 1.5709 -0.316519   -> xyz=0 0 0 rpy=0 0 0; parent neck_3 -> velodyne_motor

File: centauro_urdf/urdf/centauro_virtual_frame_robot.urdf (robot description, URDF)
Before this commit: robot centauro, 76 links, 75 joints
Links:
- removed link neck_2
- removed link neck_3
- added link velodyne_motor, mass 0.33878686; collision mesh filename=package://centauro_urdf/meshes/simple/lidar_mesh.stl scale=0.001 0.001 0.001; visual mesh filename=package://centauro_urdf/meshes/lidar_mesh.stl scale=0.001 0.001 0.001
- link neck_1: geometry collision mesh filename=package://centauro_urdf/meshes/simple/head-base_mesh.stl scale=0.001 0.001 0.001; visual mesh filename=package://centauro_urdf/meshes/head-base_mesh.stl scale=0.001 0.001 0.001
- link torso_2: geometry collision mesh filename=package://centauro_urdf/meshes/simple/link1_no_head.stl scale=0.001 0.001 0.001; visual mesh filename=package://centauro_urdf/meshes/link1_no_head.stl scale=0.001 0.001 0.001
Joints:
- removed joint neck_pitch
- removed joint neck_velodyne
- removed joint neck_yaw
- added joint neck_base: type fixed, parent torso_2, child neck_1, origin xyz=0.0030637045 0.0061607221 0.224 rpy=0 0 0, axis 0 0 1
- added joint velodyne_joint: type revolute, parent neck_1, child velodyne_motor, origin xyz=0.0825 0 0.243 rpy=0 0 0, axis 0 1 0, limit lower=-1.1 upper=1.1 effort=35 velocity=5.7
- joint T265_camera_pose_joint: origin xyz=0.252619 0.00775 -0.0206926 rpy=0.0 0.2617993 0.0 -> xyz=0.29245 0.00775 0.063 rpy=0 0 0
- joint velodyne_calib_base_mount_joint: origin xyz=0.032768 -0.01 0.048219 rpy=0 1.5709 -0.316519   -> xyz=0 0 0 rpy=0 0 0; parent neck_3 -> velodyne_motor

File: centauro_urdf/urdf/config/centauro_virtual_frame.urdf.xacro (robot description, xacro)
@@ -15,4 +15,5 @@
 <xacro:property name="USE_STICKS" value="false" />
 <xacro:property name="ADD_VELODYNE" value="true" />
+<xacro:property name="ADD_D435_HEAD" value="false" />
 <xacro:property name="ADD_INTEL_D435I" value="false" />
 <xacro:property name="ADD_INTEL_T265" value="true" />

File: centauro_urdf/urdf/parts/centauro_torso.urdf.xacro (robot description, xacro)
@@ -11,5 +11,5 @@
           <origin xyz="0.0 0 0.0"  rpy="0.0 0.0 0.0"/>
    	  <geometry>
-      	  <mesh filename="package://centauro_urdf/meshes/link1.stl" scale="0.001 0.001 0.001" />
+      	  <mesh filename="package://centauro_urdf/meshes/link1_no_head.stl" scale="0.001 0.001 0.001" />
    	  </geometry>
 	</visual>
@@ -17,5 +17,5 @@
           <origin xyz="0.0 0 0.0"  rpy="0.0 0.0 0.0"/>
    	  <geometry>
-      	  <mesh filename="package://centauro_urdf/meshes/simple/link1.stl" scale="0.001 0.001 0.001" />
+      	  <mesh filename="package://centauro_urdf/meshes/simple/link1_no_head.stl" scale="0.001 0.001 0.001" />
    	  </geometry>
 	</collision>

File: centauro_urdf/urdf/parts/head.urdf.xacro (robot description, xacro)
@@ -2,9 +2,8 @@
 <robot xmlns:xacro="http://ros.org/wiki/xacro">
 <!-- LINKS -->
-<!-- TODO: FINISH IMPLEMENTATION WITH CORRECT NUMBERS -->
 <link name="neck_1">
     <inertial>
-      <origin xyz="0.040479674 0.021377573 -0.014595112"/>
-      <mass value="0.33878686"/>
+      <origin xyz="0 0 0"/>
+      <mass value="0.33878686"/> <!-- MASS/INERTIA TO DO -->
       <inertia ixx="0.0003718568" ixy="-9.42983e-05" ixz="-2.80644e-05" iyy="0.0001886879" iyz="-1.54534e-05" izz="0.0005023443"/>
     </inertial>
@@ -12,5 +11,5 @@
       <origin rpy="0.0 0.0 0.0" xyz="0.0 0 0.0"/>
       <geometry>
-        <mesh filename="package://centauro_urdf/meshes/neck_yaw.stl" scale="0.001 0.001 0.001"/>
+        <mesh filename="package://centauro_urdf/meshes/head-base_mesh.stl" scale="0.001 0.001 0.001"/>
       </geometry>
     </visual>
@@ -18,18 +17,18 @@
       <origin rpy="0.0 0.0 0.0" xyz="0.0 0 0.0"/>
       <geometry>
-        <mesh filename="package://centauro_urdf/meshes/simple/neck_yaw.stl" scale="0.001 0.001 0.001"/>
+        <mesh filename="package://centauro_urdf/meshes/simple/head-base_mesh.stl" scale="0.001 0.001 0.001"/>
       </geometry>
     </collision>
 </link>
-<link name="neck_2">
+<link name="velodyne_motor">
     <inertial>
-      <origin xyz="0.048466918 -0.059852318 -0.0085314894"/>
-      <mass value="0.78526942"/>
-      <inertia ixx="0.0004682345" ixy="-1.05438e-05" ixz="7.24398e-05" iyy="0.0002635246" iyz="1.6904e-06" izz="0.0003763351"/>
+      <origin xyz="0 0 0"/>
+      <mass value="0.33878686"/> <!-- MASS/INERTIA TO DO -->
+      <inertia ixx="0.0003718568" ixy="-9.42983e-05" ixz="-2.80644e-05" iyy="0.0001886879" iyz="-1.54534e-05" izz="0.0005023443"/>
     </inertial>
     <visual>
       <origin rpy="0.0 0.0 0.0" xyz="0.0 0 0.0"/>
       <geometry>
-        <mesh filename="package://centauro_urdf/meshes/neck_pitch.stl" scale="0.001 0.001 0.001"/>
+        <mesh filename="package://centauro_urdf/meshes/lidar_mesh.stl" scale="0.001 0.001 0.001"/>
       </geometry>
     </visual>
@@ -37,53 +36,22 @@
       <origin rpy="0.0 0.0 0.0" xyz="0.0 0 0.0"/>
       <geometry>
-        <mesh filename="package://centauro_urdf/meshes/simple/neck_pitch.stl" scale="0.001 0.001 0.001"/>
-      </geometry>
-    </collision>
-</link>
-<!-- LINKS -->
-<link name="neck_3">
-    <inertial>
-      <origin xyz="0.048466918 -0.059852318 -0.0085314894"/>
-      <mass value="0.78526942"/>
-      <inertia ixx="0.0004682345" ixy="-1.05438e-05" ixz="7.24398e-05" iyy="0.0002635246" iyz="1.6904e-06" izz="0.0003763351"/>
-    </inertial>
-    <visual>
-      <origin rpy="0.0 0.0 0.0" xyz="0.0 0 0.0"/>
-      <geometry>
-        <mesh filename="package://centauro_urdf/meshes/lidar.stl" scale="0.001 0.001 0.001"/>
-      </geometry>
-    </visual>
-    <collision>
-      <origin rpy="0.0 0.0 0.0" xyz="0.0 0 0.0"/>
-      <geometry>
-        <mesh filename="package://centauro_urdf/meshes/simple/lidar.stl" scale="0.001 0.001 0.001"/>
+        <mesh filename="package://centauro_urdf/meshes/simple/lidar_mesh.stl" scale="0.001 0.001 0.001"/>
       </geometry>
     </collision>
 </link>
 <!--JOINTS -->
-<joint name="neck_yaw" type="revolute">
+<joint name="neck_base" type="fixed">
     <parent link="torso_2"/>
-    <origin xyz="0.0 0.0 0.2795"/>
+    <origin xyz="0.0030637045 0.0061607221 0.224" rpy="0 0 0"/>
     <child link="neck_1"/>
     <axis xyz="0 0 1"/>
-    <limit effort="35" lower="-0.78539816" upper="0.78539816" velocity="5.7"/>
+</joint>
+<joint name="velodyne_joint" type="revolute">
+    <parent link="neck_1"/>
+    <origin xyz="0.0825 0 0.243" rpy="0 0 0"/>
+    <child link="velodyne_motor"/>
+    <axis xyz="0 1 0"/>
+    <limit effort="35" lower="-1.1" upper="1.1" velocity="5.7"/>
     <dynamics friction="10.0"/>
 </joint>
-<joint name="neck_pitch" type="revolute">
-    <parent link="neck_1"/>
-    <origin xyz="0.054 0.0596 -0.0124975"/>
-    <child link="neck_2"/>
-    <axis xyz="0 1 0"/>
-    <limit effort="35" lower="-0.34906585" upper="0.78539816" velocity="5.7"/>
-    <dynamics friction="10.0"/>
-</joint>
-<joint name="neck_velodyne" type="continuous">
-    <parent link="torso_2"/>
-    <origin xyz="0.055 0.0 0.473262" rpy="0 0 -1.828"/>
-    <!--origin xyz="0.055 0.0 0.473262" rpy="0 0 -1.311481"/-->
-    <child link="neck_3"/>
-    <axis xyz="0 0 1"/>
-    <limit effort="35" velocity="5.7"/>
-    <dynamics damping="0.2" friction="10.0"/>
-</joint>
 </robot>
