Commit message: Adjust new elements position (missin mass and inertia)

File: centauro_srdf/srdf/centauro.srdf.xacro (robot description, xacro)
@@ -100,7 +100,11 @@
 	<joint name="ankle_yaw_4" value="0.746874"/>
 	<joint name="torso_yaw" value="3.56617e-13"/>
-	<joint name="velodyne_joint" value="0"/>
-	<joint name="d435_head_joint" value="0"/>
-	<joint name="j_arm1_1" value="0.520149"/>
+    <xacro:if value="${ADD_VELODYNE}">
+        <joint name="velodyne_joint" value="0"/>
+    </xacro:if>
+    <xacro:if value="${ADD_D435_HEAD}">
+        <joint name="d435_head_joint" value="0"/>
+    </xacro:if>
+    <joint name="j_arm1_1" value="0.520149"/>
 	<joint name="j_arm1_2" value="0.320865"/>
 	<joint name="j_arm1_3" value="0.274669"/>

File: centauro_urdf/urdf/_centauro_robot.urdf (robot description, URDF)
Before this commit: robot centauro, 98 links, 97 joints
Links:
- removed link D435_head_camera_accel_frame
- removed link D435_head_camera_accel_optical_frame
- removed link D435_head_camera_bottom_screw_frame
- removed link D435_head_camera_color_frame
- removed link D435_head_camera_color_optical_frame
- removed link D435_head_camera_depth_frame
- removed link D435_head_camera_depth_optical_frame
- removed link D435_head_camera_gyro_frame
- removed link D435_head_camera_gyro_optical_frame
- removed link D435_head_camera_left_ir_frame
- removed link D435_head_camera_left_ir_optical_frame
- removed link D435_head_camera_link
- removed link D435_head_camera_right_ir_frame
- removed link D435_head_camera_right_ir_optical_frame
- removed link D435i_camera_accel_frame
- removed link D435i_camera_accel_optical_frame
- removed link D435i_camera_bottom_screw_frame
- removed link D435i_camera_color_frame
- removed link D435i_camera_color_optical_frame
- removed link D435i_camera_depth_frame
- removed link D435i_camera_depth_optical_frame
- removed link D435i_camera_gyro_frame
- removed link D435i_camera_gyro_optical_frame
- removed link D435i_camera_left_ir_frame
- removed link D435i_camera_left_ir_optical_frame
- removed link D435i_camera_link
- removed link D435i_camera_right_ir_frame
- removed link D435i_camera_right_ir_optical_frame
- removed link T265_camera_accel_frame
- removed link T265_camera_accel_optical_frame
- removed link T265_camera_fisheye1_optical_frame
- removed link T265_camera_fisheye1_rgb_frame
- removed link T265_camera_fisheye2_optical_frame
- removed link T265_camera_fisheye2_rgb_frame
- removed link T265_camera_gyro_frame
- removed link T265_camera_gyro_optical_frame
- removed link T265_camera_link
- removed link T265_camera_pose_frame
- removed link d435_head_motor
Joints:
- removed joint D435_head_camera_accel_joint
- removed joint D435_head_camera_accel_optical_joint
- removed joint D435_head_camera_color_joint
- removed joint D435_head_camera_color_optical_joint
- removed joint D435_head_camera_depth_joint
- removed joint D435_head_camera_depth_optical_joint
- removed joint D435_head_camera_gyro_joint
- removed joint D435_head_camera_gyro_optical_joint
- removed joint D435_head_camera_joint
- removed joint D435_head_camera_left_ir_joint
- removed joint D435_head_camera_left_ir_optical_joint
- removed joint D435_head_camera_link_joint
- removed joint D435_head_camera_right_ir_joint
- removed joint D435_head_camera_right_ir_optical_joint
- removed joint D435i_camera_accel_joint
- removed joint D435i_camera_accel_optical_joint
- removed joint D435i_camera_color_joint
- removed joint D435i_camera_color_optical_joint
- removed joint D435i_camera_depth_joint
- removed joint D435i_camera_depth_optical_joint
- removed joint D435i_camera_gyro_joint
- removed joint D435i_camera_gyro_optical_joint
- removed joint D435i_camera_joint
- removed joint D435i_camera_left_ir_joint
- removed joint D435i_camera_left_ir_optical_joint
- removed joint D435i_camera_link_joint
- removed joint D435i_camera_right_ir_joint
- removed joint D435i_camera_right_ir_optical_joint
- removed joint T265_camera_accel_joint
- removed joint T265_camera_accel_optical_joint
- removed joint T265_camera_fisheye1_optical_joint
- removed joint T265_camera_fisheye1_rgb_joint
- removed joint T265_camera_fisheye2_optical_joint
- removed joint T265_camera_fisheye2_rgb_joint
- removed joint T265_camera_gyro_joint
- removed joint T265_camera_gyro_optical_joint
- removed joint T265_camera_link_joint
- removed joint T265_camera_pose_joint
- removed joint d435_head_joint
- joint neck_base: origin xyz=0.0030637045 0.0061607221 0.224 rpy=0 0 0 -> xyz=0.0030637045 0.0061607221 0.158 rpy=0 0 0
- joint velodyne_joint: origin xyz=0.0825 0 0.243 rpy=0 0 0 -> xyz=0.0822724 0 0.242 rpy=0 0 0

File: centauro_urdf/urdf/centauro.urdf (robot description, URDF)
Before this commit: robot centauro, 98 links, 97 joints
Links:
- removed link D435_head_camera_accel_frame
- removed link D435_head_camera_accel_optical_frame
- removed link D435_head_camera_bottom_screw_frame
- removed link D435_head_camera_color_frame
- removed link D435_head_camera_color_optical_frame
- removed link D435_head_camera_depth_frame
- removed link D435_head_camera_depth_optical_frame
- removed link D435_head_camera_gyro_frame
- removed link D435_head_camera_gyro_optical_frame
- removed link D435_head_camera_left_ir_frame
- removed link D435_head_camera_left_ir_optical_frame
- removed link D435_head_camera_link
- removed link D435_head_camera_right_ir_frame
- removed link D435_head_camera_right_ir_optical_frame
- removed link D435i_camera_accel_frame
- removed link D435i_camera_accel_optical_frame
- removed link D435i_camera_bottom_screw_frame
- removed link D435i_camera_color_frame
- removed link D435i_camera_color_optical_frame
- removed link D435i_camera_depth_frame
- removed link D435i_camera_depth_optical_frame
- removed link D435i_camera_gyro_frame
- removed link D435i_camera_gyro_optical_frame
- removed link D435i_camera_left_ir_frame
- removed link D435i_camera_left_ir_optical_frame
- removed link D435i_camera_link
- removed link D435i_camera_right_ir_frame
- removed link D435i_camera_right_ir_optical_frame
- removed link T265_camera_accel_frame
- removed link T265_camera_accel_optical_frame
- removed link T265_camera_fisheye1_optical_frame
- removed link T265_camera_fisheye1_rgb_frame
- removed link T265_camera_fisheye2_optical_frame
- removed link T265_camera_fisheye2_rgb_frame
- removed link T265_camera_gyro_frame
- removed link T265_camera_gyro_optical_frame
- removed link T265_camera_link
- removed link T265_camera_pose_frame
- removed link d435_head_motor
Joints:
- removed joint D435_head_camera_accel_joint
- removed joint D435_head_camera_accel_optical_joint
- removed joint D435_head_camera_color_joint
- removed joint D435_head_camera_color_optical_joint
- removed joint D435_head_camera_depth_joint
- removed joint D435_head_camera_depth_optical_joint
- removed joint D435_head_camera_gyro_joint
- removed joint D435_head_camera_gyro_optical_joint
- removed joint D435_head_camera_joint
- removed joint D435_head_camera_left_ir_joint
- removed joint D435_head_camera_left_ir_optical_joint
- removed joint D435_head_camera_link_joint
- removed joint D435_head_camera_right_ir_joint
- removed joint D435_head_camera_right_ir_optical_joint
- removed joint D435i_camera_accel_joint
- removed joint D435i_camera_accel_optical_joint
- removed joint D435i_camera_color_joint
- removed joint D435i_camera_color_optical_joint
- removed joint D435i_camera_depth_joint
- removed joint D435i_camera_depth_optical_joint
- removed joint D435i_camera_gyro_joint
- removed joint D435i_camera_gyro_optical_joint
- removed joint D435i_camera_joint
- removed joint D435i_camera_left_ir_joint
- removed joint D435i_camera_left_ir_optical_joint
- removed joint D435i_camera_link_joint
- removed joint D435i_camera_right_ir_joint
- removed joint D435i_camera_right_ir_optical_joint
- removed joint T265_camera_accel_joint
- removed joint T265_camera_accel_optical_joint
- removed joint T265_camera_fisheye1_optical_joint
- removed joint T265_camera_fisheye1_rgb_joint
- removed joint T265_camera_fisheye2_optical_joint
- removed joint T265_camera_fisheye2_rgb_joint
- removed joint T265_camera_gyro_joint
- removed joint T265_camera_gyro_optical_joint
- removed joint T265_camera_link_joint
- removed joint T265_camera_pose_joint
- removed joint d435_head_joint
- joint neck_base: origin xyz=0.0030637045 0.0061607221 0.224 rpy=0 0 0 -> xyz=0.0030637045 0.0061607221 0.158 rpy=0 0 0
- joint velodyne_joint: origin xyz=0.0825 0 0.243 rpy=0 0 0 -> xyz=0.0822724 0 0.242 rpy=0 0 0

File: centauro_urdf/urdf/centauro_config.urdf.xacro (robot description, xacro)
@@ -15,6 +15,6 @@
 <xacro:property name="USE_STICKS" value="false" />
 <xacro:property name="ADD_VELODYNE" value="true" />
-<xacro:property name="ADD_D435_HEAD" value="true" />
-<xacro:property name="ADD_INTEL_D435I" value="true" />
-<xacro:property name="ADD_INTEL_T265" value="true" />
+<xacro:property name="ADD_D435_HEAD" value="false" />
+<xacro:property name="ADD_INTEL_D435I" value="false" />
+<xacro:property name="ADD_INTEL_T265" value="false" />
 </robot>

File: centauro_urdf/urdf/centauro_virtual_frame.urdf (robot description, URDF)
Before this commit: robot centauro, 75 links, 74 joints
Joints:
- joint neck_base: origin xyz=0.0030637045 0.0061607221 0.224 rpy=0 0 0 -> xyz=0.0030637045 0.0061607221 0.158 rpy=0 0 0
- joint velodyne_joint: origin xyz=0.0825 0 0.243 rpy=0 0 0 -> xyz=0.0822724 0 0.242 rpy=0 0 0

File: centauro_urdf/urdf/centauro_virtual_frame_robot.urdf (robot description, URDF)
Before this commit: robot centauro, 75 links, 74 joints
Joints:
- joint neck_base: origin xyz=0.0030637045 0.0061607221 0.224 rpy=0 0 0 -> xyz=0.0030637045 0.0061607221 0.158 rpy=0 0 0
- joint velodyne_joint: origin xyz=0.0825 0 0.243 rpy=0 0 0 -> xyz=0.0822724 0 0.242 rpy=0 0 0

File: centauro_urdf/urdf/parts/head.urdf.xacro (robot description, xacro)
@@ -43,5 +43,5 @@
 <joint name="neck_base" type="fixed">
     <parent link="torso_2"/>
-    <origin xyz="0.0030637045 0.0061607221 0.224" rpy="0 0 0"/>
+    <origin xyz="0.0030637045 0.0061607221 0.158" rpy="0 0 0"/>
     <child link="neck_1"/>
     <axis xyz="0 0 1"/>
@@ -49,5 +49,5 @@
 <joint name="velodyne_joint" type="revolute">
     <parent link="neck_1"/>
-    <origin xyz="0.0825 0 0.243" rpy="0 0 0"/>
+    <origin xyz="0.0822724 0 0.242" rpy="0 0 0"/>
     <child link="velodyne_motor"/>
     <axis xyz="0 1 0"/>

Commit message: Adjust new head model (sign axis etc). Missing limits

File: centauro_srdf/srdf/centauro.srdf.xacro (robot description, xacro)
@@ -39,14 +39,10 @@
     	<chain base_link="torso_2" tip_link="neck_2" />
     </group>-->
-    <xacro:if value="${ADD_VELODYNE}">
-        <group name="velodyne">
-            <chain base_link="torso_2" tip_link="velodyne_motor" />
-        </group>
-    </xacro:if>
-    <xacro:if value="${ADD_D435_HEAD}">
-        <group name="d435_head">
-            <chain base_link="torso_2" tip_link="d435_head_motor" />
-        </group>
-    </xacro:if>
+    <group name="velodyne">
+        <chain base_link="torso_2" tip_link="velodyne_motor" />
+    </group>
+    <group name="d435_head">
+        <chain base_link="torso_2" tip_link="d435_head_motor" />
+    </group>
 </xacro:if>
 <xacro:if value="${ADD_VIRTUAL_FRAME}">
@@ -66,10 +62,6 @@
         <group name="right_arm" />
         <group name="torso" />
-        <xacro:if value="${ADD_VELODYNE}">
-            <group name="velodyne"/>
-        </xacro:if>
-        <xacro:if value="${ADD_D435_HEAD}">
-            <group name="d435_head"/>
-        </xacro:if>
+        <group name="velodyne"/>
+        <group name="d435_head"/>
     </xacro:if>
     <xacro:if value="${ADD_VIRTUAL_FRAME}">
@@ -100,10 +92,6 @@
 	<joint name="ankle_yaw_4" value="0.746874"/>
 	<joint name="torso_yaw" value="3.56617e-13"/>
-    <xacro:if value="${ADD_VELODYNE}">
-        <joint name="velodyne_joint" value="0"/>
-    </xacro:if>
-    <xacro:if value="${ADD_D435_HEAD}">
-        <joint name="d435_head_joint" value="0"/>
-    </xacro:if>
+    <joint name="velodyne_joint" value="0"/>
+    <joint name="d435_head_joint" value="0"/>
     <joint name="j_arm1_1" value="0.520149"/>
 	<joint name="j_arm1_2" value="0.320865"/>

File: centauro_urdf/urdf/_centauro_robot.urdf (robot description, URDF)
Before this commit: robot centauro, 58 links, 57 joints
Joints:
- joint d435_head_joint: axis 0 1 0 -> 0 -1 0
- joint velodyne_joint: axis 0 1 0 -> 0 -1 0

File: centauro_urdf/urdf/centauro_base.urdf.xacro (robot description, xacro)
@@ -59,31 +59,4 @@
         </xacro:VLP-16>
     </xacro:if>
-    <link name="d435_head_motor">
-        <inertial>
-        <origin xyz="0 0 0"/>
-        <mass value="0.33878686"/> <!-- MASS/INERTIA TO DO -->
-        <inertia ixx="0.0003718568" ixy="-9.42983e-05" ixz="-2.80644e-05" iyy="0.0001886879" iyz="-1.54534e-05" izz="0.0005023443"/>
-        </inertial>
-        <visual>
-        <origin rpy="0.0 0.0 0.0" xyz="0.0 0 0.0"/>
-        <geometry>
-            <mesh filename="package://centauro_urdf/meshes/neck-pitch_mesh.stl" scale="0.001 0.001 0.001"/>
-        </geometry>
-        </visual>
-        <collision>
-        <origin rpy="0.0 0.0 0.0" xyz="0.0 0 0.0"/>
-        <geometry>
-            <mesh filename="package://centauro_urdf/meshes/simple/neck-pitch_mesh.stl" scale="0.001 0.001 0.001"/>
-        </geometry>
-        </collision>
-    </link>
-    <joint name="d435_head_joint" type="revolute">
-        <parent link="neck_1"/>
-        <origin xyz="0.06 0 0.1375" rpy="0 0 0"/>
-        <child link="d435_head_motor"/>
-        <axis xyz="0 1 0"/>
-        <limit effort="35" lower="-1.1" upper="1.1" velocity="5.7"/>
-        <dynamics friction="10.0"/>
-    </joint>
     <xacro:if value="${ADD_D435_HEAD}">
         <xacro:include filename="$(find realsense_gazebo_description)/urdf/_d435i.urdf.xacro" />

File: centauro_urdf/urdf/centauro_virtual_frame.urdf (robot description, URDF)
Before this commit: robot centauro, 64 links, 63 joints
Joints:
- joint d435_head_joint: axis 0 1 0 -> 0 -1 0
- joint velodyne_joint: axis 0 1 0 -> 0 -1 0

File: centauro_urdf/urdf/centauro_virtual_frame_robot.urdf (robot description, URDF)
Before this commit: robot centauro, 64 links, 63 joints
Joints:
- joint d435_head_joint: axis 0 1 0 -> 0 -1 0
- joint velodyne_joint: axis 0 1 0 -> 0 -1 0

File: centauro_urdf/urdf/parts/head.urdf.xacro (robot description, xacro)
@@ -40,4 +40,23 @@
     </collision>
 </link>
+<link name="d435_head_motor">
+    <inertial>
+    <origin xyz="0 0 0"/>
+    <mass value="0.33878686"/> <!-- MASS/INERTIA TO DO -->
+    <inertia ixx="0.0003718568" ixy="-9.42983e-05" ixz="-2.80644e-05" iyy="0.0001886879" iyz="-1.54534e-05" izz="0.0005023443"/>
+    </inertial>
+    <visual>
+    <origin rpy="0.0 0.0 0.0" xyz="0.0 0 0.0"/>
+    <geometry>
+        <mesh filename="package://centauro_urdf/meshes/neck-pitch_mesh.stl" scale="0.001 0.001 0.001"/>
+    </geometry>
+    </visual>
+    <collision>
+    <origin rpy="0.0 0.0 0.0" xyz="0.0 0 0.0"/>
+    <geometry>
+        <mesh filename="package://centauro_urdf/meshes/simple/neck-pitch_mesh.stl" scale="0.001 0.001 0.001"/>
+    </geometry>
+    </collision>
+</link>
 <!--JOINTS -->
 <joint name="neck_base" type="fixed">
@@ -51,5 +70,13 @@
     <origin xyz="0.0822724 0 0.242" rpy="0 0 0"/>
     <child link="velodyne_motor"/>
-    <axis xyz="0 1 0"/>
+    <axis xyz="0 -1 0"/>
+    <limit effort="35" lower="-1.1" upper="1.1" velocity="5.7"/>
+    <dynamics friction="10.0"/>
+</joint>
+<joint name="d435_head_joint" type="revolute">
+    <parent link="neck_1"/>
+    <origin xyz="0.06 0 0.1375" rpy="0 0 0"/>
+    <child link="d435_head_motor"/>
+    <axis xyz="0 -1 0"/>
     <limit effort="35" lower="-1.1" upper="1.1" velocity="5.7"/>
     <dynamics friction="10.0"/>
