Commit message: xacro && meshes

File: centauro_srdf/srdf/centauro.srdf.xacro (robot description, xacro)
@@ -38,10 +38,14 @@
             <chain base_link="pelvis" tip_link="torso_2" />
         </group>
-        <group name="velodyne">
-            <chain base_link="torso_2" tip_link="neck_3" />
-        </group>
-        <group name="neck">
-            <chain base_link="torso_2" tip_link="neck_2" />
-        </group>
+        <xacro:if value="${ADD_VELODYNE}">
+            <group name="velodyne">
+                <chain base_link="torso_2" tip_link="velodyne_motor" />
+            </group>
+        </xacro:if>
+        <xacro:if value="${ADD_D435I_HEAD}">
+            <group name="d435_head">
+                <chain base_link="torso_2" tip_link="d435_head_motor" />
+            </group>
+        </xacro:if>
     </xacro:if>
     <xacro:if value="${ADD_VIRTUAL_FRAME}">
@@ -61,6 +65,10 @@
             <group name="right_arm" />
             <group name="torso" />
-            <group name="velodyne" />
-            <group name="neck" />
+            <xacro:if value="${ADD_VELODYNE}">
+                <group name="velodyne"/>
+            </xacro:if>
+            <xacro:if value="${ADD_D435I_HEAD}">
+                <group name="d435_head"/>
+            </xacro:if>
         </xacro:if>
         <xacro:if value="${ADD_VIRTUAL_FRAME}">
@@ -91,6 +99,6 @@
         <joint name="ankle_yaw_4" value="0.746874"/>
         <joint name="torso_yaw" value="3.56617e-13"/>
-        <joint name="neck_yaw" value="0."/>
-        <joint name="neck_pitch" value="0.2"/>
+        <joint name="velodyne_joint" value="0"/>
+        <joint name="d435_head_joint" value="0"/>
         <joint name="j_arm1_1" value="0.520149"/>
         <joint name="j_arm1_2" value="0.320865"/>
@@ -108,196 +116,3 @@
         <joint name="j_arm2_7" value="0.0567608"/>
     </group_state>
-    <!--DISABLE COLLISIONS: By default it is assumed that any link of the robot could potentially come into collision with any other link in the robot. This tag disables collision checking between a specified pair of links. -->
-    <disable_collisions link1="ankle1_1" link2="ankle2_1" reason="Adjacent" />
-    <disable_collisions link1="ankle1_1" link2="hip1_1" reason="Never" />
-    <disable_collisions link1="ankle1_1" link2="knee_1" reason="Adjacent" />
-    <disable_collisions link1="ankle1_1" link2="wheel_1" reason="Never" />
-    <disable_collisions link1="ankle1_2" link2="ankle2_2" reason="Adjacent" />
-    <disable_collisions link1="ankle1_2" link2="arm1_1" reason="Never" />
-    <disable_collisions link1="ankle1_2" link2="arm2_1" reason="Never" />
-    <disable_collisions link1="ankle1_2" link2="hip1_2" reason="Never" />
-    <disable_collisions link1="ankle1_2" link2="knee_2" reason="Adjacent" />
-    <disable_collisions link1="ankle1_2" link2="wheel_2" reason="Never" />
-    <disable_collisions link1="ankle1_3" link2="ankle2_3" reason="Adjacent" />
-    <disable_collisions link1="ankle1_3" link2="arm1_1" reason="Never" />
-    <disable_collisions link1="ankle1_3" link2="arm2_1" reason="Never" />
-    <disable_collisions link1="ankle1_3" link2="hip1_3" reason="Never" />
-    <disable_collisions link1="ankle1_3" link2="knee_3" reason="Adjacent" />
-    <disable_collisions link1="ankle1_3" link2="wheel_3" reason="Never" />
-    <disable_collisions link1="ankle1_4" link2="ankle2_4" reason="Adjacent" />
-    <disable_collisions link1="ankle1_4" link2="arm1_1" reason="Never" />
-    <disable_collisions link1="ankle1_4" link2="arm2_1" reason="Never" />
-    <disable_collisions link1="ankle1_4" link2="hip1_4" reason="Never" />
-    <disable_collisions link1="ankle1_4" link2="knee_4" reason="Adjacent" />
-    <disable_collisions link1="ankle1_4" link2="wheel_4" reason="Never" />
-    <disable_collisions link1="ankle2_1" link2="knee_1" reason="Never" />
-    <disable_collisions link1="ankle2_1" link2="wheel_1" reason="Adjacent" />
-    <disable_collisions link1="ankle2_2" link2="knee_2" reason="Never" />
-    <disable_collisions link1="ankle2_2" link2="wheel_2" reason="Adjacent" />
-    <disable_collisions link1="ankle2_3" link2="wheel_3" reason="Adjacent" />
-    <disable_collisions link1="ankle2_4" link2="knee_4" reason="Never" />
-    <disable_collisions link1="ankle2_4" link2="wheel_4" reason="Adjacent" />
-    <disable_collisions link1="arm1_1" link2="arm1_2" reason="Adjacent" />
-    <disable_collisions link1="arm1_1" link2="arm1_3" reason="Never" />
-    <disable_collisions link1="arm1_1" link2="arm1_4" reason="Never" />
-    <disable_collisions link1="arm1_1" link2="arm1_5" reason="Never" />
-    <disable_collisions link1="arm1_1" link2="arm2_1" reason="Never" />
-    <disable_collisions link1="arm1_1" link2="arm2_2" reason="Never" />
-    <disable_collisions link1="arm1_1" link2="arm2_3" reason="Never" />
-    <disable_collisions link1="arm1_1" link2="arm2_4" reason="Never" />
-    <disable_collisions link1="arm1_1" link2="hip1_1" reason="Never" />
-    <disable_collisions link1="arm1_1" link2="hip1_2" reason="Never" />
-    <disable_collisions link1="arm1_1" link2="hip1_3" reason="Never" />
-    <disable_collisions link1="arm1_1" link2="hip1_4" reason="Never" />
-    <disable_collisions link1="arm1_1" link2="hip2_1" reason="Never" />
-    <disable_collisions link1="arm1_1" link2="hip2_2" reason="Never" />
-    <disable_collisions link1="arm1_1" link2="hip2_3" reason="Never" />
-    <disable_collisions link1="arm1_1" link2="hip2_4" reason="Never" />
-    <disable_collisions link1="arm1_1" link2="knee_1" reason="Never" />
-    <disable_collisions link1="arm1_1" link2="knee_2" reason="Never" />
-    <disable_collisions link1="arm1_1" link2="knee_3" reason="Never" />
-    <disable_collisions link1="arm1_1" link2="knee_4" reason="Never" />
-    <disable_collisions link1="arm1_1" link2="pelvis" reason="Never" />
-    <disable_collisions link1="arm1_1" link2="torso_2" reason="Adjacent" />
-    <disable_collisions link1="arm1_2" link2="arm1_3" reason="Adjacent" />
-    <disable_collisions link1="arm1_2" link2="arm1_4" reason="Never" />
-    <disable_collisions link1="arm1_2" link2="arm1_7" reason="Never" />
-    <disable_collisions link1="arm1_2" link2="arm2_1" reason="Never" />
-    <disable_collisions link1="arm1_2" link2="arm2_2" reason="Never" />
-    <disable_collisions link1="arm1_2" link2="arm2_3" reason="Never" />
-    <disable_collisions link1="arm1_2" link2="arm2_4" reason="Never" />
-    <disable_collisions link1="arm1_2" link2="hip1_1" reason="Never" />
-    <disable_collisions link1="arm1_2" link2="hip1_2" reason="Never" />
-    <disable_collisions link1="arm1_2" link2="hip1_3" reason="Never" />
-    <disable_collisions link1="arm1_2" link2="hip1_4" reason="Never" />
-    <disable_collisions link1="arm1_2" link2="hip2_1" reason="Never" />
-    <disable_collisions link1="arm1_2" link2="hip2_2" reason="Never" />
-    <disable_collisions link1="arm1_2" link2="hip2_3" reason="Never" />
-    <disable_collisions link1="arm1_2" link2="hip2_4" reason="Never" />
-    <disable_collisions link1="arm1_2" link2="knee_1" reason="Never" />
-    <disable_collisions link1="arm1_2" link2="knee_4" reason="Never" />
-    <disable_collisions link1="arm1_3" link2="arm1_4" reason="Adjacent" />
-    <disable_collisions link1="arm1_3" link2="arm1_6" reason="Never" />
-    <disable_collisions link1="arm1_3" link2="arm1_7" reason="Never" />
-    <disable_collisions link1="arm1_3" link2="arm2_1" reason="Never" />
-    <disable_collisions link1="arm1_3" link2="arm2_2" reason="Never" />
-    <disable_collisions link1="arm1_3" link2="ft_arm1" reason="Never" />
-    <disable_collisions link1="arm1_3" link2="hip1_1" reason="Never" />
-    <disable_collisions link1="arm1_3" link2="hip1_2" reason="Never" />
-    <disable_collisions link1="arm1_3" link2="hip1_3" reason="Never" />
-    <disable_collisions link1="arm1_3" link2="hip1_4" reason="Never" />
-    <disable_collisions link1="arm1_3" link2="hip2_2" reason="Never" />
-    <disable_collisions link1="arm1_3" link2="hip2_4" reason="Never" />
-    <disable_collisions link1="arm1_4" link2="arm1_5" reason="Adjacent" />
-    <disable_collisions link1="arm1_4" link2="arm1_6" reason="Never" />
-    <disable_collisions link1="arm1_4" link2="arm1_7" reason="Never" />
-    <disable_collisions link1="arm1_4" link2="arm2_1" reason="Never" />
-    <disable_collisions link1="arm1_4" link2="arm2_2" reason="Never" />
-    <disable_collisions link1="arm1_4" link2="ft_arm1" reason="Never" />
-    <disable_collisions link1="arm1_4" link2="hip1_1" reason="Never" />
-    <disable_collisions link1="arm1_4" link2="hip1_2" reason="Never" />
-    <disable_collisions link1="arm1_4" link2="hip1_3" reason="Never" />
-    <disable_collisions link1="arm1_4" link2="hip1_4" reason="Never" />
-    <disable_collisions link1="arm1_5" link2="arm1_6" reason="Adjacent" />
-    <disable_collisions link1="arm1_5" link2="arm1_7" reason="Never" />
-    <disable_collisions link1="arm1_5" link2="ft_arm1" reason="Never" />
-    <disable_collisions link1="arm1_6" link2="arm1_7" reason="Adjacent" />
-    <disable_collisions link1="arm1_6" link2="ft_arm1" reason="Never" />
-    <disable_collisions link1="arm1_7" link2="ft_arm1" reason="Adjacent" />
-    <disable_collisions link1="arm2_1" link2="arm2_2" reason="Adjacent" />
-    <disable_collisions link1="arm2_1" link2="arm2_3" reason="Never" />
-    <disable_collisions link1="arm2_1" link2="arm2_4" reason="Never" />
-    <disable_collisions link1="arm2_1" link2="arm2_5" reason="Never" />
-    <disable_collisions link1="arm2_1" link2="arm2_7" reason="Never" />
-    <disable_collisions link1="arm2_1" link2="hip1_1" reason="Never" />
-    <disable_collisions link1="arm2_1" link2="hip1_2" reason="Never" />
-    <disable_collisions link1="arm2_1" link2="hip1_3" reason="Never" />
-    <disable_collisions link1="arm2_1" link2="hip1_4" reason="Never" />
-    <disable_collisions link1="arm2_1" link2="hip2_1" reason="Never" />
-    <disable_collisions link1="arm2_1" link2="hip2_2" reason="Never" />
-    <disable_collisions link1="arm2_1" link2="hip2_3" reason="Never" />
-    <disable_collisions link1="arm2_1" link2="hip2_4" reason="Never" />
-    <disable_collisions link1="arm2_1" link2="knee_1" reason="Never" />
-    <disable_collisions link1="arm2_1" link2="knee_2" reason="Never" />
-    <disable_collisions link1="arm2_1" link2="knee_3" reason="Never" />
-    <disable_collisions link1="arm2_1" link2="knee_4" reason="Never" />
-    <disable_collisions link1="arm2_1" link2="pelvis" reason="Never" />
-    <disable_collisions link1="arm2_1" link2="torso_2" reason="Adjacent" />
-    <disable_collisions link1="arm2_2" link2="arm2_3" reason="Adjacent" />
-    <disable_collisions link1="arm2_2" link2="arm2_4" reason="Never" />
-    <disable_collisions link1="arm2_2" link2="hip1_1" reason="Never" />
-    <disable_collisions link1="arm2_2" link2="hip1_2" reason="Never" />
-    <disable_collisions link1="arm2_2" link2="hip1_3" reason="Never" />
-    <disable_collisions link1="arm2_2" link2="hip1_4" reason="Never" />
-    <disable_collisions link1="arm2_2" link2="hip2_1" reason="Never" />
-    <disable_collisions link1="arm2_2" link2="hip2_2" reason="Never" />
-    <disable_collisions link1="arm2_2" link2="hip2_3" reason="Never" />
-    <disable_collisions link1="arm2_2" link2="hip2_4" reason="Never" />
-    <disable_collisions link1="arm2_3" link2="arm2_4" reason="Adjacent" />
-    <disable_collisions link1="arm2_3" link2="arm2_6" reason="Never" />
-    <disable_collisions link1="arm2_3" link2="arm2_7" reason="Never" />
-    <disable_collisions link1="arm2_3" link2="ft_arm2" reason="Never" />
-    <disable_collisions link1="arm2_3" link2="hip1_1" reason="Never" />
-    <disable_collisions link1="arm2_3" link2="hip1_2" reason="Never" />
-    <disable_collisions link1="arm2_3" link2="hip1_3" reason="Never" />
-    <disable_collisions link1="arm2_3" link2="hip1_4" reason="Never" />
-    <disable_collisions link1="arm2_3" link2="hip2_1" reason="Never" />
-    <disable_collisions link1="arm2_3" link2="hip2_3" reason="Never" />
-    <disable_collisions link1="arm2_4" link2="arm2_5" reason="Adjacent" />
-    <disable_collisions link1="arm2_4" link2="arm2_6" reason="Never" />
-    <disable_collisions link1="arm2_4" link2="arm2_7" reason="Never" />
-    <disable_collisions link1="arm2_4" link2="ft_arm2" reason="Never" />
-    <disable_collisions link1="arm2_4" link2="hip1_1" reason="Never" />
-    <disable_collisions link1="arm2_4" link2="hip1_2" reason="Never" />
-    <disable_collisions link1="arm2_4" link2="hip1_3" reason="Never" />
-    <disable_collisions link1="arm2_4" link2="hip1_4" reason="Never" />
-    <disable_collisions link1="arm2_5" link2="arm2_6" reason="Adjacent" />
-    <disable_collisions link1="arm2_5" link2="arm2_7" reason="Never" />
-    <disable_collisions link1="arm2_5" link2="ft_arm2" reason="Never" />
-    <disable_collisions link1="arm2_6" link2="arm2_7" reason="Adjacent" />
-    <disable_collisions link1="arm2_6" link2="ft_arm2" reason="Never" />
-    <disable_collisions link1="arm2_7" link2="ft_arm2" reason="Adjacent" />
-    <disable_collisions link1="hip1_1" link2="hip1_2" reason="Never" />
-    <disable_collisions link1="hip1_1" link2="hip1_3" reason="Never" />
-    <disable_collisions link1="hip1_1" link2="hip1_4" reason="Never" />
-    <disable_collisions link1="hip1_1" link2="hip2_1" reason="Adjacent" />
-    <disable_collisions link1="hip1_1" link2="hip2_3" reason="Never" />
-    <disable_collisions link1="hip1_1" link2="hip2_4" reason="Never" />
-    <disable_collisions link1="hip1_1" link2="knee_1" reason="Never" />
-    <disable_collisions link1="hip1_1" link2="pelvis" reason="Adjacent" />
-    <disable_collisions link1="hip1_1" link2="torso_2" reason="Never" />
-    <disable_collisions link1="hip1_2" link2="hip1_3" reason="Never" />
-    <disable_collisions link1="hip1_2" link2="hip1_4" reason="Never" />
-    <disable_collisions link1="hip1_2" link2="hip2_2" reason="Adjacent" />
-    <disable_collisions link1="hip1_2" link2="hip2_3" reason="Never" />
-    <disable_collisions link1="hip1_2" link2="hip2_4" reason="Never" />
-    <disable_collisions link1="hip1_2" link2="knee_2" reason="Never" />
-    <disable_collisions link1="hip1_2" link2="pelvis" reason="Adjacent" />
-    <disable_collisions link1="hip1_2" link2="torso_2" reason="Never" />
-    <disable_collisions link1="hip1_3" link2="hip1_4" reason="Never" />
-    <disable_collisions link1="hip1_3" link2="hip2_1" reason="Never" />
-    <disable_collisions link1="hip1_3" link2="hip2_2" reason="Never" />
-    <disable_collisions link1="hip1_3" link2="hip2_3" reason="Adjacent" />
-    <disable_collisions link1="hip1_3" link2="knee_3" reason="Never" />
-    <disable_collisions link1="hip1_3" link2="pelvis" reason="Adjacent" />
-    <disable_collisions link1="hip1_3" link2="torso_2" reason="Never" />
-    <disable_collisions link1="hip1_4" link2="hip2_1" reason="Never" />
-    <disable_collisions link1="hip1_4" link2="hip2_2" reason="Never" />
-    <disable_collisions link1="hip1_4" link2="hip2_4" reason="Adjacent" />
-    <disable_collisions link1="hip1_4" link2="knee_4" reason="Never" />
-    <disable_collisions link1="hip1_4" link2="pelvis" reason="Adjacent" />
-    <disable_collisions link1="hip1_4" link2="torso_2" reason="Never" />
-    <disable_collisions link1="hip2_1" link2="knee_1" reason="Adjacent" />
-    <disable_collisions link1="hip2_1" link2="torso_2" reason="Never" />
-    <disable_collisions link1="hip2_2" link2="knee_2" reason="Adjacent" />
-    <disable_collisions link1="hip2_2" link2="torso_2" reason="Never" />
-    <disable_collisions link1="hip2_3" link2="knee_3" reason="Adjacent" />
-    <disable_collisions link1="hip2_3" link2="torso_2" reason="Never" />
-    <disable_collisions link1="hip2_4" link2="knee_4" reason="Adjacent" />
-    <disable_collisions link1="hip2_4" link2="torso_2" reason="Never" />
-    <disable_collisions link1="knee_1" link2="wheel_1" reason="Never" />
-    <disable_collisions link1="knee_2" link2="wheel_2" reason="Never" />
-    <disable_collisions link1="knee_3" link2="wheel_3" reason="Never" />
-    <disable_collisions link1="knee_4" link2="wheel_4" reason="Never" />
-    <disable_collisions link1="pelvis" link2="torso_2" reason="Adjacent" />
 </robot>

File: centauro_urdf/urdf/centauro_base.urdf.xacro (robot description, xacro)
@@ -55,14 +55,57 @@
     <xacro:if value="${ADD_VELODYNE}">
         <xacro:include filename="$(find velodyne_description)/urdf/VLP-16.urdf.xacro"/>
-        <xacro:VLP-16 parent="neck_3" name="velodyne_calib" topic="/velodyne_points" hz="10" samples="440">
-            <origin xyz="0.032768 -0.01 0.048219" rpy="0 1.5709 -0.316519  " />
+        <xacro:VLP-16 parent="velodyne_motor" name="velodyne_calib" topic="/velodyne_points" hz="10" samples="440">
+            <origin xyz="0 0 0" rpy="0 0 0" />
         </xacro:VLP-16>
     </xacro:if>
-    <xacro:if value="${ADD_INTEL_D435I}">
+    <xacro:if value="${ADD_D435I_HEAD}">
+        <link name="d435_head_motor">
+            <inertial>
+            <origin xyz="0 0 0"/>
+            <mass value="0.33878686"/> <!-- MASS/INERTIA TO DO -->
+            <inertia ixx="0.0003718568" ixy="-9.42983e-05" ixz="-2.80644e-05" iyy="0.0001886879" iyz="-1.54534e-05" izz="0.0005023443"/>
+            </inertial>
+            <visual>
+            <origin rpy="0.0 0.0 0.0" xyz="0.0 0 0.0"/>
+            <geometry>
+                <mesh filename="package://centauro_urdf/meshes/neck-pitch_mesh.stl" scale="0.001 0.001 0.001"/>
+            </geometry>
+            </visual>
+            <collision>
+            <origin rpy="0.0 0.0 0.0" xyz="0.0 0 0.0"/>
+            <geometry>
+                <mesh filename="package://centauro_urdf/meshes/simple/neck-pitch_mesh.stl" scale="0.001 0.001 0.001"/>
+            </geometry>
+            </collision>
+        </link>
+        <joint name="d435_head_joint" type="revolute">
+            <parent link="neck_1"/>
+            <origin xyz="0.06 0 0.1375" rpy="0 0 0"/>
+            <child link="d435_head_motor"/>
+            <axis xyz="0 1 0"/>
+            <limit effort="35" lower="-1.1" upper="1.1" velocity="5.7"/>
+            <dynamics friction="10.0"/>
+        </joint>
         <xacro:include filename="$(find realsense_gazebo_description)/urdf/_d435i.urdf.xacro" />
-       <!-- <xacro:sensor_d435i parent="torso_2" name="d435i_camera" topics_ns="d435i_camera"
-                            enable_pointCloud="true" align_depth="true">
-            <origin xyz="0.13 0 0.03" rpy="0 0.25 0"/>
-        </xacro:sensor_d435i>-->
+        <xacro:sensor_d435i parent="d435_head_motor" name="D435_head_camera" topics_ns="D435/D435_head_camera"
+                      enable_pointCloud="true" align_depth="true"
+                      unite_imu_method="false"
+                      visualize="false"
+                      accel_fps="300"
+                      gyro_fps="300"
+                      depth_width="1280"
+                      depth_height="720"
+                      depth_fps="90"
+                      infra_width="1280"
+                      infra_height="720"
+                      infra_fps="90"
+                      color_width="1280"
+                      color_height="720"
+                      color_fps="30">
+            <origin xyz="0.03015 0 -0.0125" rpy="0 0 0"/>
+        </xacro:sensor_d435i>
+    </xacro:if>
+    <xacro:if value="${ADD_D435I_BASE}">
+        <xacro:include filename="$(find realsense_gazebo_description)/urdf/_d435i.urdf.xacro" />
         <xacro:sensor_d435i parent="pelvis" name="D435i_camera" topics_ns="D435i/D435i_camera"
                       enable_pointCloud="true" align_depth="true"
@@ -80,15 +123,9 @@
                       color_height="720"
                       color_fps="30">
-            <origin xyz="0.219831 0 -0.0613293" rpy="0.0 0.5585052 0.0"/>
+            <origin xyz="0.27187 0 0.0215997" rpy="0 0.5251508 0"/>
         </xacro:sensor_d435i>
     </xacro:if>
-    <xacro:if value="${ADD_INTEL_T265}">
+    <xacro:if value="${ADD_T265_BASE}">
         <xacro:include filename="$(find realsense_gazebo_description)/urdf/_t265.urdf.xacro" />
-        <!-- unite_imu_method can be false, copy or linear_interpolation -->
-        <!--<xacro:sensor_t265  parent="torso_2" name="T265_camera" topics_ns="T265_camera"
-                      xyz="0.125 0.0 0" rpy="0.0 0.25 0.0"
-                      unite_imu_method="false">
-            <origin xyz="0.125 0.0 0" rpy="0.0 0.25 0.0"/>
-        </xacro:sensor_t265>-->
         <xacro:sensor_t265  parent="pelvis" name="T265_camera" topics_ns="T265/T265_camera"
                       odom_xyz="0.0 0.0 0.25"
@@ -101,5 +138,5 @@
                       accel_fps="62.5"
                       gyro_fps="200">
-            <origin xyz="0.252619 0.00775 -0.0206926" rpy="0.0 0.2617993 0.0" />
+            <origin xyz="0.29245 0.00775 0.063" rpy="0 0 0" />
         </xacro:sensor_t265>
     </xacro:if>

File: centauro_urdf/urdf/config/centauro.urdf.xacro (robot description, xacro)
@@ -18,5 +18,6 @@
 <xacro:property name="USE_STICKS" value="false" />
 <xacro:property name="ADD_VELODYNE" value="$(arg velodyne)" />
-<xacro:property name="ADD_INTEL_D435I" value="$(arg realsense)" />
-<xacro:property name="ADD_INTEL_T265" value="$(arg realsense)" />
+<xacro:property name="ADD_D435I_HEAD" value="$(arg realsense)" />
+<xacro:property name="ADD_D435I_BASE" value="$(arg realsense)" />
+<xacro:property name="ADD_T265_BASE" value="$(arg realsense)" />
 </robot>
