Commit message: xacro && meshes

File: centauro_urdf/urdf/config/centauro_virtual_frame.urdf.xacro (robot description, xacro)
@@ -1,19 +1,20 @@
 <?xml version="1.0"?>
 <robot xmlns:xacro="http://ros.org/wiki/xacro" name="centauro">
-<xacro:property name="model_name" value="centauro" />
-<xacro:property name="model_version" value="0.1" />
-<!-- command line arguments -->
-<xacro:arg name="add_legs" default="true"/>
-<xacro:arg name="add_upper_body" default="true"/>
-<!-- ************SELECT PARTS*************-->
-<!-- *************************************-->
-<xacro:property name="ADD_LEGS" value="$(arg add_legs)" />
-<xacro:property name="ADD_UPPER_BODY" value="$(arg add_upper_body)" />
-<xacro:property name="ADD_BALL_END_EFFECTOR" value="true" />
-<xacro:property name="ADD_FLOATING_BASE" value="$(arg add_legs)" />
-<xacro:property name="ADD_VIRTUAL_FRAME" value="true" />
-<xacro:property name="USE_STICKS" value="false" />
-<xacro:property name="ADD_VELODYNE" value="true" />
-<xacro:property name="ADD_INTEL_D435I" value="true" />
-<xacro:property name="ADD_INTEL_T265" value="true" />
+    <xacro:property name="model_name" value="centauro" />
+    <xacro:property name="model_version" value="0.1" />
+    <!-- command line arguments -->
+    <xacro:arg name="add_legs" default="true"/>
+    <xacro:arg name="add_upper_body" default="true"/>
+    <!-- ************SELECT PARTS*************-->
+    <!-- *************************************-->
+    <xacro:property name="ADD_LEGS" value="$(arg add_legs)" />
+    <xacro:property name="ADD_UPPER_BODY" value="$(arg add_upper_body)" />
+    <xacro:property name="ADD_BALL_END_EFFECTOR" value="true" />
+    <xacro:property name="ADD_FLOATING_BASE" value="$(arg add_legs)" />
+    <xacro:property name="ADD_VIRTUAL_FRAME" value="true" />
+    <xacro:property name="USE_STICKS" value="false" />
+    <xacro:property name="ADD_VELODYNE" value="false" />
+    <xacro:property name="ADD_D435I_HEAD" value="false" />
+    <xacro:property name="ADD_D435I_BASE" value="false" />
+    <xacro:property name="ADD_T265_BASE" value="false" />
 </robot>

File: centauro_urdf/urdf/parts/head.urdf.xacro (robot description, xacro)
@@ -2,9 +2,8 @@
 <robot xmlns:xacro="http://ros.org/wiki/xacro">
 <!-- LINKS -->
-<!-- TODO: FINISH IMPLEMENTATION WITH CORRECT NUMBERS -->
 <link name="neck_1">
     <inertial>
-      <origin xyz="0.040479674 0.021377573 -0.014595112"/>
-      <mass value="0.33878686"/>
+      <origin xyz="0 0 0"/>
+      <mass value="0.33878686"/> <!-- MASS/INERTIA TO DO -->
       <inertia ixx="0.0003718568" ixy="-9.42983e-05" ixz="-2.80644e-05" iyy="0.0001886879" iyz="-1.54534e-05" izz="0.0005023443"/>
     </inertial>
@@ -12,5 +11,5 @@
       <origin rpy="0.0 0.0 0.0" xyz="0.0 0 0.0"/>
       <geometry>
-        <mesh filename="package://centauro_urdf/meshes/neck_yaw.stl" scale="0.001 0.001 0.001"/>
+        <mesh filename="package://centauro_urdf/meshes/head-base_mesh.stl" scale="0.001 0.001 0.001"/>
       </geometry>
     </visual>
@@ -18,18 +17,18 @@
       <origin rpy="0.0 0.0 0.0" xyz="0.0 0 0.0"/>
       <geometry>
-        <mesh filename="package://centauro_urdf/meshes/simple/neck_yaw.stl" scale="0.001 0.001 0.001"/>
+        <mesh filename="package://centauro_urdf/meshes/simple/head-base_mesh.stl" scale="0.001 0.001 0.001"/>
       </geometry>
     </collision>
 </link>
-<link name="neck_2">
+<link name="velodyne_motor">
     <inertial>
-      <origin xyz="0.048466918 -0.059852318 -0.0085314894"/>
-      <mass value="0.78526942"/>
-      <inertia ixx="0.0004682345" ixy="-1.05438e-05" ixz="7.24398e-05" iyy="0.0002635246" iyz="1.6904e-06" izz="0.0003763351"/>
+      <origin xyz="0 0 0"/>
+      <mass value="0.33878686"/> <!-- MASS/INERTIA TO DO -->
+      <inertia ixx="0.0003718568" ixy="-9.42983e-05" ixz="-2.80644e-05" iyy="0.0001886879" iyz="-1.54534e-05" izz="0.0005023443"/>
     </inertial>
     <visual>
       <origin rpy="0.0 0.0 0.0" xyz="0.0 0 0.0"/>
       <geometry>
-        <mesh filename="package://centauro_urdf/meshes/neck_pitch.stl" scale="0.001 0.001 0.001"/>
+        <mesh filename="package://centauro_urdf/meshes/lidar_mesh.stl" scale="0.001 0.001 0.001"/>
       </geometry>
     </visual>
@@ -37,52 +36,22 @@
       <origin rpy="0.0 0.0 0.0" xyz="0.0 0 0.0"/>
       <geometry>
-        <mesh filename="package://centauro_urdf/meshes/simple/neck_pitch.stl" scale="0.001 0.001 0.001"/>
-      </geometry>
-    </collision>
-</link>
-<!-- LINKS -->
-<link name="neck_3">
-    <inertial>
-      <origin xyz="0.048466918 -0.059852318 -0.0085314894"/>
-      <mass value="0.78526942"/>
-      <inertia ixx="0.0004682345" ixy="-1.05438e-05" ixz="7.24398e-05" iyy="0.0002635246" iyz="1.6904e-06" izz="0.0003763351"/>
-    </inertial>
-    <visual>
-      <origin rpy="0.0 0.0 0.0" xyz="0.0 0 0.0"/>
-      <geometry>
-        <mesh filename="package://centauro_urdf/meshes/lidar.stl" scale="0.001 0.001 0.001"/>
-      </geometry>
-    </visual>
-    <collision>
-      <origin rpy="0.0 0.0 0.0" xyz="0.0 0 0.0"/>
-      <geometry>
-        <mesh filename="package://centauro_urdf/meshes/simple/lidar.stl" scale="0.001 0.001 0.001"/>
+        <mesh filename="package://centauro_urdf/meshes/simple/lidar_mesh.stl" scale="0.001 0.001 0.001"/>
       </geometry>
     </collision>
 </link>
 <!--JOINTS -->
-<joint name="neck_yaw" type="revolute">
+<joint name="neck_base" type="fixed">
     <parent link="torso_2"/>
-    <origin xyz="0.0 0.0 0.2795"/>
+    <origin xyz="0.0030637045 0.0061607221 0.224" rpy="0 0 0"/>
     <child link="neck_1"/>
     <axis xyz="0 0 1"/>
-    <limit effort="35" lower="-0.78539816" upper="0.78539816" velocity="5.7"/>
+</joint>
+<joint name="velodyne_joint" type="revolute">
+    <parent link="neck_1"/>
+    <origin xyz="0.0825 0 0.243" rpy="0 0 0"/>
+    <child link="velodyne_motor"/>
+    <axis xyz="0 1 0"/>
+    <limit effort="35" lower="-1.1" upper="1.1" velocity="5.7"/>
     <dynamics friction="10.0"/>
 </joint>
-<joint name="neck_pitch" type="revolute">
-    <parent link="neck_1"/>
-    <origin xyz="0.054 0.0596 -0.0124975"/>
-    <child link="neck_2"/>
-    <axis xyz="0 1 0"/>
-    <limit effort="35" lower="-0.34906585" upper="0.78539816" velocity="5.7"/>
-    <dynamics friction="10.0"/>
-</joint>
-<joint name="neck_velodyne" type="continuous">
-    <parent link="torso_2"/>
-    <origin xyz="0.055 0.0 0.473262" rpy="0 0 0"/>
-    <child link="neck_3"/>
-    <axis xyz="0 0 1"/>
-    <limit effort="35" velocity="5.7"/>
-    <dynamics damping="0.2" friction="10.0"/>
-</joint>
 </robot>

Commit message: latest changes by aled96

File: centauro_srdf/srdf/centauro.srdf.xacro (robot description, xacro)
@@ -38,14 +38,10 @@
             <chain base_link="pelvis" tip_link="torso_2" />
         </group>
-        <xacro:if value="${ADD_VELODYNE}">
-            <group name="velodyne">
-                <chain base_link="torso_2" tip_link="velodyne_motor" />
-            </group>
-        </xacro:if>
-        <xacro:if value="${ADD_D435I_HEAD}">
-            <group name="d435_head">
-                <chain base_link="torso_2" tip_link="d435_head_motor" />
-            </group>
-        </xacro:if>
+        <group name="velodyne">
+            <chain base_link="torso_2" tip_link="velodyne_motor" />
+        </group>
+        <group name="d435_head">
+            <chain base_link="torso_2" tip_link="d435_head_motor" />
+        </group>
     </xacro:if>
     <xacro:if value="${ADD_VIRTUAL_FRAME}">
@@ -65,10 +61,6 @@
             <group name="right_arm" />
             <group name="torso" />
-            <xacro:if value="${ADD_VELODYNE}">
-                <group name="velodyne"/>
-            </xacro:if>
-            <xacro:if value="${ADD_D435I_HEAD}">
-                <group name="d435_head"/>
-            </xacro:if>
+            <group name="velodyne"/>
+            <group name="d435_head"/>
         </xacro:if>
         <xacro:if value="${ADD_VIRTUAL_FRAME}">

File: centauro_urdf/urdf/centauro_base.urdf.xacro (robot description, xacro)
@@ -43,67 +43,5 @@
 	<xacro:include filename="$(find centauro_urdf)/urdf/parts/centauro_torso.urdf.xacro" />
     <xacro:include filename="$(find centauro_urdf)/urdf/parts/arms.urdf.xacro" />
-	<xacro:if value="${ADD_BALL_END_EFFECTOR}">
-		<xacro:include filename="$(find centauro_urdf)/urdf/parts/ball.urdf.xacro" />
-		<xacro:ball_end_effector arm_num="1"  parent_link="arm1_7">
-      			<origin xyz="0. 0. 0." rpy="0. 0. 0."/>
-   		</xacro:ball_end_effector>
-		<xacro:ball_end_effector arm_num="2"  parent_link="arm2_7">
-      			<origin xyz="0. 0. 0." rpy="0. 0. 0."/>
-   		</xacro:ball_end_effector>
-	</xacro:if>
 	<xacro:include filename="$(find centauro_urdf)/urdf/parts/head.urdf.xacro" />
-    <xacro:if value="${ADD_VELODYNE}">
-        <xacro:include filename="$(find velodyne_description)/urdf/VLP-16.urdf.xacro"/>
-        <xacro:VLP-16 parent="velodyne_motor" name="velodyne_calib" topic="/velodyne_points" hz="10" samples="440">
-            <origin xyz="0 0 0" rpy="0 0 0" />
-        </xacro:VLP-16>
-    </xacro:if>
-    <xacro:if value="${ADD_D435I_HEAD}">
-        <link name="d435_head_motor">
-            <inertial>
-            <origin xyz="0 0 0"/>
-            <mass value="0.33878686"/> <!-- MASS/INERTIA TO DO -->
-            <inertia ixx="0.0003718568" ixy="-9.42983e-05" ixz="-2.80644e-05" iyy="0.0001886879" iyz="-1.54534e-05" izz="0.0005023443"/>
-            </inertial>
-            <visual>
-            <origin rpy="0.0 0.0 0.0" xyz="0.0 0 0.0"/>
-            <geometry>
-                <mesh filename="package://centauro_urdf/meshes/neck-pitch_mesh.stl" scale="0.001 0.001 0.001"/>
-            </geometry>
-            </visual>
-            <collision>
-            <origin rpy="0.0 0.0 0.0" xyz="0.0 0 0.0"/>
-            <geometry>
-                <mesh filename="package://centauro_urdf/meshes/simple/neck-pitch_mesh.stl" scale="0.001 0.001 0.001"/>
-            </geometry>
-            </collision>
-        </link>
-        <joint name="d435_head_joint" type="revolute">
-            <parent link="neck_1"/>
-            <origin xyz="0.06 0 0.1375" rpy="0 0 0"/>
-            <child link="d435_head_motor"/>
-            <axis xyz="0 1 0"/>
-            <limit effort="35" lower="-1.1" upper="1.1" velocity="5.7"/>
-            <dynamics friction="10.0"/>
-        </joint>
-        <xacro:include filename="$(find realsense_gazebo_description)/urdf/_d435i.urdf.xacro" />
-        <xacro:sensor_d435i parent="d435_head_motor" name="D435_head_camera" topics_ns="D435/D435_head_camera"
-                      enable_pointCloud="true" align_depth="true"
-                      unite_imu_method="false"
-                      visualize="false"
-                      accel_fps="300"
-                      gyro_fps="300"
-                      depth_width="1280"
-                      depth_height="720"
-                      depth_fps="90"
-                      infra_width="1280"
-                      infra_height="720"
-                      infra_fps="90"
-                      color_width="1280"
-                      color_height="720"
-                      color_fps="30">
-            <origin xyz="0.03015 0 -0.0125" rpy="0 0 0"/>
-        </xacro:sensor_d435i>
-    </xacro:if>
     <xacro:if value="${ADD_D435I_BASE}">
         <xacro:include filename="$(find realsense_gazebo_description)/urdf/_d435i.urdf.xacro" />

File: centauro_urdf/urdf/parts/arms.urdf.xacro (robot description, xacro)
@@ -9,3 +9,12 @@
       <origin xyz="${Shoulder_1_Ox} ${-Shoulder_1_Oy} ${Shoulder_1_Oz}" rpy="${-Shoulder_1_roll} ${Shoulder_1_pitch} ${-Shoulder_1_yaw}" />
 </xacro:centauro_arm>
+<xacro:if value="${ADD_BALL_END_EFFECTOR}">
+      <xacro:include filename="$(find centauro_urdf)/urdf/parts/ball.urdf.xacro" />
+      <xacro:ball_end_effector arm_num="1"  parent_link="arm1_7">
+                  <origin xyz="0. 0. 0." rpy="0. 0. 0."/>
+      </xacro:ball_end_effector>
+      <xacro:ball_end_effector arm_num="2"  parent_link="arm2_7">
+                  <origin xyz="0. 0. 0." rpy="0. 0. 0."/>
+      </xacro:ball_end_effector>
+</xacro:if>
 </robot>

File: centauro_urdf/urdf/parts/head.urdf.xacro (robot description, xacro)
@@ -1,9 +1,10 @@
 <?xml version="1.0"?>
 <robot xmlns:xacro="http://ros.org/wiki/xacro">
-<!-- LINKS -->
-<link name="neck_1">
+  <!-- LINKS -->
+  <link name="neck_1">
     <inertial>
       <origin xyz="0 0 0"/>
-      <mass value="0.33878686"/> <!-- MASS/INERTIA TO DO -->
+      <mass value="0.33878686"/>
+      <!-- MASS/INERTIA TO DO -->
       <inertia ixx="0.0003718568" ixy="-9.42983e-05" ixz="-2.80644e-05" iyy="0.0001886879" iyz="-1.54534e-05" izz="0.0005023443"/>
     </inertial>
@@ -20,9 +21,10 @@
       </geometry>
     </collision>
-</link>
-<link name="velodyne_motor">
+  </link>
+  <link name="velodyne_motor">
     <inertial>
       <origin xyz="0 0 0"/>
-      <mass value="0.33878686"/> <!-- MASS/INERTIA TO DO -->
+      <mass value="0.33878686"/>
+      <!-- MASS/INERTIA TO DO -->
       <inertia ixx="0.0003718568" ixy="-9.42983e-05" ixz="-2.80644e-05" iyy="0.0001886879" iyz="-1.54534e-05" izz="0.0005023443"/>
     </inertial>
@@ -39,19 +41,76 @@
       </geometry>
     </collision>
-</link>
-<!--JOINTS -->
-<joint name="neck_base" type="fixed">
+  </link>
+  <link name="d435_head_motor">
+    <inertial>
+      <origin xyz="0 0 0"/>
+      <mass value="0.33878686"/>
+      <!-- MASS/INERTIA TO DO -->
+      <inertia ixx="0.0003718568" ixy="-9.42983e-05" ixz="-2.80644e-05" iyy="0.0001886879" iyz="-1.54534e-05" izz="0.0005023443"/>
+    </inertial>
+    <visual>
+      <origin rpy="0.0 0.0 0.0" xyz="0.0 0 0.0"/>
+      <geometry>
+        <mesh filename="package://centauro_urdf/meshes/neck-pitch_mesh.stl" scale="0.001 0.001 0.001"/>
+      </geometry>
+    </visual>
+    <collision>
+      <origin rpy="0.0 0.0 0.0" xyz="0.0 0 0.0"/>
+      <geometry>
+        <mesh filename="package://centauro_urdf/meshes/simple/neck-pitch_mesh.stl" scale="0.001 0.001 0.001"/>
+      </geometry>
+    </collision>
+  </link>
+  <!--JOINTS -->
+  <joint name="neck_base" type="fixed">
     <parent link="torso_2"/>
-    <origin xyz="0.0030637045 0.0061607221 0.224" rpy="0 0 0"/>
+    <origin xyz="0.0030637045 0.0061607221 0.158" rpy="0 0 0"/>
     <child link="neck_1"/>
     <axis xyz="0 0 1"/>
-</joint>
-<joint name="velodyne_joint" type="revolute">
+  </joint>
+  <joint name="velodyne_joint" type="revolute">
     <parent link="neck_1"/>
-    <origin xyz="0.0825 0 0.243" rpy="0 0 0"/>
+    <origin xyz="0.0822724 0 0.242" rpy="0 0 0"/>
     <child link="velodyne_motor"/>
-    <axis xyz="0 1 0"/>
+    <axis xyz="0 -1 0"/>
     <limit effort="35" lower="-1.1" upper="1.1" velocity="5.7"/>
     <dynamics friction="10.0"/>
-</joint>
+  </joint>
+  <joint name="d435_head_joint" type="revolute">
+    <parent link="neck_1"/>
+    <origin xyz="0.06 0 0.1375" rpy="0 0 0"/>
+    <child link="d435_head_motor"/>
+    <axis xyz="0 -1 0"/>
+    <limit effort="35" lower="-1.1" upper="1.1" velocity="5.7"/>
+    <dynamics friction="10.0"/>
+  </joint>
+  <xacro:if value="${ADD_D435I_HEAD}">
+    <xacro:include filename="$(find realsense_gazebo_description)/urdf/_d435i.urdf.xacro" />
+    <xacro:sensor_d435i parent="d435_head_motor"
+        name="D435_head_camera"
+        topics_ns="D435/D435_head_camera"
+        enable_pointCloud="true"
+        align_depth="true"
+        unite_imu_method="false"
+        visualize="false"
+        accel_fps="300"
+        gyro_fps="300"
+        depth_width="1280"
+        depth_height="720"
+        depth_fps="90"
+        infra_width="1280"
+        infra_height="720"
+        infra_fps="90"
+        color_width="1280"
+        color_height="720"
+        color_fps="30">
+      <origin xyz="0.03015 0 -0.0125" rpy="0 0 0"/>
+    </xacro:sensor_d435i>
+  </xacro:if>
+  <xacro:if value="${ADD_VELODYNE}">
+    <xacro:include filename="$(find velodyne_description)/urdf/VLP-16.urdf.xacro"/>
+    <xacro:VLP-16 parent="velodyne_motor" name="velodyne_calib" topic="/velodyne_points" hz="10" samples="440">
+        <origin xyz="0 0 0" rpy="0 0 0" />
+    </xacro:VLP-16>
+  </xacro:if>
 </robot>
