Commit message: modification for working with reduced model

File: centauro_srdf/srdf/centauro.srdf.xacro (robot description, xacro)
@@ -51,16 +51,16 @@
     </xacro:if>
     <group name="chains">        <!--THIS HAS TO BE THE LAST GROUP IN THE FILE -->
-        <xacro:if value="${ADD_LEGS}">
+        <!--xacro:if value="${ADD_LEGS}">
             <group name="front_left_leg" />
             <group name="front_right_leg" />
             <group name="rear_right_leg" />
             <group name="rear_left_leg" />
-        </xacro:if>
+        </xacro:if-->
         <xacro:if value="${ADD_UPPER_BODY}">
             <group name="left_arm" />
-            <group name="right_arm" />
+            <!--group name="right_arm" />
             <group name="torso" />
             <group name="velodyne"/>
-            <group name="d435_head"/>
+            <group name="d435_head"/-->
         </xacro:if>
         <xacro:if value="${ADD_VIRTUAL_FRAME}">
@@ -108,3 +108,398 @@
         <joint name="j_arm2_7" value="0.0567608"/>
     </group_state>
+    <disable_collisions link1="D435_head_camera_link" link2="D435i_camera_link" reason="Never"/>
+    <disable_collisions link1="D435_head_camera_link" link2="T265_camera_pose_frame" reason="Never"/>
+    <disable_collisions link1="D435_head_camera_link" link2="ankle1_1" reason="Never"/>
+    <disable_collisions link1="D435_head_camera_link" link2="ankle1_2" reason="Never"/>
+    <disable_collisions link1="D435_head_camera_link" link2="ankle1_3" reason="Never"/>
+    <disable_collisions link1="D435_head_camera_link" link2="ankle1_4" reason="Never"/>
+    <disable_collisions link1="D435_head_camera_link" link2="ankle2_1" reason="Never"/>
+    <disable_collisions link1="D435_head_camera_link" link2="ankle2_2" reason="Never"/>
+    <disable_collisions link1="D435_head_camera_link" link2="ankle2_3" reason="Never"/>
+    <disable_collisions link1="D435_head_camera_link" link2="ankle2_4" reason="Never"/>
+    <disable_collisions link1="D435_head_camera_link" link2="arm1_1" reason="Never"/>
+    <disable_collisions link1="D435_head_camera_link" link2="arm1_2" reason="Never"/>
+    <disable_collisions link1="D435_head_camera_link" link2="arm2_1" reason="Never"/>
+    <disable_collisions link1="D435_head_camera_link" link2="arm2_2" reason="Never"/>
+    <disable_collisions link1="D435_head_camera_link" link2="d435_head_motor" reason="Adjacent"/>
+    <disable_collisions link1="D435_head_camera_link" link2="hip1_1" reason="Never"/>
+    <disable_collisions link1="D435_head_camera_link" link2="hip1_2" reason="Never"/>
+    <disable_collisions link1="D435_head_camera_link" link2="hip1_3" reason="Never"/>
+    <disable_collisions link1="D435_head_camera_link" link2="hip1_4" reason="Never"/>
+    <disable_collisions link1="D435_head_camera_link" link2="hip2_1" reason="Never"/>
+    <disable_collisions link1="D435_head_camera_link" link2="hip2_2" reason="Never"/>
+    <disable_collisions link1="D435_head_camera_link" link2="hip2_3" reason="Never"/>
+    <disable_collisions link1="D435_head_camera_link" link2="hip2_4" reason="Never"/>
+    <disable_collisions link1="D435_head_camera_link" link2="knee_1" reason="Never"/>
+    <disable_collisions link1="D435_head_camera_link" link2="knee_2" reason="Never"/>
+    <disable_collisions link1="D435_head_camera_link" link2="knee_3" reason="Never"/>
+    <disable_collisions link1="D435_head_camera_link" link2="knee_4" reason="Never"/>
+    <disable_collisions link1="D435_head_camera_link" link2="neck_1" reason="Never"/>
+    <disable_collisions link1="D435_head_camera_link" link2="pelvis" reason="Never"/>
+    <disable_collisions link1="D435_head_camera_link" link2="torso_2" reason="Never"/>
+    <disable_collisions link1="D435_head_camera_link" link2="velodyne_calib_base_link" reason="Never"/>
+    <disable_collisions link1="D435_head_camera_link" link2="velodyne_motor" reason="Never"/>
+    <disable_collisions link1="D435_head_camera_link" link2="wheel_2" reason="Never"/>
+    <disable_collisions link1="D435_head_camera_link" link2="wheel_3" reason="Never"/>
+    <disable_collisions link1="D435_head_camera_link" link2="wheel_4" reason="Never"/>
+    <disable_collisions link1="D435i_camera_link" link2="T265_camera_pose_frame" reason="Never"/>
+    <disable_collisions link1="D435i_camera_link" link2="arm1_1" reason="Never"/>
+    <disable_collisions link1="D435i_camera_link" link2="arm1_2" reason="Never"/>
+    <disable_collisions link1="D435i_camera_link" link2="arm1_3" reason="Never"/>
+    <disable_collisions link1="D435i_camera_link" link2="arm1_4" reason="Never"/>
+    <disable_collisions link1="D435i_camera_link" link2="arm2_1" reason="Never"/>
+    <disable_collisions link1="D435i_camera_link" link2="arm2_2" reason="Never"/>
+    <disable_collisions link1="D435i_camera_link" link2="arm2_3" reason="Never"/>
+    <disable_collisions link1="D435i_camera_link" link2="arm2_4" reason="Never"/>
+    <disable_collisions link1="D435i_camera_link" link2="d435_head_motor" reason="Never"/>
+    <disable_collisions link1="D435i_camera_link" link2="hip1_1" reason="Never"/>
+    <disable_collisions link1="D435i_camera_link" link2="hip1_2" reason="Never"/>
+    <disable_collisions link1="D435i_camera_link" link2="hip1_3" reason="Never"/>
+    <disable_collisions link1="D435i_camera_link" link2="hip1_4" reason="Never"/>
+    <disable_collisions link1="D435i_camera_link" link2="hip2_3" reason="Never"/>
+    <disable_collisions link1="D435i_camera_link" link2="hip2_4" reason="Never"/>
+    <disable_collisions link1="D435i_camera_link" link2="neck_1" reason="Never"/>
+    <disable_collisions link1="D435i_camera_link" link2="pelvis" reason="Adjacent"/>
+    <disable_collisions link1="D435i_camera_link" link2="torso_2" reason="Never"/>
+    <disable_collisions link1="D435i_camera_link" link2="velodyne_calib_base_link" reason="Never"/>
+    <disable_collisions link1="D435i_camera_link" link2="velodyne_motor" reason="Never"/>
+    <disable_collisions link1="T265_camera_pose_frame" link2="arm1_1" reason="Never"/>
+    <disable_collisions link1="T265_camera_pose_frame" link2="arm1_2" reason="Never"/>
+    <disable_collisions link1="T265_camera_pose_frame" link2="arm1_3" reason="Never"/>
+    <disable_collisions link1="T265_camera_pose_frame" link2="arm2_1" reason="Never"/>
+    <disable_collisions link1="T265_camera_pose_frame" link2="arm2_2" reason="Never"/>
+    <disable_collisions link1="T265_camera_pose_frame" link2="arm2_3" reason="Never"/>
+    <disable_collisions link1="T265_camera_pose_frame" link2="d435_head_motor" reason="Never"/>
+    <disable_collisions link1="T265_camera_pose_frame" link2="hip1_1" reason="Never"/>
+    <disable_collisions link1="T265_camera_pose_frame" link2="hip1_2" reason="Never"/>
+    <disable_collisions link1="T265_camera_pose_frame" link2="hip1_3" reason="Never"/>
+    <disable_collisions link1="T265_camera_pose_frame" link2="hip1_4" reason="Never"/>
+    <disable_collisions link1="T265_camera_pose_frame" link2="hip2_1" reason="Never"/>
+    <disable_collisions link1="T265_camera_pose_frame" link2="hip2_2" reason="Never"/>
+    <disable_collisions link1="T265_camera_pose_frame" link2="hip2_3" reason="Never"/>
+    <disable_collisions link1="T265_camera_pose_frame" link2="hip2_4" reason="Never"/>
+    <disable_collisions link1="T265_camera_pose_frame" link2="knee_3" reason="Never"/>
+    <disable_collisions link1="T265_camera_pose_frame" link2="knee_4" reason="Never"/>
+    <disable_collisions link1="T265_camera_pose_frame" link2="neck_1" reason="Never"/>
+    <disable_collisions link1="T265_camera_pose_frame" link2="pelvis" reason="Adjacent"/>
+    <disable_collisions link1="T265_camera_pose_frame" link2="torso_2" reason="Never"/>
+    <disable_collisions link1="T265_camera_pose_frame" link2="velodyne_calib_base_link" reason="Never"/>
+    <disable_collisions link1="T265_camera_pose_frame" link2="velodyne_motor" reason="Never"/>
+    <disable_collisions link1="ankle1_1" link2="ankle2_1" reason="Adjacent"/>
+    <disable_collisions link1="ankle1_1" link2="d435_head_motor" reason="Never"/>
+    <disable_collisions link1="ankle1_1" link2="hip1_1" reason="Never"/>
+    <disable_collisions link1="ankle1_1" link2="knee_1" reason="Adjacent"/>
+    <disable_collisions link1="ankle1_1" link2="neck_1" reason="Never"/>
+    <disable_collisions link1="ankle1_1" link2="velodyne_calib_base_link" reason="Never"/>
+    <disable_collisions link1="ankle1_1" link2="velodyne_motor" reason="Never"/>
+    <disable_collisions link1="ankle1_1" link2="wheel_1" reason="Never"/>
+    <disable_collisions link1="ankle1_2" link2="ankle2_2" reason="Adjacent"/>
+    <disable_collisions link1="ankle1_2" link2="arm1_1" reason="Never"/>
+    <disable_collisions link1="ankle1_2" link2="d435_head_motor" reason="Never"/>
+    <disable_collisions link1="ankle1_2" link2="hip1_2" reason="Never"/>
+    <disable_collisions link1="ankle1_2" link2="knee_2" reason="Adjacent"/>
+    <disable_collisions link1="ankle1_2" link2="neck_1" reason="Never"/>
+    <disable_collisions link1="ankle1_2" link2="velodyne_calib_base_link" reason="Never"/>
+    <disable_collisions link1="ankle1_2" link2="velodyne_motor" reason="Never"/>
+    <disable_collisions link1="ankle1_2" link2="wheel_2" reason="Never"/>
+    <disable_collisions link1="ankle1_3" link2="ankle2_3" reason="Adjacent"/>
+    <disable_collisions link1="ankle1_3" link2="arm1_1" reason="Never"/>
+    <disable_collisions link1="ankle1_3" link2="arm2_1" reason="Never"/>
+    <disable_collisions link1="ankle1_3" link2="d435_head_motor" reason="Never"/>
+    <disable_collisions link1="ankle1_3" link2="hip1_3" reason="Never"/>
+    <disable_collisions link1="ankle1_3" link2="knee_3" reason="Adjacent"/>
+    <disable_collisions link1="ankle1_3" link2="neck_1" reason="Never"/>
+    <disable_collisions link1="ankle1_3" link2="velodyne_calib_base_link" reason="Never"/>
+    <disable_collisions link1="ankle1_3" link2="velodyne_motor" reason="Never"/>
+    <disable_collisions link1="ankle1_3" link2="wheel_3" reason="Never"/>
+    <disable_collisions link1="ankle1_4" link2="ankle2_4" reason="Adjacent"/>
+    <disable_collisions link1="ankle1_4" link2="arm1_1" reason="Never"/>
+    <disable_collisions link1="ankle1_4" link2="arm2_1" reason="Never"/>
+    <disable_collisions link1="ankle1_4" link2="d435_head_motor" reason="Never"/>
+    <disable_collisions link1="ankle1_4" link2="hip1_4" reason="Never"/>
+    <disable_collisions link1="ankle1_4" link2="knee_4" reason="Adjacent"/>
+    <disable_collisions link1="ankle1_4" link2="neck_1" reason="Never"/>
+    <disable_collisions link1="ankle1_4" link2="velodyne_calib_base_link" reason="Never"/>
+    <disable_collisions link1="ankle1_4" link2="velodyne_motor" reason="Never"/>
+    <disable_collisions link1="ankle1_4" link2="wheel_4" reason="Never"/>
+    <disable_collisions link1="ankle2_1" link2="d435_head_motor" reason="Never"/>
+    <disable_collisions link1="ankle2_1" link2="knee_1" reason="Never"/>
+    <disable_collisions link1="ankle2_1" link2="velodyne_calib_base_link" reason="Never"/>
+    <disable_collisions link1="ankle2_1" link2="velodyne_motor" reason="Never"/>
+    <disable_collisions link1="ankle2_1" link2="wheel_1" reason="Adjacent"/>
+    <disable_collisions link1="ankle2_2" link2="d435_head_motor" reason="Never"/>
+    <disable_collisions link1="ankle2_2" link2="knee_2" reason="Never"/>
+    <disable_collisions link1="ankle2_2" link2="velodyne_calib_base_link" reason="Never"/>
+    <disable_collisions link1="ankle2_2" link2="velodyne_motor" reason="Never"/>
+    <disable_collisions link1="ankle2_2" link2="wheel_2" reason="Adjacent"/>
+    <disable_collisions link1="ankle2_3" link2="d435_head_motor" reason="Never"/>
+    <disable_collisions link1="ankle2_3" link2="velodyne_calib_base_link" reason="Never"/>
+    <disable_collisions link1="ankle2_3" link2="velodyne_motor" reason="Never"/>
+    <disable_collisions link1="ankle2_3" link2="wheel_3" reason="Adjacent"/>
+    <disable_collisions link1="ankle2_4" link2="d435_head_motor" reason="Never"/>
+    <disable_collisions link1="ankle2_4" link2="knee_4" reason="Never"/>
+    <disable_collisions link1="ankle2_4" link2="velodyne_calib_base_link" reason="Never"/>
+    <disable_collisions link1="ankle2_4" link2="velodyne_motor" reason="Never"/>
+    <disable_collisions link1="ankle2_4" link2="wheel_4" reason="Adjacent"/>
+    <disable_collisions link1="arm1_1" link2="arm1_2" reason="Adjacent"/>
+    <disable_collisions link1="arm1_1" link2="arm1_3" reason="Never"/>
+    <disable_collisions link1="arm1_1" link2="arm1_4" reason="Never"/>
+    <disable_collisions link1="arm1_1" link2="arm1_5" reason="Never"/>
+    <disable_collisions link1="arm1_1" link2="arm1_6" reason="Never"/>
+    <disable_collisions link1="arm1_1" link2="arm1_7" reason="Never"/>
+    <disable_collisions link1="arm1_1" link2="arm2_1" reason="Never"/>
+    <disable_collisions link1="arm1_1" link2="arm2_2" reason="Never"/>
+    <disable_collisions link1="arm1_1" link2="arm2_3" reason="Never"/>
+    <disable_collisions link1="arm1_1" link2="arm2_4" reason="Never"/>
+    <disable_collisions link1="arm1_1" link2="d435_head_motor" reason="Never"/>
+    <disable_collisions link1="arm1_1" link2="hip1_1" reason="Never"/>
+    <disable_collisions link1="arm1_1" link2="hip1_2" reason="Never"/>
+    <disable_collisions link1="arm1_1" link2="hip1_3" reason="Never"/>
+    <disable_collisions link1="arm1_1" link2="hip1_4" reason="Never"/>
+    <disable_collisions link1="arm1_1" link2="hip2_1" reason="Never"/>
+    <disable_collisions link1="arm1_1" link2="hip2_2" reason="Never"/>
+    <disable_collisions link1="arm1_1" link2="hip2_3" reason="Never"/>
+    <disable_collisions link1="arm1_1" link2="hip2_4" reason="Never"/>
+    <disable_collisions link1="arm1_1" link2="knee_1" reason="Never"/>
+    <disable_collisions link1="arm1_1" link2="knee_2" reason="Never"/>
+    <disable_collisions link1="arm1_1" link2="knee_3" reason="Never"/>
+    <disable_collisions link1="arm1_1" link2="knee_4" reason="Never"/>
+    <disable_collisions link1="arm1_1" link2="neck_1" reason="Never"/>
+    <disable_collisions link1="arm1_1" link2="pelvis" reason="Never"/>
+    <disable_collisions link1="arm1_1" link2="torso_2" reason="Adjacent"/>
+    <disable_collisions link1="arm1_1" link2="velodyne_calib_base_link" reason="Never"/>
+    <disable_collisions link1="arm1_1" link2="velodyne_motor" reason="Never"/>
+    <disable_collisions link1="arm1_2" link2="arm1_3" reason="Adjacent"/>
+    <disable_collisions link1="arm1_2" link2="arm1_4" reason="Never"/>
+    <disable_collisions link1="arm1_2" link2="arm1_6" reason="Never"/>
+    <disable_collisions link1="arm1_2" link2="arm1_7" reason="Never"/>
+    <disable_collisions link1="arm1_2" link2="arm2_1" reason="Never"/>
+    <disable_collisions link1="arm1_2" link2="arm2_2" reason="Never"/>
+    <disable_collisions link1="arm1_2" link2="arm2_3" reason="Never"/>
+    <disable_collisions link1="arm1_2" link2="arm2_4" reason="Never"/>
+    <disable_collisions link1="arm1_2" link2="d435_head_motor" reason="Never"/>
+    <disable_collisions link1="arm1_2" link2="hip1_1" reason="Never"/>
+    <disable_collisions link1="arm1_2" link2="hip1_2" reason="Never"/>
+    <disable_collisions link1="arm1_2" link2="hip1_3" reason="Never"/>
+    <disable_collisions link1="arm1_2" link2="hip1_4" reason="Never"/>
+    <disable_collisions link1="arm1_2" link2="hip2_1" reason="Never"/>
+    <disable_collisions link1="arm1_2" link2="hip2_2" reason="Never"/>
+    <disable_collisions link1="arm1_2" link2="hip2_3" reason="Never"/>
+    <disable_collisions link1="arm1_2" link2="hip2_4" reason="Never"/>
+    <disable_collisions link1="arm1_2" link2="neck_1" reason="Never"/>
+    <disable_collisions link1="arm1_2" link2="velodyne_calib_base_link" reason="Never"/>
+    <disable_collisions link1="arm1_2" link2="velodyne_motor" reason="Never"/>
+    <disable_collisions link1="arm1_3" link2="arm1_4" reason="Adjacent"/>
+    <disable_collisions link1="arm1_3" link2="arm1_6" reason="Never"/>
+    <disable_collisions link1="arm1_3" link2="arm1_7" reason="Never"/>
+    <disable_collisions link1="arm1_3" link2="arm2_1" reason="Never"/>
+    <disable_collisions link1="arm1_3" link2="arm2_2" reason="Never"/>
+    <disable_collisions link1="arm1_3" link2="ball1" reason="Never"/>
+    <disable_collisions link1="arm1_3" link2="hip1_1" reason="Never"/>
+    <disable_collisions link1="arm1_3" link2="hip1_2" reason="Never"/>
+    <disable_collisions link1="arm1_3" link2="hip1_3" reason="Never"/>
+    <disable_collisions link1="arm1_3" link2="hip1_4" reason="Never"/>
+    <disable_collisions link1="arm1_3" link2="hip2_1" reason="Never"/>
+    <disable_collisions link1="arm1_3" link2="hip2_3" reason="Never"/>
+    <disable_collisions link1="arm1_3" link2="torso_2" reason="Never"/>
+    <disable_collisions link1="arm1_4" link2="arm1_5" reason="Adjacent"/>
+    <disable_collisions link1="arm1_4" link2="arm1_6" reason="Never"/>
+    <disable_collisions link1="arm1_4" link2="arm1_7" reason="Never"/>
+    <disable_collisions link1="arm1_4" link2="arm2_1" reason="Never"/>
+    <disable_collisions link1="arm1_4" link2="arm2_2" reason="Never"/>
+    <disable_collisions link1="arm1_4" link2="ball1" reason="Never"/>
+    <disable_collisions link1="arm1_4" link2="hip1_1" reason="Never"/>
+    <disable_collisions link1="arm1_4" link2="hip1_2" reason="Never"/>
+    <disable_collisions link1="arm1_4" link2="hip1_3" reason="Never"/>
+    <disable_collisions link1="arm1_4" link2="hip1_4" reason="Never"/>
+    <disable_collisions link1="arm1_4" link2="torso_2" reason="Never"/>
+    <disable_collisions link1="arm1_5" link2="arm1_6" reason="Adjacent"/>
+    <disable_collisions link1="arm1_5" link2="arm1_7" reason="Never"/>
+    <disable_collisions link1="arm1_5" link2="ball1" reason="Never"/>
+    <disable_collisions link1="arm1_6" link2="arm1_7" reason="Adjacent"/>
+    <disable_collisions link1="arm1_6" link2="ball1" reason="Default"/>
+    <disable_collisions link1="arm1_7" link2="ball1" reason="Adjacent"/>
+    <disable_collisions link1="arm2_1" link2="arm2_2" reason="Adjacent"/>
+    <disable_collisions link1="arm2_1" link2="arm2_3" reason="Never"/>
+    <disable_collisions link1="arm2_1" link2="arm2_4" reason="Never"/>
+    <disable_collisions link1="arm2_1" link2="arm2_5" reason="Never"/>
+    <disable_collisions link1="arm2_1" link2="d435_head_motor" reason="Never"/>
+    <disable_collisions link1="arm2_1" link2="hip1_1" reason="Never"/>
+    <disable_collisions link1="arm2_1" link2="hip1_2" reason="Never"/>
+    <disable_collisions link1="arm2_1" link2="hip1_3" reason="Never"/>
+    <disable_collisions link1="arm2_1" link2="hip1_4" reason="Never"/>
+    <disable_collisions link1="arm2_1" link2="hip2_1" reason="Never"/>
+    <disable_collisions link1="arm2_1" link2="hip2_2" reason="Never"/>
+    <disable_collisions link1="arm2_1" link2="hip2_3" reason="Never"/>
+    <disable_collisions link1="arm2_1" link2="hip2_4" reason="Never"/>
+    <disable_collisions link1="arm2_1" link2="knee_1" reason="Never"/>
+    <disable_collisions link1="arm2_1" link2="knee_2" reason="Never"/>
+    <disable_collisions link1="arm2_1" link2="knee_3" reason="Never"/>
+    <disable_collisions link1="arm2_1" link2="knee_4" reason="Never"/>
+    <disable_collisions link1="arm2_1" link2="neck_1" reason="Never"/>
+    <disable_collisions link1="arm2_1" link2="pelvis" reason="Never"/>
+    <disable_collisions link1="arm2_1" link2="torso_2" reason="Adjacent"/>
+    <disable_collisions link1="arm2_1" link2="velodyne_calib_base_link" reason="Never"/>
+    <disable_collisions link1="arm2_1" link2="velodyne_motor" reason="Never"/>
+    <disable_collisions link1="arm2_2" link2="arm2_3" reason="Adjacent"/>
+    <disable_collisions link1="arm2_2" link2="arm2_4" reason="Never"/>
+    <disable_collisions link1="arm2_2" link2="d435_head_motor" reason="Never"/>
+    <disable_collisions link1="arm2_2" link2="hip1_1" reason="Never"/>
+    <disable_collisions link1="arm2_2" link2="hip1_2" reason="Never"/>
+    <disable_collisions link1="arm2_2" link2="hip1_3" reason="Never"/>
+    <disable_collisions link1="arm2_2" link2="hip1_4" reason="Never"/>
+    <disable_collisions link1="arm2_2" link2="hip2_1" reason="Never"/>
+    <disable_collisions link1="arm2_2" link2="hip2_2" reason="Never"/>
+    <disable_collisions link1="arm2_2" link2="hip2_3" reason="Never"/>
+    <disable_collisions link1="arm2_2" link2="hip2_4" reason="Never"/>
+    <disable_collisions link1="arm2_2" link2="knee_1" reason="Never"/>
+    <disable_collisions link1="arm2_2" link2="neck_1" reason="Never"/>
+    <disable_collisions link1="arm2_2" link2="velodyne_calib_base_link" reason="Never"/>
+    <disable_collisions link1="arm2_2" link2="velodyne_motor" reason="Never"/>
+    <disable_collisions link1="arm2_3" link2="arm2_4" reason="Adjacent"/>
+    <disable_collisions link1="arm2_3" link2="arm2_6" reason="Never"/>
+    <disable_collisions link1="arm2_3" link2="arm2_7" reason="Never"/>
+    <disable_collisions link1="arm2_3" link2="ball2" reason="Never"/>
+    <disable_collisions link1="arm2_3" link2="hip1_1" reason="Never"/>
+    <disable_collisions link1="arm2_3" link2="hip1_2" reason="Never"/>
+    <disable_collisions link1="arm2_3" link2="hip1_3" reason="Never"/>
+    <disable_collisions link1="arm2_3" link2="hip1_4" reason="Never"/>
+    <disable_collisions link1="arm2_3" link2="hip2_3" reason="Never"/>
+    <disable_collisions link1="arm2_3" link2="torso_2" reason="Never"/>
+    <disable_collisions link1="arm2_4" link2="arm2_5" reason="Adjacent"/>
+    <disable_collisions link1="arm2_4" link2="arm2_6" reason="Never"/>
+    <disable_collisions link1="arm2_4" link2="arm2_7" reason="Never"/>
+    <disable_collisions link1="arm2_4" link2="ball2" reason="Never"/>
+    <disable_collisions link1="arm2_4" link2="hip1_1" reason="Never"/>
+    <disable_collisions link1="arm2_4" link2="hip1_2" reason="Never"/>
+    <disable_collisions link1="arm2_4" link2="hip1_3" reason="Never"/>
+    <disable_collisions link1="arm2_4" link2="hip1_4" reason="Never"/>
+    <disable_collisions link1="arm2_4" link2="torso_2" reason="Never"/>
+    <disable_collisions link1="arm2_5" link2="arm2_6" reason="Adjacent"/>
+    <disable_collisions link1="arm2_5" link2="arm2_7" reason="Never"/>
+    <disable_collisions link1="arm2_5" link2="ball2" reason="Never"/>
+    <disable_collisions link1="arm2_6" link2="arm2_7" reason="Adjacent"/>
+    <disable_collisions link1="arm2_6" link2="ball2" reason="Default"/>
+    <disable_collisions link1="arm2_7" link2="ball2" reason="Adjacent"/>
+    <disable_collisions link1="d435_head_motor" link2="hip1_1" reason="Never"/>
+    <disable_collisions link1="d435_head_motor" link2="hip1_2" reason="Never"/>
+    <disable_collisions link1="d435_head_motor" link2="hip1_3" reason="Never"/>
+    <disable_collisions link1="d435_head_motor" link2="hip1_4" reason="Never"/>
+    <disable_collisions link1="d435_head_motor" link2="hip2_1" reason="Never"/>
+    <disable_collisions link1="d435_head_motor" link2="hip2_2" reason="Never"/>
+    <disable_collisions link1="d435_head_motor" link2="hip2_3" reason="Never"/>
+    <disable_collisions link1="d435_head_motor" link2="hip2_4" reason="Never"/>
+    <disable_collisions link1="d435_head_motor" link2="knee_1" reason="Never"/>
+    <disable_collisions link1="d435_head_motor" link2="knee_2" reason="Never"/>
+    <disable_collisions link1="d435_head_motor" link2="knee_3" reason="Never"/>
+    <disable_collisions link1="d435_head_motor" link2="knee_4" reason="Never"/>
+    <disable_collisions link1="d435_head_motor" link2="neck_1" reason="Adjacent"/>
+    <disable_collisions link1="d435_head_motor" link2="pelvis" reason="Never"/>
+    <disable_collisions link1="d435_head_motor" link2="torso_2" reason="Never"/>
+    <disable_collisions link1="d435_head_motor" link2="velodyne_calib_base_link" reason="Never"/>
+    <disable_collisions link1="d435_head_motor" link2="velodyne_motor" reason="Never"/>
+    <disable_collisions link1="d435_head_motor" link2="wheel_1" reason="Never"/>
+    <disable_collisions link1="d435_head_motor" link2="wheel_2" reason="Never"/>
+    <disable_collisions link1="d435_head_motor" link2="wheel_3" reason="Never"/>
+    <disable_collisions link1="d435_head_motor" link2="wheel_4" reason="Never"/>
+    <disable_collisions link1="hip1_1" link2="hip1_2" reason="Never"/>
+    <disable_collisions link1="hip1_1" link2="hip1_3" reason="Never"/>
+    <disable_collisions link1="hip1_1" link2="hip1_4" reason="Never"/>
+    <disable_collisions link1="hip1_1" link2="hip2_1" reason="Adjacent"/>
+    <disable_collisions link1="hip1_1" link2="hip2_3" reason="Never"/>
+    <disable_collisions link1="hip1_1" link2="hip2_4" reason="Never"/>
+    <disable_collisions link1="hip1_1" link2="knee_1" reason="Never"/>
+    <disable_collisions link1="hip1_1" link2="neck_1" reason="Never"/>
+    <disable_collisions link1="hip1_1" link2="pelvis" reason="Adjacent"/>
+    <disable_collisions link1="hip1_1" link2="torso_2" reason="Never"/>
+    <disable_collisions link1="hip1_1" link2="velodyne_calib_base_link" reason="Never"/>
+    <disable_collisions link1="hip1_1" link2="velodyne_motor" reason="Never"/>
+    <disable_collisions link1="hip1_2" link2="hip1_3" reason="Never"/>
+    <disable_collisions link1="hip1_2" link2="hip1_4" reason="Never"/>
+    <disable_collisions link1="hip1_2" link2="hip2_2" reason="Adjacent"/>
+    <disable_collisions link1="hip1_2" link2="hip2_3" reason="Never"/>
+    <disable_collisions link1="hip1_2" link2="hip2_4" reason="Never"/>
+    <disable_collisions link1="hip1_2" link2="knee_2" reason="Never"/>
+    <disable_collisions link1="hip1_2" link2="neck_1" reason="Never"/>
+    <disable_collisions link1="hip1_2" link2="pelvis" reason="Adjacent"/>
+    <disable_collisions link1="hip1_2" link2="torso_2" reason="Never"/>
+    <disable_collisions link1="hip1_2" link2="velodyne_calib_base_link" reason="Never"/>
+    <disable_collisions link1="hip1_2" link2="velodyne_motor" reason="Never"/>
+    <disable_collisions link1="hip1_3" link2="hip1_4" reason="Never"/>
+    <disable_collisions link1="hip1_3" link2="hip2_1" reason="Never"/>
+    <disable_collisions link1="hip1_3" link2="hip2_2" reason="Never"/>
+    <disable_collisions link1="hip1_3" link2="hip2_3" reason="Adjacent"/>
+    <disable_collisions link1="hip1_3" link2="knee_3" reason="Never"/>
+    <disable_collisions link1="hip1_3" link2="neck_1" reason="Never"/>
+    <disable_collisions link1="hip1_3" link2="pelvis" reason="Adjacent"/>
+    <disable_collisions link1="hip1_3" link2="torso_2" reason="Never"/>
+    <disable_collisions link1="hip1_3" link2="velodyne_calib_base_link" reason="Never"/>
+    <disable_collisions link1="hip1_3" link2="velodyne_motor" reason="Never"/>
+    <disable_collisions link1="hip1_4" link2="hip2_1" reason="Never"/>
+    <disable_collisions link1="hip1_4" link2="hip2_2" reason="Never"/>
+    <disable_collisions link1="hip1_4" link2="hip2_4" reason="Adjacent"/>
+    <disable_collisions link1="hip1_4" link2="knee_4" reason="Never"/>
+    <disable_collisions link1="hip1_4" link2="neck_1" reason="Never"/>
+    <disable_collisions link1="hip1_4" link2="pelvis" reason="Adjacent"/>
+    <disable_collisions link1="hip1_4" link2="torso_2" reason="Never"/>
+    <disable_collisions link1="hip1_4" link2="velodyne_calib_base_link" reason="Never"/>
+    <disable_collisions link1="hip1_4" link2="velodyne_motor" reason="Never"/>
+    <disable_collisions link1="hip2_1" link2="knee_1" reason="Adjacent"/>
+    <disable_collisions link1="hip2_1" link2="neck_1" reason="Never"/>
+    <disable_collisions link1="hip2_1" link2="torso_2" reason="Never"/>
+    <disable_collisions link1="hip2_1" link2="velodyne_calib_base_link" reason="Never"/>
+    <disable_collisions link1="hip2_1" link2="velodyne_motor" reason="Never"/>
+    <disable_collisions link1="hip2_2" link2="knee_2" reason="Adjacent"/>
+    <disable_collisions link1="hip2_2" link2="neck_1" reason="Never"/>
+    <disable_collisions link1="hip2_2" link2="torso_2" reason="Never"/>
+    <disable_collisions link1="hip2_2" link2="velodyne_calib_base_link" reason="Never"/>
+    <disable_collisions link1="hip2_2" link2="velodyne_motor" reason="Never"/>
+    <disable_collisions link1="hip2_3" link2="knee_3" reason="Adjacent"/>
+    <disable_collisions link1="hip2_3" link2="neck_1" reason="Never"/>
+    <disable_collisions link1="hip2_3" link2="torso_2" reason="Never"/>
+    <disable_collisions link1="hip2_3" link2="velodyne_calib_base_link" reason="Never"/>
+    <disable_collisions link1="hip2_3" link2="velodyne_motor" reason="Never"/>
+    <disable_collisions link1="hip2_4" link2="knee_4" reason="Adjacent"/>
+    <disable_collisions link1="hip2_4" link2="neck_1" reason="Never"/>
+    <disable_collisions link1="hip2_4" link2="torso_2" reason="Never"/>
+    <disable_collisions link1="hip2_4" link2="velodyne_calib_base_link" reason="Never"/>
+    <disable_collisions link1="hip2_4" link2="velodyne_motor" reason="Never"/>
+    <disable_collisions link1="knee_1" link2="neck_1" reason="Never"/>
+    <disable_collisions link1="knee_1" link2="velodyne_calib_base_link" reason="Never"/>
+    <disable_collisions link1="knee_1" link2="velodyne_motor" reason="Never"/>
+    <disable_collisions link1="knee_1" link2="wheel_1" reason="Never"/>
+    <disable_collisions link1="knee_2" link2="neck_1" reason="Never"/>
+    <disable_collisions link1="knee_2" link2="velodyne_calib_base_link" reason="Never"/>
+    <disable_collisions link1="knee_2" link2="velodyne_motor" reason="Never"/>
+    <disable_collisions link1="knee_2" link2="wheel_2" reason="Never"/>
+    <disable_collisions link1="knee_3" link2="neck_1" reason="Never"/>
+    <disable_collisions link1="knee_3" link2="velodyne_calib_base_link" reason="Never"/>
+    <disable_collisions link1="knee_3" link2="velodyne_motor" reason="Never"/>
+    <disable_collisions link1="knee_3" link2="wheel_3" reason="Never"/>
+    <disable_collisions link1="knee_4" link2="neck_1" reason="Never"/>
+    <disable_collisions link1="knee_4" link2="velodyne_calib_base_link" reason="Never"/>
+    <disable_collisions link1="knee_4" link2="velodyne_motor" reason="Never"/>
+    <disable_collisions link1="knee_4" link2="wheel_4" reason="Never"/>
+    <disable_collisions link1="neck_1" link2="pelvis" reason="Never"/>
+    <disable_collisions link1="neck_1" link2="torso_2" reason="Adjacent"/>
+    <disable_collisions link1="neck_1" link2="velodyne_calib_base_link" reason="Never"/>
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