Commit message: modification for working with reduced model

File: centauro_urdf/urdf/parts/ball.urdf.xacro (robot description, xacro)
@@ -13,5 +13,5 @@
         <mesh filename="package://centauro_urdf/meshes/BallHand.stl" scale="0.001 0.001 0.001" />
       </geometry>
-      <material name="grey"/>
+      <material name="dark_grey"/>
    </visual>
    <collision>

File: centauro_urdf/urdf/utils.urdf.xacro (robot description, xacro)
@@ -8,9 +8,9 @@
 <xacro:property name="toRad" value="${PI/180.0}" />
 <xacro:property name="toDeg" value="${180.0/PI}" />
-<xacro:property name="torque_scale" value="0.7" /> <!-- scaling facto for available peack torque link side, from 0 to 1 -->
+<xacro:property name="torque_scale" value="0.7" /> <!-- scaling factor for available peack torque link side, from 0 to 1 -->
 <material name="black">
     <color rgba="0.4 0.4 0.4 1"/>
 </material>
-<material name="dark">
+<material name="dark_grey">
     <color rgba="0.1 0.1 0.1 1"/>
 </material>

Commit message: few modifications

File: centauro_srdf/srdf/centauro.srdf.xacro (robot description, xacro)
@@ -507,3 +507,7 @@
     <disable_collisions link1="arm1_3" link2="arm1_5" reason="Never"/>
     <disable_collisions link1="arm1_2" link2="arm1_5" reason="Never"/>
+    <disable_collisions link1="arm2_3" link2="arm2_5" reason="Never"/>
+    <disable_collisions link1="arm2_2" link2="arm2_5" reason="Never"/>
+    <disable_collisions link1="arm2_2" link2="torso_2" reason="Never"/>
+    <disable_collisions link1="arm1_2" link2="torso_2" reason="Never"/>
 </robot>

File: centauro_urdf/urdf/config/centauro.urdf.xacro (robot description, xacro)
@@ -15,5 +15,5 @@
 <xacro:property name="ADD_BALL_END_EFFECTOR" value="true" />
 <xacro:property name="ADD_FLOATING_BASE" value="$(arg floating_joint)" />
-<xacro:property name="ADD_VIRTUAL_FRAME" value="false" />
+<xacro:property name="ADD_VIRTUAL_FRAME" value="true" />
 <xacro:property name="USE_STICKS" value="false" />
 <xacro:property name="ADD_VELODYNE" value="$(arg velodyne)" />

Commit message: setup for g2o centauro car model experiments

File: centauro_srdf/srdf/centauro.srdf.xacro (robot description, xacro)
@@ -51,13 +51,13 @@
     </xacro:if>
     <group name="chains">        <!--THIS HAS TO BE THE LAST GROUP IN THE FILE -->
-        <!--xacro:if value="${ADD_LEGS}">
+        <xacro:if value="${ADD_LEGS}">
             <group name="front_left_leg" />
             <group name="front_right_leg" />
             <group name="rear_right_leg" />
             <group name="rear_left_leg" />
-        </xacro:if-->
+        </xacro:if>
         <xacro:if value="${ADD_UPPER_BODY}">
-            <group name="left_arm" />
-            <!--group name="right_arm" />
+            <!--group name="left_arm" />
+            <group name="right_arm" />
             <group name="torso" />
             <group name="velodyne"/>
@@ -511,3 +511,147 @@
     <disable_collisions link1="arm2_2" link2="torso_2" reason="Never"/>
     <disable_collisions link1="arm1_2" link2="torso_2" reason="Never"/>
+    <disable_collisions link1="hip1_1" link2="hip1_4" reason="Never"/>
+    <disable_collisions link1="hip1_1" link2="hip2_4" reason="Never"/>
+    <disable_collisions link1="hip1_1" link2="knee_4" reason="Never"/>
+    <disable_collisions link1="hip1_1" link2="ankle1_4" reason="Never"/>
+    <disable_collisions link1="hip1_1" link2="ankle2_4" reason="Never"/>
+    <disable_collisions link1="hip1_1" link2="wheel_4" reason="Never"/>
+    <disable_collisions link1="hip2_1" link2="hip1_4" reason="Never"/>
+    <disable_collisions link1="hip2_1" link2="hip2_4" reason="Never"/>
+    <disable_collisions link1="hip2_1" link2="knee_4" reason="Never"/>
+    <disable_collisions link1="hip2_1" link2="ankle1_4" reason="Never"/>
+    <disable_collisions link1="hip2_1" link2="ankle2_4" reason="Never"/>
+    <disable_collisions link1="hip2_1" link2="wheel_4" reason="Never"/>
+    <disable_collisions link1="knee_1" link2="hip1_4" reason="Never"/>
+    <disable_collisions link1="knee_1" link2="hip2_4" reason="Never"/>
+    <disable_collisions link1="knee_1" link2="knee_4" reason="Never"/>
+    <disable_collisions link1="knee_1" link2="ankle1_4" reason="Never"/>
+    <disable_collisions link1="knee_1" link2="ankle2_4" reason="Never"/>
+    <disable_collisions link1="knee_1" link2="wheel_4" reason="Never"/>
+    <disable_collisions link1="ankle1_1" link2="hip1_4" reason="Never"/>
+    <disable_collisions link1="ankle1_1" link2="hip2_4" reason="Never"/>
+    <disable_collisions link1="ankle1_1" link2="knee_4" reason="Never"/>
+    <disable_collisions link1="ankle1_1" link2="ankle1_4" reason="Never"/>
+    <disable_collisions link1="ankle1_1" link2="ankle2_4" reason="Never"/>
+    <disable_collisions link1="ankle1_1" link2="wheel_4" reason="Never"/>
+    <disable_collisions link1="ankle2_1" link2="hip1_4" reason="Never"/>
+    <disable_collisions link1="ankle2_1" link2="hip2_4" reason="Never"/>
+    <disable_collisions link1="ankle2_1" link2="knee_4" reason="Never"/>
+    <disable_collisions link1="ankle2_1" link2="ankle1_4" reason="Never"/>
+    <disable_collisions link1="ankle2_1" link2="ankle2_4" reason="Never"/>
+    <disable_collisions link1="ankle2_1" link2="wheel_4" reason="Never"/>
+    <disable_collisions link1="wheel_1" link2="hip1_4" reason="Never"/>
+    <disable_collisions link1="wheel_1" link2="hip2_4" reason="Never"/>
+    <disable_collisions link1="wheel_1" link2="knee_4" reason="Never"/>
+    <disable_collisions link1="wheel_1" link2="ankle1_4" reason="Never"/>
+    <disable_collisions link1="wheel_1" link2="ankle2_4" reason="Never"/>
+    <disable_collisions link1="wheel_1" link2="wheel_4" reason="Never"/>
+    <disable_collisions link1="hip1_1" link2="hip1_3" reason="Never"/>
+    <disable_collisions link1="hip1_1" link2="hip2_3" reason="Never"/>
+    <disable_collisions link1="hip1_1" link2="knee_3" reason="Never"/>
+    <disable_collisions link1="hip1_1" link2="ankle1_3" reason="Never"/>
+    <disable_collisions link1="hip1_1" link2="ankle2_3" reason="Never"/>
+    <disable_collisions link1="hip1_1" link2="wheel_3" reason="Never"/>
+    <disable_collisions link1="hip2_1" link2="hip1_3" reason="Never"/>
+    <disable_collisions link1="hip2_1" link2="hip2_3" reason="Never"/>
+    <disable_collisions link1="hip2_1" link2="knee_3" reason="Never"/>
+    <disable_collisions link1="hip2_1" link2="ankle1_3" reason="Never"/>
+    <disable_collisions link1="hip2_1" link2="ankle2_3" reason="Never"/>
+    <disable_collisions link1="hip2_1" link2="wheel_3" reason="Never"/>
+    <disable_collisions link1="knee_1" link2="hip1_3" reason="Never"/>
+    <disable_collisions link1="knee_1" link2="hip2_3" reason="Never"/>
+    <disable_collisions link1="knee_1" link2="knee_3" reason="Never"/>
+    <disable_collisions link1="knee_1" link2="ankle1_3" reason="Never"/>
+    <disable_collisions link1="knee_1" link2="ankle2_3" reason="Never"/>
+    <disable_collisions link1="knee_1" link2="wheel_3" reason="Never"/>
+    <disable_collisions link1="ankle1_1" link2="hip1_3" reason="Never"/>
+    <disable_collisions link1="ankle1_1" link2="hip2_3" reason="Never"/>
+    <disable_collisions link1="ankle1_1" link2="knee_3" reason="Never"/>
+    <disable_collisions link1="ankle1_1" link2="ankle1_3" reason="Never"/>
+    <disable_collisions link1="ankle1_1" link2="ankle2_3" reason="Never"/>
+    <disable_collisions link1="ankle1_1" link2="wheel_3" reason="Never"/>
+    <disable_collisions link1="ankle2_1" link2="hip1_3" reason="Never"/>
+    <disable_collisions link1="ankle2_1" link2="hip2_3" reason="Never"/>
+    <disable_collisions link1="ankle2_1" link2="knee_3" reason="Never"/>
+    <disable_collisions link1="ankle2_1" link2="ankle1_3" reason="Never"/>
+    <disable_collisions link1="ankle2_1" link2="ankle2_3" reason="Never"/>
+    <disable_collisions link1="ankle2_1" link2="wheel_3" reason="Never"/>
+    <disable_collisions link1="wheel_1" link2="hip1_3" reason="Never"/>
+    <disable_collisions link1="wheel_1" link2="hip2_3" reason="Never"/>
+    <disable_collisions link1="wheel_1" link2="knee_3" reason="Never"/>
+    <disable_collisions link1="wheel_1" link2="ankle1_3" reason="Never"/>
+    <disable_collisions link1="wheel_1" link2="ankle2_3" reason="Never"/>
+    <disable_collisions link1="wheel_1" link2="wheel_3" reason="Never"/>
+    <disable_collisions link1="hip1_2" link2="hip1_4" reason="Never"/>
+    <disable_collisions link1="hip1_2" link2="hip2_4" reason="Never"/>
+    <disable_collisions link1="hip1_2" link2="knee_4" reason="Never"/>
+    <disable_collisions link1="hip1_2" link2="ankle1_4" reason="Never"/>
+    <disable_collisions link1="hip1_2" link2="ankle2_4" reason="Never"/>
+    <disable_collisions link1="hip1_2" link2="wheel_4" reason="Never"/>
+    <disable_collisions link1="hip2_2" link2="hip1_4" reason="Never"/>
+    <disable_collisions link1="hip2_2" link2="hip2_4" reason="Never"/>
+    <disable_collisions link1="hip2_2" link2="knee_4" reason="Never"/>
+    <disable_collisions link1="hip2_2" link2="ankle1_4" reason="Never"/>
+    <disable_collisions link1="hip2_2" link2="ankle2_4" reason="Never"/>
+    <disable_collisions link1="hip2_2" link2="wheel_4" reason="Never"/>
+    <disable_collisions link1="knee_2" link2="hip1_4" reason="Never"/>
+    <disable_collisions link1="knee_2" link2="hip2_4" reason="Never"/>
+    <disable_collisions link1="knee_2" link2="knee_4" reason="Never"/>
+    <disable_collisions link1="knee_2" link2="ankle1_4" reason="Never"/>
+    <disable_collisions link1="knee_2" link2="ankle2_4" reason="Never"/>
+    <disable_collisions link1="knee_2" link2="wheel_4" reason="Never"/>
+    <disable_collisions link1="ankle1_2" link2="hip1_4" reason="Never"/>
+    <disable_collisions link1="ankle1_2" link2="hip2_4" reason="Never"/>
+    <disable_collisions link1="ankle1_2" link2="knee_4" reason="Never"/>
+    <disable_collisions link1="ankle1_2" link2="ankle1_4" reason="Never"/>
+    <disable_collisions link1="ankle1_2" link2="ankle2_4" reason="Never"/>
+    <disable_collisions link1="ankle1_2" link2="wheel_4" reason="Never"/>
+    <disable_collisions link1="ankle2_2" link2="hip1_4" reason="Never"/>
+    <disable_collisions link1="ankle2_2" link2="hip2_4" reason="Never"/>
+    <disable_collisions link1="ankle2_2" link2="knee_4" reason="Never"/>
+    <disable_collisions link1="ankle2_2" link2="ankle1_4" reason="Never"/>
+    <disable_collisions link1="ankle2_2" link2="ankle2_4" reason="Never"/>
+    <disable_collisions link1="ankle2_2" link2="wheel_4" reason="Never"/>
+    <disable_collisions link1="wheel_2" link2="hip1_4" reason="Never"/>
+    <disable_collisions link1="wheel_2" link2="hip2_4" reason="Never"/>
+    <disable_collisions link1="wheel_2" link2="knee_4" reason="Never"/>
+    <disable_collisions link1="wheel_2" link2="ankle1_4" reason="Never"/>
+    <disable_collisions link1="wheel_2" link2="ankle2_4" reason="Never"/>
+    <disable_collisions link1="wheel_2" link2="wheel_4" reason="Never"/>
+    <disable_collisions link1="hip1_2" link2="hip1_4" reason="Never"/>
+    <disable_collisions link1="hip1_2" link2="hip2_4" reason="Never"/>
+    <disable_collisions link1="hip1_2" link2="knee_4" reason="Never"/>
+    <disable_collisions link1="hip1_2" link2="ankle1_4" reason="Never"/>
+    <disable_collisions link1="hip1_2" link2="ankle2_4" reason="Never"/>
+    <disable_collisions link1="hip1_2" link2="wheel_4" reason="Never"/>
+    <disable_collisions link1="hip2_2" link2="hip1_4" reason="Never"/>
+    <disable_collisions link1="hip2_2" link2="hip2_4" reason="Never"/>
+    <disable_collisions link1="hip2_2" link2="knee_4" reason="Never"/>
+    <disable_collisions link1="hip2_2" link2="ankle1_4" reason="Never"/>
+    <disable_collisions link1="hip2_2" link2="ankle2_4" reason="Never"/>
+    <disable_collisions link1="hip2_2" link2="wheel_4" reason="Never"/>
+    <disable_collisions link1="knee_2" link2="hip1_4" reason="Never"/>
+    <disable_collisions link1="knee_2" link2="hip2_4" reason="Never"/>
+    <disable_collisions link1="knee_2" link2="knee_4" reason="Never"/>
+    <disable_collisions link1="knee_2" link2="ankle1_4" reason="Never"/>
+    <disable_collisions link1="knee_2" link2="ankle2_4" reason="Never"/>
+    <disable_collisions link1="knee_2" link2="wheel_4" reason="Never"/>
+    <disable_collisions link1="ankle1_2" link2="hip1_4" reason="Never"/>
+    <disable_collisions link1="ankle1_2" link2="hip2_4" reason="Never"/>
+    <disable_collisions link1="ankle1_2" link2="knee_4" reason="Never"/>
+    <disable_collisions link1="ankle1_2" link2="ankle1_4" reason="Never"/>
+    <disable_collisions link1="ankle1_2" link2="ankle2_4" reason="Never"/>
+    <disable_collisions link1="ankle1_2" link2="wheel_4" reason="Never"/>
+    <disable_collisions link1="ankle2_2" link2="hip1_4" reason="Never"/>
+    <disable_collisions link1="ankle2_2" link2="hip2_4" reason="Never"/>
+    <disable_collisions link1="ankle2_2" link2="knee_4" reason="Never"/>
+    <disable_collisions link1="ankle2_2" link2="ankle1_4" reason="Never"/>
+    <disable_collisions link1="ankle2_2" link2="ankle2_4" reason="Never"/>
+    <disable_collisions link1="ankle2_2" link2="wheel_4" reason="Never"/>
+    <disable_collisions link1="wheel_2" link2="hip1_4" reason="Never"/>
+    <disable_collisions link1="wheel_2" link2="hip2_4" reason="Never"/>
+    <disable_collisions link1="wheel_2" link2="knee_4" reason="Never"/>
+    <disable_collisions link1="wheel_2" link2="ankle1_4" reason="Never"/>
+    <disable_collisions link1="wheel_2" link2="ankle2_4" reason="Never"/>
+    <disable_collisions link1="wheel_2" link2="wheel_4" reason="Never"/>
 </robot>

File: centauro_urdf/urdf/config/centauro.urdf.xacro (robot description, xacro)
@@ -15,5 +15,5 @@
 <xacro:property name="ADD_BALL_END_EFFECTOR" value="true" />
 <xacro:property name="ADD_FLOATING_BASE" value="$(arg floating_joint)" />
-<xacro:property name="ADD_VIRTUAL_FRAME" value="true" />
+<xacro:property name="ADD_VIRTUAL_FRAME" value="false" />
 <xacro:property name="USE_STICKS" value="false" />
 <xacro:property name="ADD_VELODYNE" value="$(arg velodyne)" />
