Commit message: updated arms to reflect new hardware

File: centauro_srdf/srdf/centauro.srdf.xacro (robot description, xacro)
@@ -30,8 +30,8 @@
     <xacro:if value="${ADD_UPPER_BODY}">
         <group name="left_arm">
-            <chain base_link="torso_2" tip_link="arm1_7" />
+            <chain base_link="torso_2" tip_link="arm1_8" />
         </group>
         <group name="right_arm">
-            <chain base_link="torso_2" tip_link="arm2_7" />
+            <chain base_link="torso_2" tip_link="arm2_8" />
         </group>
         <group name="torso">
@@ -99,5 +99,4 @@
         <joint name="j_arm1_5" value="0.0500815"/>
         <joint name="j_arm1_6" value="-0.781461"/>
-        <joint name="j_arm1_7" value="-0.0567608"/>
         <joint name="j_arm2_1" value="0.520149"/>
         <joint name="j_arm2_2" value="-0.320865"/>
@@ -106,5 +105,4 @@
         <joint name="j_arm2_5" value="-0.0500815"/>
         <joint name="j_arm2_6" value="-0.781461"/>
-        <joint name="j_arm2_7" value="0.0567608"/>
     </group_state>
 </robot>

File: centauro_urdf/urdf/centauro.urdf (robot description, URDF)
Before this commit: robot centauro, 98 links, 97 joints
Links:
- removed link arm1_7
- removed link arm2_7
- removed link ft_arm1
- removed link ft_arm2
- link arm1_6: geometry collision mesh filename=package://centauro_urdf/meshes/simple/wrist_pitch_right.stl scale=0.001 -0.001 0.001; visual mesh filename=package://centauro_urdf/meshes/wrist_pitch_right.stl scale=0.001 -0.001 0.001
- link arm2_6: geometry collision mesh filename=package://centauro_urdf/meshes/simple/wrist_pitch_right.stl scale=0.001 0.001 0.001; visual mesh filename=package://centauro_urdf/meshes/wrist_pitch_right.stl scale=0.001 0.001 0.001
Joints:
- removed joint j_arm1_7
- removed joint j_arm2_7
- removed joint j_ft_1
- removed joint j_ft_2
- joint j_arm1_8: origin xyz=0. 0. 0. rpy=0. 0. 0. -> xyz=0. -0.05 -0.105 rpy=0. 0. 0.; parent arm1_7 -> arm1_6
- joint j_arm2_8: origin xyz=0. 0. 0. rpy=0. 0. 0. -> xyz=0. 0.05 -0.105 rpy=0. 0. 0.; parent arm2_7 -> arm2_6

File: centauro_urdf/urdf/centauro_capsule.urdf (robot description, URDF)
Before this commit: robot centauro, 98 links, 97 joints
Links:
- removed link arm1_7
- removed link arm2_7
- removed link ft_arm1
- removed link ft_arm2
- link T265_camera_pose_frame: geometry collision cylinder length=0.1022528557886848 radius=0.0142751; collision sphere radius=0.0142751
- link ankle1_1: geometry collision cylinder length=0.049256315666076876 radius=0.0792379; collision sphere radius=0.0792379
- link ankle1_2: geometry collision cylinder length=0.04788405128558378 radius=0.0781037; collision sphere radius=0.0781037
- link ankle1_3: geometry collision cylinder length=0.049256315666076876 radius=0.0792379; collision sphere radius=0.0792379
- link ankle1_4: geometry collision cylinder length=0.04788405128558378 radius=0.0781037; collision sphere radius=0.0781037
- link ankle2_1: geometry collision cylinder length=0.07370263129636398 radius=0.0813545; collision sphere radius=0.0813545
- link ankle2_2: geometry collision cylinder length=0.07370263129636398 radius=0.0813545; collision sphere radius=0.0813545
- link ankle2_3: geometry collision cylinder length=0.07370263129636398 radius=0.0813545; collision sphere radius=0.0813545
- link ankle2_4: geometry collision cylinder length=0.07370263129636398 radius=0.0813545; collision sphere radius=0.0813545
- link arm1_1: geometry collision cylinder length=0.03739768494560427 radius=0.0698859; collision sphere radius=0.0698859
- link arm1_2: geometry collision cylinder length=0.12799269981445732 radius=0.0700645; collision sphere radius=0.0700645
- link arm1_3: geometry collision cylinder length=0.06082252644344949 radius=0.0896121; collision sphere radius=0.0896121
- link arm1_4: geometry collision cylinder length=0.08713418572944408 radius=0.0600429; collision sphere radius=0.0600429
- link arm1_5: geometry collision cylinder length=0.08434739747702645 radius=0.0804108; collision sphere radius=0.0804108
- link arm1_6: geometry collision cylinder length=0.07750977987441161 radius=0.0474698; collision sphere radius=0.0474698
- link arm2_1: geometry collision cylinder length=0.03739768494560427 radius=0.0698859; collision sphere radius=0.0698859
- link arm2_2: geometry collision cylinder length=0.12799269981445732 radius=0.0700645; collision sphere radius=0.0700645
- link arm2_3: geometry collision cylinder length=0.06082252644344949 radius=0.0896121; collision sphere radius=0.0896121
- link arm2_4: geometry collision cylinder length=0.08713418572944408 radius=0.0600429; collision sphere radius=0.0600429
- link arm2_5: geometry collision cylinder length=0.08434739747702645 radius=0.0804108; collision sphere radius=0.0804108
- link arm2_6: geometry collision cylinder length=0.07750977987441161 radius=0.0474698; collision sphere radius=0.0474698
- link ball1: geometry collision cylinder length=9.940076835940455e-05 radius=0.0709883; collision sphere radius=0.0709883
- link ball2: geometry collision cylinder length=9.940076835940455e-05 radius=0.0709883; collision sphere radius=0.0709883
- link d435_head_motor: geometry collision cylinder length=0.12134423548428976 radius=0.0261699; collision sphere radius=0.0261699
- link hip1_1: geometry collision cylinder length=0.03069545889898954 radius=0.0747223; collision sphere radius=0.0747223
- link hip1_2: geometry collision cylinder length=0.03069545889898954 radius=0.0747223; collision sphere radius=0.0747223
- link hip1_3: geometry collision cylinder length=0.03069545889898954 radius=0.0747223; collision sphere radius=0.0747223
- link hip1_4: geometry collision cylinder length=0.03069545889898954 radius=0.0747223; collision sphere radius=0.0747223
- link hip2_1: geometry collision cylinder length=0.2919804521727749 radius=0.0808941; collision sphere radius=0.0808941
- link hip2_2: geometry collision cylinder length=0.2919804521727749 radius=0.0808941; collision sphere radius=0.0808941
- link hip2_3: geometry collision cylinder length=0.2919804521727749 radius=0.0808941; collision sphere radius=0.0808941
- link hip2_4: geometry collision cylinder length=0.2919804521727749 radius=0.0808941; collision sphere radius=0.0808941
- link knee_1: geometry collision cylinder length=0.1927502246061244 radius=0.0664305; collision sphere radius=0.0664305
- link knee_2: geometry collision cylinder length=0.1927502246061244 radius=0.0664305; collision sphere radius=0.0664305
- link knee_3: geometry collision cylinder length=0.1927502246061244 radius=0.0664305; collision sphere radius=0.0664305
- link knee_4: geometry collision cylinder length=0.1927502246061244 radius=0.0664305; collision sphere radius=0.0664305
- link neck_1: geometry collision cylinder length=0.16454098025546557 radius=0.100414; collision sphere radius=0.100414
- link pelvis: geometry collision cylinder length=0.38594139791384763 radius=0.213204; collision sphere radius=0.213204
- link torso_2: geometry collision cylinder length=0.09543675990850982 radius=0.158224; collision sphere radius=0.158224
- link velodyne_motor: geometry collision cylinder length=0.032463112134515464 radius=0.0544637; collision sphere radius=0.0544637
Joints:
- removed joint j_arm1_7
- removed joint j_arm2_7
- removed joint j_ft_1
- removed joint j_ft_2
- joint D435_head_camera_accel_optical_joint: origin xyz=0.0 0.0 0.0 rpy=-1.57079632679 0.0 -1.57079632679 -> xyz=0.0 0.0 0.0 rpy=-1.5707963267948966 0.0 -1.5707963267948966
- joint D435_head_camera_color_optical_joint: origin xyz=0.0 0.0 0.0 rpy=-1.57079632679 0.0 -1.57079632679 -> xyz=0.0 0.0 0.0 rpy=-1.5707963267948966 0.0 -1.5707963267948966
- joint D435_head_camera_depth_optical_joint: origin xyz=0.0 0.0 0.0 rpy=-1.57079632679 0.0 -1.57079632679 -> xyz=0.0 0.0 0.0 rpy=-1.5707963267948966 0.0 -1.5707963267948966
- joint D435_head_camera_gyro_optical_joint: origin xyz=0.0 0.0 0.0 rpy=-1.57079632679 0.0 -1.57079632679 -> xyz=0.0 0.0 0.0 rpy=-1.5707963267948966 0.0 -1.5707963267948966
- joint D435_head_camera_left_ir_optical_joint: origin xyz=0.0 0.0 0.0 rpy=-1.57079632679 0.0 -1.57079632679 -> xyz=0.0 0.0 0.0 rpy=-1.5707963267948966 0.0 -1.5707963267948966
- joint D435_head_camera_right_ir_optical_joint: origin xyz=0.0 0.0 0.0 rpy=-1.57079632679 0.0 -1.57079632679 -> xyz=0.0 0.0 0.0 rpy=-1.5707963267948966 0.0 -1.5707963267948966
- joint D435i_camera_accel_optical_joint: origin xyz=0.0 0.0 0.0 rpy=-1.57079632679 0.0 -1.57079632679 -> xyz=0.0 0.0 0.0 rpy=-1.5707963267948966 0.0 -1.5707963267948966
- joint D435i_camera_color_optical_joint: origin xyz=0.0 0.0 0.0 rpy=-1.57079632679 0.0 -1.57079632679 -> xyz=0.0 0.0 0.0 rpy=-1.5707963267948966 0.0 -1.5707963267948966
- joint D435i_camera_depth_optical_joint: origin xyz=0.0 0.0 0.0 rpy=-1.57079632679 0.0 -1.57079632679 -> xyz=0.0 0.0 0.0 rpy=-1.5707963267948966 0.0 -1.5707963267948966
- joint D435i_camera_gyro_optical_joint: origin xyz=0.0 0.0 0.0 rpy=-1.57079632679 0.0 -1.57079632679 -> xyz=0.0 0.0 0.0 rpy=-1.5707963267948966 0.0 -1.5707963267948966
- joint D435i_camera_left_ir_optical_joint: origin xyz=0.0 0.0 0.0 rpy=-1.57079632679 0.0 -1.57079632679 -> xyz=0.0 0.0 0.0 rpy=-1.5707963267948966 0.0 -1.5707963267948966
- joint D435i_camera_right_ir_optical_joint: origin xyz=0.0 0.0 0.0 rpy=-1.57079632679 0.0 -1.57079632679 -> xyz=0.0 0.0 0.0 rpy=-1.5707963267948966 0.0 -1.5707963267948966
- joint T265_camera_accel_joint: origin xyz=-0.0311 0.0 0.00655 rpy=0.0 3.14159265359 0.0 -> xyz=-0.0311 0.0 0.00655 rpy=0.0 3.141592653589793 0.0
- joint T265_camera_accel_optical_joint: origin xyz=-0.0311 0.0 0.00655 rpy=0.0 3.14159265359 0.0 -> xyz=-0.0311 0.0 0.00655 rpy=0.0 3.141592653589793 0.0
- joint T265_camera_fisheye1_optical_joint: origin xyz=0.0 0.0 0.0 rpy=-1.57079632679 0.0 -1.57079632679 -> xyz=0.0 0.0 0.0 rpy=-1.5707963267948966 0.0 -1.5707963267948966
- joint T265_camera_fisheye1_rgb_joint: origin xyz=-0.0411 0.0 0.0 rpy=0.0 1.57079632679 1.57079632679 -> xyz=-0.0411 0.0 0.0 rpy=0.0 1.5707963267948966 1.5707963267948966
- joint T265_camera_fisheye2_optical_joint: origin xyz=0.0 0.0 0.0 rpy=-1.57079632679 0.0 -1.57079632679 -> xyz=0.0 0.0 0.0 rpy=-1.5707963267948966 0.0 -1.5707963267948966
- joint T265_camera_fisheye2_rgb_joint: origin xyz=0.0229 0.0 0.0 rpy=0.0 1.57079632679 1.57079632679 -> xyz=0.0229 0.0 0.0 rpy=0.0 1.5707963267948966 1.5707963267948966
- joint T265_camera_gyro_joint: origin xyz=-0.0311 0.0 0.00655 rpy=0.0 3.14159265359 0.0 -> xyz=-0.0311 0.0 0.00655 rpy=0.0 3.141592653589793 0.0
- joint T265_camera_link_joint: origin xyz=0.0 0.0 0.0 rpy=1.57079632679 0.0 -1.57079632679 -> xyz=0.0 0.0 0.0 rpy=1.5707963267948966 0.0 -1.5707963267948966
- joint hip_yaw_1: origin xyz=0.25 0.125 -0.0566 rpy=0.0 0.0 0.0 -> xyz=0.25 0.125 -0.056600000000000004 rpy=0.0 0.0 0.0
- joint hip_yaw_2: origin xyz=0.25 -0.125 -0.0566 rpy=0.0 0.0 0.0 -> xyz=0.25 -0.125 -0.056600000000000004 rpy=0.0 0.0 0.0
- joint hip_yaw_3: origin xyz=-0.25 0.125 -0.0566 rpy=0.0 0.0 0.0 -> xyz=-0.25 0.125 -0.056600000000000004 rpy=0.0 0.0 0.0
- joint hip_yaw_4: origin xyz=-0.25 -0.125 -0.0566 rpy=0.0 0.0 0.0 -> xyz=-0.25 -0.125 -0.056600000000000004 rpy=0.0 0.0 0.0
- joint j_arm1_8: origin xyz=0.0 0.0 0.0 rpy=0.0 0.0 0.0 -> xyz=0.0 -0.05 -0.105 rpy=0.0 0.0 0.0; parent arm1_7 -> arm1_6
- joint j_arm2_8: origin xyz=0.0 0.0 0.0 rpy=0.0 0.0 0.0 -> xyz=0.0 0.05 -0.105 rpy=0.0 0.0 0.0; parent arm2_7 -> arm2_6
- joint j_wheel_1: origin xyz=0.0 -0.0 -0.09835 rpy=1.57079632679 0.0 0.0 -> xyz=0.0 -0.0 -0.09834999999999999 rpy=1.57079632679 0.0 0.0
- joint j_wheel_2: origin xyz=0.0 0.0 -0.09835 rpy=1.57079632679 0.0 0.0 -> xyz=0.0 0.0 -0.09834999999999999 rpy=1.57079632679 0.0 0.0
- joint j_wheel_3: origin xyz=0.0 -0.0 -0.09835 rpy=1.57079632679 0.0 0.0 -> xyz=0.0 -0.0 -0.09834999999999999 rpy=1.57079632679 0.0 0.0
- joint j_wheel_4: origin xyz=0.0 0.0 -0.09835 rpy=1.57079632679 0.0 0.0 -> xyz=0.0 0.0 -0.09834999999999999 rpy=1.57079632679 0.0 0.0

File: centauro_urdf/urdf/centauro_virtual_frame.urdf (robot description, URDF)
Before this commit: robot centauro, 64 links, 63 joints
Links:
- removed link arm1_7
- removed link arm2_7
- removed link ft_arm1
- removed link ft_arm2
- added link D435_head_camera_bottom_screw_frame
- added link D435_head_camera_link, mass 0.564; collision box size=0.02505 0.09 0.025; visual mesh filename=package://centauro_urdf/meshes/realsense/d435.dae
- added link D435i_camera_bottom_screw_frame
- added link D435i_camera_link, mass 0.564; collision box size=0.02505 0.09 0.025; visual mesh filename=package://centauro_urdf/meshes/realsense/d435.dae
- link arm1_6: geometry collision mesh filename=package://centauro_urdf/meshes/simple/wrist_pitch_right.stl scale=0.001 -0.001 0.001; visual mesh filename=package://centauro_urdf/meshes/wrist_pitch_right.stl scale=0.001 -0.001 0.001
- link arm2_6: geometry collision mesh filename=package://centauro_urdf/meshes/simple/wrist_pitch_right.stl scale=0.001 0.001 0.001; visual mesh filename=package://centauro_urdf/meshes/wrist_pitch_right.stl scale=0.001 0.001 0.001
Joints:
- removed joint j_arm1_7
- removed joint j_arm2_7
- removed joint j_ft_1
- removed joint j_ft_2
- added joint D435_head_camera_joint: type fixed, parent d435_head_motor, child D435_head_camera_bottom_screw_frame, origin xyz=0.03015 0 -0.0125 rpy=0 0 0
- added joint D435_head_camera_link_joint: type fixed, parent D435_head_camera_bottom_screw_frame, child D435_head_camera_link, origin xyz=0 0.0175 0.0125 rpy=0 0 0
- added joint D435i_camera_joint: type fixed, parent pelvis, child D435i_camera_bottom_screw_frame, origin xyz=0.27187 0 0.0215997 rpy=0 0.5251508 0
- added joint D435i_camera_link_joint: type fixed, parent D435i_camera_bottom_screw_frame, child D435i_camera_link, origin xyz=0 0.0175 0.0125 rpy=0 0 0
- joint j_arm1_8: origin xyz=0. 0. 0. rpy=0. 0. 0. -> xyz=0. -0.05 -0.105 rpy=0. 0. 0.; parent arm1_7 -> arm1_6
- joint j_arm2_8: origin xyz=0. 0. 0. rpy=0. 0. 0. -> xyz=0. 0.05 -0.105 rpy=0. 0. 0.; parent arm2_7 -> arm2_6

File: centauro_urdf/urdf/parts/arms.urdf.xacro (robot description, xacro)
@@ -11,9 +11,9 @@
 <xacro:if value="${ADD_BALL_END_EFFECTOR}">
       <xacro:include filename="$(find centauro_urdf)/urdf/parts/ball.urdf.xacro" />
-      <xacro:ball_end_effector arm_num="1"  parent_link="arm1_7">
-                  <origin xyz="0. 0. 0." rpy="0. 0. 0."/>
+      <xacro:ball_end_effector arm_num="1"  parent_link="arm1_6">
+                  <origin xyz="0. -0.05 -0.105" rpy="0. 0. 0."/>
       </xacro:ball_end_effector>
-      <xacro:ball_end_effector arm_num="2"  parent_link="arm2_7">
-                  <origin xyz="0. 0. 0." rpy="0. 0. 0."/>
+      <xacro:ball_end_effector arm_num="2"  parent_link="arm2_6">
+                  <origin xyz="0. 0.05 -0.105" rpy="0. 0. 0."/>
       </xacro:ball_end_effector>
 </xacro:if>

File: centauro_urdf/urdf/parts/centauro_arm.urdf.xacro (robot description, xacro)
@@ -122,16 +122,16 @@
          <origin xyz="0.0 0.0 0.0"  rpy="0.0 0.0 0.0"/>
    <geometry>
-      <mesh filename="package://centauro_urdf/meshes/ForearmPitch.STL" scale="0.001 ${-rot*0.001} 0.001" />
-   </geometry>
-      </visual>
-      <collision>
-         <origin xyz="0.0 0.0 0.0"  rpy="0.0 0.0 0.0"/>
-   <geometry>
-      <mesh filename="package://centauro_urdf/meshes/simple/ForearmPitch.STL" scale="0.001 ${-rot*0.001} 0.001" />
+      <mesh filename="package://centauro_urdf/meshes/wrist_pitch_right.stl" scale="0.001 ${-rot*0.001} 0.001" />
+   </geometry>
+      </visual>
+      <collision>
+         <origin xyz="0.0 0.0 0.0"  rpy="0.0 0.0 0.0"/>
+   <geometry>
+      <mesh filename="package://centauro_urdf/meshes/simple/wrist_pitch_right.stl" scale="0.001 ${-rot*0.001} 0.001" />
    </geometry>
       </collision>
    </link>
 <!-- /wrist yaw-pitch -->
-   <link name="arm${arm_num}_7">
+   <!-- <link name="arm${arm_num}_7">
       <inertial>
          <origin xyz="${Wrist_3_x} ${rot*Wrist_3_y} ${Wrist_3_z}"/>
@@ -152,5 +152,5 @@
    </geometry>
       </collision>
-   </link>
+   </link> -->
 <!-- /LINKS -->
 <!-- JOINTS -->
@@ -210,5 +210,5 @@
 <!-- /wrist yaw-->
 <!-- wrist pitch-->
-   <joint name="j_arm${arm_num}_7" type="revolute">
+   <!-- <joint name="j_arm${arm_num}_7" type="fixed">
       <parent link="arm${arm_num}_6"/>
       <child link="arm${arm_num}_7"/>
@@ -216,10 +216,10 @@
       <axis xyz="0 0 1"/>
       <limit lower="${j_arm_7_lower[arm_num-1]}" upper="${j_arm_7_upper[arm_num-1]}" effort="${j_arm_7_torque[arm_num-1]}" velocity="${j_arm_7_velocity[arm_num-1]}"/>
-   </joint>
+   </joint> -->
 <!-- wrist pitch-->
 <!-- force-troque sensor -->
 <!-- end-effector -->
 <!-- wrist pitch-->
-   <joint name="j_ft_${arm_num}" type="fixed">
+   <!-- <joint name="j_ft_${arm_num}" type="fixed">
       <parent link="arm${arm_num}_7"/>
       <child link="ft_arm${arm_num}"/>
@@ -227,12 +227,12 @@
       <axis xyz="0 0 1"/>
       <limit lower="0.0" upper="0.0" effort="0" velocity="0"/>
-   </joint>
-<!-- wrist pitch-->
-   <link name="ft_arm${arm_num}">
+   </joint> -->
+<!-- wrist pitch-->
+   <!-- <link name="ft_arm${arm_num}">
       <inertial>
          <origin xyz="${Ft_arm_x} ${rot*Ft_arm_y} ${Ft_arm_z}"/>
          <mass value="${Ft_arm_mass}"/>
          <inertia ixx="${Ft_arm_xx}" ixy="${rot*Ft_arm_xy}" ixz="${Ft_arm_xz}" iyy="${Ft_arm_yy}" iyz="${rot*Ft_arm_yz}" izz="${Ft_arm_zz}"/>
-      </inertial>
+      </inertial> -->
       <!--visual>
          <origin xyz="0.0 0.0 0.0"  rpy="${PI} 0.0 0.0"/>
@@ -247,5 +247,5 @@
    </geometry>
       </collision-->
-   </link>
+   <!-- </link> -->
 </xacro:macro>
 <!-- /macro arms -->

Commit message: add F/T sensors at j_arm1_6, 100

File: centauro_srdf/srdf/centauro.srdf.xacro (robot description, xacro)
@@ -27,4 +27,10 @@
             <chain base_link="pelvis" tip_link="wheel_3" />
         </group>
+        <group name="force_torque_sensors">
+		<xacro:if value="${FORCE_TORQUE_SENSORS}">
+		    <joint name="l_arm_ft_joint"/>
+		    <joint name="r_arm_ft_joint"/>
+		</xacro:if>
+	</group>
     </xacro:if>
     <xacro:if value="${ADD_UPPER_BODY}">

File: centauro_urdf/urdf/centauro_robot.urdf.xacro (robot description, xacro)
@@ -8,4 +8,9 @@
   <xacro:include filename="$(find centauro_urdf)/urdf/centauro.urdf.xacro" />
   <xacro:include filename="$(find centauro_urdf)/urdf/gazebo/centauro.gazebo.xacro" />
+  <!-- ************ frames for force torque sensors ************ -->
+  <xacro:if value="${FORCE_TORQUE_SENSORS}">
+  <xacro:include filename="$(find centauro_urdf)/urdf/parts/arms_reference_frames.urdf.xacro"/>
+  <xacro:include filename="$(find centauro_urdf)/urdf/gazebo/force_torque.gazebo.xacro" />
+  </xacro:if>
   <xacro:include filename="$(find centauro_urdf)/urdf/gazebo/xbot.gazebo.xacro" />
   <xacro:include filename="$(find centauro_urdf)/urdf/gazebo/materials.gazebo.xacro" />

File: centauro_urdf/urdf/config/centauro.urdf.xacro (robot description, xacro)
@@ -8,4 +8,5 @@
 <xacro:arg name="velodyne" default="true"/>
 <xacro:arg name="realsense" default="true"/>
+<xacro:arg name="ft_sensors" default="true"/>
 <xacro:if value="$(arg realsense)">
 	<xacro:arg name="d435i_head" default="true"/>
@@ -21,4 +22,5 @@
 <!-- ************SELECT PARTS*************-->
 <!-- *************************************-->
+<xacro:property name="FORCE_TORQUE_SENSORS" value="$(arg ft_sensors)" />
 <xacro:property name="ADD_LEGS" value="$(arg legs)" />
 <xacro:property name="ADD_UPPER_BODY" value="$(arg upper_body)" />

Commit message: homing for dagana, if present

File: centauro_srdf/srdf/centauro.srdf.xacro (robot description, xacro)
@@ -105,4 +105,10 @@
         <joint name="j_arm2_5" value="-0.0500815"/>
         <joint name="j_arm2_6" value="-0.781461"/>
+        <xacro:if value="${END_EFFECTOR_LEFT == 'dagana'}">
+            <joint name="dagana_1_claw_joint" value="0"/>
+        </xacro:if>
+        <xacro:if value="${END_EFFECTOR_RIGHT == 'dagana'}">
+            <joint name="dagana_2_claw_joint" value="0"/>
+        </xacro:if>
     </group_state>
 </robot>

Commit message: added wheels to srdf

File: centauro_srdf/srdf/centauro.srdf.xacro (robot description, xacro)
@@ -107,4 +107,8 @@
         <joint name="j_arm2_5" value="-0.0500815"/>
         <joint name="j_arm2_6" value="-0.781461"/>
+        <joint name="wheel_1" value="0.0"/>
+        <joint name="wheel_2" value="0.0"/>
+        <joint name="wheel_3" value="0.0"/>
+        <joint name="wheel_4" value="0.0"/>
         <xacro:if value="${END_EFFECTOR_LEFT == 'dagana'}">
             <joint name="dagana_1_claw_joint" value="0"/>

Commit message: Signed-off-by: Andrea Patrizi <andreapatrizi1b6e6@gmail.com>

File: centauro_srdf/srdf/centauro.srdf.xacro (robot description, xacro)
@@ -107,8 +107,8 @@
         <joint name="j_arm2_5" value="-0.0500815"/>
         <joint name="j_arm2_6" value="-0.781461"/>
-        <joint name="wheel_1" value="0.0"/>
-        <joint name="wheel_2" value="0.0"/>
-        <joint name="wheel_3" value="0.0"/>
-        <joint name="wheel_4" value="0.0"/>
+        <joint name="j_wheel_1" value="0.0"/>
+        <joint name="j_wheel_2" value="0.0"/>
+        <joint name="j_wheel_3" value="0.0"/>
+        <joint name="j_wheel_4" value="0.0"/>
         <xacro:if value="${END_EFFECTOR_LEFT == 'dagana'}">
             <joint name="dagana_1_claw_joint" value="0"/>
