Commit message: renamed root arg

File: centauro_srdf/srdf/centauro.srdf.xacro (robot description, xacro)
@@ -6,7 +6,7 @@
 <robot xmlns:xacro="http://ros.org/wiki/xacro" name="centauro">
     <xacro:arg name="centauro_root" default="$(find centauro_urdf)" />
-    <xacro:property name="CENTAURO_ROOT" value="$(arg centauro_root)" />
+    <xacro:property name="ROOT" value="$(arg centauro_root)" />
     <!-- ************ MODEL CONFIGURATION ************ -->
-    <xacro:arg name="config" default="${CENTAURO_ROOT}/urdf/config/centauro.urdf.xacro"/>
+    <xacro:arg name="config" default="${ROOT}/urdf/config/centauro.urdf.xacro"/>
     <xacro:include filename="$(arg config)"/>
     <group name="base">

File: centauro_urdf/urdf/centauro.urdf.xacro (robot description, xacro)
@@ -4,5 +4,5 @@
 will be propagated to all its downstream childs -->
 <xacro:arg name="centauro_root" default="$(find centauro_urdf)" />
-<xacro:property name="CENTAURO_ROOT" value="$(arg centauro_root)" />
+<xacro:property name="ROOT" value="$(arg centauro_root)" />
 <!-- setting use_abs_mesh_paths should be kept to false
 for use with tools like RViz, which does not accept plain
@@ -14,8 +14,8 @@
 <xacro:if value="${USE_ABS_MESH_PATHS}">
     <xacro:if value="${USE_LOCAL_FILESYS_FOR_MESHES}">
-    <xacro:property name="MESH_PATH" value="file://${CENTAURO_ROOT}/meshes" />
+    <xacro:property name="MESH_PATH" value="file://${ROOT}/meshes" />
     </xacro:if>
     <xacro:unless value="${USE_LOCAL_FILESYS_FOR_MESHES}">
-    <xacro:property name="MESH_PATH" value="${CENTAURO_ROOT}/meshes" />
+    <xacro:property name="MESH_PATH" value="${ROOT}/meshes" />
     </xacro:unless>
 </xacro:if>
@@ -27,5 +27,5 @@
 </xacro:macro>
 <!-- configuration -->
-<xacro:arg name="config" default="${CENTAURO_ROOT}/urdf/config/centauro.urdf.xacro"/>
+<xacro:arg name="config" default="${ROOT}/urdf/config/centauro.urdf.xacro"/>
 <!-- ************ MODEL CONFIGURATION ************ -->
 <xacro:include filename="$(arg config)"/>
@@ -49,5 +49,5 @@
 </xacro:if>
 <!-- ************ Pholus plain model ************ -->
-<xacro:include filename="${CENTAURO_ROOT}/urdf/centauro_base.urdf.xacro"/>
+<xacro:include filename="${ROOT}/urdf/centauro_base.urdf.xacro"/>
 <!-- ************ Control frames ************ -->
 <xacro:if value="${ADD_FLOATING_BASE}">
@@ -61,5 +61,5 @@
 </xacro:if>
 <xacro:if value="${ADD_VIRTUAL_FRAME}">
-  <xacro:include filename="${CENTAURO_ROOT}/urdf/parts/virtual_frame.urdf.xacro"/>
+  <xacro:include filename="${ROOT}/urdf/parts/virtual_frame.urdf.xacro"/>
 </xacro:if>
 </robot>

File: centauro_urdf/urdf/centauro_base.urdf.xacro (robot description, xacro)
@@ -2,8 +2,8 @@
 <robot xmlns:xacro="http://ros.org/wiki/xacro" name="centauro">
     <!-- ROS urdf definition of the CENTAURO humanoid robot by Istituto Italiano di Tecnologia. Author Enrico Mingo Hoffman-->
-    <xacro:include filename="${CENTAURO_ROOT}/urdf/utils.urdf.xacro" />
-    <xacro:include filename="${CENTAURO_ROOT}/urdf/parts/kinematics_properties.urdf.xacro" />
-    <xacro:include filename="${CENTAURO_ROOT}/urdf/parts/inertial_properties.urdf.xacro" />
-    <xacro:include filename="${CENTAURO_ROOT}/urdf/parts/limits.urdf.xacro" />
+    <xacro:include filename="${ROOT}/urdf/utils.urdf.xacro" />
+    <xacro:include filename="${ROOT}/urdf/parts/kinematics_properties.urdf.xacro" />
+    <xacro:include filename="${ROOT}/urdf/parts/inertial_properties.urdf.xacro" />
+    <xacro:include filename="${ROOT}/urdf/parts/limits.urdf.xacro" />
     <link name="base_link" />
     <joint name="base_joint" type="fixed">
@@ -38,7 +38,7 @@
     </joint>
     <xacro:if value="${ADD_UPPER_BODY}">
-        <xacro:include filename="${CENTAURO_ROOT}/urdf/parts/centauro_torso.urdf.xacro" />
-        <xacro:include filename="${CENTAURO_ROOT}/urdf/parts/arms.urdf.xacro" />
-        <xacro:include filename="${CENTAURO_ROOT}/urdf/parts/head.urdf.xacro" />
+        <xacro:include filename="${ROOT}/urdf/parts/centauro_torso.urdf.xacro" />
+        <xacro:include filename="${ROOT}/urdf/parts/arms.urdf.xacro" />
+        <xacro:include filename="${ROOT}/urdf/parts/head.urdf.xacro" />
         <xacro:property name="d435_base_name" value="D435i_camera" />
         <xacro:property name="d435_base_parent_name" value="pelvis" />
@@ -130,5 +130,5 @@
     </xacro:if>
     <xacro:if value="${ADD_LEGS}">
-        <xacro:include filename="${CENTAURO_ROOT}/urdf/parts/legs.urdf.xacro" />
+        <xacro:include filename="${ROOT}/urdf/parts/legs.urdf.xacro" />
     </xacro:if>
 </robot>

File: centauro_urdf/urdf/centauro_robot.urdf.xacro (robot description, xacro)
@@ -9,5 +9,5 @@
   will be propagated to all its downstream childs -->
   <xacro:arg name="centauro_root" default="$(find centauro_urdf)" />
-  <xacro:property name="CENTAURO_ROOT" value="$(arg centauro_root)" />
+  <xacro:property name="ROOT" value="$(arg centauro_root)" />
   <!-- setting use_abs_mesh_paths should be kept to false
   for use with tools like RViz, which does not accept plain
@@ -16,13 +16,13 @@
   <xacro:property name="USE_ABS_MESH_PATHS" value="$(arg use_abs_mesh_paths)" />
   <xacro:if value="${USE_ABS_MESH_PATHS}">
-    <xacro:property name="MESH_PATH" value="${CENTAURO_ROOT}/meshes" />
+    <xacro:property name="MESH_PATH" value="${ROOT}/meshes" />
   </xacro:if>
   <xacro:unless value="${USE_ABS_MESH_PATHS}">
     <xacro:property name="MESH_PATH" value="package://centauro_urdf/meshes" />
   </xacro:unless>
-  <xacro:include filename="${CENTAURO_ROOT}/urdf/centauro.urdf.xacro" />
-  <xacro:include filename="${CENTAURO_ROOT}/urdf/gazebo/centauro.gazebo.xacro" />
-  <xacro:include filename="${CENTAURO_ROOT}/urdf/gazebo/xbot.gazebo.xacro" />
-  <xacro:include filename="${CENTAURO_ROOT}/urdf/gazebo/materials.gazebo.xacro" />
+  <xacro:include filename="${ROOT}/urdf/centauro.urdf.xacro" />
+  <xacro:include filename="${ROOT}/urdf/gazebo/centauro.gazebo.xacro" />
+  <xacro:include filename="${ROOT}/urdf/gazebo/xbot.gazebo.xacro" />
+  <xacro:include filename="${ROOT}/urdf/gazebo/materials.gazebo.xacro" />
   <xacro:unless value="${ADD_LEGS}">
     <link name="world"/>

File: centauro_urdf/urdf/parts/arms.urdf.xacro (robot description, xacro)
@@ -1,5 +1,5 @@
 <?xml version="1.0"?>
 <robot xmlns:xacro="http://ros.org/wiki/xacro">
-<xacro:include filename="${CENTAURO_ROOT}/urdf/parts/centauro_arm.urdf.xacro" />
+<xacro:include filename="${ROOT}/urdf/parts/centauro_arm.urdf.xacro" />
 <!-- arms -->
 <xacro:centauro_arm arm_num="1"  rot="1"  parent="torso_2">
@@ -38,5 +38,5 @@
 </xacro:if>
 <xacro:if value="${END_EFFECTOR_LEFT == 'ball'}">
-	<xacro:include filename="${CENTAURO_ROOT}/urdf/parts/ball.urdf.xacro" />
+	<xacro:include filename="${ROOT}/urdf/parts/ball.urdf.xacro" />
 	<xacro:ball_end_effector arm_num="1"  parent_link="arm1_6">
 		      <origin xyz="0. -0.05 -0.105" rpy="0. 0. 0."/>
@@ -44,5 +44,5 @@
 </xacro:if>
 <xacro:if value="${END_EFFECTOR_RIGHT == 'ball'}">
-	<xacro:include filename="${CENTAURO_ROOT}/urdf/parts/ball.urdf.xacro" />
+	<xacro:include filename="${ROOT}/urdf/parts/ball.urdf.xacro" />
 	<xacro:ball_end_effector arm_num="2"  parent_link="arm2_6">
 	 <origin xyz="0. 0.05 -0.105" rpy="0. 0. 0."/>

File: centauro_urdf/urdf/parts/centauro_leg.urdf.xacro (robot description, xacro)
@@ -1,6 +1,6 @@
 <?xml version="1.0"?>
 <robot xmlns:xacro="http://ros.org/wiki/xacro">
-<xacro:include filename="${CENTAURO_ROOT}/urdf/parts/wheel.urdf.xacro"/>
-<xacro:include filename="${CENTAURO_ROOT}/urdf/parts/wheel23.urdf.xacro"/>
+<xacro:include filename="${ROOT}/urdf/parts/wheel.urdf.xacro"/>
+<xacro:include filename="${ROOT}/urdf/parts/wheel23.urdf.xacro"/>
 <!-- macro legs -->
 <xacro:macro name="centauro_leg" params="leg_num origin_x origin_y mirror">

File: centauro_urdf/urdf/parts/legs.urdf.xacro (robot description, xacro)
@@ -1,5 +1,5 @@
 <?xml version="1.0"?>
 <robot xmlns:xacro="http://ros.org/wiki/xacro">
-<xacro:include filename="${CENTAURO_ROOT}/urdf/parts/centauro_leg.urdf.xacro" />
+<xacro:include filename="${ROOT}/urdf/parts/centauro_leg.urdf.xacro" />
 <xacro:centauro_leg leg_num="1" origin_x="1" origin_y="-1" mirror="-1">
 </xacro:centauro_leg>

Commit message: Signed-off-by: Andrea Patrizi <andreapatrizi1b6e6@gmail.com>

File: centauro_srdf/srdf/centauro.srdf.xacro (robot description, xacro)
@@ -5,6 +5,6 @@
 -->
 <robot xmlns:xacro="http://ros.org/wiki/xacro" name="centauro">
-    <xacro:arg name="centauro_root" default="$(find centauro_urdf)" />
-    <xacro:property name="ROOT" value="$(arg centauro_root)" />
+    <xacro:arg name="root" default="$(find centauro_urdf)" />
+    <xacro:property name="ROOT" value="$(arg root)" />
     <!-- ************ MODEL CONFIGURATION ************ -->
     <xacro:arg name="config" default="${ROOT}/urdf/config/centauro.urdf.xacro"/>

File: centauro_urdf/urdf/centauro.urdf.xacro (robot description, xacro)
@@ -3,6 +3,6 @@
 <!-- This argument and property should be in the top level xacro and
 will be propagated to all its downstream childs -->
-<xacro:arg name="centauro_root" default="$(find centauro_urdf)" />
-<xacro:property name="ROOT" value="$(arg centauro_root)" />
+<xacro:arg name="root" default="$(find centauro_urdf)" />
+<xacro:property name="ROOT" value="$(arg root)" />
 <!-- setting use_abs_mesh_paths should be kept to false
 for use with tools like RViz, which does not accept plain

File: centauro_urdf/urdf/centauro_robot.urdf.xacro (robot description, xacro)
@@ -8,6 +8,6 @@
   <!-- This argument and property should be in the top level xacro and
   will be propagated to all its downstream childs -->
-  <xacro:arg name="centauro_root" default="$(find centauro_urdf)" />
-  <xacro:property name="ROOT" value="$(arg centauro_root)" />
+  <xacro:arg name="root" default="$(find centauro_urdf)" />
+  <xacro:property name="ROOT" value="$(arg root)" />
   <!-- setting use_abs_mesh_paths should be kept to false
   for use with tools like RViz, which does not accept plain

Commit message: removed old CENTAURO_ROOT arg

File: centauro_srdf/srdf/centauro.srdf.xacro (robot description, xacro)
@@ -5,8 +5,8 @@
 -->
 <robot xmlns:xacro="http://ros.org/wiki/xacro" name="centauro">
-    <xacro:arg name="centauro_root" default="$(find centauro_urdf)" />
-    <xacro:property name="CENTAURO_ROOT" value="$(arg centauro_root)" />
+    <xacro:arg name="root" default="$(find centauro_urdf)" />
+    <xacro:property name="ROOT" value="$(arg root)" />
     <!-- ************ MODEL CONFIGURATION ************ -->
-    <xacro:arg name="config" default="${CENTAURO_ROOT}/urdf/config/centauro.urdf.xacro"/>
+    <xacro:arg name="config" default="${ROOT}/urdf/config/centauro.urdf.xacro"/>
     <xacro:include filename="$(arg config)"/>
     <group name="base">

File: centauro_urdf/urdf/centauro.urdf.xacro (robot description, xacro)
@@ -3,19 +3,29 @@
 <!-- This argument and property should be in the top level xacro and
 will be propagated to all its downstream childs -->
-<xacro:arg name="centauro_root" default="$(find centauro_urdf)" />
-<xacro:property name="CENTAURO_ROOT" value="$(arg centauro_root)" />
+<xacro:arg name="root" default="$(find centauro_urdf)" />
+<xacro:property name="ROOT" value="$(arg root)" />
 <!-- setting use_abs_mesh_paths should be kept to false
 for use with tools like RViz, which does not accept plain
 abolute paths for mesh paths-->
 <xacro:arg name="use_abs_mesh_paths" default="false" />
+<xacro:arg name="use_local_filesys_for_meshes" default="false" />
 <xacro:property name="USE_ABS_MESH_PATHS" value="$(arg use_abs_mesh_paths)" />
+<xacro:property name="USE_LOCAL_FILESYS_FOR_MESHES" value="$(arg use_local_filesys_for_meshes)" />
 <xacro:if value="${USE_ABS_MESH_PATHS}">
-  <xacro:property name="MESH_PATH" value="${CENTAURO_ROOT}/meshes" />
+    <xacro:if value="${USE_LOCAL_FILESYS_FOR_MESHES}">
+    <xacro:property name="MESH_PATH" value="file://${ROOT}/meshes" />
+    </xacro:if>
+    <xacro:unless value="${USE_LOCAL_FILESYS_FOR_MESHES}">
+    <xacro:property name="MESH_PATH" value="${ROOT}/meshes" />
+    </xacro:unless>
 </xacro:if>
 <xacro:unless value="${USE_ABS_MESH_PATHS}">
-  <xacro:property name="MESH_PATH" value="package://centauro_urdf/meshes" />
+    <xacro:property name="MESH_PATH" value="package://centauro_urdf/meshes" />
 </xacro:unless>
+<xacro:macro name="example_macro">
+  <example_element message="${MESH_PATH}" />
+</xacro:macro>
 <!-- configuration -->
-<xacro:arg name="config" default="${CENTAURO_ROOT}/urdf/config/centauro.urdf.xacro"/>
+<xacro:arg name="config" default="${ROOT}/urdf/config/centauro.urdf.xacro"/>
 <!-- ************ MODEL CONFIGURATION ************ -->
 <xacro:include filename="$(arg config)"/>
@@ -39,5 +49,5 @@
 </xacro:if>
 <!-- ************ Pholus plain model ************ -->
-<xacro:include filename="${CENTAURO_ROOT}/urdf/centauro_base.urdf.xacro"/>
+<xacro:include filename="${ROOT}/urdf/centauro_base.urdf.xacro"/>
 <!-- ************ Control frames ************ -->
 <xacro:if value="${ADD_FLOATING_BASE}">
@@ -51,5 +61,5 @@
 </xacro:if>
 <xacro:if value="${ADD_VIRTUAL_FRAME}">
-  <xacro:include filename="${CENTAURO_ROOT}/urdf/parts/virtual_frame.urdf.xacro"/>
+  <xacro:include filename="${ROOT}/urdf/parts/virtual_frame.urdf.xacro"/>
 </xacro:if>
 </robot>

File: centauro_urdf/urdf/centauro_base.urdf.xacro (robot description, xacro)
@@ -5,8 +5,8 @@
   Author: Enrico Mingo Hoffman
 -->
-    <xacro:include filename="${CENTAURO_ROOT}/urdf/utils.urdf.xacro" />
-    <xacro:include filename="${CENTAURO_ROOT}/urdf/parts/kinematics_properties.urdf.xacro" />
-    <xacro:include filename="${CENTAURO_ROOT}/urdf/parts/inertial_properties.urdf.xacro" />
-    <xacro:include filename="${CENTAURO_ROOT}/urdf/parts/limits.urdf.xacro" />
+    <xacro:include filename="${ROOT}/urdf/utils.urdf.xacro" />
+    <xacro:include filename="${ROOT}/urdf/parts/kinematics_properties.urdf.xacro" />
+    <xacro:include filename="${ROOT}/urdf/parts/inertial_properties.urdf.xacro" />
+    <xacro:include filename="${ROOT}/urdf/parts/limits.urdf.xacro" />
     <link name="base_link" />
     <joint name="base_joint" type="fixed">
@@ -41,7 +41,7 @@
     </joint>
     <xacro:if value="${ADD_UPPER_BODY}">
-        <xacro:include filename="${CENTAURO_ROOT}/urdf/parts/centauro_torso.urdf.xacro" />
-        <xacro:include filename="${CENTAURO_ROOT}/urdf/parts/arms.urdf.xacro" />
-        <xacro:include filename="${CENTAURO_ROOT}/urdf/parts/head.urdf.xacro" />
+        <xacro:include filename="${ROOT}/urdf/parts/centauro_torso.urdf.xacro" />
+        <xacro:include filename="${ROOT}/urdf/parts/arms.urdf.xacro" />
+        <xacro:include filename="${ROOT}/urdf/parts/head.urdf.xacro" />
         <xacro:property name="d435_base_name" value="D435i_camera" />
         <xacro:property name="d435_base_parent_name" value="pelvis" />
@@ -133,5 +133,5 @@
     </xacro:if>
     <xacro:if value="${ADD_LEGS}">
-        <xacro:include filename="${CENTAURO_ROOT}/urdf/parts/legs.urdf.xacro" />
+        <xacro:include filename="${ROOT}/urdf/parts/legs.urdf.xacro" />
     </xacro:if>
 </robot>

File: centauro_urdf/urdf/centauro_robot.urdf.xacro (robot description, xacro)
@@ -8,6 +8,6 @@
   <!-- This argument and property should be in the top level xacro and
   will be propagated to all its downstream childs -->
-  <xacro:arg name="centauro_root" default="$(find centauro_urdf)" />
-  <xacro:property name="CENTAURO_ROOT" value="$(arg centauro_root)" />
+  <xacro:arg name="root" default="$(find centauro_urdf)" />
+  <xacro:property name="ROOT" value="$(arg root)" />
   <!-- setting use_abs_mesh_paths should be kept to false
   for use with tools like RViz, which does not accept plain
@@ -16,13 +16,13 @@
   <xacro:property name="USE_ABS_MESH_PATHS" value="$(arg use_abs_mesh_paths)" />
   <xacro:if value="${USE_ABS_MESH_PATHS}">
-    <xacro:property name="MESH_PATH" value="${CENTAURO_ROOT}/meshes" />
+    <xacro:property name="MESH_PATH" value="${ROOT}/meshes" />
   </xacro:if>
   <xacro:unless value="${USE_ABS_MESH_PATHS}">
     <xacro:property name="MESH_PATH" value="package://centauro_urdf/meshes" />
   </xacro:unless>
-  <xacro:include filename="${CENTAURO_ROOT}/urdf/centauro.urdf.xacro" />
-  <xacro:include filename="${CENTAURO_ROOT}/urdf/gazebo/centauro.gazebo.xacro" />
-  <xacro:include filename="${CENTAURO_ROOT}/urdf/gazebo/xbot.gazebo.xacro" />
-  <xacro:include filename="${CENTAURO_ROOT}/urdf/gazebo/materials.gazebo.xacro" />
+  <xacro:include filename="${ROOT}/urdf/centauro.urdf.xacro" />
+  <xacro:include filename="${ROOT}/urdf/gazebo/centauro.gazebo.xacro" />
+  <xacro:include filename="${ROOT}/urdf/gazebo/xbot.gazebo.xacro" />
+  <xacro:include filename="${ROOT}/urdf/gazebo/materials.gazebo.xacro" />
   <xacro:unless value="${ADD_LEGS}">
     <link name="world"/>

File: centauro_urdf/urdf/parts/centauro_leg.urdf.xacro (robot description, xacro)
@@ -1,6 +1,6 @@
 <?xml version="1.0"?>
 <robot xmlns:xacro="http://ros.org/wiki/xacro">
-<xacro:include filename="${CENTAURO_ROOT}/urdf/parts/wheel.urdf.xacro"/>
-<xacro:include filename="${CENTAURO_ROOT}/urdf/parts/wheel23.urdf.xacro"/>
+<xacro:include filename="${ROOT}/urdf/parts/wheel.urdf.xacro"/>
+<xacro:include filename="${ROOT}/urdf/parts/wheel23.urdf.xacro"/>
 <!-- macro legs -->
 <xacro:macro name="centauro_leg" params="leg_num origin_x origin_y mirror">

Commit message: Signed-off-by: Andrea Patrizi <andreapatrizi1b6e6@gmail.com>

File: centauro_srdf/srdf/centauro.srdf.xacro (robot description, xacro)
@@ -107,4 +107,8 @@
         <joint name="j_arm2_5" value="-0.0500815"/>
         <joint name="j_arm2_6" value="-0.781461"/>
+        <joint name="j_wheel_1" value="0.0"/>
+        <joint name="j_wheel_2" value="0.0"/>
+        <joint name="j_wheel_3" value="0.0"/>
+        <joint name="j_wheel_4" value="0.0"/>
         <xacro:if value="${END_EFFECTOR_LEFT == 'dagana'}">
             <joint name="dagana_1_claw_joint" value="0"/>
