Commit message: simplify collisions (wip)

File: centauro_isaac/urdf/centauro_dagana.urdf (robot description, URDF)
Before this commit: robot centauro, 94 links, 93 joints
Links:
- link D435_head_camera_link: geometry collision box size=0.02505 0.09 0.025; visual mesh filename=/workspace/models/realsense2_description/meshes/d435.dae
- link D435i_camera_link: geometry collision box size=0.02505 0.09 0.025; visual mesh filename=/workspace/models/realsense2_description/meshes/d435.dae
- link T265_camera_pose_frame: geometry collision cylinder length=0.1022528557886848 radius=0.0142751; visual mesh filename=/workspace/models/realsense_gazebo_description/meshes/t265_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 scale=0.001 0.001 0.001
- link ankle1_1: geometry collision cylinder length=0.14 radius=0.065; visual mesh filename=/workspace/models/iit-centauro-ros-pkg/centauro_isaac/meshe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 scale=0.001 0.001 -0.001
- link ankle1_2: geometry collision cylinder length=0.14 radius=0.065; visual mesh filename=/workspace/models/iit-centauro-ros-pkg/centauro_isaac/meshe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 scale=0.001 0.001 0.001
- link ankle1_3: geometry collision cylinder length=0.14 radius=0.065; visual mesh filename=/workspace/models/iit-centauro-ros-pkg/centauro_isaac/meshe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 scale=0.001 0.001 -0.001
- link ankle1_4: geometry collision cylinder length=0.14 radius=0.065; visual mesh filename=/workspace/models/iit-centauro-ros-pkg/centauro_isaac/meshe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 scale=0.001 0.001 0.001
- link ankle2_1: geometry collision cylinder length=0.05 radius=0.08586; visual mesh filename=/workspace/models/iit-centauro-ros-pkg/centauro_isaac/meshe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 scale=0.001 -0.001 0.001
- link ankle2_2: geometry collision cylinder length=0.05 radius=0.08586; visual mesh filename=/workspace/models/iit-centauro-ros-pkg/centauro_isaac/meshe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 scale=0.001 0.001 0.001
- link ankle2_3: geometry collision cylinder length=0.05 radius=0.08586; visual mesh filename=/workspace/models/iit-centauro-ros-pkg/centauro_isaac/meshe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 scale=0.001 -0.001 0.001
- link ankle2_4: geometry collision cylinder length=0.05 radius=0.08586; visual mesh filename=/workspace/models/iit-centauro-ros-pkg/centauro_isaac/meshe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 scale=0.001 0.001 0.001
- link arm1_1: geometry collision cylinder length=0.03739768494560427 radius=0.0698859; visual mesh filename=/workspace/models/iit-centauro-ros-pkg/centauro_urdf/meshes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 scale=0.001 -0.001 0.001
- link arm1_2: geometry collision cylinder length=0.12799269981445732 radius=0.0700645; visual mesh filename=/workspace/models/iit-centauro-ros-pkg/centauro_urdf/meshes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 scale=0.001 -0.001 0.001
- link arm1_3: geometry collision cylinder length=0.06082252644344949 radius=0.0896121; visual mesh filename=/workspace/models/iit-centauro-ros-pkg/centauro_urdf/meshes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 scale=0.001 -0.001 0.001
- link arm1_4: geometry collision cylinder length=0.08713418572944408 radius=0.0600429; visual mesh filename=/workspace/models/iit-centauro-ros-pkg/centauro_urdf/meshes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 scale=0.001 -0.001 0.001
- link arm1_5: geometry collision cylinder length=0.08434739747702548 radius=0.0804108; visual mesh filename=/workspace/models/iit-centauro-ros-pkg/centauro_urdf/meshes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 scale=0.001 -0.001 0.001
- link arm1_6: geometry collision cylinder length=0.07750977987441161 radius=0.0474698; visual mesh filename=/workspace/models/iit-centauro-ros-pkg/centauro_urdf/meshes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 scale=0.001 -0.001 0.001
- link arm2_1: geometry collision cylinder length=0.03739768494560427 radius=0.0698859; visual mesh filename=/workspace/models/iit-centauro-ros-pkg/centauro_urdf/meshes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 scale=0.001 0.001 0.001
- link arm2_2: geometry collision cylinder length=0.12799269981445732 radius=0.0700645; visual mesh filename=/workspace/models/iit-centauro-ros-pkg/centauro_urdf/meshes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 scale=0.001 0.001 0.001
- link arm2_3: geometry collision cylinder length=0.06082252644344949 radius=0.0896121; visual mesh filename=/workspace/models/iit-centauro-ros-pkg/centauro_urdf/meshes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 scale=0.001 0.001 0.001
- link arm2_4: geometry collision cylinder length=0.08713418572944408 radius=0.0600429; visual mesh filename=/workspace/models/iit-centauro-ros-pkg/centauro_urdf/meshes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 scale=0.001 0.001 0.001
- link arm2_5: geometry collision cylinder length=0.08434739747702548 radius=0.0804108; visual mesh filename=/workspace/models/iit-centauro-ros-pkg/centauro_urdf/meshes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 scale=0.001 0.001 0.001
- link arm2_6: geometry collision cylinder length=0.07750977987441161 radius=0.0474698; visual mesh filename=/workspace/models/iit-centauro-ros-pkg/centauro_urdf/meshes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 scale=0.001 0.001 0.001
- link ball1: geometry collision cylinder length=9.940076835940455e-05 radius=0.0709883; visual mesh filename=/workspace/models/iit-centauro-ros-pkg/centauro_urdf/meshes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 scale=0.001 0.001 0.001
- link base_link: geometry collision mesh filename=/workspace/models/iit-centauro-ros-pkg/centauro_urdf/meshes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 scale=0.001 0.001 0.001; visual mesh filename=/workspace/models/iit-centauro-ros-pkg/centauro_urdf/meshes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 scale=0.001 0.001 0.001
- link d435_head_motor: geometry collision cylinder length=0.12134423548428976 radius=0.0261699; visual mesh filename=/workspace/models/iit-centauro-ros-pkg/centauro_isaac/meshe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 scale=0.001 0.001 0.001
- link dagana_2_bottom_link: geometry visual mesh filename=/workspace/models/iit-dagana-ros-pkg/dagana_urdf/meshes/dg0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 scale=0.001 0.001 0.001
- link dagana_2_top_link: geometry collision cylinder length=0.10212404260993166 radius=0.0760764; visual mesh filename=/workspace/models/iit-centauro-ros-pkg/centauro_isaac/meshe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 scale=0.001 0.001 0.001
- link hip1_1: geometry collision cylinder length=0.09 radius=0.05; visual mesh filename=/workspace/models/iit-centauro-ros-pkg/centauro_isaac/meshe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 scale=0.001 -0.001 0.001
- link hip1_2: geometry collision cylinder length=0.09 radius=0.05; visual mesh filename=/workspace/models/iit-centauro-ros-pkg/centauro_isaac/meshe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 scale=0.001 0.001 0.001
- link hip1_3: geometry collision cylinder length=0.09 radius=0.05; visual mesh filename=/workspace/models/iit-centauro-ros-pkg/centauro_isaac/meshe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 scale=0.001 -0.001 0.001
- link hip1_4: geometry collision cylinder length=0.09 radius=0.05; visual mesh filename=/workspace/models/iit-centauro-ros-pkg/centauro_isaac/meshe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 scale=0.001 0.001 0.001
- link hip2_1: geometry collision box size=0.12 0.10 0.4; visual mesh filename=/workspace/models/iit-centauro-ros-pkg/centauro_isaac/meshe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 scale=0.001 0.001 -0.001
- link hip2_2: geometry collision box size=0.12 0.10 0.4; visual mesh filename=/workspace/models/iit-centauro-ros-pkg/centauro_isaac/meshe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 scale=0.001 0.001 0.001
- link hip2_3: geometry collision box size=0.12 0.10 0.4; visual mesh filename=/workspace/models/iit-centauro-ros-pkg/centauro_isaac/meshe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 scale=0.001 0.001 -0.001
- link hip2_4: geometry collision box size=0.12 0.10 0.4; visual mesh filename=/workspace/models/iit-centauro-ros-pkg/centauro_isaac/meshe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 scale=0.001 0.001 0.001
- link knee_1: geometry collision box size=0.08 0.08 0.3; visual mesh filename=/workspace/models/iit-centauro-ros-pkg/centauro_urdf/meshes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 scale=0.001 0.001 -0.001
- link knee_2: geometry collision box size=0.08 0.08 0.3; visual mesh filename=/workspace/models/iit-centauro-ros-pkg/centauro_urdf/meshes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 scale=0.001 0.001 0.001
- link knee_3: geometry collision box size=0.08 0.08 0.3; visual mesh filename=/workspace/models/iit-centauro-ros-pkg/centauro_urdf/meshes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 scale=0.001 0.001 -0.001
- link knee_4: geometry collision box size=0.08 0.08 0.3; visual mesh filename=/workspace/models/iit-centauro-ros-pkg/centauro_urdf/meshes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 scale=0.001 0.001 0.001
- link neck_1: geometry collision cylinder length=0.16454098025546557 radius=0.100414; visual mesh filename=/workspace/models/iit-centauro-ros-pkg/centauro_isaac/meshe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 scale=0.001 0.001 0.001
- link torso_2: geometry collision cylinder length=0.09543675990850982 radius=0.158224; visual mesh filename=/workspace/models/iit-centauro-ros-pkg/centauro_urdf/meshes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 scale=0.001 0.001 0.001
- link velodyne_calib: geometry visual mesh filename=/workspace/models/velodyne_simulator/velodyne_description/m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
- link velodyne_calib_base_link: geometry collision cylinder length=0.0717 radius=0.0516; visual mesh filename=/workspace/models/velodyne_simulator/velodyne_description/m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
- link velodyne_motor: geometry collision cylinder length=0.032463112134515464 radius=0.0544637; visual mesh filename=/workspace/models/iit-centauro-ros-pkg/centauro_urdf/meshes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 scale=0.001 0.001 0.001
- link wheel_1: geometry collision mesh filename=/workspace/models/iit-centauro-ros-pkg/centauro_urdf/meshes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 scale=0.001 0.001 -0.001; visual mesh filename=/workspace/models/iit-centauro-ros-pkg/centauro_urdf/meshes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 scale=0.001 0.001 -0.001
- link wheel_2: geometry collision mesh filename=/workspace/models/iit-centauro-ros-pkg/centauro_urdf/meshes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 scale=0.001 0.001 -0.001; visual mesh filename=/workspace/models/iit-centauro-ros-pkg/centauro_urdf/meshes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 scale=0.001 0.001 0.001
- link wheel_3: geometry collision mesh filename=/workspace/models/iit-centauro-ros-pkg/centauro_urdf/meshes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 scale=0.001 0.001 -0.001; visual mesh filename=/workspace/models/iit-centauro-ros-pkg/centauro_urdf/meshes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 scale=0.001 0.001 -0.001
- link wheel_4: geometry collision mesh filename=/workspace/models/iit-centauro-ros-pkg/centauro_urdf/meshes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 scale=0.001 0.001 -0.001; visual mesh filename=/workspace/models/iit-centauro-ros-pkg/centauro_urdf/meshes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 scale=0.001 0.001 0.001

Commit message: fix isaac leg and base collisions

File: centauro_isaac/urdf/centauro_dagana.urdf (robot description, URDF)
Before this commit: robot centauro, 94 links, 93 joints
Links:
- link ankle1_1: geometry collision cylinder length=0.14 radius=0.05; visual mesh filename=/workspace/models/iit-centauro-ros-pkg/centauro_isaac/meshe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 scale=0.001 0.001 -0.001
- link ankle1_2: geometry collision cylinder length=0.14 radius=0.05; visual mesh filename=/workspace/models/iit-centauro-ros-pkg/centauro_isaac/meshe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 scale=0.001 0.001 0.001
- link ankle1_3: geometry collision cylinder length=0.14 radius=0.05; visual mesh filename=/workspace/models/iit-centauro-ros-pkg/centauro_isaac/meshe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 scale=0.001 0.001 -0.001
- link ankle1_4: geometry collision cylinder length=0.14 radius=0.05; visual mesh filename=/workspace/models/iit-centauro-ros-pkg/centauro_isaac/meshe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 scale=0.001 0.001 0.001
- link ankle2_1: geometry collision cylinder length=0.05 radius=0.075; visual mesh filename=/workspace/models/iit-centauro-ros-pkg/centauro_isaac/meshe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 scale=0.001 -0.001 0.001
- link ankle2_2: geometry collision cylinder length=0.05 radius=0.075; visual mesh filename=/workspace/models/iit-centauro-ros-pkg/centauro_isaac/meshe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 scale=0.001 0.001 0.001
- link ankle2_3: geometry collision cylinder length=0.05 radius=0.075; visual mesh filename=/workspace/models/iit-centauro-ros-pkg/centauro_isaac/meshe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 scale=0.001 -0.001 0.001
- link ankle2_4: geometry collision cylinder length=0.05 radius=0.075; visual mesh filename=/workspace/models/iit-centauro-ros-pkg/centauro_isaac/meshe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 scale=0.001 0.001 0.001
- link base_link: geometry collision box size=0.6 0.3 0.22; visual mesh filename=/workspace/models/iit-centauro-ros-pkg/centauro_urdf/meshes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 scale=0.001 0.001 0.001
- link torso_2: geometry collision cylinder length=0.20 radius=0.15; visual mesh filename=/workspace/models/iit-centauro-ros-pkg/centauro_urdf/meshes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 scale=0.001 0.001 0.001
