Commit message: crazy hack for sensors waiting for alovato's help

File: centauro_gazebo/urdf/centauro_sensors.urdf.xacro (robot description, xacro)
@@ -43,34 +43,55 @@
     </xacro:if>
     <xacro:if value="${ADD_D435I_HEAD}">
-        <link name="D435_head_camera_gz_optical_frame"/>
+        <link name="D435_head_camera_gz_optical_frame" />
         <joint name="D435_head_camera_gz_optical_frame_joint" type="fixed">
-            <parent link="D435_head_camera_link"/>
-            <child link="D435_head_camera_gz_optical_frame"/>
-            <origin xyz="0 0 0" rpy="${-PI_2} 0 ${-PI_2}"/>
+            <parent link="D435_head_camera_link" />
+            <child link="D435_head_camera_gz_optical_frame" />
+            <origin xyz="0 0 0" rpy="${-PI_2} 0 ${-PI_2}" />
         </joint>
         <gazebo reference="D435_head_camera_link">
-        <sensor name="rgbd_camera" type="rgbd_camera">
-            <!-- rotate 180° around X to match ROS optical frame convention (Y down in image) -->
-            <!-- <pose relative_to="D435_head_camera_link">0 0 0 3.14159265 0 0</pose> -->
-            <camera>
-              <horizontal_fov>1.047</horizontal_fov>
-              <image>
-                <width>320</width>
-                <height>240</height>
-              </image>
-              <clip>
-                <near>0.3</near>
-                <far>10</far>
-              </clip>
-              <optical_frame_id>D435_head_camera_gz_optical_frame</optical_frame_id>
-            </camera>
-            <gz_frame_id>D435_head_camera_gz_optical_frame</gz_frame_id>
-            <always_on>1</always_on>
-            <update_rate>30</update_rate>
-            <visualize>true</visualize>
-            <topic>D435_head_camera</topic>
-            <enable_metrics>true</enable_metrics>
-          </sensor>
-          </gazebo>
+            <sensor name="rgbd_camera_depth" type="depth_camera">
+                <camera>
+                    <horizontal_fov>1.047</horizontal_fov>
+                    <image>
+                        <width>320</width>
+                        <height>240</height>
+                    </image>
+                    <clip>
+                        <near>0.3</near>
+                        <far>10</far>
+                    </clip>
+                    <camera_info_topic>D435_head_camera/depth/camera_info</camera_info_topic>
+                </camera>
+                <gz_frame_id>D435_head_camera_link</gz_frame_id>
+                <always_on>1</always_on>
+                <update_rate>30</update_rate>
+                <visualize>true</visualize>
+                <topic>D435_head_camera/depth</topic>
+                <enable_metrics>true</enable_metrics>
+            </sensor>
+        </gazebo>
+        <gazebo reference="D435_head_camera_link">
+            <sensor name="rgbd_camera_color" type="camera">
+                <camera>
+                    <horizontal_fov>1.047</horizontal_fov>
+                    <image>
+                        <width>320</width>
+                        <height>240</height>
+                    </image>
+                    <clip>
+                        <near>0.3</near>
+                        <far>10</far>
+                    </clip>
+                    <optical_frame_id>D435_head_camera_gz_optical_frame</optical_frame_id>
+                    <camera_info_topic>D435_head_camera/color/camera_info</camera_info_topic>
+                </camera>
+                <gz_frame_id>D435_head_camera_gz_optical_frame</gz_frame_id>
+                <always_on>1</always_on>
+                <update_rate>30</update_rate>
+                <visualize>true</visualize>
+                <topic>D435_head_camera/color</topic>
+                <enable_metrics>true</enable_metrics>
+            </sensor>
+        </gazebo>
     </xacro:if>
 </robot>
